File: KiMBo/rf.sch (KiCad schematic (older format))
At the start: 7 parts

Commit message: Update to use OSD335x as the main chipset
Parts:
- removed AE? (x2): UFL, symbol UFL
- removed AE? (x2): ANTENNA, symbol ANTENNA
- removed T? (x2): 2450BL15B100, symbol 2450BL15B100
- removed U?: MT7620N, symbol MT7620N
Changed lines of the file:
@@
 Comment4 ""
 $EndDescr
-$Comp
-L MT7620N U?
-U 4 1 581F0159
-P 4300 3700
-AR Path="/581F0159" Ref="U?"  Part="4"
-AR Path="/581E2C5F/581F0159" Ref="U?"  Part="4"
-F 0 "U?" H 3900 4837 60  0000 C CNN
-F 1 "MT7620N" H 3900 4731 60  0000 C CNN
-F 2 "" H 2600 4200 60  0000 C CNN
-F 3 "" H 2600 4200 60  0000 C CNN
-	4    4300 3700
-	-1   0    0    -1
-$EndComp
-$Comp
-L 2450BL15B100 T?
-U 1 1 581F4FDC
-P 8500 2600
-F 0 "T?" H 8500 3087 60  0000 C CNN
-F 1 "2450BL15B100" H 8500 2981 60  0000 C CNN
-F 2 "" H 8500 2600 60  0000 C CNN
-F 3 "" H 8500 2600 60  0000 C CNN
-	1    8500 2600
-	1    0    0    -1
-$EndComp
-$Comp
-L 2450BL15B100 T?
-U 1 1 581F5012
-P 8500 3850
-F 0 "T?" H 8500 4337 60  0000 C CNN
-F 1 "2450BL15B100" H 8500 4231 60  0000 C CNN
-F 2 "" H 8500 3850 60  0000 C CNN
-F 3 "" H 8500 3850 60  0000 C CNN
-	1    8500 3850
-	1    0    0    -1
-$EndComp
-$Comp
-L UFL AE?
-U 1 1 582F1376
-P 10100 2850
-F 0 "AE?" H 10341 2972 60  0000 L CNN
-F 1 "UFL" H 10341 2866 60  0000 L CNN
-F 2 "" H 9950 2850 60  0000 C CNN
-F 3 "" H 9950 2850 60  0000 C CNN
-	1    10100 2850
-	1    0    0    -1
-$EndComp
-$Comp
-L ANTENNA AE?
-U 1 1 582F1398
-P 9850 3750
-F 0 "AE?" H 9968 4287 60  0000 C CNN
-F 1 "ANTENNA" H 9968 4181 60  0000 C CNN
-F 2 "" H 9950 3750 60  0000 C CNN
-F 3 "" H 9950 3750 60  0000 C CNN
-	1    9850 3750
-	1    0    0    -1
-$EndComp
-$Comp
-L UFL AE?
-U 1 1 582F1981
-P 10100 4700
-F 0 "AE?" H 10341 4822 60  0000 L CNN
-F 1 "UFL" H 10341 4716 60  0000 L CNN
-F 2 "" H 9950 4700 60  0000 C CNN
-F 3 "" H 9950 4700 60  0000 C CNN
-	1    10100 4700
-	1    0    0    -1
-$EndComp
-$Comp
-L ANTENNA AE?
-U 1 1 582F1988
-P 9850 5600
-F 0 "AE?" H 9968 6137 60  0000 C CNN
-F 1 "ANTENNA" H 9968 6031 60  0000 C CNN
-F 2 "" H 9950 5600 60  0000 C CNN
-F 3 "" H 9950 5600 60  0000 C CNN
-	1    9850 5600
-	1    0    0    -1
-$EndComp
 $EndSCHEMATC
