File: KiMBo/sdram.sch (KiCad schematic (older format))
At the start: 2 parts

Commit message: Update to use OSD335x as the main chipset
Parts:
- removed U?: MT7620N, symbol MT7620N
- removed U?: W9751G6KB-25, symbol W9751G6KB-25
Changed lines of the file:
@@
 Comment4 ""
 $EndDescr
-$Comp
-L MT7620N U?
-U 2 1 581F255A
-P 8100 5100
-AR Path="/581F255A" Ref="U?"  Part="2"
-AR Path="/581A9C89/581F255A" Ref="U?"  Part="2"
-F 0 "U?" H 7775 6237 60  0000 C CNN
-F 1 "MT7620N" H 7775 6131 60  0000 C CNN
-F 2 "" H 6400 5600 60  0000 C CNN
-F 3 "" H 6400 5600 60  0000 C CNN
-	2    8100 5100
-	1    0    0    -1
-$EndComp
-$Comp
-L W9751G6KB-25 U?
-U 1 1 581F54E2
-P 10650 4700
-F 0 "U?" H 10650 6800 60  0000 C CNN
-F 1 "W9751G6KB-25" H 10650 6694 60  0000 C CNN
-F 2 "" H 9050 5100 60  0000 C CNN
-F 3 "" H 9050 5100 60  0000 C CNN
-	1    10650 4700
-	1    0    0    -1
-$EndComp
 $EndSCHEMATC
