File: KiMBo/x1_stepper.sch (KiCad schematic (older format))
At the start: 25 parts, among them U28 TMC2130

Commit message: Reorder the SS and EN lines from the shift registers such that the previously enabled/disabled motors stay enabled/disabled whilst writting to the shift register
Change 10k resistors to 4.7k, flip the open-drain inverter connected to B15 (PMTC_PGOOD)

Update the links in the README

Update the PDF schematic
Parts:
- R188, R189, R190: value 10kΩ -> 4.7kΩ
Changed lines of the file:
@@
 F 0 "C199" H 7386 3054 50  0000 R CNN
 F 1 "100nF" H 7386 3145 50  0000 R CNN
-F 2 "" H 7538 2950 50  0000 C CNN
+F 2 "" H 7538 2950 50  0001 C CNN
 F 3 "" H 7500 3100 50  0000 C CNN
 	1    7500 3100
@@
 F 0 "C204" V 9250 3550 50  0000 C CNN
 F 1 "100nF" V 9250 3825 50  0000 C CNN
-F 2 "" H 9338 3500 50  0000 C CNN
+F 2 "" H 9338 3500 50  0001 C CNN
 F 3 "" H 9300 3650 50  0000 C CNN
 	1    9300 3650
@@
 F 0 "C211" H 10700 3200 50  0000 C CNN
 F 1 "100μF" H 10800 3000 50  0000 C CNN
-F 2 "" H 10650 3100 50  0000 C CNN
+F 2 "" H 10650 3100 50  0001 C CNN
 F 3 "" H 10650 3100 50  0000 C CNN
 	1    10650 3100
@@
 F 0 "C207" H 9700 3200 50  0000 C CNN
 F 1 "100nF" H 9625 3000 50  0000 C CNN
-F 2 "" H 9788 2950 50  0000 C CNN
+F 2 "" H 9788 2950 50  0001 C CNN
 F 3 "" H 9750 3100 50  0000 C CNN
 	1    9750 3100
@@
 F 0 "C208" H 10000 3200 50  0000 C CNN
 F 1 "100nF" H 9925 3000 50  0000 C CNN
-F 2 "" H 10088 2950 50  0000 C CNN
+F 2 "" H 10088 2950 50  0001 C CNN
 F 3 "" H 10050 3100 50  0000 C CNN
 	1    10050 3100
@@
 F 0 "C201" H 9265 4196 50  0000 L CNN
 F 1 "22nF" H 9265 4105 50  0000 L CNN
-F 2 "" H 9188 4000 50  0000 C CNN
+F 2 "" H 9188 4000 50  0001 C CNN
 F 3 "" H 9150 4150 50  0000 C CNN
 	1    9150 4150
@@
 F 0 "R195" H 10700 6650 50  0000 R CNN
 F 1 "220mΩ" H 10700 6750 50  0000 R CNN
-F 2 "" V 10680 6700 50  0000 C CNN
+F 2 "" V 10680 6700 50  0001 C CNN
 F 3 "" H 10750 6700 50  0000 C CNN
 	1    10750 6700
@@
 F 0 "R194" H 9900 6650 50  0000 R CNN
 F 1 "220mΩ" H 9900 6750 50  0000 R CNN
-F 2 "" V 9880 6700 50  0000 C CNN
+F 2 "" V 9880 6700 50  0001 C CNN
 F 3 "" H 9950 6700 50  0000 C CNN
 	1    9950 6700
@@
 F 0 "R191" V 7200 3750 50  0000 C CNN
 F 1 "2.2Ω" V 7300 3750 50  0000 C CNN
-F 2 "" V 7230 3750 50  0000 C CNN
+F 2 "" V 7230 3750 50  0001 C CNN
 F 3 "" H 7300 3750 50  0000 C CNN
 	1    7300 3750
@@
 F 0 "C198" H 7150 4050 50  0000 L CNN
 F 1 "470nF" H 7125 3850 50  0000 L CNN
-F 2 "" H 7138 3800 50  0000 C CNN
+F 2 "" H 7138 3800 50  0001 C CNN
 F 3 "" H 7100 3950 50  0000 C CNN
 	1    7100 3950
@@
 F 0 "C209" H 10150 6800 50  0000 L CNN
 F 1 "100nF" H 10150 6600 50  0000 L CNN
-F 2 "" H 10138 6550 50  0000 C CNN
+F 2 "" H 10138 6550 50  0001 C CNN
 F 3 "" H 10100 6700 50  0000 C CNN
 	1    10100 6700
@@
 P 6050 4250
 F 0 "R189" H 6119 4296 50  0000 L CNN
-F 1 "10kΩ" H 6119 4205 50  0000 L CNN
-F 2 "" V 5980 4250 50  0000 C CNN
+F 1 "4.7kΩ" H 6119 4205 50  0000 L CNN
+F 2 "" V 5980 4250 50  0001 C CNN
 F 3 "" H 6050 4250 50  0000 C CNN
 	1    6050 4250
@@
 F 0 "C200" H 7550 4050 50  0000 L CNN
 F 1 "4.7μF" H 7550 3850 50  0000 L CNN
-F 2 "" H 7538 3800 50  0000 C CNN
+F 2 "" H 7538 3800 50  0001 C CNN
 F 3 "" H 7500 3950 50  0000 C CNN
 	1    7500 3950
@@
 F 0 "R192" H 9319 6746 50  0000 L CNN
 F 1 "5.23kΩ" H 9319 6655 50  0000 L CNN
-F 2 "" V 9180 6700 50  0000 C CNN
+F 2 "" V 9180 6700 50  0001 C CNN
 F 3 "" H 9250 6700 50  0000 C CNN
 	1    9250 6700
@@
 F 0 "R193" V 9250 6900 50  0000 C CNN
 F 1 "4.75kΩ" V 9350 6900 50  0000 C CNN
-F 2 "" V 9380 6900 50  0000 C CNN
+F 2 "" V 9380 6900 50  0001 C CNN
 F 3 "" H 9450 6900 50  0000 C CNN
 	1    9450 6900
@@
 P 6400 4250
 F 0 "R190" H 6469 4296 50  0000 L CNN
-F 1 "10kΩ" H 6469 4205 50  0000 L CNN
-F 2 "" V 6330 4250 50  0000 C CNN
+F 1 "4.7kΩ" H 6469 4205 50  0000 L CNN
+F 2 "" V 6330 4250 50  0001 C CNN
 F 3 "" H 6400 4250 50  0000 C CNN
 	1    6400 4250
@@
 F 0 "C212" H 10950 6800 50  0000 L CNN
 F 1 "100nF" H 10950 6600 50  0000 L CNN
-F 2 "" H 10938 6550 50  0000 C CNN
+F 2 "" H 10938 6550 50  0001 C CNN
 F 3 "" H 10900 6700 50  0000 C CNN
 	1    10900 6700
@@
 F 0 "C202" H 9175 5050 50  0000 L CNN
 F 1 "470pF" H 9150 4850 50  0000 L CNN
-F 2 "" H 9188 4800 50  0000 C CNN
+F 2 "" H 9188 4800 50  0001 C CNN
 F 3 "" H 9150 4950 50  0000 C CNN
 	1    9150 4950
@@
 F 0 "C205" H 9375 5050 50  0000 L CNN
 F 1 "470pF" H 9375 4850 50  0000 L CNN
-F 2 "" H 9388 4800 50  0000 C CNN
+F 2 "" H 9388 4800 50  0001 C CNN
 F 3 "" H 9350 4950 50  0000 C CNN
 	1    9350 4950
@@
 F 0 "C203" H 9175 5900 50  0000 L CNN
 F 1 "470pF" H 9150 5700 50  0000 L CNN
-F 2 "" H 9188 5650 50  0000 C CNN
+F 2 "" H 9188 5650 50  0001 C CNN
 F 3 "" H 9150 5800 50  0000 C CNN
 	1    9150 5800
@@
 F 0 "C206" H 9375 5900 50  0000 L CNN
 F 1 "470pF" H 9375 5700 50  0000 L CNN
-F 2 "" H 9388 5650 50  0000 C CNN
+F 2 "" H 9388 5650 50  0001 C CNN
 F 3 "" H 9350 5800 50  0000 C CNN
 	1    9350 5800
@@
 F 0 "U28" H 7950 6200 60  0000 C CNN
 F 1 "TMC2130" H 8700 6200 60  0000 C CNN
-F 2 "" H 8400 5000 60  0000 C CNN
+F 2 "" H 8400 5000 60  0001 C CNN
 F 3 "" H 8400 5000 60  0000 C CNN
 	1    8400 4700
@@
 P 5700 4250
 F 0 "R188" H 5769 4296 50  0000 L CNN
-F 1 "10kΩ" H 5769 4205 50  0000 L CNN
-F 2 "" V 5630 4250 50  0000 C CNN
+F 1 "4.7kΩ" H 5769 4205 50  0000 L CNN
+F 2 "" V 5630 4250 50  0001 C CNN
 F 3 "" H 5700 4250 50  0000 C CNN
 	1    5700 4250
@@
 F 0 "C210" H 10300 3200 50  0000 C CNN
 F 1 "4.7μF" H 10225 3000 50  0000 C CNN
-F 2 "" H 10388 2950 50  0000 C CNN
+F 2 "" H 10388 2950 50  0001 C CNN
 F 3 "" H 10350 3100 50  0000 C CNN
 	1    10350 3100
@@
 F 0 "C197" H 6800 4050 50  0000 L CNN
 F 1 "100nF" H 6775 3850 50  0000 L CNN
-F 2 "" H 6788 3800 50  0000 C CNN
+F 2 "" H 6788 3800 50  0001 C CNN
 F 3 "" H 6750 3950 50  0000 C CNN
 	1    6750 3950

Commit message: Entry of additional component values
Parts:
- renumbered R188 to R187, R189 to R188, R190 to R189, R191 to R190, R192 to R191, R193 to R192, R194 to R193, R195 to R194
Changed lines of the file:
@@
 $EndComp
 $Comp
-L GND #PWR0264
+L GND #PWR0265
 U 1 1 5BA7E13F
 P 7500 3300
-F 0 "#PWR0264" H 7500 3050 50  0001 C CNN
+F 0 "#PWR0265" H 7500 3050 50  0001 C CNN
 F 1 "GND" H 7500 3150 50  0000 C CNN
 F 2 "" H 7500 3300 50  0000 C CNN
@@
 $EndComp
 $Comp
-L GND #PWR0265
+L GND #PWR0266
 U 1 1 58C092DF
 P 10350 3350
-F 0 "#PWR0265" H 10350 3100 50  0001 C CNN
+F 0 "#PWR0266" H 10350 3100 50  0001 C CNN
 F 1 "GND" H 10355 3177 50  0000 C CNN
 F 2 "" H 10350 3350 50  0000 C CNN
@@
 $EndComp
 $Comp
-L +24V #PWR0266
+L +24V #PWR0267
 U 1 1 5BA7E142
 P 8550 2850
-F 0 "#PWR0266" H 8550 2700 50  0001 C CNN
+F 0 "#PWR0267" H 8550 2700 50  0001 C CNN
 F 1 "+24V" H 8565 3023 50  0000 C CNN
 F 2 "" H 8550 2850 50  0000 C CNN
@@
 $EndComp
 $Comp
-L R R195
+L R R194
 U 1 1 5BA7E144
 P 10750 6700
-F 0 "R195" H 10700 6650 50  0000 R CNN
+F 0 "R194" H 10700 6650 50  0000 R CNN
 F 1 "220mΩ" H 10700 6750 50  0000 R CNN
 F 2 "" V 10680 6700 50  0001 C CNN
@@
 $EndComp
 $Comp
-L R R194
+L R R193
 U 1 1 5BA7E145
 P 9950 6700
-F 0 "R194" H 9900 6650 50  0000 R CNN
+F 0 "R193" H 9900 6650 50  0000 R CNN
 F 1 "220mΩ" H 9900 6750 50  0000 R CNN
 F 2 "" V 9880 6700 50  0001 C CNN
@@
 $EndComp
 $Comp
-L GND #PWR0267
+L GND #PWR0268
 U 1 1 58C09300
 P 9650 7050
-F 0 "#PWR0267" H 9650 6800 50  0001 C CNN
+F 0 "#PWR0268" H 9650 6800 50  0001 C CNN
 F 1 "GND" H 9655 6877 50  0000 C CNN
 F 2 "" H 9650 7050 50  0000 C CNN
@@
 NoConn ~ 7700 5600
 $Comp
-L R R191
+L R R190
 U 1 1 58C09307
 P 7300 3750
-F 0 "R191" V 7200 3750 50  0000 C CNN
+F 0 "R190" V 7200 3750 50  0000 C CNN
 F 1 "2.2Ω" V 7300 3750 50  0000 C CNN
 F 2 "" V 7230 3750 50  0001 C CNN
@@
 NoConn ~ 7700 5700
 $Comp
-L GND #PWR0268
+L GND #PWR0269
 U 1 1 58C09323
 P 7650 6100
-F 0 "#PWR0268" H 7650 5850 50  0001 C CNN
+F 0 "#PWR0269" H 7650 5850 50  0001 C CNN
 F 1 "GND" H 7655 5927 50  0000 C CNN
 F 2 "" H 7650 6100 50  0000 C CNN
@@
 X1_FAULT
 $Comp
-L R R189
+L R R188
 U 1 1 5BA7E14B
 P 6050 4250
-F 0 "R189" H 6119 4296 50  0000 L CNN
+F 0 "R188" H 6119 4296 50  0000 L CNN
 F 1 "4.7kΩ" H 6119 4205 50  0000 L CNN
 F 2 "" V 5980 4250 50  0001 C CNN
@@
 5VOUT
 $Comp
-L R R192
+L R R191
 U 1 1 58C09343
 P 9250 6700
-F 0 "R192" H 9319 6746 50  0000 L CNN
+F 0 "R191" H 9319 6746 50  0000 L CNN
 F 1 "5.23kΩ" H 9319 6655 50  0000 L CNN
 F 2 "" V 9180 6700 50  0001 C CNN
@@
 5VOUT
 $Comp
-L R R193
+L R R192
 U 1 1 58C0934B
 P 9450 6900
-F 0 "R193" V 9250 6900 50  0000 C CNN
+F 0 "R192" V 9250 6900 50  0000 C CNN
 F 1 "4.75kΩ" V 9350 6900 50  0000 C CNN
 F 2 "" V 9380 6900 50  0001 C CNN
@@
 $EndComp
 $Comp
-L R R190
+L R R189
 U 1 1 5BA7E14F
 P 6400 4250
-F 0 "R190" H 6469 4296 50  0000 L CNN
+F 0 "R189" H 6469 4296 50  0000 L CNN
 F 1 "4.7kΩ" H 6469 4205 50  0000 L CNN
 F 2 "" V 6330 4250 50  0001 C CNN
@@
 $EndComp
 $Comp
-L GND #PWR0269
+L GND #PWR0270
 U 1 1 5BA7E152
 P 9250 5200
-F 0 "#PWR0269" H 9250 4950 50  0001 C CNN
+F 0 "#PWR0270" H 9250 4950 50  0001 C CNN
 F 1 "GND" H 9250 5050 50  0000 C CNN
 F 2 "" H 9250 5200 50  0000 C CNN
@@
 $EndComp
 $Comp
-L GND #PWR0270
+L GND #PWR0271
 U 1 1 5BA7E155
 P 9250 6050
-F 0 "#PWR0270" H 9250 5800 50  0001 C CNN
+F 0 "#PWR0271" H 9250 5800 50  0001 C CNN
 F 1 "GND" H 9250 5900 50  0000 C CNN
 F 2 "" H 9250 6050 50  0000 C CNN
@@
 	9150 6000 9150 5950
 $Comp
-L R R188
+L R R187
 U 1 1 58C093FF
 P 5700 4250
-F 0 "R188" H 5769 4296 50  0000 L CNN
+F 0 "R187" H 5769 4296 50  0000 L CNN
 F 1 "4.7kΩ" H 5769 4205 50  0000 L CNN
 F 2 "" V 5630 4250 50  0001 C CNN
@@
 	5700 3500 7700 3500
 $Comp
-L VDD_3V3B #PWR0271
+L VDD_3V3B #PWR0272
 U 1 1 5BA7E15A
 P 6750 3450
-F 0 "#PWR0271" H 6750 3300 50  0001 C CNN
+F 0 "#PWR0272" H 6750 3300 50  0001 C CNN
 F 1 "VDD_3V3B" H 6765 3623 50  0000 C CNN
 F 2 "" H 6750 3450 50  0000 C CNN

Commit message: Add equivalent annotations document, associate more footprints
Parts:
- C199: renamed from C197; footprint (none) -> Capacitors_SMD:C_0603
- C200: renamed from C198; footprint (none) -> Capacitors_SMD:C_0603
- C201: renamed from C199; footprint (none) -> Capacitors_SMD:C_0603
- C202: renamed from C200; footprint (none) -> Capacitors_SMD:C_0402
- C203: renamed from C201; footprint (none) -> Capacitors_SMD:C_0402
- C204: renamed from C202; footprint (none) -> Capacitors_SMD:C_0603
- C205: renamed from C203; footprint (none) -> Capacitors_SMD:C_0603
- C206: renamed from C204; footprint (none) -> Capacitors_SMD:C_0603
- C207: renamed from C205; footprint (none) -> Capacitors_SMD:C_0603
- C208: renamed from C206; footprint (none) -> Capacitors_SMD:C_0603
- C209: renamed from C207; footprint (none) -> Capacitors_SMD:C_0603
- C210: renamed from C208; footprint (none) -> Capacitors_SMD:C_0603
- C211: renamed from C209; footprint (none) -> Capacitors_SMD:C_0603
- C212: renamed from C210; value 4.7μF -> 10μF; footprint (none) -> Capacitors_SMD:C_0805
- C213: renamed from C211; footprint (none) -> Capacitors_SMD:c_elec_8x10
- C214: renamed from C212; footprint (none) -> Capacitors_SMD:C_0603
- renumbered R187 to R186, R188 to R187, R189 to R188, R190 to R189, R191 to R190, R192 to R191, R193 to R192, R194 to R193
Changed lines of the file:
@@
 X1_SG
 $Comp
-L C C199
+L C C201
 U 1 1 58C092B6
 P 7500 3100
-F 0 "C199" H 7386 3054 50  0000 R CNN
+F 0 "C201" H 7386 3054 50  0000 R CNN
 F 1 "100nF" H 7386 3145 50  0000 R CNN
-F 2 "" H 7538 2950 50  0001 C CNN
+F 2 "Capacitors_SMD:C_0603" H 7538 2950 50  0001 C CNN
 F 3 "" H 7500 3100 50  0000 C CNN
 	1    7500 3100
@@
 $EndComp
 $Comp
-L C C204
+L C C206
 U 1 1 58C092BD
 P 9300 3650
-F 0 "C204" V 9250 3550 50  0000 C CNN
+F 0 "C206" V 9250 3550 50  0000 C CNN
 F 1 "100nF" V 9250 3825 50  0000 C CNN
-F 2 "" H 9338 3500 50  0001 C CNN
+F 2 "Capacitors_SMD:C_0603" H 9338 3500 50  0001 C CNN
 F 3 "" H 9300 3650 50  0000 C CNN
 	1    9300 3650
@@
 $EndComp
 $Comp
-L CP1 C211
+L CP1 C213
 U 1 1 5BA7E13D
 P 10650 3100
-F 0 "C211" H 10700 3200 50  0000 C CNN
+F 0 "C213" H 10750 3200 50  0000 C CNN
 F 1 "100μF" H 10800 3000 50  0000 C CNN
-F 2 "" H 10650 3100 50  0001 C CNN
+F 2 "Capacitors_SMD:c_elec_8x10" H 10650 3100 50  0001 C CNN
 F 3 "" H 10650 3100 50  0000 C CNN
 	1    10650 3100
@@
 $EndComp
 $Comp
-L C C207
+L C C209
 U 1 1 5BA7E13E
 P 9750 3100
-F 0 "C207" H 9700 3200 50  0000 C CNN
+F 0 "C209" H 9650 3200 50  0000 C CNN
 F 1 "100nF" H 9625 3000 50  0000 C CNN
-F 2 "" H 9788 2950 50  0001 C CNN
+F 2 "Capacitors_SMD:C_0603" H 9788 2950 50  0001 C CNN
 F 3 "" H 9750 3100 50  0000 C CNN
 	1    9750 3100
@@
 $EndComp
 $Comp
-L GND #PWR0265
+L GND #PWR0266
 U 1 1 5BA7E13F
 P 7500 3300
-F 0 "#PWR0265" H 7500 3050 50  0001 C CNN
+F 0 "#PWR0266" H 7500 3050 50  0001 C CNN
 F 1 "GND" H 7500 3150 50  0000 C CNN
 F 2 "" H 7500 3300 50  0000 C CNN
@@
 $EndComp
 $Comp
-L C C208
+L C C210
 U 1 1 58C092D8
 P 10050 3100
-F 0 "C208" H 10000 3200 50  0000 C CNN
+F 0 "C210" H 9950 3200 50  0000 C CNN
 F 1 "100nF" H 9925 3000 50  0000 C CNN
-F 2 "" H 10088 2950 50  0001 C CNN
+F 2 "Capacitors_SMD:C_0603" H 10088 2950 50  0001 C CNN
 F 3 "" H 10050 3100 50  0000 C CNN
 	1    10050 3100
@@
 $EndComp
 $Comp
-L GND #PWR0266
+L GND #PWR0267
 U 1 1 58C092DF
 P 10350 3350
-F 0 "#PWR0266" H 10350 3100 50  0001 C CNN
+F 0 "#PWR0267" H 10350 3100 50  0001 C CNN
 F 1 "GND" H 10355 3177 50  0000 C CNN
 F 2 "" H 10350 3350 50  0000 C CNN
@@
 $EndComp
 $Comp
-L +24V #PWR0267
+L +24V #PWR0268
 U 1 1 5BA7E142
 P 8550 2850
-F 0 "#PWR0267" H 8550 2700 50  0001 C CNN
+F 0 "#PWR0268" H 8550 2700 50  0001 C CNN
 F 1 "+24V" H 8565 3023 50  0000 C CNN
 F 2 "" H 8550 2850 50  0000 C CNN
@@
 $EndComp
 $Comp
-L C C201
+L C C203
 U 1 1 5BA7E143
 P 9150 4150
-F 0 "C201" H 9265 4196 50  0000 L CNN
+F 0 "C203" H 9265 4196 50  0000 L CNN
 F 1 "22nF" H 9265 4105 50  0000 L CNN
-F 2 "" H 9188 4000 50  0001 C CNN
+F 2 "Capacitors_SMD:C_0402" H 9188 4000 50  0001 C CNN
 F 3 "" H 9150 4150 50  0000 C CNN
 	1    9150 4150
@@
 $EndComp
 $Comp
-L R R194
+L R R193
 U 1 1 5BA7E144
 P 10750 6700
-F 0 "R194" H 10700 6650 50  0000 R CNN
+F 0 "R193" H 10700 6650 50  0000 R CNN
 F 1 "220mΩ" H 10700 6750 50  0000 R CNN
 F 2 "" V 10680 6700 50  0001 C CNN
@@
 $EndComp
 $Comp
-L R R193
+L R R192
 U 1 1 5BA7E145
 P 9950 6700
-F 0 "R193" H 9900 6650 50  0000 R CNN
+F 0 "R192" H 9900 6650 50  0000 R CNN
 F 1 "220mΩ" H 9900 6750 50  0000 R CNN
 F 2 "" V 9880 6700 50  0001 C CNN
@@
 $EndComp
 $Comp
-L GND #PWR0268
+L GND #PWR0269
 U 1 1 58C09300
 P 9650 7050
-F 0 "#PWR0268" H 9650 6800 50  0001 C CNN
+F 0 "#PWR0269" H 9650 6800 50  0001 C CNN
 F 1 "GND" H 9655 6877 50  0000 C CNN
 F 2 "" H 9650 7050 50  0000 C CNN
@@
 NoConn ~ 7700 5600
 $Comp
-L R R190
+L R R189
 U 1 1 58C09307
 P 7300 3750
-F 0 "R190" V 7200 3750 50  0000 C CNN
+F 0 "R189" V 7200 3750 50  0000 C CNN
 F 1 "2.2Ω" V 7300 3750 50  0000 C CNN
 F 2 "" V 7230 3750 50  0001 C CNN
@@
 $EndComp
 $Comp
-L C C198
+L C C200
 U 1 1 58C0930E
 P 7100 3950
-F 0 "C198" H 7150 4050 50  0000 L CNN
+F 0 "C200" H 7150 4050 50  0000 L CNN
 F 1 "470nF" H 7125 3850 50  0000 L CNN
-F 2 "" H 7138 3800 50  0001 C CNN
+F 2 "Capacitors_SMD:C_0603" H 7138 3800 50  0001 C CNN
 F 3 "" H 7100 3950 50  0000 C CNN
 	1    7100 3950
@@
 NoConn ~ 7700 5700
 $Comp
-L GND #PWR0269
+L GND #PWR0270
 U 1 1 58C09323
 P 7650 6100
-F 0 "#PWR0269" H 7650 5850 50  0001 C CNN
+F 0 "#PWR0270" H 7650 5850 50  0001 C CNN
 F 1 "GND" H 7655 5927 50  0000 C CNN
 F 2 "" H 7650 6100 50  0000 C CNN
@@
 $EndComp
 $Comp
-L C C209
+L C C211
 U 1 1 58C09329
 P 10100 6700
-F 0 "C209" H 10150 6800 50  0000 L CNN
+F 0 "C211" H 10150 6800 50  0000 L CNN
 F 1 "100nF" H 10150 6600 50  0000 L CNN
-F 2 "" H 10138 6550 50  0001 C CNN
+F 2 "Capacitors_SMD:C_0603" H 10138 6550 50  0001 C CNN
 F 3 "" H 10100 6700 50  0000 C CNN
 	1    10100 6700
@@
 X1_FAULT
 $Comp
-L R R188
+L R R187
 U 1 1 5BA7E14B
 P 6050 4250
-F 0 "R188" H 6119 4296 50  0000 L CNN
+F 0 "R187" H 6119 4296 50  0000 L CNN
 F 1 "4.7kΩ" H 6119 4205 50  0000 L CNN
 F 2 "" V 5980 4250 50  0001 C CNN
@@
 NoConn ~ 7700 4550
 $Comp
-L C C200
+L C C202
 U 1 1 58C0933B
 P 7500 3950
-F 0 "C200" H 7550 4050 50  0000 L CNN
+F 0 "C202" H 7550 4050 50  0000 L CNN
 F 1 "4.7μF" H 7550 3850 50  0000 L CNN
-F 2 "" H 7538 3800 50  0001 C CNN
+F 2 "Capacitors_SMD:C_0402" H 7538 3800 50  0001 C CNN
 F 3 "" H 7500 3950 50  0000 C CNN
 	1    7500 3950
@@
 5VOUT
 $Comp
-L R R191
+L R R190
 U 1 1 58C09343
 P 9250 6700
-F 0 "R191" H 9319 6746 50  0000 L CNN
+F 0 "R190" H 9319 6746 50  0000 L CNN
 F 1 "5.23kΩ" H 9319 6655 50  0000 L CNN
 F 2 "" V 9180 6700 50  0001 C CNN
@@
 5VOUT
 $Comp
-L R R192
+L R R191
 U 1 1 58C0934B
 P 9450 6900
-F 0 "R192" V 9250 6900 50  0000 C CNN
+F 0 "R191" V 9250 6900 50  0000 C CNN
 F 1 "4.75kΩ" V 9350 6900 50  0000 C CNN
 F 2 "" V 9380 6900 50  0001 C CNN
@@
 $EndComp
 $Comp
-L R R189
+L R R188
 U 1 1 5BA7E14F
 P 6400 4250
-F 0 "R189" H 6469 4296 50  0000 L CNN
+F 0 "R188" H 6469 4296 50  0000 L CNN
 F 1 "4.7kΩ" H 6469 4205 50  0000 L CNN
 F 2 "" V 6330 4250 50  0001 C CNN
@@
 $EndComp
 $Comp
-L C C212
+L C C214
 U 1 1 5BA7E150
 P 10900 6700
-F 0 "C212" H 10950 6800 50  0000 L CNN
+F 0 "C214" H 10950 6800 50  0000 L CNN
 F 1 "100nF" H 10950 6600 50  0000 L CNN
-F 2 "" H 10938 6550 50  0001 C CNN
+F 2 "Capacitors_SMD:C_0603" H 10938 6550 50  0001 C CNN
 F 3 "" H 10900 6700 50  0000 C CNN
 	1    10900 6700
@@
 $EndComp
 $Comp
-L C C202
+L C C204
 U 1 1 5BA7E151
 P 9150 4950
-F 0 "C202" H 9175 5050 50  0000 L CNN
+F 0 "C204" H 9175 5050 50  0000 L CNN
 F 1 "470pF" H 9150 4850 50  0000 L CNN
-F 2 "" H 9188 4800 50  0001 C CNN
+F 2 "Capacitors_SMD:C_0603" H 9188 4800 50  0001 C CNN
 F 3 "" H 9150 4950 50  0000 C CNN
 	1    9150 4950
@@
 $EndComp
 $Comp
-L GND #PWR0270
+L GND #PWR0271
 U 1 1 5BA7E152
 P 9250 5200
-F 0 "#PWR0270" H 9250 4950 50  0001 C CNN
+F 0 "#PWR0271" H 9250 4950 50  0001 C CNN
 F 1 "GND" H 9250 5050 50  0000 C CNN
 F 2 "" H 9250 5200 50  0000 C CNN
@@
 $EndComp
 $Comp
-L C C205
+L C C207
 U 1 1 5BA7E153
 P 9350 4950
-F 0 "C205" H 9375 5050 50  0000 L CNN
+F 0 "C207" H 9375 5050 50  0000 L CNN
 F 1 "470pF" H 9375 4850 50  0000 L CNN
-F 2 "" H 9388 4800 50  0001 C CNN
+F 2 "Capacitors_SMD:C_0603" H 9388 4800 50  0001 C CNN
 F 3 "" H 9350 4950 50  0000 C CNN
 	1    9350 4950
@@
 $EndComp
 $Comp
-L C C203
+L C C205
 U 1 1 58C09377
 P 9150 5800
-F 0 "C203" H 9175 5900 50  0000 L CNN
+F 0 "C205" H 9175 5900 50  0000 L CNN
 F 1 "470pF" H 9150 5700 50  0000 L CNN
-F 2 "" H 9188 5650 50  0001 C CNN
+F 2 "Capacitors_SMD:C_0603" H 9188 5650 50  0001 C CNN
 F 3 "" H 9150 5800 50  0000 C CNN
 	1    9150 5800
@@
 $EndComp
 $Comp
-L GND #PWR0271
+L GND #PWR0272
 U 1 1 5BA7E155
 P 9250 6050
-F 0 "#PWR0271" H 9250 5800 50  0001 C CNN
+F 0 "#PWR0272" H 9250 5800 50  0001 C CNN
 F 1 "GND" H 9250 5900 50  0000 C CNN
 F 2 "" H 9250 6050 50  0000 C CNN
@@
 $EndComp
 $Comp
-L C C206
+L C C208
 U 1 1 5BA7E156
 P 9350 5800
-F 0 "C206" H 9375 5900 50  0000 L CNN
+F 0 "C208" H 9375 5900 50  0000 L CNN
 F 1 "470pF" H 9375 5700 50  0000 L CNN
-F 2 "" H 9388 5650 50  0001 C CNN
+F 2 "Capacitors_SMD:C_0603" H 9388 5650 50  0001 C CNN
 F 3 "" H 9350 5800 50  0000 C CNN
 	1    9350 5800
@@
 	9150 6000 9150 5950
 $Comp
-L R R187
+L R R186
 U 1 1 58C093FF
 P 5700 4250
-F 0 "R187" H 5769 4296 50  0000 L CNN
+F 0 "R186" H 5769 4296 50  0000 L CNN
 F 1 "4.7kΩ" H 5769 4205 50  0000 L CNN
 F 2 "" V 5630 4250 50  0001 C CNN
@@
 Connection ~ 6050 3500
 $Comp
-L C C210
+L C C212
 U 1 1 58C0940A
 P 10350 3100
-F 0 "C210" H 10300 3200 50  0000 C CNN
-F 1 "4.7μF" H 10225 3000 50  0000 C CNN
-F 2 "" H 10388 2950 50  0001 C CNN
+F 0 "C212" H 10250 3200 50  0000 C CNN
+F 1 "10μF" H 10225 3000 50  0000 C CNN
+F 2 "Capacitors_SMD:C_0805" H 10388 2950 50  0001 C CNN
 F 3 "" H 10350 3100 50  0000 C CNN
 	1    10350 3100
@@
 	5700 3500 7700 3500
 $Comp
-L VDD_3V3B #PWR0272
+L VDD_3V3B #PWR0273
 U 1 1 5BA7E15A
 P 6750 3450
-F 0 "#PWR0272" H 6750 3300 50  0001 C CNN
+F 0 "#PWR0273" H 6750 3300 50  0001 C CNN
 F 1 "VDD_3V3B" H 6765 3623 50  0000 C CNN
 F 2 "" H 6750 3450 50  0000 C CNN
@@
 $EndComp
 $Comp
-L C C197
+L C C199
 U 1 1 5A89A0A1
 P 6750 3950
-F 0 "C197" H 6800 4050 50  0000 L CNN
+F 0 "C199" H 6800 4050 50  0000 L CNN
 F 1 "100nF" H 6775 3850 50  0000 L CNN
-F 2 "" H 6788 3800 50  0001 C CNN
+F 2 "Capacitors_SMD:C_0603" H 6788 3800 50  0001 C CNN
 F 3 "" H 6750 3950 50  0000 C CNN
 	1    6750 3950
