File: KiMBo/y_stepper.sch (KiCad schematic (older format))
At the start: 26 parts

Commit message: Use only one driver on Y, NAND X and Z FAULT and SG signals
Dual X carriage will need to be tested to determine if two seperate drivers are required for X
Parts:
- removed C?: 100nF, symbol C
- removed R?: 10kΩ, symbol R
- added C?: 100nF, symbol C
Connections:
- net GND: now also C?.2
- net VDD_3V3B: now also C?.1
- net Y1_A1 renamed Y_A1
- net Y1_A2 renamed Y_A2
- net Y1_B1 renamed Y_B1
- net Y1_B2 renamed Y_B2
- net Y1_DIR renamed Y_DIR
- net Y1_FAULT renamed Y_FAULT
- net Y1_SG renamed Y_SG
- net Y1_STEP renamed Y_STEP
- net ~Y1_EN renamed ~Y_EN
- net ~Y1_SS renamed ~Y_SS
Changed lines of the file:
@@
 $Descr A3 16535 11693
 encoding utf-8
-Sheet 26 27
+Sheet 25 26
 Title ""
 Date ""
@@
 $EndDescr
 Text HLabel 8450 4750 2    60   Output ~ 0
-Y1_A1
+Y_A1
 Text HLabel 8450 4900 2    60   Output ~ 0
-Y1_A2
+Y_A2
 Text HLabel 8450 5600 2    60   Output ~ 0
-Y1_B1
+Y_B1
 Text HLabel 8450 5750 2    60   Output ~ 0
-Y1_B2
+Y_B2
 Text HLabel 6650 6100 0    60   Input ~ 0
-Y1_STEP
+Y_STEP
 Text HLabel 6650 6200 0    60   Input ~ 0
-Y1_DIR
+Y_DIR
 Text HLabel 5400 5200 0    60   Input ~ 0
-~Y1_SS
+~Y_SS
 Text HLabel 6650 5300 0    60   Input ~ 0
 SCLK
@@
 MOSI
 Text HLabel 4700 4950 0    60   Output ~ 0
-Y1_SG
+Y_SG
 $Comp
 L C C?
@@
 	-1   0    0    -1
 $EndComp
-$Comp
-L C C?
-U 1 1 58C0B274
-P 5800 4100
-AR Path="/57AC927F/58BF2D49/58C0B274" Ref="C?"  Part="1"
-AR Path="/57AC927F/5A2A6632/58C0B274" Ref="C?"  Part="1"
-AR Path="/57AC927F/5A2D12A2/58C0B274" Ref="C?"  Part="1"
-F 0 "C?" H 5850 4200 50  0000 L CNN
-F 1 "100nF" H 5800 4000 50  0000 L CNN
-F 2 "" H 5838 3950 50  0000 C CNN
-F 3 "" H 5800 4100 50  0000 C CNN
-	1    5800 4100
-	-1   0    0    -1
-$EndComp
 NoConn ~ 6750 5850
 $Comp
@@
 $EndComp
 Text HLabel 5050 5050 0    60   Output ~ 0
-Y1_FAULT
+Y_FAULT
 $Comp
 L R R?
@@
 	-1   0    0    -1
 $EndComp
-Text HLabel 4300 4600 0    60   Input ~ 0
-~Y1_EN
+Text HLabel 4700 4600 0    60   Input ~ 0
+~Y_EN
 NoConn ~ 6750 4700
 $Comp
@@
 Connection ~ 6700 4350
 Wire Wire Line
-	5800 4350 6750 4350
+	5800 4350 6150 4350
+Wire Wire Line
+	6150 4350 6550 4350
+Wire Wire Line
+	6550 4350 6700 4350
+Wire Wire Line
+	6700 4350 6750 4350
 Wire Wire Line
 	6700 4450 6750 4450
@@
 Connection ~ 6700 4250
 Wire Wire Line
-	6700 4050 6700 6250
+	6700 4050 6700 4150
+Wire Wire Line
+	6700 4150 6700 4250
+Wire Wire Line
+	6700 4250 6700 4350
+Wire Wire Line
+	6700 4350 6700 4450
+Wire Wire Line
+	6700 4450 6700 5650
+Wire Wire Line
+	6700 5650 6700 5950
+Wire Wire Line
+	6700 5950 6700 6250
 Wire Wire Line
 	6750 4050 6700 4050
@@
 	6700 5650 6750 5650
 Wire Wire Line
-	8150 6400 9950 6400
-Wire Wire Line
-	8150 5750 8450 5750
+	8150 6400 9800 6400
+Wire Wire Line
+	9800 6400 9950 6400
+Wire Wire Line
+	8150 5750 8200 5750
+Wire Wire Line
+	8200 5750 8450 5750
 Wire Wire Line
 	8200 4100 8150 4100
@@
 	9700 3450 9700 3400
 Wire Wire Line
-	8800 3450 9700 3450
+	8800 3450 9100 3450
+Wire Wire Line
+	9100 3450 9400 3450
+Wire Wire Line
+	9400 3450 9700 3450
 Wire Wire Line
 	8800 3400 8800 3450
@@
 	6550 3400 6550 3450
 Wire Wire Line
-	8650 3050 8650 3800
+	8650 3050 8650 3500
+Wire Wire Line
+	8650 3500 8650 3600
+Wire Wire Line
+	8650 3600 8650 3800
 Wire Wire Line
 	8650 3800 8500 3800
@@
 	8150 3800 8200 3800
 Wire Wire Line
-	6550 3050 9700 3050
+	6550 3050 6700 3050
+Wire Wire Line
+	6700 3050 7600 3050
+Wire Wire Line
+	7600 3050 8650 3050
+Wire Wire Line
+	8650 3050 8800 3050
+Wire Wire Line
+	8800 3050 9100 3050
+Wire Wire Line
+	9100 3050 9400 3050
+Wire Wire Line
+	9400 3050 9700 3050
 Wire Wire Line
 	6700 3500 6700 3050
 Wire Wire Line
-	6500 3900 6750 3900
+	6500 3900 6550 3900
+Wire Wire Line
+	6550 3900 6750 3900
 Wire Wire Line
 	6750 4250 6700 4250
@@
 	6150 4250 6150 4350
 Wire Wire Line
-	6150 3750 6150 3950
+	6150 3750 6150 3900
+Wire Wire Line
+	6150 3900 6150 3950
 Wire Wire Line
 	6150 3900 6200 3900
@@
 Connection ~ 6150 3900
 Wire Wire Line
-	5800 3600 5800 3950
+	5800 3600 5800 3650
+Wire Wire Line
+	5800 3650 5800 3950
 Wire Wire Line
 	5800 4250 5800 4350
@@
 Connection ~ 9800 7150
 Wire Wire Line
-	8150 6550 9150 6550
+	8150 6550 9000 6550
+Wire Wire Line
+	9000 6550 9150 6550
 Connection ~ 9800 6400
 Wire Wire Line
-	5050 5050 6750 5050
+	5050 5050 5100 5050
+Wire Wire Line
+	5100 5050 6750 5050
 Wire Wire Line
 	5100 4550 5100 5050
@@
 Connection ~ 5100 5050
 Wire Wire Line
-	4300 4600 6750 4600
+	4700 4600 6750 4600
 Wire Wire Line
 	6550 3950 6550 3900
 Wire Wire Line
-	8150 7050 8350 7050
+	8150 7050 8300 7050
+Wire Wire Line
+	8300 7050 8350 7050
 Wire Wire Line
 	8300 6700 8300 6650
@@
 Connection ~ 8300 7050
 Wire Wire Line
-	8700 7050 8700 7200
+	8700 7050 8700 7150
+Wire Wire Line
+	8700 7150 8700 7200
 Connection ~ 8700 7150
 Wire Wire Line
 	8700 7050 8650 7050
 Wire Wire Line
-	5400 5200 6750 5200
+	5400 5200 5450 5200
+Wire Wire Line
+	5450 5200 6750 5200
 Wire Wire Line
 	5450 5200 5450 4550
@@
 Connection ~ 5450 3650
 Wire Wire Line
-	4700 4950 6750 4950
-Wire Wire Line
-	8200 5300 8400 5300
+	4700 4950 4750 4950
+Wire Wire Line
+	4750 4950 6750 4950
+Wire Wire Line
+	8200 5300 8300 5300
+Wire Wire Line
+	8300 5300 8400 5300
 Wire Wire Line
 	8200 4900 8200 4950
 Connection ~ 8200 4900
 Wire Wire Line
-	8200 6150 8400 6150
+	8200 6150 8300 6150
+Wire Wire Line
+	8300 6150 8400 6150
 Wire Wire Line
 	8200 5750 8200 5800
 Connection ~ 8200 5750
 Wire Wire Line
-	8150 7150 9950 7150
+	8150 7150 8700 7150
+Wire Wire Line
+	8700 7150 9000 7150
+Wire Wire Line
+	9000 7150 9150 7150
+Wire Wire Line
+	9150 7150 9800 7150
+Wire Wire Line
+	9800 7150 9950 7150
 Wire Wire Line
 	8300 6650 8550 6650
@@
 Connection ~ 9400 3050
 Wire Wire Line
-	9400 3400 9400 3500
+	9400 3400 9400 3450
+Wire Wire Line
+	9400 3450 9400 3500
 Connection ~ 9400 3450
 Wire Wire Line
 	9100 3400 9100 3450
 Wire Wire Line
-	8150 5600 8450 5600
+	8150 5600 8400 5600
+Wire Wire Line
+	8400 5600 8450 5600
 Wire Wire Line
 	8400 6150 8400 6100
@@
 	8400 5300 8400 5250
 Wire Wire Line
-	8150 4900 8450 4900
-Wire Wire Line
-	8150 4750 8450 4750
-$Comp
-L R R?
-U 1 1 58C0B37C
-P 4350 4800
-AR Path="/57AC927F/58BF2D49/58C0B37C" Ref="R?"  Part="1"
-AR Path="/57AC927F/5A2A6632/58C0B37C" Ref="R?"  Part="1"
-AR Path="/57AC927F/5A2D12A2/58C0B37C" Ref="R?"  Part="1"
-F 0 "R?" H 4419 4846 50  0000 L CNN
-F 1 "10kΩ" H 4419 4755 50  0000 L CNN
-F 2 "" V 4280 4800 50  0000 C CNN
-F 3 "" H 4350 4800 50  0000 C CNN
-	1    4350 4800
-	-1   0    0    -1
-$EndComp
-Connection ~ 4350 4600
-Wire Wire Line
-	4750 3650 6750 3650
-$Comp
-L GND #PWR?
-U 1 1 58C0B385
-P 4350 5000
-AR Path="/57AC927F/58BF2D49/58C0B385" Ref="#PWR?"  Part="1"
-AR Path="/57AC927F/5A2A6632/58C0B385" Ref="#PWR?"  Part="1"
-AR Path="/57AC927F/5A2D12A2/58C0B385" Ref="#PWR?"  Part="1"
-F 0 "#PWR?" H 4350 4750 50  0001 C CNN
-F 1 "GND" H 4355 4827 50  0000 C CNN
-F 2 "" H 4350 5000 50  0000 C CNN
-F 3 "" H 4350 5000 50  0000 C CNN
-	1    4350 5000
-	1    0    0    -1
-$EndComp
-Wire Wire Line
-	4350 5000 4350 4950
-Wire Wire Line
-	4350 4600 4350 4650
+	8150 4900 8200 4900
+Wire Wire Line
+	8200 4900 8450 4900
+Wire Wire Line
+	8150 4750 8400 4750
+Wire Wire Line
+	8400 4750 8450 4750
+Wire Wire Line
+	4750 3650 5100 3650
+Wire Wire Line
+	5100 3650 5450 3650
+Wire Wire Line
+	5450 3650 5800 3650
+Wire Wire Line
+	5800 3650 6750 3650
 $Comp
 L VDD_3V3B #PWR?
@@
 	1    0    0    -1
 $EndComp
+$Comp
+L C C?
+U 1 1 5A89AE9E
+P 5800 4100
+F 0 "C?" H 5850 4200 50  0000 L CNN
+F 1 "100nF" H 5825 4000 50  0000 L CNN
+F 2 "" H 5838 3950 50  0000 C CNN
+F 3 "" H 5800 4100 50  0000 C CNN
+	1    5800 4100
+	-1   0    0    -1
+$EndComp
 $EndSCHEMATC

Commit message: Annotate all components, now passing ERC, added ferrites to the rest of the connectors
Parts:
- gave numbers to parts that had none: 25

Commit message: Reorder the SS and EN lines from the shift registers such that the previously enabled/disabled motors stay enabled/disabled whilst writting to the shift register
Change 10k resistors to 4.7k, flip the open-drain inverter connected to B15 (PMTC_PGOOD)

Update the links in the README

Update the PDF schematic
Parts:
- R180, R181, R182: value 10kΩ -> 4.7kΩ
Changed lines of the file:
@@
 F 0 "C183" H 6436 3204 50  0000 R CNN
 F 1 "100nF" H 6436 3295 50  0000 R CNN
-F 2 "" H 6588 3100 50  0000 C CNN
+F 2 "" H 6588 3100 50  0001 C CNN
 F 3 "" H 6550 3250 50  0000 C CNN
 	1    6550 3250
@@
 F 0 "C188" V 8300 3700 50  0000 C CNN
 F 1 "100nF" V 8300 3975 50  0000 C CNN
-F 2 "" H 8388 3650 50  0000 C CNN
+F 2 "" H 8388 3650 50  0001 C CNN
 F 3 "" H 8350 3800 50  0000 C CNN
 	1    8350 3800
@@
 F 0 "C195" H 9750 3350 50  0000 C CNN
 F 1 "100μF" H 9850 3150 50  0000 C CNN
-F 2 "" H 9700 3250 50  0000 C CNN
+F 2 "" H 9700 3250 50  0001 C CNN
 F 3 "" H 9700 3250 50  0000 C CNN
 	1    9700 3250
@@
 F 0 "C191" H 8750 3350 50  0000 C CNN
 F 1 "100nF" H 8675 3150 50  0000 C CNN
-F 2 "" H 8838 3100 50  0000 C CNN
+F 2 "" H 8838 3100 50  0001 C CNN
 F 3 "" H 8800 3250 50  0000 C CNN
 	1    8800 3250
@@
 F 0 "C192" H 9050 3350 50  0000 C CNN
 F 1 "100nF" H 8975 3150 50  0000 C CNN
-F 2 "" H 9138 3100 50  0000 C CNN
+F 2 "" H 9138 3100 50  0001 C CNN
 F 3 "" H 9100 3250 50  0000 C CNN
 	1    9100 3250
@@
 F 0 "C185" H 8315 4346 50  0000 L CNN
 F 1 "22nF" H 8315 4255 50  0000 L CNN
-F 2 "" H 8238 4150 50  0000 C CNN
+F 2 "" H 8238 4150 50  0001 C CNN
 F 3 "" H 8200 4300 50  0000 C CNN
 	1    8200 4300
@@
 F 0 "R187" H 9750 6800 50  0000 R CNN
 F 1 "220mΩ" H 9750 6900 50  0000 R CNN
-F 2 "" V 9730 6850 50  0000 C CNN
+F 2 "" V 9730 6850 50  0001 C CNN
 F 3 "" H 9800 6850 50  0000 C CNN
 	1    9800 6850
@@
 F 0 "R186" H 8950 6800 50  0000 R CNN
 F 1 "220mΩ" H 8950 6900 50  0000 R CNN
-F 2 "" V 8930 6850 50  0000 C CNN
+F 2 "" V 8930 6850 50  0001 C CNN
 F 3 "" H 9000 6850 50  0000 C CNN
 	1    9000 6850
@@
 F 0 "R183" V 6250 3900 50  0000 C CNN
 F 1 "2.2Ω" V 6350 3900 50  0000 C CNN
-F 2 "" V 6280 3900 50  0000 C CNN
+F 2 "" V 6280 3900 50  0001 C CNN
 F 3 "" H 6350 3900 50  0000 C CNN
 	1    6350 3900
@@
 F 0 "C182" H 6200 4200 50  0000 L CNN
 F 1 "470nF" H 6175 4000 50  0000 L CNN
-F 2 "" H 6188 3950 50  0000 C CNN
+F 2 "" H 6188 3950 50  0001 C CNN
 F 3 "" H 6150 4100 50  0000 C CNN
 	1    6150 4100
@@
 F 0 "C193" H 9200 6950 50  0000 L CNN
 F 1 "100nF" H 9200 6750 50  0000 L CNN
-F 2 "" H 9188 6700 50  0000 C CNN
+F 2 "" H 9188 6700 50  0001 C CNN
 F 3 "" H 9150 6850 50  0000 C CNN
 	1    9150 6850
@@
 P 5100 4400
 F 0 "R181" H 5169 4446 50  0000 L CNN
-F 1 "10kΩ" H 5169 4355 50  0000 L CNN
-F 2 "" V 5030 4400 50  0000 C CNN
+F 1 "4.7kΩ" H 5169 4355 50  0000 L CNN
+F 2 "" V 5030 4400 50  0001 C CNN
 F 3 "" H 5100 4400 50  0000 C CNN
 	1    5100 4400
@@
 F 0 "C184" H 6600 4200 50  0000 L CNN
 F 1 "4.7μF" H 6600 4000 50  0000 L CNN
-F 2 "" H 6588 3950 50  0000 C CNN
+F 2 "" H 6588 3950 50  0001 C CNN
 F 3 "" H 6550 4100 50  0000 C CNN
 	1    6550 4100
@@
 F 0 "R184" H 8369 6896 50  0000 L CNN
 F 1 "5.23kΩ" H 8369 6805 50  0000 L CNN
-F 2 "" V 8230 6850 50  0000 C CNN
+F 2 "" V 8230 6850 50  0001 C CNN
 F 3 "" H 8300 6850 50  0000 C CNN
 	1    8300 6850
@@
 F 0 "R185" V 8300 7050 50  0000 C CNN
 F 1 "4.75kΩ" V 8400 7050 50  0000 C CNN
-F 2 "" V 8430 7050 50  0000 C CNN
+F 2 "" V 8430 7050 50  0001 C CNN
 F 3 "" H 8500 7050 50  0000 C CNN
 	1    8500 7050
@@
 P 5450 4400
 F 0 "R182" H 5519 4446 50  0000 L CNN
-F 1 "10kΩ" H 5519 4355 50  0000 L CNN
-F 2 "" V 5380 4400 50  0000 C CNN
+F 1 "4.7kΩ" H 5519 4355 50  0000 L CNN
+F 2 "" V 5380 4400 50  0001 C CNN
 F 3 "" H 5450 4400 50  0000 C CNN
 	1    5450 4400
@@
 F 0 "C196" H 10000 6950 50  0000 L CNN
 F 1 "100nF" H 10000 6750 50  0000 L CNN
-F 2 "" H 9988 6700 50  0000 C CNN
+F 2 "" H 9988 6700 50  0001 C CNN
 F 3 "" H 9950 6850 50  0000 C CNN
 	1    9950 6850
@@
 F 0 "C186" H 8225 5200 50  0000 L CNN
 F 1 "470pF" H 8200 5000 50  0000 L CNN
-F 2 "" H 8238 4950 50  0000 C CNN
+F 2 "" H 8238 4950 50  0001 C CNN
 F 3 "" H 8200 5100 50  0000 C CNN
 	1    8200 5100
@@
 F 0 "C189" H 8425 5200 50  0000 L CNN
 F 1 "470pF" H 8425 5000 50  0000 L CNN
-F 2 "" H 8438 4950 50  0000 C CNN
+F 2 "" H 8438 4950 50  0001 C CNN
 F 3 "" H 8400 5100 50  0000 C CNN
 	1    8400 5100
@@
 F 0 "C187" H 8225 6050 50  0000 L CNN
 F 1 "470pF" H 8200 5850 50  0000 L CNN
-F 2 "" H 8238 5800 50  0000 C CNN
+F 2 "" H 8238 5800 50  0001 C CNN
 F 3 "" H 8200 5950 50  0000 C CNN
 	1    8200 5950
@@
 F 0 "C190" H 8425 6050 50  0000 L CNN
 F 1 "470pF" H 8425 5850 50  0000 L CNN
-F 2 "" H 8438 5800 50  0000 C CNN
+F 2 "" H 8438 5800 50  0001 C CNN
 F 3 "" H 8400 5950 50  0000 C CNN
 	1    8400 5950
@@
 F 0 "U27" H 7000 6350 60  0000 C CNN
 F 1 "TMC2130" H 7750 6350 60  0000 C CNN
-F 2 "" H 7450 5150 60  0000 C CNN
+F 2 "" H 7450 5150 60  0001 C CNN
 F 3 "" H 7450 5150 60  0000 C CNN
 	1    7450 4850
@@
 P 4750 4400
 F 0 "R180" H 4819 4446 50  0000 L CNN
-F 1 "10kΩ" H 4819 4355 50  0000 L CNN
-F 2 "" V 4680 4400 50  0000 C CNN
+F 1 "4.7kΩ" H 4819 4355 50  0000 L CNN
+F 2 "" V 4680 4400 50  0001 C CNN
 F 3 "" H 4750 4400 50  0000 C CNN
 	1    4750 4400
@@
 F 0 "C194" H 9350 3350 50  0000 C CNN
 F 1 "4.7μF" H 9275 3150 50  0000 C CNN
-F 2 "" H 9438 3100 50  0000 C CNN
+F 2 "" H 9438 3100 50  0001 C CNN
 F 3 "" H 9400 3250 50  0000 C CNN
 	1    9400 3250
@@
 F 0 "C181" H 5850 4200 50  0000 L CNN
 F 1 "100nF" H 5825 4000 50  0000 L CNN
-F 2 "" H 5838 3950 50  0000 C CNN
+F 2 "" H 5838 3950 50  0001 C CNN
 F 3 "" H 5800 4100 50  0000 C CNN
 	1    5800 4100

Commit message: Entry of additional component values
Parts:
- renumbered R180 to R179, R181 to R180, R182 to R181, R183 to R182, R184 to R183, R185 to R184, R186 to R185, R187 to R186
Changed lines of the file:
@@
 $EndComp
 $Comp
-L GND #PWR0256
+L GND #PWR0257
 U 1 1 58C0B231
 P 6550 3450
-F 0 "#PWR0256" H 6550 3200 50  0001 C CNN
+F 0 "#PWR0257" H 6550 3200 50  0001 C CNN
 F 1 "GND" H 6550 3300 50  0000 C CNN
 F 2 "" H 6550 3450 50  0000 C CNN
@@
 $EndComp
 $Comp
-L GND #PWR0257
+L GND #PWR0258
 U 1 1 58C0B23E
 P 9400 3500
-F 0 "#PWR0257" H 9400 3250 50  0001 C CNN
+F 0 "#PWR0258" H 9400 3250 50  0001 C CNN
 F 1 "GND" H 9405 3327 50  0000 C CNN
 F 2 "" H 9400 3500 50  0000 C CNN
@@
 $EndComp
 $Comp
-L +24V #PWR0258
+L +24V #PWR0259
 U 1 1 58C0B244
 P 7600 3000
-F 0 "#PWR0258" H 7600 2850 50  0001 C CNN
+F 0 "#PWR0259" H 7600 2850 50  0001 C CNN
 F 1 "+24V" H 7615 3173 50  0000 C CNN
 F 2 "" H 7600 3000 50  0000 C CNN
@@
 $EndComp
 $Comp
-L R R187
+L R R186
 U 1 1 58C0B251
 P 9800 6850
-F 0 "R187" H 9750 6800 50  0000 R CNN
+F 0 "R186" H 9750 6800 50  0000 R CNN
 F 1 "220mΩ" H 9750 6900 50  0000 R CNN
 F 2 "" V 9730 6850 50  0001 C CNN
@@
 $EndComp
 $Comp
-L R R186
+L R R185
 U 1 1 58C0B258
 P 9000 6850
-F 0 "R186" H 8950 6800 50  0000 R CNN
+F 0 "R185" H 8950 6800 50  0000 R CNN
 F 1 "220mΩ" H 8950 6900 50  0000 R CNN
 F 2 "" V 8930 6850 50  0001 C CNN
@@
 $EndComp
 $Comp
-L GND #PWR0259
+L GND #PWR0260
 U 1 1 58C0B25F
 P 8700 7200
-F 0 "#PWR0259" H 8700 6950 50  0001 C CNN
+F 0 "#PWR0260" H 8700 6950 50  0001 C CNN
 F 1 "GND" H 8705 7027 50  0000 C CNN
 F 2 "" H 8700 7200 50  0000 C CNN
@@
 NoConn ~ 6750 5750
 $Comp
-L R R183
+L R R182
 U 1 1 58C0B266
 P 6350 3900
-F 0 "R183" V 6250 3900 50  0000 C CNN
+F 0 "R182" V 6250 3900 50  0000 C CNN
 F 1 "2.2Ω" V 6350 3900 50  0000 C CNN
 F 2 "" V 6280 3900 50  0001 C CNN
@@
 NoConn ~ 6750 5850
 $Comp
-L GND #PWR0260
+L GND #PWR0261
 U 1 1 58C0B282
 P 6700 6250
-F 0 "#PWR0260" H 6700 6000 50  0001 C CNN
+F 0 "#PWR0261" H 6700 6000 50  0001 C CNN
 F 1 "GND" H 6705 6077 50  0000 C CNN
 F 2 "" H 6700 6250 50  0000 C CNN
@@
 Y_FAULT
 $Comp
-L R R181
+L R R180
 U 1 1 58C0B290
 P 5100 4400
-F 0 "R181" H 5169 4446 50  0000 L CNN
+F 0 "R180" H 5169 4446 50  0000 L CNN
 F 1 "4.7kΩ" H 5169 4355 50  0000 L CNN
 F 2 "" V 5030 4400 50  0001 C CNN
@@
 5VOUT
 $Comp
-L R R184
+L R R183
 U 1 1 58C0B2A2
 P 8300 6850
-F 0 "R184" H 8369 6896 50  0000 L CNN
+F 0 "R183" H 8369 6896 50  0000 L CNN
 F 1 "5.23kΩ" H 8369 6805 50  0000 L CNN
 F 2 "" V 8230 6850 50  0001 C CNN
@@
 5VOUT
 $Comp
-L R R185
+L R R184
 U 1 1 58C0B2AA
 P 8500 7050
-F 0 "R185" V 8300 7050 50  0000 C CNN
+F 0 "R184" V 8300 7050 50  0000 C CNN
 F 1 "4.75kΩ" V 8400 7050 50  0000 C CNN
 F 2 "" V 8430 7050 50  0001 C CNN
@@
 $EndComp
 $Comp
-L R R182
+L R R181
 U 1 1 58C0B2B1
 P 5450 4400
-F 0 "R182" H 5519 4446 50  0000 L CNN
+F 0 "R181" H 5519 4446 50  0000 L CNN
 F 1 "4.7kΩ" H 5519 4355 50  0000 L CNN
 F 2 "" V 5380 4400 50  0001 C CNN
@@
 $EndComp
 $Comp
-L GND #PWR0261
+L GND #PWR0262
 U 1 1 58C0B2C6
 P 8300 5350
-F 0 "#PWR0261" H 8300 5100 50  0001 C CNN
+F 0 "#PWR0262" H 8300 5100 50  0001 C CNN
 F 1 "GND" H 8300 5200 50  0000 C CNN
 F 2 "" H 8300 5350 50  0000 C CNN
@@
 $EndComp
 $Comp
-L GND #PWR0262
+L GND #PWR0263
 U 1 1 58C0B2DA
 P 8300 6200
-F 0 "#PWR0262" H 8300 5950 50  0001 C CNN
+F 0 "#PWR0263" H 8300 5950 50  0001 C CNN
 F 1 "GND" H 8300 6050 50  0000 C CNN
 F 2 "" H 8300 6200 50  0000 C CNN
@@
 	8200 6150 8200 6100
 $Comp
-L R R180
+L R R179
 U 1 1 58C0B35B
 P 4750 4400
-F 0 "R180" H 4819 4446 50  0000 L CNN
+F 0 "R179" H 4819 4446 50  0000 L CNN
 F 1 "4.7kΩ" H 4819 4355 50  0000 L CNN
 F 2 "" V 4680 4400 50  0001 C CNN
@@
 	4750 3650 6750 3650
 $Comp
-L VDD_3V3B #PWR0263
+L VDD_3V3B #PWR0264
 U 1 1 5A300CA5
 P 5800 3600
-F 0 "#PWR0263" H 5800 3450 50  0001 C CNN
+F 0 "#PWR0264" H 5800 3450 50  0001 C CNN
 F 1 "VDD_3V3B" H 5815 3773 50  0000 C CNN
 F 2 "" H 5800 3600 50  0000 C CNN
