File: KiMBo/y_stepper.sch (KiCad schematic (older format))
At the start: 25 parts, among them U27 TMC2130

Commit message: Add equivalent annotations document, associate more footprints
Parts:
- C183: renamed from C181; footprint (none) -> Capacitors_SMD:C_0603
- C184: renamed from C182; footprint (none) -> Capacitors_SMD:C_0603
- C185: renamed from C183; footprint (none) -> Capacitors_SMD:C_0603
- C186: renamed from C184; footprint (none) -> Capacitors_SMD:C_0402
- C187: renamed from C185; footprint (none) -> Capacitors_SMD:C_0402
- C188: renamed from C186; footprint (none) -> Capacitors_SMD:C_0603
- C189: renamed from C187; footprint (none) -> Capacitors_SMD:C_0603
- C190: renamed from C188; footprint (none) -> Capacitors_SMD:C_0603
- C191: renamed from C189; footprint (none) -> Capacitors_SMD:C_0603
- C192: renamed from C190; footprint (none) -> Capacitors_SMD:C_0603
- C193: renamed from C191; footprint (none) -> Capacitors_SMD:C_0603
- C194: renamed from C192; footprint (none) -> Capacitors_SMD:C_0603
- C195: renamed from C193; footprint (none) -> Capacitors_SMD:C_0603
- C196: renamed from C194; value 4.7μF -> 10μF; footprint (none) -> Capacitors_SMD:C_0805
- C197: renamed from C195; footprint (none) -> Capacitors_SMD:c_elec_8x10
- C198: renamed from C196; footprint (none) -> Capacitors_SMD:C_0603
- renumbered R179 to R178, R180 to R179, R181 to R180, R182 to R181, R183 to R182, R184 to R183, R185 to R184, R186 to R185
Changed lines of the file:
@@
 Y_SG
 $Comp
-L C C183
+L C C185
 U 1 1 58C0B215
 P 6550 3250
-F 0 "C183" H 6436 3204 50  0000 R CNN
+F 0 "C185" H 6436 3204 50  0000 R CNN
 F 1 "100nF" H 6436 3295 50  0000 R CNN
-F 2 "" H 6588 3100 50  0001 C CNN
+F 2 "Capacitors_SMD:C_0603" H 6588 3100 50  0001 C CNN
 F 3 "" H 6550 3250 50  0000 C CNN
 	1    6550 3250
@@
 $EndComp
 $Comp
-L C C188
+L C C190
 U 1 1 58C0B21C
 P 8350 3800
-F 0 "C188" V 8300 3700 50  0000 C CNN
+F 0 "C190" V 8300 3700 50  0000 C CNN
 F 1 "100nF" V 8300 3975 50  0000 C CNN
-F 2 "" H 8388 3650 50  0001 C CNN
+F 2 "Capacitors_SMD:C_0603" H 8388 3650 50  0001 C CNN
 F 3 "" H 8350 3800 50  0000 C CNN
 	1    8350 3800
@@
 $EndComp
 $Comp
-L CP1 C195
+L CP1 C197
 U 1 1 58C0B223
 P 9700 3250
-F 0 "C195" H 9750 3350 50  0000 C CNN
+F 0 "C197" H 9800 3350 50  0000 C CNN
 F 1 "100μF" H 9850 3150 50  0000 C CNN
-F 2 "" H 9700 3250 50  0001 C CNN
+F 2 "Capacitors_SMD:c_elec_8x10" H 9700 3250 50  0001 C CNN
 F 3 "" H 9700 3250 50  0000 C CNN
 	1    9700 3250
@@
 $EndComp
 $Comp
-L C C191
+L C C193
 U 1 1 58C0B22A
 P 8800 3250
-F 0 "C191" H 8750 3350 50  0000 C CNN
+F 0 "C193" H 8700 3350 50  0000 C CNN
 F 1 "100nF" H 8675 3150 50  0000 C CNN
-F 2 "" H 8838 3100 50  0001 C CNN
+F 2 "Capacitors_SMD:C_0603" H 8838 3100 50  0001 C CNN
 F 3 "" H 8800 3250 50  0000 C CNN
 	1    8800 3250
@@
 $EndComp
 $Comp
-L GND #PWR0257
+L GND #PWR0258
 U 1 1 58C0B231
 P 6550 3450
-F 0 "#PWR0257" H 6550 3200 50  0001 C CNN
+F 0 "#PWR0258" H 6550 3200 50  0001 C CNN
 F 1 "GND" H 6550 3300 50  0000 C CNN
 F 2 "" H 6550 3450 50  0000 C CNN
@@
 $EndComp
 $Comp
-L C C192
+L C C194
 U 1 1 58C0B237
 P 9100 3250
-F 0 "C192" H 9050 3350 50  0000 C CNN
+F 0 "C194" H 9000 3350 50  0000 C CNN
 F 1 "100nF" H 8975 3150 50  0000 C CNN
-F 2 "" H 9138 3100 50  0001 C CNN
+F 2 "Capacitors_SMD:C_0603" H 9138 3100 50  0001 C CNN
 F 3 "" H 9100 3250 50  0000 C CNN
 	1    9100 3250
@@
 $EndComp
 $Comp
-L GND #PWR0258
+L GND #PWR0259
 U 1 1 58C0B23E
 P 9400 3500
-F 0 "#PWR0258" H 9400 3250 50  0001 C CNN
+F 0 "#PWR0259" H 9400 3250 50  0001 C CNN
 F 1 "GND" H 9405 3327 50  0000 C CNN
 F 2 "" H 9400 3500 50  0000 C CNN
@@
 $EndComp
 $Comp
-L +24V #PWR0259
+L +24V #PWR0260
 U 1 1 58C0B244
 P 7600 3000
-F 0 "#PWR0259" H 7600 2850 50  0001 C CNN
+F 0 "#PWR0260" H 7600 2850 50  0001 C CNN
 F 1 "+24V" H 7615 3173 50  0000 C CNN
 F 2 "" H 7600 3000 50  0000 C CNN
@@
 $EndComp
 $Comp
-L C C185
+L C C187
 U 1 1 58C0B24A
 P 8200 4300
-F 0 "C185" H 8315 4346 50  0000 L CNN
+F 0 "C187" H 8315 4346 50  0000 L CNN
 F 1 "22nF" H 8315 4255 50  0000 L CNN
-F 2 "" H 8238 4150 50  0001 C CNN
+F 2 "Capacitors_SMD:C_0402" H 8238 4150 50  0001 C CNN
 F 3 "" H 8200 4300 50  0000 C CNN
 	1    8200 4300
@@
 $EndComp
 $Comp
-L R R186
+L R R185
 U 1 1 58C0B251
 P 9800 6850
-F 0 "R186" H 9750 6800 50  0000 R CNN
+F 0 "R185" H 9750 6800 50  0000 R CNN
 F 1 "220mΩ" H 9750 6900 50  0000 R CNN
 F 2 "" V 9730 6850 50  0001 C CNN
@@
 $EndComp
 $Comp
-L R R185
+L R R184
 U 1 1 58C0B258
 P 9000 6850
-F 0 "R185" H 8950 6800 50  0000 R CNN
+F 0 "R184" H 8950 6800 50  0000 R CNN
 F 1 "220mΩ" H 8950 6900 50  0000 R CNN
 F 2 "" V 8930 6850 50  0001 C CNN
@@
 $EndComp
 $Comp
-L GND #PWR0260
+L GND #PWR0261
 U 1 1 58C0B25F
 P 8700 7200
-F 0 "#PWR0260" H 8700 6950 50  0001 C CNN
+F 0 "#PWR0261" H 8700 6950 50  0001 C CNN
 F 1 "GND" H 8705 7027 50  0000 C CNN
 F 2 "" H 8700 7200 50  0000 C CNN
@@
 NoConn ~ 6750 5750
 $Comp
-L R R182
+L R R181
 U 1 1 58C0B266
 P 6350 3900
-F 0 "R182" V 6250 3900 50  0000 C CNN
+F 0 "R181" V 6250 3900 50  0000 C CNN
 F 1 "2.2Ω" V 6350 3900 50  0000 C CNN
 F 2 "" V 6280 3900 50  0001 C CNN
@@
 $EndComp
 $Comp
-L C C182
+L C C184
 U 1 1 58C0B26D
 P 6150 4100
-F 0 "C182" H 6200 4200 50  0000 L CNN
+F 0 "C184" H 6200 4200 50  0000 L CNN
 F 1 "470nF" H 6175 4000 50  0000 L CNN
-F 2 "" H 6188 3950 50  0001 C CNN
+F 2 "Capacitors_SMD:C_0603" H 6188 3950 50  0001 C CNN
 F 3 "" H 6150 4100 50  0000 C CNN
 	1    6150 4100
@@
 NoConn ~ 6750 5850
 $Comp
-L GND #PWR0261
+L GND #PWR0262
 U 1 1 58C0B282
 P 6700 6250
-F 0 "#PWR0261" H 6700 6000 50  0001 C CNN
+F 0 "#PWR0262" H 6700 6000 50  0001 C CNN
 F 1 "GND" H 6705 6077 50  0000 C CNN
 F 2 "" H 6700 6250 50  0000 C CNN
@@
 $EndComp
 $Comp
-L C C193
+L C C195
 U 1 1 58C0B288
 P 9150 6850
-F 0 "C193" H 9200 6950 50  0000 L CNN
+F 0 "C195" H 9200 6950 50  0000 L CNN
 F 1 "100nF" H 9200 6750 50  0000 L CNN
-F 2 "" H 9188 6700 50  0001 C CNN
+F 2 "Capacitors_SMD:C_0603" H 9188 6700 50  0001 C CNN
 F 3 "" H 9150 6850 50  0000 C CNN
 	1    9150 6850
@@
 Y_FAULT
 $Comp
-L R R180
+L R R179
 U 1 1 58C0B290
 P 5100 4400
-F 0 "R180" H 5169 4446 50  0000 L CNN
+F 0 "R179" H 5169 4446 50  0000 L CNN
 F 1 "4.7kΩ" H 5169 4355 50  0000 L CNN
 F 2 "" V 5030 4400 50  0001 C CNN
@@
 NoConn ~ 6750 4700
 $Comp
-L C C184
+L C C186
 U 1 1 58C0B29A
 P 6550 4100
-F 0 "C184" H 6600 4200 50  0000 L CNN
+F 0 "C186" H 6600 4200 50  0000 L CNN
 F 1 "4.7μF" H 6600 4000 50  0000 L CNN
-F 2 "" H 6588 3950 50  0001 C CNN
+F 2 "Capacitors_SMD:C_0402" H 6588 3950 50  0001 C CNN
 F 3 "" H 6550 4100 50  0000 C CNN
 	1    6550 4100
@@
 5VOUT
 $Comp
-L R R183
+L R R182
 U 1 1 58C0B2A2
 P 8300 6850
-F 0 "R183" H 8369 6896 50  0000 L CNN
+F 0 "R182" H 8369 6896 50  0000 L CNN
 F 1 "5.23kΩ" H 8369 6805 50  0000 L CNN
 F 2 "" V 8230 6850 50  0001 C CNN
@@
 5VOUT
 $Comp
-L R R184
+L R R183
 U 1 1 58C0B2AA
 P 8500 7050
-F 0 "R184" V 8300 7050 50  0000 C CNN
+F 0 "R183" V 8300 7050 50  0000 C CNN
 F 1 "4.75kΩ" V 8400 7050 50  0000 C CNN
 F 2 "" V 8430 7050 50  0001 C CNN
@@
 $EndComp
 $Comp
-L R R181
+L R R180
 U 1 1 58C0B2B1
 P 5450 4400
-F 0 "R181" H 5519 4446 50  0000 L CNN
+F 0 "R180" H 5519 4446 50  0000 L CNN
 F 1 "4.7kΩ" H 5519 4355 50  0000 L CNN
 F 2 "" V 5380 4400 50  0001 C CNN
@@
 $EndComp
 $Comp
-L C C196
+L C C198
 U 1 1 58C0B2B8
 P 9950 6850
-F 0 "C196" H 10000 6950 50  0000 L CNN
+F 0 "C198" H 10000 6950 50  0000 L CNN
 F 1 "100nF" H 10000 6750 50  0000 L CNN
-F 2 "" H 9988 6700 50  0001 C CNN
+F 2 "Capacitors_SMD:C_0603" H 9988 6700 50  0001 C CNN
 F 3 "" H 9950 6850 50  0000 C CNN
 	1    9950 6850
@@
 $EndComp
 $Comp
-L C C186
+L C C188
 U 1 1 58C0B2BF
 P 8200 5100
-F 0 "C186" H 8225 5200 50  0000 L CNN
+F 0 "C188" H 8225 5200 50  0000 L CNN
 F 1 "470pF" H 8200 5000 50  0000 L CNN
-F 2 "" H 8238 4950 50  0001 C CNN
+F 2 "Capacitors_SMD:C_0603" H 8238 4950 50  0001 C CNN
 F 3 "" H 8200 5100 50  0000 C CNN
 	1    8200 5100
@@
 $EndComp
 $Comp
-L GND #PWR0262
+L GND #PWR0263
 U 1 1 58C0B2C6
 P 8300 5350
-F 0 "#PWR0262" H 8300 5100 50  0001 C CNN
+F 0 "#PWR0263" H 8300 5100 50  0001 C CNN
 F 1 "GND" H 8300 5200 50  0000 C CNN
 F 2 "" H 8300 5350 50  0000 C CNN
@@
 $EndComp
 $Comp
-L C C189
+L C C191
 U 1 1 58C0B2CC
 P 8400 5100
-F 0 "C189" H 8425 5200 50  0000 L CNN
+F 0 "C191" H 8425 5200 50  0000 L CNN
 F 1 "470pF" H 8425 5000 50  0000 L CNN
-F 2 "" H 8438 4950 50  0001 C CNN
+F 2 "Capacitors_SMD:C_0603" H 8438 4950 50  0001 C CNN
 F 3 "" H 8400 5100 50  0000 C CNN
 	1    8400 5100
@@
 $EndComp
 $Comp
-L C C187
+L C C189
 U 1 1 58C0B2D3
 P 8200 5950
-F 0 "C187" H 8225 6050 50  0000 L CNN
+F 0 "C189" H 8225 6050 50  0000 L CNN
 F 1 "470pF" H 8200 5850 50  0000 L CNN
-F 2 "" H 8238 5800 50  0001 C CNN
+F 2 "Capacitors_SMD:C_0603" H 8238 5800 50  0001 C CNN
 F 3 "" H 8200 5950 50  0000 C CNN
 	1    8200 5950
@@
 $EndComp
 $Comp
-L GND #PWR0263
+L GND #PWR0264
 U 1 1 58C0B2DA
 P 8300 6200
-F 0 "#PWR0263" H 8300 5950 50  0001 C CNN
+F 0 "#PWR0264" H 8300 5950 50  0001 C CNN
 F 1 "GND" H 8300 6050 50  0000 C CNN
 F 2 "" H 8300 6200 50  0000 C CNN
@@
 $EndComp
 $Comp
-L C C190
+L C C192
 U 1 1 58C0B2E0
 P 8400 5950
-F 0 "C190" H 8425 6050 50  0000 L CNN
+F 0 "C192" H 8425 6050 50  0000 L CNN
 F 1 "470pF" H 8425 5850 50  0000 L CNN
-F 2 "" H 8438 5800 50  0001 C CNN
+F 2 "Capacitors_SMD:C_0603" H 8438 5800 50  0001 C CNN
 F 3 "" H 8400 5950 50  0000 C CNN
 	1    8400 5950
@@
 	8200 6150 8200 6100
 $Comp
-L R R179
+L R R178
 U 1 1 58C0B35B
 P 4750 4400
-F 0 "R179" H 4819 4446 50  0000 L CNN
+F 0 "R178" H 4819 4446 50  0000 L CNN
 F 1 "4.7kΩ" H 4819 4355 50  0000 L CNN
 F 2 "" V 4680 4400 50  0001 C CNN
@@
 Connection ~ 5100 3650
 $Comp
-L C C194
+L C C196
 U 1 1 58C0B366
 P 9400 3250
-F 0 "C194" H 9350 3350 50  0000 C CNN
-F 1 "4.7μF" H 9275 3150 50  0000 C CNN
-F 2 "" H 9438 3100 50  0001 C CNN
+F 0 "C196" H 9300 3350 50  0000 C CNN
+F 1 "10μF" H 9275 3150 50  0000 C CNN
+F 2 "Capacitors_SMD:C_0805" H 9438 3100 50  0001 C CNN
 F 3 "" H 9400 3250 50  0000 C CNN
 	1    9400 3250
@@
 	4750 3650 6750 3650
 $Comp
-L VDD_3V3B #PWR0264
+L VDD_3V3B #PWR0265
 U 1 1 5A300CA5
 P 5800 3600
-F 0 "#PWR0264" H 5800 3450 50  0001 C CNN
+F 0 "#PWR0265" H 5800 3450 50  0001 C CNN
 F 1 "VDD_3V3B" H 5815 3773 50  0000 C CNN
 F 2 "" H 5800 3600 50  0000 C CNN
@@
 $EndComp
 $Comp
-L C C181
+L C C183
 U 1 1 5A89AE9E
 P 5800 4100
-F 0 "C181" H 5850 4200 50  0000 L CNN
+F 0 "C183" H 5850 4200 50  0000 L CNN
 F 1 "100nF" H 5825 4000 50  0000 L CNN
-F 2 "" H 5838 3950 50  0001 C CNN
+F 2 "Capacitors_SMD:C_0603" H 5838 3950 50  0001 C CNN
 F 3 "" H 5800 4100 50  0000 C CNN
 	1    5800 4100

Commit message: Connect X and Z stepper driver open-drain DIAG0 and DIAG1 lines together
Parts:
- renumbered C183 to C181, C184 to C182, C185 to C183, C186 to C184, C187 to C185, C188 to C186, C189 to C187, C190 to C188, C191 to C189, C192 to C190, C193 to C191, C194 to C192, C195 to C193, C196 to C194, C197 to C195, C198 to C196, R178 to R174, R179 to R175, R180 to R176, R181 to R177, R182 to R178, R183 to R179, R184 to R180, R185 to R181, U27 to U25
Changed lines of the file:
@@
 Y_SG
 $Comp
-L C C185
+L C C183
 U 1 1 58C0B215
 P 6550 3250
-F 0 "C185" H 6436 3204 50  0000 R CNN
+F 0 "C183" H 6436 3204 50  0000 R CNN
 F 1 "100nF" H 6436 3295 50  0000 R CNN
 F 2 "Capacitors_SMD:C_0603" H 6588 3100 50  0001 C CNN
@@
 $EndComp
 $Comp
-L C C190
+L C C188
 U 1 1 58C0B21C
 P 8350 3800
-F 0 "C190" V 8300 3700 50  0000 C CNN
+F 0 "C188" V 8300 3700 50  0000 C CNN
 F 1 "100nF" V 8300 3975 50  0000 C CNN
 F 2 "Capacitors_SMD:C_0603" H 8388 3650 50  0001 C CNN
@@
 $EndComp
 $Comp
-L CP1 C197
+L CP1 C195
 U 1 1 58C0B223
 P 9700 3250
-F 0 "C197" H 9800 3350 50  0000 C CNN
+F 0 "C195" H 9800 3350 50  0000 C CNN
 F 1 "100μF" H 9850 3150 50  0000 C CNN
 F 2 "Capacitors_SMD:c_elec_8x10" H 9700 3250 50  0001 C CNN
@@
 $EndComp
 $Comp
-L C C193
+L C C191
 U 1 1 58C0B22A
 P 8800 3250
-F 0 "C193" H 8700 3350 50  0000 C CNN
+F 0 "C191" H 8700 3350 50  0000 C CNN
 F 1 "100nF" H 8675 3150 50  0000 C CNN
 F 2 "Capacitors_SMD:C_0603" H 8838 3100 50  0001 C CNN
@@
 $EndComp
 $Comp
-L GND #PWR0258
+L GND #PWR0248
 U 1 1 58C0B231
 P 6550 3450
-F 0 "#PWR0258" H 6550 3200 50  0001 C CNN
+F 0 "#PWR0248" H 6550 3200 50  0001 C CNN
 F 1 "GND" H 6550 3300 50  0000 C CNN
 F 2 "" H 6550 3450 50  0000 C CNN
@@
 $EndComp
 $Comp
-L C C194
+L C C192
 U 1 1 58C0B237
 P 9100 3250
-F 0 "C194" H 9000 3350 50  0000 C CNN
+F 0 "C192" H 9000 3350 50  0000 C CNN
 F 1 "100nF" H 8975 3150 50  0000 C CNN
 F 2 "Capacitors_SMD:C_0603" H 9138 3100 50  0001 C CNN
@@
 $EndComp
 $Comp
-L GND #PWR0259
+L GND #PWR0249
 U 1 1 58C0B23E
 P 9400 3500
-F 0 "#PWR0259" H 9400 3250 50  0001 C CNN
+F 0 "#PWR0249" H 9400 3250 50  0001 C CNN
 F 1 "GND" H 9405 3327 50  0000 C CNN
 F 2 "" H 9400 3500 50  0000 C CNN
@@
 $EndComp
 $Comp
-L +24V #PWR0260
+L +24V #PWR0250
 U 1 1 58C0B244
 P 7600 3000
-F 0 "#PWR0260" H 7600 2850 50  0001 C CNN
+F 0 "#PWR0250" H 7600 2850 50  0001 C CNN
 F 1 "+24V" H 7615 3173 50  0000 C CNN
 F 2 "" H 7600 3000 50  0000 C CNN
@@
 $EndComp
 $Comp
-L C C187
+L C C185
 U 1 1 58C0B24A
 P 8200 4300
-F 0 "C187" H 8315 4346 50  0000 L CNN
+F 0 "C185" H 8315 4346 50  0000 L CNN
 F 1 "22nF" H 8315 4255 50  0000 L CNN
 F 2 "Capacitors_SMD:C_0402" H 8238 4150 50  0001 C CNN
@@
 $EndComp
 $Comp
-L R R185
+L R R181
 U 1 1 58C0B251
 P 9800 6850
-F 0 "R185" H 9750 6800 50  0000 R CNN
+F 0 "R181" H 9750 6800 50  0000 R CNN
 F 1 "220mΩ" H 9750 6900 50  0000 R CNN
 F 2 "" V 9730 6850 50  0001 C CNN
@@
 $EndComp
 $Comp
-L R R184
+L R R180
 U 1 1 58C0B258
 P 9000 6850
-F 0 "R184" H 8950 6800 50  0000 R CNN
+F 0 "R180" H 8950 6800 50  0000 R CNN
 F 1 "220mΩ" H 8950 6900 50  0000 R CNN
 F 2 "" V 8930 6850 50  0001 C CNN
@@
 $EndComp
 $Comp
-L GND #PWR0261
+L GND #PWR0251
 U 1 1 58C0B25F
 P 8700 7200
-F 0 "#PWR0261" H 8700 6950 50  0001 C CNN
+F 0 "#PWR0251" H 8700 6950 50  0001 C CNN
 F 1 "GND" H 8705 7027 50  0000 C CNN
 F 2 "" H 8700 7200 50  0000 C CNN
@@
 NoConn ~ 6750 5750
 $Comp
-L R R181
+L R R177
 U 1 1 58C0B266
 P 6350 3900
-F 0 "R181" V 6250 3900 50  0000 C CNN
+F 0 "R177" V 6250 3900 50  0000 C CNN
 F 1 "2.2Ω" V 6350 3900 50  0000 C CNN
 F 2 "" V 6280 3900 50  0001 C CNN
@@
 $EndComp
 $Comp
-L C C184
+L C C182
 U 1 1 58C0B26D
 P 6150 4100
-F 0 "C184" H 6200 4200 50  0000 L CNN
+F 0 "C182" H 6200 4200 50  0000 L CNN
 F 1 "470nF" H 6175 4000 50  0000 L CNN
 F 2 "Capacitors_SMD:C_0603" H 6188 3950 50  0001 C CNN
@@
 NoConn ~ 6750 5850
 $Comp
-L GND #PWR0262
+L GND #PWR0252
 U 1 1 58C0B282
 P 6700 6250
-F 0 "#PWR0262" H 6700 6000 50  0001 C CNN
+F 0 "#PWR0252" H 6700 6000 50  0001 C CNN
 F 1 "GND" H 6705 6077 50  0000 C CNN
 F 2 "" H 6700 6250 50  0000 C CNN
@@
 $EndComp
 $Comp
-L C C195
+L C C193
 U 1 1 58C0B288
 P 9150 6850
-F 0 "C195" H 9200 6950 50  0000 L CNN
+F 0 "C193" H 9200 6950 50  0000 L CNN
 F 1 "100nF" H 9200 6750 50  0000 L CNN
 F 2 "Capacitors_SMD:C_0603" H 9188 6700 50  0001 C CNN
@@
 Y_FAULT
 $Comp
-L R R179
+L R R175
 U 1 1 58C0B290
 P 5100 4400
-F 0 "R179" H 5169 4446 50  0000 L CNN
+F 0 "R175" H 5169 4446 50  0000 L CNN
 F 1 "4.7kΩ" H 5169 4355 50  0000 L CNN
 F 2 "" V 5030 4400 50  0001 C CNN
@@
 NoConn ~ 6750 4700
 $Comp
-L C C186
+L C C184
 U 1 1 58C0B29A
 P 6550 4100
-F 0 "C186" H 6600 4200 50  0000 L CNN
+F 0 "C184" H 6600 4200 50  0000 L CNN
 F 1 "4.7μF" H 6600 4000 50  0000 L CNN
 F 2 "Capacitors_SMD:C_0402" H 6588 3950 50  0001 C CNN
@@
 5VOUT
 $Comp
-L R R182
+L R R178
 U 1 1 58C0B2A2
 P 8300 6850
-F 0 "R182" H 8369 6896 50  0000 L CNN
+F 0 "R178" H 8369 6896 50  0000 L CNN
 F 1 "5.23kΩ" H 8369 6805 50  0000 L CNN
 F 2 "" V 8230 6850 50  0001 C CNN
@@
 5VOUT
 $Comp
-L R R183
+L R R179
 U 1 1 58C0B2AA
 P 8500 7050
-F 0 "R183" V 8300 7050 50  0000 C CNN
+F 0 "R179" V 8300 7050 50  0000 C CNN
 F 1 "4.75kΩ" V 8400 7050 50  0000 C CNN
 F 2 "" V 8430 7050 50  0001 C CNN
@@
 $EndComp
 $Comp
-L R R180
+L R R176
 U 1 1 58C0B2B1
 P 5450 4400
-F 0 "R180" H 5519 4446 50  0000 L CNN
+F 0 "R176" H 5519 4446 50  0000 L CNN
 F 1 "4.7kΩ" H 5519 4355 50  0000 L CNN
 F 2 "" V 5380 4400 50  0001 C CNN
@@
 $EndComp
 $Comp
-L C C198
+L C C196
 U 1 1 58C0B2B8
 P 9950 6850
-F 0 "C198" H 10000 6950 50  0000 L CNN
+F 0 "C196" H 10000 6950 50  0000 L CNN
 F 1 "100nF" H 10000 6750 50  0000 L CNN
 F 2 "Capacitors_SMD:C_0603" H 9988 6700 50  0001 C CNN
@@
 $EndComp
 $Comp
-L C C188
+L C C186
 U 1 1 58C0B2BF
 P 8200 5100
-F 0 "C188" H 8225 5200 50  0000 L CNN
+F 0 "C186" H 8225 5200 50  0000 L CNN
 F 1 "470pF" H 8200 5000 50  0000 L CNN
 F 2 "Capacitors_SMD:C_0603" H 8238 4950 50  0001 C CNN
@@
 $EndComp
 $Comp
-L GND #PWR0263
+L GND #PWR0253
 U 1 1 58C0B2C6
 P 8300 5350
-F 0 "#PWR0263" H 8300 5100 50  0001 C CNN
+F 0 "#PWR0253" H 8300 5100 50  0001 C CNN
 F 1 "GND" H 8300 5200 50  0000 C CNN
 F 2 "" H 8300 5350 50  0000 C CNN
@@
 $EndComp
 $Comp
-L C C191
+L C C189
 U 1 1 58C0B2CC
 P 8400 5100
-F 0 "C191" H 8425 5200 50  0000 L CNN
+F 0 "C189" H 8425 5200 50  0000 L CNN
 F 1 "470pF" H 8425 5000 50  0000 L CNN
 F 2 "Capacitors_SMD:C_0603" H 8438 4950 50  0001 C CNN
@@
 $EndComp
 $Comp
-L C C189
+L C C187
 U 1 1 58C0B2D3
 P 8200 5950
-F 0 "C189" H 8225 6050 50  0000 L CNN
+F 0 "C187" H 8225 6050 50  0000 L CNN
 F 1 "470pF" H 8200 5850 50  0000 L CNN
 F 2 "Capacitors_SMD:C_0603" H 8238 5800 50  0001 C CNN
@@
 $EndComp
 $Comp
-L GND #PWR0264
+L GND #PWR0254
 U 1 1 58C0B2DA
 P 8300 6200
-F 0 "#PWR0264" H 8300 5950 50  0001 C CNN
+F 0 "#PWR0254" H 8300 5950 50  0001 C CNN
 F 1 "GND" H 8300 6050 50  0000 C CNN
 F 2 "" H 8300 6200 50  0000 C CNN
@@
 $EndComp
 $Comp
-L C C192
+L C C190
 U 1 1 58C0B2E0
 P 8400 5950
-F 0 "C192" H 8425 6050 50  0000 L CNN
+F 0 "C190" H 8425 6050 50  0000 L CNN
 F 1 "470pF" H 8425 5850 50  0000 L CNN
 F 2 "Capacitors_SMD:C_0603" H 8438 5800 50  0001 C CNN
@@
 $EndComp
 $Comp
-L TMC2130 U27
+L TMC2130 U25
 U 1 1 58C0B2E7
 P 7450 4850
-F 0 "U27" H 7000 6350 60  0000 C CNN
+F 0 "U25" H 7000 6350 60  0000 C CNN
 F 1 "TMC2130" H 7750 6350 60  0000 C CNN
 F 2 "" H 7450 5150 60  0001 C CNN
@@
 	8200 6150 8200 6100
 $Comp
-L R R178
+L R R174
 U 1 1 58C0B35B
 P 4750 4400
-F 0 "R178" H 4819 4446 50  0000 L CNN
+F 0 "R174" H 4819 4446 50  0000 L CNN
 F 1 "4.7kΩ" H 4819 4355 50  0000 L CNN
 F 2 "" V 4680 4400 50  0001 C CNN
@@
 Connection ~ 5100 3650
 $Comp
-L C C196
+L C C194
 U 1 1 58C0B366
 P 9400 3250
-F 0 "C196" H 9300 3350 50  0000 C CNN
+F 0 "C194" H 9300 3350 50  0000 C CNN
 F 1 "10μF" H 9275 3150 50  0000 C CNN
 F 2 "Capacitors_SMD:C_0805" H 9438 3100 50  0001 C CNN
@@
 	4750 3650 6750 3650
 $Comp
-L VDD_3V3B #PWR0265
+L VDD_3V3B #PWR0255
 U 1 1 5A300CA5
 P 5800 3600
-F 0 "#PWR0265" H 5800 3450 50  0001 C CNN
+F 0 "#PWR0255" H 5800 3450 50  0001 C CNN
 F 1 "VDD_3V3B" H 5815 3773 50  0000 C CNN
 F 2 "" H 5800 3600 50  0000 C CNN
@@
 $EndComp
 $Comp
-L C C183
+L C C181
 U 1 1 5A89AE9E
 P 5800 4100
-F 0 "C183" H 5850 4200 50  0000 L CNN
+F 0 "C181" H 5850 4200 50  0000 L CNN
 F 1 "100nF" H 5825 4000 50  0000 L CNN
 F 2 "Capacitors_SMD:C_0603" H 5838 3950 50  0001 C CNN
