File: KiMBo/endstop.sch (KiCad schematic (older format))
At the start: 19 parts

Commit message: Annotate all components, now passing ERC, added ferrites to the rest of the connectors
Parts:
- gave numbers to parts that had none: 19
Changed lines of the file:
@@
 X1
 $Comp
-L C C?
+L C C36
 U 1 1 58129032
 P 6150 5500
-F 0 "C?" H 6264 5546 50  0000 L CNN
+F 0 "C36" H 6264 5546 50  0000 L CNN
 F 1 "4.7μF" H 6264 5455 50  0000 L CNN
 F 2 "" H 6188 5350 50  0000 C CNN
@@
 $EndComp
 $Comp
-L R R?
+L R R64
 U 1 1 58129040
 P 6150 5100
-F 0 "R?" H 6081 5054 50  0000 R CNN
+F 0 "R64" H 6081 5054 50  0000 R CNN
 F 1 "4.7kΩ" H 6081 5145 50  0000 R CNN
 F 2 "" V 6080 5100 50  0000 C CNN
@@
 $EndComp
 Wire Wire Line
-	6100 5300 6150 5300
-Wire Wire Line
-	6150 5300 6200 5300
+	6100 5300 6200 5300
 Wire Wire Line
 	6150 5650 6150 5700
 Connection ~ 6150 5300
 Wire Wire Line
-	6150 5250 6150 5300
-Wire Wire Line
-	6150 5300 6150 5350
+	6150 5250 6150 5350
 Wire Wire Line
 	6150 4950 6150 4900
 $Comp
-L R R?
+L R R63
 U 1 1 5812D30B
 P 5950 5300
-F 0 "R?" V 6157 5300 50  0000 C CNN
+F 0 "R63" V 6157 5300 50  0000 C CNN
 F 1 "4.7kΩ" V 6066 5300 50  0000 C CNN
 F 2 "" V 5880 5300 50  0000 C CNN
@@
 Y1
 $Comp
-L C C?
+L C C37
 U 1 1 589415E7
 P 7700 5500
-F 0 "C?" H 7814 5546 50  0000 L CNN
+F 0 "C37" H 7814 5546 50  0000 L CNN
 F 1 "4.7μF" H 7814 5455 50  0000 L CNN
 F 2 "" H 7738 5350 50  0000 C CNN
@@
 $EndComp
 $Comp
-L R R?
+L R R66
 U 1 1 589415EE
 P 7700 5100
-F 0 "R?" H 7631 5054 50  0000 R CNN
+F 0 "R66" H 7631 5054 50  0000 R CNN
 F 1 "4.7kΩ" H 7631 5145 50  0000 R CNN
 F 2 "" V 7630 5100 50  0000 C CNN
@@
 $EndComp
 Wire Wire Line
-	7650 5300 7700 5300
-Wire Wire Line
-	7700 5300 7750 5300
+	7650 5300 7750 5300
 Wire Wire Line
 	7700 5650 7700 5700
 Connection ~ 7700 5300
 Wire Wire Line
-	7700 5250 7700 5300
-Wire Wire Line
-	7700 5300 7700 5350
+	7700 5250 7700 5350
 Wire Wire Line
 	7700 4950 7700 4900
 $Comp
-L R R?
+L R R65
 U 1 1 58941610
 P 7500 5300
-F 0 "R?" V 7707 5300 50  0000 C CNN
+F 0 "R65" V 7707 5300 50  0000 C CNN
 F 1 "4.7kΩ" V 7616 5300 50  0000 C CNN
 F 2 "" V 7430 5300 50  0000 C CNN
@@
 Z1
 $Comp
-L C C?
+L C C38
 U 1 1 58941879
 P 9300 5500
-F 0 "C?" H 9414 5546 50  0000 L CNN
+F 0 "C38" H 9414 5546 50  0000 L CNN
 F 1 "4.7μF" H 9414 5455 50  0000 L CNN
 F 2 "" H 9338 5350 50  0000 C CNN
@@
 $EndComp
 $Comp
-L R R?
+L R R68
 U 1 1 58941880
 P 9300 5100
-F 0 "R?" H 9231 5054 50  0000 R CNN
+F 0 "R68" H 9231 5054 50  0000 R CNN
 F 1 "4.7kΩ" H 9231 5145 50  0000 R CNN
 F 2 "" V 9230 5100 50  0000 C CNN
@@
 $EndComp
 Wire Wire Line
-	9250 5300 9300 5300
-Wire Wire Line
-	9300 5300 9350 5300
+	9250 5300 9350 5300
 Wire Wire Line
 	9300 5650 9300 5700
 Connection ~ 9300 5300
 Wire Wire Line
-	9300 5250 9300 5300
-Wire Wire Line
-	9300 5300 9300 5350
+	9300 5250 9300 5350
 Wire Wire Line
 	9300 4950 9300 4900
 $Comp
-L R R?
+L R R67
 U 1 1 589418A2
 P 9100 5300
-F 0 "R?" V 9307 5300 50  0000 C CNN
+F 0 "R67" V 9307 5300 50  0000 C CNN
 F 1 "4.7kΩ" V 9216 5300 50  0000 C CNN
 F 2 "" V 9030 5300 50  0000 C CNN
@@
 ENC_A
 $Comp
-L C C?
+L C C39
 U 1 1 5894C248
 P 11100 5000
-F 0 "C?" H 11214 5046 50  0000 L CNN
+F 0 "C39" H 11214 5046 50  0000 L CNN
 F 1 "4.7μF" H 11214 4955 50  0000 L CNN
 F 2 "" H 11138 4850 50  0000 C CNN
@@
 $EndComp
 Wire Wire Line
-	11050 4800 11100 4800
-Wire Wire Line
-	11100 4800 11150 4800
+	11050 4800 11150 4800
 Wire Wire Line
 	11100 5150 11100 5200
@@
 	11100 6000 11100 6050
 $Comp
-L C C?
+L C C40
 U 1 1 5894C2A4
 P 11100 6200
-F 0 "C?" H 11214 6246 50  0000 L CNN
+F 0 "C40" H 11214 6246 50  0000 L CNN
 F 1 "4.7μF" H 11214 6155 50  0000 L CNN
 F 2 "" H 11138 6050 50  0000 C CNN
@@
 ENC_B_IN
 $Comp
-L VDD_3V3B #PWR0131
+L VDD_3V3B #PWR0179
 U 1 1 59E67523
 P 6150 4900
-F 0 "#PWR0131" H 6150 4750 50  0001 C CNN
+F 0 "#PWR0179" H 6150 4750 50  0001 C CNN
 F 1 "VDD_3V3B" H 6165 5073 50  0000 C CNN
 F 2 "" H 6150 4900 50  0000 C CNN
@@
 $EndComp
 $Comp
-L VDD_3V3B #PWR0132
+L VDD_3V3B #PWR0180
 U 1 1 59E6755C
 P 7700 4900
-F 0 "#PWR0132" H 7700 4750 50  0001 C CNN
+F 0 "#PWR0180" H 7700 4750 50  0001 C CNN
 F 1 "VDD_3V3B" H 7715 5073 50  0000 C CNN
 F 2 "" H 7700 4900 50  0000 C CNN
@@
 $EndComp
 $Comp
-L VDD_3V3B #PWR0133
+L VDD_3V3B #PWR0181
 U 1 1 59E6758E
 P 9300 4900
-F 0 "#PWR0133" H 9300 4750 50  0001 C CNN
+F 0 "#PWR0181" H 9300 4750 50  0001 C CNN
 F 1 "VDD_3V3B" H 9315 5073 50  0000 C CNN
 F 2 "" H 9300 4900 50  0000 C CNN
@@
 $EndComp
 Wire Wire Line
-	11050 6000 11100 6000
-Wire Wire Line
-	11100 6000 11150 6000
-$Comp
-L GND #PWR0134
+	11050 6000 11150 6000
+$Comp
+L GND #PWR0182
 U 1 1 59E68F88
 P 11100 5200
-F 0 "#PWR0134" H 11100 4950 50  0001 C CNN
+F 0 "#PWR0182" H 11100 4950 50  0001 C CNN
 F 1 "GND" H 11105 5027 50  0000 C CNN
 F 2 "" H 11100 5200 50  0000 C CNN
@@
 $EndComp
 $Comp
-L GND #PWR0135
+L GND #PWR0183
 U 1 1 59E68FBB
 P 11100 6400
-F 0 "#PWR0135" H 11100 6150 50  0001 C CNN
+F 0 "#PWR0183" H 11100 6150 50  0001 C CNN
 F 1 "GND" H 11105 6227 50  0000 C CNN
 F 2 "" H 11100 6400 50  0000 C CNN
@@
 $EndComp
 $Comp
-L GND #PWR0136
+L GND #PWR0184
 U 1 1 59E68FE7
 P 9300 5700
-F 0 "#PWR0136" H 9300 5450 50  0001 C CNN
+F 0 "#PWR0184" H 9300 5450 50  0001 C CNN
 F 1 "GND" H 9305 5527 50  0000 C CNN
 F 2 "" H 9300 5700 50  0000 C CNN
@@
 $EndComp
 $Comp
-L GND #PWR0137
+L GND #PWR0185
 U 1 1 59E69013
 P 7700 5700
-F 0 "#PWR0137" H 7700 5450 50  0001 C CNN
+F 0 "#PWR0185" H 7700 5450 50  0001 C CNN
 F 1 "GND" H 7705 5527 50  0000 C CNN
 F 2 "" H 7700 5700 50  0000 C CNN
@@
 $EndComp
 $Comp
-L GND #PWR0138
+L GND #PWR0186
 U 1 1 59E6903F
 P 6150 5700
-F 0 "#PWR0138" H 6150 5450 50  0001 C CNN
+F 0 "#PWR0186" H 6150 5450 50  0001 C CNN
 F 1 "GND" H 6155 5527 50  0000 C CNN
 F 2 "" H 6150 5700 50  0000 C CNN
@@
 RC=22.09ms
 Wire Wire Line
-	8400 5300 8450 5300
-Wire Wire Line
-	8450 5300 8500 5300
+	8400 5300 8500 5300
 Wire Wire Line
 	8950 5300 8700 5300
@@
 	7100 5300 7350 5300
 $Comp
-L INDUCTOR_Small FB?
+L INDUCTOR_Small FB13
 U 1 1 5B28F416
 P 5450 5300
-F 0 "FB?" V 5635 5300 50  0000 C CNN
+F 0 "FB13" V 5635 5300 50  0000 C CNN
 F 1 "MMZ1608A252BTA00" V 5544 5300 50  0000 C CNN
 F 2 "" H 5450 5300 50  0000 C CNN
@@
 	5550 5300 5800 5300
 $Comp
-L INDUCTOR_Small FB?
+L INDUCTOR_Small FB16
 U 1 1 5B292FBD
 P 10400 4800
-F 0 "FB?" V 10585 4800 50  0000 C CNN
+F 0 "FB16" V 10585 4800 50  0000 C CNN
 F 1 "MMZ1608A252BTA00" V 10494 4800 50  0000 C CNN
 F 2 "" H 10400 4800 50  0000 C CNN
@@
 $EndComp
 $Comp
-L INDUCTOR_Small FB?
+L INDUCTOR_Small FB17
 U 1 1 5B293036
 P 10400 6000
-F 0 "FB?" V 10585 6000 50  0000 C CNN
+F 0 "FB17" V 10585 6000 50  0000 C CNN
 F 1 "MMZ1608A252BTA00" V 10494 6000 50  0000 C CNN
 F 2 "" H 10400 6000 50  0000 C CNN
@@
 	10300 6000 10250 6000
 $Comp
-L R R?
+L R R69
 U 1 1 5B2944CE
 P 10900 4800
-F 0 "R?" V 11107 4800 50  0000 C CNN
+F 0 "R69" V 11107 4800 50  0000 C CNN
 F 1 "4.7kΩ" V 11016 4800 50  0000 C CNN
 F 2 "" V 10830 4800 50  0000 C CNN
@@
 $EndComp
 $Comp
-L R R?
+L R R70
 U 1 1 5B294BC6
 P 10900 6000
-F 0 "R?" V 11107 6000 50  0000 C CNN
+F 0 "R70" V 11107 6000 50  0000 C CNN
 F 1 "4.7kΩ" V 11016 6000 50  0000 C CNN
 F 2 "" V 10830 6000 50  0000 C CNN
@@
 	10750 4800 10500 4800
 $Comp
-L ZENER D?
+L ZENER D13
 U 1 1 5B4EDDEC
 P 8450 5550
-F 0 "D?" V 8404 5629 50  0000 L CNN
+F 0 "D13" V 8404 5629 50  0000 L CNN
 F 1 "ZENER" V 8495 5629 50  0000 L CNN
 F 2 "" H 8450 5550 50  0000 C CNN
@@
 Connection ~ 8450 5300
 $Comp
-L GND #PWR0139
+L GND #PWR0187
 U 1 1 5B4EDFC5
 P 8450 5800
-F 0 "#PWR0139" H 8450 5550 50  0001 C CNN
+F 0 "#PWR0187" H 8450 5550 50  0001 C CNN
 F 1 "GND" H 8455 5627 50  0000 C CNN
 F 2 "" H 8450 5800 50  0000 C CNN
@@
 	8450 5800 8450 5750
 $Comp
-L INDUCTOR_Small FB?
+L INDUCTOR_Small FB14
 U 1 1 5B9752EE
 P 7000 5300
-F 0 "FB?" V 7185 5300 50  0000 C CNN
+F 0 "FB14" V 7185 5300 50  0000 C CNN
 F 1 "MMZ1608A252BTA00" V 7094 5300 50  0000 C CNN
 F 2 "" H 7000 5300 50  0000 C CNN
@@
 $EndComp
 $Comp
-L INDUCTOR_Small FB?
+L INDUCTOR_Small FB15
 U 1 1 5B975719
 P 8600 5300
-F 0 "FB?" V 8785 5300 50  0000 C CNN
+F 0 "FB15" V 8785 5300 50  0000 C CNN
 F 1 "MMZ1608A252BTA00" V 8694 5300 50  0000 C CNN
 F 2 "" H 8600 5300 50  0000 C CNN

Commit message: Clean up various parts of the schematic, high level sheet has annoated modules
Parts:
- renumbered C36 to C74, C37 to C75, C38 to C76, C39 to C77, C40 to C78, D13 to D14, FB13 to FB26, FB14 to FB27, FB15 to FB28, FB16 to FB29, FB17 to FB30, R63 to R126, R64 to R127, R65 to R128, R66 to R129, R67 to R130, R68 to R131, R69 to R132, R70 to R133
Changed lines of the file:
@@
 $Descr A3 16535 11693
 encoding utf-8
-Sheet 10 26
+Sheet 14 26
 Title ""
 Date ""
@@
 X1
 $Comp
-L C C36
+L C C74
 U 1 1 58129032
 P 6150 5500
-F 0 "C36" H 6264 5546 50  0000 L CNN
+F 0 "C74" H 6264 5546 50  0000 L CNN
 F 1 "4.7μF" H 6264 5455 50  0000 L CNN
 F 2 "" H 6188 5350 50  0000 C CNN
@@
 $EndComp
 $Comp
-L R R64
+L R R127
 U 1 1 58129040
 P 6150 5100
-F 0 "R64" H 6081 5054 50  0000 R CNN
+F 0 "R127" H 6081 5054 50  0000 R CNN
 F 1 "4.7kΩ" H 6081 5145 50  0000 R CNN
 F 2 "" V 6080 5100 50  0000 C CNN
@@
 	6150 4950 6150 4900
 $Comp
-L R R63
+L R R126
 U 1 1 5812D30B
 P 5950 5300
-F 0 "R63" V 6157 5300 50  0000 C CNN
+F 0 "R126" V 6157 5300 50  0000 C CNN
 F 1 "4.7kΩ" V 6066 5300 50  0000 C CNN
 F 2 "" V 5880 5300 50  0000 C CNN
@@
 Y1
 $Comp
-L C C37
+L C C75
 U 1 1 589415E7
 P 7700 5500
-F 0 "C37" H 7814 5546 50  0000 L CNN
+F 0 "C75" H 7814 5546 50  0000 L CNN
 F 1 "4.7μF" H 7814 5455 50  0000 L CNN
 F 2 "" H 7738 5350 50  0000 C CNN
@@
 $EndComp
 $Comp
-L R R66
+L R R129
 U 1 1 589415EE
 P 7700 5100
-F 0 "R66" H 7631 5054 50  0000 R CNN
+F 0 "R129" H 7631 5054 50  0000 R CNN
 F 1 "4.7kΩ" H 7631 5145 50  0000 R CNN
 F 2 "" V 7630 5100 50  0000 C CNN
@@
 	7700 4950 7700 4900
 $Comp
-L R R65
+L R R128
 U 1 1 58941610
 P 7500 5300
-F 0 "R65" V 7707 5300 50  0000 C CNN
+F 0 "R128" V 7707 5300 50  0000 C CNN
 F 1 "4.7kΩ" V 7616 5300 50  0000 C CNN
 F 2 "" V 7430 5300 50  0000 C CNN
@@
 Z1
 $Comp
-L C C38
+L C C76
 U 1 1 58941879
 P 9300 5500
-F 0 "C38" H 9414 5546 50  0000 L CNN
+F 0 "C76" H 9414 5546 50  0000 L CNN
 F 1 "4.7μF" H 9414 5455 50  0000 L CNN
 F 2 "" H 9338 5350 50  0000 C CNN
@@
 $EndComp
 $Comp
-L R R68
+L R R131
 U 1 1 58941880
 P 9300 5100
-F 0 "R68" H 9231 5054 50  0000 R CNN
+F 0 "R131" H 9231 5054 50  0000 R CNN
 F 1 "4.7kΩ" H 9231 5145 50  0000 R CNN
 F 2 "" V 9230 5100 50  0000 C CNN
@@
 	9300 4950 9300 4900
 $Comp
-L R R67
+L R R130
 U 1 1 589418A2
 P 9100 5300
-F 0 "R67" V 9307 5300 50  0000 C CNN
+F 0 "R130" V 9307 5300 50  0000 C CNN
 F 1 "4.7kΩ" V 9216 5300 50  0000 C CNN
 F 2 "" V 9030 5300 50  0000 C CNN
@@
 ENC_A
 $Comp
-L C C39
+L C C77
 U 1 1 5894C248
 P 11100 5000
-F 0 "C39" H 11214 5046 50  0000 L CNN
+F 0 "C77" H 11214 5046 50  0000 L CNN
 F 1 "4.7μF" H 11214 4955 50  0000 L CNN
 F 2 "" H 11138 4850 50  0000 C CNN
@@
 	11100 6000 11100 6050
 $Comp
-L C C40
+L C C78
 U 1 1 5894C2A4
 P 11100 6200
-F 0 "C40" H 11214 6246 50  0000 L CNN
+F 0 "C78" H 11214 6246 50  0000 L CNN
 F 1 "4.7μF" H 11214 6155 50  0000 L CNN
 F 2 "" H 11138 6050 50  0000 C CNN
@@
 	7100 5300 7350 5300
 $Comp
-L INDUCTOR_Small FB13
+L INDUCTOR_Small FB26
 U 1 1 5B28F416
 P 5450 5300
-F 0 "FB13" V 5635 5300 50  0000 C CNN
+F 0 "FB26" V 5635 5300 50  0000 C CNN
 F 1 "MMZ1608A252BTA00" V 5544 5300 50  0000 C CNN
 F 2 "" H 5450 5300 50  0000 C CNN
@@
 	5550 5300 5800 5300
 $Comp
-L INDUCTOR_Small FB16
+L INDUCTOR_Small FB29
 U 1 1 5B292FBD
 P 10400 4800
-F 0 "FB16" V 10585 4800 50  0000 C CNN
+F 0 "FB29" V 10585 4800 50  0000 C CNN
 F 1 "MMZ1608A252BTA00" V 10494 4800 50  0000 C CNN
 F 2 "" H 10400 4800 50  0000 C CNN
@@
 $EndComp
 $Comp
-L INDUCTOR_Small FB17
+L INDUCTOR_Small FB30
 U 1 1 5B293036
 P 10400 6000
-F 0 "FB17" V 10585 6000 50  0000 C CNN
+F 0 "FB30" V 10585 6000 50  0000 C CNN
 F 1 "MMZ1608A252BTA00" V 10494 6000 50  0000 C CNN
 F 2 "" H 10400 6000 50  0000 C CNN
@@
 	10300 6000 10250 6000
 $Comp
-L R R69
+L R R132
 U 1 1 5B2944CE
 P 10900 4800
-F 0 "R69" V 11107 4800 50  0000 C CNN
+F 0 "R132" V 11107 4800 50  0000 C CNN
 F 1 "4.7kΩ" V 11016 4800 50  0000 C CNN
 F 2 "" V 10830 4800 50  0000 C CNN
@@
 $EndComp
 $Comp
-L R R70
+L R R133
 U 1 1 5B294BC6
 P 10900 6000
-F 0 "R70" V 11107 6000 50  0000 C CNN
+F 0 "R133" V 11107 6000 50  0000 C CNN
 F 1 "4.7kΩ" V 11016 6000 50  0000 C CNN
 F 2 "" V 10830 6000 50  0000 C CNN
@@
 	10750 4800 10500 4800
 $Comp
-L ZENER D13
+L ZENER D14
 U 1 1 5B4EDDEC
 P 8450 5550
-F 0 "D13" V 8404 5629 50  0000 L CNN
+F 0 "D14" V 8404 5629 50  0000 L CNN
 F 1 "ZENER" V 8495 5629 50  0000 L CNN
 F 2 "" H 8450 5550 50  0000 C CNN
@@
 	8450 5800 8450 5750
 $Comp
-L INDUCTOR_Small FB14
+L INDUCTOR_Small FB27
 U 1 1 5B9752EE
 P 7000 5300
-F 0 "FB14" V 7185 5300 50  0000 C CNN
+F 0 "FB27" V 7185 5300 50  0000 C CNN
 F 1 "MMZ1608A252BTA00" V 7094 5300 50  0000 C CNN
 F 2 "" H 7000 5300 50  0000 C CNN
@@
 $EndComp
 $Comp
-L INDUCTOR_Small FB15
+L INDUCTOR_Small FB28
 U 1 1 5B975719
 P 8600 5300
-F 0 "FB15" V 8785 5300 50  0000 C CNN
+F 0 "FB28" V 8785 5300 50  0000 C CNN
 F 1 "MMZ1608A252BTA00" V 8694 5300 50  0000 C CNN
 F 2 "" H 8600 5300 50  0000 C CNN

Commit message: Entry of additional component values
Parts:
- D15: renamed from D14; value ZENER -> TPD1E04U04DPYR
- renumbered FB26 to FB27, FB27 to FB28, FB28 to FB29, FB29 to FB30, FB30 to FB31, R126 to R125, R127 to R126, R128 to R127, R129 to R128, R130 to R129, R131 to R130, R132 to R131, R133 to R132
Changed lines of the file:
@@
 $EndComp
 $Comp
-L R R127
+L R R126
 U 1 1 58129040
 P 6150 5100
-F 0 "R127" H 6081 5054 50  0000 R CNN
+F 0 "R126" H 6081 5054 50  0000 R CNN
 F 1 "4.7kΩ" H 6081 5145 50  0000 R CNN
 F 2 "" V 6080 5100 50  0001 C CNN
@@
 	6150 4950 6150 4900
 $Comp
-L R R126
+L R R125
 U 1 1 5812D30B
 P 5950 5300
-F 0 "R126" V 6157 5300 50  0000 C CNN
+F 0 "R125" V 6157 5300 50  0000 C CNN
 F 1 "4.7kΩ" V 6066 5300 50  0000 C CNN
 F 2 "" V 5880 5300 50  0001 C CNN
@@
 $EndComp
 $Comp
-L R R129
+L R R128
 U 1 1 589415EE
 P 7700 5100
-F 0 "R129" H 7631 5054 50  0000 R CNN
+F 0 "R128" H 7631 5054 50  0000 R CNN
 F 1 "4.7kΩ" H 7631 5145 50  0000 R CNN
 F 2 "" V 7630 5100 50  0001 C CNN
@@
 	7700 4950 7700 4900
 $Comp
-L R R128
+L R R127
 U 1 1 58941610
 P 7500 5300
-F 0 "R128" V 7707 5300 50  0000 C CNN
+F 0 "R127" V 7707 5300 50  0000 C CNN
 F 1 "4.7kΩ" V 7616 5300 50  0000 C CNN
 F 2 "" V 7430 5300 50  0001 C CNN
@@
 $EndComp
 $Comp
-L R R131
+L R R130
 U 1 1 58941880
 P 9300 5100
-F 0 "R131" H 9231 5054 50  0000 R CNN
+F 0 "R130" H 9231 5054 50  0000 R CNN
 F 1 "4.7kΩ" H 9231 5145 50  0000 R CNN
 F 2 "" V 9230 5100 50  0001 C CNN
@@
 	9300 4950 9300 4900
 $Comp
-L R R130
+L R R129
 U 1 1 589418A2
 P 9100 5300
-F 0 "R130" V 9307 5300 50  0000 C CNN
+F 0 "R129" V 9307 5300 50  0000 C CNN
 F 1 "4.7kΩ" V 9216 5300 50  0000 C CNN
 F 2 "" V 9030 5300 50  0001 C CNN
@@
 ENC_B_IN
 $Comp
-L VDD_3V3B #PWR0179
+L VDD_3V3B #PWR0180
 U 1 1 59E67523
 P 6150 4900
-F 0 "#PWR0179" H 6150 4750 50  0001 C CNN
+F 0 "#PWR0180" H 6150 4750 50  0001 C CNN
 F 1 "VDD_3V3B" H 6165 5073 50  0000 C CNN
 F 2 "" H 6150 4900 50  0000 C CNN
@@
 $EndComp
 $Comp
-L VDD_3V3B #PWR0180
+L VDD_3V3B #PWR0181
 U 1 1 59E6755C
 P 7700 4900
-F 0 "#PWR0180" H 7700 4750 50  0001 C CNN
+F 0 "#PWR0181" H 7700 4750 50  0001 C CNN
 F 1 "VDD_3V3B" H 7715 5073 50  0000 C CNN
 F 2 "" H 7700 4900 50  0000 C CNN
@@
 $EndComp
 $Comp
-L VDD_3V3B #PWR0181
+L VDD_3V3B #PWR0182
 U 1 1 59E6758E
 P 9300 4900
-F 0 "#PWR0181" H 9300 4750 50  0001 C CNN
+F 0 "#PWR0182" H 9300 4750 50  0001 C CNN
 F 1 "VDD_3V3B" H 9315 5073 50  0000 C CNN
 F 2 "" H 9300 4900 50  0000 C CNN
@@
 	11050 6000 11150 6000
 $Comp
-L GND #PWR0182
+L GND #PWR0183
 U 1 1 59E68F88
 P 11100 5200
-F 0 "#PWR0182" H 11100 4950 50  0001 C CNN
+F 0 "#PWR0183" H 11100 4950 50  0001 C CNN
 F 1 "GND" H 11105 5027 50  0000 C CNN
 F 2 "" H 11100 5200 50  0000 C CNN
@@
 $EndComp
 $Comp
-L GND #PWR0183
+L GND #PWR0184
 U 1 1 59E68FBB
 P 11100 6400
-F 0 "#PWR0183" H 11100 6150 50  0001 C CNN
+F 0 "#PWR0184" H 11100 6150 50  0001 C CNN
 F 1 "GND" H 11105 6227 50  0000 C CNN
 F 2 "" H 11100 6400 50  0000 C CNN
@@
 $EndComp
 $Comp
-L GND #PWR0184
+L GND #PWR0185
 U 1 1 59E68FE7
 P 9300 5700
-F 0 "#PWR0184" H 9300 5450 50  0001 C CNN
+F 0 "#PWR0185" H 9300 5450 50  0001 C CNN
 F 1 "GND" H 9305 5527 50  0000 C CNN
 F 2 "" H 9300 5700 50  0000 C CNN
@@
 $EndComp
 $Comp
-L GND #PWR0185
+L GND #PWR0186
 U 1 1 59E69013
 P 7700 5700
-F 0 "#PWR0185" H 7700 5450 50  0001 C CNN
+F 0 "#PWR0186" H 7700 5450 50  0001 C CNN
 F 1 "GND" H 7705 5527 50  0000 C CNN
 F 2 "" H 7700 5700 50  0000 C CNN
@@
 $EndComp
 $Comp
-L GND #PWR0186
+L GND #PWR0187
 U 1 1 59E6903F
 P 6150 5700
-F 0 "#PWR0186" H 6150 5450 50  0001 C CNN
+F 0 "#PWR0187" H 6150 5450 50  0001 C CNN
 F 1 "GND" H 6155 5527 50  0000 C CNN
 F 2 "" H 6150 5700 50  0000 C CNN
@@
 	7100 5300 7350 5300
 $Comp
-L INDUCTOR_Small FB26
+L INDUCTOR_Small FB27
 U 1 1 5B28F416
 P 5450 5300
-F 0 "FB26" V 5635 5300 50  0000 C CNN
+F 0 "FB27" V 5635 5300 50  0000 C CNN
 F 1 "MMZ1608A252BTA00" V 5544 5300 50  0000 C CNN
 F 2 "" H 5450 5300 50  0001 C CNN
@@
 	5550 5300 5800 5300
 $Comp
-L INDUCTOR_Small FB29
+L INDUCTOR_Small FB30
 U 1 1 5B292FBD
 P 10400 4800
-F 0 "FB29" V 10585 4800 50  0000 C CNN
+F 0 "FB30" V 10585 4800 50  0000 C CNN
 F 1 "MMZ1608A252BTA00" V 10494 4800 50  0000 C CNN
 F 2 "" H 10400 4800 50  0001 C CNN
@@
 $EndComp
 $Comp
-L INDUCTOR_Small FB30
+L INDUCTOR_Small FB31
 U 1 1 5B293036
 P 10400 6000
-F 0 "FB30" V 10585 6000 50  0000 C CNN
+F 0 "FB31" V 10585 6000 50  0000 C CNN
 F 1 "MMZ1608A252BTA00" V 10494 6000 50  0000 C CNN
 F 2 "" H 10400 6000 50  0001 C CNN
@@
 	10300 6000 10250 6000
 $Comp
-L R R132
+L R R131
 U 1 1 5B2944CE
 P 10900 4800
-F 0 "R132" V 11107 4800 50  0000 C CNN
+F 0 "R131" V 11107 4800 50  0000 C CNN
 F 1 "4.7kΩ" V 11016 4800 50  0000 C CNN
 F 2 "" V 10830 4800 50  0001 C CNN
@@
 $EndComp
 $Comp
-L R R133
+L R R132
 U 1 1 5B294BC6
 P 10900 6000
-F 0 "R133" V 11107 6000 50  0000 C CNN
+F 0 "R132" V 11107 6000 50  0000 C CNN
 F 1 "4.7kΩ" V 11016 6000 50  0000 C CNN
 F 2 "" V 10830 6000 50  0001 C CNN
@@
 	10750 4800 10500 4800
 $Comp
-L ZENER D14
+L ZENER D15
 U 1 1 5B4EDDEC
 P 8450 5550
-F 0 "D14" V 8404 5629 50  0000 L CNN
-F 1 "ZENER" V 8495 5629 50  0000 L CNN
+F 0 "D15" V 8404 5629 50  0000 L CNN
+F 1 "TPD1E04U04DPYR" V 8495 5629 50  0000 L CNN
 F 2 "" H 8450 5550 50  0001 C CNN
 F 3 "" H 8450 5550 50  0000 C CNN
@@
 Connection ~ 8450 5300
 $Comp
-L GND #PWR0187
+L GND #PWR0188
 U 1 1 5B4EDFC5
 P 8450 5800
-F 0 "#PWR0187" H 8450 5550 50  0001 C CNN
+F 0 "#PWR0188" H 8450 5550 50  0001 C CNN
 F 1 "GND" H 8455 5627 50  0000 C CNN
 F 2 "" H 8450 5800 50  0000 C CNN
@@
 	8450 5800 8450 5750
 $Comp
-L INDUCTOR_Small FB27
+L INDUCTOR_Small FB28
 U 1 1 5B9752EE
 P 7000 5300
-F 0 "FB27" V 7185 5300 50  0000 C CNN
+F 0 "FB28" V 7185 5300 50  0000 C CNN
 F 1 "MMZ1608A252BTA00" V 7094 5300 50  0000 C CNN
 F 2 "" H 7000 5300 50  0001 C CNN
@@
 $EndComp
 $Comp
-L INDUCTOR_Small FB28
+L INDUCTOR_Small FB29
 U 1 1 5B975719
 P 8600 5300
-F 0 "FB28" V 8785 5300 50  0000 C CNN
+F 0 "FB29" V 8785 5300 50  0000 C CNN
 F 1 "MMZ1608A252BTA00" V 8694 5300 50  0000 C CNN
 F 2 "" H 8600 5300 50  0001 C CNN
