File: KiMBo/endstop.sch (KiCad schematic (older format))
At the start: 19 parts

Commit message: Add equivalent annotations document, associate more footprints
Parts:
- C74, C75, C76, C77, C78: footprint (none) -> Capacitors_SMD:C_0402
- renumbered R125 to R124, R126 to R125, R127 to R126, R128 to R127, R129 to R128, R130 to R129, R131 to R130, R132 to R131
Changed lines of the file:
@@
 F 0 "C74" H 6264 5546 50  0000 L CNN
 F 1 "4.7μF" H 6264 5455 50  0000 L CNN
-F 2 "" H 6188 5350 50  0001 C CNN
+F 2 "Capacitors_SMD:C_0402" H 6188 5350 50  0001 C CNN
 F 3 "" H 6150 5500 50  0000 C CNN
 	1    6150 5500
@@
 $EndComp
 $Comp
-L R R126
+L R R125
 U 1 1 58129040
 P 6150 5100
-F 0 "R126" H 6081 5054 50  0000 R CNN
+F 0 "R125" H 6081 5054 50  0000 R CNN
 F 1 "4.7kΩ" H 6081 5145 50  0000 R CNN
 F 2 "" V 6080 5100 50  0001 C CNN
@@
 	6150 4950 6150 4900
 $Comp
-L R R125
+L R R124
 U 1 1 5812D30B
 P 5950 5300
-F 0 "R125" V 6157 5300 50  0000 C CNN
+F 0 "R124" V 6157 5300 50  0000 C CNN
 F 1 "4.7kΩ" V 6066 5300 50  0000 C CNN
 F 2 "" V 5880 5300 50  0001 C CNN
@@
 F 0 "C75" H 7814 5546 50  0000 L CNN
 F 1 "4.7μF" H 7814 5455 50  0000 L CNN
-F 2 "" H 7738 5350 50  0001 C CNN
+F 2 "Capacitors_SMD:C_0402" H 7738 5350 50  0001 C CNN
 F 3 "" H 7700 5500 50  0000 C CNN
 	1    7700 5500
@@
 $EndComp
 $Comp
-L R R128
+L R R127
 U 1 1 589415EE
 P 7700 5100
-F 0 "R128" H 7631 5054 50  0000 R CNN
+F 0 "R127" H 7631 5054 50  0000 R CNN
 F 1 "4.7kΩ" H 7631 5145 50  0000 R CNN
 F 2 "" V 7630 5100 50  0001 C CNN
@@
 	7700 4950 7700 4900
 $Comp
-L R R127
+L R R126
 U 1 1 58941610
 P 7500 5300
-F 0 "R127" V 7707 5300 50  0000 C CNN
+F 0 "R126" V 7707 5300 50  0000 C CNN
 F 1 "4.7kΩ" V 7616 5300 50  0000 C CNN
 F 2 "" V 7430 5300 50  0001 C CNN
@@
 F 0 "C76" H 9414 5546 50  0000 L CNN
 F 1 "4.7μF" H 9414 5455 50  0000 L CNN
-F 2 "" H 9338 5350 50  0001 C CNN
+F 2 "Capacitors_SMD:C_0402" H 9338 5350 50  0001 C CNN
 F 3 "" H 9300 5500 50  0000 C CNN
 	1    9300 5500
@@
 $EndComp
 $Comp
-L R R130
+L R R129
 U 1 1 58941880
 P 9300 5100
-F 0 "R130" H 9231 5054 50  0000 R CNN
+F 0 "R129" H 9231 5054 50  0000 R CNN
 F 1 "4.7kΩ" H 9231 5145 50  0000 R CNN
 F 2 "" V 9230 5100 50  0001 C CNN
@@
 	9300 4950 9300 4900
 $Comp
-L R R129
+L R R128
 U 1 1 589418A2
 P 9100 5300
-F 0 "R129" V 9307 5300 50  0000 C CNN
+F 0 "R128" V 9307 5300 50  0000 C CNN
 F 1 "4.7kΩ" V 9216 5300 50  0000 C CNN
 F 2 "" V 9030 5300 50  0001 C CNN
@@
 F 0 "C77" H 11214 5046 50  0000 L CNN
 F 1 "4.7μF" H 11214 4955 50  0000 L CNN
-F 2 "" H 11138 4850 50  0001 C CNN
+F 2 "Capacitors_SMD:C_0402" H 11138 4850 50  0001 C CNN
 F 3 "" H 11100 5000 50  0000 C CNN
 	1    11100 5000
@@
 F 0 "C78" H 11214 6246 50  0000 L CNN
 F 1 "4.7μF" H 11214 6155 50  0000 L CNN
-F 2 "" H 11138 6050 50  0001 C CNN
+F 2 "Capacitors_SMD:C_0402" H 11138 6050 50  0001 C CNN
 F 3 "" H 11100 6200 50  0000 C CNN
 	1    11100 6200
@@
 ENC_B_IN
 $Comp
-L VDD_3V3B #PWR0180
+L VDD_3V3B #PWR0179
 U 1 1 59E67523
 P 6150 4900
-F 0 "#PWR0180" H 6150 4750 50  0001 C CNN
+F 0 "#PWR0179" H 6150 4750 50  0001 C CNN
 F 1 "VDD_3V3B" H 6165 5073 50  0000 C CNN
 F 2 "" H 6150 4900 50  0000 C CNN
@@
 $EndComp
 $Comp
-L VDD_3V3B #PWR0181
+L VDD_3V3B #PWR0180
 U 1 1 59E6755C
 P 7700 4900
-F 0 "#PWR0181" H 7700 4750 50  0001 C CNN
+F 0 "#PWR0180" H 7700 4750 50  0001 C CNN
 F 1 "VDD_3V3B" H 7715 5073 50  0000 C CNN
 F 2 "" H 7700 4900 50  0000 C CNN
@@
 $EndComp
 $Comp
-L VDD_3V3B #PWR0182
+L VDD_3V3B #PWR0181
 U 1 1 59E6758E
 P 9300 4900
-F 0 "#PWR0182" H 9300 4750 50  0001 C CNN
+F 0 "#PWR0181" H 9300 4750 50  0001 C CNN
 F 1 "VDD_3V3B" H 9315 5073 50  0000 C CNN
 F 2 "" H 9300 4900 50  0000 C CNN
@@
 	11050 6000 11150 6000
 $Comp
-L GND #PWR0183
+L GND #PWR0182
 U 1 1 59E68F88
 P 11100 5200
-F 0 "#PWR0183" H 11100 4950 50  0001 C CNN
+F 0 "#PWR0182" H 11100 4950 50  0001 C CNN
 F 1 "GND" H 11105 5027 50  0000 C CNN
 F 2 "" H 11100 5200 50  0000 C CNN
@@
 $EndComp
 $Comp
-L GND #PWR0184
+L GND #PWR0183
 U 1 1 59E68FBB
 P 11100 6400
-F 0 "#PWR0184" H 11100 6150 50  0001 C CNN
+F 0 "#PWR0183" H 11100 6150 50  0001 C CNN
 F 1 "GND" H 11105 6227 50  0000 C CNN
 F 2 "" H 11100 6400 50  0000 C CNN
@@
 $EndComp
 $Comp
-L GND #PWR0185
+L GND #PWR0184
 U 1 1 59E68FE7
 P 9300 5700
-F 0 "#PWR0185" H 9300 5450 50  0001 C CNN
+F 0 "#PWR0184" H 9300 5450 50  0001 C CNN
 F 1 "GND" H 9305 5527 50  0000 C CNN
 F 2 "" H 9300 5700 50  0000 C CNN
@@
 $EndComp
 $Comp
-L GND #PWR0186
+L GND #PWR0185
 U 1 1 59E69013
 P 7700 5700
-F 0 "#PWR0186" H 7700 5450 50  0001 C CNN
+F 0 "#PWR0185" H 7700 5450 50  0001 C CNN
 F 1 "GND" H 7705 5527 50  0000 C CNN
 F 2 "" H 7700 5700 50  0000 C CNN
@@
 $EndComp
 $Comp
-L GND #PWR0187
+L GND #PWR0186
 U 1 1 59E6903F
 P 6150 5700
-F 0 "#PWR0187" H 6150 5450 50  0001 C CNN
+F 0 "#PWR0186" H 6150 5450 50  0001 C CNN
 F 1 "GND" H 6155 5527 50  0000 C CNN
 F 2 "" H 6150 5700 50  0000 C CNN
@@
 	10300 6000 10250 6000
 $Comp
-L R R131
+L R R130
 U 1 1 5B2944CE
 P 10900 4800
-F 0 "R131" V 11107 4800 50  0000 C CNN
+F 0 "R130" V 11107 4800 50  0000 C CNN
 F 1 "4.7kΩ" V 11016 4800 50  0000 C CNN
 F 2 "" V 10830 4800 50  0001 C CNN
@@
 $EndComp
 $Comp
-L R R132
+L R R131
 U 1 1 5B294BC6
 P 10900 6000
-F 0 "R132" V 11107 6000 50  0000 C CNN
+F 0 "R131" V 11107 6000 50  0000 C CNN
 F 1 "4.7kΩ" V 11016 6000 50  0000 C CNN
 F 2 "" V 10830 6000 50  0001 C CNN
@@
 Connection ~ 8450 5300
 $Comp
-L GND #PWR0188
+L GND #PWR0187
 U 1 1 5B4EDFC5
 P 8450 5800
-F 0 "#PWR0188" H 8450 5550 50  0001 C CNN
+F 0 "#PWR0187" H 8450 5550 50  0001 C CNN
 F 1 "GND" H 8455 5627 50  0000 C CNN
 F 2 "" H 8450 5800 50  0000 C CNN

Commit message: Change the endstop RC filter
Lower the time constant

Reduce the series resistor to 100Ohms
Parts:
- C74, C75, C76, C77, C78: value 4.7μF -> 0.1μF
- R124, R126, R128: value 4.7kΩ -> 100Ω
Other:
- note added: "RC_rise=10μs"
- note added: "RC_rise=470μs"
- note removed: "RC=22.09ms"
Changed lines of the file:
@@
 P 6150 5500
 F 0 "C74" H 6264 5546 50  0000 L CNN
-F 1 "4.7μF" H 6264 5455 50  0000 L CNN
+F 1 "0.1μF" H 6264 5455 50  0000 L CNN
 F 2 "Capacitors_SMD:C_0402" H 6188 5350 50  0001 C CNN
 F 3 "" H 6150 5500 50  0000 C CNN
@@
 P 5950 5300
 F 0 "R124" V 6157 5300 50  0000 C CNN
-F 1 "4.7kΩ" V 6066 5300 50  0000 C CNN
+F 1 "100Ω" V 6066 5300 50  0000 C CNN
 F 2 "" V 5880 5300 50  0001 C CNN
 F 3 "" H 5950 5300 50  0000 C CNN
@@
 P 7700 5500
 F 0 "C75" H 7814 5546 50  0000 L CNN
-F 1 "4.7μF" H 7814 5455 50  0000 L CNN
+F 1 "0.1μF" H 7814 5455 50  0000 L CNN
 F 2 "Capacitors_SMD:C_0402" H 7738 5350 50  0001 C CNN
 F 3 "" H 7700 5500 50  0000 C CNN
@@
 P 7500 5300
 F 0 "R126" V 7707 5300 50  0000 C CNN
-F 1 "4.7kΩ" V 7616 5300 50  0000 C CNN
+F 1 "100Ω" V 7616 5300 50  0000 C CNN
 F 2 "" V 7430 5300 50  0001 C CNN
 F 3 "" H 7500 5300 50  0000 C CNN
@@
 P 9300 5500
 F 0 "C76" H 9414 5546 50  0000 L CNN
-F 1 "4.7μF" H 9414 5455 50  0000 L CNN
+F 1 "0.1μF" H 9414 5455 50  0000 L CNN
 F 2 "Capacitors_SMD:C_0402" H 9338 5350 50  0001 C CNN
 F 3 "" H 9300 5500 50  0000 C CNN
@@
 P 9100 5300
 F 0 "R128" V 9307 5300 50  0000 C CNN
-F 1 "4.7kΩ" V 9216 5300 50  0000 C CNN
+F 1 "100Ω" V 9216 5300 50  0000 C CNN
 F 2 "" V 9030 5300 50  0001 C CNN
 F 3 "" H 9100 5300 50  0000 C CNN
@@
 P 11100 5000
 F 0 "C77" H 11214 5046 50  0000 L CNN
-F 1 "4.7μF" H 11214 4955 50  0000 L CNN
+F 1 "0.1μF" H 11214 4955 50  0000 L CNN
 F 2 "Capacitors_SMD:C_0402" H 11138 4850 50  0001 C CNN
 F 3 "" H 11100 5000 50  0000 C CNN
@@
 P 11100 6200
 F 0 "C78" H 11214 6246 50  0000 L CNN
-F 1 "4.7μF" H 11214 6155 50  0000 L CNN
+F 1 "0.1μF" H 11214 6155 50  0000 L CNN
 F 2 "Capacitors_SMD:C_0402" H 11138 6050 50  0001 C CNN
 F 3 "" H 11100 6200 50  0000 C CNN
@@
 $EndComp
 Text Notes 7950 4600 0    60   ~ 0
-RC=22.09ms
+RC_rise=470μs
 Wire Wire Line
 	8400 5300 8500 5300
@@
 	0    -1   -1   0
 $EndComp
+Text Notes 7950 4700 0    60   ~ 0
+RC_rise=10μs
 $EndSCHEMATC

Commit message: Leave SPI0 free for a display, reassign pins so SPI1 is available
Fix some typos/errors
Parts:
- renumbered R124 to R126, R125 to R127, R126 to R128, R127 to R129, R128 to R130, R129 to R131, R130 to R132, R131 to R133
Changed lines of the file:
@@
 $EndComp
 $Comp
-L R R125
+L R R127
 U 1 1 58129040
 P 6150 5100
-F 0 "R125" H 6081 5054 50  0000 R CNN
+F 0 "R127" H 6081 5054 50  0000 R CNN
 F 1 "4.7kΩ" H 6081 5145 50  0000 R CNN
 F 2 "" V 6080 5100 50  0001 C CNN
@@
 	6150 4950 6150 4900
 $Comp
-L R R124
+L R R126
 U 1 1 5812D30B
 P 5950 5300
-F 0 "R124" V 6157 5300 50  0000 C CNN
+F 0 "R126" V 6157 5300 50  0000 C CNN
 F 1 "100Ω" V 6066 5300 50  0000 C CNN
 F 2 "" V 5880 5300 50  0001 C CNN
@@
 $EndComp
 $Comp
-L R R127
+L R R129
 U 1 1 589415EE
 P 7700 5100
-F 0 "R127" H 7631 5054 50  0000 R CNN
+F 0 "R129" H 7631 5054 50  0000 R CNN
 F 1 "4.7kΩ" H 7631 5145 50  0000 R CNN
 F 2 "" V 7630 5100 50  0001 C CNN
@@
 	7700 4950 7700 4900
 $Comp
-L R R126
+L R R128
 U 1 1 58941610
 P 7500 5300
-F 0 "R126" V 7707 5300 50  0000 C CNN
+F 0 "R128" V 7707 5300 50  0000 C CNN
 F 1 "100Ω" V 7616 5300 50  0000 C CNN
 F 2 "" V 7430 5300 50  0001 C CNN
@@
 $EndComp
 $Comp
-L R R129
+L R R131
 U 1 1 58941880
 P 9300 5100
-F 0 "R129" H 9231 5054 50  0000 R CNN
+F 0 "R131" H 9231 5054 50  0000 R CNN
 F 1 "4.7kΩ" H 9231 5145 50  0000 R CNN
 F 2 "" V 9230 5100 50  0001 C CNN
@@
 	9300 4950 9300 4900
 $Comp
-L R R128
+L R R130
 U 1 1 589418A2
 P 9100 5300
-F 0 "R128" V 9307 5300 50  0000 C CNN
+F 0 "R130" V 9307 5300 50  0000 C CNN
 F 1 "100Ω" V 9216 5300 50  0000 C CNN
 F 2 "" V 9030 5300 50  0001 C CNN
@@
 ENC_B_IN
 $Comp
-L VDD_3V3B #PWR0179
+L VDD_3V3B #PWR0178
 U 1 1 59E67523
 P 6150 4900
-F 0 "#PWR0179" H 6150 4750 50  0001 C CNN
+F 0 "#PWR0178" H 6150 4750 50  0001 C CNN
 F 1 "VDD_3V3B" H 6165 5073 50  0000 C CNN
 F 2 "" H 6150 4900 50  0000 C CNN
@@
 $EndComp
 $Comp
-L VDD_3V3B #PWR0180
+L VDD_3V3B #PWR0179
 U 1 1 59E6755C
 P 7700 4900
-F 0 "#PWR0180" H 7700 4750 50  0001 C CNN
+F 0 "#PWR0179" H 7700 4750 50  0001 C CNN
 F 1 "VDD_3V3B" H 7715 5073 50  0000 C CNN
 F 2 "" H 7700 4900 50  0000 C CNN
@@
 $EndComp
 $Comp
-L VDD_3V3B #PWR0181
+L VDD_3V3B #PWR0180
 U 1 1 59E6758E
 P 9300 4900
-F 0 "#PWR0181" H 9300 4750 50  0001 C CNN
+F 0 "#PWR0180" H 9300 4750 50  0001 C CNN
 F 1 "VDD_3V3B" H 9315 5073 50  0000 C CNN
 F 2 "" H 9300 4900 50  0000 C CNN
@@
 	11050 6000 11150 6000
 $Comp
-L GND #PWR0182
+L GND #PWR0181
 U 1 1 59E68F88
 P 11100 5200
-F 0 "#PWR0182" H 11100 4950 50  0001 C CNN
+F 0 "#PWR0181" H 11100 4950 50  0001 C CNN
 F 1 "GND" H 11105 5027 50  0000 C CNN
 F 2 "" H 11100 5200 50  0000 C CNN
@@
 $EndComp
 $Comp
-L GND #PWR0183
+L GND #PWR0182
 U 1 1 59E68FBB
 P 11100 6400
-F 0 "#PWR0183" H 11100 6150 50  0001 C CNN
+F 0 "#PWR0182" H 11100 6150 50  0001 C CNN
 F 1 "GND" H 11105 6227 50  0000 C CNN
 F 2 "" H 11100 6400 50  0000 C CNN
@@
 $EndComp
 $Comp
-L GND #PWR0184
+L GND #PWR0183
 U 1 1 59E68FE7
 P 9300 5700
-F 0 "#PWR0184" H 9300 5450 50  0001 C CNN
+F 0 "#PWR0183" H 9300 5450 50  0001 C CNN
 F 1 "GND" H 9305 5527 50  0000 C CNN
 F 2 "" H 9300 5700 50  0000 C CNN
@@
 $EndComp
 $Comp
-L GND #PWR0185
+L GND #PWR0184
 U 1 1 59E69013
 P 7700 5700
-F 0 "#PWR0185" H 7700 5450 50  0001 C CNN
+F 0 "#PWR0184" H 7700 5450 50  0001 C CNN
 F 1 "GND" H 7705 5527 50  0000 C CNN
 F 2 "" H 7700 5700 50  0000 C CNN
@@
 $EndComp
 $Comp
-L GND #PWR0186
+L GND #PWR0185
 U 1 1 59E6903F
 P 6150 5700
-F 0 "#PWR0186" H 6150 5450 50  0001 C CNN
+F 0 "#PWR0185" H 6150 5450 50  0001 C CNN
 F 1 "GND" H 6155 5527 50  0000 C CNN
 F 2 "" H 6150 5700 50  0000 C CNN
@@
 	10300 6000 10250 6000
 $Comp
-L R R130
+L R R132
 U 1 1 5B2944CE
 P 10900 4800
-F 0 "R130" V 11107 4800 50  0000 C CNN
+F 0 "R132" V 11107 4800 50  0000 C CNN
 F 1 "4.7kΩ" V 11016 4800 50  0000 C CNN
 F 2 "" V 10830 4800 50  0001 C CNN
@@
 $EndComp
 $Comp
-L R R131
+L R R133
 U 1 1 5B294BC6
 P 10900 6000
-F 0 "R131" V 11107 6000 50  0000 C CNN
+F 0 "R133" V 11107 6000 50  0000 C CNN
 F 1 "4.7kΩ" V 11016 6000 50  0000 C CNN
 F 2 "" V 10830 6000 50  0001 C CNN
@@
 Connection ~ 8450 5300
 $Comp
-L GND #PWR0187
+L GND #PWR0186
 U 1 1 5B4EDFC5
 P 8450 5800
-F 0 "#PWR0187" H 8450 5550 50  0001 C CNN
+F 0 "#PWR0186" H 8450 5550 50  0001 C CNN
 F 1 "GND" H 8455 5627 50  0000 C CNN
 F 2 "" H 8450 5800 50  0000 C CNN
