File: KiMBo/z2_stepper.sch (KiCad schematic (older format))
At the start: 25 parts

Commit message: Annotate all components, now passing ERC, added ferrites to the rest of the connectors
Parts:
- gave numbers to parts that had none: 25

Commit message: Reorder the SS and EN lines from the shift registers such that the previously enabled/disabled motors stay enabled/disabled whilst writting to the shift register
Change 10k resistors to 4.7k, flip the open-drain inverter connected to B15 (PMTC_PGOOD)

Update the links in the README

Update the PDF schematic
Parts:
- R165, R166, R167: value 10kΩ -> 4.7kΩ
Changed lines of the file:
@@
 F 0 "C151" H 7086 3154 50  0000 R CNN
 F 1 "100nF" H 7086 3245 50  0000 R CNN
-F 2 "" H 7238 3050 50  0000 C CNN
+F 2 "" H 7238 3050 50  0001 C CNN
 F 3 "" H 7200 3200 50  0000 C CNN
 	1    7200 3200
@@
 F 0 "C156" V 8950 3650 50  0000 C CNN
 F 1 "100nF" V 8950 3925 50  0000 C CNN
-F 2 "" H 9038 3600 50  0000 C CNN
+F 2 "" H 9038 3600 50  0001 C CNN
 F 3 "" H 9000 3750 50  0000 C CNN
 	1    9000 3750
@@
 F 0 "C163" H 10400 3300 50  0000 C CNN
 F 1 "100μF" H 10500 3100 50  0000 C CNN
-F 2 "" H 10350 3200 50  0000 C CNN
+F 2 "" H 10350 3200 50  0001 C CNN
 F 3 "" H 10350 3200 50  0000 C CNN
 	1    10350 3200
@@
 F 0 "C159" H 9400 3300 50  0000 C CNN
 F 1 "100nF" H 9325 3100 50  0000 C CNN
-F 2 "" H 9488 3050 50  0000 C CNN
+F 2 "" H 9488 3050 50  0001 C CNN
 F 3 "" H 9450 3200 50  0000 C CNN
 	1    9450 3200
@@
 F 0 "C160" H 9700 3300 50  0000 C CNN
 F 1 "100nF" H 9625 3100 50  0000 C CNN
-F 2 "" H 9788 3050 50  0000 C CNN
+F 2 "" H 9788 3050 50  0001 C CNN
 F 3 "" H 9750 3200 50  0000 C CNN
 	1    9750 3200
@@
 F 0 "C153" H 8965 4296 50  0000 L CNN
 F 1 "22nF" H 8965 4205 50  0000 L CNN
-F 2 "" H 8888 4100 50  0000 C CNN
+F 2 "" H 8888 4100 50  0001 C CNN
 F 3 "" H 8850 4250 50  0000 C CNN
 	1    8850 4250
@@
 F 0 "R172" H 10400 6750 50  0000 R CNN
 F 1 "220mΩ" H 10400 6850 50  0000 R CNN
-F 2 "" V 10380 6800 50  0000 C CNN
+F 2 "" V 10380 6800 50  0001 C CNN
 F 3 "" H 10450 6800 50  0000 C CNN
 	1    10450 6800
@@
 F 0 "R171" H 9600 6750 50  0000 R CNN
 F 1 "220mΩ" H 9600 6850 50  0000 R CNN
-F 2 "" V 9580 6800 50  0000 C CNN
+F 2 "" V 9580 6800 50  0001 C CNN
 F 3 "" H 9650 6800 50  0000 C CNN
 	1    9650 6800
@@
 F 0 "R168" V 6900 3850 50  0000 C CNN
 F 1 "2.2Ω" V 7000 3850 50  0000 C CNN
-F 2 "" V 6930 3850 50  0000 C CNN
+F 2 "" V 6930 3850 50  0001 C CNN
 F 3 "" H 7000 3850 50  0000 C CNN
 	1    7000 3850
@@
 F 0 "C150" H 6850 4150 50  0000 L CNN
 F 1 "470nF" H 6825 3950 50  0000 L CNN
-F 2 "" H 6838 3900 50  0000 C CNN
+F 2 "" H 6838 3900 50  0001 C CNN
 F 3 "" H 6800 4050 50  0000 C CNN
 	1    6800 4050
@@
 F 0 "C161" H 9850 6900 50  0000 L CNN
 F 1 "100nF" H 9850 6700 50  0000 L CNN
-F 2 "" H 9838 6650 50  0000 C CNN
+F 2 "" H 9838 6650 50  0001 C CNN
 F 3 "" H 9800 6800 50  0000 C CNN
 	1    9800 6800
@@
 P 5750 4350
 F 0 "R166" H 5819 4396 50  0000 L CNN
-F 1 "10kΩ" H 5819 4305 50  0000 L CNN
-F 2 "" V 5680 4350 50  0000 C CNN
+F 1 "4.7kΩ" H 5819 4305 50  0000 L CNN
+F 2 "" V 5680 4350 50  0001 C CNN
 F 3 "" H 5750 4350 50  0000 C CNN
 	1    5750 4350
@@
 F 0 "C152" H 7250 4150 50  0000 L CNN
 F 1 "4.7μF" H 7250 3950 50  0000 L CNN
-F 2 "" H 7238 3900 50  0000 C CNN
+F 2 "" H 7238 3900 50  0001 C CNN
 F 3 "" H 7200 4050 50  0000 C CNN
 	1    7200 4050
@@
 F 0 "R169" H 9019 6846 50  0000 L CNN
 F 1 "5.23kΩ" H 9019 6755 50  0000 L CNN
-F 2 "" V 8880 6800 50  0000 C CNN
+F 2 "" V 8880 6800 50  0001 C CNN
 F 3 "" H 8950 6800 50  0000 C CNN
 	1    8950 6800
@@
 F 0 "R170" V 8950 7000 50  0000 C CNN
 F 1 "4.75kΩ" V 9050 7000 50  0000 C CNN
-F 2 "" V 9080 7000 50  0000 C CNN
+F 2 "" V 9080 7000 50  0001 C CNN
 F 3 "" H 9150 7000 50  0000 C CNN
 	1    9150 7000
@@
 P 6100 4350
 F 0 "R167" H 6169 4396 50  0000 L CNN
-F 1 "10kΩ" H 6169 4305 50  0000 L CNN
-F 2 "" V 6030 4350 50  0000 C CNN
+F 1 "4.7kΩ" H 6169 4305 50  0000 L CNN
+F 2 "" V 6030 4350 50  0001 C CNN
 F 3 "" H 6100 4350 50  0000 C CNN
 	1    6100 4350
@@
 F 0 "C164" H 10650 6900 50  0000 L CNN
 F 1 "100nF" H 10650 6700 50  0000 L CNN
-F 2 "" H 10638 6650 50  0000 C CNN
+F 2 "" H 10638 6650 50  0001 C CNN
 F 3 "" H 10600 6800 50  0000 C CNN
 	1    10600 6800
@@
 F 0 "C154" H 8875 5150 50  0000 L CNN
 F 1 "470pF" H 8850 4950 50  0000 L CNN
-F 2 "" H 8888 4900 50  0000 C CNN
+F 2 "" H 8888 4900 50  0001 C CNN
 F 3 "" H 8850 5050 50  0000 C CNN
 	1    8850 5050
@@
 F 0 "C157" H 9075 5150 50  0000 L CNN
 F 1 "470pF" H 9075 4950 50  0000 L CNN
-F 2 "" H 9088 4900 50  0000 C CNN
+F 2 "" H 9088 4900 50  0001 C CNN
 F 3 "" H 9050 5050 50  0000 C CNN
 	1    9050 5050
@@
 F 0 "C155" H 8875 6000 50  0000 L CNN
 F 1 "470pF" H 8850 5800 50  0000 L CNN
-F 2 "" H 8888 5750 50  0000 C CNN
+F 2 "" H 8888 5750 50  0001 C CNN
 F 3 "" H 8850 5900 50  0000 C CNN
 	1    8850 5900
@@
 F 0 "C158" H 9075 6000 50  0000 L CNN
 F 1 "470pF" H 9075 5800 50  0000 L CNN
-F 2 "" H 9088 5750 50  0000 C CNN
+F 2 "" H 9088 5750 50  0001 C CNN
 F 3 "" H 9050 5900 50  0000 C CNN
 	1    9050 5900
@@
 F 0 "U25" H 7650 6300 60  0000 C CNN
 F 1 "TMC2130" H 8400 6300 60  0000 C CNN
-F 2 "" H 8100 5100 60  0000 C CNN
+F 2 "" H 8100 5100 60  0001 C CNN
 F 3 "" H 8100 5100 60  0000 C CNN
 	1    8100 4800
@@
 P 5400 4350
 F 0 "R165" H 5469 4396 50  0000 L CNN
-F 1 "10kΩ" H 5469 4305 50  0000 L CNN
-F 2 "" V 5330 4350 50  0000 C CNN
+F 1 "4.7kΩ" H 5469 4305 50  0000 L CNN
+F 2 "" V 5330 4350 50  0001 C CNN
 F 3 "" H 5400 4350 50  0000 C CNN
 	1    5400 4350
@@
 F 0 "C162" H 10000 3300 50  0000 C CNN
 F 1 "4.7μF" H 9925 3100 50  0000 C CNN
-F 2 "" H 10088 3050 50  0000 C CNN
+F 2 "" H 10088 3050 50  0001 C CNN
 F 3 "" H 10050 3200 50  0000 C CNN
 	1    10050 3200
@@
 F 0 "C149" H 6500 4150 50  0000 L CNN
 F 1 "100nF" H 6475 3950 50  0000 L CNN
-F 2 "" H 6488 3900 50  0000 C CNN
+F 2 "" H 6488 3900 50  0001 C CNN
 F 3 "" H 6450 4050 50  0000 C CNN
 	1    6450 4050

Commit message: Entry of additional component values
Parts:
- renumbered R165 to R164, R166 to R165, R167 to R166, R168 to R167, R169 to R168, R170 to R169, R171 to R170, R172 to R171
Changed lines of the file:
@@
 $EndComp
 $Comp
-L GND #PWR0240
+L GND #PWR0241
 U 1 1 58C0DF31
 P 7200 3400
-F 0 "#PWR0240" H 7200 3150 50  0001 C CNN
+F 0 "#PWR0241" H 7200 3150 50  0001 C CNN
 F 1 "GND" H 7200 3250 50  0000 C CNN
 F 2 "" H 7200 3400 50  0000 C CNN
@@
 $EndComp
 $Comp
-L GND #PWR0241
+L GND #PWR0242
 U 1 1 58C0DF3E
 P 10050 3450
-F 0 "#PWR0241" H 10050 3200 50  0001 C CNN
+F 0 "#PWR0242" H 10050 3200 50  0001 C CNN
 F 1 "GND" H 10055 3277 50  0000 C CNN
 F 2 "" H 10050 3450 50  0000 C CNN
@@
 $EndComp
 $Comp
-L +24V #PWR0242
+L +24V #PWR0243
 U 1 1 58C0DF44
 P 8250 2950
-F 0 "#PWR0242" H 8250 2800 50  0001 C CNN
+F 0 "#PWR0243" H 8250 2800 50  0001 C CNN
 F 1 "+24V" H 8265 3123 50  0000 C CNN
 F 2 "" H 8250 2950 50  0000 C CNN
@@
 $EndComp
 $Comp
-L R R172
+L R R171
 U 1 1 58C0DF51
 P 10450 6800
-F 0 "R172" H 10400 6750 50  0000 R CNN
+F 0 "R171" H 10400 6750 50  0000 R CNN
 F 1 "220mΩ" H 10400 6850 50  0000 R CNN
 F 2 "" V 10380 6800 50  0001 C CNN
@@
 $EndComp
 $Comp
-L R R171
+L R R170
 U 1 1 58C0DF58
 P 9650 6800
-F 0 "R171" H 9600 6750 50  0000 R CNN
+F 0 "R170" H 9600 6750 50  0000 R CNN
 F 1 "220mΩ" H 9600 6850 50  0000 R CNN
 F 2 "" V 9580 6800 50  0001 C CNN
@@
 $EndComp
 $Comp
-L GND #PWR0243
+L GND #PWR0244
 U 1 1 58C0DF5F
 P 9350 7150
-F 0 "#PWR0243" H 9350 6900 50  0001 C CNN
+F 0 "#PWR0244" H 9350 6900 50  0001 C CNN
 F 1 "GND" H 9355 6977 50  0000 C CNN
 F 2 "" H 9350 7150 50  0000 C CNN
@@
 NoConn ~ 7400 5700
 $Comp
-L R R168
+L R R167
 U 1 1 58C0DF66
 P 7000 3850
-F 0 "R168" V 6900 3850 50  0000 C CNN
+F 0 "R167" V 6900 3850 50  0000 C CNN
 F 1 "2.2Ω" V 7000 3850 50  0000 C CNN
 F 2 "" V 6930 3850 50  0001 C CNN
@@
 NoConn ~ 7400 5800
 $Comp
-L GND #PWR0244
+L GND #PWR0245
 U 1 1 58C0DF82
 P 7350 6200
-F 0 "#PWR0244" H 7350 5950 50  0001 C CNN
+F 0 "#PWR0245" H 7350 5950 50  0001 C CNN
 F 1 "GND" H 7355 6027 50  0000 C CNN
 F 2 "" H 7350 6200 50  0000 C CNN
@@
 Z2_FAULT
 $Comp
-L R R166
+L R R165
 U 1 1 58C0DF90
 P 5750 4350
-F 0 "R166" H 5819 4396 50  0000 L CNN
+F 0 "R165" H 5819 4396 50  0000 L CNN
 F 1 "4.7kΩ" H 5819 4305 50  0000 L CNN
 F 2 "" V 5680 4350 50  0001 C CNN
@@
 5VOUT
 $Comp
-L R R169
+L R R168
 U 1 1 58C0DFA2
 P 8950 6800
-F 0 "R169" H 9019 6846 50  0000 L CNN
+F 0 "R168" H 9019 6846 50  0000 L CNN
 F 1 "5.23kΩ" H 9019 6755 50  0000 L CNN
 F 2 "" V 8880 6800 50  0001 C CNN
@@
 5VOUT
 $Comp
-L R R170
+L R R169
 U 1 1 58C0DFAA
 P 9150 7000
-F 0 "R170" V 8950 7000 50  0000 C CNN
+F 0 "R169" V 8950 7000 50  0000 C CNN
 F 1 "4.75kΩ" V 9050 7000 50  0000 C CNN
 F 2 "" V 9080 7000 50  0001 C CNN
@@
 $EndComp
 $Comp
-L R R167
+L R R166
 U 1 1 58C0DFB1
 P 6100 4350
-F 0 "R167" H 6169 4396 50  0000 L CNN
+F 0 "R166" H 6169 4396 50  0000 L CNN
 F 1 "4.7kΩ" H 6169 4305 50  0000 L CNN
 F 2 "" V 6030 4350 50  0001 C CNN
@@
 $EndComp
 $Comp
-L GND #PWR0245
+L GND #PWR0246
 U 1 1 58C0DFC6
 P 8950 5300
-F 0 "#PWR0245" H 8950 5050 50  0001 C CNN
+F 0 "#PWR0246" H 8950 5050 50  0001 C CNN
 F 1 "GND" H 8950 5150 50  0000 C CNN
 F 2 "" H 8950 5300 50  0000 C CNN
@@
 $EndComp
 $Comp
-L GND #PWR0246
+L GND #PWR0247
 U 1 1 58C0DFDA
 P 8950 6150
-F 0 "#PWR0246" H 8950 5900 50  0001 C CNN
+F 0 "#PWR0247" H 8950 5900 50  0001 C CNN
 F 1 "GND" H 8950 6000 50  0000 C CNN
 F 2 "" H 8950 6150 50  0000 C CNN
@@
 	8850 6100 8850 6050
 $Comp
-L R R165
+L R R164
 U 1 1 58C0E05B
 P 5400 4350
-F 0 "R165" H 5469 4396 50  0000 L CNN
+F 0 "R164" H 5469 4396 50  0000 L CNN
 F 1 "4.7kΩ" H 5469 4305 50  0000 L CNN
 F 2 "" V 5330 4350 50  0001 C CNN
@@
 	5400 3600 7400 3600
 $Comp
-L VDD_3V3B #PWR0247
+L VDD_3V3B #PWR0248
 U 1 1 5A315EF4
 P 6450 3550
-F 0 "#PWR0247" H 6450 3400 50  0001 C CNN
+F 0 "#PWR0248" H 6450 3400 50  0001 C CNN
 F 1 "VDD_3V3B" H 6465 3723 50  0000 C CNN
 F 2 "" H 6450 3550 50  0000 C CNN

Commit message: Add equivalent annotations document, associate more footprints
Parts:
- C151: renamed from C149; footprint (none) -> Capacitors_SMD:C_0603
- C152: renamed from C150; footprint (none) -> Capacitors_SMD:C_0603
- C153: renamed from C151; footprint (none) -> Capacitors_SMD:C_0603
- C154: renamed from C152; footprint (none) -> Capacitors_SMD:C_0402
- C155: renamed from C153; footprint (none) -> Capacitors_SMD:C_0402
- C156: renamed from C154; footprint (none) -> Capacitors_SMD:C_0603
- C157: renamed from C155; footprint (none) -> Capacitors_SMD:C_0603
- C158: renamed from C156; footprint (none) -> Capacitors_SMD:C_0603
- C159: renamed from C157; footprint (none) -> Capacitors_SMD:C_0603
- C160: renamed from C158; footprint (none) -> Capacitors_SMD:C_0603
- C161: renamed from C159; footprint (none) -> Capacitors_SMD:C_0603
- C162: renamed from C160; footprint (none) -> Capacitors_SMD:C_0603
- C163: renamed from C161; footprint (none) -> Capacitors_SMD:C_0603
- C164: renamed from C162; value 4.7μF -> 10μF; footprint (none) -> Capacitors_SMD:C_0805
- C165: renamed from C163; footprint (none) -> Capacitors_SMD:c_elec_8x10
- C166: renamed from C164; footprint (none) -> Capacitors_SMD:C_0603
- renumbered R164 to R163, R165 to R164, R166 to R165, R167 to R166, R168 to R167, R169 to R168, R170 to R169, R171 to R170
Changed lines of the file:
@@
 Z2_SG
 $Comp
-L C C151
+L C C153
 U 1 1 58C0DF15
 P 7200 3200
-F 0 "C151" H 7086 3154 50  0000 R CNN
+F 0 "C153" H 7086 3154 50  0000 R CNN
 F 1 "100nF" H 7086 3245 50  0000 R CNN
-F 2 "" H 7238 3050 50  0001 C CNN
+F 2 "Capacitors_SMD:C_0603" H 7238 3050 50  0001 C CNN
 F 3 "" H 7200 3200 50  0000 C CNN
 	1    7200 3200
@@
 $EndComp
 $Comp
-L C C156
+L C C158
 U 1 1 58C0DF1C
 P 9000 3750
-F 0 "C156" V 8950 3650 50  0000 C CNN
+F 0 "C158" V 8950 3650 50  0000 C CNN
 F 1 "100nF" V 8950 3925 50  0000 C CNN
-F 2 "" H 9038 3600 50  0001 C CNN
+F 2 "Capacitors_SMD:C_0603" H 9038 3600 50  0001 C CNN
 F 3 "" H 9000 3750 50  0000 C CNN
 	1    9000 3750
@@
 $EndComp
 $Comp
-L CP1 C163
+L CP1 C165
 U 1 1 58C0DF23
 P 10350 3200
-F 0 "C163" H 10400 3300 50  0000 C CNN
+F 0 "C165" H 10450 3300 50  0000 C CNN
 F 1 "100μF" H 10500 3100 50  0000 C CNN
-F 2 "" H 10350 3200 50  0001 C CNN
+F 2 "Capacitors_SMD:c_elec_8x10" H 10350 3200 50  0001 C CNN
 F 3 "" H 10350 3200 50  0000 C CNN
 	1    10350 3200
@@
 $EndComp
 $Comp
-L C C159
+L C C161
 U 1 1 58C0DF2A
 P 9450 3200
-F 0 "C159" H 9400 3300 50  0000 C CNN
+F 0 "C161" H 9350 3300 50  0000 C CNN
 F 1 "100nF" H 9325 3100 50  0000 C CNN
-F 2 "" H 9488 3050 50  0001 C CNN
+F 2 "Capacitors_SMD:C_0603" H 9488 3050 50  0001 C CNN
 F 3 "" H 9450 3200 50  0000 C CNN
 	1    9450 3200
@@
 $EndComp
 $Comp
-L GND #PWR0241
+L GND #PWR0242
 U 1 1 58C0DF31
 P 7200 3400
-F 0 "#PWR0241" H 7200 3150 50  0001 C CNN
+F 0 "#PWR0242" H 7200 3150 50  0001 C CNN
 F 1 "GND" H 7200 3250 50  0000 C CNN
 F 2 "" H 7200 3400 50  0000 C CNN
@@
 $EndComp
 $Comp
-L C C160
+L C C162
 U 1 1 58C0DF37
 P 9750 3200
-F 0 "C160" H 9700 3300 50  0000 C CNN
+F 0 "C162" H 9650 3300 50  0000 C CNN
 F 1 "100nF" H 9625 3100 50  0000 C CNN
-F 2 "" H 9788 3050 50  0001 C CNN
+F 2 "Capacitors_SMD:C_0603" H 9788 3050 50  0001 C CNN
 F 3 "" H 9750 3200 50  0000 C CNN
 	1    9750 3200
@@
 $EndComp
 $Comp
-L GND #PWR0242
+L GND #PWR0243
 U 1 1 58C0DF3E
 P 10050 3450
-F 0 "#PWR0242" H 10050 3200 50  0001 C CNN
+F 0 "#PWR0243" H 10050 3200 50  0001 C CNN
 F 1 "GND" H 10055 3277 50  0000 C CNN
 F 2 "" H 10050 3450 50  0000 C CNN
@@
 $EndComp
 $Comp
-L +24V #PWR0243
+L +24V #PWR0244
 U 1 1 58C0DF44
 P 8250 2950
-F 0 "#PWR0243" H 8250 2800 50  0001 C CNN
+F 0 "#PWR0244" H 8250 2800 50  0001 C CNN
 F 1 "+24V" H 8265 3123 50  0000 C CNN
 F 2 "" H 8250 2950 50  0000 C CNN
@@
 $EndComp
 $Comp
-L C C153
+L C C155
 U 1 1 58C0DF4A
 P 8850 4250
-F 0 "C153" H 8965 4296 50  0000 L CNN
+F 0 "C155" H 8965 4296 50  0000 L CNN
 F 1 "22nF" H 8965 4205 50  0000 L CNN
-F 2 "" H 8888 4100 50  0001 C CNN
+F 2 "Capacitors_SMD:C_0402" H 8888 4100 50  0001 C CNN
 F 3 "" H 8850 4250 50  0000 C CNN
 	1    8850 4250
@@
 $EndComp
 $Comp
-L R R171
+L R R170
 U 1 1 58C0DF51
 P 10450 6800
-F 0 "R171" H 10400 6750 50  0000 R CNN
+F 0 "R170" H 10400 6750 50  0000 R CNN
 F 1 "220mΩ" H 10400 6850 50  0000 R CNN
 F 2 "" V 10380 6800 50  0001 C CNN
@@
 $EndComp
 $Comp
-L R R170
+L R R169
 U 1 1 58C0DF58
 P 9650 6800
-F 0 "R170" H 9600 6750 50  0000 R CNN
+F 0 "R169" H 9600 6750 50  0000 R CNN
 F 1 "220mΩ" H 9600 6850 50  0000 R CNN
 F 2 "" V 9580 6800 50  0001 C CNN
@@
 $EndComp
 $Comp
-L GND #PWR0244
+L GND #PWR0245
 U 1 1 58C0DF5F
 P 9350 7150
-F 0 "#PWR0244" H 9350 6900 50  0001 C CNN
+F 0 "#PWR0245" H 9350 6900 50  0001 C CNN
 F 1 "GND" H 9355 6977 50  0000 C CNN
 F 2 "" H 9350 7150 50  0000 C CNN
@@
 NoConn ~ 7400 5700
 $Comp
-L R R167
+L R R166
 U 1 1 58C0DF66
 P 7000 3850
-F 0 "R167" V 6900 3850 50  0000 C CNN
+F 0 "R166" V 6900 3850 50  0000 C CNN
 F 1 "2.2Ω" V 7000 3850 50  0000 C CNN
 F 2 "" V 6930 3850 50  0001 C CNN
@@
 $EndComp
 $Comp
-L C C150
+L C C152
 U 1 1 58C0DF6D
 P 6800 4050
-F 0 "C150" H 6850 4150 50  0000 L CNN
+F 0 "C152" H 6850 4150 50  0000 L CNN
 F 1 "470nF" H 6825 3950 50  0000 L CNN
-F 2 "" H 6838 3900 50  0001 C CNN
+F 2 "Capacitors_SMD:C_0603" H 6838 3900 50  0001 C CNN
 F 3 "" H 6800 4050 50  0000 C CNN
 	1    6800 4050
@@
 NoConn ~ 7400 5800
 $Comp
-L GND #PWR0245
+L GND #PWR0246
 U 1 1 58C0DF82
 P 7350 6200
-F 0 "#PWR0245" H 7350 5950 50  0001 C CNN
+F 0 "#PWR0246" H 7350 5950 50  0001 C CNN
 F 1 "GND" H 7355 6027 50  0000 C CNN
 F 2 "" H 7350 6200 50  0000 C CNN
@@
 $EndComp
 $Comp
-L C C161
+L C C163
 U 1 1 58C0DF88
 P 9800 6800
-F 0 "C161" H 9850 6900 50  0000 L CNN
+F 0 "C163" H 9850 6900 50  0000 L CNN
 F 1 "100nF" H 9850 6700 50  0000 L CNN
-F 2 "" H 9838 6650 50  0001 C CNN
+F 2 "Capacitors_SMD:C_0603" H 9838 6650 50  0001 C CNN
 F 3 "" H 9800 6800 50  0000 C CNN
 	1    9800 6800
@@
 Z2_FAULT
 $Comp
-L R R165
+L R R164
 U 1 1 58C0DF90
 P 5750 4350
-F 0 "R165" H 5819 4396 50  0000 L CNN
+F 0 "R164" H 5819 4396 50  0000 L CNN
 F 1 "4.7kΩ" H 5819 4305 50  0000 L CNN
 F 2 "" V 5680 4350 50  0001 C CNN
@@
 NoConn ~ 7400 4650
 $Comp
-L C C152
+L C C154
 U 1 1 58C0DF9A
 P 7200 4050
-F 0 "C152" H 7250 4150 50  0000 L CNN
+F 0 "C154" H 7250 4150 50  0000 L CNN
 F 1 "4.7μF" H 7250 3950 50  0000 L CNN
-F 2 "" H 7238 3900 50  0001 C CNN
+F 2 "Capacitors_SMD:C_0402" H 7238 3900 50  0001 C CNN
 F 3 "" H 7200 4050 50  0000 C CNN
 	1    7200 4050
@@
 5VOUT
 $Comp
-L R R168
+L R R167
 U 1 1 58C0DFA2
 P 8950 6800
-F 0 "R168" H 9019 6846 50  0000 L CNN
+F 0 "R167" H 9019 6846 50  0000 L CNN
 F 1 "5.23kΩ" H 9019 6755 50  0000 L CNN
 F 2 "" V 8880 6800 50  0001 C CNN
@@
 5VOUT
 $Comp
-L R R169
+L R R168
 U 1 1 58C0DFAA
 P 9150 7000
-F 0 "R169" V 8950 7000 50  0000 C CNN
+F 0 "R168" V 8950 7000 50  0000 C CNN
 F 1 "4.75kΩ" V 9050 7000 50  0000 C CNN
 F 2 "" V 9080 7000 50  0001 C CNN
@@
 $EndComp
 $Comp
-L R R166
+L R R165
 U 1 1 58C0DFB1
 P 6100 4350
-F 0 "R166" H 6169 4396 50  0000 L CNN
+F 0 "R165" H 6169 4396 50  0000 L CNN
 F 1 "4.7kΩ" H 6169 4305 50  0000 L CNN
 F 2 "" V 6030 4350 50  0001 C CNN
@@
 $EndComp
 $Comp
-L C C164
+L C C166
 U 1 1 58C0DFB8
 P 10600 6800
-F 0 "C164" H 10650 6900 50  0000 L CNN
+F 0 "C166" H 10650 6900 50  0000 L CNN
 F 1 "100nF" H 10650 6700 50  0000 L CNN
-F 2 "" H 10638 6650 50  0001 C CNN
+F 2 "Capacitors_SMD:C_0603" H 10638 6650 50  0001 C CNN
 F 3 "" H 10600 6800 50  0000 C CNN
 	1    10600 6800
@@
 $EndComp
 $Comp
-L C C154
+L C C156
 U 1 1 58C0DFBF
 P 8850 5050
-F 0 "C154" H 8875 5150 50  0000 L CNN
+F 0 "C156" H 8875 5150 50  0000 L CNN
 F 1 "470pF" H 8850 4950 50  0000 L CNN
-F 2 "" H 8888 4900 50  0001 C CNN
+F 2 "Capacitors_SMD:C_0603" H 8888 4900 50  0001 C CNN
 F 3 "" H 8850 5050 50  0000 C CNN
 	1    8850 5050
@@
 $EndComp
 $Comp
-L GND #PWR0246
+L GND #PWR0247
 U 1 1 58C0DFC6
 P 8950 5300
-F 0 "#PWR0246" H 8950 5050 50  0001 C CNN
+F 0 "#PWR0247" H 8950 5050 50  0001 C CNN
 F 1 "GND" H 8950 5150 50  0000 C CNN
 F 2 "" H 8950 5300 50  0000 C CNN
@@
 $EndComp
 $Comp
-L C C157
+L C C159
 U 1 1 58C0DFCC
 P 9050 5050
-F 0 "C157" H 9075 5150 50  0000 L CNN
+F 0 "C159" H 9075 5150 50  0000 L CNN
 F 1 "470pF" H 9075 4950 50  0000 L CNN
-F 2 "" H 9088 4900 50  0001 C CNN
+F 2 "Capacitors_SMD:C_0603" H 9088 4900 50  0001 C CNN
 F 3 "" H 9050 5050 50  0000 C CNN
 	1    9050 5050
@@
 $EndComp
 $Comp
-L C C155
+L C C157
 U 1 1 58C0DFD3
 P 8850 5900
-F 0 "C155" H 8875 6000 50  0000 L CNN
+F 0 "C157" H 8875 6000 50  0000 L CNN
 F 1 "470pF" H 8850 5800 50  0000 L CNN
-F 2 "" H 8888 5750 50  0001 C CNN
+F 2 "Capacitors_SMD:C_0603" H 8888 5750 50  0001 C CNN
 F 3 "" H 8850 5900 50  0000 C CNN
 	1    8850 5900
@@
 $EndComp
 $Comp
-L GND #PWR0247
+L GND #PWR0248
 U 1 1 58C0DFDA
 P 8950 6150
-F 0 "#PWR0247" H 8950 5900 50  0001 C CNN
+F 0 "#PWR0248" H 8950 5900 50  0001 C CNN
 F 1 "GND" H 8950 6000 50  0000 C CNN
 F 2 "" H 8950 6150 50  0000 C CNN
@@
 $EndComp
 $Comp
-L C C158
+L C C160
 U 1 1 58C0DFE0
 P 9050 5900
-F 0 "C158" H 9075 6000 50  0000 L CNN
+F 0 "C160" H 9075 6000 50  0000 L CNN
 F 1 "470pF" H 9075 5800 50  0000 L CNN
-F 2 "" H 9088 5750 50  0001 C CNN
+F 2 "Capacitors_SMD:C_0603" H 9088 5750 50  0001 C CNN
 F 3 "" H 9050 5900 50  0000 C CNN
 	1    9050 5900
@@
 	8850 6100 8850 6050
 $Comp
-L R R164
+L R R163
 U 1 1 58C0E05B
 P 5400 4350
-F 0 "R164" H 5469 4396 50  0000 L CNN
+F 0 "R163" H 5469 4396 50  0000 L CNN
 F 1 "4.7kΩ" H 5469 4305 50  0000 L CNN
 F 2 "" V 5330 4350 50  0001 C CNN
@@
 Connection ~ 5750 3600
 $Comp
-L C C162
+L C C164
 U 1 1 58C0E066
 P 10050 3200
-F 0 "C162" H 10000 3300 50  0000 C CNN
-F 1 "4.7μF" H 9925 3100 50  0000 C CNN
-F 2 "" H 10088 3050 50  0001 C CNN
+F 0 "C164" H 9950 3300 50  0000 C CNN
+F 1 "10μF" H 9925 3100 50  0000 C CNN
+F 2 "Capacitors_SMD:C_0805" H 10088 3050 50  0001 C CNN
 F 3 "" H 10050 3200 50  0000 C CNN
 	1    10050 3200
@@
 	5400 3600 7400 3600
 $Comp
-L VDD_3V3B #PWR0248
+L VDD_3V3B #PWR0249
 U 1 1 5A315EF4
 P 6450 3550
-F 0 "#PWR0248" H 6450 3400 50  0001 C CNN
+F 0 "#PWR0249" H 6450 3400 50  0001 C CNN
 F 1 "VDD_3V3B" H 6465 3723 50  0000 C CNN
 F 2 "" H 6450 3550 50  0000 C CNN
@@
 $EndComp
 $Comp
-L C C149
+L C C151
 U 1 1 5A89C77B
 P 6450 4050
-F 0 "C149" H 6500 4150 50  0000 L CNN
+F 0 "C151" H 6500 4150 50  0000 L CNN
 F 1 "100nF" H 6475 3950 50  0000 L CNN
-F 2 "" H 6488 3900 50  0001 C CNN
+F 2 "Capacitors_SMD:C_0603" H 6488 3900 50  0001 C CNN
 F 3 "" H 6450 4050 50  0000 C CNN
 	1    6450 4050
