File: KiMBo/z2_stepper.sch (KiCad schematic (older format))
At the start: 25 parts, among them U25 TMC2130

Commit message: Connect X and Z stepper driver open-drain DIAG0 and DIAG1 lines together
Parts:
- removed R163, R164: 4.7kΩ, symbol R
- renumbered C151 to C149, C152 to C150, C153 to C151, C154 to C152, C155 to C153, C156 to C154, C157 to C155, C158 to C156, C159 to C157, C160 to C158, C161 to C159, C162 to C160, C163 to C161, C164 to C162, C165 to C163, C166 to C164, R165 to R161, R166 to R162, R167 to R163, R168 to R164, R169 to R165, R170 to R166, U25 to U23
Changed lines of the file:
@@
 Z2_SG
 $Comp
-L C C153
+L C C151
 U 1 1 58C0DF15
 P 7200 3200
-F 0 "C153" H 7086 3154 50  0000 R CNN
+F 0 "C151" H 7086 3154 50  0000 R CNN
 F 1 "100nF" H 7086 3245 50  0000 R CNN
 F 2 "Capacitors_SMD:C_0603" H 7238 3050 50  0001 C CNN
@@
 $EndComp
 $Comp
-L C C158
+L C C156
 U 1 1 58C0DF1C
 P 9000 3750
-F 0 "C158" V 8950 3650 50  0000 C CNN
+F 0 "C156" V 8950 3650 50  0000 C CNN
 F 1 "100nF" V 8950 3925 50  0000 C CNN
 F 2 "Capacitors_SMD:C_0603" H 9038 3600 50  0001 C CNN
@@
 $EndComp
 $Comp
-L CP1 C165
+L CP1 C163
 U 1 1 58C0DF23
 P 10350 3200
-F 0 "C165" H 10450 3300 50  0000 C CNN
+F 0 "C163" H 10450 3300 50  0000 C CNN
 F 1 "100μF" H 10500 3100 50  0000 C CNN
 F 2 "Capacitors_SMD:c_elec_8x10" H 10350 3200 50  0001 C CNN
@@
 $EndComp
 $Comp
-L C C161
+L C C159
 U 1 1 58C0DF2A
 P 9450 3200
-F 0 "C161" H 9350 3300 50  0000 C CNN
+F 0 "C159" H 9350 3300 50  0000 C CNN
 F 1 "100nF" H 9325 3100 50  0000 C CNN
 F 2 "Capacitors_SMD:C_0603" H 9488 3050 50  0001 C CNN
@@
 $EndComp
 $Comp
-L GND #PWR0242
+L GND #PWR0232
 U 1 1 58C0DF31
 P 7200 3400
-F 0 "#PWR0242" H 7200 3150 50  0001 C CNN
+F 0 "#PWR0232" H 7200 3150 50  0001 C CNN
 F 1 "GND" H 7200 3250 50  0000 C CNN
 F 2 "" H 7200 3400 50  0000 C CNN
@@
 $EndComp
 $Comp
-L C C162
+L C C160
 U 1 1 58C0DF37
 P 9750 3200
-F 0 "C162" H 9650 3300 50  0000 C CNN
+F 0 "C160" H 9650 3300 50  0000 C CNN
 F 1 "100nF" H 9625 3100 50  0000 C CNN
 F 2 "Capacitors_SMD:C_0603" H 9788 3050 50  0001 C CNN
@@
 $EndComp
 $Comp
-L GND #PWR0243
+L GND #PWR0233
 U 1 1 58C0DF3E
 P 10050 3450
-F 0 "#PWR0243" H 10050 3200 50  0001 C CNN
+F 0 "#PWR0233" H 10050 3200 50  0001 C CNN
 F 1 "GND" H 10055 3277 50  0000 C CNN
 F 2 "" H 10050 3450 50  0000 C CNN
@@
 $EndComp
 $Comp
-L +24V #PWR0244
+L +24V #PWR0234
 U 1 1 58C0DF44
 P 8250 2950
-F 0 "#PWR0244" H 8250 2800 50  0001 C CNN
+F 0 "#PWR0234" H 8250 2800 50  0001 C CNN
 F 1 "+24V" H 8265 3123 50  0000 C CNN
 F 2 "" H 8250 2950 50  0000 C CNN
@@
 $EndComp
 $Comp
-L C C155
+L C C153
 U 1 1 58C0DF4A
 P 8850 4250
-F 0 "C155" H 8965 4296 50  0000 L CNN
+F 0 "C153" H 8965 4296 50  0000 L CNN
 F 1 "22nF" H 8965 4205 50  0000 L CNN
 F 2 "Capacitors_SMD:C_0402" H 8888 4100 50  0001 C CNN
@@
 $EndComp
 $Comp
-L R R170
+L R R166
 U 1 1 58C0DF51
 P 10450 6800
-F 0 "R170" H 10400 6750 50  0000 R CNN
+F 0 "R166" H 10400 6750 50  0000 R CNN
 F 1 "220mΩ" H 10400 6850 50  0000 R CNN
 F 2 "" V 10380 6800 50  0001 C CNN
@@
 $EndComp
 $Comp
-L R R169
+L R R165
 U 1 1 58C0DF58
 P 9650 6800
-F 0 "R169" H 9600 6750 50  0000 R CNN
+F 0 "R165" H 9600 6750 50  0000 R CNN
 F 1 "220mΩ" H 9600 6850 50  0000 R CNN
 F 2 "" V 9580 6800 50  0001 C CNN
@@
 $EndComp
 $Comp
-L GND #PWR0245
+L GND #PWR0235
 U 1 1 58C0DF5F
 P 9350 7150
-F 0 "#PWR0245" H 9350 6900 50  0001 C CNN
+F 0 "#PWR0235" H 9350 6900 50  0001 C CNN
 F 1 "GND" H 9355 6977 50  0000 C CNN
 F 2 "" H 9350 7150 50  0000 C CNN
@@
 NoConn ~ 7400 5700
 $Comp
-L R R166
+L R R162
 U 1 1 58C0DF66
 P 7000 3850
-F 0 "R166" V 6900 3850 50  0000 C CNN
+F 0 "R162" V 6900 3850 50  0000 C CNN
 F 1 "2.2Ω" V 7000 3850 50  0000 C CNN
 F 2 "" V 6930 3850 50  0001 C CNN
@@
 $EndComp
 $Comp
-L C C152
+L C C150
 U 1 1 58C0DF6D
 P 6800 4050
-F 0 "C152" H 6850 4150 50  0000 L CNN
+F 0 "C150" H 6850 4150 50  0000 L CNN
 F 1 "470nF" H 6825 3950 50  0000 L CNN
 F 2 "Capacitors_SMD:C_0603" H 6838 3900 50  0001 C CNN
@@
 NoConn ~ 7400 5800
 $Comp
-L GND #PWR0246
+L GND #PWR0236
 U 1 1 58C0DF82
 P 7350 6200
-F 0 "#PWR0246" H 7350 5950 50  0001 C CNN
+F 0 "#PWR0236" H 7350 5950 50  0001 C CNN
 F 1 "GND" H 7355 6027 50  0000 C CNN
 F 2 "" H 7350 6200 50  0000 C CNN
@@
 $EndComp
 $Comp
-L C C163
+L C C161
 U 1 1 58C0DF88
 P 9800 6800
-F 0 "C163" H 9850 6900 50  0000 L CNN
+F 0 "C161" H 9850 6900 50  0000 L CNN
 F 1 "100nF" H 9850 6700 50  0000 L CNN
 F 2 "Capacitors_SMD:C_0603" H 9838 6650 50  0001 C CNN
@@
 Text HLabel 5700 5000 0    60   Output ~ 0
 Z2_FAULT
-$Comp
-L R R164
-U 1 1 58C0DF90
-P 5750 4350
-F 0 "R164" H 5819 4396 50  0000 L CNN
-F 1 "4.7kΩ" H 5819 4305 50  0000 L CNN
-F 2 "" V 5680 4350 50  0001 C CNN
-F 3 "" H 5750 4350 50  0000 C CNN
-	1    5750 4350
-	-1   0    0    -1
-$EndComp
 Text HLabel 5350 4550 0    60   Input ~ 0
 ~Z2_EN
 NoConn ~ 7400 4650
 $Comp
-L C C154
+L C C152
 U 1 1 58C0DF9A
 P 7200 4050
-F 0 "C154" H 7250 4150 50  0000 L CNN
+F 0 "C152" H 7250 4150 50  0000 L CNN
 F 1 "4.7μF" H 7250 3950 50  0000 L CNN
 F 2 "Capacitors_SMD:C_0402" H 7238 3900 50  0001 C CNN
@@
 5VOUT
 $Comp
-L R R167
+L R R163
 U 1 1 58C0DFA2
 P 8950 6800
-F 0 "R167" H 9019 6846 50  0000 L CNN
+F 0 "R163" H 9019 6846 50  0000 L CNN
 F 1 "5.23kΩ" H 9019 6755 50  0000 L CNN
 F 2 "" V 8880 6800 50  0001 C CNN
@@
 5VOUT
 $Comp
-L R R168
+L R R164
 U 1 1 58C0DFAA
 P 9150 7000
-F 0 "R168" V 8950 7000 50  0000 C CNN
+F 0 "R164" V 8950 7000 50  0000 C CNN
 F 1 "4.75kΩ" V 9050 7000 50  0000 C CNN
 F 2 "" V 9080 7000 50  0001 C CNN
@@
 $EndComp
 $Comp
-L R R165
+L R R161
 U 1 1 58C0DFB1
 P 6100 4350
-F 0 "R165" H 6169 4396 50  0000 L CNN
+F 0 "R161" H 6169 4396 50  0000 L CNN
 F 1 "4.7kΩ" H 6169 4305 50  0000 L CNN
 F 2 "" V 6030 4350 50  0001 C CNN
@@
 $EndComp
 $Comp
-L C C166
+L C C164
 U 1 1 58C0DFB8
 P 10600 6800
-F 0 "C166" H 10650 6900 50  0000 L CNN
+F 0 "C164" H 10650 6900 50  0000 L CNN
 F 1 "100nF" H 10650 6700 50  0000 L CNN
 F 2 "Capacitors_SMD:C_0603" H 10638 6650 50  0001 C CNN
@@
 $EndComp
 $Comp
-L C C156
+L C C154
 U 1 1 58C0DFBF
 P 8850 5050
-F 0 "C156" H 8875 5150 50  0000 L CNN
+F 0 "C154" H 8875 5150 50  0000 L CNN
 F 1 "470pF" H 8850 4950 50  0000 L CNN
 F 2 "Capacitors_SMD:C_0603" H 8888 4900 50  0001 C CNN
@@
 $EndComp
 $Comp
-L GND #PWR0247
+L GND #PWR0237
 U 1 1 58C0DFC6
 P 8950 5300
-F 0 "#PWR0247" H 8950 5050 50  0001 C CNN
+F 0 "#PWR0237" H 8950 5050 50  0001 C CNN
 F 1 "GND" H 8950 5150 50  0000 C CNN
 F 2 "" H 8950 5300 50  0000 C CNN
@@
 $EndComp
 $Comp
-L C C159
+L C C157
 U 1 1 58C0DFCC
 P 9050 5050
-F 0 "C159" H 9075 5150 50  0000 L CNN
+F 0 "C157" H 9075 5150 50  0000 L CNN
 F 1 "470pF" H 9075 4950 50  0000 L CNN
 F 2 "Capacitors_SMD:C_0603" H 9088 4900 50  0001 C CNN
@@
 $EndComp
 $Comp
-L C C157
+L C C155
 U 1 1 58C0DFD3
 P 8850 5900
-F 0 "C157" H 8875 6000 50  0000 L CNN
+F 0 "C155" H 8875 6000 50  0000 L CNN
 F 1 "470pF" H 8850 5800 50  0000 L CNN
 F 2 "Capacitors_SMD:C_0603" H 8888 5750 50  0001 C CNN
@@
 $EndComp
 $Comp
-L GND #PWR0248
+L GND #PWR0238
 U 1 1 58C0DFDA
 P 8950 6150
-F 0 "#PWR0248" H 8950 5900 50  0001 C CNN
+F 0 "#PWR0238" H 8950 5900 50  0001 C CNN
 F 1 "GND" H 8950 6000 50  0000 C CNN
 F 2 "" H 8950 6150 50  0000 C CNN
@@
 $EndComp
 $Comp
-L C C160
+L C C158
 U 1 1 58C0DFE0
 P 9050 5900
-F 0 "C160" H 9075 6000 50  0000 L CNN
+F 0 "C158" H 9075 6000 50  0000 L CNN
 F 1 "470pF" H 9075 5800 50  0000 L CNN
 F 2 "Capacitors_SMD:C_0603" H 9088 5750 50  0001 C CNN
@@
 $EndComp
 $Comp
-L TMC2130 U25
+L TMC2130 U23
 U 1 1 58C0DFE7
 P 8100 4800
-F 0 "U25" H 7650 6300 60  0000 C CNN
+F 0 "U23" H 7650 6300 60  0000 C CNN
 F 1 "TMC2130" H 8400 6300 60  0000 C CNN
 F 2 "" H 8100 5100 60  0001 C CNN
@@
 	5700 5000 7400 5000
 Wire Wire Line
-	5750 4500 5750 5000
-Wire Wire Line
-	5750 4200 5750 3600
-Connection ~ 5750 5000
-Wire Wire Line
 	5350 4550 7400 4550
 Wire Wire Line
@@
 Wire Wire Line
 	6100 3600 6100 4200
-Connection ~ 6100 3600
 Wire Wire Line
 	5350 4900 7400 4900
@@
 	8850 6100 8850 6050
 $Comp
-L R R163
-U 1 1 58C0E05B
-P 5400 4350
-F 0 "R163" H 5469 4396 50  0000 L CNN
-F 1 "4.7kΩ" H 5469 4305 50  0000 L CNN
-F 2 "" V 5330 4350 50  0001 C CNN
-F 3 "" H 5400 4350 50  0000 C CNN
-	1    5400 4350
-	-1   0    0    -1
-$EndComp
-Wire Wire Line
-	5400 4500 5400 4900
-Connection ~ 5400 4900
-Wire Wire Line
-	5400 4200 5400 3600
-Connection ~ 5750 3600
-$Comp
-L C C164
+L C C162
 U 1 1 58C0E066
 P 10050 3200
-F 0 "C164" H 9950 3300 50  0000 C CNN
+F 0 "C162" H 9950 3300 50  0000 C CNN
 F 1 "10μF" H 9925 3100 50  0000 C CNN
 F 2 "Capacitors_SMD:C_0805" H 10088 3050 50  0001 C CNN
@@
 Wire Wire Line
 	8800 4700 9100 4700
-Wire Wire Line
-	5400 3600 7400 3600
-$Comp
-L VDD_3V3B #PWR0249
+$Comp
+L VDD_3V3B #PWR0239
 U 1 1 5A315EF4
 P 6450 3550
-F 0 "#PWR0249" H 6450 3400 50  0001 C CNN
+F 0 "#PWR0239" H 6450 3400 50  0001 C CNN
 F 1 "VDD_3V3B" H 6465 3723 50  0000 C CNN
 F 2 "" H 6450 3550 50  0000 C CNN
@@
 $EndComp
 $Comp
-L C C151
+L C C149
 U 1 1 5A89C77B
 P 6450 4050
-F 0 "C151" H 6500 4150 50  0000 L CNN
+F 0 "C149" H 6500 4150 50  0000 L CNN
 F 1 "100nF" H 6475 3950 50  0000 L CNN
 F 2 "Capacitors_SMD:C_0603" H 6488 3900 50  0001 C CNN
@@
 	-1   0    0    -1
 $EndComp
+Wire Wire Line
+	6100 3600 7400 3600
 $EndSCHEMATC

Commit message: Leave SPI0 free for a display, reassign pins so SPI1 is available
Fix some typos/errors
Parts:
- renumbered R161 to R163, R162 to R164, R163 to R165, R164 to R166, R165 to R167, R166 to R168, U23 to U22
Changed lines of the file:
@@
 $EndComp
 $Comp
-L GND #PWR0232
+L GND #PWR0231
 U 1 1 58C0DF31
 P 7200 3400
-F 0 "#PWR0232" H 7200 3150 50  0001 C CNN
+F 0 "#PWR0231" H 7200 3150 50  0001 C CNN
 F 1 "GND" H 7200 3250 50  0000 C CNN
 F 2 "" H 7200 3400 50  0000 C CNN
@@
 $EndComp
 $Comp
-L GND #PWR0233
+L GND #PWR0232
 U 1 1 58C0DF3E
 P 10050 3450
-F 0 "#PWR0233" H 10050 3200 50  0001 C CNN
+F 0 "#PWR0232" H 10050 3200 50  0001 C CNN
 F 1 "GND" H 10055 3277 50  0000 C CNN
 F 2 "" H 10050 3450 50  0000 C CNN
@@
 $EndComp
 $Comp
-L +24V #PWR0234
+L +24V #PWR0233
 U 1 1 58C0DF44
 P 8250 2950
-F 0 "#PWR0234" H 8250 2800 50  0001 C CNN
+F 0 "#PWR0233" H 8250 2800 50  0001 C CNN
 F 1 "+24V" H 8265 3123 50  0000 C CNN
 F 2 "" H 8250 2950 50  0000 C CNN
@@
 $EndComp
 $Comp
-L R R166
+L R R168
 U 1 1 58C0DF51
 P 10450 6800
-F 0 "R166" H 10400 6750 50  0000 R CNN
+F 0 "R168" H 10400 6750 50  0000 R CNN
 F 1 "220mΩ" H 10400 6850 50  0000 R CNN
 F 2 "" V 10380 6800 50  0001 C CNN
@@
 $EndComp
 $Comp
-L R R165
+L R R167
 U 1 1 58C0DF58
 P 9650 6800
-F 0 "R165" H 9600 6750 50  0000 R CNN
+F 0 "R167" H 9600 6750 50  0000 R CNN
 F 1 "220mΩ" H 9600 6850 50  0000 R CNN
 F 2 "" V 9580 6800 50  0001 C CNN
@@
 $EndComp
 $Comp
-L GND #PWR0235
+L GND #PWR0234
 U 1 1 58C0DF5F
 P 9350 7150
-F 0 "#PWR0235" H 9350 6900 50  0001 C CNN
+F 0 "#PWR0234" H 9350 6900 50  0001 C CNN
 F 1 "GND" H 9355 6977 50  0000 C CNN
 F 2 "" H 9350 7150 50  0000 C CNN
@@
 NoConn ~ 7400 5700
 $Comp
-L R R162
+L R R164
 U 1 1 58C0DF66
 P 7000 3850
-F 0 "R162" V 6900 3850 50  0000 C CNN
+F 0 "R164" V 6900 3850 50  0000 C CNN
 F 1 "2.2Ω" V 7000 3850 50  0000 C CNN
 F 2 "" V 6930 3850 50  0001 C CNN
@@
 NoConn ~ 7400 5800
 $Comp
-L GND #PWR0236
+L GND #PWR0235
 U 1 1 58C0DF82
 P 7350 6200
-F 0 "#PWR0236" H 7350 5950 50  0001 C CNN
+F 0 "#PWR0235" H 7350 5950 50  0001 C CNN
 F 1 "GND" H 7355 6027 50  0000 C CNN
 F 2 "" H 7350 6200 50  0000 C CNN
@@
 5VOUT
 $Comp
-L R R163
+L R R165
 U 1 1 58C0DFA2
 P 8950 6800
-F 0 "R163" H 9019 6846 50  0000 L CNN
+F 0 "R165" H 9019 6846 50  0000 L CNN
 F 1 "5.23kΩ" H 9019 6755 50  0000 L CNN
 F 2 "" V 8880 6800 50  0001 C CNN
@@
 5VOUT
 $Comp
-L R R164
+L R R166
 U 1 1 58C0DFAA
 P 9150 7000
-F 0 "R164" V 8950 7000 50  0000 C CNN
+F 0 "R166" V 8950 7000 50  0000 C CNN
 F 1 "4.75kΩ" V 9050 7000 50  0000 C CNN
 F 2 "" V 9080 7000 50  0001 C CNN
@@
 $EndComp
 $Comp
-L R R161
+L R R163
 U 1 1 58C0DFB1
 P 6100 4350
-F 0 "R161" H 6169 4396 50  0000 L CNN
+F 0 "R163" H 6169 4396 50  0000 L CNN
 F 1 "4.7kΩ" H 6169 4305 50  0000 L CNN
 F 2 "" V 6030 4350 50  0001 C CNN
@@
 $EndComp
 $Comp
-L GND #PWR0237
+L GND #PWR0236
 U 1 1 58C0DFC6
 P 8950 5300
-F 0 "#PWR0237" H 8950 5050 50  0001 C CNN
+F 0 "#PWR0236" H 8950 5050 50  0001 C CNN
 F 1 "GND" H 8950 5150 50  0000 C CNN
 F 2 "" H 8950 5300 50  0000 C CNN
@@
 $EndComp
 $Comp
-L GND #PWR0238
+L GND #PWR0237
 U 1 1 58C0DFDA
 P 8950 6150
-F 0 "#PWR0238" H 8950 5900 50  0001 C CNN
+F 0 "#PWR0237" H 8950 5900 50  0001 C CNN
 F 1 "GND" H 8950 6000 50  0000 C CNN
 F 2 "" H 8950 6150 50  0000 C CNN
@@
 $EndComp
 $Comp
-L TMC2130 U23
+L TMC2130 U22
 U 1 1 58C0DFE7
 P 8100 4800
-F 0 "U23" H 7650 6300 60  0000 C CNN
+F 0 "U22" H 7650 6300 60  0000 C CNN
 F 1 "TMC2130" H 8400 6300 60  0000 C CNN
 F 2 "" H 8100 5100 60  0001 C CNN
@@
 	8800 4700 9100 4700
 $Comp
-L VDD_3V3B #PWR0239
+L VDD_3V3B #PWR0238
 U 1 1 5A315EF4
 P 6450 3550
-F 0 "#PWR0239" H 6450 3400 50  0001 C CNN
+F 0 "#PWR0238" H 6450 3400 50  0001 C CNN
 F 1 "VDD_3V3B" H 6465 3723 50  0000 C CNN
 F 2 "" H 6450 3550 50  0000 C CNN

Commit message: Use fixed 5V LM2592HV Buck, include SPI0 header for LCD
Parts:
- renumbered C149 to C146, C150 to C147, C151 to C148, C152 to C149, C153 to C150, C154 to C151, C155 to C152, C156 to C153, C157 to C154, C158 to C155, C159 to C156, C160 to C157, C161 to C158, C162 to C159, C163 to C160, C164 to C161, R163 to R160, R164 to R161, R165 to R162, R166 to R163, R167 to R164, R168 to R165
Changed lines of the file:
@@
 Z2_SG
 $Comp
-L C C151
+L C C148
 U 1 1 58C0DF15
 P 7200 3200
-F 0 "C151" H 7086 3154 50  0000 R CNN
+F 0 "C148" H 7086 3154 50  0000 R CNN
 F 1 "100nF" H 7086 3245 50  0000 R CNN
 F 2 "Capacitors_SMD:C_0603" H 7238 3050 50  0001 C CNN
@@
 $EndComp
 $Comp
-L C C156
+L C C153
 U 1 1 58C0DF1C
 P 9000 3750
-F 0 "C156" V 8950 3650 50  0000 C CNN
+F 0 "C153" V 8950 3650 50  0000 C CNN
 F 1 "100nF" V 8950 3925 50  0000 C CNN
 F 2 "Capacitors_SMD:C_0603" H 9038 3600 50  0001 C CNN
@@
 $EndComp
 $Comp
-L CP1 C163
+L CP1 C160
 U 1 1 58C0DF23
 P 10350 3200
-F 0 "C163" H 10450 3300 50  0000 C CNN
+F 0 "C160" H 10450 3300 50  0000 C CNN
 F 1 "100μF" H 10500 3100 50  0000 C CNN
 F 2 "Capacitors_SMD:c_elec_8x10" H 10350 3200 50  0001 C CNN
@@
 $EndComp
 $Comp
-L C C159
+L C C156
 U 1 1 58C0DF2A
 P 9450 3200
-F 0 "C159" H 9350 3300 50  0000 C CNN
+F 0 "C156" H 9350 3300 50  0000 C CNN
 F 1 "100nF" H 9325 3100 50  0000 C CNN
 F 2 "Capacitors_SMD:C_0603" H 9488 3050 50  0001 C CNN
@@
 $EndComp
 $Comp
-L GND #PWR0231
+L GND #PWR0226
 U 1 1 58C0DF31
 P 7200 3400
-F 0 "#PWR0231" H 7200 3150 50  0001 C CNN
+F 0 "#PWR0226" H 7200 3150 50  0001 C CNN
 F 1 "GND" H 7200 3250 50  0000 C CNN
 F 2 "" H 7200 3400 50  0000 C CNN
@@
 $EndComp
 $Comp
-L C C160
+L C C157
 U 1 1 58C0DF37
 P 9750 3200
-F 0 "C160" H 9650 3300 50  0000 C CNN
+F 0 "C157" H 9650 3300 50  0000 C CNN
 F 1 "100nF" H 9625 3100 50  0000 C CNN
 F 2 "Capacitors_SMD:C_0603" H 9788 3050 50  0001 C CNN
@@
 $EndComp
 $Comp
-L GND #PWR0232
+L GND #PWR0227
 U 1 1 58C0DF3E
 P 10050 3450
-F 0 "#PWR0232" H 10050 3200 50  0001 C CNN
+F 0 "#PWR0227" H 10050 3200 50  0001 C CNN
 F 1 "GND" H 10055 3277 50  0000 C CNN
 F 2 "" H 10050 3450 50  0000 C CNN
@@
 $EndComp
 $Comp
-L +24V #PWR0233
+L +24V #PWR0228
 U 1 1 58C0DF44
 P 8250 2950
-F 0 "#PWR0233" H 8250 2800 50  0001 C CNN
+F 0 "#PWR0228" H 8250 2800 50  0001 C CNN
 F 1 "+24V" H 8265 3123 50  0000 C CNN
 F 2 "" H 8250 2950 50  0000 C CNN
@@
 $EndComp
 $Comp
-L C C153
+L C C150
 U 1 1 58C0DF4A
 P 8850 4250
-F 0 "C153" H 8965 4296 50  0000 L CNN
+F 0 "C150" H 8965 4296 50  0000 L CNN
 F 1 "22nF" H 8965 4205 50  0000 L CNN
 F 2 "Capacitors_SMD:C_0402" H 8888 4100 50  0001 C CNN
@@
 $EndComp
 $Comp
-L R R168
+L R R165
 U 1 1 58C0DF51
 P 10450 6800
-F 0 "R168" H 10400 6750 50  0000 R CNN
+F 0 "R165" H 10400 6750 50  0000 R CNN
 F 1 "220mΩ" H 10400 6850 50  0000 R CNN
 F 2 "" V 10380 6800 50  0001 C CNN
@@
 $EndComp
 $Comp
-L R R167
+L R R164
 U 1 1 58C0DF58
 P 9650 6800
-F 0 "R167" H 9600 6750 50  0000 R CNN
+F 0 "R164" H 9600 6750 50  0000 R CNN
 F 1 "220mΩ" H 9600 6850 50  0000 R CNN
 F 2 "" V 9580 6800 50  0001 C CNN
@@
 $EndComp
 $Comp
-L GND #PWR0234
+L GND #PWR0229
 U 1 1 58C0DF5F
 P 9350 7150
-F 0 "#PWR0234" H 9350 6900 50  0001 C CNN
+F 0 "#PWR0229" H 9350 6900 50  0001 C CNN
 F 1 "GND" H 9355 6977 50  0000 C CNN
 F 2 "" H 9350 7150 50  0000 C CNN
@@
 NoConn ~ 7400 5700
 $Comp
-L R R164
+L R R161
 U 1 1 58C0DF66
 P 7000 3850
-F 0 "R164" V 6900 3850 50  0000 C CNN
+F 0 "R161" V 6900 3850 50  0000 C CNN
 F 1 "2.2Ω" V 7000 3850 50  0000 C CNN
 F 2 "" V 6930 3850 50  0001 C CNN
@@
 $EndComp
 $Comp
-L C C150
+L C C147
 U 1 1 58C0DF6D
 P 6800 4050
-F 0 "C150" H 6850 4150 50  0000 L CNN
+F 0 "C147" H 6850 4150 50  0000 L CNN
 F 1 "470nF" H 6825 3950 50  0000 L CNN
 F 2 "Capacitors_SMD:C_0603" H 6838 3900 50  0001 C CNN
@@
 NoConn ~ 7400 5800
 $Comp
-L GND #PWR0235
+L GND #PWR0230
 U 1 1 58C0DF82
 P 7350 6200
-F 0 "#PWR0235" H 7350 5950 50  0001 C CNN
+F 0 "#PWR0230" H 7350 5950 50  0001 C CNN
 F 1 "GND" H 7355 6027 50  0000 C CNN
 F 2 "" H 7350 6200 50  0000 C CNN
@@
 $EndComp
 $Comp
-L C C161
+L C C158
 U 1 1 58C0DF88
 P 9800 6800
-F 0 "C161" H 9850 6900 50  0000 L CNN
+F 0 "C158" H 9850 6900 50  0000 L CNN
 F 1 "100nF" H 9850 6700 50  0000 L CNN
 F 2 "Capacitors_SMD:C_0603" H 9838 6650 50  0001 C CNN
@@
 NoConn ~ 7400 4650
 $Comp
-L C C152
+L C C149
 U 1 1 58C0DF9A
 P 7200 4050
-F 0 "C152" H 7250 4150 50  0000 L CNN
+F 0 "C149" H 7250 4150 50  0000 L CNN
 F 1 "4.7μF" H 7250 3950 50  0000 L CNN
 F 2 "Capacitors_SMD:C_0402" H 7238 3900 50  0001 C CNN
@@
 5VOUT
 $Comp
-L R R165
+L R R162
 U 1 1 58C0DFA2
 P 8950 6800
-F 0 "R165" H 9019 6846 50  0000 L CNN
+F 0 "R162" H 9019 6846 50  0000 L CNN
 F 1 "5.23kΩ" H 9019 6755 50  0000 L CNN
 F 2 "" V 8880 6800 50  0001 C CNN
@@
 5VOUT
 $Comp
-L R R166
+L R R163
 U 1 1 58C0DFAA
 P 9150 7000
-F 0 "R166" V 8950 7000 50  0000 C CNN
+F 0 "R163" V 8950 7000 50  0000 C CNN
 F 1 "4.75kΩ" V 9050 7000 50  0000 C CNN
 F 2 "" V 9080 7000 50  0001 C CNN
@@
 $EndComp
 $Comp
-L R R163
+L R R160
 U 1 1 58C0DFB1
 P 6100 4350
-F 0 "R163" H 6169 4396 50  0000 L CNN
+F 0 "R160" H 6169 4396 50  0000 L CNN
 F 1 "4.7kΩ" H 6169 4305 50  0000 L CNN
 F 2 "" V 6030 4350 50  0001 C CNN
@@
 $EndComp
 $Comp
-L C C164
+L C C161
 U 1 1 58C0DFB8
 P 10600 6800
-F 0 "C164" H 10650 6900 50  0000 L CNN
+F 0 "C161" H 10650 6900 50  0000 L CNN
 F 1 "100nF" H 10650 6700 50  0000 L CNN
 F 2 "Capacitors_SMD:C_0603" H 10638 6650 50  0001 C CNN
@@
 $EndComp
 $Comp
-L C C154
+L C C151
 U 1 1 58C0DFBF
 P 8850 5050
-F 0 "C154" H 8875 5150 50  0000 L CNN
+F 0 "C151" H 8875 5150 50  0000 L CNN
 F 1 "470pF" H 8850 4950 50  0000 L CNN
 F 2 "Capacitors_SMD:C_0603" H 8888 4900 50  0001 C CNN
@@
 $EndComp
 $Comp
-L GND #PWR0236
+L GND #PWR0231
 U 1 1 58C0DFC6
 P 8950 5300
-F 0 "#PWR0236" H 8950 5050 50  0001 C CNN
+F 0 "#PWR0231" H 8950 5050 50  0001 C CNN
 F 1 "GND" H 8950 5150 50  0000 C CNN
 F 2 "" H 8950 5300 50  0000 C CNN
@@
 $EndComp
 $Comp
-L C C157
+L C C154
 U 1 1 58C0DFCC
 P 9050 5050
-F 0 "C157" H 9075 5150 50  0000 L CNN
+F 0 "C154" H 9075 5150 50  0000 L CNN
 F 1 "470pF" H 9075 4950 50  0000 L CNN
 F 2 "Capacitors_SMD:C_0603" H 9088 4900 50  0001 C CNN
@@
 $EndComp
 $Comp
-L C C155
+L C C152
 U 1 1 58C0DFD3
 P 8850 5900
-F 0 "C155" H 8875 6000 50  0000 L CNN
+F 0 "C152" H 8875 6000 50  0000 L CNN
 F 1 "470pF" H 8850 5800 50  0000 L CNN
 F 2 "Capacitors_SMD:C_0603" H 8888 5750 50  0001 C CNN
@@
 $EndComp
 $Comp
-L GND #PWR0237
+L GND #PWR0232
 U 1 1 58C0DFDA
 P 8950 6150
-F 0 "#PWR0237" H 8950 5900 50  0001 C CNN
+F 0 "#PWR0232" H 8950 5900 50  0001 C CNN
 F 1 "GND" H 8950 6000 50  0000 C CNN
 F 2 "" H 8950 6150 50  0000 C CNN
@@
 $EndComp
 $Comp
-L C C158
+L C C155
 U 1 1 58C0DFE0
 P 9050 5900
-F 0 "C158" H 9075 6000 50  0000 L CNN
+F 0 "C155" H 9075 6000 50  0000 L CNN
 F 1 "470pF" H 9075 5800 50  0000 L CNN
 F 2 "Capacitors_SMD:C_0603" H 9088 5750 50  0001 C CNN
@@
 	8850 6100 8850 6050
 $Comp
-L C C162
+L C C159
 U 1 1 58C0E066
 P 10050 3200
-F 0 "C162" H 9950 3300 50  0000 C CNN
+F 0 "C159" H 9950 3300 50  0000 C CNN
 F 1 "10μF" H 9925 3100 50  0000 C CNN
 F 2 "Capacitors_SMD:C_0805" H 10088 3050 50  0001 C CNN
@@
 	8800 4700 9100 4700
 $Comp
-L VDD_3V3B #PWR0238
+L VDD_3V3B #PWR0233
 U 1 1 5A315EF4
 P 6450 3550
-F 0 "#PWR0238" H 6450 3400 50  0001 C CNN
+F 0 "#PWR0233" H 6450 3400 50  0001 C CNN
 F 1 "VDD_3V3B" H 6465 3723 50  0000 C CNN
 F 2 "" H 6450 3550 50  0000 C CNN
@@
 $EndComp
 $Comp
-L C C149
+L C C146
 U 1 1 5A89C77B
 P 6450 4050
-F 0 "C149" H 6500 4150 50  0000 L CNN
+F 0 "C146" H 6500 4150 50  0000 L CNN
 F 1 "100nF" H 6475 3950 50  0000 L CNN
 F 2 "Capacitors_SMD:C_0603" H 6488 3900 50  0001 C CNN
