File: KiMBo/z2_stepper.sch (KiCad schematic (older format))
At the start: 23 parts, among them U22 TMC2130

Commit message: Assocate more footprints
Parts:
- C149, C150: footprint Capacitors_SMD:C_0402 -> Capacitors_SMD:C_0603
- R160, R161, R162, R163: footprint (none) -> Resistors_SMD:R_0603
Changed lines of the file:
@@
 F 0 "C150" H 8965 4296 50  0000 L CNN
 F 1 "22nF" H 8965 4205 50  0000 L CNN
-F 2 "Capacitors_SMD:C_0402" H 8888 4100 50  0001 C CNN
+F 2 "Capacitors_SMD:C_0603" H 8888 4100 50  0001 C CNN
 F 3 "" H 8850 4250 50  0000 C CNN
 	1    8850 4250
@@
 F 0 "R161" V 6900 3850 50  0000 C CNN
 F 1 "2.2Ω" V 7000 3850 50  0000 C CNN
-F 2 "" V 6930 3850 50  0001 C CNN
+F 2 "Resistors_SMD:R_0603" V 6930 3850 50  0001 C CNN
 F 3 "" H 7000 3850 50  0000 C CNN
 	1    7000 3850
@@
 F 0 "C149" H 7250 4150 50  0000 L CNN
 F 1 "4.7μF" H 7250 3950 50  0000 L CNN
-F 2 "Capacitors_SMD:C_0402" H 7238 3900 50  0001 C CNN
+F 2 "Capacitors_SMD:C_0603" H 7238 3900 50  0001 C CNN
 F 3 "" H 7200 4050 50  0000 C CNN
 	1    7200 4050
@@
 F 0 "R162" H 9019 6846 50  0000 L CNN
 F 1 "5.23kΩ" H 9019 6755 50  0000 L CNN
-F 2 "" V 8880 6800 50  0001 C CNN
+F 2 "Resistors_SMD:R_0603" V 8880 6800 50  0001 C CNN
 F 3 "" H 8950 6800 50  0000 C CNN
 	1    8950 6800
@@
 F 0 "R163" V 8950 7000 50  0000 C CNN
 F 1 "4.75kΩ" V 9050 7000 50  0000 C CNN
-F 2 "" V 9080 7000 50  0001 C CNN
+F 2 "Resistors_SMD:R_0603" V 9080 7000 50  0001 C CNN
 F 3 "" H 9150 7000 50  0000 C CNN
 	1    9150 7000
@@
 F 0 "R160" H 6169 4396 50  0000 L CNN
 F 1 "4.7kΩ" H 6169 4305 50  0000 L CNN
-F 2 "" V 6030 4350 50  0001 C CNN
+F 2 "Resistors_SMD:R_0603" V 6030 4350 50  0001 C CNN
 F 3 "" H 6100 4350 50  0000 C CNN
 	1    6100 4350

Commit message: More footprint association
Parts:
- R164, R165: footprint (none) -> Resistors_SMD:R_0805
- U22: footprint (none) -> KiMBo:QFN36_5X6
Changed lines of the file:
@@
 $EndComp
 $Comp
-L GND #PWR0226
+L GND #PWR0227
 U 1 1 58C0DF31
 P 7200 3400
-F 0 "#PWR0226" H 7200 3150 50  0001 C CNN
+F 0 "#PWR0227" H 7200 3150 50  0001 C CNN
 F 1 "GND" H 7200 3250 50  0000 C CNN
 F 2 "" H 7200 3400 50  0000 C CNN
@@
 $EndComp
 $Comp
-L GND #PWR0227
+L GND #PWR0228
 U 1 1 58C0DF3E
 P 10050 3450
-F 0 "#PWR0227" H 10050 3200 50  0001 C CNN
+F 0 "#PWR0228" H 10050 3200 50  0001 C CNN
 F 1 "GND" H 10055 3277 50  0000 C CNN
 F 2 "" H 10050 3450 50  0000 C CNN
@@
 $EndComp
 $Comp
-L +24V #PWR0228
+L +24V #PWR0229
 U 1 1 58C0DF44
 P 8250 2950
-F 0 "#PWR0228" H 8250 2800 50  0001 C CNN
+F 0 "#PWR0229" H 8250 2800 50  0001 C CNN
 F 1 "+24V" H 8265 3123 50  0000 C CNN
 F 2 "" H 8250 2950 50  0000 C CNN
@@
 F 0 "R165" H 10400 6750 50  0000 R CNN
 F 1 "220mΩ" H 10400 6850 50  0000 R CNN
-F 2 "" V 10380 6800 50  0001 C CNN
+F 2 "Resistors_SMD:R_0805" V 10380 6800 50  0001 C CNN
 F 3 "" H 10450 6800 50  0000 C CNN
 	1    10450 6800
@@
 F 0 "R164" H 9600 6750 50  0000 R CNN
 F 1 "220mΩ" H 9600 6850 50  0000 R CNN
-F 2 "" V 9580 6800 50  0001 C CNN
+F 2 "Resistors_SMD:R_0805" V 9580 6800 50  0001 C CNN
 F 3 "" H 9650 6800 50  0000 C CNN
 	1    9650 6800
@@
 $EndComp
 $Comp
-L GND #PWR0229
+L GND #PWR0230
 U 1 1 58C0DF5F
 P 9350 7150
-F 0 "#PWR0229" H 9350 6900 50  0001 C CNN
+F 0 "#PWR0230" H 9350 6900 50  0001 C CNN
 F 1 "GND" H 9355 6977 50  0000 C CNN
 F 2 "" H 9350 7150 50  0000 C CNN
@@
 NoConn ~ 7400 5800
 $Comp
-L GND #PWR0230
+L GND #PWR0231
 U 1 1 58C0DF82
 P 7350 6200
-F 0 "#PWR0230" H 7350 5950 50  0001 C CNN
+F 0 "#PWR0231" H 7350 5950 50  0001 C CNN
 F 1 "GND" H 7355 6027 50  0000 C CNN
 F 2 "" H 7350 6200 50  0000 C CNN
@@
 $EndComp
 $Comp
-L GND #PWR0231
+L GND #PWR0232
 U 1 1 58C0DFC6
 P 8950 5300
-F 0 "#PWR0231" H 8950 5050 50  0001 C CNN
+F 0 "#PWR0232" H 8950 5050 50  0001 C CNN
 F 1 "GND" H 8950 5150 50  0000 C CNN
 F 2 "" H 8950 5300 50  0000 C CNN
@@
 $EndComp
 $Comp
-L GND #PWR0232
+L GND #PWR0233
 U 1 1 58C0DFDA
 P 8950 6150
-F 0 "#PWR0232" H 8950 5900 50  0001 C CNN
+F 0 "#PWR0233" H 8950 5900 50  0001 C CNN
 F 1 "GND" H 8950 6000 50  0000 C CNN
 F 2 "" H 8950 6150 50  0000 C CNN
@@
 F 0 "U22" H 7650 6300 60  0000 C CNN
 F 1 "TMC2130" H 8400 6300 60  0000 C CNN
-F 2 "" H 8100 5100 60  0001 C CNN
+F 2 "KiMBo:QFN36_5X6" H 8100 5100 60  0001 C CNN
 F 3 "" H 8100 5100 60  0000 C CNN
 	1    8100 4800
@@
 	8800 4700 9100 4700
 $Comp
-L VDD_3V3B #PWR0233
+L VDD_3V3B #PWR0234
 U 1 1 5A315EF4
 P 6450 3550
-F 0 "#PWR0233" H 6450 3400 50  0001 C CNN
+F 0 "#PWR0234" H 6450 3400 50  0001 C CNN
 F 1 "VDD_3V3B" H 6465 3723 50  0000 C CNN
 F 2 "" H 6450 3550 50  0000 C CNN

Commit message: Add more footprints and more associations, one association left!
Parts:
- R172: renamed from R163; footprint Resistors_SMD:R_0603 -> Resistors_SMD:R_0805
- R174: renamed from R165; footprint Resistors_SMD:R_0805 -> Resistors_SMD:R_0603
- renumbered R160 to R169, R161 to R170, R162 to R171, R164 to R173
Changed lines of the file:
@@
 $EndComp
 $Comp
-L GND #PWR0227
+L GND #PWR0229
 U 1 1 58C0DF31
 P 7200 3400
-F 0 "#PWR0227" H 7200 3150 50  0001 C CNN
+F 0 "#PWR0229" H 7200 3150 50  0001 C CNN
 F 1 "GND" H 7200 3250 50  0000 C CNN
 F 2 "" H 7200 3400 50  0000 C CNN
@@
 $EndComp
 $Comp
-L GND #PWR0228
+L GND #PWR0230
 U 1 1 58C0DF3E
 P 10050 3450
-F 0 "#PWR0228" H 10050 3200 50  0001 C CNN
+F 0 "#PWR0230" H 10050 3200 50  0001 C CNN
 F 1 "GND" H 10055 3277 50  0000 C CNN
 F 2 "" H 10050 3450 50  0000 C CNN
@@
 $EndComp
 $Comp
-L +24V #PWR0229
+L +24V #PWR0231
 U 1 1 58C0DF44
 P 8250 2950
-F 0 "#PWR0229" H 8250 2800 50  0001 C CNN
+F 0 "#PWR0231" H 8250 2800 50  0001 C CNN
 F 1 "+24V" H 8265 3123 50  0000 C CNN
 F 2 "" H 8250 2950 50  0000 C CNN
@@
 $EndComp
 $Comp
-L R R165
+L R R174
 U 1 1 58C0DF51
 P 10450 6800
-F 0 "R165" H 10400 6750 50  0000 R CNN
+F 0 "R174" H 10400 6750 50  0000 R CNN
 F 1 "220mΩ" H 10400 6850 50  0000 R CNN
-F 2 "Resistors_SMD:R_0805" V 10380 6800 50  0001 C CNN
+F 2 "Resistors_SMD:R_0603" V 10380 6800 50  0001 C CNN
 F 3 "" H 10450 6800 50  0000 C CNN
 	1    10450 6800
@@
 $EndComp
 $Comp
-L R R164
+L R R173
 U 1 1 58C0DF58
 P 9650 6800
-F 0 "R164" H 9600 6750 50  0000 R CNN
+F 0 "R173" H 9600 6750 50  0000 R CNN
 F 1 "220mΩ" H 9600 6850 50  0000 R CNN
 F 2 "Resistors_SMD:R_0805" V 9580 6800 50  0001 C CNN
@@
 $EndComp
 $Comp
-L GND #PWR0230
+L GND #PWR0232
 U 1 1 58C0DF5F
 P 9350 7150
-F 0 "#PWR0230" H 9350 6900 50  0001 C CNN
+F 0 "#PWR0232" H 9350 6900 50  0001 C CNN
 F 1 "GND" H 9355 6977 50  0000 C CNN
 F 2 "" H 9350 7150 50  0000 C CNN
@@
 NoConn ~ 7400 5700
 $Comp
-L R R161
+L R R170
 U 1 1 58C0DF66
 P 7000 3850
-F 0 "R161" V 6900 3850 50  0000 C CNN
+F 0 "R170" V 6900 3850 50  0000 C CNN
 F 1 "2.2Ω" V 7000 3850 50  0000 C CNN
 F 2 "Resistors_SMD:R_0603" V 6930 3850 50  0001 C CNN
@@
 NoConn ~ 7400 5800
 $Comp
-L GND #PWR0231
+L GND #PWR0233
 U 1 1 58C0DF82
 P 7350 6200
-F 0 "#PWR0231" H 7350 5950 50  0001 C CNN
+F 0 "#PWR0233" H 7350 5950 50  0001 C CNN
 F 1 "GND" H 7355 6027 50  0000 C CNN
 F 2 "" H 7350 6200 50  0000 C CNN
@@
 5VOUT
 $Comp
-L R R162
+L R R171
 U 1 1 58C0DFA2
 P 8950 6800
-F 0 "R162" H 9019 6846 50  0000 L CNN
+F 0 "R171" H 9019 6846 50  0000 L CNN
 F 1 "5.23kΩ" H 9019 6755 50  0000 L CNN
 F 2 "Resistors_SMD:R_0603" V 8880 6800 50  0001 C CNN
@@
 5VOUT
 $Comp
-L R R163
+L R R172
 U 1 1 58C0DFAA
 P 9150 7000
-F 0 "R163" V 8950 7000 50  0000 C CNN
+F 0 "R172" V 8950 7000 50  0000 C CNN
 F 1 "4.75kΩ" V 9050 7000 50  0000 C CNN
-F 2 "Resistors_SMD:R_0603" V 9080 7000 50  0001 C CNN
+F 2 "Resistors_SMD:R_0805" V 9080 7000 50  0001 C CNN
 F 3 "" H 9150 7000 50  0000 C CNN
 	1    9150 7000
@@
 $EndComp
 $Comp
-L R R160
+L R R169
 U 1 1 58C0DFB1
 P 6100 4350
-F 0 "R160" H 6169 4396 50  0000 L CNN
+F 0 "R169" H 6169 4396 50  0000 L CNN
 F 1 "4.7kΩ" H 6169 4305 50  0000 L CNN
 F 2 "Resistors_SMD:R_0603" V 6030 4350 50  0001 C CNN
@@
 $EndComp
 $Comp
-L GND #PWR0232
+L GND #PWR0234
 U 1 1 58C0DFC6
 P 8950 5300
-F 0 "#PWR0232" H 8950 5050 50  0001 C CNN
+F 0 "#PWR0234" H 8950 5050 50  0001 C CNN
 F 1 "GND" H 8950 5150 50  0000 C CNN
 F 2 "" H 8950 5300 50  0000 C CNN
@@
 $EndComp
 $Comp
-L GND #PWR0233
+L GND #PWR0235
 U 1 1 58C0DFDA
 P 8950 6150
-F 0 "#PWR0233" H 8950 5900 50  0001 C CNN
+F 0 "#PWR0235" H 8950 5900 50  0001 C CNN
 F 1 "GND" H 8950 6000 50  0000 C CNN
 F 2 "" H 8950 6150 50  0000 C CNN
@@
 	8800 4700 9100 4700
 $Comp
-L VDD_3V3B #PWR0234
+L VDD_3V3B #PWR0236
 U 1 1 5A315EF4
 P 6450 3550
-F 0 "#PWR0234" H 6450 3400 50  0001 C CNN
+F 0 "#PWR0236" H 6450 3400 50  0001 C CNN
 F 1 "VDD_3V3B" H 6465 3723 50  0000 C CNN
 F 2 "" H 6450 3550 50  0000 C CNN

Commit message: Begin layout
Arrange all connectors to get a feel for the area.
Parts:
- renumbered C146 to C148, C147 to C149, C148 to C150, C149 to C151, C150 to C152, C151 to C153, C152 to C154, C153 to C155, C154 to C156, C155 to C157, C156 to C158, C157 to C159, C158 to C160, C159 to C161, C160 to C162, C161 to C163
Changed lines of the file:
@@
 Z2_SG
 $Comp
-L C C148
+L C C150
 U 1 1 58C0DF15
 P 7200 3200
-F 0 "C148" H 7086 3154 50  0000 R CNN
+F 0 "C150" H 7086 3154 50  0000 R CNN
 F 1 "100nF" H 7086 3245 50  0000 R CNN
 F 2 "Capacitors_SMD:C_0603" H 7238 3050 50  0001 C CNN
@@
 $EndComp
 $Comp
-L C C153
+L C C155
 U 1 1 58C0DF1C
 P 9000 3750
-F 0 "C153" V 8950 3650 50  0000 C CNN
+F 0 "C155" V 8950 3650 50  0000 C CNN
 F 1 "100nF" V 8950 3925 50  0000 C CNN
 F 2 "Capacitors_SMD:C_0603" H 9038 3600 50  0001 C CNN
@@
 $EndComp
 $Comp
-L CP1 C160
+L CP1 C162
 U 1 1 58C0DF23
 P 10350 3200
-F 0 "C160" H 10450 3300 50  0000 C CNN
+F 0 "C162" H 10450 3300 50  0000 C CNN
 F 1 "100μF" H 10500 3100 50  0000 C CNN
 F 2 "Capacitors_SMD:c_elec_8x10" H 10350 3200 50  0001 C CNN
@@
 $EndComp
 $Comp
-L C C156
+L C C158
 U 1 1 58C0DF2A
 P 9450 3200
-F 0 "C156" H 9350 3300 50  0000 C CNN
+F 0 "C158" H 9350 3300 50  0000 C CNN
 F 1 "100nF" H 9325 3100 50  0000 C CNN
 F 2 "Capacitors_SMD:C_0603" H 9488 3050 50  0001 C CNN
@@
 $EndComp
 $Comp
-L GND #PWR0229
+L GND #PWR0232
 U 1 1 58C0DF31
 P 7200 3400
-F 0 "#PWR0229" H 7200 3150 50  0001 C CNN
+F 0 "#PWR0232" H 7200 3150 50  0001 C CNN
 F 1 "GND" H 7200 3250 50  0000 C CNN
 F 2 "" H 7200 3400 50  0000 C CNN
@@
 $EndComp
 $Comp
-L C C157
+L C C159
 U 1 1 58C0DF37
 P 9750 3200
-F 0 "C157" H 9650 3300 50  0000 C CNN
+F 0 "C159" H 9650 3300 50  0000 C CNN
 F 1 "100nF" H 9625 3100 50  0000 C CNN
 F 2 "Capacitors_SMD:C_0603" H 9788 3050 50  0001 C CNN
@@
 $EndComp
 $Comp
-L GND #PWR0230
+L GND #PWR0233
 U 1 1 58C0DF3E
 P 10050 3450
-F 0 "#PWR0230" H 10050 3200 50  0001 C CNN
+F 0 "#PWR0233" H 10050 3200 50  0001 C CNN
 F 1 "GND" H 10055 3277 50  0000 C CNN
 F 2 "" H 10050 3450 50  0000 C CNN
@@
 $EndComp
 $Comp
-L +24V #PWR0231
+L +24V #PWR0234
 U 1 1 58C0DF44
 P 8250 2950
-F 0 "#PWR0231" H 8250 2800 50  0001 C CNN
+F 0 "#PWR0234" H 8250 2800 50  0001 C CNN
 F 1 "+24V" H 8265 3123 50  0000 C CNN
 F 2 "" H 8250 2950 50  0000 C CNN
@@
 $EndComp
 $Comp
-L C C150
+L C C152
 U 1 1 58C0DF4A
 P 8850 4250
-F 0 "C150" H 8965 4296 50  0000 L CNN
+F 0 "C152" H 8965 4296 50  0000 L CNN
 F 1 "22nF" H 8965 4205 50  0000 L CNN
 F 2 "Capacitors_SMD:C_0603" H 8888 4100 50  0001 C CNN
@@
 $EndComp
 $Comp
-L GND #PWR0232
+L GND #PWR0235
 U 1 1 58C0DF5F
 P 9350 7150
-F 0 "#PWR0232" H 9350 6900 50  0001 C CNN
+F 0 "#PWR0235" H 9350 6900 50  0001 C CNN
 F 1 "GND" H 9355 6977 50  0000 C CNN
 F 2 "" H 9350 7150 50  0000 C CNN
@@
 $EndComp
 $Comp
-L C C147
+L C C149
 U 1 1 58C0DF6D
 P 6800 4050
-F 0 "C147" H 6850 4150 50  0000 L CNN
+F 0 "C149" H 6850 4150 50  0000 L CNN
 F 1 "470nF" H 6825 3950 50  0000 L CNN
 F 2 "Capacitors_SMD:C_0603" H 6838 3900 50  0001 C CNN
@@
 NoConn ~ 7400 5800
 $Comp
-L GND #PWR0233
+L GND #PWR0236
 U 1 1 58C0DF82
 P 7350 6200
-F 0 "#PWR0233" H 7350 5950 50  0001 C CNN
+F 0 "#PWR0236" H 7350 5950 50  0001 C CNN
 F 1 "GND" H 7355 6027 50  0000 C CNN
 F 2 "" H 7350 6200 50  0000 C CNN
@@
 $EndComp
 $Comp
-L C C158
+L C C160
 U 1 1 58C0DF88
 P 9800 6800
-F 0 "C158" H 9850 6900 50  0000 L CNN
+F 0 "C160" H 9850 6900 50  0000 L CNN
 F 1 "100nF" H 9850 6700 50  0000 L CNN
 F 2 "Capacitors_SMD:C_0603" H 9838 6650 50  0001 C CNN
@@
 NoConn ~ 7400 4650
 $Comp
-L C C149
+L C C151
 U 1 1 58C0DF9A
 P 7200 4050
-F 0 "C149" H 7250 4150 50  0000 L CNN
+F 0 "C151" H 7250 4150 50  0000 L CNN
 F 1 "4.7μF" H 7250 3950 50  0000 L CNN
 F 2 "Capacitors_SMD:C_0603" H 7238 3900 50  0001 C CNN
@@
 $EndComp
 $Comp
-L C C161
+L C C163
 U 1 1 58C0DFB8
 P 10600 6800
-F 0 "C161" H 10650 6900 50  0000 L CNN
+F 0 "C163" H 10650 6900 50  0000 L CNN
 F 1 "100nF" H 10650 6700 50  0000 L CNN
 F 2 "Capacitors_SMD:C_0603" H 10638 6650 50  0001 C CNN
@@
 $EndComp
 $Comp
-L C C151
+L C C153
 U 1 1 58C0DFBF
 P 8850 5050
-F 0 "C151" H 8875 5150 50  0000 L CNN
+F 0 "C153" H 8875 5150 50  0000 L CNN
 F 1 "470pF" H 8850 4950 50  0000 L CNN
 F 2 "Capacitors_SMD:C_0603" H 8888 4900 50  0001 C CNN
@@
 $EndComp
 $Comp
-L GND #PWR0234
+L GND #PWR0237
 U 1 1 58C0DFC6
 P 8950 5300
-F 0 "#PWR0234" H 8950 5050 50  0001 C CNN
+F 0 "#PWR0237" H 8950 5050 50  0001 C CNN
 F 1 "GND" H 8950 5150 50  0000 C CNN
 F 2 "" H 8950 5300 50  0000 C CNN
@@
 $EndComp
 $Comp
-L C C154
+L C C156
 U 1 1 58C0DFCC
 P 9050 5050
-F 0 "C154" H 9075 5150 50  0000 L CNN
+F 0 "C156" H 9075 5150 50  0000 L CNN
 F 1 "470pF" H 9075 4950 50  0000 L CNN
 F 2 "Capacitors_SMD:C_0603" H 9088 4900 50  0001 C CNN
@@
 $EndComp
 $Comp
-L C C152
+L C C154
 U 1 1 58C0DFD3
 P 8850 5900
-F 0 "C152" H 8875 6000 50  0000 L CNN
+F 0 "C154" H 8875 6000 50  0000 L CNN
 F 1 "470pF" H 8850 5800 50  0000 L CNN
 F 2 "Capacitors_SMD:C_0603" H 8888 5750 50  0001 C CNN
@@
 $EndComp
 $Comp
-L GND #PWR0235
+L GND #PWR0238
 U 1 1 58C0DFDA
 P 8950 6150
-F 0 "#PWR0235" H 8950 5900 50  0001 C CNN
+F 0 "#PWR0238" H 8950 5900 50  0001 C CNN
 F 1 "GND" H 8950 6000 50  0000 C CNN
 F 2 "" H 8950 6150 50  0000 C CNN
@@
 $EndComp
 $Comp
-L C C155
+L C C157
 U 1 1 58C0DFE0
 P 9050 5900
-F 0 "C155" H 9075 6000 50  0000 L CNN
+F 0 "C157" H 9075 6000 50  0000 L CNN
 F 1 "470pF" H 9075 5800 50  0000 L CNN
 F 2 "Capacitors_SMD:C_0603" H 9088 5750 50  0001 C CNN
@@
 	8850 6100 8850 6050
 $Comp
-L C C159
+L C C161
 U 1 1 58C0E066
 P 10050 3200
-F 0 "C159" H 9950 3300 50  0000 C CNN
+F 0 "C161" H 9950 3300 50  0000 C CNN
 F 1 "10μF" H 9925 3100 50  0000 C CNN
 F 2 "Capacitors_SMD:C_0805" H 10088 3050 50  0001 C CNN
@@
 	8800 4700 9100 4700
 $Comp
-L VDD_3V3B #PWR0236
+L VDD_3V3B #PWR0239
 U 1 1 5A315EF4
 P 6450 3550
-F 0 "#PWR0236" H 6450 3400 50  0001 C CNN
+F 0 "#PWR0239" H 6450 3400 50  0001 C CNN
 F 1 "VDD_3V3B" H 6465 3723 50  0000 C CNN
 F 2 "" H 6450 3550 50  0000 C CNN
@@
 $EndComp
 $Comp
-L C C146
+L C C148
 U 1 1 5A89C77B
 P 6450 4050
-F 0 "C146" H 6500 4150 50  0000 L CNN
+F 0 "C148" H 6500 4150 50  0000 L CNN
 F 1 "100nF" H 6475 3950 50  0000 L CNN
 F 2 "Capacitors_SMD:C_0603" H 6488 3900 50  0001 C CNN

Commit message: Arrange connectors and E-stepper circuit
Parts:
- R172: footprint Resistors_SMD:R_0805 -> Resistors_SMD:R_0603
- R174: footprint Resistors_SMD:R_0603 -> Resistors_SMD:R_0805
Changed lines of the file:
@@
 F 0 "R174" H 10400 6750 50  0000 R CNN
 F 1 "220mΩ" H 10400 6850 50  0000 R CNN
-F 2 "Resistors_SMD:R_0603" V 10380 6800 50  0001 C CNN
+F 2 "Resistors_SMD:R_0805" V 10380 6800 50  0001 C CNN
 F 3 "" H 10450 6800 50  0000 C CNN
 	1    10450 6800
@@
 F 0 "R172" V 8950 7000 50  0000 C CNN
 F 1 "4.75kΩ" V 9050 7000 50  0000 C CNN
-F 2 "Resistors_SMD:R_0805" V 9080 7000 50  0001 C CNN
+F 2 "Resistors_SMD:R_0603" V 9080 7000 50  0001 C CNN
 F 3 "" H 9150 7000 50  0000 C CNN
 	1    9150 7000

Commit message: Remove HDMI from the schematic
Parts:
- renumbered C148 to C123, C149 to C124, C150 to C125, C151 to C126, C152 to C127, C153 to C128, C154 to C129, C155 to C130, C156 to C131, C157 to C132, C158 to C133, C159 to C134, C160 to C135, C161 to C136, C162 to C137, C163 to C138, R169 to R142, R170 to R143, R171 to R144, R172 to R145, R173 to R146, R174 to R147, U22 to U18
Changed lines of the file:
@@
 $Descr A3 16535 11693
 encoding utf-8
-Sheet 20 26
+Sheet 20 25
 Title ""
 Date ""
@@
 Z2_SG
 $Comp
-L C C150
+L C C125
 U 1 1 58C0DF15
 P 7200 3200
-F 0 "C150" H 7086 3154 50  0000 R CNN
+F 0 "C125" H 7086 3154 50  0000 R CNN
 F 1 "100nF" H 7086 3245 50  0000 R CNN
 F 2 "Capacitors_SMD:C_0603" H 7238 3050 50  0001 C CNN
@@
 $EndComp
 $Comp
-L C C155
+L C C130
 U 1 1 58C0DF1C
 P 9000 3750
-F 0 "C155" V 8950 3650 50  0000 C CNN
+F 0 "C130" V 8950 3650 50  0000 C CNN
 F 1 "100nF" V 8950 3925 50  0000 C CNN
 F 2 "Capacitors_SMD:C_0603" H 9038 3600 50  0001 C CNN
@@
 $EndComp
 $Comp
-L CP1 C162
+L CP1 C137
 U 1 1 58C0DF23
 P 10350 3200
-F 0 "C162" H 10450 3300 50  0000 C CNN
+F 0 "C137" H 10450 3300 50  0000 C CNN
 F 1 "100μF" H 10500 3100 50  0000 C CNN
 F 2 "Capacitors_SMD:c_elec_8x10" H 10350 3200 50  0001 C CNN
@@
 $EndComp
 $Comp
-L C C158
+L C C133
 U 1 1 58C0DF2A
 P 9450 3200
-F 0 "C158" H 9350 3300 50  0000 C CNN
+F 0 "C133" H 9350 3300 50  0000 C CNN
 F 1 "100nF" H 9325 3100 50  0000 C CNN
 F 2 "Capacitors_SMD:C_0603" H 9488 3050 50  0001 C CNN
@@
 $EndComp
 $Comp
-L GND #PWR0232
+L GND #PWR0201
 U 1 1 58C0DF31
 P 7200 3400
-F 0 "#PWR0232" H 7200 3150 50  0001 C CNN
+F 0 "#PWR0201" H 7200 3150 50  0001 C CNN
 F 1 "GND" H 7200 3250 50  0000 C CNN
 F 2 "" H 7200 3400 50  0000 C CNN
@@
 $EndComp
 $Comp
-L C C159
+L C C134
 U 1 1 58C0DF37
 P 9750 3200
-F 0 "C159" H 9650 3300 50  0000 C CNN
+F 0 "C134" H 9650 3300 50  0000 C CNN
 F 1 "100nF" H 9625 3100 50  0000 C CNN
 F 2 "Capacitors_SMD:C_0603" H 9788 3050 50  0001 C CNN
@@
 $EndComp
 $Comp
-L GND #PWR0233
+L GND #PWR0202
 U 1 1 58C0DF3E
 P 10050 3450
-F 0 "#PWR0233" H 10050 3200 50  0001 C CNN
+F 0 "#PWR0202" H 10050 3200 50  0001 C CNN
 F 1 "GND" H 10055 3277 50  0000 C CNN
 F 2 "" H 10050 3450 50  0000 C CNN
@@
 $EndComp
 $Comp
-L +24V #PWR0234
+L +24V #PWR0203
 U 1 1 58C0DF44
 P 8250 2950
-F 0 "#PWR0234" H 8250 2800 50  0001 C CNN
+F 0 "#PWR0203" H 8250 2800 50  0001 C CNN
 F 1 "+24V" H 8265 3123 50  0000 C CNN
 F 2 "" H 8250 2950 50  0000 C CNN
@@
 $EndComp
 $Comp
-L C C152
+L C C127
 U 1 1 58C0DF4A
 P 8850 4250
-F 0 "C152" H 8965 4296 50  0000 L CNN
+F 0 "C127" H 8965 4296 50  0000 L CNN
 F 1 "22nF" H 8965 4205 50  0000 L CNN
 F 2 "Capacitors_SMD:C_0603" H 8888 4100 50  0001 C CNN
@@
 $EndComp
 $Comp
-L R R174
+L R R147
 U 1 1 58C0DF51
 P 10450 6800
-F 0 "R174" H 10400 6750 50  0000 R CNN
+F 0 "R147" H 10400 6750 50  0000 R CNN
 F 1 "220mΩ" H 10400 6850 50  0000 R CNN
 F 2 "Resistors_SMD:R_0805" V 10380 6800 50  0001 C CNN
@@
 $EndComp
 $Comp
-L R R173
+L R R146
 U 1 1 58C0DF58
 P 9650 6800
-F 0 "R173" H 9600 6750 50  0000 R CNN
+F 0 "R146" H 9600 6750 50  0000 R CNN
 F 1 "220mΩ" H 9600 6850 50  0000 R CNN
 F 2 "Resistors_SMD:R_0805" V 9580 6800 50  0001 C CNN
@@
 $EndComp
 $Comp
-L GND #PWR0235
+L GND #PWR0204
 U 1 1 58C0DF5F
 P 9350 7150
-F 0 "#PWR0235" H 9350 6900 50  0001 C CNN
+F 0 "#PWR0204" H 9350 6900 50  0001 C CNN
 F 1 "GND" H 9355 6977 50  0000 C CNN
 F 2 "" H 9350 7150 50  0000 C CNN
@@
 NoConn ~ 7400 5700
 $Comp
-L R R170
+L R R143
 U 1 1 58C0DF66
 P 7000 3850
-F 0 "R170" V 6900 3850 50  0000 C CNN
+F 0 "R143" V 6900 3850 50  0000 C CNN
 F 1 "2.2Ω" V 7000 3850 50  0000 C CNN
 F 2 "Resistors_SMD:R_0603" V 6930 3850 50  0001 C CNN
@@
 $EndComp
 $Comp
-L C C149
+L C C124
 U 1 1 58C0DF6D
 P 6800 4050
-F 0 "C149" H 6850 4150 50  0000 L CNN
+F 0 "C124" H 6850 4150 50  0000 L CNN
 F 1 "470nF" H 6825 3950 50  0000 L CNN
 F 2 "Capacitors_SMD:C_0603" H 6838 3900 50  0001 C CNN
@@
 NoConn ~ 7400 5800
 $Comp
-L GND #PWR0236
+L GND #PWR0205
 U 1 1 58C0DF82
 P 7350 6200
-F 0 "#PWR0236" H 7350 5950 50  0001 C CNN
+F 0 "#PWR0205" H 7350 5950 50  0001 C CNN
 F 1 "GND" H 7355 6027 50  0000 C CNN
 F 2 "" H 7350 6200 50  0000 C CNN
@@
 $EndComp
 $Comp
-L C C160
+L C C135
 U 1 1 58C0DF88
 P 9800 6800
-F 0 "C160" H 9850 6900 50  0000 L CNN
+F 0 "C135" H 9850 6900 50  0000 L CNN
 F 1 "100nF" H 9850 6700 50  0000 L CNN
 F 2 "Capacitors_SMD:C_0603" H 9838 6650 50  0001 C CNN
@@
 NoConn ~ 7400 4650
 $Comp
-L C C151
+L C C126
 U 1 1 58C0DF9A
 P 7200 4050
-F 0 "C151" H 7250 4150 50  0000 L CNN
+F 0 "C126" H 7250 4150 50  0000 L CNN
 F 1 "4.7μF" H 7250 3950 50  0000 L CNN
 F 2 "Capacitors_SMD:C_0603" H 7238 3900 50  0001 C CNN
@@
 5VOUT
 $Comp
-L R R171
+L R R144
 U 1 1 58C0DFA2
 P 8950 6800
-F 0 "R171" H 9019 6846 50  0000 L CNN
+F 0 "R144" H 9019 6846 50  0000 L CNN
 F 1 "5.23kΩ" H 9019 6755 50  0000 L CNN
 F 2 "Resistors_SMD:R_0603" V 8880 6800 50  0001 C CNN
@@
 5VOUT
 $Comp
-L R R172
+L R R145
 U 1 1 58C0DFAA
 P 9150 7000
-F 0 "R172" V 8950 7000 50  0000 C CNN
+F 0 "R145" V 8950 7000 50  0000 C CNN
 F 1 "4.75kΩ" V 9050 7000 50  0000 C CNN
 F 2 "Resistors_SMD:R_0603" V 9080 7000 50  0001 C CNN
@@
 $EndComp
 $Comp
-L R R169
+L R R142
 U 1 1 58C0DFB1
 P 6100 4350
-F 0 "R169" H 6169 4396 50  0000 L CNN
+F 0 "R142" H 6169 4396 50  0000 L CNN
 F 1 "4.7kΩ" H 6169 4305 50  0000 L CNN
 F 2 "Resistors_SMD:R_0603" V 6030 4350 50  0001 C CNN
@@
 $EndComp
 $Comp
-L C C163
+L C C138
 U 1 1 58C0DFB8
 P 10600 6800
-F 0 "C163" H 10650 6900 50  0000 L CNN
+F 0 "C138" H 10650 6900 50  0000 L CNN
 F 1 "100nF" H 10650 6700 50  0000 L CNN
 F 2 "Capacitors_SMD:C_0603" H 10638 6650 50  0001 C CNN
@@
 $EndComp
 $Comp
-L C C153
+L C C128
 U 1 1 58C0DFBF
 P 8850 5050
-F 0 "C153" H 8875 5150 50  0000 L CNN
+F 0 "C128" H 8875 5150 50  0000 L CNN
 F 1 "470pF" H 8850 4950 50  0000 L CNN
 F 2 "Capacitors_SMD:C_0603" H 8888 4900 50  0001 C CNN
@@
 $EndComp
 $Comp
-L GND #PWR0237
+L GND #PWR0206
 U 1 1 58C0DFC6
 P 8950 5300
-F 0 "#PWR0237" H 8950 5050 50  0001 C CNN
+F 0 "#PWR0206" H 8950 5050 50  0001 C CNN
 F 1 "GND" H 8950 5150 50  0000 C CNN
 F 2 "" H 8950 5300 50  0000 C CNN
@@
 $EndComp
 $Comp
-L C C156
+L C C131
 U 1 1 58C0DFCC
 P 9050 5050
-F 0 "C156" H 9075 5150 50  0000 L CNN
+F 0 "C131" H 9075 5150 50  0000 L CNN
 F 1 "470pF" H 9075 4950 50  0000 L CNN
 F 2 "Capacitors_SMD:C_0603" H 9088 4900 50  0001 C CNN
@@
 $EndComp
 $Comp
-L C C154
+L C C129
 U 1 1 58C0DFD3
 P 8850 5900
-F 0 "C154" H 8875 6000 50  0000 L CNN
+F 0 "C129" H 8875 6000 50  0000 L CNN
 F 1 "470pF" H 8850 5800 50  0000 L CNN
 F 2 "Capacitors_SMD:C_0603" H 8888 5750 50  0001 C CNN
@@
 $EndComp
 $Comp
-L GND #PWR0238
+L GND #PWR0207
 U 1 1 58C0DFDA
 P 8950 6150
-F 0 "#PWR0238" H 8950 5900 50  0001 C CNN
+F 0 "#PWR0207" H 8950 5900 50  0001 C CNN
 F 1 "GND" H 8950 6000 50  0000 C CNN
 F 2 "" H 8950 6150 50  0000 C CNN
@@
 $EndComp
 $Comp
-L C C157
+L C C132
 U 1 1 58C0DFE0
 P 9050 5900
-F 0 "C157" H 9075 6000 50  0000 L CNN
+F 0 "C132" H 9075 6000 50  0000 L CNN
 F 1 "470pF" H 9075 5800 50  0000 L CNN
 F 2 "Capacitors_SMD:C_0603" H 9088 5750 50  0001 C CNN
@@
 $EndComp
 $Comp
-L TMC2130 U22
+L TMC2130 U18
 U 1 1 58C0DFE7
 P 8100 4800
-F 0 "U22" H 7650 6300 60  0000 C CNN
+F 0 "U18" H 7650 6300 60  0000 C CNN
 F 1 "TMC2130" H 8400 6300 60  0000 C CNN
 F 2 "KiMBo:QFN36_5X6" H 8100 5100 60  0001 C CNN
@@
 	8850 6100 8850 6050
 $Comp
-L C C161
+L C C136
 U 1 1 58C0E066
 P 10050 3200
-F 0 "C161" H 9950 3300 50  0000 C CNN
+F 0 "C136" H 9950 3300 50  0000 C CNN
 F 1 "10μF" H 9925 3100 50  0000 C CNN
 F 2 "Capacitors_SMD:C_0805" H 10088 3050 50  0001 C CNN
@@
 	8800 4700 9100 4700
 $Comp
-L VDD_3V3B #PWR0239
+L VDD_3V3B #PWR0208
 U 1 1 5A315EF4
 P 6450 3550
-F 0 "#PWR0239" H 6450 3400 50  0001 C CNN
+F 0 "#PWR0208" H 6450 3400 50  0001 C CNN
 F 1 "VDD_3V3B" H 6465 3723 50  0000 C CNN
 F 2 "" H 6450 3550 50  0000 C CNN
@@
 $EndComp
 $Comp
-L C C148
+L C C123
 U 1 1 5A89C77B
 P 6450 4050
-F 0 "C148" H 6500 4150 50  0000 L CNN
+F 0 "C123" H 6500 4150 50  0000 L CNN
 F 1 "100nF" H 6475 3950 50  0000 L CNN
 F 2 "Capacitors_SMD:C_0603" H 6488 3900 50  0001 C CNN
