File: KiMBo/z2_stepper.sch (KiCad schematic (older format))
At the start: 23 parts, among them U18 TMC2130

Commit message: More stepper motor driver progress
Parts:
- renumbered R142 to R144, R143 to R145, R144 to R146, R145 to R147, R146 to R148, R147 to R149
Changed lines of the file:
@@
 $Descr A3 16535 11693
 encoding utf-8
-Sheet 20 25
+Sheet 18 25
 Title ""
 Date ""
@@
 $EndComp
 $Comp
-L R R147
+L R R149
 U 1 1 58C0DF51
 P 10450 6800
-F 0 "R147" H 10400 6750 50  0000 R CNN
+F 0 "R149" H 10400 6750 50  0000 R CNN
 F 1 "220mΩ" H 10400 6850 50  0000 R CNN
 F 2 "Resistors_SMD:R_0805" V 10380 6800 50  0001 C CNN
@@
 $EndComp
 $Comp
-L R R146
+L R R148
 U 1 1 58C0DF58
 P 9650 6800
-F 0 "R146" H 9600 6750 50  0000 R CNN
+F 0 "R148" H 9600 6750 50  0000 R CNN
 F 1 "220mΩ" H 9600 6850 50  0000 R CNN
 F 2 "Resistors_SMD:R_0805" V 9580 6800 50  0001 C CNN
@@
 NoConn ~ 7400 5700
 $Comp
-L R R143
+L R R145
 U 1 1 58C0DF66
 P 7000 3850
-F 0 "R143" V 6900 3850 50  0000 C CNN
+F 0 "R145" V 6900 3850 50  0000 C CNN
 F 1 "2.2Ω" V 7000 3850 50  0000 C CNN
 F 2 "Resistors_SMD:R_0603" V 6930 3850 50  0001 C CNN
@@
 5VOUT
 $Comp
-L R R144
+L R R146
 U 1 1 58C0DFA2
 P 8950 6800
-F 0 "R144" H 9019 6846 50  0000 L CNN
+F 0 "R146" H 9019 6846 50  0000 L CNN
 F 1 "5.23kΩ" H 9019 6755 50  0000 L CNN
 F 2 "Resistors_SMD:R_0603" V 8880 6800 50  0001 C CNN
@@
 5VOUT
 $Comp
-L R R145
+L R R147
 U 1 1 58C0DFAA
 P 9150 7000
-F 0 "R145" V 8950 7000 50  0000 C CNN
+F 0 "R147" V 8950 7000 50  0000 C CNN
 F 1 "4.75kΩ" V 9050 7000 50  0000 C CNN
 F 2 "Resistors_SMD:R_0603" V 9080 7000 50  0001 C CNN
@@
 $EndComp
 $Comp
-L R R142
+L R R144
 U 1 1 58C0DFB1
 P 6100 4350
-F 0 "R142" H 6169 4396 50  0000 L CNN
+F 0 "R144" H 6169 4396 50  0000 L CNN
 F 1 "4.7kΩ" H 6169 4305 50  0000 L CNN
 F 2 "Resistors_SMD:R_0603" V 6030 4350 50  0001 C CNN

Commit message: Daisy chain the SPI stepper motor driver interface, continue work on the E-heater layout
Parts:
- renumbered C123 to C121, C124 to C122, C125 to C123, C126 to C124, C127 to C125, C128 to C126, C129 to C127, C130 to C128, C131 to C129, C132 to C130, C133 to C131, C134 to C132, C135 to C133, C136 to C134, C137 to C135, C138 to C136, U18 to U17
Changed lines of the file:
@@
 Z2_SG
 $Comp
-L C C125
+L C C123
 U 1 1 58C0DF15
 P 7200 3200
-F 0 "C125" H 7086 3154 50  0000 R CNN
+F 0 "C123" H 7086 3154 50  0000 R CNN
 F 1 "100nF" H 7086 3245 50  0000 R CNN
 F 2 "Capacitors_SMD:C_0603" H 7238 3050 50  0001 C CNN
@@
 $EndComp
 $Comp
-L C C130
+L C C128
 U 1 1 58C0DF1C
 P 9000 3750
-F 0 "C130" V 8950 3650 50  0000 C CNN
+F 0 "C128" V 8950 3650 50  0000 C CNN
 F 1 "100nF" V 8950 3925 50  0000 C CNN
 F 2 "Capacitors_SMD:C_0603" H 9038 3600 50  0001 C CNN
@@
 $EndComp
 $Comp
-L CP1 C137
+L CP1 C135
 U 1 1 58C0DF23
 P 10350 3200
-F 0 "C137" H 10450 3300 50  0000 C CNN
+F 0 "C135" H 10450 3300 50  0000 C CNN
 F 1 "100μF" H 10500 3100 50  0000 C CNN
 F 2 "Capacitors_SMD:c_elec_8x10" H 10350 3200 50  0001 C CNN
@@
 $EndComp
 $Comp
-L C C133
+L C C131
 U 1 1 58C0DF2A
 P 9450 3200
-F 0 "C133" H 9350 3300 50  0000 C CNN
+F 0 "C131" H 9350 3300 50  0000 C CNN
 F 1 "100nF" H 9325 3100 50  0000 C CNN
 F 2 "Capacitors_SMD:C_0603" H 9488 3050 50  0001 C CNN
@@
 $EndComp
 $Comp
-L GND #PWR0201
+L GND #PWR181
 U 1 1 58C0DF31
 P 7200 3400
-F 0 "#PWR0201" H 7200 3150 50  0001 C CNN
+F 0 "#PWR181" H 7200 3150 50  0001 C CNN
 F 1 "GND" H 7200 3250 50  0000 C CNN
 F 2 "" H 7200 3400 50  0000 C CNN
@@
 $EndComp
 $Comp
-L C C134
+L C C132
 U 1 1 58C0DF37
 P 9750 3200
-F 0 "C134" H 9650 3300 50  0000 C CNN
+F 0 "C132" H 9650 3300 50  0000 C CNN
 F 1 "100nF" H 9625 3100 50  0000 C CNN
 F 2 "Capacitors_SMD:C_0603" H 9788 3050 50  0001 C CNN
@@
 $EndComp
 $Comp
-L GND #PWR0202
+L GND #PWR187
 U 1 1 58C0DF3E
 P 10050 3450
-F 0 "#PWR0202" H 10050 3200 50  0001 C CNN
+F 0 "#PWR187" H 10050 3200 50  0001 C CNN
 F 1 "GND" H 10055 3277 50  0000 C CNN
 F 2 "" H 10050 3450 50  0000 C CNN
@@
 $EndComp
 $Comp
-L +24V #PWR0203
+L +24V #PWR183
 U 1 1 58C0DF44
 P 8250 2950
-F 0 "#PWR0203" H 8250 2800 50  0001 C CNN
+F 0 "#PWR183" H 8250 2800 50  0001 C CNN
 F 1 "+24V" H 8265 3123 50  0000 C CNN
 F 2 "" H 8250 2950 50  0000 C CNN
@@
 $EndComp
 $Comp
-L C C127
+L C C125
 U 1 1 58C0DF4A
 P 8850 4250
-F 0 "C127" H 8965 4296 50  0000 L CNN
+F 0 "C125" H 8965 4296 50  0000 L CNN
 F 1 "22nF" H 8965 4205 50  0000 L CNN
 F 2 "Capacitors_SMD:C_0603" H 8888 4100 50  0001 C CNN
@@
 $EndComp
 $Comp
-L GND #PWR0204
+L GND #PWR186
 U 1 1 58C0DF5F
 P 9350 7150
-F 0 "#PWR0204" H 9350 6900 50  0001 C CNN
+F 0 "#PWR186" H 9350 6900 50  0001 C CNN
 F 1 "GND" H 9355 6977 50  0000 C CNN
 F 2 "" H 9350 7150 50  0000 C CNN
@@
 $EndComp
 $Comp
-L C C124
+L C C122
 U 1 1 58C0DF6D
 P 6800 4050
-F 0 "C124" H 6850 4150 50  0000 L CNN
+F 0 "C122" H 6850 4150 50  0000 L CNN
 F 1 "470nF" H 6825 3950 50  0000 L CNN
 F 2 "Capacitors_SMD:C_0603" H 6838 3900 50  0001 C CNN
@@
 NoConn ~ 7400 5800
 $Comp
-L GND #PWR0205
+L GND #PWR182
 U 1 1 58C0DF82
 P 7350 6200
-F 0 "#PWR0205" H 7350 5950 50  0001 C CNN
+F 0 "#PWR182" H 7350 5950 50  0001 C CNN
 F 1 "GND" H 7355 6027 50  0000 C CNN
 F 2 "" H 7350 6200 50  0000 C CNN
@@
 $EndComp
 $Comp
-L C C135
+L C C133
 U 1 1 58C0DF88
 P 9800 6800
-F 0 "C135" H 9850 6900 50  0000 L CNN
+F 0 "C133" H 9850 6900 50  0000 L CNN
 F 1 "100nF" H 9850 6700 50  0000 L CNN
 F 2 "Capacitors_SMD:C_0603" H 9838 6650 50  0001 C CNN
@@
 NoConn ~ 7400 4650
 $Comp
-L C C126
+L C C124
 U 1 1 58C0DF9A
 P 7200 4050
-F 0 "C126" H 7250 4150 50  0000 L CNN
+F 0 "C124" H 7250 4150 50  0000 L CNN
 F 1 "4.7μF" H 7250 3950 50  0000 L CNN
 F 2 "Capacitors_SMD:C_0603" H 7238 3900 50  0001 C CNN
@@
 $EndComp
 $Comp
-L C C138
+L C C136
 U 1 1 58C0DFB8
 P 10600 6800
-F 0 "C138" H 10650 6900 50  0000 L CNN
+F 0 "C136" H 10650 6900 50  0000 L CNN
 F 1 "100nF" H 10650 6700 50  0000 L CNN
 F 2 "Capacitors_SMD:C_0603" H 10638 6650 50  0001 C CNN
@@
 $EndComp
 $Comp
-L C C128
+L C C126
 U 1 1 58C0DFBF
 P 8850 5050
-F 0 "C128" H 8875 5150 50  0000 L CNN
+F 0 "C126" H 8875 5150 50  0000 L CNN
 F 1 "470pF" H 8850 4950 50  0000 L CNN
 F 2 "Capacitors_SMD:C_0603" H 8888 4900 50  0001 C CNN
@@
 $EndComp
 $Comp
-L GND #PWR0206
+L GND #PWR184
 U 1 1 58C0DFC6
 P 8950 5300
-F 0 "#PWR0206" H 8950 5050 50  0001 C CNN
+F 0 "#PWR184" H 8950 5050 50  0001 C CNN
 F 1 "GND" H 8950 5150 50  0000 C CNN
 F 2 "" H 8950 5300 50  0000 C CNN
@@
 $EndComp
 $Comp
-L C C131
+L C C129
 U 1 1 58C0DFCC
 P 9050 5050
-F 0 "C131" H 9075 5150 50  0000 L CNN
+F 0 "C129" H 9075 5150 50  0000 L CNN
 F 1 "470pF" H 9075 4950 50  0000 L CNN
 F 2 "Capacitors_SMD:C_0603" H 9088 4900 50  0001 C CNN
@@
 $EndComp
 $Comp
-L C C129
+L C C127
 U 1 1 58C0DFD3
 P 8850 5900
-F 0 "C129" H 8875 6000 50  0000 L CNN
+F 0 "C127" H 8875 6000 50  0000 L CNN
 F 1 "470pF" H 8850 5800 50  0000 L CNN
 F 2 "Capacitors_SMD:C_0603" H 8888 5750 50  0001 C CNN
@@
 $EndComp
 $Comp
-L GND #PWR0207
+L GND #PWR185
 U 1 1 58C0DFDA
 P 8950 6150
-F 0 "#PWR0207" H 8950 5900 50  0001 C CNN
+F 0 "#PWR185" H 8950 5900 50  0001 C CNN
 F 1 "GND" H 8950 6000 50  0000 C CNN
 F 2 "" H 8950 6150 50  0000 C CNN
@@
 $EndComp
 $Comp
-L C C132
+L C C130
 U 1 1 58C0DFE0
 P 9050 5900
-F 0 "C132" H 9075 6000 50  0000 L CNN
+F 0 "C130" H 9075 6000 50  0000 L CNN
 F 1 "470pF" H 9075 5800 50  0000 L CNN
 F 2 "Capacitors_SMD:C_0603" H 9088 5750 50  0001 C CNN
@@
 $EndComp
 $Comp
-L TMC2130 U18
+L TMC2130 U17
 U 1 1 58C0DFE7
 P 8100 4800
-F 0 "U18" H 7650 6300 60  0000 C CNN
+F 0 "U17" H 7650 6300 60  0000 C CNN
 F 1 "TMC2130" H 8400 6300 60  0000 C CNN
 F 2 "KiMBo:QFN36_5X6" H 8100 5100 60  0001 C CNN
@@
 	8850 6100 8850 6050
 $Comp
-L C C136
+L C C134
 U 1 1 58C0E066
 P 10050 3200
-F 0 "C136" H 9950 3300 50  0000 C CNN
+F 0 "C134" H 9950 3300 50  0000 C CNN
 F 1 "10μF" H 9925 3100 50  0000 C CNN
 F 2 "Capacitors_SMD:C_0805" H 10088 3050 50  0001 C CNN
@@
 	8800 4700 9100 4700
 $Comp
-L VDD_3V3B #PWR0208
+L VDD_3V3B #PWR180
 U 1 1 5A315EF4
 P 6450 3550
-F 0 "#PWR0208" H 6450 3400 50  0001 C CNN
+F 0 "#PWR180" H 6450 3400 50  0001 C CNN
 F 1 "VDD_3V3B" H 6465 3723 50  0000 C CNN
 F 2 "" H 6450 3550 50  0000 C CNN
@@
 $EndComp
 $Comp
-L C C123
+L C C121
 U 1 1 5A89C77B
 P 6450 4050
-F 0 "C123" H 6500 4150 50  0000 L CNN
+F 0 "C121" H 6500 4150 50  0000 L CNN
 F 1 "100nF" H 6475 3950 50  0000 L CNN
 F 2 "Capacitors_SMD:C_0603" H 6488 3900 50  0001 C CNN
