File: KiMBo/pwm.sch (KiCad schematic (older format))
At the start: 3 parts, among them U29 PCA9685

Commit message: Reorder the SS and EN lines from the shift registers such that the previously enabled/disabled motors stay enabled/disabled whilst writting to the shift register
Change 10k resistors to 4.7k, flip the open-drain inverter connected to B15 (PMTC_PGOOD)

Update the links in the README

Update the PDF schematic
Parts:
- R196: value 4.7k -> 4.7kΩ
Changed lines of the file:
@@
 F 0 "U29" H 5450 4587 60  0000 C CNN
 F 1 "PCA9685" H 5450 4481 60  0000 C CNN
-F 2 "" H 5450 3600 60  0000 C CNN
+F 2 "" H 5450 3600 60  0001 C CNN
 F 3 "" H 5450 3600 60  0000 C CNN
 	1    5450 3600
@@
 F 0 "C213" H 4214 3146 50  0000 L CNN
 F 1 "C" H 4214 3055 50  0000 L CNN
-F 2 "" H 4138 2950 50  0000 C CNN
+F 2 "" H 4138 2950 50  0001 C CNN
 F 3 "" H 4100 3100 50  0000 C CNN
 	1    4100 3100
@@
 P 4500 3900
 F 0 "R196" H 4570 3946 50  0000 L CNN
-F 1 "4.7k" H 4570 3855 50  0000 L CNN
-F 2 "" V 4430 3900 50  0000 C CNN
+F 1 "4.7kΩ" H 4570 3855 50  0000 L CNN
+F 2 "" V 4430 3900 50  0001 C CNN
 F 3 "" H 4500 3900 50  0000 C CNN
 	1    4500 3900

Commit message: Entry of additional component values
Parts:
- C213: value C -> 100nF
- renumbered R196 to R195
Changed lines of the file:
@@
 P 4100 3100
 F 0 "C213" H 4214 3146 50  0000 L CNN
-F 1 "C" H 4214 3055 50  0000 L CNN
+F 1 "100nF" H 4214 3055 50  0000 L CNN
 F 2 "" H 4138 2950 50  0001 C CNN
 F 3 "" H 4100 3100 50  0000 C CNN
@@
 $EndComp
 $Comp
-L GND #PWR0272
+L GND #PWR0273
 U 1 1 595584AE
 P 4100 3300
-F 0 "#PWR0272" H 4100 3050 50  0001 C CNN
+F 0 "#PWR0273" H 4100 3050 50  0001 C CNN
 F 1 "GND" H 4105 3127 50  0000 C CNN
 F 2 "" H 4100 3300 50  0000 C CNN
@@
 	4450 4100 4750 4100
 $Comp
-L GND #PWR0273
+L GND #PWR0274
 U 1 1 595593D7
 P 4700 4450
-F 0 "#PWR0273" H 4700 4200 50  0001 C CNN
+F 0 "#PWR0274" H 4700 4200 50  0001 C CNN
 F 1 "GND" H 4705 4277 50  0000 C CNN
 F 2 "" H 4700 4450 50  0000 C CNN
@@
 ~PWM_EN
 $Comp
-L R R196
+L R R195
 U 1 1 5970A901
 P 4500 3900
-F 0 "R196" H 4570 3946 50  0000 L CNN
+F 0 "R195" H 4570 3946 50  0000 L CNN
 F 1 "4.7kΩ" H 4570 3855 50  0000 L CNN
 F 2 "" V 4430 3900 50  0001 C CNN
@@
 DOCK1_HEAT
 $Comp
-L VDD_3V3B #PWR0274
+L VDD_3V3B #PWR0275
 U 1 1 5A115F67
 P 4500 3700
-F 0 "#PWR0274" H 4500 3550 50  0001 C CNN
+F 0 "#PWR0275" H 4500 3550 50  0001 C CNN
 F 1 "VDD_3V3B" H 4500 3850 50  0000 C CNN
 F 2 "" H 4500 3700 50  0000 C CNN
@@
 $EndComp
 $Comp
-L VDD_3V3B #PWR0275
+L VDD_3V3B #PWR0276
 U 1 1 5A118229
 P 4100 2850
-F 0 "#PWR0275" H 4100 2700 50  0001 C CNN
+F 0 "#PWR0276" H 4100 2700 50  0001 C CNN
 F 1 "VDD_3V3B" H 4115 3023 50  0000 C CNN
 F 2 "" H 4100 2850 50  0000 C CNN

Commit message: Add equivalent annotations document, associate more footprints
Parts:
- C215: renamed from C213; footprint (none) -> Capacitors_SMD:C_0603
- renumbered R195 to R194
Other:
- note added: "CL10B104KB8NNND-ND"
Changed lines of the file:
@@
 $EndComp
 $Comp
-L C C213
+L C C215
 U 1 1 59558467
 P 4100 3100
-F 0 "C213" H 4214 3146 50  0000 L CNN
+F 0 "C215" H 4214 3146 50  0000 L CNN
 F 1 "100nF" H 4214 3055 50  0000 L CNN
-F 2 "" H 4138 2950 50  0001 C CNN
+F 2 "Capacitors_SMD:C_0603" H 4138 2950 50  0001 C CNN
 F 3 "" H 4100 3100 50  0000 C CNN
 	1    4100 3100
@@
 $EndComp
 $Comp
-L GND #PWR0273
+L GND #PWR0274
 U 1 1 595584AE
 P 4100 3300
-F 0 "#PWR0273" H 4100 3050 50  0001 C CNN
+F 0 "#PWR0274" H 4100 3050 50  0001 C CNN
 F 1 "GND" H 4105 3127 50  0000 C CNN
 F 2 "" H 4100 3300 50  0000 C CNN
@@
 	4450 4100 4750 4100
 $Comp
-L GND #PWR0274
+L GND #PWR0275
 U 1 1 595593D7
 P 4700 4450
-F 0 "#PWR0274" H 4700 4200 50  0001 C CNN
+F 0 "#PWR0275" H 4700 4200 50  0001 C CNN
 F 1 "GND" H 4705 4277 50  0000 C CNN
 F 2 "" H 4700 4450 50  0000 C CNN
@@
 ~PWM_EN
 $Comp
-L R R195
+L R R194
 U 1 1 5970A901
 P 4500 3900
-F 0 "R195" H 4570 3946 50  0000 L CNN
+F 0 "R194" H 4570 3946 50  0000 L CNN
 F 1 "4.7kΩ" H 4570 3855 50  0000 L CNN
 F 2 "" V 4430 3900 50  0001 C CNN
@@
 DOCK1_HEAT
 $Comp
-L VDD_3V3B #PWR0275
+L VDD_3V3B #PWR0276
 U 1 1 5A115F67
 P 4500 3700
-F 0 "#PWR0275" H 4500 3550 50  0001 C CNN
+F 0 "#PWR0276" H 4500 3550 50  0001 C CNN
 F 1 "VDD_3V3B" H 4500 3850 50  0000 C CNN
 F 2 "" H 4500 3700 50  0000 C CNN
@@
 $EndComp
 $Comp
-L VDD_3V3B #PWR0276
+L VDD_3V3B #PWR0277
 U 1 1 5A118229
 P 4100 2850
-F 0 "#PWR0276" H 4100 2700 50  0001 C CNN
+F 0 "#PWR0277" H 4100 2700 50  0001 C CNN
 F 1 "VDD_3V3B" H 4115 3023 50  0000 C CNN
 F 2 "" H 4100 2850 50  0000 C CNN
@@
 $EndComp
 NoConn ~ 6150 3900
+Text Notes 3550 2600 0    60   ~ 0
+CL10B104KB8NNND-ND
 $EndSCHEMATC

Commit message: Connect X and Z stepper driver open-drain DIAG0 and DIAG1 lines together
Parts:
- renumbered C215 to C213, R194 to R188, U29 to U27
Changed lines of the file:
@@
 $EndDescr
 $Comp
-L PCA9685 U29
+L PCA9685 U27
 U 1 1 595289D2
 P 5450 3600
-F 0 "U29" H 5450 4587 60  0000 C CNN
+F 0 "U27" H 5450 4587 60  0000 C CNN
 F 1 "PCA9685" H 5450 4481 60  0000 C CNN
 F 2 "" H 5450 3600 60  0001 C CNN
@@
 $EndComp
 $Comp
-L C C215
+L C C213
 U 1 1 59558467
 P 4100 3100
-F 0 "C215" H 4214 3146 50  0000 L CNN
+F 0 "C213" H 4214 3146 50  0000 L CNN
 F 1 "100nF" H 4214 3055 50  0000 L CNN
 F 2 "Capacitors_SMD:C_0603" H 4138 2950 50  0001 C CNN
@@
 $EndComp
 $Comp
-L GND #PWR0274
+L GND #PWR0264
 U 1 1 595584AE
 P 4100 3300
-F 0 "#PWR0274" H 4100 3050 50  0001 C CNN
+F 0 "#PWR0264" H 4100 3050 50  0001 C CNN
 F 1 "GND" H 4105 3127 50  0000 C CNN
 F 2 "" H 4100 3300 50  0000 C CNN
@@
 	4450 4100 4750 4100
 $Comp
-L GND #PWR0275
+L GND #PWR0265
 U 1 1 595593D7
 P 4700 4450
-F 0 "#PWR0275" H 4700 4200 50  0001 C CNN
+F 0 "#PWR0265" H 4700 4200 50  0001 C CNN
 F 1 "GND" H 4705 4277 50  0000 C CNN
 F 2 "" H 4700 4450 50  0000 C CNN
@@
 ~PWM_EN
 $Comp
-L R R194
+L R R188
 U 1 1 5970A901
 P 4500 3900
-F 0 "R194" H 4570 3946 50  0000 L CNN
+F 0 "R188" H 4570 3946 50  0000 L CNN
 F 1 "4.7kΩ" H 4570 3855 50  0000 L CNN
 F 2 "" V 4430 3900 50  0001 C CNN
@@
 DOCK1_HEAT
 $Comp
-L VDD_3V3B #PWR0276
+L VDD_3V3B #PWR0266
 U 1 1 5A115F67
 P 4500 3700
-F 0 "#PWR0276" H 4500 3550 50  0001 C CNN
+F 0 "#PWR0266" H 4500 3550 50  0001 C CNN
 F 1 "VDD_3V3B" H 4500 3850 50  0000 C CNN
 F 2 "" H 4500 3700 50  0000 C CNN
@@
 $EndComp
 $Comp
-L VDD_3V3B #PWR0277
+L VDD_3V3B #PWR0267
 U 1 1 5A118229
 P 4100 2850
-F 0 "#PWR0277" H 4100 2700 50  0001 C CNN
+F 0 "#PWR0267" H 4100 2700 50  0001 C CNN
 F 1 "VDD_3V3B" H 4115 3023 50  0000 C CNN
 F 2 "" H 4100 2850 50  0000 C CNN

Commit message: Leave SPI0 free for a display, reassign pins so SPI1 is available
Fix some typos/errors
Parts:
- renumbered R188 to R190, U27 to U26
Changed lines of the file:
@@
 $EndDescr
 $Comp
-L PCA9685 U27
+L PCA9685 U26
 U 1 1 595289D2
 P 5450 3600
-F 0 "U27" H 5450 4587 60  0000 C CNN
+F 0 "U26" H 5450 4587 60  0000 C CNN
 F 1 "PCA9685" H 5450 4481 60  0000 C CNN
 F 2 "" H 5450 3600 60  0001 C CNN
@@
 $EndComp
 $Comp
-L GND #PWR0264
+L GND #PWR0263
 U 1 1 595584AE
 P 4100 3300
-F 0 "#PWR0264" H 4100 3050 50  0001 C CNN
+F 0 "#PWR0263" H 4100 3050 50  0001 C CNN
 F 1 "GND" H 4105 3127 50  0000 C CNN
 F 2 "" H 4100 3300 50  0000 C CNN
@@
 	4450 4100 4750 4100
 $Comp
-L GND #PWR0265
+L GND #PWR0264
 U 1 1 595593D7
 P 4700 4450
-F 0 "#PWR0265" H 4700 4200 50  0001 C CNN
+F 0 "#PWR0264" H 4700 4200 50  0001 C CNN
 F 1 "GND" H 4705 4277 50  0000 C CNN
 F 2 "" H 4700 4450 50  0000 C CNN
@@
 ~PWM_EN
 $Comp
-L R R188
+L R R190
 U 1 1 5970A901
 P 4500 3900
-F 0 "R188" H 4570 3946 50  0000 L CNN
+F 0 "R190" H 4570 3946 50  0000 L CNN
 F 1 "4.7kΩ" H 4570 3855 50  0000 L CNN
 F 2 "" V 4430 3900 50  0001 C CNN
@@
 DOCK1_HEAT
 $Comp
-L VDD_3V3B #PWR0266
+L VDD_3V3B #PWR0265
 U 1 1 5A115F67
 P 4500 3700
-F 0 "#PWR0266" H 4500 3550 50  0001 C CNN
+F 0 "#PWR0265" H 4500 3550 50  0001 C CNN
 F 1 "VDD_3V3B" H 4500 3850 50  0000 C CNN
 F 2 "" H 4500 3700 50  0000 C CNN
@@
 $EndComp
 $Comp
-L VDD_3V3B #PWR0267
+L VDD_3V3B #PWR0266
 U 1 1 5A118229
 P 4100 2850
-F 0 "#PWR0267" H 4100 2700 50  0001 C CNN
+F 0 "#PWR0266" H 4100 2700 50  0001 C CNN
 F 1 "VDD_3V3B" H 4115 3023 50  0000 C CNN
 F 2 "" H 4100 2850 50  0000 C CNN

Commit message: Use fixed 5V LM2592HV Buck, include SPI0 header for LCD
Parts:
- renumbered C213 to C210, R190 to R187
Changed lines of the file:
@@
 $EndComp
 $Comp
-L C C213
+L C C210
 U 1 1 59558467
 P 4100 3100
-F 0 "C213" H 4214 3146 50  0000 L CNN
+F 0 "C210" H 4214 3146 50  0000 L CNN
 F 1 "100nF" H 4214 3055 50  0000 L CNN
 F 2 "Capacitors_SMD:C_0603" H 4138 2950 50  0001 C CNN
@@
 $EndComp
 $Comp
-L GND #PWR0263
+L GND #PWR0258
 U 1 1 595584AE
 P 4100 3300
-F 0 "#PWR0263" H 4100 3050 50  0001 C CNN
+F 0 "#PWR0258" H 4100 3050 50  0001 C CNN
 F 1 "GND" H 4105 3127 50  0000 C CNN
 F 2 "" H 4100 3300 50  0000 C CNN
@@
 	4450 4100 4750 4100
 $Comp
-L GND #PWR0264
+L GND #PWR0259
 U 1 1 595593D7
 P 4700 4450
-F 0 "#PWR0264" H 4700 4200 50  0001 C CNN
+F 0 "#PWR0259" H 4700 4200 50  0001 C CNN
 F 1 "GND" H 4705 4277 50  0000 C CNN
 F 2 "" H 4700 4450 50  0000 C CNN
@@
 ~PWM_EN
 $Comp
-L R R190
+L R R187
 U 1 1 5970A901
 P 4500 3900
-F 0 "R190" H 4570 3946 50  0000 L CNN
+F 0 "R187" H 4570 3946 50  0000 L CNN
 F 1 "4.7kΩ" H 4570 3855 50  0000 L CNN
 F 2 "" V 4430 3900 50  0001 C CNN
@@
 DOCK1_HEAT
 $Comp
-L VDD_3V3B #PWR0265
+L VDD_3V3B #PWR0260
 U 1 1 5A115F67
 P 4500 3700
-F 0 "#PWR0265" H 4500 3550 50  0001 C CNN
+F 0 "#PWR0260" H 4500 3550 50  0001 C CNN
 F 1 "VDD_3V3B" H 4500 3850 50  0000 C CNN
 F 2 "" H 4500 3700 50  0000 C CNN
@@
 $EndComp
 $Comp
-L VDD_3V3B #PWR0266
+L VDD_3V3B #PWR0261
 U 1 1 5A118229
 P 4100 2850
-F 0 "#PWR0266" H 4100 2700 50  0001 C CNN
+F 0 "#PWR0261" H 4100 2700 50  0001 C CNN
 F 1 "VDD_3V3B" H 4115 3023 50  0000 C CNN
 F 2 "" H 4100 2850 50  0000 C CNN

Commit message: Assocate more footprints
Parts:
- R187: footprint (none) -> Resistors_SMD:R_0603
Changed lines of the file:
@@
 F 0 "R187" H 4570 3946 50  0000 L CNN
 F 1 "4.7kΩ" H 4570 3855 50  0000 L CNN
-F 2 "" V 4430 3900 50  0001 C CNN
+F 2 "Resistors_SMD:R_0603" V 4430 3900 50  0001 C CNN
 F 3 "" H 4500 3900 50  0000 C CNN
 	1    4500 3900
