File: KiMBo/config.sch (KiCad schematic (older format))
At the start: 18 parts, among them SW3 μSD_Boot

Commit message: Create more footprints and add more associations
Parts:
- SW3: footprint (none) -> KiMBo:KMR_SW_SPST_EVQP7A
Changed lines of the file:
@@
 F 0 "SW3" H 7900 2975 50  0000 C CNN
 F 1 "μSD_Boot" H 7900 2884 50  0000 C CNN
-F 2 "" H 7900 2650 50  0001 C CNN
+F 2 "KiMBo:KMR_SW_SPST_EVQP7A" H 7900 2650 50  0001 C CNN
 F 3 "" H 7900 2650 50  0000 C CNN
 	1    7900 2650
