File: KiMBo/usb.sch (KiCad schematic (older format))
At the start: 19 parts, among them U1 OSD3358, U10 TPD4S012, U7 TPS2051B, U8 TPD4S012, U9 74LVC2G241

Commit message: Use fixed 5V LM2592HV Buck, include SPI0 header for LCD
Parts:
- renumbered C26 to C23, C27 to C24, C28 to C25, C29 to C26, FB22 to FB27, R49 to R46, R50 to R47, R51 to R48, R52 to R49, R53 to R50, R54 to R51, R55 to R52, R56 to R53
Changed lines of the file:
@@
 $EndComp
 $Comp
-L GND #PWR0106
+L GND #PWR0101
 U 1 1 584F5078
 P 7550 2500
-F 0 "#PWR0106" H 7550 2250 50  0001 C CNN
+F 0 "#PWR0101" H 7550 2250 50  0001 C CNN
 F 1 "GND" H 7555 2327 50  0000 C CNN
 F 2 "" H 7550 2500 50  0000 C CNN
@@
 UART0_RXD_IN
 $Comp
-L R R56
+L R R53
 U 1 1 584F5085
 P 7700 1800
-F 0 "R56" H 7770 1846 50  0000 L CNN
+F 0 "R53" H 7770 1846 50  0000 L CNN
 F 1 "100kΩ" H 7770 1755 50  0000 L CNN
 F 2 "Resistors_SMD:R_0402" V 7630 1800 50  0001 C CNN
@@
 $EndComp
 $Comp
-L GND #PWR0107
+L GND #PWR0102
 U 1 1 584F508C
 P 6450 2050
-F 0 "#PWR0107" H 6450 1800 50  0001 C CNN
+F 0 "#PWR0102" H 6450 1800 50  0001 C CNN
 F 1 "GND" H 6455 1877 50  0000 C CNN
 F 2 "" H 6450 2050 50  0000 C CNN
@@
 UART0_TXD_OUT
 $Comp
-L GND #PWR0108
+L GND #PWR0103
 U 1 1 584F509A
 P 7700 2000
-F 0 "#PWR0108" H 7700 1750 50  0001 C CNN
+F 0 "#PWR0103" H 7700 1750 50  0001 C CNN
 F 1 "GND" H 7705 1827 50  0000 C CNN
 F 2 "" H 7700 2000 50  0000 C CNN
@@
 $EndComp
 $Comp
-L C C29
+L C C26
 U 1 1 584F50A3
 P 8150 1650
-F 0 "C29" H 8265 1696 50  0000 L CNN
+F 0 "C26" H 8265 1696 50  0000 L CNN
 F 1 "100nF" H 8265 1605 50  0000 L CNN
 F 2 "Capacitors_SMD:C_0402" H 8150 1650 50  0001 C CNN
@@
 $EndComp
 $Comp
-L GND #PWR0109
+L GND #PWR0104
 U 1 1 584F50AA
 P 8150 1850
-F 0 "#PWR0109" H 8150 1600 50  0001 C CNN
+F 0 "#PWR0104" H 8150 1600 50  0001 C CNN
 F 1 "GND" H 8155 1677 50  0000 C CNN
 F 2 "" H 8150 1850 50  0000 C CNN
@@
 NoConn ~ 5450 2150
 $Comp
-L R R55
+L R R52
 U 1 1 584F50C1
 P 6250 1650
-F 0 "R55" H 6320 1696 50  0000 L CNN
+F 0 "R52" H 6320 1696 50  0000 L CNN
 F 1 "0Ω" H 6320 1605 50  0000 L CNN
 F 2 "Resistors_SMD:R_0402" V 6180 1650 50  0001 C CNN
@@
 NoConn ~ 3650 1950
 $Comp
-L R R49
+L R R46
 U 1 1 584F50D1
 P 2850 2250
-F 0 "R49" H 2920 2296 50  0000 L CNN
+F 0 "R46" H 2920 2296 50  0000 L CNN
 F 1 "0Ω" H 2920 2205 50  0000 L CNN
 F 2 "Resistors_SMD:R_0402" V 2780 2250 50  0001 C CNN
@@
 $EndComp
 $Comp
-L GND #PWR0110
+L GND #PWR0105
 U 1 1 584F50D8
 P 2850 2450
-F 0 "#PWR0110" H 2850 2200 50  0001 C CNN
+F 0 "#PWR0105" H 2850 2200 50  0001 C CNN
 F 1 "GND" H 2855 2277 50  0000 C CNN
 F 2 "" H 2850 2450 50  0000 C CNN
@@
 USB1_DRVVBUS
 $Comp
-L R R50
+L R R47
 U 1 1 584F50E0
 P 3500 1450
-F 0 "R50" H 3569 1496 50  0000 L CNN
+F 0 "R47" H 3569 1496 50  0000 L CNN
 F 1 "1.5kΩ" H 3569 1405 50  0000 L CNN
 F 2 "Resistors_SMD:R_0402" V 3430 1450 50  0001 C CNN
@@
 $EndComp
 $Comp
-L R R52
+L R R49
 U 1 1 584F50E7
 P 3600 1450
-F 0 "R52" H 3670 1496 50  0000 L CNN
+F 0 "R49" H 3670 1496 50  0000 L CNN
 F 1 "1.5kΩ" H 3670 1405 50  0000 L CNN
 F 2 "Resistors_SMD:R_0402" V 3530 1450 50  0001 C CNN
@@
 $EndComp
 $Comp
-L C C27
+L C C24
 U 1 1 58524285
 P 6300 4600
-F 0 "C27" H 6415 4646 50  0000 L CNN
+F 0 "C24" H 6415 4646 50  0000 L CNN
 F 1 "100nF" H 6415 4555 50  0000 L CNN
 F 2 "Capacitors_SMD:C_0402" H 6300 4600 50  0001 C CNN
@@
 $EndComp
 $Comp
-L GND #PWR0111
+L GND #PWR0106
 U 1 1 585243B8
 P 6300 4850
-F 0 "#PWR0111" H 6300 4600 50  0001 C CNN
+F 0 "#PWR0106" H 6300 4600 50  0001 C CNN
 F 1 "GND" H 6305 4677 50  0000 C CNN
 F 2 "" H 6300 4850 50  0000 C CNN
@@
 $EndComp
 $Comp
-L GND #PWR0112
+L GND #PWR0107
 U 1 1 58528602
 P 4500 4550
-F 0 "#PWR0112" H 4500 4300 50  0001 C CNN
+F 0 "#PWR0107" H 4500 4300 50  0001 C CNN
 F 1 "GND" H 4505 4377 50  0000 C CNN
 F 2 "" H 4500 4550 50  0000 C CNN
@@
 $EndComp
 $Comp
-L R R53
+L R R50
 U 1 1 58528C30
 P 4850 4400
-F 0 "R53" V 4700 4400 50  0000 C CNN
+F 0 "R50" V 4700 4400 50  0000 C CNN
 F 1 "0Ω" V 4775 4400 50  0000 C CNN
 F 2 "Resistors_SMD:R_0402" V 4780 4400 50  0001 C CNN
@@
 $EndComp
 $Comp
-L GND #PWR0113
+L GND #PWR0108
 U 1 1 5852A6BE
 P 2500 4600
-F 0 "#PWR0113" H 2500 4350 50  0001 C CNN
+F 0 "#PWR0108" H 2500 4350 50  0001 C CNN
 F 1 "GND" H 2505 4427 50  0000 C CNN
 F 2 "" H 2500 4600 50  0000 C CNN
@@
 $EndComp
 $Comp
-L GND #PWR0114
+L GND #PWR0109
 U 1 1 5852A82F
 P 2700 4250
-F 0 "#PWR0114" H 2700 4000 50  0001 C CNN
+F 0 "#PWR0109" H 2700 4000 50  0001 C CNN
 F 1 "GND" H 2705 4077 50  0000 C CNN
 F 2 "" H 2700 4250 50  0000 C CNN
@@
 USB1_DRVVBUS
 $Comp
-L R R51
+L R R48
 U 1 1 5852B51B
 P 3500 4600
-F 0 "R51" H 3570 4646 50  0000 L CNN
+F 0 "R48" H 3570 4646 50  0000 L CNN
 F 1 "10kΩ" H 3570 4555 50  0000 L CNN
 F 2 "Resistors_SMD:R_0402" V 3430 4600 50  0001 C CNN
@@
 $EndComp
 $Comp
-L GND #PWR0115
+L GND #PWR0110
 U 1 1 5852B68C
 P 3500 4800
-F 0 "#PWR0115" H 3500 4550 50  0001 C CNN
+F 0 "#PWR0110" H 3500 4550 50  0001 C CNN
 F 1 "GND" H 3505 4627 50  0000 C CNN
 F 2 "" H 3500 4800 50  0000 C CNN
@@
 $EndComp
 $Comp
-L C C28
+L C C25
 U 1 1 5852C2E6
 P 7950 4100
-F 0 "C28" H 8065 4146 50  0000 L CNN
+F 0 "C25" H 8065 4146 50  0000 L CNN
 F 1 "100nF" H 8065 4055 50  0000 L CNN
 F 2 "Capacitors_SMD:C_0402" H 7950 4100 50  0001 C CNN
@@
 USB.CLIENT.ID
 $Comp
-L INDUCTOR_Small FB22
+L INDUCTOR_Small FB27
 U 1 1 58E84972
 P 5950 4100
-F 0 "FB22" V 6135 4100 50  0000 C CNN
+F 0 "FB27" V 6135 4100 50  0000 C CNN
 F 1 "LI0805H151R-10" V 6050 3900 50  0000 C CNN
 F 2 "" H 5950 4100 50  0001 C CNN
@@
 I2C2_SDA
 $Comp
-L USB_DC #PWR0116
+L USB_DC #PWR0111
 U 1 1 59F94F9A
 P 8100 3850
-F 0 "#PWR0116" H 8100 3700 50  0001 C CNN
+F 0 "#PWR0111" H 8100 3700 50  0001 C CNN
 F 1 "USB_DC" H 8115 4023 50  0000 C CNN
 F 2 "" H 8100 3850 50  0000 C CNN
@@
 $EndComp
 $Comp
-L SYS_5V #PWR0117
+L SYS_5V #PWR0112
 U 1 1 59F970D0
 P 2500 4150
-F 0 "#PWR0117" H 2500 4000 50  0001 C CNN
+F 0 "#PWR0112" H 2500 4000 50  0001 C CNN
 F 1 "SYS_5V" H 2515 4323 50  0000 C CNN
 F 2 "" H 2500 4150 50  0000 C CNN
@@
 $EndComp
 $Comp
-L VDD_3V3B #PWR0118
+L VDD_3V3B #PWR0113
 U 1 1 59FBF8B1
 P 6350 2100
-F 0 "#PWR0118" H 6350 1950 50  0001 C CNN
+F 0 "#PWR0113" H 6350 1950 50  0001 C CNN
 F 1 "VDD_3V3B" H 6350 2250 50  0000 C CNN
 F 2 "" H 6350 2100 50  0000 C CNN
@@
 $EndComp
 $Comp
-L VDD_3V3B #PWR0119
+L VDD_3V3B #PWR0114
 U 1 1 59FBF8FC
 P 7450 1950
-F 0 "#PWR0119" H 7450 1800 50  0001 C CNN
+F 0 "#PWR0114" H 7450 1800 50  0001 C CNN
 F 1 "VDD_3V3B" H 7400 2100 50  0000 C CNN
 F 2 "" H 7450 1950 50  0000 C CNN
@@
 $EndComp
 $Comp
-L VDD_3V3B #PWR0120
+L VDD_3V3B #PWR0115
 U 1 1 59FC0162
 P 8150 1450
-F 0 "#PWR0120" H 8150 1300 50  0001 C CNN
+F 0 "#PWR0115" H 8150 1300 50  0001 C CNN
 F 1 "VDD_3V3B" H 8165 1623 50  0000 C CNN
 F 2 "" H 8150 1450 50  0000 C CNN
@@
 $EndComp
 $Comp
-L USB_DC #PWR0121
+L USB_DC #PWR0116
 U 1 1 59FEDDB0
 P 6250 1450
-F 0 "#PWR0121" H 6250 1300 50  0001 C CNN
+F 0 "#PWR0116" H 6250 1300 50  0001 C CNN
 F 1 "USB_DC" H 6265 1623 50  0000 C CNN
 F 2 "" H 6250 1450 50  0000 C CNN
@@
 $EndComp
 $Comp
-L VDD_3V3B #PWR0122
+L VDD_3V3B #PWR0117
 U 1 1 5A01DA26
 P 3550 1200
-F 0 "#PWR0122" H 3550 1050 50  0001 C CNN
+F 0 "#PWR0117" H 3550 1050 50  0001 C CNN
 F 1 "VDD_3V3B" H 3565 1373 50  0000 C CNN
 F 2 "" H 3550 1200 50  0000 C CNN
@@
 Used a tantalum cap instead\nof the large aluminium cap\nTAJD227M010RNJ\ninstead of\nAVE107M06D16T-F (100μF)
 $Comp
-L VDD_3V3B #PWR0123
+L VDD_3V3B #PWR0118
 U 1 1 5AF563FC
 P 5050 4350
-F 0 "#PWR0123" H 5050 4200 50  0001 C CNN
+F 0 "#PWR0118" H 5050 4200 50  0001 C CNN
 F 1 "VDD_3V3B" H 5065 4523 50  0000 C CNN
 F 2 "" H 5050 4350 50  0000 C CNN
@@
 $EndComp
 $Comp
-L GND #PWR0124
+L GND #PWR0119
 U 1 1 5BC77EEA
 P 7950 4350
-F 0 "#PWR0124" H 7950 4100 50  0001 C CNN
+F 0 "#PWR0119" H 7950 4100 50  0001 C CNN
 F 1 "GND" H 7955 4177 50  0000 C CNN
 F 2 "" H 7950 4350 50  0000 C CNN
@@
 	6200 2350 6200 2300
 $Comp
-L R R54
+L R R51
 U 1 1 58DC7D9A
 P 5750 3900
-F 0 "R54" H 5819 3946 50  0000 L CNN
+F 0 "R51" H 5819 3946 50  0000 L CNN
 F 1 "100mΩ" H 5819 3855 50  0000 L CNN
 F 2 "Resistors_SMD:R_0402" V 5680 3900 50  0001 C CNN
@@
 73L3R10J
 $Comp
-L CP1 C26
+L CP1 C23
 U 1 1 58EB0DF2
 P 2500 4400
-F 0 "C26" H 2615 4446 50  0000 L CNN
+F 0 "C23" H 2615 4446 50  0000 L CNN
 F 1 "220μF" H 2615 4355 50  0000 L CNN
 F 2 "" H 2500 4400 50  0001 C CNN

Commit message: Assocate more footprints
Parts:
- C24, C25, C26: footprint Capacitors_SMD:C_0402 -> Capacitors_SMD:C_0603
- FB27: footprint (none) -> Resistors_SMD:R_0805
- R46, R47, R48, R49, R50, R51, R52, R53: footprint Resistors_SMD:R_0402 -> Resistors_SMD:R_0603
- U1: footprint (none) -> KiMBo:BGA-400-1-27mm
Changed lines of the file:
@@
 F 0 "U1" H 4550 1940 60  0000 C CNN
 F 1 "OSD3358" H 4550 1834 60  0000 C CNN
-F 2 "" H 3650 1650 60  0001 C CNN
+F 2 "KiMBo:BGA-400-1-27mm" H 3650 1650 60  0001 C CNN
 F 3 "" H 3650 1650 60  0001 C CNN
 	7    3650 1650
@@
 F 0 "R53" H 7770 1846 50  0000 L CNN
 F 1 "100kΩ" H 7770 1755 50  0000 L CNN
-F 2 "Resistors_SMD:R_0402" V 7630 1800 50  0001 C CNN
+F 2 "Resistors_SMD:R_0603" V 7630 1800 50  0001 C CNN
 F 3 "" H 7700 1800 50  0000 C CNN
 	1    7700 1800
@@
 F 0 "C26" H 8265 1696 50  0000 L CNN
 F 1 "100nF" H 8265 1605 50  0000 L CNN
-F 2 "Capacitors_SMD:C_0402" H 8150 1650 50  0001 C CNN
+F 2 "Capacitors_SMD:C_0603" H 8150 1650 50  0001 C CNN
 F 3 "" H 8150 1650 50  0000 C CNN
 	1    8150 1650
@@
 F 0 "R52" H 6320 1696 50  0000 L CNN
 F 1 "0Ω" H 6320 1605 50  0000 L CNN
-F 2 "Resistors_SMD:R_0402" V 6180 1650 50  0001 C CNN
+F 2 "Resistors_SMD:R_0603" V 6180 1650 50  0001 C CNN
 F 3 "" H 6250 1650 50  0000 C CNN
 	1    6250 1650
@@
 F 0 "R46" H 2920 2296 50  0000 L CNN
 F 1 "0Ω" H 2920 2205 50  0000 L CNN
-F 2 "Resistors_SMD:R_0402" V 2780 2250 50  0001 C CNN
+F 2 "Resistors_SMD:R_0603" V 2780 2250 50  0001 C CNN
 F 3 "" H 2850 2250 50  0000 C CNN
 	1    2850 2250
@@
 F 0 "R47" H 3569 1496 50  0000 L CNN
 F 1 "1.5kΩ" H 3569 1405 50  0000 L CNN
-F 2 "Resistors_SMD:R_0402" V 3430 1450 50  0001 C CNN
+F 2 "Resistors_SMD:R_0603" V 3430 1450 50  0001 C CNN
 F 3 "" H 3500 1450 50  0000 C CNN
 	1    3500 1450
@@
 F 0 "R49" H 3670 1496 50  0000 L CNN
 F 1 "1.5kΩ" H 3670 1405 50  0000 L CNN
-F 2 "Resistors_SMD:R_0402" V 3530 1450 50  0001 C CNN
+F 2 "Resistors_SMD:R_0603" V 3530 1450 50  0001 C CNN
 F 3 "" H 3600 1450 50  0000 C CNN
 	1    3600 1450
@@
 F 0 "C24" H 6415 4646 50  0000 L CNN
 F 1 "100nF" H 6415 4555 50  0000 L CNN
-F 2 "Capacitors_SMD:C_0402" H 6300 4600 50  0001 C CNN
+F 2 "Capacitors_SMD:C_0603" H 6300 4600 50  0001 C CNN
 F 3 "" H 6300 4600 50  0000 C CNN
 	1    6300 4600
@@
 F 0 "R50" V 4700 4400 50  0000 C CNN
 F 1 "0Ω" V 4775 4400 50  0000 C CNN
-F 2 "Resistors_SMD:R_0402" V 4780 4400 50  0001 C CNN
+F 2 "Resistors_SMD:R_0603" V 4780 4400 50  0001 C CNN
 F 3 "" H 4850 4400 50  0000 C CNN
 	1    4850 4400
@@
 F 0 "R48" H 3570 4646 50  0000 L CNN
 F 1 "10kΩ" H 3570 4555 50  0000 L CNN
-F 2 "Resistors_SMD:R_0402" V 3430 4600 50  0001 C CNN
+F 2 "Resistors_SMD:R_0603" V 3430 4600 50  0001 C CNN
 F 3 "" H 3500 4600 50  0000 C CNN
 	1    3500 4600
@@
 F 0 "C25" H 8065 4146 50  0000 L CNN
 F 1 "100nF" H 8065 4055 50  0000 L CNN
-F 2 "Capacitors_SMD:C_0402" H 7950 4100 50  0001 C CNN
+F 2 "Capacitors_SMD:C_0603" H 7950 4100 50  0001 C CNN
 F 3 "" H 7950 4100 50  0000 C CNN
 	1    7950 4100
@@
 F 0 "FB27" V 6135 4100 50  0000 C CNN
 F 1 "LI0805H151R-10" V 6050 3900 50  0000 C CNN
-F 2 "" H 5950 4100 50  0001 C CNN
+F 2 "Resistors_SMD:R_0805" H 5950 4100 50  0001 C CNN
 F 3 "" H 5950 4100 50  0000 C CNN
 	1    5950 4100
@@
 F 0 "R51" H 5819 3946 50  0000 L CNN
 F 1 "100mΩ" H 5819 3855 50  0000 L CNN
-F 2 "Resistors_SMD:R_0402" V 5680 3900 50  0001 C CNN
+F 2 "Resistors_SMD:R_0603" V 5680 3900 50  0001 C CNN
 F 3 "" H 5750 3900 50  0000 C CNN
 	1    5750 3900

Commit message: More footprint association
Parts:
- C23: footprint (none) -> Capacitors_Tantalum_SMD:TantalC_SizeD_EIA-7343_Reflow
Changed lines of the file:
@@
 $EndComp
 $Comp
-L GND #PWR0101
+L GND #PWR0102
 U 1 1 584F5078
 P 7550 2500
-F 0 "#PWR0101" H 7550 2250 50  0001 C CNN
+F 0 "#PWR0102" H 7550 2250 50  0001 C CNN
 F 1 "GND" H 7555 2327 50  0000 C CNN
 F 2 "" H 7550 2500 50  0000 C CNN
@@
 $EndComp
 $Comp
-L GND #PWR0102
+L GND #PWR0103
 U 1 1 584F508C
 P 6450 2050
-F 0 "#PWR0102" H 6450 1800 50  0001 C CNN
+F 0 "#PWR0103" H 6450 1800 50  0001 C CNN
 F 1 "GND" H 6455 1877 50  0000 C CNN
 F 2 "" H 6450 2050 50  0000 C CNN
@@
 UART0_TXD_OUT
 $Comp
-L GND #PWR0103
+L GND #PWR0104
 U 1 1 584F509A
 P 7700 2000
-F 0 "#PWR0103" H 7700 1750 50  0001 C CNN
+F 0 "#PWR0104" H 7700 1750 50  0001 C CNN
 F 1 "GND" H 7705 1827 50  0000 C CNN
 F 2 "" H 7700 2000 50  0000 C CNN
@@
 $EndComp
 $Comp
-L GND #PWR0104
+L GND #PWR0105
 U 1 1 584F50AA
 P 8150 1850
-F 0 "#PWR0104" H 8150 1600 50  0001 C CNN
+F 0 "#PWR0105" H 8150 1600 50  0001 C CNN
 F 1 "GND" H 8155 1677 50  0000 C CNN
 F 2 "" H 8150 1850 50  0000 C CNN
@@
 $EndComp
 $Comp
-L GND #PWR0105
+L GND #PWR0106
 U 1 1 584F50D8
 P 2850 2450
-F 0 "#PWR0105" H 2850 2200 50  0001 C CNN
+F 0 "#PWR0106" H 2850 2200 50  0001 C CNN
 F 1 "GND" H 2855 2277 50  0000 C CNN
 F 2 "" H 2850 2450 50  0000 C CNN
@@
 $EndComp
 $Comp
-L GND #PWR0106
+L GND #PWR0107
 U 1 1 585243B8
 P 6300 4850
-F 0 "#PWR0106" H 6300 4600 50  0001 C CNN
+F 0 "#PWR0107" H 6300 4600 50  0001 C CNN
 F 1 "GND" H 6305 4677 50  0000 C CNN
 F 2 "" H 6300 4850 50  0000 C CNN
@@
 $EndComp
 $Comp
-L GND #PWR0107
+L GND #PWR0108
 U 1 1 58528602
 P 4500 4550
-F 0 "#PWR0107" H 4500 4300 50  0001 C CNN
+F 0 "#PWR0108" H 4500 4300 50  0001 C CNN
 F 1 "GND" H 4505 4377 50  0000 C CNN
 F 2 "" H 4500 4550 50  0000 C CNN
@@
 $EndComp
 $Comp
-L GND #PWR0108
+L GND #PWR0109
 U 1 1 5852A6BE
 P 2500 4600
-F 0 "#PWR0108" H 2500 4350 50  0001 C CNN
+F 0 "#PWR0109" H 2500 4350 50  0001 C CNN
 F 1 "GND" H 2505 4427 50  0000 C CNN
 F 2 "" H 2500 4600 50  0000 C CNN
@@
 $EndComp
 $Comp
-L GND #PWR0109
+L GND #PWR0110
 U 1 1 5852A82F
 P 2700 4250
-F 0 "#PWR0109" H 2700 4000 50  0001 C CNN
+F 0 "#PWR0110" H 2700 4000 50  0001 C CNN
 F 1 "GND" H 2705 4077 50  0000 C CNN
 F 2 "" H 2700 4250 50  0000 C CNN
@@
 $EndComp
 $Comp
-L GND #PWR0110
+L GND #PWR0111
 U 1 1 5852B68C
 P 3500 4800
-F 0 "#PWR0110" H 3500 4550 50  0001 C CNN
+F 0 "#PWR0111" H 3500 4550 50  0001 C CNN
 F 1 "GND" H 3505 4627 50  0000 C CNN
 F 2 "" H 3500 4800 50  0000 C CNN
@@
 I2C2_SDA
 $Comp
-L USB_DC #PWR0111
+L USB_DC #PWR0112
 U 1 1 59F94F9A
 P 8100 3850
-F 0 "#PWR0111" H 8100 3700 50  0001 C CNN
+F 0 "#PWR0112" H 8100 3700 50  0001 C CNN
 F 1 "USB_DC" H 8115 4023 50  0000 C CNN
 F 2 "" H 8100 3850 50  0000 C CNN
@@
 $EndComp
 $Comp
-L SYS_5V #PWR0112
+L SYS_5V #PWR0113
 U 1 1 59F970D0
 P 2500 4150
-F 0 "#PWR0112" H 2500 4000 50  0001 C CNN
+F 0 "#PWR0113" H 2500 4000 50  0001 C CNN
 F 1 "SYS_5V" H 2515 4323 50  0000 C CNN
 F 2 "" H 2500 4150 50  0000 C CNN
@@
 $EndComp
 $Comp
-L VDD_3V3B #PWR0113
+L VDD_3V3B #PWR0114
 U 1 1 59FBF8B1
 P 6350 2100
-F 0 "#PWR0113" H 6350 1950 50  0001 C CNN
+F 0 "#PWR0114" H 6350 1950 50  0001 C CNN
 F 1 "VDD_3V3B" H 6350 2250 50  0000 C CNN
 F 2 "" H 6350 2100 50  0000 C CNN
@@
 $EndComp
 $Comp
-L VDD_3V3B #PWR0114
+L VDD_3V3B #PWR0115
 U 1 1 59FBF8FC
 P 7450 1950
-F 0 "#PWR0114" H 7450 1800 50  0001 C CNN
+F 0 "#PWR0115" H 7450 1800 50  0001 C CNN
 F 1 "VDD_3V3B" H 7400 2100 50  0000 C CNN
 F 2 "" H 7450 1950 50  0000 C CNN
@@
 $EndComp
 $Comp
-L VDD_3V3B #PWR0115
+L VDD_3V3B #PWR0116
 U 1 1 59FC0162
 P 8150 1450
-F 0 "#PWR0115" H 8150 1300 50  0001 C CNN
+F 0 "#PWR0116" H 8150 1300 50  0001 C CNN
 F 1 "VDD_3V3B" H 8165 1623 50  0000 C CNN
 F 2 "" H 8150 1450 50  0000 C CNN
@@
 $EndComp
 $Comp
-L USB_DC #PWR0116
+L USB_DC #PWR0117
 U 1 1 59FEDDB0
 P 6250 1450
-F 0 "#PWR0116" H 6250 1300 50  0001 C CNN
+F 0 "#PWR0117" H 6250 1300 50  0001 C CNN
 F 1 "USB_DC" H 6265 1623 50  0000 C CNN
 F 2 "" H 6250 1450 50  0000 C CNN
@@
 $EndComp
 $Comp
-L VDD_3V3B #PWR0117
+L VDD_3V3B #PWR0118
 U 1 1 5A01DA26
 P 3550 1200
-F 0 "#PWR0117" H 3550 1050 50  0001 C CNN
+F 0 "#PWR0118" H 3550 1050 50  0001 C CNN
 F 1 "VDD_3V3B" H 3565 1373 50  0000 C CNN
 F 2 "" H 3550 1200 50  0000 C CNN
@@
 Used a tantalum cap instead\nof the large aluminium cap\nTAJD227M010RNJ\ninstead of\nAVE107M06D16T-F (100μF)
 $Comp
-L VDD_3V3B #PWR0118
+L VDD_3V3B #PWR0119
 U 1 1 5AF563FC
 P 5050 4350
-F 0 "#PWR0118" H 5050 4200 50  0001 C CNN
+F 0 "#PWR0119" H 5050 4200 50  0001 C CNN
 F 1 "VDD_3V3B" H 5065 4523 50  0000 C CNN
 F 2 "" H 5050 4350 50  0000 C CNN
@@
 $EndComp
 $Comp
-L GND #PWR0119
+L GND #PWR0120
 U 1 1 5BC77EEA
 P 7950 4350
-F 0 "#PWR0119" H 7950 4100 50  0001 C CNN
+F 0 "#PWR0120" H 7950 4100 50  0001 C CNN
 F 1 "GND" H 7955 4177 50  0000 C CNN
 F 2 "" H 7950 4350 50  0000 C CNN
@@
 F 0 "C23" H 2615 4446 50  0000 L CNN
 F 1 "220μF" H 2615 4355 50  0000 L CNN
-F 2 "" H 2500 4400 50  0001 C CNN
+F 2 "Capacitors_Tantalum_SMD:TantalC_SizeD_EIA-7343_Reflow" H 2500 4400 50  0001 C CNN
 F 3 "" H 2500 4400 50  0000 C CNN
 	1    2500 4400

Commit message: Create more footprints and add more associations
Parts:
- TP6: footprint (none) -> Measurement_Points:Measurement_Point_Round-SMD-Pad_Small
- U10, U8: footprint (none) -> KiMBo:DRY-DFN-6-1EP_2x2mm_Pitch0.5mm
- U7: footprint (none) -> KiMBo:DGN-MSOP-8_3x3mm_Pitch0.65mm
- U9: footprint (none) -> KiMBo:DCT-MSOP-8_3x3mm_Pitch0.65mm
Changed lines of the file:
@@
 F 0 "U9" H 7000 2647 60  0000 C CNN
 F 1 "74LVC2G241" H 7000 2541 60  0000 C CNN
-F 2 "" H 7050 1950 60  0001 C CNN
+F 2 "KiMBo:DCT-MSOP-8_3x3mm_Pitch0.65mm" H 7050 1950 60  0001 C CNN
 F 3 "" H 7050 1950 60  0001 C CNN
 	1    7000 2200
@@
 F 0 "U8" H 5675 4900 60  0000 C CNN
 F 1 "TPD4S012" H 5675 4500 60  0000 C CNN
-F 2 "" H 5650 4700 60  0001 C CNN
+F 2 "KiMBo:DRY-DFN-6-1EP_2x2mm_Pitch0.5mm" H 5650 4700 60  0001 C CNN
 F 3 "" H 5650 4700 60  0001 C CNN
 	1    5650 4700
@@
 F 0 "U7" H 4000 4647 60  0000 C CNN
 F 1 "TPS2051B" H 4000 4541 60  0000 C CNN
-F 2 "" H 4000 4200 60  0001 C CNN
+F 2 "KiMBo:DGN-MSOP-8_3x3mm_Pitch0.65mm" H 4000 4200 60  0001 C CNN
 F 3 "" H 4000 4200 60  0001 C CNN
 	1    4000 4250
@@
 F 0 "U10" H 8625 4547 60  0000 C CNN
 F 1 "TPD4S012" H 8625 4441 60  0000 C CNN
-F 2 "" H 8600 4200 60  0001 C CNN
+F 2 "KiMBo:DRY-DFN-6-1EP_2x2mm_Pitch0.5mm" H 8600 4200 60  0001 C CNN
 F 3 "" H 8600 4200 60  0001 C CNN
 	1    8600 4200
@@
 F 0 "TP6" H 6150 2500 50  0000 L CNN
 F 1 "Test_Point" H 6258 2329 50  0001 L CNN
-F 2 "" H 6400 2300 50  0001 C CNN
+F 2 "Measurement_Points:Measurement_Point_Round-SMD-Pad_Small" H 6400 2300 50  0001 C CNN
 F 3 "" H 6400 2300 50  0000 C CNN
 	1    6200 2300
