File: KiMBo/h_stepper.sch (KiCad schematic (older format))
At the start: 24 parts, among them U26 TMC2130

Commit message: Add equivalent annotations document, associate more footprints
Parts:
- C167: renamed from C165; footprint (none) -> Capacitors_SMD:C_0603
- C168: renamed from C166; footprint (none) -> Capacitors_SMD:C_0603
- C169: renamed from C167; footprint (none) -> Capacitors_SMD:C_0603
- C170: renamed from C168; footprint (none) -> Capacitors_SMD:C_0402
- C171: renamed from C169; footprint (none) -> Capacitors_SMD:C_0402
- C172: renamed from C170; footprint (none) -> Capacitors_SMD:C_0603
- C173: renamed from C171; footprint (none) -> Capacitors_SMD:C_0603
- C174: renamed from C172; footprint (none) -> Capacitors_SMD:C_0603
- C175: renamed from C173; footprint (none) -> Capacitors_SMD:C_0603
- C176: renamed from C174; footprint (none) -> Capacitors_SMD:C_0603
- C177: renamed from C175; footprint (none) -> Capacitors_SMD:C_0603
- C178: renamed from C176; footprint (none) -> Capacitors_SMD:C_0603
- C179: renamed from C177; footprint (none) -> Capacitors_SMD:C_0603
- C180: renamed from C178; value 4.7μF -> 10μF; footprint (none) -> Capacitors_SMD:C_0805
- C181: renamed from C179; footprint (none) -> Capacitors_SMD:c_elec_8x10
- C182: renamed from C180; footprint (none) -> Capacitors_SMD:C_0603
- renumbered R172 to R171, R173 to R172, R174 to R173, R175 to R174, R176 to R175, R177 to R176, R178 to R177
Changed lines of the file:
@@
 MOSI
 $Comp
-L C C167
+L C C169
 U 1 1 5BA7E11E
 P 7300 3950
-F 0 "C167" H 7186 3904 50  0000 R CNN
+F 0 "C169" H 7186 3904 50  0000 R CNN
 F 1 "100nF" H 7186 3995 50  0000 R CNN
-F 2 "" H 7338 3800 50  0001 C CNN
+F 2 "Capacitors_SMD:C_0603" H 7338 3800 50  0001 C CNN
 F 3 "" H 7300 3950 50  0000 C CNN
 	1    7300 3950
@@
 $EndComp
 $Comp
-L C C172
+L C C174
 U 1 1 589B8C70
 P 9100 4500
-F 0 "C172" V 9050 4400 50  0000 C CNN
+F 0 "C174" V 9050 4400 50  0000 C CNN
 F 1 "100nF" V 9050 4675 50  0000 C CNN
-F 2 "" H 9138 4350 50  0001 C CNN
+F 2 "Capacitors_SMD:C_0603" H 9138 4350 50  0001 C CNN
 F 3 "" H 9100 4500 50  0000 C CNN
 	1    9100 4500
@@
 $EndComp
 $Comp
-L CP1 C179
+L CP1 C181
 U 1 1 589B8CBD
 P 10450 3950
-F 0 "C179" H 10500 4050 50  0000 C CNN
+F 0 "C181" H 10550 4050 50  0000 C CNN
 F 1 "100μF" H 10600 3850 50  0000 C CNN
-F 2 "" H 10450 3950 50  0001 C CNN
+F 2 "Capacitors_SMD:c_elec_8x10" H 10450 3950 50  0001 C CNN
 F 3 "" H 10450 3950 50  0000 C CNN
 	1    10450 3950
@@
 $EndComp
 $Comp
-L C C175
+L C C177
 U 1 1 5BA7E121
 P 9550 3950
-F 0 "C175" H 9500 4050 50  0000 C CNN
+F 0 "C177" H 9450 4050 50  0000 C CNN
 F 1 "100nF" H 9425 3850 50  0000 C CNN
-F 2 "" H 9588 3800 50  0001 C CNN
+F 2 "Capacitors_SMD:C_0603" H 9588 3800 50  0001 C CNN
 F 3 "" H 9550 3950 50  0000 C CNN
 	1    9550 3950
@@
 $EndComp
 $Comp
-L GND #PWR0249
+L GND #PWR0250
 U 1 1 5BA7E122
 P 7300 4150
-F 0 "#PWR0249" H 7300 3900 50  0001 C CNN
+F 0 "#PWR0250" H 7300 3900 50  0001 C CNN
 F 1 "GND" H 7300 4000 50  0000 C CNN
 F 2 "" H 7300 4150 50  0000 C CNN
@@
 $EndComp
 $Comp
-L C C176
+L C C178
 U 1 1 5BA7E123
 P 9850 3950
-F 0 "C176" H 9800 4050 50  0000 C CNN
+F 0 "C178" H 9750 4050 50  0000 C CNN
 F 1 "100nF" H 9725 3850 50  0000 C CNN
-F 2 "" H 9888 3800 50  0001 C CNN
+F 2 "Capacitors_SMD:C_0603" H 9888 3800 50  0001 C CNN
 F 3 "" H 9850 3950 50  0000 C CNN
 	1    9850 3950
@@
 $EndComp
 $Comp
-L GND #PWR0250
+L GND #PWR0251
 U 1 1 5BA7E124
 P 10150 4200
-F 0 "#PWR0250" H 10150 3950 50  0001 C CNN
+F 0 "#PWR0251" H 10150 3950 50  0001 C CNN
 F 1 "GND" H 10155 4027 50  0000 C CNN
 F 2 "" H 10150 4200 50  0000 C CNN
@@
 $EndComp
 $Comp
-L +24V #PWR0251
+L +24V #PWR0252
 U 1 1 589BEDE1
 P 8350 3700
-F 0 "#PWR0251" H 8350 3550 50  0001 C CNN
+F 0 "#PWR0252" H 8350 3550 50  0001 C CNN
 F 1 "+24V" H 8365 3873 50  0000 C CNN
 F 2 "" H 8350 3700 50  0000 C CNN
@@
 $EndComp
 $Comp
-L C C169
+L C C171
 U 1 1 5BA7E126
 P 8950 5000
-F 0 "C169" H 9065 5046 50  0000 L CNN
+F 0 "C171" H 9065 5046 50  0000 L CNN
 F 1 "22nF" H 9065 4955 50  0000 L CNN
-F 2 "" H 8988 4850 50  0001 C CNN
+F 2 "Capacitors_SMD:C_0402" H 8988 4850 50  0001 C CNN
 F 3 "" H 8950 5000 50  0000 C CNN
 	1    8950 5000
@@
 $EndComp
 $Comp
-L R R178
+L R R177
 U 1 1 5BA7E127
 P 10550 7550
-F 0 "R178" H 10500 7500 50  0000 R CNN
+F 0 "R177" H 10500 7500 50  0000 R CNN
 F 1 "220mΩ" H 10500 7600 50  0000 R CNN
 F 2 "" V 10480 7550 50  0001 C CNN
@@
 $EndComp
 $Comp
-L R R177
+L R R176
 U 1 1 5BA7E128
 P 9750 7550
-F 0 "R177" H 9700 7500 50  0000 R CNN
+F 0 "R176" H 9700 7500 50  0000 R CNN
 F 1 "220mΩ" H 9700 7600 50  0000 R CNN
 F 2 "" V 9680 7550 50  0001 C CNN
@@
 $EndComp
 $Comp
-L GND #PWR0252
+L GND #PWR0253
 U 1 1 589C2B70
 P 9450 7900
-F 0 "#PWR0252" H 9450 7650 50  0001 C CNN
+F 0 "#PWR0253" H 9450 7650 50  0001 C CNN
 F 1 "GND" H 9455 7727 50  0000 C CNN
 F 2 "" H 9450 7900 50  0000 C CNN
@@
 NoConn ~ 7500 6450
 $Comp
-L R R174
+L R R173
 U 1 1 589C4ED8
 P 7100 4600
-F 0 "R174" V 7000 4600 50  0000 C CNN
+F 0 "R173" V 7000 4600 50  0000 C CNN
 F 1 "2.2Ω" V 7100 4600 50  0000 C CNN
 F 2 "" V 7030 4600 50  0001 C CNN
@@
 $EndComp
 $Comp
-L C C166
+L C C168
 U 1 1 5BA7E12C
 P 6900 4800
-F 0 "C166" H 6950 4900 50  0000 L CNN
+F 0 "C168" H 6950 4900 50  0000 L CNN
 F 1 "470nF" H 6925 4700 50  0000 L CNN
-F 2 "" H 6938 4650 50  0001 C CNN
+F 2 "Capacitors_SMD:C_0603" H 6938 4650 50  0001 C CNN
 F 3 "" H 6900 4800 50  0000 C CNN
 	1    6900 4800
@@
 NoConn ~ 7500 6550
 $Comp
-L GND #PWR0253
+L GND #PWR0254
 U 1 1 5BA7E12D
 P 7450 6950
-F 0 "#PWR0253" H 7450 6700 50  0001 C CNN
+F 0 "#PWR0254" H 7450 6700 50  0001 C CNN
 F 1 "GND" H 7455 6777 50  0000 C CNN
 F 2 "" H 7450 6950 50  0000 C CNN
@@
 $EndComp
 $Comp
-L C C177
+L C C179
 U 1 1 589CC9B9
 P 9900 7550
-F 0 "C177" H 9950 7650 50  0000 L CNN
+F 0 "C179" H 9950 7650 50  0000 L CNN
 F 1 "100nF" H 9950 7450 50  0000 L CNN
-F 2 "" H 9938 7400 50  0001 C CNN
+F 2 "Capacitors_SMD:C_0603" H 9938 7400 50  0001 C CNN
 F 3 "" H 9900 7550 50  0000 C CNN
 	1    9900 7550
@@
 H_FAULT
 $Comp
-L R R172
+L R R171
 U 1 1 5BA7E12F
 P 5850 5100
-F 0 "R172" H 5919 5146 50  0000 L CNN
+F 0 "R171" H 5919 5146 50  0000 L CNN
 F 1 "4.7kΩ" H 5919 5055 50  0000 L CNN
 F 2 "" V 5780 5100 50  0001 C CNN
@@
 NoConn ~ 7500 5400
 $Comp
-L C C168
+L C C170
 U 1 1 589C396E
 P 7300 4800
-F 0 "C168" H 7350 4900 50  0000 L CNN
+F 0 "C170" H 7350 4900 50  0000 L CNN
 F 1 "4.7μF" H 7350 4700 50  0000 L CNN
-F 2 "" H 7338 4650 50  0001 C CNN
+F 2 "Capacitors_SMD:C_0402" H 7338 4650 50  0001 C CNN
 F 3 "" H 7300 4800 50  0000 C CNN
 	1    7300 4800
@@
 5VOUT
 $Comp
-L R R175
+L R R174
 U 1 1 5BA7E130
 P 9050 7550
-F 0 "R175" H 9119 7596 50  0000 L CNN
+F 0 "R174" H 9119 7596 50  0000 L CNN
 F 1 "5.23kΩ" H 9119 7505 50  0000 L CNN
 F 2 "" V 8980 7550 50  0001 C CNN
@@
 5VOUT
 $Comp
-L R R176
+L R R175
 U 1 1 5BA7E131
 P 9250 7750
-F 0 "R176" V 9050 7750 50  0000 C CNN
+F 0 "R175" V 9050 7750 50  0000 C CNN
 F 1 "4.75kΩ" V 9150 7750 50  0000 C CNN
 F 2 "" V 9180 7750 50  0001 C CNN
@@
 $EndComp
 $Comp
-L R R173
+L R R172
 U 1 1 58A47723
 P 6200 5100
-F 0 "R173" H 6269 5146 50  0000 L CNN
+F 0 "R172" H 6269 5146 50  0000 L CNN
 F 1 "4.7kΩ" H 6269 5055 50  0000 L CNN
 F 2 "" V 6130 5100 50  0001 C CNN
@@
 $EndComp
 $Comp
-L C C180
+L C C182
 U 1 1 58AF169E
 P 10700 7550
-F 0 "C180" H 10750 7650 50  0000 L CNN
+F 0 "C182" H 10750 7650 50  0000 L CNN
 F 1 "100nF" H 10750 7450 50  0000 L CNN
-F 2 "" H 10738 7400 50  0001 C CNN
+F 2 "Capacitors_SMD:C_0603" H 10738 7400 50  0001 C CNN
 F 3 "" H 10700 7550 50  0000 C CNN
 	1    10700 7550
@@
 $EndComp
 $Comp
-L C C170
+L C C172
 U 1 1 58B19CCF
 P 8950 5800
-F 0 "C170" H 8975 5900 50  0000 L CNN
+F 0 "C172" H 8975 5900 50  0000 L CNN
 F 1 "470pF" H 8950 5700 50  0000 L CNN
-F 2 "" H 8988 5650 50  0001 C CNN
+F 2 "Capacitors_SMD:C_0603" H 8988 5650 50  0001 C CNN
 F 3 "" H 8950 5800 50  0000 C CNN
 	1    8950 5800
@@
 $EndComp
 $Comp
-L GND #PWR0254
+L GND #PWR0255
 U 1 1 5BA7E135
 P 9050 6050
-F 0 "#PWR0254" H 9050 5800 50  0001 C CNN
+F 0 "#PWR0255" H 9050 5800 50  0001 C CNN
 F 1 "GND" H 9050 5900 50  0000 C CNN
 F 2 "" H 9050 6050 50  0000 C CNN
@@
 $EndComp
 $Comp
-L C C173
+L C C175
 U 1 1 5BA7E136
 P 9150 5800
-F 0 "C173" H 9175 5900 50  0000 L CNN
+F 0 "C175" H 9175 5900 50  0000 L CNN
 F 1 "470pF" H 9175 5700 50  0000 L CNN
-F 2 "" H 9188 5650 50  0001 C CNN
+F 2 "Capacitors_SMD:C_0603" H 9188 5650 50  0001 C CNN
 F 3 "" H 9150 5800 50  0000 C CNN
 	1    9150 5800
@@
 $EndComp
 $Comp
-L C C171
+L C C173
 U 1 1 5BA7E137
 P 8950 6650
-F 0 "C171" H 8975 6750 50  0000 L CNN
+F 0 "C173" H 8975 6750 50  0000 L CNN
 F 1 "470pF" H 8950 6550 50  0000 L CNN
-F 2 "" H 8988 6500 50  0001 C CNN
+F 2 "Capacitors_SMD:C_0603" H 8988 6500 50  0001 C CNN
 F 3 "" H 8950 6650 50  0000 C CNN
 	1    8950 6650
@@
 $EndComp
 $Comp
-L GND #PWR0255
+L GND #PWR0256
 U 1 1 5BA7E138
 P 9050 6900
-F 0 "#PWR0255" H 9050 6650 50  0001 C CNN
+F 0 "#PWR0256" H 9050 6650 50  0001 C CNN
 F 1 "GND" H 9050 6750 50  0000 C CNN
 F 2 "" H 9050 6900 50  0000 C CNN
@@
 $EndComp
 $Comp
-L C C174
+L C C176
 U 1 1 5BA7E139
 P 9150 6650
-F 0 "C174" H 9175 6750 50  0000 L CNN
+F 0 "C176" H 9175 6750 50  0000 L CNN
 F 1 "470pF" H 9175 6550 50  0000 L CNN
-F 2 "" H 9188 6500 50  0001 C CNN
+F 2 "Capacitors_SMD:C_0603" H 9188 6500 50  0001 C CNN
 F 3 "" H 9150 6650 50  0000 C CNN
 	1    9150 6650
@@
 	8950 6850 8950 6800
 $Comp
-L C C178
+L C C180
 U 1 1 5BA7E13A
 P 10150 3950
-F 0 "C178" H 10100 4050 50  0000 C CNN
-F 1 "4.7μF" H 10025 3850 50  0000 C CNN
-F 2 "" H 10188 3800 50  0001 C CNN
+F 0 "C180" H 10050 4050 50  0000 C CNN
+F 1 "10μF" H 10025 3850 50  0000 C CNN
+F 2 "Capacitors_SMD:C_0805" H 10188 3800 50  0001 C CNN
 F 3 "" H 10150 3950 50  0000 C CNN
 	1    10150 3950
@@
 	5850 4350 7500 4350
 $Comp
-L VDD_3V3B #PWR0256
+L VDD_3V3B #PWR0257
 U 1 1 5A2FEA7A
 P 6550 4300
-F 0 "#PWR0256" H 6550 4150 50  0001 C CNN
+F 0 "#PWR0257" H 6550 4150 50  0001 C CNN
 F 1 "VDD_3V3B" H 6565 4473 50  0000 C CNN
 F 2 "" H 6550 4300 50  0000 C CNN
@@
 $EndComp
 $Comp
-L C C165
+L C C167
 U 1 1 5A897FB1
 P 6550 4800
-F 0 "C165" H 6600 4900 50  0000 L CNN
+F 0 "C167" H 6600 4900 50  0000 L CNN
 F 1 "100nF" H 6575 4700 50  0000 L CNN
-F 2 "" H 6588 4650 50  0001 C CNN
+F 2 "Capacitors_SMD:C_0603" H 6588 4650 50  0001 C CNN
 F 3 "" H 6550 4800 50  0000 C CNN
 	1    6550 4800

Commit message: Connect X and Z stepper driver open-drain DIAG0 and DIAG1 lines together
Parts:
- renumbered C167 to C165, C168 to C166, C169 to C167, C170 to C168, C171 to C169, C172 to C170, C173 to C171, C174 to C172, C175 to C173, C176 to C174, C177 to C175, C178 to C176, C179 to C177, C180 to C178, C181 to C179, C182 to C180, R171 to R167, R172 to R168, R173 to R169, R174 to R170, R175 to R171, R176 to R172, R177 to R173, U26 to U24
Changed lines of the file:
@@
 MOSI
 $Comp
-L C C169
+L C C167
 U 1 1 5BA7E11E
 P 7300 3950
-F 0 "C169" H 7186 3904 50  0000 R CNN
+F 0 "C167" H 7186 3904 50  0000 R CNN
 F 1 "100nF" H 7186 3995 50  0000 R CNN
 F 2 "Capacitors_SMD:C_0603" H 7338 3800 50  0001 C CNN
@@
 $EndComp
 $Comp
-L C C174
+L C C172
 U 1 1 589B8C70
 P 9100 4500
-F 0 "C174" V 9050 4400 50  0000 C CNN
+F 0 "C172" V 9050 4400 50  0000 C CNN
 F 1 "100nF" V 9050 4675 50  0000 C CNN
 F 2 "Capacitors_SMD:C_0603" H 9138 4350 50  0001 C CNN
@@
 $EndComp
 $Comp
-L CP1 C181
+L CP1 C179
 U 1 1 589B8CBD
 P 10450 3950
-F 0 "C181" H 10550 4050 50  0000 C CNN
+F 0 "C179" H 10550 4050 50  0000 C CNN
 F 1 "100μF" H 10600 3850 50  0000 C CNN
 F 2 "Capacitors_SMD:c_elec_8x10" H 10450 3950 50  0001 C CNN
@@
 $EndComp
 $Comp
-L C C177
+L C C175
 U 1 1 5BA7E121
 P 9550 3950
-F 0 "C177" H 9450 4050 50  0000 C CNN
+F 0 "C175" H 9450 4050 50  0000 C CNN
 F 1 "100nF" H 9425 3850 50  0000 C CNN
 F 2 "Capacitors_SMD:C_0603" H 9588 3800 50  0001 C CNN
@@
 $EndComp
 $Comp
-L GND #PWR0250
+L GND #PWR0240
 U 1 1 5BA7E122
 P 7300 4150
-F 0 "#PWR0250" H 7300 3900 50  0001 C CNN
+F 0 "#PWR0240" H 7300 3900 50  0001 C CNN
 F 1 "GND" H 7300 4000 50  0000 C CNN
 F 2 "" H 7300 4150 50  0000 C CNN
@@
 $EndComp
 $Comp
-L C C178
+L C C176
 U 1 1 5BA7E123
 P 9850 3950
-F 0 "C178" H 9750 4050 50  0000 C CNN
+F 0 "C176" H 9750 4050 50  0000 C CNN
 F 1 "100nF" H 9725 3850 50  0000 C CNN
 F 2 "Capacitors_SMD:C_0603" H 9888 3800 50  0001 C CNN
@@
 $EndComp
 $Comp
-L GND #PWR0251
+L GND #PWR0241
 U 1 1 5BA7E124
 P 10150 4200
-F 0 "#PWR0251" H 10150 3950 50  0001 C CNN
+F 0 "#PWR0241" H 10150 3950 50  0001 C CNN
 F 1 "GND" H 10155 4027 50  0000 C CNN
 F 2 "" H 10150 4200 50  0000 C CNN
@@
 $EndComp
 $Comp
-L +24V #PWR0252
+L +24V #PWR0242
 U 1 1 589BEDE1
 P 8350 3700
-F 0 "#PWR0252" H 8350 3550 50  0001 C CNN
+F 0 "#PWR0242" H 8350 3550 50  0001 C CNN
 F 1 "+24V" H 8365 3873 50  0000 C CNN
 F 2 "" H 8350 3700 50  0000 C CNN
@@
 $EndComp
 $Comp
-L C C171
+L C C169
 U 1 1 5BA7E126
 P 8950 5000
-F 0 "C171" H 9065 5046 50  0000 L CNN
+F 0 "C169" H 9065 5046 50  0000 L CNN
 F 1 "22nF" H 9065 4955 50  0000 L CNN
 F 2 "Capacitors_SMD:C_0402" H 8988 4850 50  0001 C CNN
@@
 $EndComp
 $Comp
-L R R177
+L R R173
 U 1 1 5BA7E127
 P 10550 7550
-F 0 "R177" H 10500 7500 50  0000 R CNN
+F 0 "R173" H 10500 7500 50  0000 R CNN
 F 1 "220mΩ" H 10500 7600 50  0000 R CNN
 F 2 "" V 10480 7550 50  0001 C CNN
@@
 $EndComp
 $Comp
-L R R176
+L R R172
 U 1 1 5BA7E128
 P 9750 7550
-F 0 "R176" H 9700 7500 50  0000 R CNN
+F 0 "R172" H 9700 7500 50  0000 R CNN
 F 1 "220mΩ" H 9700 7600 50  0000 R CNN
 F 2 "" V 9680 7550 50  0001 C CNN
@@
 $EndComp
 $Comp
-L GND #PWR0253
+L GND #PWR0243
 U 1 1 589C2B70
 P 9450 7900
-F 0 "#PWR0253" H 9450 7650 50  0001 C CNN
+F 0 "#PWR0243" H 9450 7650 50  0001 C CNN
 F 1 "GND" H 9455 7727 50  0000 C CNN
 F 2 "" H 9450 7900 50  0000 C CNN
@@
 NoConn ~ 7500 6450
 $Comp
-L R R173
+L R R169
 U 1 1 589C4ED8
 P 7100 4600
-F 0 "R173" V 7000 4600 50  0000 C CNN
+F 0 "R169" V 7000 4600 50  0000 C CNN
 F 1 "2.2Ω" V 7100 4600 50  0000 C CNN
 F 2 "" V 7030 4600 50  0001 C CNN
@@
 $EndComp
 $Comp
-L C C168
+L C C166
 U 1 1 5BA7E12C
 P 6900 4800
-F 0 "C168" H 6950 4900 50  0000 L CNN
+F 0 "C166" H 6950 4900 50  0000 L CNN
 F 1 "470nF" H 6925 4700 50  0000 L CNN
 F 2 "Capacitors_SMD:C_0603" H 6938 4650 50  0001 C CNN
@@
 NoConn ~ 7500 6550
 $Comp
-L GND #PWR0254
+L GND #PWR0244
 U 1 1 5BA7E12D
 P 7450 6950
-F 0 "#PWR0254" H 7450 6700 50  0001 C CNN
+F 0 "#PWR0244" H 7450 6700 50  0001 C CNN
 F 1 "GND" H 7455 6777 50  0000 C CNN
 F 2 "" H 7450 6950 50  0000 C CNN
@@
 $EndComp
 $Comp
-L C C179
+L C C177
 U 1 1 589CC9B9
 P 9900 7550
-F 0 "C179" H 9950 7650 50  0000 L CNN
+F 0 "C177" H 9950 7650 50  0000 L CNN
 F 1 "100nF" H 9950 7450 50  0000 L CNN
 F 2 "Capacitors_SMD:C_0603" H 9938 7400 50  0001 C CNN
@@
 H_FAULT
 $Comp
-L R R171
+L R R167
 U 1 1 5BA7E12F
 P 5850 5100
-F 0 "R171" H 5919 5146 50  0000 L CNN
+F 0 "R167" H 5919 5146 50  0000 L CNN
 F 1 "4.7kΩ" H 5919 5055 50  0000 L CNN
 F 2 "" V 5780 5100 50  0001 C CNN
@@
 NoConn ~ 7500 5400
 $Comp
-L C C170
+L C C168
 U 1 1 589C396E
 P 7300 4800
-F 0 "C170" H 7350 4900 50  0000 L CNN
+F 0 "C168" H 7350 4900 50  0000 L CNN
 F 1 "4.7μF" H 7350 4700 50  0000 L CNN
 F 2 "Capacitors_SMD:C_0402" H 7338 4650 50  0001 C CNN
@@
 5VOUT
 $Comp
-L R R174
+L R R170
 U 1 1 5BA7E130
 P 9050 7550
-F 0 "R174" H 9119 7596 50  0000 L CNN
+F 0 "R170" H 9119 7596 50  0000 L CNN
 F 1 "5.23kΩ" H 9119 7505 50  0000 L CNN
 F 2 "" V 8980 7550 50  0001 C CNN
@@
 5VOUT
 $Comp
-L R R175
+L R R171
 U 1 1 5BA7E131
 P 9250 7750
-F 0 "R175" V 9050 7750 50  0000 C CNN
+F 0 "R171" V 9050 7750 50  0000 C CNN
 F 1 "4.75kΩ" V 9150 7750 50  0000 C CNN
 F 2 "" V 9180 7750 50  0001 C CNN
@@
 $EndComp
 $Comp
-L R R172
+L R R168
 U 1 1 58A47723
 P 6200 5100
-F 0 "R172" H 6269 5146 50  0000 L CNN
+F 0 "R168" H 6269 5146 50  0000 L CNN
 F 1 "4.7kΩ" H 6269 5055 50  0000 L CNN
 F 2 "" V 6130 5100 50  0001 C CNN
@@
 $EndComp
 $Comp
-L C C182
+L C C180
 U 1 1 58AF169E
 P 10700 7550
-F 0 "C182" H 10750 7650 50  0000 L CNN
+F 0 "C180" H 10750 7650 50  0000 L CNN
 F 1 "100nF" H 10750 7450 50  0000 L CNN
 F 2 "Capacitors_SMD:C_0603" H 10738 7400 50  0001 C CNN
@@
 $EndComp
 $Comp
-L C C172
+L C C170
 U 1 1 58B19CCF
 P 8950 5800
-F 0 "C172" H 8975 5900 50  0000 L CNN
+F 0 "C170" H 8975 5900 50  0000 L CNN
 F 1 "470pF" H 8950 5700 50  0000 L CNN
 F 2 "Capacitors_SMD:C_0603" H 8988 5650 50  0001 C CNN
@@
 $EndComp
 $Comp
-L GND #PWR0255
+L GND #PWR0245
 U 1 1 5BA7E135
 P 9050 6050
-F 0 "#PWR0255" H 9050 5800 50  0001 C CNN
+F 0 "#PWR0245" H 9050 5800 50  0001 C CNN
 F 1 "GND" H 9050 5900 50  0000 C CNN
 F 2 "" H 9050 6050 50  0000 C CNN
@@
 $EndComp
 $Comp
-L C C175
+L C C173
 U 1 1 5BA7E136
 P 9150 5800
-F 0 "C175" H 9175 5900 50  0000 L CNN
+F 0 "C173" H 9175 5900 50  0000 L CNN
 F 1 "470pF" H 9175 5700 50  0000 L CNN
 F 2 "Capacitors_SMD:C_0603" H 9188 5650 50  0001 C CNN
@@
 $EndComp
 $Comp
-L C C173
+L C C171
 U 1 1 5BA7E137
 P 8950 6650
-F 0 "C173" H 8975 6750 50  0000 L CNN
+F 0 "C171" H 8975 6750 50  0000 L CNN
 F 1 "470pF" H 8950 6550 50  0000 L CNN
 F 2 "Capacitors_SMD:C_0603" H 8988 6500 50  0001 C CNN
@@
 $EndComp
 $Comp
-L GND #PWR0256
+L GND #PWR0246
 U 1 1 5BA7E138
 P 9050 6900
-F 0 "#PWR0256" H 9050 6650 50  0001 C CNN
+F 0 "#PWR0246" H 9050 6650 50  0001 C CNN
 F 1 "GND" H 9050 6750 50  0000 C CNN
 F 2 "" H 9050 6900 50  0000 C CNN
@@
 $EndComp
 $Comp
-L C C176
+L C C174
 U 1 1 5BA7E139
 P 9150 6650
-F 0 "C176" H 9175 6750 50  0000 L CNN
+F 0 "C174" H 9175 6750 50  0000 L CNN
 F 1 "470pF" H 9175 6550 50  0000 L CNN
 F 2 "Capacitors_SMD:C_0603" H 9188 6500 50  0001 C CNN
@@
 $EndComp
 $Comp
-L TMC2130 U26
+L TMC2130 U24
 U 1 1 589A7425
 P 8200 5550
-F 0 "U26" H 7750 7050 60  0000 C CNN
+F 0 "U24" H 7750 7050 60  0000 C CNN
 F 1 "TMC2130" H 8500 7050 60  0000 C CNN
 F 2 "" H 8200 5850 60  0001 C CNN
@@
 	8950 6850 8950 6800
 $Comp
-L C C180
+L C C178
 U 1 1 5BA7E13A
 P 10150 3950
-F 0 "C180" H 10050 4050 50  0000 C CNN
+F 0 "C178" H 10050 4050 50  0000 C CNN
 F 1 "10μF" H 10025 3850 50  0000 C CNN
 F 2 "Capacitors_SMD:C_0805" H 10188 3800 50  0001 C CNN
@@
 	5850 4350 7500 4350
 $Comp
-L VDD_3V3B #PWR0257
+L VDD_3V3B #PWR0247
 U 1 1 5A2FEA7A
 P 6550 4300
-F 0 "#PWR0257" H 6550 4150 50  0001 C CNN
+F 0 "#PWR0247" H 6550 4150 50  0001 C CNN
 F 1 "VDD_3V3B" H 6565 4473 50  0000 C CNN
 F 2 "" H 6550 4300 50  0000 C CNN
@@
 $EndComp
 $Comp
-L C C167
+L C C165
 U 1 1 5A897FB1
 P 6550 4800
-F 0 "C167" H 6600 4900 50  0000 L CNN
+F 0 "C165" H 6600 4900 50  0000 L CNN
 F 1 "100nF" H 6575 4700 50  0000 L CNN
 F 2 "Capacitors_SMD:C_0603" H 6588 4650 50  0001 C CNN

Commit message: Leave SPI0 free for a display, reassign pins so SPI1 is available
Fix some typos/errors
Parts:
- renumbered R167 to R169, R168 to R170, R169 to R171, R170 to R172, R171 to R173, R172 to R174, R173 to R175, U24 to U23
Changed lines of the file:
@@
 $EndComp
 $Comp
-L GND #PWR0240
+L GND #PWR0239
 U 1 1 5BA7E122
 P 7300 4150
-F 0 "#PWR0240" H 7300 3900 50  0001 C CNN
+F 0 "#PWR0239" H 7300 3900 50  0001 C CNN
 F 1 "GND" H 7300 4000 50  0000 C CNN
 F 2 "" H 7300 4150 50  0000 C CNN
@@
 $EndComp
 $Comp
-L GND #PWR0241
+L GND #PWR0240
 U 1 1 5BA7E124
 P 10150 4200
-F 0 "#PWR0241" H 10150 3950 50  0001 C CNN
+F 0 "#PWR0240" H 10150 3950 50  0001 C CNN
 F 1 "GND" H 10155 4027 50  0000 C CNN
 F 2 "" H 10150 4200 50  0000 C CNN
@@
 $EndComp
 $Comp
-L +24V #PWR0242
+L +24V #PWR0241
 U 1 1 589BEDE1
 P 8350 3700
-F 0 "#PWR0242" H 8350 3550 50  0001 C CNN
+F 0 "#PWR0241" H 8350 3550 50  0001 C CNN
 F 1 "+24V" H 8365 3873 50  0000 C CNN
 F 2 "" H 8350 3700 50  0000 C CNN
@@
 $EndComp
 $Comp
-L R R173
+L R R175
 U 1 1 5BA7E127
 P 10550 7550
-F 0 "R173" H 10500 7500 50  0000 R CNN
+F 0 "R175" H 10500 7500 50  0000 R CNN
 F 1 "220mΩ" H 10500 7600 50  0000 R CNN
 F 2 "" V 10480 7550 50  0001 C CNN
@@
 $EndComp
 $Comp
-L R R172
+L R R174
 U 1 1 5BA7E128
 P 9750 7550
-F 0 "R172" H 9700 7500 50  0000 R CNN
+F 0 "R174" H 9700 7500 50  0000 R CNN
 F 1 "220mΩ" H 9700 7600 50  0000 R CNN
 F 2 "" V 9680 7550 50  0001 C CNN
@@
 $EndComp
 $Comp
-L GND #PWR0243
+L GND #PWR0242
 U 1 1 589C2B70
 P 9450 7900
-F 0 "#PWR0243" H 9450 7650 50  0001 C CNN
+F 0 "#PWR0242" H 9450 7650 50  0001 C CNN
 F 1 "GND" H 9455 7727 50  0000 C CNN
 F 2 "" H 9450 7900 50  0000 C CNN
@@
 NoConn ~ 7500 6450
 $Comp
-L R R169
+L R R171
 U 1 1 589C4ED8
 P 7100 4600
-F 0 "R169" V 7000 4600 50  0000 C CNN
+F 0 "R171" V 7000 4600 50  0000 C CNN
 F 1 "2.2Ω" V 7100 4600 50  0000 C CNN
 F 2 "" V 7030 4600 50  0001 C CNN
@@
 NoConn ~ 7500 6550
 $Comp
-L GND #PWR0244
+L GND #PWR0243
 U 1 1 5BA7E12D
 P 7450 6950
-F 0 "#PWR0244" H 7450 6700 50  0001 C CNN
+F 0 "#PWR0243" H 7450 6700 50  0001 C CNN
 F 1 "GND" H 7455 6777 50  0000 C CNN
 F 2 "" H 7450 6950 50  0000 C CNN
@@
 H_FAULT
 $Comp
-L R R167
+L R R169
 U 1 1 5BA7E12F
 P 5850 5100
-F 0 "R167" H 5919 5146 50  0000 L CNN
+F 0 "R169" H 5919 5146 50  0000 L CNN
 F 1 "4.7kΩ" H 5919 5055 50  0000 L CNN
 F 2 "" V 5780 5100 50  0001 C CNN
@@
 5VOUT
 $Comp
-L R R170
+L R R172
 U 1 1 5BA7E130
 P 9050 7550
-F 0 "R170" H 9119 7596 50  0000 L CNN
+F 0 "R172" H 9119 7596 50  0000 L CNN
 F 1 "5.23kΩ" H 9119 7505 50  0000 L CNN
 F 2 "" V 8980 7550 50  0001 C CNN
@@
 5VOUT
 $Comp
-L R R171
+L R R173
 U 1 1 5BA7E131
 P 9250 7750
-F 0 "R171" V 9050 7750 50  0000 C CNN
+F 0 "R173" V 9050 7750 50  0000 C CNN
 F 1 "4.75kΩ" V 9150 7750 50  0000 C CNN
 F 2 "" V 9180 7750 50  0001 C CNN
@@
 $EndComp
 $Comp
-L R R168
+L R R170
 U 1 1 58A47723
 P 6200 5100
-F 0 "R168" H 6269 5146 50  0000 L CNN
+F 0 "R170" H 6269 5146 50  0000 L CNN
 F 1 "4.7kΩ" H 6269 5055 50  0000 L CNN
 F 2 "" V 6130 5100 50  0001 C CNN
@@
 $EndComp
 $Comp
-L GND #PWR0245
+L GND #PWR0244
 U 1 1 5BA7E135
 P 9050 6050
-F 0 "#PWR0245" H 9050 5800 50  0001 C CNN
+F 0 "#PWR0244" H 9050 5800 50  0001 C CNN
 F 1 "GND" H 9050 5900 50  0000 C CNN
 F 2 "" H 9050 6050 50  0000 C CNN
@@
 $EndComp
 $Comp
-L GND #PWR0246
+L GND #PWR0245
 U 1 1 5BA7E138
 P 9050 6900
-F 0 "#PWR0246" H 9050 6650 50  0001 C CNN
+F 0 "#PWR0245" H 9050 6650 50  0001 C CNN
 F 1 "GND" H 9050 6750 50  0000 C CNN
 F 2 "" H 9050 6900 50  0000 C CNN
@@
 $EndComp
 $Comp
-L TMC2130 U24
+L TMC2130 U23
 U 1 1 589A7425
 P 8200 5550
-F 0 "U24" H 7750 7050 60  0000 C CNN
+F 0 "U23" H 7750 7050 60  0000 C CNN
 F 1 "TMC2130" H 8500 7050 60  0000 C CNN
 F 2 "" H 8200 5850 60  0001 C CNN
@@
 	5850 4350 7500 4350
 $Comp
-L VDD_3V3B #PWR0247
+L VDD_3V3B #PWR0246
 U 1 1 5A2FEA7A
 P 6550 4300
-F 0 "#PWR0247" H 6550 4150 50  0001 C CNN
+F 0 "#PWR0246" H 6550 4150 50  0001 C CNN
 F 1 "VDD_3V3B" H 6565 4473 50  0000 C CNN
 F 2 "" H 6550 4300 50  0000 C CNN
