File: KiMBo/h_stepper.sch (KiCad schematic (older format))
At the start: 24 parts, among them U23 TMC2130

Commit message: Use fixed 5V LM2592HV Buck, include SPI0 header for LCD
Parts:
- renumbered C165 to C162, C166 to C163, C167 to C164, C168 to C165, C169 to C166, C170 to C167, C171 to C168, C172 to C169, C173 to C170, C174 to C171, C175 to C172, C176 to C173, C177 to C174, C178 to C175, C179 to C176, C180 to C177, R169 to R166, R170 to R167, R171 to R168, R172 to R169, R173 to R170, R174 to R171, R175 to R172
Changed lines of the file:
@@
 MOSI
 $Comp
-L C C167
+L C C164
 U 1 1 5BA7E11E
 P 7300 3950
-F 0 "C167" H 7186 3904 50  0000 R CNN
+F 0 "C164" H 7186 3904 50  0000 R CNN
 F 1 "100nF" H 7186 3995 50  0000 R CNN
 F 2 "Capacitors_SMD:C_0603" H 7338 3800 50  0001 C CNN
@@
 $EndComp
 $Comp
-L C C172
+L C C169
 U 1 1 589B8C70
 P 9100 4500
-F 0 "C172" V 9050 4400 50  0000 C CNN
+F 0 "C169" V 9050 4400 50  0000 C CNN
 F 1 "100nF" V 9050 4675 50  0000 C CNN
 F 2 "Capacitors_SMD:C_0603" H 9138 4350 50  0001 C CNN
@@
 $EndComp
 $Comp
-L CP1 C179
+L CP1 C176
 U 1 1 589B8CBD
 P 10450 3950
-F 0 "C179" H 10550 4050 50  0000 C CNN
+F 0 "C176" H 10550 4050 50  0000 C CNN
 F 1 "100μF" H 10600 3850 50  0000 C CNN
 F 2 "Capacitors_SMD:c_elec_8x10" H 10450 3950 50  0001 C CNN
@@
 $EndComp
 $Comp
-L C C175
+L C C172
 U 1 1 5BA7E121
 P 9550 3950
-F 0 "C175" H 9450 4050 50  0000 C CNN
+F 0 "C172" H 9450 4050 50  0000 C CNN
 F 1 "100nF" H 9425 3850 50  0000 C CNN
 F 2 "Capacitors_SMD:C_0603" H 9588 3800 50  0001 C CNN
@@
 $EndComp
 $Comp
-L GND #PWR0239
+L GND #PWR0234
 U 1 1 5BA7E122
 P 7300 4150
-F 0 "#PWR0239" H 7300 3900 50  0001 C CNN
+F 0 "#PWR0234" H 7300 3900 50  0001 C CNN
 F 1 "GND" H 7300 4000 50  0000 C CNN
 F 2 "" H 7300 4150 50  0000 C CNN
@@
 $EndComp
 $Comp
-L C C176
+L C C173
 U 1 1 5BA7E123
 P 9850 3950
-F 0 "C176" H 9750 4050 50  0000 C CNN
+F 0 "C173" H 9750 4050 50  0000 C CNN
 F 1 "100nF" H 9725 3850 50  0000 C CNN
 F 2 "Capacitors_SMD:C_0603" H 9888 3800 50  0001 C CNN
@@
 $EndComp
 $Comp
-L GND #PWR0240
+L GND #PWR0235
 U 1 1 5BA7E124
 P 10150 4200
-F 0 "#PWR0240" H 10150 3950 50  0001 C CNN
+F 0 "#PWR0235" H 10150 3950 50  0001 C CNN
 F 1 "GND" H 10155 4027 50  0000 C CNN
 F 2 "" H 10150 4200 50  0000 C CNN
@@
 $EndComp
 $Comp
-L +24V #PWR0241
+L +24V #PWR0236
 U 1 1 589BEDE1
 P 8350 3700
-F 0 "#PWR0241" H 8350 3550 50  0001 C CNN
+F 0 "#PWR0236" H 8350 3550 50  0001 C CNN
 F 1 "+24V" H 8365 3873 50  0000 C CNN
 F 2 "" H 8350 3700 50  0000 C CNN
@@
 $EndComp
 $Comp
-L C C169
+L C C166
 U 1 1 5BA7E126
 P 8950 5000
-F 0 "C169" H 9065 5046 50  0000 L CNN
+F 0 "C166" H 9065 5046 50  0000 L CNN
 F 1 "22nF" H 9065 4955 50  0000 L CNN
 F 2 "Capacitors_SMD:C_0402" H 8988 4850 50  0001 C CNN
@@
 $EndComp
 $Comp
-L R R175
+L R R172
 U 1 1 5BA7E127
 P 10550 7550
-F 0 "R175" H 10500 7500 50  0000 R CNN
+F 0 "R172" H 10500 7500 50  0000 R CNN
 F 1 "220mΩ" H 10500 7600 50  0000 R CNN
 F 2 "" V 10480 7550 50  0001 C CNN
@@
 $EndComp
 $Comp
-L R R174
+L R R171
 U 1 1 5BA7E128
 P 9750 7550
-F 0 "R174" H 9700 7500 50  0000 R CNN
+F 0 "R171" H 9700 7500 50  0000 R CNN
 F 1 "220mΩ" H 9700 7600 50  0000 R CNN
 F 2 "" V 9680 7550 50  0001 C CNN
@@
 $EndComp
 $Comp
-L GND #PWR0242
+L GND #PWR0237
 U 1 1 589C2B70
 P 9450 7900
-F 0 "#PWR0242" H 9450 7650 50  0001 C CNN
+F 0 "#PWR0237" H 9450 7650 50  0001 C CNN
 F 1 "GND" H 9455 7727 50  0000 C CNN
 F 2 "" H 9450 7900 50  0000 C CNN
@@
 NoConn ~ 7500 6450
 $Comp
-L R R171
+L R R168
 U 1 1 589C4ED8
 P 7100 4600
-F 0 "R171" V 7000 4600 50  0000 C CNN
+F 0 "R168" V 7000 4600 50  0000 C CNN
 F 1 "2.2Ω" V 7100 4600 50  0000 C CNN
 F 2 "" V 7030 4600 50  0001 C CNN
@@
 $EndComp
 $Comp
-L C C166
+L C C163
 U 1 1 5BA7E12C
 P 6900 4800
-F 0 "C166" H 6950 4900 50  0000 L CNN
+F 0 "C163" H 6950 4900 50  0000 L CNN
 F 1 "470nF" H 6925 4700 50  0000 L CNN
 F 2 "Capacitors_SMD:C_0603" H 6938 4650 50  0001 C CNN
@@
 NoConn ~ 7500 6550
 $Comp
-L GND #PWR0243
+L GND #PWR0238
 U 1 1 5BA7E12D
 P 7450 6950
-F 0 "#PWR0243" H 7450 6700 50  0001 C CNN
+F 0 "#PWR0238" H 7450 6700 50  0001 C CNN
 F 1 "GND" H 7455 6777 50  0000 C CNN
 F 2 "" H 7450 6950 50  0000 C CNN
@@
 $EndComp
 $Comp
-L C C177
+L C C174
 U 1 1 589CC9B9
 P 9900 7550
-F 0 "C177" H 9950 7650 50  0000 L CNN
+F 0 "C174" H 9950 7650 50  0000 L CNN
 F 1 "100nF" H 9950 7450 50  0000 L CNN
 F 2 "Capacitors_SMD:C_0603" H 9938 7400 50  0001 C CNN
@@
 H_FAULT
 $Comp
-L R R169
+L R R166
 U 1 1 5BA7E12F
 P 5850 5100
-F 0 "R169" H 5919 5146 50  0000 L CNN
+F 0 "R166" H 5919 5146 50  0000 L CNN
 F 1 "4.7kΩ" H 5919 5055 50  0000 L CNN
 F 2 "" V 5780 5100 50  0001 C CNN
@@
 NoConn ~ 7500 5400
 $Comp
-L C C168
+L C C165
 U 1 1 589C396E
 P 7300 4800
-F 0 "C168" H 7350 4900 50  0000 L CNN
+F 0 "C165" H 7350 4900 50  0000 L CNN
 F 1 "4.7μF" H 7350 4700 50  0000 L CNN
 F 2 "Capacitors_SMD:C_0402" H 7338 4650 50  0001 C CNN
@@
 5VOUT
 $Comp
-L R R172
+L R R169
 U 1 1 5BA7E130
 P 9050 7550
-F 0 "R172" H 9119 7596 50  0000 L CNN
+F 0 "R169" H 9119 7596 50  0000 L CNN
 F 1 "5.23kΩ" H 9119 7505 50  0000 L CNN
 F 2 "" V 8980 7550 50  0001 C CNN
@@
 5VOUT
 $Comp
-L R R173
+L R R170
 U 1 1 5BA7E131
 P 9250 7750
-F 0 "R173" V 9050 7750 50  0000 C CNN
+F 0 "R170" V 9050 7750 50  0000 C CNN
 F 1 "4.75kΩ" V 9150 7750 50  0000 C CNN
 F 2 "" V 9180 7750 50  0001 C CNN
@@
 $EndComp
 $Comp
-L R R170
+L R R167
 U 1 1 58A47723
 P 6200 5100
-F 0 "R170" H 6269 5146 50  0000 L CNN
+F 0 "R167" H 6269 5146 50  0000 L CNN
 F 1 "4.7kΩ" H 6269 5055 50  0000 L CNN
 F 2 "" V 6130 5100 50  0001 C CNN
@@
 $EndComp
 $Comp
-L C C180
+L C C177
 U 1 1 58AF169E
 P 10700 7550
-F 0 "C180" H 10750 7650 50  0000 L CNN
+F 0 "C177" H 10750 7650 50  0000 L CNN
 F 1 "100nF" H 10750 7450 50  0000 L CNN
 F 2 "Capacitors_SMD:C_0603" H 10738 7400 50  0001 C CNN
@@
 $EndComp
 $Comp
-L C C170
+L C C167
 U 1 1 58B19CCF
 P 8950 5800
-F 0 "C170" H 8975 5900 50  0000 L CNN
+F 0 "C167" H 8975 5900 50  0000 L CNN
 F 1 "470pF" H 8950 5700 50  0000 L CNN
 F 2 "Capacitors_SMD:C_0603" H 8988 5650 50  0001 C CNN
@@
 $EndComp
 $Comp
-L GND #PWR0244
+L GND #PWR0239
 U 1 1 5BA7E135
 P 9050 6050
-F 0 "#PWR0244" H 9050 5800 50  0001 C CNN
+F 0 "#PWR0239" H 9050 5800 50  0001 C CNN
 F 1 "GND" H 9050 5900 50  0000 C CNN
 F 2 "" H 9050 6050 50  0000 C CNN
@@
 $EndComp
 $Comp
-L C C173
+L C C170
 U 1 1 5BA7E136
 P 9150 5800
-F 0 "C173" H 9175 5900 50  0000 L CNN
+F 0 "C170" H 9175 5900 50  0000 L CNN
 F 1 "470pF" H 9175 5700 50  0000 L CNN
 F 2 "Capacitors_SMD:C_0603" H 9188 5650 50  0001 C CNN
@@
 $EndComp
 $Comp
-L C C171
+L C C168
 U 1 1 5BA7E137
 P 8950 6650
-F 0 "C171" H 8975 6750 50  0000 L CNN
+F 0 "C168" H 8975 6750 50  0000 L CNN
 F 1 "470pF" H 8950 6550 50  0000 L CNN
 F 2 "Capacitors_SMD:C_0603" H 8988 6500 50  0001 C CNN
@@
 $EndComp
 $Comp
-L GND #PWR0245
+L GND #PWR0240
 U 1 1 5BA7E138
 P 9050 6900
-F 0 "#PWR0245" H 9050 6650 50  0001 C CNN
+F 0 "#PWR0240" H 9050 6650 50  0001 C CNN
 F 1 "GND" H 9050 6750 50  0000 C CNN
 F 2 "" H 9050 6900 50  0000 C CNN
@@
 $EndComp
 $Comp
-L C C174
+L C C171
 U 1 1 5BA7E139
 P 9150 6650
-F 0 "C174" H 9175 6750 50  0000 L CNN
+F 0 "C171" H 9175 6750 50  0000 L CNN
 F 1 "470pF" H 9175 6550 50  0000 L CNN
 F 2 "Capacitors_SMD:C_0603" H 9188 6500 50  0001 C CNN
@@
 	8950 6850 8950 6800
 $Comp
-L C C178
+L C C175
 U 1 1 5BA7E13A
 P 10150 3950
-F 0 "C178" H 10050 4050 50  0000 C CNN
+F 0 "C175" H 10050 4050 50  0000 C CNN
 F 1 "10μF" H 10025 3850 50  0000 C CNN
 F 2 "Capacitors_SMD:C_0805" H 10188 3800 50  0001 C CNN
@@
 	5850 4350 7500 4350
 $Comp
-L VDD_3V3B #PWR0246
+L VDD_3V3B #PWR0241
 U 1 1 5A2FEA7A
 P 6550 4300
-F 0 "#PWR0246" H 6550 4150 50  0001 C CNN
+F 0 "#PWR0241" H 6550 4150 50  0001 C CNN
 F 1 "VDD_3V3B" H 6565 4473 50  0000 C CNN
 F 2 "" H 6550 4300 50  0000 C CNN
@@
 $EndComp
 $Comp
-L C C165
+L C C162
 U 1 1 5A897FB1
 P 6550 4800
-F 0 "C165" H 6600 4900 50  0000 L CNN
+F 0 "C162" H 6600 4900 50  0000 L CNN
 F 1 "100nF" H 6575 4700 50  0000 L CNN
 F 2 "Capacitors_SMD:C_0603" H 6588 4650 50  0001 C CNN

Commit message: Assocate more footprints
Parts:
- C165, C166: footprint Capacitors_SMD:C_0402 -> Capacitors_SMD:C_0603
- R166, R167, R168, R169, R170: footprint (none) -> Resistors_SMD:R_0603
Changed lines of the file:
@@
 F 0 "C166" H 9065 5046 50  0000 L CNN
 F 1 "22nF" H 9065 4955 50  0000 L CNN
-F 2 "Capacitors_SMD:C_0402" H 8988 4850 50  0001 C CNN
+F 2 "Capacitors_SMD:C_0603" H 8988 4850 50  0001 C CNN
 F 3 "" H 8950 5000 50  0000 C CNN
 	1    8950 5000
@@
 F 0 "R168" V 7000 4600 50  0000 C CNN
 F 1 "2.2Ω" V 7100 4600 50  0000 C CNN
-F 2 "" V 7030 4600 50  0001 C CNN
+F 2 "Resistors_SMD:R_0603" V 7030 4600 50  0001 C CNN
 F 3 "" H 7100 4600 50  0000 C CNN
 	1    7100 4600
@@
 F 0 "R166" H 5919 5146 50  0000 L CNN
 F 1 "4.7kΩ" H 5919 5055 50  0000 L CNN
-F 2 "" V 5780 5100 50  0001 C CNN
+F 2 "Resistors_SMD:R_0603" V 5780 5100 50  0001 C CNN
 F 3 "" H 5850 5100 50  0000 C CNN
 	1    5850 5100
@@
 F 0 "C165" H 7350 4900 50  0000 L CNN
 F 1 "4.7μF" H 7350 4700 50  0000 L CNN
-F 2 "Capacitors_SMD:C_0402" H 7338 4650 50  0001 C CNN
+F 2 "Capacitors_SMD:C_0603" H 7338 4650 50  0001 C CNN
 F 3 "" H 7300 4800 50  0000 C CNN
 	1    7300 4800
@@
 F 0 "R169" H 9119 7596 50  0000 L CNN
 F 1 "5.23kΩ" H 9119 7505 50  0000 L CNN
-F 2 "" V 8980 7550 50  0001 C CNN
+F 2 "Resistors_SMD:R_0603" V 8980 7550 50  0001 C CNN
 F 3 "" H 9050 7550 50  0000 C CNN
 	1    9050 7550
@@
 F 0 "R170" V 9050 7750 50  0000 C CNN
 F 1 "4.75kΩ" V 9150 7750 50  0000 C CNN
-F 2 "" V 9180 7750 50  0001 C CNN
+F 2 "Resistors_SMD:R_0603" V 9180 7750 50  0001 C CNN
 F 3 "" H 9250 7750 50  0000 C CNN
 	1    9250 7750
@@
 F 0 "R167" H 6269 5146 50  0000 L CNN
 F 1 "4.7kΩ" H 6269 5055 50  0000 L CNN
-F 2 "" V 6130 5100 50  0001 C CNN
+F 2 "Resistors_SMD:R_0603" V 6130 5100 50  0001 C CNN
 F 3 "" H 6200 5100 50  0000 C CNN
 	1    6200 5100

Commit message: More footprint association
Parts:
- R171, R172: footprint (none) -> Resistors_SMD:R_0805
- U23: footprint (none) -> KiMBo:QFN36_5X6
Changed lines of the file:
@@
 $EndComp
 $Comp
-L GND #PWR0234
+L GND #PWR0235
 U 1 1 5BA7E122
 P 7300 4150
-F 0 "#PWR0234" H 7300 3900 50  0001 C CNN
+F 0 "#PWR0235" H 7300 3900 50  0001 C CNN
 F 1 "GND" H 7300 4000 50  0000 C CNN
 F 2 "" H 7300 4150 50  0000 C CNN
@@
 $EndComp
 $Comp
-L GND #PWR0235
+L GND #PWR0236
 U 1 1 5BA7E124
 P 10150 4200
-F 0 "#PWR0235" H 10150 3950 50  0001 C CNN
+F 0 "#PWR0236" H 10150 3950 50  0001 C CNN
 F 1 "GND" H 10155 4027 50  0000 C CNN
 F 2 "" H 10150 4200 50  0000 C CNN
@@
 $EndComp
 $Comp
-L +24V #PWR0236
+L +24V #PWR0237
 U 1 1 589BEDE1
 P 8350 3700
-F 0 "#PWR0236" H 8350 3550 50  0001 C CNN
+F 0 "#PWR0237" H 8350 3550 50  0001 C CNN
 F 1 "+24V" H 8365 3873 50  0000 C CNN
 F 2 "" H 8350 3700 50  0000 C CNN
@@
 F 0 "R172" H 10500 7500 50  0000 R CNN
 F 1 "220mΩ" H 10500 7600 50  0000 R CNN
-F 2 "" V 10480 7550 50  0001 C CNN
+F 2 "Resistors_SMD:R_0805" V 10480 7550 50  0001 C CNN
 F 3 "" H 10550 7550 50  0000 C CNN
 	1    10550 7550
@@
 F 0 "R171" H 9700 7500 50  0000 R CNN
 F 1 "220mΩ" H 9700 7600 50  0000 R CNN
-F 2 "" V 9680 7550 50  0001 C CNN
+F 2 "Resistors_SMD:R_0805" V 9680 7550 50  0001 C CNN
 F 3 "" H 9750 7550 50  0000 C CNN
 	1    9750 7550
@@
 $EndComp
 $Comp
-L GND #PWR0237
+L GND #PWR0238
 U 1 1 589C2B70
 P 9450 7900
-F 0 "#PWR0237" H 9450 7650 50  0001 C CNN
+F 0 "#PWR0238" H 9450 7650 50  0001 C CNN
 F 1 "GND" H 9455 7727 50  0000 C CNN
 F 2 "" H 9450 7900 50  0000 C CNN
@@
 NoConn ~ 7500 6550
 $Comp
-L GND #PWR0238
+L GND #PWR0239
 U 1 1 5BA7E12D
 P 7450 6950
-F 0 "#PWR0238" H 7450 6700 50  0001 C CNN
+F 0 "#PWR0239" H 7450 6700 50  0001 C CNN
 F 1 "GND" H 7455 6777 50  0000 C CNN
 F 2 "" H 7450 6950 50  0000 C CNN
@@
 $EndComp
 $Comp
-L GND #PWR0239
+L GND #PWR0240
 U 1 1 5BA7E135
 P 9050 6050
-F 0 "#PWR0239" H 9050 5800 50  0001 C CNN
+F 0 "#PWR0240" H 9050 5800 50  0001 C CNN
 F 1 "GND" H 9050 5900 50  0000 C CNN
 F 2 "" H 9050 6050 50  0000 C CNN
@@
 $EndComp
 $Comp
-L GND #PWR0240
+L GND #PWR0241
 U 1 1 5BA7E138
 P 9050 6900
-F 0 "#PWR0240" H 9050 6650 50  0001 C CNN
+F 0 "#PWR0241" H 9050 6650 50  0001 C CNN
 F 1 "GND" H 9050 6750 50  0000 C CNN
 F 2 "" H 9050 6900 50  0000 C CNN
@@
 F 0 "U23" H 7750 7050 60  0000 C CNN
 F 1 "TMC2130" H 8500 7050 60  0000 C CNN
-F 2 "" H 8200 5850 60  0001 C CNN
+F 2 "KiMBo:QFN36_5X6" H 8200 5850 60  0001 C CNN
 F 3 "" H 8200 5850 60  0000 C CNN
 	1    8200 5550
@@
 	5850 4350 7500 4350
 $Comp
-L VDD_3V3B #PWR0241
+L VDD_3V3B #PWR0242
 U 1 1 5A2FEA7A
 P 6550 4300
-F 0 "#PWR0241" H 6550 4150 50  0001 C CNN
+F 0 "#PWR0242" H 6550 4150 50  0001 C CNN
 F 1 "VDD_3V3B" H 6565 4473 50  0000 C CNN
 F 2 "" H 6550 4300 50  0000 C CNN

Commit message: Add more footprints and more associations, one association left!
Parts:
- R179: renamed from R170; footprint Resistors_SMD:R_0603 -> Resistors_SMD:R_0805
- R181: renamed from R172; footprint Resistors_SMD:R_0805 -> Resistors_SMD:R_0603
- renumbered R166 to R175, R167 to R176, R168 to R177, R169 to R178, R171 to R180
Changed lines of the file:
@@
 $EndComp
 $Comp
-L GND #PWR0235
+L GND #PWR0237
 U 1 1 5BA7E122
 P 7300 4150
-F 0 "#PWR0235" H 7300 3900 50  0001 C CNN
+F 0 "#PWR0237" H 7300 3900 50  0001 C CNN
 F 1 "GND" H 7300 4000 50  0000 C CNN
 F 2 "" H 7300 4150 50  0000 C CNN
@@
 $EndComp
 $Comp
-L GND #PWR0236
+L GND #PWR0238
 U 1 1 5BA7E124
 P 10150 4200
-F 0 "#PWR0236" H 10150 3950 50  0001 C CNN
+F 0 "#PWR0238" H 10150 3950 50  0001 C CNN
 F 1 "GND" H 10155 4027 50  0000 C CNN
 F 2 "" H 10150 4200 50  0000 C CNN
@@
 $EndComp
 $Comp
-L +24V #PWR0237
+L +24V #PWR0239
 U 1 1 589BEDE1
 P 8350 3700
-F 0 "#PWR0237" H 8350 3550 50  0001 C CNN
+F 0 "#PWR0239" H 8350 3550 50  0001 C CNN
 F 1 "+24V" H 8365 3873 50  0000 C CNN
 F 2 "" H 8350 3700 50  0000 C CNN
@@
 $EndComp
 $Comp
-L R R172
+L R R181
 U 1 1 5BA7E127
 P 10550 7550
-F 0 "R172" H 10500 7500 50  0000 R CNN
+F 0 "R181" H 10500 7500 50  0000 R CNN
 F 1 "220mΩ" H 10500 7600 50  0000 R CNN
-F 2 "Resistors_SMD:R_0805" V 10480 7550 50  0001 C CNN
+F 2 "Resistors_SMD:R_0603" V 10480 7550 50  0001 C CNN
 F 3 "" H 10550 7550 50  0000 C CNN
 	1    10550 7550
@@
 $EndComp
 $Comp
-L R R171
+L R R180
 U 1 1 5BA7E128
 P 9750 7550
-F 0 "R171" H 9700 7500 50  0000 R CNN
+F 0 "R180" H 9700 7500 50  0000 R CNN
 F 1 "220mΩ" H 9700 7600 50  0000 R CNN
 F 2 "Resistors_SMD:R_0805" V 9680 7550 50  0001 C CNN
@@
 $EndComp
 $Comp
-L GND #PWR0238
+L GND #PWR0240
 U 1 1 589C2B70
 P 9450 7900
-F 0 "#PWR0238" H 9450 7650 50  0001 C CNN
+F 0 "#PWR0240" H 9450 7650 50  0001 C CNN
 F 1 "GND" H 9455 7727 50  0000 C CNN
 F 2 "" H 9450 7900 50  0000 C CNN
@@
 NoConn ~ 7500 6450
 $Comp
-L R R168
+L R R177
 U 1 1 589C4ED8
 P 7100 4600
-F 0 "R168" V 7000 4600 50  0000 C CNN
+F 0 "R177" V 7000 4600 50  0000 C CNN
 F 1 "2.2Ω" V 7100 4600 50  0000 C CNN
 F 2 "Resistors_SMD:R_0603" V 7030 4600 50  0001 C CNN
@@
 NoConn ~ 7500 6550
 $Comp
-L GND #PWR0239
+L GND #PWR0241
 U 1 1 5BA7E12D
 P 7450 6950
-F 0 "#PWR0239" H 7450 6700 50  0001 C CNN
+F 0 "#PWR0241" H 7450 6700 50  0001 C CNN
 F 1 "GND" H 7455 6777 50  0000 C CNN
 F 2 "" H 7450 6950 50  0000 C CNN
@@
 H_FAULT
 $Comp
-L R R166
+L R R175
 U 1 1 5BA7E12F
 P 5850 5100
-F 0 "R166" H 5919 5146 50  0000 L CNN
+F 0 "R175" H 5919 5146 50  0000 L CNN
 F 1 "4.7kΩ" H 5919 5055 50  0000 L CNN
 F 2 "Resistors_SMD:R_0603" V 5780 5100 50  0001 C CNN
@@
 5VOUT
 $Comp
-L R R169
+L R R178
 U 1 1 5BA7E130
 P 9050 7550
-F 0 "R169" H 9119 7596 50  0000 L CNN
+F 0 "R178" H 9119 7596 50  0000 L CNN
 F 1 "5.23kΩ" H 9119 7505 50  0000 L CNN
 F 2 "Resistors_SMD:R_0603" V 8980 7550 50  0001 C CNN
@@
 5VOUT
 $Comp
-L R R170
+L R R179
 U 1 1 5BA7E131
 P 9250 7750
-F 0 "R170" V 9050 7750 50  0000 C CNN
+F 0 "R179" V 9050 7750 50  0000 C CNN
 F 1 "4.75kΩ" V 9150 7750 50  0000 C CNN
-F 2 "Resistors_SMD:R_0603" V 9180 7750 50  0001 C CNN
+F 2 "Resistors_SMD:R_0805" V 9180 7750 50  0001 C CNN
 F 3 "" H 9250 7750 50  0000 C CNN
 	1    9250 7750
@@
 $EndComp
 $Comp
-L R R167
+L R R176
 U 1 1 58A47723
 P 6200 5100
-F 0 "R167" H 6269 5146 50  0000 L CNN
+F 0 "R176" H 6269 5146 50  0000 L CNN
 F 1 "4.7kΩ" H 6269 5055 50  0000 L CNN
 F 2 "Resistors_SMD:R_0603" V 6130 5100 50  0001 C CNN
@@
 $EndComp
 $Comp
-L GND #PWR0240
+L GND #PWR0242
 U 1 1 5BA7E135
 P 9050 6050
-F 0 "#PWR0240" H 9050 5800 50  0001 C CNN
+F 0 "#PWR0242" H 9050 5800 50  0001 C CNN
 F 1 "GND" H 9050 5900 50  0000 C CNN
 F 2 "" H 9050 6050 50  0000 C CNN
@@
 $EndComp
 $Comp
-L GND #PWR0241
+L GND #PWR0243
 U 1 1 5BA7E138
 P 9050 6900
-F 0 "#PWR0241" H 9050 6650 50  0001 C CNN
+F 0 "#PWR0243" H 9050 6650 50  0001 C CNN
 F 1 "GND" H 9050 6750 50  0000 C CNN
 F 2 "" H 9050 6900 50  0000 C CNN
@@
 	5850 4350 7500 4350
 $Comp
-L VDD_3V3B #PWR0242
+L VDD_3V3B #PWR0244
 U 1 1 5A2FEA7A
 P 6550 4300
-F 0 "#PWR0242" H 6550 4150 50  0001 C CNN
+F 0 "#PWR0244" H 6550 4150 50  0001 C CNN
 F 1 "VDD_3V3B" H 6565 4473 50  0000 C CNN
 F 2 "" H 6550 4300 50  0000 C CNN

Commit message: Begin layout
Arrange all connectors to get a feel for the area.
Parts:
- renumbered C162 to C164, C163 to C165, C164 to C166, C165 to C167, C166 to C168, C167 to C169, C168 to C170, C169 to C171, C170 to C172, C171 to C173, C172 to C174, C173 to C175, C174 to C176, C175 to C177, C176 to C178, C177 to C179
Changed lines of the file:
@@
 MOSI
 $Comp
-L C C164
+L C C166
 U 1 1 5BA7E11E
 P 7300 3950
-F 0 "C164" H 7186 3904 50  0000 R CNN
+F 0 "C166" H 7186 3904 50  0000 R CNN
 F 1 "100nF" H 7186 3995 50  0000 R CNN
 F 2 "Capacitors_SMD:C_0603" H 7338 3800 50  0001 C CNN
@@
 $EndComp
 $Comp
-L C C169
+L C C171
 U 1 1 589B8C70
 P 9100 4500
-F 0 "C169" V 9050 4400 50  0000 C CNN
+F 0 "C171" V 9050 4400 50  0000 C CNN
 F 1 "100nF" V 9050 4675 50  0000 C CNN
 F 2 "Capacitors_SMD:C_0603" H 9138 4350 50  0001 C CNN
@@
 $EndComp
 $Comp
-L CP1 C176
+L CP1 C178
 U 1 1 589B8CBD
 P 10450 3950
-F 0 "C176" H 10550 4050 50  0000 C CNN
+F 0 "C178" H 10550 4050 50  0000 C CNN
 F 1 "100μF" H 10600 3850 50  0000 C CNN
 F 2 "Capacitors_SMD:c_elec_8x10" H 10450 3950 50  0001 C CNN
@@
 $EndComp
 $Comp
-L C C172
+L C C174
 U 1 1 5BA7E121
 P 9550 3950
-F 0 "C172" H 9450 4050 50  0000 C CNN
+F 0 "C174" H 9450 4050 50  0000 C CNN
 F 1 "100nF" H 9425 3850 50  0000 C CNN
 F 2 "Capacitors_SMD:C_0603" H 9588 3800 50  0001 C CNN
@@
 $EndComp
 $Comp
-L GND #PWR0237
+L GND #PWR0240
 U 1 1 5BA7E122
 P 7300 4150
-F 0 "#PWR0237" H 7300 3900 50  0001 C CNN
+F 0 "#PWR0240" H 7300 3900 50  0001 C CNN
 F 1 "GND" H 7300 4000 50  0000 C CNN
 F 2 "" H 7300 4150 50  0000 C CNN
@@
 $EndComp
 $Comp
-L C C173
+L C C175
 U 1 1 5BA7E123
 P 9850 3950
-F 0 "C173" H 9750 4050 50  0000 C CNN
+F 0 "C175" H 9750 4050 50  0000 C CNN
 F 1 "100nF" H 9725 3850 50  0000 C CNN
 F 2 "Capacitors_SMD:C_0603" H 9888 3800 50  0001 C CNN
@@
 $EndComp
 $Comp
-L GND #PWR0238
+L GND #PWR0241
 U 1 1 5BA7E124
 P 10150 4200
-F 0 "#PWR0238" H 10150 3950 50  0001 C CNN
+F 0 "#PWR0241" H 10150 3950 50  0001 C CNN
 F 1 "GND" H 10155 4027 50  0000 C CNN
 F 2 "" H 10150 4200 50  0000 C CNN
@@
 $EndComp
 $Comp
-L +24V #PWR0239
+L +24V #PWR0242
 U 1 1 589BEDE1
 P 8350 3700
-F 0 "#PWR0239" H 8350 3550 50  0001 C CNN
+F 0 "#PWR0242" H 8350 3550 50  0001 C CNN
 F 1 "+24V" H 8365 3873 50  0000 C CNN
 F 2 "" H 8350 3700 50  0000 C CNN
@@
 $EndComp
 $Comp
-L C C166
+L C C168
 U 1 1 5BA7E126
 P 8950 5000
-F 0 "C166" H 9065 5046 50  0000 L CNN
+F 0 "C168" H 9065 5046 50  0000 L CNN
 F 1 "22nF" H 9065 4955 50  0000 L CNN
 F 2 "Capacitors_SMD:C_0603" H 8988 4850 50  0001 C CNN
@@
 $EndComp
 $Comp
-L GND #PWR0240
+L GND #PWR0243
 U 1 1 589C2B70
 P 9450 7900
-F 0 "#PWR0240" H 9450 7650 50  0001 C CNN
+F 0 "#PWR0243" H 9450 7650 50  0001 C CNN
 F 1 "GND" H 9455 7727 50  0000 C CNN
 F 2 "" H 9450 7900 50  0000 C CNN
@@
 $EndComp
 $Comp
-L C C163
+L C C165
 U 1 1 5BA7E12C
 P 6900 4800
-F 0 "C163" H 6950 4900 50  0000 L CNN
+F 0 "C165" H 6950 4900 50  0000 L CNN
 F 1 "470nF" H 6925 4700 50  0000 L CNN
 F 2 "Capacitors_SMD:C_0603" H 6938 4650 50  0001 C CNN
@@
 NoConn ~ 7500 6550
 $Comp
-L GND #PWR0241
+L GND #PWR0244
 U 1 1 5BA7E12D
 P 7450 6950
-F 0 "#PWR0241" H 7450 6700 50  0001 C CNN
+F 0 "#PWR0244" H 7450 6700 50  0001 C CNN
 F 1 "GND" H 7455 6777 50  0000 C CNN
 F 2 "" H 7450 6950 50  0000 C CNN
@@
 $EndComp
 $Comp
-L C C174
+L C C176
 U 1 1 589CC9B9
 P 9900 7550
-F 0 "C174" H 9950 7650 50  0000 L CNN
+F 0 "C176" H 9950 7650 50  0000 L CNN
 F 1 "100nF" H 9950 7450 50  0000 L CNN
 F 2 "Capacitors_SMD:C_0603" H 9938 7400 50  0001 C CNN
@@
 NoConn ~ 7500 5400
 $Comp
-L C C165
+L C C167
 U 1 1 589C396E
 P 7300 4800
-F 0 "C165" H 7350 4900 50  0000 L CNN
+F 0 "C167" H 7350 4900 50  0000 L CNN
 F 1 "4.7μF" H 7350 4700 50  0000 L CNN
 F 2 "Capacitors_SMD:C_0603" H 7338 4650 50  0001 C CNN
@@
 $EndComp
 $Comp
-L C C177
+L C C179
 U 1 1 58AF169E
 P 10700 7550
-F 0 "C177" H 10750 7650 50  0000 L CNN
+F 0 "C179" H 10750 7650 50  0000 L CNN
 F 1 "100nF" H 10750 7450 50  0000 L CNN
 F 2 "Capacitors_SMD:C_0603" H 10738 7400 50  0001 C CNN
@@
 $EndComp
 $Comp
-L C C167
+L C C169
 U 1 1 58B19CCF
 P 8950 5800
-F 0 "C167" H 8975 5900 50  0000 L CNN
+F 0 "C169" H 8975 5900 50  0000 L CNN
 F 1 "470pF" H 8950 5700 50  0000 L CNN
 F 2 "Capacitors_SMD:C_0603" H 8988 5650 50  0001 C CNN
@@
 $EndComp
 $Comp
-L GND #PWR0242
+L GND #PWR0245
 U 1 1 5BA7E135
 P 9050 6050
-F 0 "#PWR0242" H 9050 5800 50  0001 C CNN
+F 0 "#PWR0245" H 9050 5800 50  0001 C CNN
 F 1 "GND" H 9050 5900 50  0000 C CNN
 F 2 "" H 9050 6050 50  0000 C CNN
@@
 $EndComp
 $Comp
-L C C170
+L C C172
 U 1 1 5BA7E136
 P 9150 5800
-F 0 "C170" H 9175 5900 50  0000 L CNN
+F 0 "C172" H 9175 5900 50  0000 L CNN
 F 1 "470pF" H 9175 5700 50  0000 L CNN
 F 2 "Capacitors_SMD:C_0603" H 9188 5650 50  0001 C CNN
@@
 $EndComp
 $Comp
-L C C168
+L C C170
 U 1 1 5BA7E137
 P 8950 6650
-F 0 "C168" H 8975 6750 50  0000 L CNN
+F 0 "C170" H 8975 6750 50  0000 L CNN
 F 1 "470pF" H 8950 6550 50  0000 L CNN
 F 2 "Capacitors_SMD:C_0603" H 8988 6500 50  0001 C CNN
@@
 $EndComp
 $Comp
-L GND #PWR0243
+L GND #PWR0246
 U 1 1 5BA7E138
 P 9050 6900
-F 0 "#PWR0243" H 9050 6650 50  0001 C CNN
+F 0 "#PWR0246" H 9050 6650 50  0001 C CNN
 F 1 "GND" H 9050 6750 50  0000 C CNN
 F 2 "" H 9050 6900 50  0000 C CNN
@@
 $EndComp
 $Comp
-L C C171
+L C C173
 U 1 1 5BA7E139
 P 9150 6650
-F 0 "C171" H 9175 6750 50  0000 L CNN
+F 0 "C173" H 9175 6750 50  0000 L CNN
 F 1 "470pF" H 9175 6550 50  0000 L CNN
 F 2 "Capacitors_SMD:C_0603" H 9188 6500 50  0001 C CNN
@@
 	8950 6850 8950 6800
 $Comp
-L C C175
+L C C177
 U 1 1 5BA7E13A
 P 10150 3950
-F 0 "C175" H 10050 4050 50  0000 C CNN
+F 0 "C177" H 10050 4050 50  0000 C CNN
 F 1 "10μF" H 10025 3850 50  0000 C CNN
 F 2 "Capacitors_SMD:C_0805" H 10188 3800 50  0001 C CNN
@@
 	5850 4350 7500 4350
 $Comp
-L VDD_3V3B #PWR0244
+L VDD_3V3B #PWR0247
 U 1 1 5A2FEA7A
 P 6550 4300
-F 0 "#PWR0244" H 6550 4150 50  0001 C CNN
+F 0 "#PWR0247" H 6550 4150 50  0001 C CNN
 F 1 "VDD_3V3B" H 6565 4473 50  0000 C CNN
 F 2 "" H 6550 4300 50  0000 C CNN
@@
 $EndComp
 $Comp
-L C C162
+L C C164
 U 1 1 5A897FB1
 P 6550 4800
-F 0 "C162" H 6600 4900 50  0000 L CNN
+F 0 "C164" H 6600 4900 50  0000 L CNN
 F 1 "100nF" H 6575 4700 50  0000 L CNN
 F 2 "Capacitors_SMD:C_0603" H 6588 4650 50  0001 C CNN
