File: KiMBo/hdmi.sch (KiCad schematic (older format))
At the start: 41 parts, among them U13 TDA19988BHN/C1,557, U14 IP4283CZ10-TBR, U15 IP4283CZ10-TBR, U2 OSD3358

Commit message: Associate more footprints
Parts:
- C44, C46, C51, C57: footprint (none) -> Capacitors_SMD:C_0402
- C45, C60: footprint (none) -> Capacitors_SMD:C_0805
- C48, C54: footprint (none) -> Capacitors_SMD:C_0603
Changed lines of the file:
@@
 F 0 "C44" H 1715 1496 50  0000 L CNN
 F 1 "100nF" H 1715 1405 50  0000 L CNN
-F 2 "" H 1600 1450 50  0001 C CNN
+F 2 "Capacitors_SMD:C_0402" H 1600 1450 50  0001 C CNN
 F 3 "" H 1600 1450 50  0000 C CNN
 	1    1600 1450
@@
 F 0 "C45" H 2015 1746 50  0000 L CNN
 F 1 "2.2μF" H 1975 1650 50  0000 L CNN
-F 2 "" H 1900 1700 50  0001 C CNN
+F 2 "Capacitors_SMD:C_0805" H 1900 1700 50  0001 C CNN
 F 3 "" H 1900 1700 50  0000 C CNN
 	1    1900 1700
@@
 F 0 "C46" H 2315 1496 50  0000 L CNN
 F 1 "100nF" H 2260 1420 50  0000 L CNN
-F 2 "" H 2200 1450 50  0001 C CNN
+F 2 "Capacitors_SMD:C_0402" H 2200 1450 50  0001 C CNN
 F 3 "" H 2200 1450 50  0000 C CNN
 	1    2200 1450
@@
 F 0 "C48" H 2615 1746 50  0000 L CNN
 F 1 "2.2μF" H 2575 1650 50  0000 L CNN
-F 2 "" H 2500 1700 50  0001 C CNN
+F 2 "Capacitors_SMD:C_0603" H 2500 1700 50  0001 C CNN
 F 3 "" H 2500 1700 50  0000 C CNN
 	1    2500 1700
@@
 F 0 "C51" H 2915 1496 50  0000 L CNN
 F 1 "100nF" H 2860 1420 50  0000 L CNN
-F 2 "" H 2800 1450 50  0001 C CNN
+F 2 "Capacitors_SMD:C_0402" H 2800 1450 50  0001 C CNN
 F 3 "" H 2800 1450 50  0000 C CNN
 	1    2800 1450
@@
 F 0 "C54" H 3215 1746 50  0000 L CNN
 F 1 "2.2μF" H 3175 1650 50  0000 L CNN
-F 2 "" H 3100 1700 50  0001 C CNN
+F 2 "Capacitors_SMD:C_0603" H 3100 1700 50  0001 C CNN
 F 3 "" H 3100 1700 50  0000 C CNN
 	1    3100 1700
@@
 F 0 "C57" H 3515 1496 50  0000 L CNN
 F 1 "100nF" H 3460 1420 50  0000 L CNN
-F 2 "" H 3400 1450 50  0001 C CNN
+F 2 "Capacitors_SMD:C_0402" H 3400 1450 50  0001 C CNN
 F 3 "" H 3400 1450 50  0000 C CNN
 	1    3400 1450
@@
 F 0 "C60" H 3815 1746 50  0000 L CNN
 F 1 "2.2μF" H 3775 1650 50  0000 L CNN
-F 2 "" H 3700 1700 50  0001 C CNN
+F 2 "Capacitors_SMD:C_0805" H 3700 1700 50  0001 C CNN
 F 3 "" H 3700 1700 50  0000 C CNN
 	1    3700 1700

Commit message: Add equivalent annotations document, associate more footprints
Parts:
- C47, C49, C50, C52, C53, C55, C56, C58, C59, C61, C62, C63, C64, C65, C66, C67: footprint (none) -> Capacitors_SMD:C_0402
- R100: renamed from R101; footprint (none) -> Resistors_SMD:R_0402
- R91: renamed from R92; footprint (none) -> Resistors_SMD:R_0402
- R92: renamed from R93; footprint (none) -> Resistors_SMD:R_0402
- R93: renamed from R94; footprint (none) -> Resistors_SMD:R_0402
- R94: renamed from R95; footprint (none) -> Resistors_SMD:R_0402
- R95: renamed from R96; footprint (none) -> Resistors_SMD:R_0402
- R96: renamed from R97; footprint (none) -> Resistors_SMD:R_0402
- R97: renamed from R98; footprint (none) -> Resistors_SMD:R_0402
- R98: renamed from R99; footprint (none) -> Resistors_SMD:R_0402
- R99: renamed from R100; footprint (none) -> Resistors_SMD:R_0402

Commit message: Leave SPI0 free for a display, reassign pins so SPI1 is available
Fix some typos/errors
Parts:
- renumbered R98 to R100, R99 to R101, R100 to R102, R91 to R93, R92 to R94, R93 to R95, R94 to R96, R95 to R97, R96 to R98, R97 to R99, U2 to U1, U13 to U12, U14 to U13, U15 to U14
Changed lines of the file:
@@
 $EndDescr
 $Comp
-L TDA19988BHN/C1,557 U13
+L TDA19988BHN/C1,557 U12
 U 1 1 5895FD47
 P 6400 2700
-F 0 "U13" H 6300 2700 60  0000 L CNN
+F 0 "U12" H 6300 2700 60  0000 L CNN
 F 1 "TDA19988BHN/C1,557" H 5800 2600 60  0000 L CNN
 F 2 "" H 5850 2850 60  0001 C CNN
@@
 $EndComp
 $Comp
-L GND #PWR0149
+L GND #PWR0148
 U 1 1 5896044E
 P 4200 2800
-F 0 "#PWR0149" H 4200 2550 50  0001 C CNN
+F 0 "#PWR0148" H 4200 2550 50  0001 C CNN
 F 1 "GND" H 4200 2650 50  0000 C CNN
 F 2 "" H 4200 2800 50  0000 C CNN
@@
 HDMI
 $Comp
-L GND #PWR0150
+L GND #PWR0149
 U 1 1 5898A6BE
 P 5100 4200
-F 0 "#PWR0150" H 5100 3950 50  0001 C CNN
+F 0 "#PWR0149" H 5100 3950 50  0001 C CNN
 F 1 "GND" H 5100 4050 50  0000 C CNN
 F 2 "" H 5100 4200 50  0000 C CNN
@@
 $EndComp
 $Comp
-L R R96
+L R R98
 U 1 1 5898DA3A
 P 7500 4650
-F 0 "R96" V 7350 4650 50  0000 C CNN
+F 0 "R98" V 7350 4650 50  0000 C CNN
 F 1 "27kΩ" V 7425 4650 50  0000 C CNN
 F 2 "Resistors_SMD:R_0402" V 7430 4650 50  0001 C CNN
@@
 HPD
 $Comp
-L R R99
+L R R101
 U 1 1 5898E81F
 P 8150 4150
-F 0 "R99" V 7943 4150 50  0000 C CNN
+F 0 "R101" V 7943 4150 50  0000 C CNN
 F 1 "1.5kΩ" V 8034 4150 50  0000 C CNN
 F 2 "Resistors_SMD:R_0402" V 8080 4150 50  0001 C CNN
@@
 $EndComp
 $Comp
-L R R98
+L R R100
 U 1 1 5898E892
 P 8150 3800
-F 0 "R98" V 7943 3800 50  0000 C CNN
+F 0 "R100" V 7943 3800 50  0000 C CNN
 F 1 "1.5kΩ" V 8034 3800 50  0000 C CNN
 F 2 "Resistors_SMD:R_0402" V 8080 3800 50  0001 C CNN
@@
 $EndComp
 $Comp
-L GND #PWR0151
+L GND #PWR0150
 U 1 1 58990275
 P 5400 1250
-F 0 "#PWR0151" H 5400 1000 50  0001 C CNN
+F 0 "#PWR0150" H 5400 1000 50  0001 C CNN
 F 1 "GND" H 5400 1100 50  0000 C CNN
 F 2 "" H 5400 1250 50  0000 C CNN
@@
 $EndComp
 $Comp
-L GND #PWR0152
+L GND #PWR0151
 U 1 1 58990A45
 P 5850 1050
-F 0 "#PWR0152" H 5850 800 50  0001 C CNN
+F 0 "#PWR0151" H 5850 800 50  0001 C CNN
 F 1 "GND" H 5850 900 50  0000 C CNN
 F 2 "" H 5850 1050 50  0000 C CNN
@@
 LCD.D15.R4--R7
 $Comp
-L GND #PWR0153
+L GND #PWR0152
 U 1 1 589952D6
 P 6850 1050
-F 0 "#PWR0153" H 6850 800 50  0001 C CNN
+F 0 "#PWR0152" H 6850 800 50  0001 C CNN
 F 1 "GND" H 6850 900 50  0000 C CNN
 F 2 "" H 6850 1050 50  0000 C CNN
@@
 $EndComp
 $Comp
-L R R97
+L R R99
 U 1 1 58996377
 P 7600 1250
-F 0 "R97" V 7393 1250 50  0000 C CNN
+F 0 "R99" V 7393 1250 50  0000 C CNN
 F 1 "0Ω" V 7484 1250 50  0000 C CNN
 F 2 "Resistors_SMD:R_0402" V 7530 1250 50  0001 C CNN
@@
 TEST
 $Comp
-L GND #PWR0154
+L GND #PWR0153
 U 1 1 58996432
 P 7800 1300
-F 0 "#PWR0154" H 7800 1050 50  0001 C CNN
+F 0 "#PWR0153" H 7800 1050 50  0001 C CNN
 F 1 "GND" H 7800 1150 50  0000 C CNN
 F 2 "" H 7800 1300 50  0000 C CNN
@@
 $EndComp
 $Comp
-L R R95
+L R R97
 U 1 1 58996A35
 P 7350 1050
-F 0 "R95" V 7143 1050 50  0000 C CNN
+F 0 "R97" V 7143 1050 50  0000 C CNN
 F 1 "10kΩ" V 7234 1050 50  0000 C CNN
 F 2 "Resistors_SMD:R_0402" V 7280 1050 50  0001 C CNN
@@
 $EndComp
 $Comp
-L R R100
+L R R102
 U 1 1 5899782C
 P 8300 3350
-F 0 "R100" V 8093 3350 50  0000 C CNN
+F 0 "R102" V 8093 3350 50  0000 C CNN
 F 1 "10kΩ" V 8184 3350 50  0000 C CNN
 F 2 "Resistors_SMD:R_0402" V 8230 3350 50  0001 C CNN
@@
 $EndComp
 $Comp
-L GND #PWR0155
+L GND #PWR0154
 U 1 1 589978DF
 P 8550 3600
-F 0 "#PWR0155" H 8550 3350 50  0001 C CNN
+F 0 "#PWR0154" H 8550 3350 50  0001 C CNN
 F 1 "GND" H 8550 3450 50  0000 C CNN
 F 2 "" H 8550 3600 50  0000 C CNN
@@
 EXT_SWING
 $Comp
-L IP4283CZ10-TBR U14
+L IP4283CZ10-TBR U13
 U 1 1 589AA3AA
 P 9550 3950
-F 0 "U14" V 9200 3700 60  0000 L CNN
+F 0 "U13" V 9200 3700 60  0000 L CNN
 F 1 "IP4283CZ10-TBR" V 9900 3550 60  0000 L CNN
 F 2 "" H 9600 4250 60  0001 C CNN
@@
 $EndComp
 $Comp
-L IP4283CZ10-TBR U15
+L IP4283CZ10-TBR U14
 U 1 1 589AA56A
 P 10350 3950
-F 0 "U15" V 10000 3700 60  0000 L CNN
+F 0 "U14" V 10000 3700 60  0000 L CNN
 F 1 "IP4283CZ10-TBR" V 10700 3550 60  0000 L CNN
 F 2 "" H 10400 4250 60  0001 C CNN
@@
 $EndComp
 $Comp
-L GND #PWR0156
+L GND #PWR0155
 U 1 1 589AAAC6
 P 10350 4400
-F 0 "#PWR0156" H 10350 4150 50  0001 C CNN
+F 0 "#PWR0155" H 10350 4150 50  0001 C CNN
 F 1 "GND" H 10355 4227 50  0000 C CNN
 F 2 "" H 10350 4400 50  0000 C CNN
@@
 $EndComp
 $Comp
-L GND #PWR0157
+L GND #PWR0156
 U 1 1 589AAAF2
 P 9550 4400
-F 0 "#PWR0157" H 9550 4150 50  0001 C CNN
+F 0 "#PWR0156" H 9550 4150 50  0001 C CNN
 F 1 "GND" H 9555 4227 50  0000 C CNN
 F 2 "" H 9550 4400 50  0000 C CNN
@@
 $EndComp
 $Comp
-L GND #PWR0158
+L GND #PWR0157
 U 1 1 589B56E5
 P 3600 7500
-F 0 "#PWR0158" H 3600 7250 50  0001 C CNN
+F 0 "#PWR0157" H 3600 7250 50  0001 C CNN
 F 1 "GND" H 3605 7327 50  0000 C CNN
 F 2 "" H 3600 7500 50  0000 C CNN
@@
 SPI1_SCLK
 $Comp
-L VDD_3V3B #PWR0159
+L VDD_3V3B #PWR0158
 U 1 1 5A077125
 P 7550 1000
-F 0 "#PWR0159" H 7550 850 50  0001 C CNN
+F 0 "#PWR0158" H 7550 850 50  0001 C CNN
 F 1 "VDD_3V3B" H 7650 1150 50  0000 C CNN
 F 2 "" H 7550 1000 50  0000 C CNN
@@
 $EndComp
 $Comp
-L VDD_3V3B #PWR0160
+L VDD_3V3B #PWR0159
 U 1 1 5A078B10
 P 7700 4600
-F 0 "#PWR0160" H 7700 4450 50  0001 C CNN
+F 0 "#PWR0159" H 7700 4450 50  0001 C CNN
 F 1 "VDD_3V3B" H 7715 4773 50  0000 C CNN
 F 2 "" H 7700 4600 50  0000 C CNN
@@
 $EndComp
 $Comp
-L SYS_5V #PWR0161
+L SYS_5V #PWR0160
 U 1 1 5A079ADB
 P 9800 1600
-F 0 "#PWR0161" H 9800 1450 50  0001 C CNN
+F 0 "#PWR0160" H 9800 1450 50  0001 C CNN
 F 1 "SYS_5V" H 9815 1773 50  0000 C CNN
 F 2 "" H 9800 1600 50  0000 C CNN
@@
 $EndComp
 $Comp
-L HDMI_1V8 #PWR0162
+L HDMI_1V8 #PWR0161
 U 1 1 5A07ADDF
 P 4200 2300
-F 0 "#PWR0162" H 4200 2150 50  0001 C CNN
+F 0 "#PWR0161" H 4200 2150 50  0001 C CNN
 F 1 "HDMI_1V8" H 4200 2450 50  0000 C CNN
 F 2 "" H 4200 2300 50  0000 C CNN
@@
 $EndComp
 $Comp
-L HDMI_1V8 #PWR0163
+L HDMI_1V8 #PWR0162
 U 1 1 5A07B406
 P 4200 3200
-F 0 "#PWR0163" H 4200 3050 50  0001 C CNN
+F 0 "#PWR0162" H 4200 3050 50  0001 C CNN
 F 1 "HDMI_1V8" H 4200 3350 50  0000 C CNN
 F 2 "" H 4200 3200 50  0000 C CNN
@@
 $EndComp
 $Comp
-L HDMI_1V8 #PWR0164
+L HDMI_1V8 #PWR0163
 U 1 1 5A07C429
 P 7800 2000
-F 0 "#PWR0164" H 7800 1850 50  0001 C CNN
+F 0 "#PWR0163" H 7800 1850 50  0001 C CNN
 F 1 "HDMI_1V8" H 7800 2150 50  0000 C CNN
 F 2 "" H 7800 2000 50  0000 C CNN
@@
 $EndComp
 $Comp
-L HDMI_1V8 #PWR0165
+L HDMI_1V8 #PWR0164
 U 1 1 5A07C4AF
 P 8550 2600
-F 0 "#PWR0165" H 8550 2450 50  0001 C CNN
+F 0 "#PWR0164" H 8550 2450 50  0001 C CNN
 F 1 "HDMI_1V8" H 8750 2700 50  0000 C CNN
 F 2 "" H 8550 2600 50  0000 C CNN
@@
 $EndComp
 $Comp
-L HDMI_1V8 #PWR0166
+L HDMI_1V8 #PWR0165
 U 1 1 5A07C535
 P 8550 3200
-F 0 "#PWR0166" H 8550 3050 50  0001 C CNN
+F 0 "#PWR0165" H 8550 3050 50  0001 C CNN
 F 1 "HDMI_1V8" H 8750 3300 50  0000 C CNN
 F 2 "" H 8550 3200 50  0000 C CNN
@@
 $EndComp
 $Comp
-L HDMI_1V8 #PWR0167
+L HDMI_1V8 #PWR0166
 U 1 1 5A0922CB
 P 6750 4850
-F 0 "#PWR0167" H 6750 4700 50  0001 C CNN
+F 0 "#PWR0166" H 6750 4700 50  0001 C CNN
 F 1 "HDMI_1V8" H 6650 5000 50  0000 C CNN
 F 2 "" H 6750 4850 50  0000 C CNN
@@
 $EndComp
 $Comp
-L HDMI_1V8 #PWR0168
+L HDMI_1V8 #PWR0167
 U 1 1 5A094D61
 P 2500 1200
-F 0 "#PWR0168" H 2500 1050 50  0001 C CNN
+F 0 "#PWR0167" H 2500 1050 50  0001 C CNN
 F 1 "HDMI_1V8" H 2515 1373 50  0000 C CNN
 F 2 "" H 2500 1200 50  0000 C CNN
@@
 $EndComp
 $Comp
-L PWR_FLAG #FLG0169
+L PWR_FLAG #FLG0168
 U 1 1 5A0B0393
 P 1900 1200
-F 0 "#FLG0169" H 1900 1295 50  0001 C CNN
+F 0 "#FLG0168" H 1900 1295 50  0001 C CNN
 F 1 "PWR_FLAG" H 1900 1424 50  0000 C CNN
 F 2 "" H 1900 1200 50  0000 C CNN
@@
 $EndComp
 $Comp
-L VDD_1V8 #PWR0170
+L VDD_1V8 #PWR0169
 U 1 1 5A0B0EAC
 P 1050 1200
-F 0 "#PWR0170" H 1050 1050 50  0001 C CNN
+F 0 "#PWR0169" H 1050 1050 50  0001 C CNN
 F 1 "VDD_1V8" H 1065 1373 50  0000 C CNN
 F 2 "" H 1050 1200 50  0000 C CNN
@@
 P 400 6300
 AR Path="/581AEC7B/5AD9EF75" Ref="U?"  Part="4"
-AR Path="/58958D2E/5AD9EF75" Ref="U2"  Part="4"
-F 0 "U2" H 1105 6590 60  0000 C CNN
+AR Path="/58958D2E/5AD9EF75" Ref="U1"  Part="4"
+F 0 "U1" H 1105 6590 60  0000 C CNN
 F 1 "OSD3358" H 1105 6484 60  0000 C CNN
 F 2 "" H 400 6300 60  0001 C CNN
@@
 MCUJ_CD.HS
 $Comp
-L R R94
+L R R96
 U 1 1 5ADA169F
 P 2450 4700
-F 0 "R94" V 2500 4525 50  0000 C CNN
+F 0 "R96" V 2500 4525 50  0000 C CNN
 F 1 "0Ω" V 2500 4900 50  0000 C CNN
 F 2 "Resistors_SMD:R_0402" V 2380 4700 50  0001 C CNN
@@
 $EndComp
 $Comp
-L R R93
+L R R95
 U 1 1 5ADA16A6
 P 2450 4600
-F 0 "R93" V 2500 4425 50  0000 C CNN
+F 0 "R95" V 2500 4425 50  0000 C CNN
 F 1 "0Ω" V 2500 4800 50  0000 C CNN
 F 2 "Resistors_SMD:R_0402" V 2380 4600 50  0001 C CNN
@@
 $EndComp
 $Comp
-L R R92
+L R R94
 U 1 1 5ADA16AD
 P 2450 4500
-F 0 "R92" V 2500 4325 50  0000 C CNN
+F 0 "R94" V 2500 4325 50  0000 C CNN
 F 1 "0Ω" V 2500 4700 50  0000 C CNN
 F 2 "Resistors_SMD:R_0402" V 2380 4500 50  0001 C CNN
@@
 $EndComp
 $Comp
-L R R91
+L R R93
 U 1 1 5ADA16B4
 P 2450 4400
-F 0 "R91" V 2500 4225 50  0000 C CNN
+F 0 "R93" V 2500 4225 50  0000 C CNN
 F 1 "22Ω" V 2500 4600 50  0000 C CNN
 F 2 "Resistors_SMD:R_0402" V 2380 4400 50  0001 C CNN
@@
 HDMI_INT
 $Comp
-L VDD_1V8 #PWR0171
+L VDD_1V8 #PWR0170
 U 1 1 5BC7F01E
 P 6650 1100
-F 0 "#PWR0171" H 6650 950 50  0001 C CNN
+F 0 "#PWR0170" H 6650 950 50  0001 C CNN
 F 1 "VDD_1V8" H 6725 1250 50  0000 C CNN
 F 2 "" H 6650 1100 50  0000 C CNN

Commit message: Use fixed 5V LM2592HV Buck, include SPI0 header for LCD
Parts:
- renumbered C44 to C41, C45 to C42, C46 to C43, C47 to C44, C48 to C45, C49 to C46, C50 to C47, C51 to C48, C52 to C49, C53 to C50, C54 to C51, C55 to C52, C56 to C53, C57 to C54, C58 to C55, C59 to C56, C60 to C57, C61 to C58, C62 to C59, C63 to C60, C64 to C61, C65 to C62, C66 to C63, C67 to C64, FB24 to FB29, R93 to R90, R94 to R91, R95 to R92, R96 to R93, R97 to R94, R98 to R95, R99 to R96, R100 to R97, R101 to R98, R102 to R99

Commit message: Assocate more footprints
Parts:
- C41, C43, C44, C46, C47, C48, C49, C50, C52, C53, C54, C55, C56, C58, C59, C60, C61, C62, C63, C64: footprint Capacitors_SMD:C_0402 -> Capacitors_SMD:C_0603
- FB29: value BLM18BD252SN1D -> ?H
- R90, R91, R92, R93, R94, R95, R96, R97, R98, R99: footprint Resistors_SMD:R_0402 -> Resistors_SMD:R_0603
- U1: footprint (none) -> KiMBo:BGA-400-1-27mm
- renumbered D14 to D15
Changed lines of the file:
@@
 NoConn ~ 6750 4100
 $Comp
-L D_Schottky D14
+L D_Schottky D15
 U 1 1 5898D395
 P 7150 4650
-F 0 "D14" H 7150 4866 50  0000 C CNN
+F 0 "D15" H 7150 4866 50  0000 C CNN
 F 1 "RB751V40,115" H 7150 4775 50  0000 C CNN
 F 2 "" H 7150 4650 50  0001 C CNN
@@
 F 0 "R95" V 7350 4650 50  0000 C CNN
 F 1 "27kΩ" V 7425 4650 50  0000 C CNN
-F 2 "Resistors_SMD:R_0402" V 7430 4650 50  0001 C CNN
+F 2 "Resistors_SMD:R_0603" V 7430 4650 50  0001 C CNN
 F 3 "" H 7500 4650 50  0000 C CNN
 	1    7500 4650
@@
 F 0 "R98" V 7943 4150 50  0000 C CNN
 F 1 "1.5kΩ" V 8034 4150 50  0000 C CNN
-F 2 "Resistors_SMD:R_0402" V 8080 4150 50  0001 C CNN
+F 2 "Resistors_SMD:R_0603" V 8080 4150 50  0001 C CNN
 F 3 "" H 8150 4150 50  0000 C CNN
 	1    8150 4150
@@
 F 0 "R97" V 7943 3800 50  0000 C CNN
 F 1 "1.5kΩ" V 8034 3800 50  0000 C CNN
-F 2 "Resistors_SMD:R_0402" V 8080 3800 50  0001 C CNN
+F 2 "Resistors_SMD:R_0603" V 8080 3800 50  0001 C CNN
 F 3 "" H 8150 3800 50  0000 C CNN
 	1    8150 3800
@@
 F 0 "R96" V 7393 1250 50  0000 C CNN
 F 1 "0Ω" V 7484 1250 50  0000 C CNN
-F 2 "Resistors_SMD:R_0402" V 7530 1250 50  0001 C CNN
+F 2 "Resistors_SMD:R_0603" V 7530 1250 50  0001 C CNN
 F 3 "" H 7600 1250 50  0000 C CNN
 	1    7600 1250
@@
 F 0 "R94" V 7143 1050 50  0000 C CNN
 F 1 "10kΩ" V 7234 1050 50  0000 C CNN
-F 2 "Resistors_SMD:R_0402" V 7280 1050 50  0001 C CNN
+F 2 "Resistors_SMD:R_0603" V 7280 1050 50  0001 C CNN
 F 3 "" H 7350 1050 50  0000 C CNN
 	1    7350 1050
@@
 F 0 "R99" V 8093 3350 50  0000 C CNN
 F 1 "10kΩ" V 8184 3350 50  0000 C CNN
-F 2 "Resistors_SMD:R_0402" V 8230 3350 50  0001 C CNN
+F 2 "Resistors_SMD:R_0603" V 8230 3350 50  0001 C CNN
 F 3 "" H 8300 3350 50  0000 C CNN
 	1    8300 3350
@@
 F 0 "C44" H 2515 6546 50  0000 L CNN
 F 1 "47pF" H 2515 6455 50  0000 L CNN
-F 2 "Capacitors_SMD:C_0402" H 2400 6500 50  0001 C CNN
+F 2 "Capacitors_SMD:C_0603" H 2400 6500 50  0001 C CNN
 F 3 "" H 2400 6500 50  0000 C CNN
 	1    2400 6500
@@
 F 0 "C46" H 2665 6796 50  0000 L CNN
 F 1 "47pF" H 2665 6705 50  0000 L CNN
-F 2 "Capacitors_SMD:C_0402" H 2550 6750 50  0001 C CNN
+F 2 "Capacitors_SMD:C_0603" H 2550 6750 50  0001 C CNN
 F 3 "" H 2550 6750 50  0000 C CNN
 	1    2550 6750
@@
 F 0 "C47" H 2815 7046 50  0000 L CNN
 F 1 "47pF" H 2815 6955 50  0000 L CNN
-F 2 "Capacitors_SMD:C_0402" H 2700 7000 50  0001 C CNN
+F 2 "Capacitors_SMD:C_0603" H 2700 7000 50  0001 C CNN
 F 3 "" H 2700 7000 50  0000 C CNN
 	1    2700 7000
@@
 F 0 "C49" H 2965 7296 50  0000 L CNN
 F 1 "47pF" H 2965 7205 50  0000 L CNN
-F 2 "Capacitors_SMD:C_0402" H 2850 7250 50  0001 C CNN
+F 2 "Capacitors_SMD:C_0603" H 2850 7250 50  0001 C CNN
 F 3 "" H 2850 7250 50  0000 C CNN
 	1    2850 7250
@@
 F 0 "C50" H 3115 6546 50  0000 L CNN
 F 1 "47pF" H 3115 6455 50  0000 L CNN
-F 2 "Capacitors_SMD:C_0402" H 3000 6500 50  0001 C CNN
+F 2 "Capacitors_SMD:C_0603" H 3000 6500 50  0001 C CNN
 F 3 "" H 3000 6500 50  0000 C CNN
 	1    3000 6500
@@
 F 0 "C52" H 3265 6796 50  0000 L CNN
 F 1 "47pF" H 3265 6705 50  0000 L CNN
-F 2 "Capacitors_SMD:C_0402" H 3150 6750 50  0001 C CNN
+F 2 "Capacitors_SMD:C_0603" H 3150 6750 50  0001 C CNN
 F 3 "" H 3150 6750 50  0000 C CNN
 	1    3150 6750
@@
 F 0 "C53" H 3415 7046 50  0000 L CNN
 F 1 "47pF" H 3415 6955 50  0000 L CNN
-F 2 "Capacitors_SMD:C_0402" H 3300 7000 50  0001 C CNN
+F 2 "Capacitors_SMD:C_0603" H 3300 7000 50  0001 C CNN
 F 3 "" H 3300 7000 50  0000 C CNN
 	1    3300 7000
@@
 F 0 "C55" H 3565 7296 50  0000 L CNN
 F 1 "47pF" H 3565 7205 50  0000 L CNN
-F 2 "Capacitors_SMD:C_0402" H 3450 7250 50  0001 C CNN
+F 2 "Capacitors_SMD:C_0603" H 3450 7250 50  0001 C CNN
 F 3 "" H 3450 7250 50  0000 C CNN
 	1    3450 7250
@@
 F 0 "C56" H 3715 6546 50  0000 L CNN
 F 1 "47pF" H 3715 6455 50  0000 L CNN
-F 2 "Capacitors_SMD:C_0402" H 3600 6500 50  0001 C CNN
+F 2 "Capacitors_SMD:C_0603" H 3600 6500 50  0001 C CNN
 F 3 "" H 3600 6500 50  0000 C CNN
 	1    3600 6500
@@
 F 0 "C58" H 3865 6796 50  0000 L CNN
 F 1 "47pF" H 3865 6705 50  0000 L CNN
-F 2 "Capacitors_SMD:C_0402" H 3750 6750 50  0001 C CNN
+F 2 "Capacitors_SMD:C_0603" H 3750 6750 50  0001 C CNN
 F 3 "" H 3750 6750 50  0000 C CNN
 	1    3750 6750
@@
 F 0 "C59" H 4015 7046 50  0000 L CNN
 F 1 "47pF" H 4015 6955 50  0000 L CNN
-F 2 "Capacitors_SMD:C_0402" H 3900 7000 50  0001 C CNN
+F 2 "Capacitors_SMD:C_0603" H 3900 7000 50  0001 C CNN
 F 3 "" H 3900 7000 50  0000 C CNN
 	1    3900 7000
@@
 F 0 "C60" H 4165 7296 50  0000 L CNN
 F 1 "47pF" H 4165 7205 50  0000 L CNN
-F 2 "Capacitors_SMD:C_0402" H 4050 7250 50  0001 C CNN
+F 2 "Capacitors_SMD:C_0603" H 4050 7250 50  0001 C CNN
 F 3 "" H 4050 7250 50  0000 C CNN
 	1    4050 7250
@@
 F 0 "C61" H 4315 6546 50  0000 L CNN
 F 1 "47pF" H 4315 6455 50  0000 L CNN
-F 2 "Capacitors_SMD:C_0402" H 4200 6500 50  0001 C CNN
+F 2 "Capacitors_SMD:C_0603" H 4200 6500 50  0001 C CNN
 F 3 "" H 4200 6500 50  0000 C CNN
 	1    4200 6500
@@
 F 0 "C62" H 4465 6796 50  0000 L CNN
 F 1 "47pF" H 4465 6705 50  0000 L CNN
-F 2 "Capacitors_SMD:C_0402" H 4350 6750 50  0001 C CNN
+F 2 "Capacitors_SMD:C_0603" H 4350 6750 50  0001 C CNN
 F 3 "" H 4350 6750 50  0000 C CNN
 	1    4350 6750
@@
 F 0 "C63" H 4615 7046 50  0000 L CNN
 F 1 "47pF" H 4615 6955 50  0000 L CNN
-F 2 "Capacitors_SMD:C_0402" H 4500 7000 50  0001 C CNN
+F 2 "Capacitors_SMD:C_0603" H 4500 7000 50  0001 C CNN
 F 3 "" H 4500 7000 50  0000 C CNN
 	1    4500 7000
@@
 F 0 "C64" H 4765 7296 50  0000 L CNN
 F 1 "47pF" H 4765 7205 50  0000 L CNN
-F 2 "Capacitors_SMD:C_0402" H 4650 7250 50  0001 C CNN
+F 2 "Capacitors_SMD:C_0603" H 4650 7250 50  0001 C CNN
 F 3 "" H 4650 7250 50  0000 C CNN
 	1    4650 7250
@@
 P 1450 1250
 F 0 "FB29" V 1635 1250 50  0000 C CNN
-F 1 "BLM18BD252SN1D" V 1544 1250 50  0000 C CNN
+F 1 "?H" V 1544 1250 50  0000 C CNN
 F 2 "" H 1450 1250 50  0001 C CNN
 F 3 "" H 1450 1250 50  0000 C CNN
@@
 F 0 "C41" H 1715 1496 50  0000 L CNN
 F 1 "100nF" H 1715 1405 50  0000 L CNN
-F 2 "Capacitors_SMD:C_0402" H 1600 1450 50  0001 C CNN
+F 2 "Capacitors_SMD:C_0603" H 1600 1450 50  0001 C CNN
 F 3 "" H 1600 1450 50  0000 C CNN
 	1    1600 1450
@@
 F 0 "C43" H 2315 1496 50  0000 L CNN
 F 1 "100nF" H 2260 1420 50  0000 L CNN
-F 2 "Capacitors_SMD:C_0402" H 2200 1450 50  0001 C CNN
+F 2 "Capacitors_SMD:C_0603" H 2200 1450 50  0001 C CNN
 F 3 "" H 2200 1450 50  0000 C CNN
 	1    2200 1450
@@
 F 0 "C48" H 2915 1496 50  0000 L CNN
 F 1 "100nF" H 2860 1420 50  0000 L CNN
-F 2 "Capacitors_SMD:C_0402" H 2800 1450 50  0001 C CNN
+F 2 "Capacitors_SMD:C_0603" H 2800 1450 50  0001 C CNN
 F 3 "" H 2800 1450 50  0000 C CNN
 	1    2800 1450
@@
 F 0 "C54" H 3515 1496 50  0000 L CNN
 F 1 "100nF" H 3460 1420 50  0000 L CNN
-F 2 "Capacitors_SMD:C_0402" H 3400 1450 50  0001 C CNN
+F 2 "Capacitors_SMD:C_0603" H 3400 1450 50  0001 C CNN
 F 3 "" H 3400 1450 50  0000 C CNN
 	1    3400 1450
@@
 F 0 "U1" H 1105 6590 60  0000 C CNN
 F 1 "OSD3358" H 1105 6484 60  0000 C CNN
-F 2 "" H 400 6300 60  0001 C CNN
+F 2 "KiMBo:BGA-400-1-27mm" H 400 6300 60  0001 C CNN
 F 3 "" H 400 6300 60  0001 C CNN
 	4    400  6300
@@
 F 0 "R93" V 2500 4525 50  0000 C CNN
 F 1 "0Ω" V 2500 4900 50  0000 C CNN
-F 2 "Resistors_SMD:R_0402" V 2380 4700 50  0001 C CNN
+F 2 "Resistors_SMD:R_0603" V 2380 4700 50  0001 C CNN
 F 3 "" H 2450 4700 50  0000 C CNN
 	1    2450 4700
@@
 F 0 "R92" V 2500 4425 50  0000 C CNN
 F 1 "0Ω" V 2500 4800 50  0000 C CNN
-F 2 "Resistors_SMD:R_0402" V 2380 4600 50  0001 C CNN
+F 2 "Resistors_SMD:R_0603" V 2380 4600 50  0001 C CNN
 F 3 "" H 2450 4600 50  0000 C CNN
 	1    2450 4600
@@
 F 0 "R91" V 2500 4325 50  0000 C CNN
 F 1 "0Ω" V 2500 4700 50  0000 C CNN
-F 2 "Resistors_SMD:R_0402" V 2380 4500 50  0001 C CNN
+F 2 "Resistors_SMD:R_0603" V 2380 4500 50  0001 C CNN
 F 3 "" H 2450 4500 50  0000 C CNN
 	1    2450 4500
@@
 F 0 "R90" V 2500 4225 50  0000 C CNN
 F 1 "22Ω" V 2500 4600 50  0000 C CNN
-F 2 "Resistors_SMD:R_0402" V 2380 4400 50  0001 C CNN
+F 2 "Resistors_SMD:R_0603" V 2380 4400 50  0001 C CNN
 F 3 "" H 2450 4400 50  0000 C CNN
 	1    2450 4400
