File: KiMBo/hdmi.sch (KiCad schematic (older format))
At the start: 41 parts, among them U1 OSD3358, U12 TDA19988BHN/C1,557, U13 IP4283CZ10-TBR, U14 IP4283CZ10-TBR

Commit message: More footprint association
Parts:
- D16: renamed from D15; footprint (none) -> Diodes_SMD:SOD-323
- FB29: value ?H -> BLM18BD252SN1D; footprint (none) -> Resistors_SMD:R_0603
Changed lines of the file:
@@
 $EndComp
 $Comp
-L GND #PWR0143
+L GND #PWR0144
 U 1 1 5896044E
 P 4200 2800
-F 0 "#PWR0143" H 4200 2550 50  0001 C CNN
+F 0 "#PWR0144" H 4200 2550 50  0001 C CNN
 F 1 "GND" H 4200 2650 50  0000 C CNN
 F 2 "" H 4200 2800 50  0000 C CNN
@@
 HDMI
 $Comp
-L GND #PWR0144
+L GND #PWR0145
 U 1 1 5898A6BE
 P 5100 4200
-F 0 "#PWR0144" H 5100 3950 50  0001 C CNN
+F 0 "#PWR0145" H 5100 3950 50  0001 C CNN
 F 1 "GND" H 5100 4050 50  0000 C CNN
 F 2 "" H 5100 4200 50  0000 C CNN
@@
 NoConn ~ 6750 4100
 $Comp
-L D_Schottky D15
+L D_Schottky D16
 U 1 1 5898D395
 P 7150 4650
-F 0 "D15" H 7150 4866 50  0000 C CNN
+F 0 "D16" H 7150 4866 50  0000 C CNN
 F 1 "RB751V40,115" H 7150 4775 50  0000 C CNN
-F 2 "" H 7150 4650 50  0001 C CNN
+F 2 "Diodes_SMD:SOD-323" H 7150 4650 50  0001 C CNN
 F 3 "" H 7150 4650 50  0000 C CNN
 	1    7150 4650
@@
 $EndComp
 $Comp
-L GND #PWR0145
+L GND #PWR0146
 U 1 1 58990275
 P 5400 1250
-F 0 "#PWR0145" H 5400 1000 50  0001 C CNN
+F 0 "#PWR0146" H 5400 1000 50  0001 C CNN
 F 1 "GND" H 5400 1100 50  0000 C CNN
 F 2 "" H 5400 1250 50  0000 C CNN
@@
 $EndComp
 $Comp
-L GND #PWR0146
+L GND #PWR0147
 U 1 1 58990A45
 P 5850 1050
-F 0 "#PWR0146" H 5850 800 50  0001 C CNN
+F 0 "#PWR0147" H 5850 800 50  0001 C CNN
 F 1 "GND" H 5850 900 50  0000 C CNN
 F 2 "" H 5850 1050 50  0000 C CNN
@@
 LCD.D15.R4--R7
 $Comp
-L GND #PWR0147
+L GND #PWR0148
 U 1 1 589952D6
 P 6850 1050
-F 0 "#PWR0147" H 6850 800 50  0001 C CNN
+F 0 "#PWR0148" H 6850 800 50  0001 C CNN
 F 1 "GND" H 6850 900 50  0000 C CNN
 F 2 "" H 6850 1050 50  0000 C CNN
@@
 TEST
 $Comp
-L GND #PWR0148
+L GND #PWR0149
 U 1 1 58996432
 P 7800 1300
-F 0 "#PWR0148" H 7800 1050 50  0001 C CNN
+F 0 "#PWR0149" H 7800 1050 50  0001 C CNN
 F 1 "GND" H 7800 1150 50  0000 C CNN
 F 2 "" H 7800 1300 50  0000 C CNN
@@
 $EndComp
 $Comp
-L GND #PWR0149
+L GND #PWR0150
 U 1 1 589978DF
 P 8550 3600
-F 0 "#PWR0149" H 8550 3350 50  0001 C CNN
+F 0 "#PWR0150" H 8550 3350 50  0001 C CNN
 F 1 "GND" H 8550 3450 50  0000 C CNN
 F 2 "" H 8550 3600 50  0000 C CNN
@@
 $EndComp
 $Comp
-L GND #PWR0150
+L GND #PWR0151
 U 1 1 589AAAC6
 P 10350 4400
-F 0 "#PWR0150" H 10350 4150 50  0001 C CNN
+F 0 "#PWR0151" H 10350 4150 50  0001 C CNN
 F 1 "GND" H 10355 4227 50  0000 C CNN
 F 2 "" H 10350 4400 50  0000 C CNN
@@
 $EndComp
 $Comp
-L GND #PWR0151
+L GND #PWR0152
 U 1 1 589AAAF2
 P 9550 4400
-F 0 "#PWR0151" H 9550 4150 50  0001 C CNN
+F 0 "#PWR0152" H 9550 4150 50  0001 C CNN
 F 1 "GND" H 9555 4227 50  0000 C CNN
 F 2 "" H 9550 4400 50  0000 C CNN
@@
 $EndComp
 $Comp
-L GND #PWR0152
+L GND #PWR0153
 U 1 1 589B56E5
 P 3600 7500
-F 0 "#PWR0152" H 3600 7250 50  0001 C CNN
+F 0 "#PWR0153" H 3600 7250 50  0001 C CNN
 F 1 "GND" H 3605 7327 50  0000 C CNN
 F 2 "" H 3600 7500 50  0000 C CNN
@@
 P 1450 1250
 F 0 "FB29" V 1635 1250 50  0000 C CNN
-F 1 "?H" V 1544 1250 50  0000 C CNN
-F 2 "" H 1450 1250 50  0001 C CNN
+F 1 "BLM18BD252SN1D" V 1544 1250 50  0000 C CNN
+F 2 "Resistors_SMD:R_0603" H 1450 1250 50  0001 C CNN
 F 3 "" H 1450 1250 50  0000 C CNN
 	1    1450 1250
@@
 SPI1_SCLK
 $Comp
-L VDD_3V3B #PWR0153
+L VDD_3V3B #PWR0154
 U 1 1 5A077125
 P 7550 1000
-F 0 "#PWR0153" H 7550 850 50  0001 C CNN
+F 0 "#PWR0154" H 7550 850 50  0001 C CNN
 F 1 "VDD_3V3B" H 7650 1150 50  0000 C CNN
 F 2 "" H 7550 1000 50  0000 C CNN
@@
 $EndComp
 $Comp
-L VDD_3V3B #PWR0154
+L VDD_3V3B #PWR0155
 U 1 1 5A078B10
 P 7700 4600
-F 0 "#PWR0154" H 7700 4450 50  0001 C CNN
+F 0 "#PWR0155" H 7700 4450 50  0001 C CNN
 F 1 "VDD_3V3B" H 7715 4773 50  0000 C CNN
 F 2 "" H 7700 4600 50  0000 C CNN
@@
 $EndComp
 $Comp
-L SYS_5V #PWR0155
+L SYS_5V #PWR0156
 U 1 1 5A079ADB
 P 9800 1600
-F 0 "#PWR0155" H 9800 1450 50  0001 C CNN
+F 0 "#PWR0156" H 9800 1450 50  0001 C CNN
 F 1 "SYS_5V" H 9815 1773 50  0000 C CNN
 F 2 "" H 9800 1600 50  0000 C CNN
@@
 $EndComp
 $Comp
-L HDMI_1V8 #PWR0156
+L HDMI_1V8 #PWR0157
 U 1 1 5A07ADDF
 P 4200 2300
-F 0 "#PWR0156" H 4200 2150 50  0001 C CNN
+F 0 "#PWR0157" H 4200 2150 50  0001 C CNN
 F 1 "HDMI_1V8" H 4200 2450 50  0000 C CNN
 F 2 "" H 4200 2300 50  0000 C CNN
@@
 $EndComp
 $Comp
-L HDMI_1V8 #PWR0157
+L HDMI_1V8 #PWR0158
 U 1 1 5A07B406
 P 4200 3200
-F 0 "#PWR0157" H 4200 3050 50  0001 C CNN
+F 0 "#PWR0158" H 4200 3050 50  0001 C CNN
 F 1 "HDMI_1V8" H 4200 3350 50  0000 C CNN
 F 2 "" H 4200 3200 50  0000 C CNN
@@
 $EndComp
 $Comp
-L HDMI_1V8 #PWR0158
+L HDMI_1V8 #PWR0159
 U 1 1 5A07C429
 P 7800 2000
-F 0 "#PWR0158" H 7800 1850 50  0001 C CNN
+F 0 "#PWR0159" H 7800 1850 50  0001 C CNN
 F 1 "HDMI_1V8" H 7800 2150 50  0000 C CNN
 F 2 "" H 7800 2000 50  0000 C CNN
@@
 $EndComp
 $Comp
-L HDMI_1V8 #PWR0159
+L HDMI_1V8 #PWR0160
 U 1 1 5A07C4AF
 P 8550 2600
-F 0 "#PWR0159" H 8550 2450 50  0001 C CNN
+F 0 "#PWR0160" H 8550 2450 50  0001 C CNN
 F 1 "HDMI_1V8" H 8750 2700 50  0000 C CNN
 F 2 "" H 8550 2600 50  0000 C CNN
@@
 $EndComp
 $Comp
-L HDMI_1V8 #PWR0160
+L HDMI_1V8 #PWR0161
 U 1 1 5A07C535
 P 8550 3200
-F 0 "#PWR0160" H 8550 3050 50  0001 C CNN
+F 0 "#PWR0161" H 8550 3050 50  0001 C CNN
 F 1 "HDMI_1V8" H 8750 3300 50  0000 C CNN
 F 2 "" H 8550 3200 50  0000 C CNN
@@
 $EndComp
 $Comp
-L HDMI_1V8 #PWR0161
+L HDMI_1V8 #PWR0162
 U 1 1 5A0922CB
 P 6750 4850
-F 0 "#PWR0161" H 6750 4700 50  0001 C CNN
+F 0 "#PWR0162" H 6750 4700 50  0001 C CNN
 F 1 "HDMI_1V8" H 6650 5000 50  0000 C CNN
 F 2 "" H 6750 4850 50  0000 C CNN
@@
 $EndComp
 $Comp
-L HDMI_1V8 #PWR0162
+L HDMI_1V8 #PWR0163
 U 1 1 5A094D61
 P 2500 1200
-F 0 "#PWR0162" H 2500 1050 50  0001 C CNN
+F 0 "#PWR0163" H 2500 1050 50  0001 C CNN
 F 1 "HDMI_1V8" H 2515 1373 50  0000 C CNN
 F 2 "" H 2500 1200 50  0000 C CNN
@@
 $EndComp
 $Comp
-L PWR_FLAG #FLG0163
+L PWR_FLAG #FLG0164
 U 1 1 5A0B0393
 P 1900 1200
-F 0 "#FLG0163" H 1900 1295 50  0001 C CNN
+F 0 "#FLG0164" H 1900 1295 50  0001 C CNN
 F 1 "PWR_FLAG" H 1900 1424 50  0000 C CNN
 F 2 "" H 1900 1200 50  0000 C CNN
@@
 $EndComp
 $Comp
-L VDD_1V8 #PWR0164
+L VDD_1V8 #PWR0165
 U 1 1 5A0B0EAC
 P 1050 1200
-F 0 "#PWR0164" H 1050 1050 50  0001 C CNN
+F 0 "#PWR0165" H 1050 1050 50  0001 C CNN
 F 1 "VDD_1V8" H 1065 1373 50  0000 C CNN
 F 2 "" H 1050 1200 50  0000 C CNN
@@
 HDMI_INT
 $Comp
-L VDD_1V8 #PWR0165
+L VDD_1V8 #PWR0166
 U 1 1 5BC7F01E
 P 6650 1100
-F 0 "#PWR0165" H 6650 950 50  0001 C CNN
+F 0 "#PWR0166" H 6650 950 50  0001 C CNN
 F 1 "VDD_1V8" H 6725 1250 50  0000 C CNN
 F 2 "" H 6650 1100 50  0000 C CNN

Commit message: Create more footprints and add more associations
Parts:
- F2: footprint (none) -> KiMBo:F_1206
- U12: footprint (none) -> KiMBo:SOT804-4
- U13, U14: footprint (none) -> KiMBo:XFDFN-10-1EP_2x3mm_Pitch0.5mm
Changed lines of the file:
@@
 F 0 "U12" H 6300 2700 60  0000 L CNN
 F 1 "TDA19988BHN/C1,557" H 5800 2600 60  0000 L CNN
-F 2 "" H 5850 2850 60  0001 C CNN
+F 2 "KiMBo:SOT804-4" H 5850 2850 60  0001 C CNN
 F 3 "" H 5850 2850 60  0001 C CNN
 	1    6400 2700
@@
 F 0 "F2" H 9500 1835 50  0000 C CNN
 F 1 "1206L025YR" H 9500 1744 50  0000 C CNN
-F 2 "" H 9500 1650 50  0001 C CNN
+F 2 "KiMBo:F_1206" H 9500 1650 50  0001 C CNN
 F 3 "" H 9500 1650 50  0000 C CNN
 	1    9500 1650
@@
 F 0 "U13" V 9200 3700 60  0000 L CNN
 F 1 "IP4283CZ10-TBR" V 9900 3550 60  0000 L CNN
-F 2 "" H 9600 4250 60  0001 C CNN
+F 2 "KiMBo:XFDFN-10-1EP_2x3mm_Pitch0.5mm" H 9600 4250 60  0001 C CNN
 F 3 "" H 9600 4250 60  0001 C CNN
 	1    9550 3950
@@
 F 0 "U14" V 10000 3700 60  0000 L CNN
 F 1 "IP4283CZ10-TBR" V 10700 3550 60  0000 L CNN
-F 2 "" H 10400 4250 60  0001 C CNN
+F 2 "KiMBo:XFDFN-10-1EP_2x3mm_Pitch0.5mm" H 10400 4250 60  0001 C CNN
 F 3 "" H 10400 4250 60  0001 C CNN
 	1    10350 3950

Commit message: Begin layout
Arrange all connectors to get a feel for the area.
Parts:
- renumbered C41 to C43, C42 to C44, C43 to C45, C44 to C46, C45 to C47, C46 to C48, C47 to C49, C48 to C50, C49 to C51, C50 to C52, C51 to C53, C52 to C54, C53 to C55, C54 to C56, C55 to C57, C56 to C58, C57 to C59, C58 to C60, C59 to C61, C60 to C62, C61 to C63, C62 to C64, C63 to C65, C64 to C66, D16 to D17
