File: KiMBo/mpu.sch (KiCad schematic (older format))
At the start: 11 parts, among them U2 OSD3358, U5 74LVC1G74

Commit message: Associate more footprints
Changed lines of the file:
@@
 	8950 3550 8950 3450
 Wire Wire Line
-	8950 3450 10350 3450
-Wire Wire Line
-	10350 3450 11150 3450
+	8950 3450 11150 3450
 Wire Wire Line
 	11150 3450 11150 3500
@@
 	7200 7350 6750 7350
 Wire Wire Line
-	6100 7400 6100 7450
-Wire Wire Line
-	6100 7450 6100 7500
+	6100 7400 6100 7500
 Wire Wire Line
 	6100 7450 7200 7450
@@
 	7150 6550 7200 6550
 Wire Wire Line
-	7150 6400 7150 6450
-Wire Wire Line
-	7150 6450 7150 6550
-Wire Wire Line
-	7150 6550 7150 6650
+	7150 6400 7150 6650
 Connection ~ 7150 6450
 Wire Wire Line
 	7050 6450 7050 6500
 Wire Wire Line
-	7050 6450 7150 6450
-Wire Wire Line
-	7150 6450 7200 6450
-Wire Wire Line
-	7350 3850 8150 3850
-Wire Wire Line
-	8150 3850 8250 3850
+	7050 6450 7200 6450
+Wire Wire Line
+	7350 3850 8250 3850
 Wire Wire Line
 	6150 4050 6100 4050
@@
 	6900 4150 6900 4100
 Wire Wire Line
-	6900 2850 6900 2900
-Wire Wire Line
-	6900 2900 6900 3250
-Wire Wire Line
-	6900 3250 6900 3550
-Wire Wire Line
-	6900 3550 6900 3600
+	6900 2850 6900 3600
 Wire Wire Line
 	6150 3650 6000 3650
@@
 F 0 "C15" H 7165 3146 50  0000 L CNN
 F 1 "100nF" H 7165 3055 50  0000 L CNN
-F 2 "" H 7088 2950 50  0000 C CNN
+F 2 "" H 7088 2950 50  0001 C CNN
 F 3 "" H 7050 3100 50  0000 C CNN
 	1    7050 3100

Commit message: Add equivalent annotations document, associate more footprints
Parts:
- C15: footprint (none) -> Capacitors_SMD:C_0402
- R27: renamed from R28; footprint (none) -> Resistors_SMD:R_0402
- R28: renamed from R29; footprint (none) -> Resistors_SMD:R_0402
- R29: renamed from R30; footprint (none) -> Resistors_SMD:R_0402
- R30: renamed from R31; footprint (none) -> Resistors_SMD:R_0402
- R31: renamed from R32; footprint (none) -> Resistors_SMD:R_0402
Changed lines of the file:
@@
 I2C1_SCL
 $Comp
-L R R31
+L R R30
 U 1 1 5834D6F6
 P 11150 3650
-F 0 "R31" H 11220 3696 50  0000 L CNN
+F 0 "R30" H 11220 3696 50  0000 L CNN
 F 1 "0Ω" H 11220 3605 50  0000 L CNN
-F 2 "" V 11080 3650 50  0001 C CNN
+F 2 "Resistors_SMD:R_0402" V 11080 3650 50  0001 C CNN
 F 3 "" H 11150 3650 50  0000 C CNN
 	1    11150 3650
@@
 AIN6
 $Comp
-L R R28
+L R R27
 U 1 1 584B72FD
 P 6100 7250
-F 0 "R28" H 6169 7296 50  0000 L CNN
+F 0 "R27" H 6169 7296 50  0000 L CNN
 F 1 "4.75kΩ" H 6169 7205 50  0000 L CNN
-F 2 "" V 6030 7250 50  0001 C CNN
+F 2 "Resistors_SMD:R_0402" V 6030 7250 50  0001 C CNN
 F 3 "" H 6100 7250 50  0000 C CNN
 	1    6100 7250
@@
 $EndComp
 $Comp
-L R R29
+L R R28
 U 1 1 584B7384
 P 6100 7650
-F 0 "R29" H 6169 7696 50  0000 L CNN
+F 0 "R28" H 6169 7696 50  0000 L CNN
 F 1 "4.75kΩ" H 6169 7605 50  0000 L CNN
-F 2 "" V 6030 7650 50  0001 C CNN
+F 2 "Resistors_SMD:R_0402" V 6030 7650 50  0001 C CNN
 F 3 "" H 6100 7650 50  0000 C CNN
 	1    6100 7650
@@
 $EndComp
 $Comp
-L GND #PWR091
+L GND #PWR090
 U 1 1 584B7680
 P 6100 7850
-F 0 "#PWR091" H 6100 7600 50  0001 C CNN
+F 0 "#PWR090" H 6100 7600 50  0001 C CNN
 F 1 "GND" H 6105 7677 50  0000 C CNN
 F 2 "" H 6100 7850 50  0000 C CNN
@@
 $EndComp
 $Comp
-L GND #PWR092
+L GND #PWR091
 U 1 1 584D67FE
 P 6900 4150
-F 0 "#PWR092" H 6900 3900 50  0001 C CNN
+F 0 "#PWR091" H 6900 3900 50  0001 C CNN
 F 1 "GND" H 6905 3977 50  0000 C CNN
 F 2 "" H 6900 4150 50  0000 C CNN
@@
 $EndComp
 $Comp
-L GND #PWR093
+L GND #PWR092
 U 1 1 584DD3A5
 P 7050 3300
-F 0 "#PWR093" H 7050 3050 50  0001 C CNN
+F 0 "#PWR092" H 7050 3050 50  0001 C CNN
 F 1 "GND" H 7055 3127 50  0000 C CNN
 F 2 "" H 7050 3300 50  0000 C CNN
@@
 12M_LOOP
 $Comp
-L R R30
+L R R29
 U 1 1 584E01E5
 P 9500 7550
-F 0 "R30" V 9293 7550 50  0000 C CNN
+F 0 "R29" V 9293 7550 50  0000 C CNN
 F 1 "0Ω" V 9384 7550 50  0000 C CNN
-F 2 "" V 9430 7550 50  0001 C CNN
+F 2 "Resistors_SMD:R_0402" V 9430 7550 50  0001 C CNN
 F 3 "" H 9500 7550 50  0000 C CNN
 	1    9500 7550
@@
 $EndComp
 $Comp
-L R R32
+L R R31
 U 1 1 584E0761
 P 11300 4150
-F 0 "R32" V 11250 4000 50  0000 C CNN
+F 0 "R31" V 11250 4000 50  0000 C CNN
 F 1 "0Ω" V 11300 4150 50  0000 C CNN
-F 2 "" V 11230 4150 50  0001 C CNN
+F 2 "Resistors_SMD:R_0402" V 11230 4150 50  0001 C CNN
 F 3 "" H 11300 4150 50  0000 C CNN
 	1    11300 4150
@@
 ENC_B
 $Comp
-L VDD_ADC #PWR094
+L VDD_ADC #PWR093
 U 1 1 59E85302
 P 7000 7650
-F 0 "#PWR094" H 7150 7600 50  0001 C CNN
+F 0 "#PWR093" H 7150 7600 50  0001 C CNN
 F 1 "VDD_ADC" H 7020 7793 50  0000 C CNN
 F 2 "" H 7000 7650 50  0000 C CNN
@@
 $EndComp
 $Comp
-L VDD_3V3B #PWR095
+L VDD_3V3B #PWR094
 U 1 1 59F9CAE6
 P 6900 2850
-F 0 "#PWR095" H 6900 2700 50  0001 C CNN
+F 0 "#PWR094" H 6900 2700 50  0001 C CNN
 F 1 "VDD_3V3B" H 6915 3023 50  0000 C CNN
 F 2 "" H 6900 2850 50  0000 C CNN
@@
 $EndComp
 $Comp
-L VDD_3V3B #PWR096
+L VDD_3V3B #PWR095
 U 1 1 59FC1115
 P 6100 7050
-F 0 "#PWR096" H 6100 6900 50  0001 C CNN
+F 0 "#PWR095" H 6100 6900 50  0001 C CNN
 F 1 "VDD_3V3B" H 6115 7223 50  0000 C CNN
 F 2 "" H 6100 7050 50  0000 C CNN
@@
 $EndComp
 $Comp
-L GNDA #PWR097
+L GNDA #PWR096
 U 1 1 59FCC96D
 P 7050 6500
-F 0 "#PWR097" H 7050 6250 50  0001 C CNN
+F 0 "#PWR096" H 7050 6250 50  0001 C CNN
 F 1 "GNDA" H 7055 6327 50  0000 C CNN
 F 2 "" H 7050 6500 50  0000 C CNN
@@
 Internal 150Ω FB\nfrom E8 to VSS\nunused on Replicape
 $Comp
-L PWR_FLAG #FLG098
+L PWR_FLAG #FLG097
 U 1 1 59FD3D41
 P 7150 6400
-F 0 "#FLG098" H 7150 6495 50  0001 C CNN
+F 0 "#FLG097" H 7150 6495 50  0001 C CNN
 F 1 "PWR_FLAG" H 7150 6624 50  0000 C CNN
 F 2 "" H 7150 6400 50  0000 C CNN
@@
 F 0 "C15" H 7165 3146 50  0000 L CNN
 F 1 "100nF" H 7165 3055 50  0000 L CNN
-F 2 "" H 7088 2950 50  0001 C CNN
+F 2 "Capacitors_SMD:C_0402" H 7088 2950 50  0001 C CNN
 F 3 "" H 7050 3100 50  0000 C CNN
 	1    7050 3100

Commit message: Leave SPI0 free for a display, reassign pins so SPI1 is available
Fix some typos/errors
Parts:
- renumbered R27 to R29, R28 to R30, R29 to R31, R30 to R32, R31 to R33, U2 to U1, U5 to U4
Connections:
- net GPIO3_19 is gone; now on net Z2_ENDSTOP: U1.C13 (MCASP0_FSR)
- net Z2_ENDSTOP: no longer U1.B16 (SPI0_D1)
- net ENC_B renamed SPI0_CS0
- net UART2_TXD renamed SPI0_MISO
- new net SPI0_MOSI: U1.B16 (SPI0_D1)
- no-connect marks 7 -> 5
Other:
- note removed: "potential GPIO"
Changed lines of the file:
@@
 $EndDescr
 $Comp
-L OSD3358 U2
+L OSD3358 U1
 U 6 1 582FD785
 P 7200 6450
-F 0 "U2" H 8250 6740 60  0000 C CNN
+F 0 "U1" H 8250 6740 60  0000 C CNN
 F 1 "OSD3358" H 8250 6634 60  0000 C CNN
 F 2 "" H 7200 6450 60  0001 C CNN
@@
 $EndComp
 $Comp
-L OSD3358 U2
+L OSD3358 U1
 U 5 1 582FE5A0
 P 9000 3850
-F 0 "U2" H 10050 4140 60  0000 C CNN
+F 0 "U1" H 10050 4140 60  0000 C CNN
 F 1 "OSD3358" H 10050 4034 60  0000 C CNN
 F 2 "" H 9000 3850 60  0001 C CNN
@@
 I2C1_SCL
 $Comp
-L R R30
+L R R32
 U 1 1 5834D6F6
 P 11150 3650
-F 0 "R30" H 11220 3696 50  0000 L CNN
+F 0 "R32" H 11220 3696 50  0000 L CNN
 F 1 "0Ω" H 11220 3605 50  0000 L CNN
 F 2 "Resistors_SMD:R_0402" V 11080 3650 50  0001 C CNN
@@
 AIN6
 $Comp
-L R R27
+L R R29
 U 1 1 584B72FD
 P 6100 7250
-F 0 "R27" H 6169 7296 50  0000 L CNN
+F 0 "R29" H 6169 7296 50  0000 L CNN
 F 1 "4.75kΩ" H 6169 7205 50  0000 L CNN
 F 2 "Resistors_SMD:R_0402" V 6030 7250 50  0001 C CNN
@@
 $EndComp
 $Comp
-L R R28
+L R R30
 U 1 1 584B7384
 P 6100 7650
-F 0 "R28" H 6169 7696 50  0000 L CNN
+F 0 "R30" H 6169 7696 50  0000 L CNN
 F 1 "4.75kΩ" H 6169 7605 50  0000 L CNN
 F 2 "Resistors_SMD:R_0402" V 6030 7650 50  0001 C CNN
@@
 $EndComp
 $Comp
-L GND #PWR090
+L GND #PWR089
 U 1 1 584B7680
 P 6100 7850
-F 0 "#PWR090" H 6100 7600 50  0001 C CNN
+F 0 "#PWR089" H 6100 7600 50  0001 C CNN
 F 1 "GND" H 6105 7677 50  0000 C CNN
 F 2 "" H 6100 7850 50  0000 C CNN
@@
 $EndComp
 $Comp
-L 74LVC1G74 U5
+L 74LVC1G74 U4
 U 1 1 584D5286
 P 6750 3850
-F 0 "U5" H 6850 4250 50  0000 L CNN
+F 0 "U4" H 6850 4250 50  0000 L CNN
 F 1 "74LVC1G74" H 6800 4150 50  0000 L CNN
 F 2 "" H 6750 3850 50  0001 C CNN
@@
 $EndComp
 $Comp
-L GND #PWR091
+L GND #PWR090
 U 1 1 584D67FE
 P 6900 4150
-F 0 "#PWR091" H 6900 3900 50  0001 C CNN
+F 0 "#PWR090" H 6900 3900 50  0001 C CNN
 F 1 "GND" H 6905 3977 50  0000 C CNN
 F 2 "" H 6900 4150 50  0000 C CNN
@@
 $EndComp
 $Comp
-L GND #PWR092
+L GND #PWR091
 U 1 1 584DD3A5
 P 7050 3300
-F 0 "#PWR092" H 7050 3050 50  0001 C CNN
+F 0 "#PWR091" H 7050 3050 50  0001 C CNN
 F 1 "GND" H 7055 3127 50  0000 C CNN
 F 2 "" H 7050 3300 50  0000 C CNN
@@
 12M_LOOP
 $Comp
-L R R29
+L R R31
 U 1 1 584E01E5
 P 9500 7550
-F 0 "R29" V 9293 7550 50  0000 C CNN
+F 0 "R31" V 9293 7550 50  0000 C CNN
 F 1 "0Ω" V 9384 7550 50  0000 C CNN
 F 2 "Resistors_SMD:R_0402" V 9430 7550 50  0001 C CNN
@@
 $EndComp
 $Comp
-L R R31
+L R R33
 U 1 1 584E0761
 P 11300 4150
-F 0 "R31" V 11250 4000 50  0000 C CNN
+F 0 "R33" V 11250 4000 50  0000 C CNN
 F 1 "0Ω" V 11300 4150 50  0000 C CNN
 F 2 "Resistors_SMD:R_0402" V 11230 4150 50  0001 C CNN
@@
 P 2250 3900
 AR Path="/58F3251C" Ref="U?"  Part="12"
-AR Path="/581AEC7B/58F3251C" Ref="U2"  Part="12"
-F 0 "U2" H 2900 4190 60  0000 C CNN
+AR Path="/581AEC7B/58F3251C" Ref="U1"  Part="12"
+F 0 "U1" H 2900 4190 60  0000 C CNN
 F 1 "OSD3358" H 2900 4084 60  0000 C CNN
 F 2 "" H 2250 3900 60  0001 C CNN
@@
 Text HLabel 11850 4050 2    60   BiDi ~ 0
 SPI1_CS0
-Text HLabel 8500 4450 0    60   Input ~ 0
+Text HLabel 11850 4250 2    60   Input ~ 0
 Z2_ENDSTOP
 Text HLabel 6750 7350 0    60   Input ~ 0
@@
 Text HLabel 10000 7550 2    60   Output ~ 0
 SPI1_CS1
-Text HLabel 8500 4150 0    60   Input ~ 0
-ENC_B
-$Comp
-L VDD_ADC #PWR093
+$Comp
+L VDD_ADC #PWR092
 U 1 1 59E85302
 P 7000 7650
-F 0 "#PWR093" H 7150 7600 50  0001 C CNN
+F 0 "#PWR092" H 7150 7600 50  0001 C CNN
 F 1 "VDD_ADC" H 7020 7793 50  0000 C CNN
 F 2 "" H 7000 7650 50  0000 C CNN
@@
 $EndComp
 $Comp
-L VDD_3V3B #PWR094
+L VDD_3V3B #PWR093
 U 1 1 59F9CAE6
 P 6900 2850
-F 0 "#PWR094" H 6900 2700 50  0001 C CNN
+F 0 "#PWR093" H 6900 2700 50  0001 C CNN
 F 1 "VDD_3V3B" H 6915 3023 50  0000 C CNN
 F 2 "" H 6900 2850 50  0000 C CNN
@@
 $EndComp
 $Comp
-L VDD_3V3B #PWR095
+L VDD_3V3B #PWR094
 U 1 1 59FC1115
 P 6100 7050
-F 0 "#PWR095" H 6100 6900 50  0001 C CNN
+F 0 "#PWR094" H 6100 6900 50  0001 C CNN
 F 1 "VDD_3V3B" H 6115 7223 50  0000 C CNN
 F 2 "" H 6100 7050 50  0000 C CNN
@@
 $EndComp
 $Comp
-L GNDA #PWR096
+L GNDA #PWR095
 U 1 1 59FCC96D
 P 7050 6500
-F 0 "#PWR096" H 7050 6250 50  0001 C CNN
+F 0 "#PWR095" H 7050 6250 50  0001 C CNN
 F 1 "GNDA" H 7055 6327 50  0000 C CNN
 F 2 "" H 7050 6500 50  0000 C CNN
@@
 Internal 150Ω FB\nfrom E8 to VSS\nunused on Replicape
 $Comp
-L PWR_FLAG #FLG097
+L PWR_FLAG #FLG096
 U 1 1 59FD3D41
 P 7150 6400
-F 0 "#FLG097" H 7150 6495 50  0001 C CNN
+F 0 "#FLG096" H 7150 6495 50  0001 C CNN
 F 1 "PWR_FLAG" H 7150 6624 50  0000 C CNN
 F 2 "" H 7150 6400 50  0000 C CNN
@@
 	1    0    0    -1
 $EndComp
-Text Notes 8500 4375 2    60   ~ 0
-potential GPIO
-Text Notes 11850 4250 0    60   ~ 0
-potential GPIO
 $Comp
 L INDUCTOR_Small FB19
@@
 Wire Wire Line
 	8500 4050 9000 4050
-NoConn ~ 8500 4350
 Text HLabel 5750 3650 0    60   Output ~ 0
 12MHz
-NoConn ~ 11850 4250
 $Comp
 L INDUCTOR_Small FB21
@@
 	1    0    0    -1
 $EndComp
+Text HLabel 8500 4350 0    60   Output ~ 0
+SPI0_MISO
+Text Label 8500 4250 0    60   ~ 0
+SPI0_CS1
+Text HLabel 8500 4450 0    60   Input ~ 0
+SPI0_MOSI
+Text HLabel 11850 4150 2    60   Output ~ 0
+SPI1_CS1
+Text HLabel 8500 4150 0    60   Input ~ 0
+SPI0_CS0
 $EndSCHEMATC

Commit message: Use fixed 5V LM2592HV Buck, include SPI0 header for LCD
Parts:
- renumbered C15 to C12, FB19 to FB24, FB20 to FB25, FB21 to FB26, R29 to R26, R30 to R27, R31 to R28, R32 to R29, R33 to R30
Changed lines of the file:
@@
 I2C1_SCL
 $Comp
-L R R32
+L R R29
 U 1 1 5834D6F6
 P 11150 3650
-F 0 "R32" H 11220 3696 50  0000 L CNN
+F 0 "R29" H 11220 3696 50  0000 L CNN
 F 1 "0Ω" H 11220 3605 50  0000 L CNN
 F 2 "Resistors_SMD:R_0402" V 11080 3650 50  0001 C CNN
@@
 AIN6
 $Comp
-L R R29
+L R R26
 U 1 1 584B72FD
 P 6100 7250
-F 0 "R29" H 6169 7296 50  0000 L CNN
+F 0 "R26" H 6169 7296 50  0000 L CNN
 F 1 "4.75kΩ" H 6169 7205 50  0000 L CNN
 F 2 "Resistors_SMD:R_0402" V 6030 7250 50  0001 C CNN
@@
 $EndComp
 $Comp
-L R R30
+L R R27
 U 1 1 584B7384
 P 6100 7650
-F 0 "R30" H 6169 7696 50  0000 L CNN
+F 0 "R27" H 6169 7696 50  0000 L CNN
 F 1 "4.75kΩ" H 6169 7605 50  0000 L CNN
 F 2 "Resistors_SMD:R_0402" V 6030 7650 50  0001 C CNN
@@
 $EndComp
 $Comp
-L GND #PWR089
+L GND #PWR084
 U 1 1 584B7680
 P 6100 7850
-F 0 "#PWR089" H 6100 7600 50  0001 C CNN
+F 0 "#PWR084" H 6100 7600 50  0001 C CNN
 F 1 "GND" H 6105 7677 50  0000 C CNN
 F 2 "" H 6100 7850 50  0000 C CNN
@@
 $EndComp
 $Comp
-L GND #PWR090
+L GND #PWR085
 U 1 1 584D67FE
 P 6900 4150
-F 0 "#PWR090" H 6900 3900 50  0001 C CNN
+F 0 "#PWR085" H 6900 3900 50  0001 C CNN
 F 1 "GND" H 6905 3977 50  0000 C CNN
 F 2 "" H 6900 4150 50  0000 C CNN
@@
 $EndComp
 $Comp
-L GND #PWR091
+L GND #PWR086
 U 1 1 584DD3A5
 P 7050 3300
-F 0 "#PWR091" H 7050 3050 50  0001 C CNN
+F 0 "#PWR086" H 7050 3050 50  0001 C CNN
 F 1 "GND" H 7055 3127 50  0000 C CNN
 F 2 "" H 7050 3300 50  0000 C CNN
@@
 12M_LOOP
 $Comp
-L R R31
+L R R28
 U 1 1 584E01E5
 P 9500 7550
-F 0 "R31" V 9293 7550 50  0000 C CNN
+F 0 "R28" V 9293 7550 50  0000 C CNN
 F 1 "0Ω" V 9384 7550 50  0000 C CNN
 F 2 "Resistors_SMD:R_0402" V 9430 7550 50  0001 C CNN
@@
 $EndComp
 $Comp
-L R R33
+L R R30
 U 1 1 584E0761
 P 11300 4150
-F 0 "R33" V 11250 4000 50  0000 C CNN
+F 0 "R30" V 11250 4000 50  0000 C CNN
 F 1 "0Ω" V 11300 4150 50  0000 C CNN
 F 2 "Resistors_SMD:R_0402" V 11230 4150 50  0001 C CNN
@@
 SPI1_CS1
 $Comp
-L VDD_ADC #PWR092
+L VDD_ADC #PWR087
 U 1 1 59E85302
 P 7000 7650
-F 0 "#PWR092" H 7150 7600 50  0001 C CNN
+F 0 "#PWR087" H 7150 7600 50  0001 C CNN
 F 1 "VDD_ADC" H 7020 7793 50  0000 C CNN
 F 2 "" H 7000 7650 50  0000 C CNN
@@
 $EndComp
 $Comp
-L VDD_3V3B #PWR093
+L VDD_3V3B #PWR088
 U 1 1 59F9CAE6
 P 6900 2850
-F 0 "#PWR093" H 6900 2700 50  0001 C CNN
+F 0 "#PWR088" H 6900 2700 50  0001 C CNN
 F 1 "VDD_3V3B" H 6915 3023 50  0000 C CNN
 F 2 "" H 6900 2850 50  0000 C CNN
@@
 $EndComp
 $Comp
-L VDD_3V3B #PWR094
+L VDD_3V3B #PWR089
 U 1 1 59FC1115
 P 6100 7050
-F 0 "#PWR094" H 6100 6900 50  0001 C CNN
+F 0 "#PWR089" H 6100 6900 50  0001 C CNN
 F 1 "VDD_3V3B" H 6115 7223 50  0000 C CNN
 F 2 "" H 6100 7050 50  0000 C CNN
@@
 $EndComp
 $Comp
-L GNDA #PWR095
+L GNDA #PWR090
 U 1 1 59FCC96D
 P 7050 6500
-F 0 "#PWR095" H 7050 6250 50  0001 C CNN
+F 0 "#PWR090" H 7050 6250 50  0001 C CNN
 F 1 "GNDA" H 7055 6327 50  0000 C CNN
 F 2 "" H 7050 6500 50  0000 C CNN
@@
 Internal 150Ω FB\nfrom E8 to VSS\nunused on Replicape
 $Comp
-L PWR_FLAG #FLG096
+L PWR_FLAG #FLG091
 U 1 1 59FD3D41
 P 7150 6400
-F 0 "#FLG096" H 7150 6495 50  0001 C CNN
+F 0 "#FLG091" H 7150 6495 50  0001 C CNN
 F 1 "PWR_FLAG" H 7150 6624 50  0000 C CNN
 F 2 "" H 7150 6400 50  0000 C CNN
@@
 $EndComp
 $Comp
-L INDUCTOR_Small FB19
+L INDUCTOR_Small FB24
 U 1 1 5B034EFC
 P 5900 3650
-F 0 "FB19" V 6085 3650 50  0000 C CNN
+F 0 "FB24" V 6085 3650 50  0000 C CNN
 F 1 "BLM15AG102SN1D" V 6000 3800 50  0000 C CNN
 F 2 "" H 5900 3650 50  0001 C CNN
@@
 12MHz
 $Comp
-L INDUCTOR_Small FB21
+L INDUCTOR_Small FB26
 U 1 1 58CEF5B5
 P 8950 3650
-F 0 "FB21" H 9000 3650 50  0000 L CNN
+F 0 "FB26" H 9000 3650 50  0000 L CNN
 F 1 "BLM15AG102SN1D" H 8250 3650 50  0000 L CNN
 F 2 "" H 8950 3650 50  0001 C CNN
@@
 $EndComp
 $Comp
-L INDUCTOR_Small FB20
+L INDUCTOR_Small FB25
 U 1 1 58CF0E6E
 P 8350 3850
-F 0 "FB20" V 8300 3750 50  0000 L CNN
+F 0 "FB25" V 8300 3750 50  0000 L CNN
 F 1 "BLM15AG102SN1D" V 8400 3700 50  0000 L CNN
 F 2 "" H 8350 3850 50  0001 C CNN
@@
 $EndComp
 $Comp
-L C C15
+L C C12
 U 1 1 58EAE0AA
 P 7050 3100
-F 0 "C15" H 7165 3146 50  0000 L CNN
+F 0 "C12" H 7165 3146 50  0000 L CNN
 F 1 "100nF" H 7165 3055 50  0000 L CNN
 F 2 "Capacitors_SMD:C_0402" H 7088 2950 50  0001 C CNN

Commit message: Assocate more footprints
Parts:
- C12: footprint Capacitors_SMD:C_0402 -> Capacitors_SMD:C_0603
- FB24, FB25, FB26: value BLM15AG102SN1D -> ?H
- R26, R27, R28, R29, R30: footprint Resistors_SMD:R_0402 -> Resistors_SMD:R_0603
- U1: footprint (none) -> KiMBo:BGA-400-1-27mm
Changed lines of the file:
@@
 F 0 "U1" H 8250 6740 60  0000 C CNN
 F 1 "OSD3358" H 8250 6634 60  0000 C CNN
-F 2 "" H 7200 6450 60  0001 C CNN
+F 2 "KiMBo:BGA-400-1-27mm" H 7200 6450 60  0001 C CNN
 F 3 "" H 7200 6450 60  0001 C CNN
 	6    7200 6450
@@
 F 0 "U1" H 10050 4140 60  0000 C CNN
 F 1 "OSD3358" H 10050 4034 60  0000 C CNN
-F 2 "" H 9000 3850 60  0001 C CNN
+F 2 "KiMBo:BGA-400-1-27mm" H 9000 3850 60  0001 C CNN
 F 3 "" H 9000 3850 60  0001 C CNN
 	5    9000 3850
@@
 F 0 "R29" H 11220 3696 50  0000 L CNN
 F 1 "0Ω" H 11220 3605 50  0000 L CNN
-F 2 "Resistors_SMD:R_0402" V 11080 3650 50  0001 C CNN
+F 2 "Resistors_SMD:R_0603" V 11080 3650 50  0001 C CNN
 F 3 "" H 11150 3650 50  0000 C CNN
 	1    11150 3650
@@
 F 0 "R26" H 6169 7296 50  0000 L CNN
 F 1 "4.75kΩ" H 6169 7205 50  0000 L CNN
-F 2 "Resistors_SMD:R_0402" V 6030 7250 50  0001 C CNN
+F 2 "Resistors_SMD:R_0603" V 6030 7250 50  0001 C CNN
 F 3 "" H 6100 7250 50  0000 C CNN
 	1    6100 7250
@@
 F 0 "R27" H 6169 7696 50  0000 L CNN
 F 1 "4.75kΩ" H 6169 7605 50  0000 L CNN
-F 2 "Resistors_SMD:R_0402" V 6030 7650 50  0001 C CNN
+F 2 "Resistors_SMD:R_0603" V 6030 7650 50  0001 C CNN
 F 3 "" H 6100 7650 50  0000 C CNN
 	1    6100 7650
@@
 F 0 "R28" V 9293 7550 50  0000 C CNN
 F 1 "0Ω" V 9384 7550 50  0000 C CNN
-F 2 "Resistors_SMD:R_0402" V 9430 7550 50  0001 C CNN
+F 2 "Resistors_SMD:R_0603" V 9430 7550 50  0001 C CNN
 F 3 "" H 9500 7550 50  0000 C CNN
 	1    9500 7550
@@
 F 0 "R30" V 11250 4000 50  0000 C CNN
 F 1 "0Ω" V 11300 4150 50  0000 C CNN
-F 2 "Resistors_SMD:R_0402" V 11230 4150 50  0001 C CNN
+F 2 "Resistors_SMD:R_0603" V 11230 4150 50  0001 C CNN
 F 3 "" H 11300 4150 50  0000 C CNN
 	1    11300 4150
@@
 F 0 "U1" H 2900 4190 60  0000 C CNN
 F 1 "OSD3358" H 2900 4084 60  0000 C CNN
-F 2 "" H 2250 3900 60  0001 C CNN
+F 2 "KiMBo:BGA-400-1-27mm" H 2250 3900 60  0001 C CNN
 F 3 "" H 2250 3900 60  0001 C CNN
 	12   2250 3900
@@
 P 5900 3650
 F 0 "FB24" V 6085 3650 50  0000 C CNN
-F 1 "BLM15AG102SN1D" V 6000 3800 50  0000 C CNN
+F 1 "?H" V 6000 3800 50  0000 C CNN
 F 2 "" H 5900 3650 50  0001 C CNN
 F 3 "" H 5900 3650 50  0000 C CNN
@@
 P 8950 3650
 F 0 "FB26" H 9000 3650 50  0000 L CNN
-F 1 "BLM15AG102SN1D" H 8250 3650 50  0000 L CNN
+F 1 "?H" H 8800 3650 50  0000 L CNN
 F 2 "" H 8950 3650 50  0001 C CNN
 F 3 "" H 8950 3650 50  0000 C CNN
@@
 P 8350 3850
 F 0 "FB25" V 8300 3750 50  0000 L CNN
-F 1 "BLM15AG102SN1D" V 8400 3700 50  0000 L CNN
+F 1 "?H" V 8400 3700 50  0000 L CNN
 F 2 "" H 8350 3850 50  0001 C CNN
 F 3 "" H 8350 3850 50  0000 C CNN
@@
 F 0 "C12" H 7165 3146 50  0000 L CNN
 F 1 "100nF" H 7165 3055 50  0000 L CNN
-F 2 "Capacitors_SMD:C_0402" H 7088 2950 50  0001 C CNN
+F 2 "Capacitors_SMD:C_0603" H 7088 2950 50  0001 C CNN
 F 3 "" H 7050 3100 50  0000 C CNN
 	1    7050 3100
