File: KiMBo/KiMBo.kicad_pcb (KiCad board)
At the start: 2 copper layers, 0 parts

Commit message: Import the netlist
Parts:
- added C1: 100nF, Capacitors_SMD:C_0603, F.Cu at (157.8, 2.86)
- added C10: 22μF, Capacitors_SMD:C_0805, F.Cu at (101.1, 142.3)
- added C100: 100nF, Capacitors_SMD:C_0603, F.Cu at (317.4, 8.71)
- added C101: 4.7μF, Capacitors_SMD:C_0603, F.Cu at (313.8, 2.86)
- added C102: 22nF, Capacitors_SMD:C_0603, F.Cu at (326.9, 14.6)
- added C103: 470pF, Capacitors_SMD:C_0603, F.Cu at (317.7, 20.8)
- added C104: 470pF, Capacitors_SMD:C_0603, F.Cu at (327.7, 8.71)
- added C105: 100nF, Capacitors_SMD:C_0603, F.Cu at (312.6, 20.8)
- added C106: 470pF, Capacitors_SMD:C_0603, F.Cu at (297.9, 15.4)
- added C107: 470pF, Capacitors_SMD:C_0603, F.Cu at (329.5, 2.86)
- added C108: 100nF, Capacitors_SMD:C_0603, F.Cu at (316.9, 15.0)
- added C109: 100nF, Capacitors_SMD:C_0603, F.Cu at (307.4, 20.8)
- added C11: 22μF, Capacitors_SMD:C_0805, F.Cu at (115.1, 135.6)
- added C110: 100nF, Capacitors_SMD:C_0603, F.Cu at (311.8, 15.0)
- added C111: 10μF, Capacitors_SMD:C_0805, F.Cu at (301.8, 9.31)
- added C112: 100μF, Capacitors_SMD:c_elec_8x10, F.Cu at (294.1, 6.04)
- added C113: 100nF, Capacitors_SMD:C_0603, F.Cu at (322.5, 8.71)
- added C114: 100nF, Capacitors_SMD:C_0603, F.Cu at (176.1, 137.9)
- added C115: 470nF, Capacitors_SMD:C_0603, F.Cu at (186.9, 125.8)
- added C116: 100nF, Capacitors_SMD:C_0603, F.Cu at (180.1, 131.7)
- added C117: 4.7μF, Capacitors_SMD:C_0603, F.Cu at (171.1, 137.9)
- added C118: 22nF, Capacitors_SMD:C_0603, F.Cu at (187.0, 120.0)
- added C119: 470pF, Capacitors_SMD:C_0603, F.Cu at (185.2, 131.7)
- added C12: 100nF, Capacitors_SMD:C_0603, F.Cu at (260.3, 170.8)
- added C120: 470pF, Capacitors_SMD:C_0603, F.Cu at (177.1, 120.0)
- added C121: 100nF, Capacitors_SMD:C_0603, F.Cu at (161.0, 137.9)
- added C122: 470pF, Capacitors_SMD:C_0603, F.Cu at (182.2, 120.0)
- added C123: 470pF, Capacitors_SMD:C_0603, F.Cu at (169.8, 132.1)
- added C124: 100nF, Capacitors_SMD:C_0603, F.Cu at (176.6, 125.8)
- added C125: 100nF, Capacitors_SMD:C_0603, F.Cu at (166.2, 137.9)
- added C126: 100nF, Capacitors_SMD:C_0603, F.Cu at (181.7, 125.8)
- added C127: 10μF, Capacitors_SMD:C_0805, F.Cu at (160.1, 126.4)
- added C128: 100μF, Capacitors_SMD:c_elec_8x10, F.Cu at (152.3, 123.2)
- added C129: 100nF, Capacitors_SMD:C_0603, F.Cu at (174.9, 132.1)
- added C13: 100nF, Capacitors_SMD:C_0603, F.Cu at (262.2, 127.4)
- added C130: 100nF, Capacitors_SMD:C_0603, F.Cu at (226.1, 149.3)
- added C131: 470nF, Capacitors_SMD:C_0603, F.Cu at (204.9, 155.9)
- added C132: 100nF, Capacitors_SMD:C_0603, F.Cu at (225.5, 137.6)
- added C133: 4.7μF, Capacitors_SMD:C_0603, F.Cu at (215.0, 149.7)
- added C134: 22nF, Capacitors_SMD:C_0603, F.Cu at (220.6, 143.4)
- added C135: 470pF, Capacitors_SMD:C_0603, F.Cu at (210.1, 155.9)
- added C136: 470pF, Capacitors_SMD:C_0603, F.Cu at (204.9, 150.1)
- added C137: 100nF, Capacitors_SMD:C_0603, F.Cu at (230.6, 137.6)
- added C138: 470pF, Capacitors_SMD:C_0603, F.Cu at (221.0, 149.3)
- added C139: 470pF, Capacitors_SMD:C_0603, F.Cu at (215.3, 155.5)
- added C14: 2.2μF, Capacitors_SMD:C_0805, F.Cu at (261.1, 115.5)
- added C140: 100nF, Capacitors_SMD:C_0603, F.Cu at (235.8, 137.6)
- added C141: 100nF, Capacitors_SMD:C_0603, F.Cu at (230.5, 143.4)
- added C142: 100nF, Capacitors_SMD:C_0603, F.Cu at (225.4, 143.4)
- added C143: 10μF, Capacitors_SMD:C_0805, F.Cu at (208.9, 137.8)
- added C144: 100μF, Capacitors_SMD:c_elec_8x10, F.Cu at (201.1, 140.7)
- added C145: 100nF, Capacitors_SMD:C_0603, F.Cu at (235.7, 143.4)
- added C146: 100nF, Capacitors_SMD:C_0603, F.Cu at (226.7, 120.9)
- added C147: 470nF, Capacitors_SMD:C_0603, F.Cu at (226.6, 109.2)
- added C148: 100nF, Capacitors_SMD:C_0603, F.Cu at (216.4, 121.3)
- added C149: 4.7μF, Capacitors_SMD:C_0603, F.Cu at (220.6, 115.1)
- added C15: 100nF, Capacitors_SMD:C_0603, F.Cu at (274.9, 115.1)
- added C150: 22nF, Capacitors_SMD:C_0603, F.Cu at (211.6, 127.6)
- added C151: 470pF, Capacitors_SMD:C_0603, F.Cu at (225.6, 115.1)
- added C152: 470pF, Capacitors_SMD:C_0603, F.Cu at (206.2, 121.7)
- added C153: 100nF, Capacitors_SMD:C_0603, F.Cu at (216.4, 127.2)
- added C154: 470pF, Capacitors_SMD:C_0603, F.Cu at (221.6, 120.9)
- added C155: 470pF, Capacitors_SMD:C_0603, F.Cu at (236.0, 115.1)
- added C156: 100nF, Capacitors_SMD:C_0603, F.Cu at (237.0, 109.2)
- added C157: 100nF, Capacitors_SMD:C_0603, F.Cu at (230.8, 115.1)
- added C158: 100nF, Capacitors_SMD:C_0603, F.Cu at (231.8, 109.2)
- added C159: 10μF, Capacitors_SMD:C_0805, F.Cu at (210.2, 109.4)
- added C16: 100nF, Capacitors_SMD:C_0603, F.Cu at (266.4, 121.3)
- added C160: 100μF, Capacitors_SMD:c_elec_8x10, F.Cu at (202.4, 112.4)
- added C161: 100nF, Capacitors_SMD:C_0603, F.Cu at (221.6, 126.8)
- added C162: 100nF, Capacitors_SMD:C_0603, F.Cu at (158.0, 166.8)
- added C163: 470nF, Capacitors_SMD:C_0603, F.Cu at (167.2, 154.7)
- added C164: 100nF, Capacitors_SMD:C_0603, F.Cu at (158.3, 148.8)
- added C165: 4.7μF, Capacitors_SMD:C_0603, F.Cu at (142.7, 166.8)
- added C166: 22nF, Capacitors_SMD:C_0603, F.Cu at (163.1, 148.8)
- added C167: 470pF, Capacitors_SMD:C_0603, F.Cu at (153.1, 148.8)
- added C168: 470pF, Capacitors_SMD:C_0603, F.Cu at (160.3, 160.5)
- added C169: 100nF, Capacitors_SMD:C_0603, F.Cu at (151.7, 155.1)
- added C17: 2.2μF, Capacitors_SMD:C_0805, F.Cu at (256.2, 116.4)
- added C170: 470pF, Capacitors_SMD:C_0603, F.Cu at (156.9, 154.7)
- added C171: 470pF, Capacitors_SMD:C_0603, F.Cu at (152.9, 166.8)
- added C172: 100nF, Capacitors_SMD:C_0603, F.Cu at (167.9, 148.8)
- added C173: 100nF, Capacitors_SMD:C_0603, F.Cu at (155.1, 160.9)
- added C174: 100nF, Capacitors_SMD:C_0603, F.Cu at (162.0, 154.7)
- added C175: 10μF, Capacitors_SMD:C_0805, F.Cu at (141.0, 155.3)
- added C176: 100μF, Capacitors_SMD:c_elec_8x10, F.Cu at (133.3, 152.0)
- added C177: 100nF, Capacitors_SMD:C_0603, F.Cu at (147.7, 166.8)
- added C178: 100nF, Capacitors_SMD:C_0603, F.Cu at (251.1, 51.9)
- added C179: 470nF, Capacitors_SMD:C_0603, F.Cu at (245.5, 58.2)
- added C18: 100nF, Capacitors_SMD:C_0603, F.Cu at (261.2, 121.5)
- added C180: 100nF, Capacitors_SMD:C_0603, F.Cu at (231.6, 58.6)
- added C181: 4.7μF, Capacitors_SMD:C_0603, F.Cu at (241.0, 64.0)
- added C182: 22nF, Capacitors_SMD:C_0603, F.Cu at (255.9, 51.9)
- added C183: 470pF, Capacitors_SMD:C_0603, F.Cu at (250.7, 58.2)
- added C184: 470pF, Capacitors_SMD:C_0603, F.Cu at (263.5, 46.1)
- added C185: 100nF, Capacitors_SMD:C_0603, F.Cu at (246.0, 64.0)
- added C186: 470pF, Capacitors_SMD:C_0603, F.Cu at (255.8, 57.8)
- added C187: 470pF, Capacitors_SMD:C_0603, F.Cu at (260.7, 51.9)
- added C188: 100nF, Capacitors_SMD:C_0603, F.Cu at (251.1, 64.0)
- added C189: 100nF, Capacitors_SMD:C_0603, F.Cu at (261.0, 57.8)
- added C19: 2.2μF, Capacitors_SMD:C_0805, F.Cu at (252.8, 123.0)
- added C190: 100nF, Capacitors_SMD:C_0603, F.Cu at (240.3, 58.2)
- added C191: 10μF, Capacitors_SMD:C_0805, F.Cu at (235.6, 52.5)
- added C192: 100μF, Capacitors_SMD:c_elec_8x10, F.Cu at (227.8, 49.3)
- added C193: 100nF, Capacitors_SMD:C_0603, F.Cu at (247.6, 46.1)
- added C194: 100nF, Capacitors_SMD:C_0603, F.Cu at (299.2, 73.3)
- added C195: 470nF, Capacitors_SMD:C_0603, F.Cu at (304.6, 67.1)
- added C196: 100nF, Capacitors_SMD:C_0603, F.Cu at (290.7, 79.2)
- added C197: 4.7μF, Capacitors_SMD:C_0603, F.Cu at (294.2, 73.3)
- added C198: 22nF, Capacitors_SMD:C_0603, F.Cu at (299.8, 67.1)
- added C199: 470pF, Capacitors_SMD:C_0603, F.Cu at (306.8, 61.2)
- added C2: 10nF, Capacitors_SMD:C_0603, F.Cu at (156.3, 15.6)
- added C20: 4.7μF, Capacitors_SMD:C_0805, F.Cu at (267.8, 109.4)
- added C200: 470pF, Capacitors_SMD:C_0603, F.Cu at (285.6, 79.2)
- added C201: 100nF, Capacitors_SMD:C_0603, F.Cu at (301.6, 61.2)
- added C202: 470pF, Capacitors_SMD:C_0603, F.Cu at (295.0, 67.5)
- added C203: 470pF, Capacitors_SMD:C_0603, F.Cu at (295.9, 79.2)
- added C204: 100nF, Capacitors_SMD:C_0603, F.Cu at (312.0, 61.2)
- added C205: 100nF, Capacitors_SMD:C_0603, F.Cu at (296.5, 61.2)
- added C206: 100nF, Capacitors_SMD:C_0603, F.Cu at (289.2, 73.3)
- added C207: 10μF, Capacitors_SMD:C_0805, F.Cu at (284.4, 67.7)
- added C208: 100μF, Capacitors_SMD:c_elec_8x10, F.Cu at (276.6, 64.4)
- added C209: 100nF, Capacitors_SMD:C_0603, F.Cu at (280.4, 79.6)
- added C21: 100nF, Capacitors_SMD:C_0603, F.Cu at (281.6, 109.2)
- added C210: 100nF, Capacitors_SMD:C_0603, F.Cu at (222.6, 165.9)
- added C211: 4.7nF, Capacitors_SMD:C_0603, F.Cu at (81.9, 96.3)
- added C212: 4.7nF, Capacitors_SMD:C_0603, F.Cu at (74.3, 104.4)
- added C213: 4.7nF, Capacitors_SMD:C_0603, F.Cu at (57.3, 123.5)
- added C214: 4.7nF, Capacitors_SMD:C_0603, F.Cu at (64.8, 116.8)
- added C215: 4.7nF, Capacitors_SMD:C_0603, F.Cu at (52.6, 123.5)
- added C216: 4.7nF, Capacitors_SMD:C_0603, F.Cu at (118.3, 102.9)
- added C217: 4.7nF, Capacitors_SMD:C_0603, F.Cu at (118.2, 97.0)
- added C218: 4.7nF, Capacitors_SMD:C_0603, F.Cu at (118.8, 108.7)
- added C22: 100nF, Capacitors_SMD:C_0603, F.Cu at (271.5, 121.3)
- added C23: 220μF, Capacitors_Tantalum_SMD:TantalC_SizeD_EIA-7343_Reflow, F.Cu at (215.3, 81.9)
- added C24: 100nF, Capacitors_SMD:C_0603, F.Cu at (226.0, 92.5)
- added C25: 100nF, Capacitors_SMD:C_0603, F.Cu at (230.8, 80.5)
- added C26: 100nF, Capacitors_SMD:C_0603, F.Cu at (217.4, 89.5)
- added C27: 30pF, Capacitors_SMD:C_0603, F.Cu at (205.2, 46.1)
- added C28: 30pF, Capacitors_SMD:C_0603, F.Cu at (192.2, 58.2)
- added C29: 100nF, Capacitors_SMD:C_0603, F.Cu at (201.2, 51.9)
- added C3: 100nF, Capacitors_SMD:C_0603, F.Cu at (157.8, 8.71)
- added C30: 100nF, Capacitors_SMD:C_0603, F.Cu at (185.9, 69.5)
- added C31: 100nF, Capacitors_SMD:C_0603, F.Cu at (209.9, 46.1)
- added C32: 470pF, Capacitors_SMD:C_0603, F.Cu at (191.6, 64.0)
- added C33: 10μF, Capacitors_SMD:C_0805, F.Cu at (196.4, 46.3)
- added C34: 1μF, Capacitors_SMD:C_0603, F.Cu at (205.5, 51.9)
- added C35: DNP-15pF, Capacitors_SMD:C_0603, F.Cu at (167.6, 65.9)
- added C36: DNP-15pF, Capacitors_SMD:C_0603, F.Cu at (181.3, 55.6)
- added C37: DNP-15pF, Capacitors_SMD:C_0603, F.Cu at (190.0, 46.1)
- added C38: DNP-15pF, Capacitors_SMD:C_0603, F.Cu at (167.6, 60.1)
- added C39: 10μF, Capacitors_SMD:C_0603, F.Cu at (294.1, 119.6)
- added C4: 22nF, Capacitors_SMD:C_0603, F.Cu at (156.3, 21.4)
- added C40: 10μF, Capacitors_SMD:C_0603, F.Cu at (298.5, 113.7)
- added C41: 100nF, Capacitors_SMD:C_0603, F.Cu at (34.8, 142.6)
- added C42: 2.2μF, Capacitors_SMD:C_0805, F.Cu at (43.5, 135.6)
- added C43: 100nF, Capacitors_SMD:C_0603, F.Cu at (38.3, 154.3)
- added C44: 47pF, Capacitors_SMD:C_0603, F.Cu at (43.0, 159.2)
- added C45: 2.2μF, Capacitors_SMD:C_0603, F.Cu at (48.3, 135.4)
- added C46: 47pF, Capacitors_SMD:C_0603, F.Cu at (39.4, 142.6)
- added C47: 47pF, Capacitors_SMD:C_0603, F.Cu at (25.8, 161.4)
- added C48: 100nF, Capacitors_SMD:C_0603, F.Cu at (30.5, 155.5)
- added C49: 47pF, Capacitors_SMD:C_0603, F.Cu at (37.8, 148.4)
- added C5: 100nF, Capacitors_SMD:C_0603, F.Cu at (128.7, 50.3)
- added C50: 47pF, Capacitors_SMD:C_0603, F.Cu at (25.8, 155.5)
- added C51: 2.2μF, Capacitors_SMD:C_0603, F.Cu at (52.6, 147.1)
- added C52: 47pF, Capacitors_SMD:C_0603, F.Cu at (52.8, 135.4)
- added C53: 47pF, Capacitors_SMD:C_0603, F.Cu at (43.7, 147.5)
- added C54: 100nF, Capacitors_SMD:C_0603, F.Cu at (30.5, 161.3)
- added C55: 47pF, Capacitors_SMD:C_0603, F.Cu at (43.7, 141.7)
- added C56: 47pF, Capacitors_SMD:C_0603, F.Cu at (48.0, 141.3)
- added C57: 2.2μF, Capacitors_SMD:C_0805, F.Cu at (29.8, 142.8)
- added C58: 47pF, Capacitors_SMD:C_0603, F.Cu at (55.7, 153.0)
- added C59: 47pF, Capacitors_SMD:C_0603, F.Cu at (47.2, 159.2)
- added C6: 2.2μF, Capacitors_SMD:C_0603, F.Cu at (225.0, 16.5)
- added C60: 47pF, Capacitors_SMD:C_0603, F.Cu at (64.0, 141.3)
- added C61: 47pF, Capacitors_SMD:C_0603, F.Cu at (51.4, 153.0)
- added C62: 47pF, Capacitors_SMD:C_0603, F.Cu at (57.1, 147.1)
- added C63: 47pF, Capacitors_SMD:C_0603, F.Cu at (57.0, 135.4)
- added C64: 47pF, Capacitors_SMD:C_0603, F.Cu at (35.2, 160.1)
- added C65: 18pF, Capacitors_SMD:C_0603, F.Cu at (192.5, 173.6)
- added C66: 18pF, Capacitors_SMD:C_0603, F.Cu at (200.7, 165.9)
- added C67: 18pF, Capacitors_SMD:C_0603, F.Cu at (205.0, 165.9)
- added C68: 18pF, Capacitors_SMD:C_0603, F.Cu at (196.7, 171.7)
- added C69: 4.7μF, Capacitors_SMD:C_0603, F.Cu at (91.8, 173.0)
- added C7: 100nF, Capacitors_SMD:C_0603, F.Cu at (207.8, 31.7)
- added C70: 4.7μF, Capacitors_SMD:C_0603, F.Cu at (91.8, 167.2)
- added C71: 0.1μF, Capacitors_SMD:C_0603, F.Cu at (180.8, 96.3)
- added C72: 0.1μF, Capacitors_SMD:C_0603, F.Cu at (165.0, 104.5)
- added C73: 0.1μF, Capacitors_SMD:C_0603, F.Cu at (179.2, 108.0)
- added C74: 0.1μF, Capacitors_SMD:C_0603, F.Cu at (174.4, 104.5)
- added C75: 0.1μF, Capacitors_SMD:C_0603, F.Cu at (169.9, 110.4)
- added C76: 100nF, Capacitors_SMD:C_0603, F.Cu at (254.5, 152.6)
- added C77: 100nF, Capacitors_SMD:C_0603, F.Cu at (277.8, 137.6)
- added C78: 100nF, Capacitors_SMD:C_0603, F.Cu at (267.8, 137.6)
- added C79: 100nF, Capacitors_SMD:C_0603, F.Cu at (262.9, 143.4)
- added C8: 470μF, KiMBo:c_elec_16x16.5, F.Cu at (247.6, 7.31)
- added C80: 100nF, Capacitors_SMD:C_0603, F.Cu at (254.5, 146.7)
- added C81: 100nF, Capacitors_SMD:C_0603, F.Cu at (259.7, 149.3)
- added C82: 100nF, Capacitors_SMD:C_0603, F.Cu at (280.4, 45.1)
- added C83: 470nF, Capacitors_SMD:C_0603, F.Cu at (285.6, 45.1)
- added C84: 100nF, Capacitors_SMD:C_0603, F.Cu at (280.4, 51.0)
- added C85: 4.7μF, Capacitors_SMD:C_0603, F.Cu at (295.7, 44.3)
- added C86: 22nF, Capacitors_SMD:C_0603, F.Cu at (300.4, 32.6)
- added C87: 470pF, Capacitors_SMD:C_0603, F.Cu at (295.8, 38.5)
- added C88: 470pF, Capacitors_SMD:C_0603, F.Cu at (300.9, 38.5)
- added C89: 100nF, Capacitors_SMD:C_0603, F.Cu at (305.1, 32.6)
- added C9: 220μF, KiMBo:c_elec_8x10.2, F.Cu at (263.0, 19.8)
- added C90: 470pF, Capacitors_SMD:C_0603, F.Cu at (290.7, 44.7)
- added C91: 470pF, Capacitors_SMD:C_0603, F.Cu at (285.6, 51.0)
- added C92: 100nF, Capacitors_SMD:C_0603, F.Cu at (305.6, 44.3)
- added C93: 100nF, Capacitors_SMD:C_0603, F.Cu at (290.6, 38.9)
- added C94: 100nF, Capacitors_SMD:C_0603, F.Cu at (311.2, 38.5)
- added C95: 10μF, Capacitors_SMD:C_0805, F.Cu at (284.4, 32.8)
- added C96: 100μF, Capacitors_SMD:c_elec_8x10, F.Cu at (276.6, 35.8)
- added C97: 100nF, Capacitors_SMD:C_0603, F.Cu at (306.1, 38.5)
- added C98: 100nF, Capacitors_SMD:C_0603, F.Cu at (306.6, 15.0)
- added C99: 470nF, Capacitors_SMD:C_0603, F.Cu at (322.1, 14.6)
- added D1: LED, LEDs:LED_0603, F.Cu at (84.5, 32.2)
- added D10: LED, LEDs:LED_0603, F.Cu at (206.4, 2.46)
- added D11: DNP-TLVH431, TO_SOT_Packages_SMD:SOT-23, F.Cu at (184.6, 34.3)
- added D12: SK54A-LTP, KiMBo:SK-DO-214AC, F.Cu at (279.9, 3.89)
- added D13: D5V0F1U2S9, KiMBo:SOD-923, F.Cu at (273.8, 16.2)
- added D14: SMAZ10, KiMBo:SMA-DO-214AC, F.Cu at (114.1, 156.4)
- added D15: SMAJ26A, KiMBo:SK-DO-214AC, F.Cu at (99.9, 156.6)
- added D16: RB751V40,115, Diodes_SMD:SOD-323, F.Cu at (29.9, 149.6)
- added D17: TPD1E04U04DPYR, KiMBo:TPD_PX1SON, F.Cu at (153.7, 111.2)
- added D18: SK1545-TP, KiMBo:SK-DO-214AB, F.Cu at (43.9, 107.2)
- added D19: LED, LEDs:LED_0603, F.Cu at (22.2, 126.5)
- added D2: LED, LEDs:LED_0603, F.Cu at (87.8, 32.2)
- added D20: MBRA340T3, KiMBo:MBR-DO-214AC, F.Cu at (24.0, 119.8)
- added D21: MBRA340T3, KiMBo:MBR-DO-214AC, F.Cu at (69.0, 91.5)
- added D22: LED, LEDs:LED_0603, F.Cu at (82.8, 101.7)
- added D23: LED, LEDs:LED_0603, F.Cu at (32.6, 126.5)
- added D24: MBRA340T3, KiMBo:MBR-DO-214AC, F.Cu at (31.1, 119.8)
- added D25: MBRA340T3, KiMBo:MBR-DO-214AC, F.Cu at (53.5, 98.1)
- added D26: LED, LEDs:LED_0603, F.Cu at (29.1, 126.5)
- added D27: LED, LEDs:LED_0603, F.Cu at (25.7, 126.5)
- added D28: MBRA340T3, KiMBo:MBR-DO-214AC, F.Cu at (91.1, 110.6)
- added D29: LED, LEDs:LED_0603, F.Cu at (122.3, 102.5)
- added D3: LED, LEDs:LED_0603, F.Cu at (107.3, 46.9)
- added D30: MBRA340T3, KiMBo:MBR-DO-214AC, F.Cu at (101.6, 104.3)
- added D31: LED, LEDs:LED_0603, F.Cu at (112.5, 116.4)
- added D32: MBRA340T3, KiMBo:MBR-DO-214AC, F.Cu at (112.3, 98.1)
- added D33: LED, LEDs:LED_0603, F.Cu at (141.6, 90.0)
- added D4: LED, LEDs:LED_0603, F.Cu at (110.6, 46.9)
- added D5: TPD1E04U04DPYR, KiMBo:TPD_PX1SON, F.Cu at (64.1, 81.5)
- added D6: D5V0F1U2S9, KiMBo:SOD-923, F.Cu at (68.6, 37.7)
- added D7: D5V0F1U2S9, KiMBo:SOD-923, F.Cu at (76.0, 81.5)
- added D8: TLVH431, TO_SOT_Packages_SMD:SOT-23, F.Cu at (226.2, 3.21)
- added D9: TPD1E04U04DPYR, KiMBo:TPD_PX1SON, F.Cu at (197.8, 2.46)
- added F1: 0891020.NXS, KiMBo:3557-2-Fuseholder, F.Cu at (86.2, 138.6)
- added F2: 1206L025YR, KiMBo:F_1206, F.Cu at (14.9, 163.1)
- added FB1: MPZ1608S102ATA00, KiMBo:Ferrite_Bead_0603, F.Cu at (33.9, 76.5)
- added FB10: MMZ1608A252BTA00, KiMBo:Ferrite_Bead_0603, F.Cu at (31.8, 62.4)
- added FB11: MMZ1608A252BTA00, KiMBo:Ferrite_Bead_0603, F.Cu at (71.7, 24.4)
- added FB12: MMZ1608A252BTA00, KiMBo:Ferrite_Bead_0603, F.Cu at (18.1, 80.1)
- added FB13: MMZ1608A252BTA00, KiMBo:Ferrite_Bead_0603, F.Cu at (75.6, 17.4)
- added FB14: MMZ1608A252BTA00, KiMBo:Ferrite_Bead_0603, F.Cu at (69.1, 43.9)
- added FB15: MMZ1608A252BTA00, KiMBo:Ferrite_Bead_0603, F.Cu at (51.2, 50.9)
- added FB16: MMZ1608A252BTA00, KiMBo:Ferrite_Bead_0603, F.Cu at (91.4, 10.3)
- added FB17: MMZ1608A252BTA00, KiMBo:Ferrite_Bead_0603, F.Cu at (71.7, 31.5)
- added FB18: MPZ1608S102ATA00, KiMBo:Ferrite_Bead_0603, F.Cu at (49.5, 76.5)
- added FB19: MMZ1608A252BTA00, KiMBo:Ferrite_Bead_0603, F.Cu at (33.9, 69.5)
- added FB2: MMZ1608A252BTA00, KiMBo:Ferrite_Bead_0603, F.Cu at (18.1, 73.1)
- added FB20: MPZ1608S102ATA00, KiMBo:Ferrite_Bead_0603, F.Cu at (99.8, 34.6)
- added FB21: MPZ1608S102ATA00, KiMBo:Ferrite_Bead_0603, F.Cu at (171.4, 34.4)
- added FB22: BLM31SN500SN1L, Resistors_SMD:R_1206_HandSoldering, F.Cu at (103.6, 149.3)
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
Commit message: Begin layout
Arrange all connectors to get a feel for the area.
Parts:
- removed P38: PWR_Input, KiMBo:euro_header_4_angled
- added C219: 4.7nF, Capacitors_SMD:C_0603, F.Cu at (144.1, -276.5)
- added C220: 4.7nF, Capacitors_SMD:C_0603, F.Cu at (148.8, -276.5)
- added D34: LED, LEDs:LED_0603, F.Cu at (152.8, -276.9)
- added REF** (x2): MountingHole_3mm_Pad, KiMBo:MountingHole_3mm_Pad, F.Cu at (255.0, 46.0)
- added REF**: MountingHole_3mm_Pad, KiMBo:MountingHole_3mm_Pad, F.Cu at (227.0, 155.0)
- added REF**: MountingHole_3mm_Pad, KiMBo:MountingHole_3mm_Pad, F.Cu at (69.0, 168.0)
- added REF**: MountingHole_3mm_Pad, KiMBo:MountingHole_3mm_Pad, F.Cu at (57.0, 28.0)
- C10: value 22μF -> 470μF; footprint Capacitors_SMD:C_0805 -> KiMBo:c_elec_16x16.5
- C101, C117, C133, C149, C165, C181, C197, C85: value 4.7μF -> 470nF
- C102, C118, C134, C150, C166, C182, C198, C86: value 22nF -> 100nF
- C103, C119, C135, C151, C167, C183, C199, C87: value 470pF -> 4.7μF
- C104, C120, C136, C152, C168, C184, C200, C88: value 470pF -> 22nF
- C105, C108, C109, C121, C124, C125, C137, C140, C141, C153, C156, C157, C169, C172, C173, C185, C188, C189, C201, C204, C205, C89, C92, C93: value 100nF -> 470pF
- C107, C123, C139, C155, C171, C187, C203, C32, C91: value 470pF -> 100nF
- C11: value 22μF -> 220μF; footprint Capacitors_SMD:C_0805 -> KiMBo:c_elec_8x10.2
- C111, C127, C143, C159, C175, C191, C207, C33, C95: value 10μF -> 100nF; footprint Capacitors_SMD:C_0805 -> Capacitors_SMD:C_0603
- C112, C128, C144, C160, C176, C192, C208, C96: value 100μF -> 100nF; footprint Capacitors_SMD:c_elec_8x10 -> Capacitors_SMD:C_0603
- C113, C129, C145, C161, C177, C193, C209, C97: value 100nF -> 10μF; footprint Capacitors_SMD:C_0603 -> Capacitors_SMD:C_0805
- C114, C130, C146, C162, C178, C194, C210, C98: value 100nF -> 100μF; footprint Capacitors_SMD:C_0603 -> Capacitors_SMD:c_elec_8x10
- C115, C131, C147, C163, C179, C195, C83, C99: value 470nF -> 100nF
- C12, C13: value 100nF -> 22μF; footprint Capacitors_SMD:C_0603 -> Capacitors_SMD:C_0805
- C14, C17: value 2.2μF -> 100nF; footprint Capacitors_SMD:C_0805 -> Capacitors_SMD:C_0603
- C16, C21: value 100nF -> 2.2μF; footprint Capacitors_SMD:C_0603 -> Capacitors_SMD:C_0805
- C2: value 10nF -> 100nF
- C20: value 4.7μF -> 100nF; footprint Capacitors_SMD:C_0805 -> Capacitors_SMD:C_0603
- C211, C212: value 4.7nF -> 100nF
- C22: value 100nF -> 4.7μF; footprint Capacitors_SMD:C_0603 -> Capacitors_SMD:C_0805
- C23: value 220μF -> 100nF; footprint Capacitors_Tantalum_SMD:TantalC_SizeD_EIA-7343_Reflow -> Capacitors_SMD:C_0603
- C25: value 100nF -> 220μF; footprint Capacitors_SMD:C_0603 -> Capacitors_Tantalum_SMD:TantalC_SizeD_EIA-7343_Reflow
- C27, C28: value 30pF -> 100nF
- C29, C30: value 100nF -> 30pF
- C3: value 100nF -> 10nF
- C34: value 1μF -> 470pF
- C35: value DNP-15pF -> 10μF; footprint Capacitors_SMD:C_0603 -> Capacitors_SMD:C_0805
- C36: value DNP-15pF -> 1μF
- C39, C40: value 10μF -> DNP-15pF
- C4: value 22nF -> 10nF
- C41: value 100nF -> 10μF
- C42: value 2.2μF -> 10μF; footprint Capacitors_SMD:C_0805 -> Capacitors_SMD:C_0603
- C44, C59: value 47pF -> 2.2μF; footprint Capacitors_SMD:C_0603 -> Capacitors_SMD:C_0805
- C45: value 2.2μF -> 100nF
- C47, C53: value 47pF -> 2.2μF
- C48, C54: value 100nF -> 47pF
- C50, C56: value 47pF -> 100nF
- C51: value 2.2μF -> 47pF
- C57: value 2.2μF -> 47pF; footprint Capacitors_SMD:C_0805 -> Capacitors_SMD:C_0603
- C6: value 2.2μF -> 22nF
- C65, C66: value 18pF -> 47pF
- C69, C70: value 4.7μF -> 18pF
- C71, C72: value 0.1μF -> 4.7μF
- C76, C77: value 100nF -> 0.1μF
- C8: value 470μF -> 2.2μF; footprint KiMBo:c_elec_16x16.5 -> Capacitors_SMD:C_0603
- C9: value 220μF -> 100nF; footprint KiMBo:c_elec_8x10.2 -> Capacitors_SMD:C_0603
- D1: value LED -> D5V0F1U2S9; footprint LEDs:LED_0603 -> KiMBo:SOD-923
- D10, D2: value LED -> TPD1E04U04DPYR; footprint LEDs:LED_0603 -> KiMBo:TPD_PX1SON
- D11: value DNP-TLVH431 -> LED; footprint TO_SOT_Packages_SMD:SOT-23 -> LEDs:LED_0603
- D12: value SK54A-LTP -> DNP-TLVH431; footprint KiMBo:SK-DO-214AC -> TO_SOT_Packages_SMD:SOT-23
- D13: value D5V0F1U2S9 -> SK54A-LTP; footprint KiMBo:SOD-923 -> KiMBo:SK-DO-214AC
- D14: value SMAZ10 -> D5V0F1U2S9; footprint KiMBo:SMA-DO-214AC -> KiMBo:SOD-923
- D15: value SMAJ26A -> SMAZ10; footprint KiMBo:SK-DO-214AC -> KiMBo:SMA-DO-214AC
- D16: value RB751V40,115 -> SMAJ26A; footprint Diodes_SMD:SOD-323 -> KiMBo:SK-DO-214AC
- D17: value TPD1E04U04DPYR -> RB751V40,115; footprint KiMBo:TPD_PX1SON -> Diodes_SMD:SOD-323
- D18: value SK1545-TP -> TPD1E04U04DPYR; footprint KiMBo:SK-DO-214AB -> KiMBo:TPD_PX1SON
- D19: value LED -> SK1545-TP; footprint LEDs:LED_0603 -> KiMBo:SK-DO-214AB
- D20, D24, D28, D30, D32: value MBRA340T3 -> LED; footprint KiMBo:MBR-DO-214AC -> LEDs:LED_0603
- D22, D26, D29, D31, D33: value LED -> MBRA340T3; footprint LEDs:LED_0603 -> KiMBo:MBR-DO-214AC
- D5: value TPD1E04U04DPYR -> LED; footprint KiMBo:TPD_PX1SON -> LEDs:LED_0603
- D6: value D5V0F1U2S9 -> LED; footprint KiMBo:SOD-923 -> LEDs:LED_0603
- D8: value TLVH431 -> D5V0F1U2S9; footprint TO_SOT_Packages_SMD:SOT-23 -> KiMBo:SOD-923
- D9: value TPD1E04U04DPYR -> TLVH431; footprint KiMBo:TPD_PX1SON -> TO_SOT_Packages_SMD:SOT-23
- FB18, FB20: value MPZ1608S102ATA00 -> MMZ1608A252BTA00
- FB19, FB2: value MMZ1608A252BTA00 -> MPZ1608S102ATA00
- P1: value BED_THERM -> TOOLHEAD0; footprint Pin_Headers:Pin_Header_Angled_1x02 -> Pin_Headers:Pin_Header_Angled_1x08
- P10: value ENC -> ADC
- P15, P17: moved to B.Cu
- P2: value ADC -> TOOLHEAD1; footprint Pin_Headers:Pin_Header_Angled_1x02 -> Pin_Headers:Pin_Header_Angled_1x08
- P3: value TOOLHEAD0 -> DOCK0; footprint Pin_Headers:Pin_Header_Angled_1x07 -> Pin_Headers:Pin_Header_Angled_1x08
- P37: value HS_FAN -> PWR_Input; footprint Pin_Headers:Pin_Header_Angled_1x02 -> KiMBo:euro_header_4_angled
- P4: value TOOLHEAD1 -> DOCK1; footprint Pin_Headers:Pin_Header_Angled_1x07 -> Pin_Headers:Pin_Header_Angled_1x08
- P5: value DOCK0 -> X1; footprint Pin_Headers:Pin_Header_Angled_1x07 -> Pin_Headers:Pin_Header_Angled_1x02
- P6: value DOCK1 -> Y1; footprint Pin_Headers:Pin_Header_Angled_1x07 -> Pin_Headers:Pin_Header_Angled_1x02
- P7: value X1 -> Z1
- P8: value Y1 -> ENC
- P9: value Z1 -> BED_THERM
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Connections:
- C100 pad 1: CGND -> VCC
- C100 pad 2: +24V -> CGND
- C101 pad 1: /Stepper Drivers/X0 Stepper Driver/5VOUT -> Net-(C101-Pad1)
- C102 pad 1: Net-(C102-Pad1) -> CGND
- C102 pad 2: Net-(C102-Pad2) -> +24V
- C103 pad 1: /Stepper Drivers/X0_A2 -> /Stepper Drivers/X0 Stepper Driver/5VOUT
- C104 pad 1: /Stepper Drivers/X0_B2 -> Net-(C104-Pad1)
- C104 pad 2: CGND -> Net-(C104-Pad2)
- C105 pad 1: +24V -> /Stepper Drivers/X0_A2
- C105 pad 2: Net-(C105-Pad2) -> CGND
- C106 pad 1: /Stepper Drivers/X0_A1 -> /Stepper Drivers/X0_B2
- C107 pad 1: /Stepper Drivers/X0_B1 -> +24V
- C107 pad 2: CGND -> Net-(C107-Pad2)
- C108 pad 1: +24V -> /Stepper Drivers/X0_A1
- C109 pad 1: +24V -> /Stepper Drivers/X0_B1
- C11 pad 1: +24V -> VDD_5V
- C110 pad 1: Net-(C110-Pad1) -> +24V
- C112 pad 1: +24V -> Net-(C112-Pad1)
- C113 pad 1: Net-(C113-Pad1) -> +24V
- C114 pad 1: VCC -> +24V
- C116 pad 1: CGND -> VCC
- C116 pad 2: +24V -> CGND
- C117 pad 1: /Stepper Drivers/Z0 Stepper Driver/5VOUT -> Net-(C117-Pad1)
- C118 pad 1: Net-(C118-Pad1) -> CGND
- C118 pad 2: Net-(C118-Pad2) -> +24V
- C119 pad 1: /Stepper Drivers/Z0_A2 -> /Stepper Drivers/Z0 Stepper Driver/5VOUT
- C12 pad 1: VCC -> +24V
- C120 pad 1: /Stepper Drivers/Z0_B2 -> Net-(C120-Pad1)
- C120 pad 2: CGND -> Net-(C120-Pad2)
- C121 pad 1: +24V -> /Stepper Drivers/Z0_A2
- C121 pad 2: Net-(C121-Pad2) -> CGND
- C122 pad 1: /Stepper Drivers/Z0_A1 -> /Stepper Drivers/Z0_B2
- C123 pad 1: /Stepper Drivers/Z0_B1 -> +24V
- C123 pad 2: CGND -> Net-(C123-Pad2)
- C124 pad 1: +24V -> /Stepper Drivers/Z0_A1
- C125 pad 1: +24V -> /Stepper Drivers/Z0_B1
- C126 pad 1: Net-(C126-Pad1) -> +24V
- C128 pad 1: +24V -> Net-(C128-Pad1)
- C129 pad 1: Net-(C129-Pad1) -> +24V
- C13 pad 1: VCC -> +24V
- C130 pad 1: VCC -> +24V
- C132 pad 1: CGND -> VCC
- C132 pad 2: +24V -> CGND
- C133 pad 1: /Stepper Drivers/Z1 Stepper Driver/5VOUT -> Net-(C133-Pad1)
- C134 pad 1: Net-(C134-Pad1) -> CGND
- C134 pad 2: Net-(C134-Pad2) -> +24V
- C135 pad 1: /Stepper Drivers/Z1_A2 -> /Stepper Drivers/Z1 Stepper Driver/5VOUT
- C136 pad 1: /Stepper Drivers/Z1_B2 -> Net-(C136-Pad1)
- C136 pad 2: CGND -> Net-(C136-Pad2)
- C137 pad 1: +24V -> /Stepper Drivers/Z1_A2
- C137 pad 2: Net-(C137-Pad2) -> CGND
- C138 pad 1: /Stepper Drivers/Z1_A1 -> /Stepper Drivers/Z1_B2
- C139 pad 1: /Stepper Drivers/Z1_B1 -> +24V
- C139 pad 2: CGND -> Net-(C139-Pad2)
- C14 pad 1: CGND -> VCC
- C140 pad 1: +24V -> /Stepper Drivers/Z1_A1
- C141 pad 1: +24V -> /Stepper Drivers/Z1_B1
- C142 pad 1: Net-(C142-Pad1) -> +24V
- C144 pad 1: +24V -> Net-(C144-Pad1)
- C145 pad 1: Net-(C145-Pad1) -> +24V
- C146 pad 1: VCC -> +24V
- C148 pad 1: CGND -> VCC
- C148 pad 2: +24V -> CGND
- C149 pad 1: /Stepper Drivers/Z2 Stepper Driver/5VOUT -> Net-(C149-Pad1)
- C150 pad 1: Net-(C150-Pad1) -> CGND
- C150 pad 2: Net-(C150-Pad2) -> +24V
- C151 pad 1: /Stepper Drivers/Z2_A2 -> /Stepper Drivers/Z2 Stepper Driver/5VOUT
- C152 pad 1: /Stepper Drivers/Z2_B2 -> Net-(C152-Pad1)
- C152 pad 2: CGND -> Net-(C152-Pad2)
- C153 pad 1: +24V -> /Stepper Drivers/Z2_A2
- C153 pad 2: Net-(C153-Pad2) -> CGND
- C154 pad 1: /Stepper Drivers/Z2_A1 -> /Stepper Drivers/Z2_B2
- C155 pad 1: /Stepper Drivers/Z2_B1 -> +24V
- C155 pad 2: CGND -> Net-(C155-Pad2)
- C156 pad 1: +24V -> /Stepper Drivers/Z2_A1
- C157 pad 1: +24V -> /Stepper Drivers/Z2_B1
- C158 pad 1: Net-(C158-Pad1) -> +24V
- C160 pad 1: +24V -> Net-(C160-Pad1)
- C161 pad 1: Net-(C161-Pad1) -> +24V
- C162 pad 1: VCC -> +24V
- C164 pad 1: CGND -> VCC
- C164 pad 2: +24V -> CGND
- C165 pad 1: /Stepper Drivers/H Stepper Driver/5VOUT -> Net-(C165-Pad1)
- C166 pad 1: Net-(C166-Pad1) -> CGND
- C166 pad 2: Net-(C166-Pad2) -> +24V
- C167 pad 1: /Stepper Drivers/H_A2 -> /Stepper Drivers/H Stepper Driver/5VOUT
- C168 pad 1: /Stepper Drivers/H_B2 -> Net-(C168-Pad1)
- C168 pad 2: CGND -> Net-(C168-Pad2)
- C169 pad 1: +24V -> /Stepper Drivers/H_A2
- C169 pad 2: Net-(C169-Pad2) -> CGND
- C17 pad 1: CGND -> VCC
- C170 pad 1: /Stepper Drivers/H_A1 -> /Stepper Drivers/H_B2
- C171 pad 1: /Stepper Drivers/H_B1 -> +24V
- C171 pad 2: CGND -> Net-(C171-Pad2)
- C172 pad 1: +24V -> /Stepper Drivers/H_A1
- C173 pad 1: +24V -> /Stepper Drivers/H_B1
- C174 pad 1: Net-(C174-Pad1) -> +24V
- C176 pad 1: +24V -> Net-(C176-Pad1)
- C177 pad 1: Net-(C177-Pad1) -> +24V
- C178 pad 1: VCC -> +24V
- C180 pad 1: CGND -> VCC
- C180 pad 2: +24V -> CGND
- C181 pad 1: /Stepper Drivers/Y Stepper Driver/5VOUT -> Net-(C181-Pad1)
- C182 pad 1: Net-(C182-Pad1) -> CGND
- C182 pad 2: Net-(C182-Pad2) -> +24V
- C183 pad 1: /Stepper Drivers/Y_A2 -> /Stepper Drivers/Y Stepper Driver/5VOUT
- C184 pad 1: /Stepper Drivers/Y_B2 -> Net-(C184-Pad1)
- C184 pad 2: CGND -> Net-(C184-Pad2)
- C185 pad 1: +24V -> /Stepper Drivers/Y_A2
- C185 pad 2: Net-(C185-Pad2) -> CGND
- C186 pad 1: /Stepper Drivers/Y_A1 -> /Stepper Drivers/Y_B2
- C187 pad 1: /Stepper Drivers/Y_B1 -> +24V
- C187 pad 2: CGND -> Net-(C187-Pad2)
- C188 pad 1: +24V -> /Stepper Drivers/Y_A1
- C189 pad 1: +24V -> /Stepper Drivers/Y_B1
- C190 pad 1: Net-(C190-Pad1) -> +24V
- C192 pad 1: +24V -> Net-(C192-Pad1)
- C193 pad 1: Net-(C193-Pad1) -> +24V
- C194 pad 1: VCC -> +24V
- C196 pad 1: CGND -> VCC
- C196 pad 2: +24V -> CGND
- C197 pad 1: /Stepper Drivers/X1 Stepper Driver/5VOUT -> Net-(C197-Pad1)
- C198 pad 1: Net-(C198-Pad1) -> CGND
- C198 pad 2: Net-(C198-Pad2) -> +24V
- C199 pad 1: /Stepper Drivers/X1_A2 -> /Stepper Drivers/X1 Stepper Driver/5VOUT
- C2 pad 1: /3V3_FILTERED -> Net-(C2-Pad1)
- C20 pad 1: Net-(C20-Pad1) -> CGND
- C200 pad 1: /Stepper Drivers/X1_B2 -> Net-(C200-Pad1)
- C200 pad 2: CGND -> Net-(C200-Pad2)
- C201 pad 1: +24V -> /Stepper Drivers/X1_A2
- C201 pad 2: Net-(C201-Pad2) -> CGND
- C202 pad 1: /Stepper Drivers/X1_A1 -> /Stepper Drivers/X1_B2
- C203 pad 1: /Stepper Drivers/X1_B1 -> +24V
- C203 pad 2: CGND -> Net-(C203-Pad2)
- C204 pad 1: +24V -> /Stepper Drivers/X1_A1
- C205 pad 1: +24V -> /Stepper Drivers/X1_B1
- C206 pad 1: Net-(C206-Pad1) -> +24V
- C208 pad 1: +24V -> Net-(C208-Pad1)
- C209 pad 1: Net-(C209-Pad1) -> +24V
- C21 pad 1: Net-(C20-Pad1) -> CGND
- C210 pad 1: VCC -> +24V
- C211 pad 1: +24V -> Net-(C211-Pad1)
- C211 pad 2: /Heaters/BED_HEAT -> CGND
- C212 pad 1: +24V -> VCC
- C212 pad 2: /Heaters/E_HEAT -> CGND
- C213 pad 2: /Heaters/DOCK0_HEAT -> /Heaters/BED_HEAT
- C214 pad 2: /Heaters/H_HEAT -> /Heaters/E_HEAT
- C215 pad 2: /Heaters/DOCK1_HEAT -> /Heaters/DOCK0_HEAT
- C216 pad 2: /Fans/E_FAN -> /Heaters/H_HEAT
- C217 pad 2: /Fans/H_FAN -> /Heaters/DOCK1_HEAT
- C218 pad 2: /Fans/CASE_FAN -> /Fans/E_FAN
- C22 pad 1: VCC -> Net-(C22-Pad1)
- C23 pad 1: SYS_5V -> Net-(C22-Pad1)
- C24 pad 1: Net-(C24-Pad1) -> VCC
- C25 pad 1: USB_DC -> SYS_5V
- C26 pad 1: VCC -> Net-(C26-Pad1)
- C27 pad 1: Net-(C27-Pad1) -> USB_DC
- C28 pad 1: Net-(C28-Pad1) -> VCC
- C29 pad 1: VCC -> Net-(C29-Pad1)
- C3 pad 1: /~SYS_RESET -> /3V3_FILTERED
- C30 pad 1: VDD_PHYA -> Net-(C30-Pad1)
- C31 pad 1: VDD_PHYA -> VCC
- C32 pad 1: /Ethernet/PHY_VDDCR -> VDD_PHYA
- C35 pad 1: /Ethernet/RD+ -> VDD_PHYA
- C36 pad 1: /Ethernet/RD- -> /Ethernet/PHY_VDDCR
- C37 pad 1: /Ethernet/TD+ -> /Ethernet/RD+
- C38 pad 1: /Ethernet/TD- -> /Ethernet/RD-
- C39 pad 1: VCC -> /Ethernet/TD+
- C4 pad 1: Net-(C4-Pad1) -> Net-(C2-Pad1)
- C40 pad 1: VCC -> /Ethernet/TD-
- C41 pad 1: HDMI_1V8 -> VCC
- C41 pad 2: Net-(C41-Pad2) -> CGND
- C42 pad 1: HDMI_1V8 -> VCC
- C42 pad 2: Net-(C41-Pad2) -> CGND
- C43 pad 2: Net-(C41-Pad2) -> Net-(C43-Pad2)
- C44 pad 1: /HDMI/LCD.D15.R4--R7 -> HDMI_1V8
- C44 pad 2: CGND -> Net-(C43-Pad2)
- C45 pad 2: Net-(C41-Pad2) -> Net-(C43-Pad2)
- C46 pad 1: /HDMI/LCD.D14.R3--R6 -> /HDMI/LCD.D15.R4--R7
- C47 pad 1: /HDMI/LCD.D13.R2--R5 -> HDMI_1V8
- C47 pad 2: CGND -> Net-(C43-Pad2)
- C48 pad 1: HDMI_1V8 -> /HDMI/LCD.D14.R3--R6
- C48 pad 2: Net-(C41-Pad2) -> CGND
- C49 pad 1: /HDMI/LCD.D12.R1--R4 -> /HDMI/LCD.D13.R2--R5
- C5 pad 1: VCC -> /~SYS_RESET
- C50 pad 1: /HDMI/LCD.D11.R0--R3 -> HDMI_1V8
- C50 pad 2: CGND -> Net-(C43-Pad2)
- C51 pad 1: HDMI_1V8 -> /HDMI/LCD.D12.R1--R4
- C51 pad 2: Net-(C41-Pad2) -> CGND
- C52 pad 1: /HDMI/LCD.D10.G5--G7 -> /HDMI/LCD.D11.R0--R3
- C53 pad 1: /HDMI/LCD.D9.G4--G6 -> HDMI_1V8
- C53 pad 2: CGND -> Net-(C43-Pad2)
- C54 pad 1: HDMI_1V8 -> /HDMI/LCD.D10.G5--G7
- C54 pad 2: Net-(C41-Pad2) -> CGND
- C55 pad 1: /HDMI/LCD.D8.G3--G5 -> /HDMI/LCD.D9.G4--G6
- C56 pad 1: /HDMI/LCD.D7.G2--G4 -> HDMI_1V8
- C56 pad 2: CGND -> Net-(C43-Pad2)
- C57 pad 1: HDMI_1V8 -> /HDMI/LCD.D8.G3--G5
- C57 pad 2: Net-(C41-Pad2) -> CGND
- C58 pad 1: /HDMI/LCD.D6.G1--G3 -> /HDMI/LCD.D7.G2--G4
- C59 pad 1: /HDMI/LCD.D5.G0--G2 -> HDMI_1V8
- C59 pad 2: CGND -> Net-(C43-Pad2)
- C6 pad 1: /~SYS_RESET -> Net-(C6-Pad1)
- C60 pad 1: /HDMI/LCD.D4.B4--B7 -> /HDMI/LCD.D6.G1--G3
- C61 pad 1: /HDMI/LCD.D3.B3--B6 -> /HDMI/LCD.D5.G0--G2
- C62 pad 1: /HDMI/LCD.D2.B2--B5 -> /HDMI/LCD.D4.B4--B7
- C63 pad 1: /HDMI/LCD.D1.B1--B4 -> /HDMI/LCD.D3.B3--B6
- C64 pad 1: /HDMI/LCD.D0.B0--B3 -> /HDMI/LCD.D2.B2--B5
- C65 pad 1: Net-(C65-Pad1) -> /HDMI/LCD.D1.B1--B4
- C65 pad 2: Net-(C65-Pad2) -> CGND
- C66 pad 1: Net-(C66-Pad1) -> /HDMI/LCD.D0.B0--B3
- C66 pad 2: Net-(C65-Pad2) -> CGND
- C69 pad 1: CGND -> Net-(C69-Pad1)
- C69 pad 2: /BED_THERM -> Net-(C69-Pad2)
- C7 pad 1: Net-(C7-Pad1) -> VCC
- C70 pad 1: CGND -> Net-(C70-Pad1)
- C70 pad 2: /ADC -> Net-(C69-Pad2)
- C71 pad 1: /X1_ENDSTOP -> CGND
- C71 pad 2: CGND -> /BED_THERM
- C72 pad 1: /Y1_ENDSTOP -> CGND
- C72 pad 2: CGND -> /ADC
- C73 pad 1: /Z1_ENDSTOP -> /X1_ENDSTOP
- C74 pad 1: /ENC_A -> /Y1_ENDSTOP
- C75 pad 1: /ENC_B -> /Z1_ENDSTOP
- C76 pad 1: VCC -> /ENC_A
- C77 pad 1: VCC -> /ENC_B
- C79 pad 1: CGND -> VCC
- C79 pad 2: VCC -> CGND
- C8 pad 1: +24V -> /~SYS_RESET
- C81 pad 1: VCC -> CGND
- C81 pad 2: CGND -> VCC
- C83 pad 1: Net-(C83-Pad1) -> VCC
- C84 pad 1: CGND -> VCC
- C84 pad 2: +24V -> CGND
- C85 pad 1: /Stepper Drivers/E Stepper Driver/5VOUT -> Net-(C85-Pad1)
- C86 pad 1: Net-(C86-Pad1) -> CGND
- C86 pad 2: Net-(C86-Pad2) -> +24V
- C87 pad 1: /Stepper Drivers/E_A2 -> /Stepper Drivers/E Stepper Driver/5VOUT
- C88 pad 1: /Stepper Drivers/E_B2 -> Net-(C88-Pad1)
- C88 pad 2: CGND -> Net-(C88-Pad2)
- C89 pad 1: +24V -> /Stepper Drivers/E_A2
- C89 pad 2: Net-(C89-Pad2) -> CGND
- C9 pad 1: VDD_5V -> Net-(C9-Pad1)
- C90 pad 1: /Stepper Drivers/E_A1 -> /Stepper Drivers/E_B2
- C91 pad 1: /Stepper Drivers/E_B1 -> +24V
- C91 pad 2: CGND -> Net-(C91-Pad2)
- C92 pad 1: +24V -> /Stepper Drivers/E_A1
- C93 pad 1: +24V -> /Stepper Drivers/E_B1
- C94 pad 1: Net-(C94-Pad1) -> +24V
- C96 pad 1: +24V -> Net-(C96-Pad1)
- C97 pad 1: Net-(C97-Pad1) -> +24V
- C98 pad 1: VCC -> +24V
- D1 pad 1: CGND -> Net-(C2-Pad1)
- D1 pad 2: Net-(D1-Pad2) -> CGND
- D10 pad 1: Net-(D10-Pad1) -> VCC
- D10 pad 2: VDD_3V3AUX -> CGND
- D11 pad 2: VDD_1V8 -> VDD_3V3AUX
- D12 pad 2: CGND -> VDD_1V8
- D13 pad 1: VDD_5V -> Net-(D13-Pad1)
- D14 pad 1: Net-(D14-Pad1) -> VDD_5V
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Other:
- board text added: "24V_FANS"
- board text added: "ADC"
- board text added: "BED_HEAT"
- board text added: "BED_T"
- board text added: "DOCK0_HEAT"
- board text added: "DOCK1_HEAT"
- board text added: "E"
- board text added: "END/ENC"
- board text added: "EPM"
- board text added: "E_HEAT"
- board text added: "Ethernet"
- board text added: "H"
- board text added: "H_HEAT"
- board text added: "PWR_IN"
- board text added: "SPI"
- board text added: "USB-Host"
- board text added: "X0"
- board text added: "X1"
- board text added: "Y0"
- board text added: "Y1"
- board text added: "Z0"
- board text added: "Z1"
- board text added: "Z2"
- board text added: "μHDMI"
- board text added: "μSD"
- board text added: "μUSB-OTG"

Commit message: Arrange connectors and E-stepper circuit
Parts:
- removed REF** (x5): MountingHole_3mm_Pad, KiMBo:MountingHole_3mm_Pad
- R144, R152, R160, R166, R172, R179, R187, R193: footprint Resistors_SMD:R_0805 -> Resistors_SMD:R_0603
- R146, R154, R162, R168, R174, R181, R189, R195: footprint Resistors_SMD:R_0603 -> Resistors_SMD:R_0805
- moved C82 403.6 mm to (243.0, -84.0)
- moved C83 398.9 mm to (242.0, -78.0)
- moved C98 300.7 mm to (318.4, 335.5)
- moved C99 289.1 mm to (322.8, 325.8), turned to 90 degrees
- moved R145 59.1 mm to (324.7, 359.7), turned to 90 degrees
- moved C96 57.0 mm to (322.5, 359.7), turned to 270 degrees
- moved C95 51.4 mm to (329.8, 351.1), turned to 270 degrees
- moved R143 48.4 mm to (334.4, 347.2), turned to 180 degrees
- moved C90 47.4 mm to (327.0, 359.9), turned to 270 degrees
- moved R144 44.3 mm to (334.4, 349.1), turned to 180 degrees
- moved C93 42.7 mm to (323.9, 349.3), turned to 180 degrees
- moved C86 39.6 mm to (329.2, 339.3), turned to 270 degrees
- moved R140 39.0 mm to (333.5, 351.0), turned to 180 degrees
- moved C87 38.5 mm to (333.8, 344.7), turned to 270 degrees
- moved C94 36.9 mm to (330.9, 339.3), turned to 90 degrees
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Routing:
- net +24V: track 0.00 -> 10.4 mm
- net Net-(C85-Pad1): track 0.00 -> 7.77 mm
- net CGND: track 0.00 -> 7.41 mm
- net /Stepper Drivers/E Stepper Driver/5VOUT: track 0.00 -> 6.92 mm
- net Net-(C91-Pad2): track 0.00 -> 5.29 mm
- net /E_FAULT: track 0.00 -> 5.14 mm
- net Net-(R143-Pad2): track 0.00 -> 4.91 mm
- net Net-(C88-Pad2): track 0.00 -> 4.74 mm
- net /Stepper Drivers/E_B1: track 0.00 -> 4.60 mm
- net /Stepper Drivers/E_A1: track 0.00 -> 4.45 mm
- net Net-(C88-Pad1): track 0.00 -> 2.81 mm
- net Net-(C99-Pad1): track 0.00 -> 2.32 mm
- net Net-(C96-Pad1): track 0.00 -> 2.32 mm
- net /Stepper Drivers/~E_SS: track 0.00 -> 1.69 mm
- net VCC: track 0.00 -> 1.69 mm
Other:
- board outline added: 187 x 127 mm
- copper layers 2 -> 6

Commit message: More progress on the stepper driver layout
Parts:
- moved R140 288.6 mm to (161.3, 119.4), turned to 270 degrees
- moved R141 274.6 mm to (164.8, 119.6), turned to 270 degrees
- moved C96 264.6 mm to (180.1, 136.7), turned to 180 degrees
- moved R145 264.1 mm to (180.1, 138.7), turned to 0 degrees
- moved C90 263.5 mm to (180.4, 141.0), turned to 180 degrees
- moved C95 255.7 mm to (181.0, 143.1), turned to 180 degrees
- moved C93 254.1 mm to (183.0, 137.8), turned to 90 degrees
- moved R144 252.1 mm to (183.0, 147.5), turned to 90 degrees
- moved C84 251.1 mm to (185.4, 137.0), turned to 90 degrees
- moved R143 249.5 mm to (184.9, 147.5), turned to 90 degrees
- moved U18 247.9 mm to (186.9, 142.1), turned to 270 degrees
- moved C87 246.1 mm to (187.4, 146.9), turned to 180 degrees
- moved R142 245.7 mm to (187.4, 148.9), turned to 0 degrees
- moved C98 244.2 mm to (186.9, 129.7), turned to 180 degrees
- moved C92 242.9 mm to (190.8, 137.8), turned to 90 degrees
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Routing:
- net CGND: track 7.41 -> 37.1 mm
- net /Stepper Drivers/~E_EN: track 0.00 -> 19.9 mm
- net /E_FAULT: track 5.14 -> 17.7 mm
- net +24V: track 10.4 -> 17.4 mm, vias 0 -> 10
- net /Stepper Drivers/E_A2: track 0.04 -> 5.95 mm, vias 0 -> 2
- net /Stepper Drivers/E_B2: track 0.00 -> 5.87 mm, vias 0 -> 2
- net Net-(C99-Pad1): track 2.32 -> 6.88 mm
- net Net-(C96-Pad1): track 2.32 -> 6.85 mm
- net Net-(C85-Pad1): track 7.77 -> 5.77 mm
- net /Stepper Drivers/E_B1: track 4.60 -> 6.16 mm, vias 0 -> 2
- net /Stepper Drivers/E_A1: track 4.45 -> 6.00 mm, vias 0 -> 2
- net /E_STEP: track 0.00 -> 1.40 mm
- net /SPI1_MOSI: track 0.00 -> 1.40 mm
- net /E_DIR: track 0.00 -> 1.40 mm
- net /SPI1_MISO: track 0.00 -> 1.40 mm
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- added copper zone on F.Cu, net +24V
- added copper zone on F.Cu, net /Stepper Drivers/E_A1
- added copper zone on F.Cu, net /Stepper Drivers/E_A2
- added copper zone on F.Cu, net /Stepper Drivers/E_B1
- added copper zone on F.Cu, net /Stepper Drivers/E_B2
- added copper zone on F.Cu, net CGND

Commit message: Tune in the stepper motor circuit, prior to removing HDMI
Parts:
- moved P14 76.7 mm to (241.7, 63.9)
- moved R140 28.2 mm to (187.3, 108.4)
- moved R141 28.2 mm to (190.8, 108.6)
- moved U12 23.6 mm to (234.5, 52.0)
- moved P15 19.5 mm to (241.4, 50.8)
- moved P12 15.1 mm to (239.7, 93.3)
- moved P16 14.9 mm to (231.7, 109.2)
- moved U11 14.7 mm to (215.2, 109.4)
- moved P13 12.3 mm to (229.3, 81.2)
- moved C86 1.77 mm to (193.3, 144.6)
- moved C94 1.77 mm to (193.3, 142.9)
- moved C92 0.40 mm to (190.8, 137.4)
- moved C93 0.40 mm to (183.0, 137.4)
- moved C98 0.40 mm to (186.9, 130.1)
- moved R142 0.20 mm to (187.4, 148.7)
Routing:
- net CGND: track 37.1 -> 101.4 mm
- net /Stepper Drivers/~E_EN: track 19.9 -> 5.28 mm, vias 0 -> 1
- net /E_FAULT: track 17.7 -> 4.86 mm, vias 0 -> 1
- net +24V: track 17.4 -> 26.5 mm
- net /SPI1_MISO: track 1.40 -> 4.99 mm, vias 0 -> 1
- net /E_STEP: track 1.40 -> 4.92 mm, vias 0 -> 1
- net /SPI1_MOSI: track 1.40 -> 4.25 mm, vias 0 -> 1
- net /E_DIR: track 1.40 -> 4.20 mm, vias 0 -> 1
- net /SPI1_SCLK: track 1.35 -> 3.51 mm, vias 0 -> 1
- net /Stepper Drivers/~E_SS: track 1.20 -> 2.68 mm, vias 0 -> 1
- net VCC: track 1.76 -> 3.18 mm, vias 0 -> 1
- net /Stepper Drivers/E_B1: track 6.16 -> 7.17 mm
- net /Stepper Drivers/E_A1: track 6.00 -> 7.02 mm
Other:
- rule trace_min: 0.2 -> 0.1016
- rule via_min_drill: 0.3 -> 0.2
- rule via_min_size: 0.4 -> 0.327
