File: KiMBo/KiMBo.kicad_pcb (KiCad board)
At the start: 6 copper layers, 187 x 127 mm, 643 parts, among them IC1 24LC32AT-I/OT, P1 TOOLHEAD0, P10 ADC, P11 Serial, P12 μUSB, P13 USB_Type_A, P14 HDMI, P15 μSD, P16 Ethernet, P17 JTAG, P18 LCD, P19 E_MOTOR, P2 TOOLHEAD1, P20 H_MOTOR, P21 X0_MOTOR, P22 X1_MOTOR, P23 Y0_MOTOR, P24 Y1_MOTOR, P25 Z0_MOTOR, P26 Z1_MOTOR, P27 Z2_MOTOR, P28 BED_HEAT, P29 E_HEAT, P3 DOCK0, P30 H_HEAT, P31 DOCK0_HEAT, P32 DOCK1_HEAT, P33 E_FAN, P34 H_FAN, P35 CASE_FAN, P36 PWM, P37 PWR_Input, P4 DOCK1, P5 X1, P6 Y1, P7 Z1, P8 ENC, P9 BED_THERM, Q1 2N7002, Q10 DMP3098L-7, Q11 2N7002, Q12 2N7002, Q13 DMP3098L-7, Q14 DMP3098L-7, Q15 2N7002, Q16 DMP3098L-7, Q17 2N7002, Q18 DMP3098L-7, Q19 2N7002, Q2 MMBT2907, Q20 DMP3098L-7, Q3 DNP-MMBT2907, Q4 IPD90P03P4-04, Q5 2N7002, Q6 IPD90P03P4-04, Q7 2N7002, Q8 2N7002, Q9 DMP3098L-7, SW1 RESET, SW2 Power, SW3 μSD_Boot, U1 OSD3358, U10 TPD4S012, U11 LAN8710A, U12 TDA19988BHN/C1,557, U13 IP4283CZ10-TBR, U14 IP4283CZ10-TBR, U15 74HC595, U16 74HC595, U17 74HC595, U18 TMC2130, U19 TMC2130, U2 74LVC1G06, U20 TMC2130, U21 TMC2130, U22 TMC2130, U23 TMC2130, U24 TMC2130, U25 TMC2130, U26 PCA9685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

Commit message: Remove HDMI from the schematic
Parts:
- removed C212: 100nF, Capacitors_SMD:C_0603
- removed C213, C214, C215, C216, C217, C218, C219, C220: 4.7nF, Capacitors_SMD:C_0603
- removed the C59 at (386.2, 106.2)
- removed the C60 at (403.0, 88.3)
- removed the C61 at (390.4, 100.0)
- removed the C62 at (396.1, 94.1)
- removed the C63 at (396.0, 82.4)
- removed the C64 at (374.2, 107.1)
- removed the C65 at (5.54, -309.4)
- removed the C66 at (13.7, -317.1)
- removed the C67 at (18.0, -317.1)
- removed the C68 at (9.75, -311.3)
- removed the C69 at (-14.2, -158.0)
- removed the C70 at (-14.2, -163.8)
- removed the C71 at (74.8, -234.7)
- removed the C72 at (59.0, -226.5)
- removed the C73 at (73.2, -223.0)
- removed the C74 at (68.4, -226.5)
- removed D34: LED, LEDs:LED_0603
- removed F2: 1206L025YR, KiMBo:F_1206
- removed FB44, FB45: CIM21J202NE, Resistors_SMD:R_0805
- removed P37: PWR_Input, KiMBo:euro_header_4_angled
- removed the R115 at (212.3, -235.6)
- removed the R116 at (217.3, -241.4)
- removed the R117 at (7.61, -317.1)
- removed the R118 at (14.1, -311.3)
- removed the R119 at (-9.30, -163.8)
- removed R235, R236, R237, R238, R240, R241, R242, R243, R244: 4.7kΩ, Resistors_SMD:R_0603
- removed R239: 10Ω, Resistors_SMD:R_0603
- removed the U14 at (355.8, 103.2)
- removed U23, U24, U25: TMC2130, KiMBo:QFN36_5X6
- removed U26: PCA9685, Housings_SSOP:TSSOP-28_4.4x9.7mm_Pitch0.65mm
- added C84: 470pF, Capacitors_SMD:C_0603, F.Cu at (529.4, 63.2)
- added C85: 100nF, Capacitors_SMD:C_0603, F.Cu at (544.9, 62.8)
- added C86: 100nF, Capacitors_SMD:C_0603, F.Cu at (550.1, 62.8)
- added C87: 100nF, Capacitors_SMD:C_0603, F.Cu at (534.6, 69.1)
- added C88: 10μF, Capacitors_SMD:C_0805, F.Cu at (524.7, 63.4)
- added C89: 100μF, Capacitors_SMD:c_elec_8x10, F.Cu at (516.9, 60.2)
- added C90: 100nF, Capacitors_SMD:C_0603, F.Cu at (539.8, 62.8)
- added C91: 100nF, Capacitors_SMD:C_0603, F.Cu at (443.2, 128.7)
- added C92: 470nF, Capacitors_SMD:C_0603, F.Cu at (467.4, 122.4)
- added C93: 100nF, Capacitors_SMD:C_0603, F.Cu at (458.0, 122.4)
- added C94: 4.7μF, Capacitors_SMD:C_0603, F.Cu at (458.5, 128.3)
- added C95: 22nF, Capacitors_SMD:C_0603, F.Cu at (462.7, 122.4)
- added C96: 470pF, Capacitors_SMD:C_0603, F.Cu at (453.5, 128.7)
- added C97: 470pF, Capacitors_SMD:C_0603, F.Cu at (463.2, 116.6)
- added C98: 100nF, Capacitors_SMD:C_0603, F.Cu at (448.3, 128.7)
- added C99: 470pF, Capacitors_SMD:C_0603, F.Cu at (458.0, 116.6)
- added R142: 4.7kΩ, Resistors_SMD:R_0603, F.Cu at (442.1, 168.2)
- added R143: 2.2Ω, Resistors_SMD:R_0603, F.Cu at (399.9, 162.1)
- added R144: 5.23kΩ, Resistors_SMD:R_0603, F.Cu at (410.2, 162.1)
- added R145: 4.75kΩ, Resistors_SMD:R_0603, F.Cu at (416.0, 156.3)
- added R146: 220mΩ, Resistors_SMD:R_0805, F.Cu at (379.2, 168.7)
- added U18: TMC2130, KiMBo:QFN36_5X6, F.Cu at (426.7, 169.2)
- C100, C112, C115, C116, C128, C131, C132, C144, C147, C148, C160, C163, C164, C176, C179, C180, C33, C80, C81, C83: value 100nF -> 470pF
- C101, C117, C133, C149, C165, C181: value 470nF -> 100nF
- C103, C119, C135, C151, C167, C183: value 4.7μF -> 100nF
- C104, C120, C136, C152, C168, C184: value 22nF -> 10μF; footprint Capacitors_SMD:C_0603 -> Capacitors_SMD:C_0805
- C105, C121, C137, C153, C169, C185: value 470pF -> 100μF; footprint Capacitors_SMD:C_0603 -> Capacitors_SMD:c_elec_8x10
- C106, C109, C122, C125, C138, C141, C154, C157, C170, C173, C186: value 470pF -> 100nF
- C108, C124, C140, C156, C172: value 470pF -> 470nF
- C110, C126, C142, C158, C174, C78: value 100nF -> 4.7μF
- C111, C127, C143, C159, C175, C7, C79: value 100nF -> 22nF
- C113, C129, C145, C161, C177: value 10μF -> 470pF; footprint Capacitors_SMD:C_0805 -> Capacitors_SMD:C_0603
- C114, C130, C146, C162, C178: value 100μF -> 100nF; footprint Capacitors_SMD:c_elec_8x10 -> Capacitors_SMD:C_0603
- C15, C18, C20: value 100nF -> 2.2μF; footprint Capacitors_SMD:C_0603 -> Capacitors_SMD:C_0805
- C16, C19: value 2.2μF -> 100nF; footprint Capacitors_SMD:C_0805 -> Capacitors_SMD:C_0603
- C188, C189: value 470pF -> 4.7nF
- C190, C191, C192, C195: value 100nF -> 4.7nF
- C193: value 10μF -> 4.7nF; footprint Capacitors_SMD:C_0805 -> Capacitors_SMD:C_0603
- C194: value 100μF -> 4.7nF; footprint Capacitors_SMD:c_elec_8x10 -> Capacitors_SMD:C_0603
- C196, C198, C203, C206, C207, C208, C211: value 100nF -> 47pF
- C197: value 470nF -> 47pF
- C199: value 4.7μF -> 47pF
- C200: value 22nF -> 47pF
- C201, C202, C204, C205: value 470pF -> 47pF
- C209: value 10μF -> 47pF; footprint Capacitors_SMD:C_0805 -> Capacitors_SMD:C_0603
- C21, C47: value 2.2μF -> 4.7μF
- C210: value 100μF -> 47pF; footprint Capacitors_SMD:c_elec_8x10 -> Capacitors_SMD:C_0603
- C22: value 4.7μF -> 100nF; footprint Capacitors_SMD:C_0805 -> Capacitors_SMD:C_0603
- C24: value 100nF -> 220μF; footprint Capacitors_SMD:C_0603 -> Capacitors_Tantalum_SMD:TantalC_SizeD_EIA-7343_Reflow
- C25: value 220μF -> 100nF; footprint Capacitors_Tantalum_SMD:TantalC_SizeD_EIA-7343_Reflow -> Capacitors_SMD:C_0603
- C28: value 100nF -> 30pF
- C30: value 30pF -> 100nF
- C34: value 470pF -> 10μF; footprint Capacitors_SMD:C_0603 -> Capacitors_SMD:C_0805
- C35: value 10μF -> 1μF; footprint Capacitors_SMD:C_0805 -> Capacitors_SMD:C_0603
- C36: value 1μF -> DNP-15pF
- C40: value DNP-15pF -> 10μF
- C42: value 10μF -> 18pF
- C43, C45: value 100nF -> 18pF
- C44: value 2.2μF -> 18pF; footprint Capacitors_SMD:C_0805 -> Capacitors_SMD:C_0603
- C46: value 47pF -> 4.7μF
- C48, C49, C51, C52: value 47pF -> 0.1μF
- C50: value 100nF -> 0.1μF
- C53: value 2.2μF -> 100nF
- C54, C55, C57, C58: value 47pF -> 100nF
- C6: value 22nF -> 100nF
- C75, C77: value 0.1μF -> 100nF
- C76: value 0.1μF -> 470nF
- D17: value RB751V40,115 -> TPD1E04U04DPYR; footprint Diodes_SMD:SOD-323 -> KiMBo:TPD_PX1SON
- D18: value TPD1E04U04DPYR -> SK1545-TP; footprint KiMBo:TPD_PX1SON -> KiMBo:SK-DO-214AB
- D19: value SK1545-TP -> LED; footprint KiMBo:SK-DO-214AB -> LEDs:LED_0603
- D20, D24, D28, D30, D32: value LED -> MBRA340T3; footprint LEDs:LED_0603 -> KiMBo:MBR-DO-214AC
- D22, D26, D29, D31, D33: value MBRA340T3 -> LED; footprint KiMBo:MBR-DO-214AC -> LEDs:LED_0603
- FB26: value BLM15AG102SN1D -> LI0805H151R-10; footprint Resistors_SMD:R_0402 -> Resistors_SMD:R_0805
- FB28: value LI0805H151R-10 -> MMZ1608A252BTA00; footprint Resistors_SMD:R_0805 -> KiMBo:Ferrite_Bead_0603
- FB29: value BLM18BD252SN1D -> MMZ1608A252BTA00; footprint Resistors_SMD:R_0603 -> KiMBo:Ferrite_Bead_0603
- FB35, FB36: value MMZ1608A252BTA00 -> BLM31SN500SN1L; footprint KiMBo:Ferrite_Bead_0603 -> Resistors_SMD:R_1206_HandSoldering
- FB37, FB38: value BLM31SN500SN1L -> FBMH4532HM132-T; footprint Resistors_SMD:R_1206_HandSoldering -> KiMBo:Ferrite_Bead_1812
- FB41, FB42: value FBMH4532HM132-T -> CIM21J202NE; footprint KiMBo:Ferrite_Bead_1812 -> Resistors_SMD:R_0805
- P14: value HDMI -> JTAG; footprint KiMBo:MICRO-HDMI-D -> KiMBo:JTAG
- P17: value JTAG -> LCD; footprint KiMBo:JTAG -> Pin_Headers:Pin_Header_Angled_1x07
- P18: value LCD -> E_MOTOR; footprint Pin_Headers:Pin_Header_Angled_1x07 -> Pin_Headers:Pin_Header_Angled_1x04
- P19: value E_MOTOR -> H_MOTOR
- P20: value H_MOTOR -> X0_MOTOR
- P21: value X0_MOTOR -> X1_MOTOR
- P22: value X1_MOTOR -> Y0_MOTOR
- P23: value Y0_MOTOR -> Y1_MOTOR
- P24: value Y1_MOTOR -> Z0_MOTOR
- P25: value Z0_MOTOR -> Z1_MOTOR
- P26: value Z1_MOTOR -> Z2_MOTOR
- P27: value Z2_MOTOR -> BED_HEAT; footprint Pin_Headers:Pin_Header_Angled_1x04 -> KiMBo:euro_header_2_angled
- P28: value BED_HEAT -> E_HEAT
- P29: value E_HEAT -> H_HEAT
- P30: value H_HEAT -> DOCK0_HEAT
- P31: value DOCK0_HEAT -> DOCK1_HEAT
- P32: value DOCK1_HEAT -> E_FAN; footprint KiMBo:euro_header_2_angled -> Pin_Headers:Pin_Header_Angled_1x02
- P33: value E_FAN -> H_FAN
- P34: value H_FAN -> CASE_FAN
- P35: value CASE_FAN -> PWM; footprint Pin_Headers:Pin_Header_Angled_1x02 -> Pin_Headers:Pin_Header_Angled_1x03
- P36: value PWM -> PWR_Input; footprint Pin_Headers:Pin_Header_Angled_1x03 -> KiMBo:euro_header_4_angled
- R100: value 100kΩ -> 100Ω
- R101, R102, R103, R104, R105, R106, R107, R108, R109, R110, R111, R112, R113, R114: value 100kΩ -> 4.7kΩ
- R120, R122, R94, R99: value 10kΩ -> 4.7kΩ
- R123: value 100Ω -> 2.2Ω
- R124, R132, R138: value 4.7kΩ -> 5.23kΩ
- R125: value 100Ω -> 4.75kΩ
- R126, R134, R135, R140, R141, R147: value 4.7kΩ -> 220mΩ; footprint Resistors_SMD:R_0603 -> Resistors_SMD:R_0805
- R127: value 100Ω -> 220mΩ; footprint Resistors_SMD:R_0603 -> Resistors_SMD:R_0805
- R131, R137: value 4.7kΩ -> 2.2Ω
- R133, R139: value 4.7kΩ -> 4.75kΩ
- R170, R177: value 2.2Ω -> 10Ω
- R171, R178, R186, R192: value 5.23kΩ -> 4.7kΩ
- R172, R179, R187, R193: value 4.75kΩ -> 4.7kΩ
- R173, R174, R180, R181, R194, R195: value 220mΩ -> 4.7kΩ; footprint Resistors_SMD:R_0805 -> Resistors_SMD:R_0603
- R176, R200, R206, R212: value 4.7kΩ -> 10Ω
- R185, R191: value 2.2Ω -> 4.7kΩ
- R188, R189: value 220mΩ -> 10Ω; footprint Resistors_SMD:R_0805 -> Resistors_SMD:R_0603
- R197, R203, R204, R215, R216: value 10Ω -> 4.7kΩ
- R218, R220, R221, R222, R223, R224, R225, R226, R228, R229, R230, R231, R232, R234: value 4.7kΩ -> 100kΩ
- R219: value 4.7kΩ -> 100Ω
- R227, R233: value 10Ω -> 100kΩ
- R5: value 470Ω -> 4.75kΩ
- R6: value 4.75kΩ -> 470Ω
- R90: value 22Ω -> DNP-1MΩ
- R91: value 0Ω -> 1MΩ
- R92: value 0Ω -> 4.7kΩ
- R93: value 0Ω -> 10kΩ
- R95: value 27kΩ -> 10kΩ
- R96: value 0Ω -> 100Ω
- R97: value 1.5kΩ -> 4.7kΩ
- R98: value 1.5kΩ -> 100Ω
- U10: value TPD4S012 -> LAN8710A; footprint KiMBo:DRY-DFN-6-1EP_2x2mm_Pitch0.5mm -> Housings_DFN_QFN:QFN-32-1EP_5x5mm_Pitch0.5mm
- U11: value LAN8710A -> 74HC595; footprint Housings_DFN_QFN:QFN-32-1EP_5x5mm_Pitch0.5mm -> Housings_SSOP:TSSOP-16_4.4x5mm_Pitch0.65mm
- U12: value TDA19988BHN/C1,557 -> 74HC595; footprint KiMBo:SOT804-4 -> Housings_SSOP:TSSOP-16_4.4x5mm_Pitch0.65mm
- U13: value IP4283CZ10-TBR -> 74HC595; footprint KiMBo:XFDFN-10-1EP_2x3mm_Pitch0.5mm -> Housings_SSOP:TSSOP-16_4.4x5mm_Pitch0.65mm
- U15, U16, U17: value 74HC595 -> TMC2130; footprint Housings_SSOP:TSSOP-16_4.4x5mm_Pitch0.65mm -> KiMBo:QFN36_5X6
- U22: value TMC2130 -> PCA9685; footprint KiMBo:QFN36_5X6 -> Housings_SSOP:TSSOP-28_4.4x9.7mm_Pitch0.65mm
- U4: value SN74AUC1G74DCTR -> 74LVC1G06; footprint KiMBo:DCT-MSOP-8_3x3mm_Pitch0.65mm -> TO_SOT_Packages_SMD:SC-70-5
- U5: value 74LVC1G06 -> EMMC**G-S100; footprint TO_SOT_Packages_SMD:SC-70-5 -> KiMBo:EMMCxxG-S100
- U6: value EMMC**G-S100 -> TPS2051B; footprint KiMBo:EMMCxxG-S100 -> KiMBo:DGN-MSOP-8_3x3mm_Pitch0.65mm
- U7: value TPS2051B -> TPD4S012; footprint KiMBo:DGN-MSOP-8_3x3mm_Pitch0.65mm -> KiMBo:DRY-DFN-6-1EP_2x2mm_Pitch0.5mm
- U8: value TPD4S012 -> 74LVC2G241; footprint KiMBo:DRY-DFN-6-1EP_2x2mm_Pitch0.5mm -> KiMBo:DCT-MSOP-8_3x3mm_Pitch0.65mm
- U9: value 74LVC2G241 -> TPD4S012; footprint KiMBo:DCT-MSOP-8_3x3mm_Pitch0.65mm -> KiMBo:DRY-DFN-6-1EP_2x2mm_Pitch0.5mm
- Y2: value TXC CORPORATION -> AH-32.768KDZY-T
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- renumbered C84 to C59, C85 to C60, C86 to C61, C87 to C62, C88 to C63, C89 to C64, C90 to C65, C91 to C66, C92 to C67, C93 to C68, C94 to C69, C95 to C70, C96 to C71, C97 to C72, C98 to C73, C99 to C74, R142 to R115, R143 to R116, R144 to R117, R145 to R118, R146 to R119, U18 to U14
Connections:
- C100 pad 1: VCC -> /Stepper Drivers/Z0_B1
- C101 pad 1: Net-(C101-Pad1) -> +24V
- C102 pad 1: CGND -> +24V
- C102 pad 2: +24V -> CGND
- C103 pad 1: /Stepper Drivers/X0 Stepper Driver/5VOUT -> Net-(C103-Pad1)
- C104 pad 1: Net-(C104-Pad1) -> +24V
- C104 pad 2: Net-(C104-Pad2) -> CGND
- C105 pad 1: /Stepper Drivers/X0_A2 -> +24V
- C106 pad 1: /Stepper Drivers/X0_B2 -> Net-(C106-Pad1)
- C107 pad 1: +24V -> VCC
- C107 pad 2: Net-(C107-Pad2) -> CGND
- C108 pad 1: /Stepper Drivers/X0_A1 -> Net-(C108-Pad1)
- C109 pad 1: /Stepper Drivers/X0_B1 -> CGND
- C109 pad 2: CGND -> +24V
- C110 pad 1: +24V -> /Stepper Drivers/Z1 Stepper Driver/5VOUT
- C111 pad 1: +24V -> Net-(C111-Pad1)
- C111 pad 2: CGND -> Net-(C111-Pad2)
- C112 pad 1: Net-(C112-Pad1) -> /Stepper Drivers/Z1_A2
- C113 pad 1: +24V -> /Stepper Drivers/Z1_B2
- C114 pad 2: CGND -> Net-(C114-Pad2)
- C115 pad 1: Net-(C115-Pad1) -> /Stepper Drivers/Z1_A1
- C116 pad 1: VCC -> /Stepper Drivers/Z1_B1
- C117 pad 1: Net-(C117-Pad1) -> +24V
- C118 pad 1: CGND -> +24V
- C118 pad 2: +24V -> CGND
- C119 pad 1: /Stepper Drivers/Z0 Stepper Driver/5VOUT -> Net-(C119-Pad1)
- C120 pad 1: Net-(C120-Pad1) -> +24V
- C120 pad 2: Net-(C120-Pad2) -> CGND
- C121 pad 1: /Stepper Drivers/Z0_A2 -> +24V
- C122 pad 1: /Stepper Drivers/Z0_B2 -> Net-(C122-Pad1)
- C123 pad 1: +24V -> VCC
- C123 pad 2: Net-(C123-Pad2) -> CGND
- C124 pad 1: /Stepper Drivers/Z0_A1 -> Net-(C124-Pad1)
- C125 pad 1: /Stepper Drivers/Z0_B1 -> CGND
- C125 pad 2: CGND -> +24V
- C126 pad 1: +24V -> /Stepper Drivers/Z2 Stepper Driver/5VOUT
- C127 pad 1: +24V -> Net-(C127-Pad1)
- C127 pad 2: CGND -> Net-(C127-Pad2)
- C128 pad 1: Net-(C128-Pad1) -> /Stepper Drivers/Z2_A2
- C129 pad 1: +24V -> /Stepper Drivers/Z2_B2
- C130 pad 2: CGND -> Net-(C130-Pad2)
- C131 pad 1: Net-(C131-Pad1) -> /Stepper Drivers/Z2_A1
- C132 pad 1: VCC -> /Stepper Drivers/Z2_B1
- C133 pad 1: Net-(C133-Pad1) -> +24V
- C134 pad 1: CGND -> +24V
- C134 pad 2: +24V -> CGND
- C135 pad 1: /Stepper Drivers/Z1 Stepper Driver/5VOUT -> Net-(C135-Pad1)
- C136 pad 1: Net-(C136-Pad1) -> +24V
- C136 pad 2: Net-(C136-Pad2) -> CGND
- C137 pad 1: /Stepper Drivers/Z1_A2 -> +24V
- C138 pad 1: /Stepper Drivers/Z1_B2 -> Net-(C138-Pad1)
- C139 pad 1: +24V -> VCC
- C139 pad 2: Net-(C139-Pad2) -> CGND
- C140 pad 1: /Stepper Drivers/Z1_A1 -> Net-(C140-Pad1)
- C141 pad 1: /Stepper Drivers/Z1_B1 -> CGND
- C141 pad 2: CGND -> +24V
- C142 pad 1: +24V -> /Stepper Drivers/H Stepper Driver/5VOUT
- C143 pad 1: +24V -> Net-(C143-Pad1)
- C143 pad 2: CGND -> Net-(C143-Pad2)
- C144 pad 1: Net-(C144-Pad1) -> /Stepper Drivers/H_A2
- C145 pad 1: +24V -> /Stepper Drivers/H_B2
- C146 pad 2: CGND -> Net-(C146-Pad2)
- C147 pad 1: Net-(C147-Pad1) -> /Stepper Drivers/H_A1
- C148 pad 1: VCC -> /Stepper Drivers/H_B1
- C149 pad 1: Net-(C149-Pad1) -> +24V
- C15 pad 1: VCC -> CGND
- C150 pad 1: CGND -> +24V
- C150 pad 2: +24V -> CGND
- C151 pad 1: /Stepper Drivers/Z2 Stepper Driver/5VOUT -> Net-(C151-Pad1)
- C152 pad 1: Net-(C152-Pad1) -> +24V
- C152 pad 2: Net-(C152-Pad2) -> CGND
- C153 pad 1: /Stepper Drivers/Z2_A2 -> +24V
- C154 pad 1: /Stepper Drivers/Z2_B2 -> Net-(C154-Pad1)
- C155 pad 1: +24V -> VCC
- C155 pad 2: Net-(C155-Pad2) -> CGND
- C156 pad 1: /Stepper Drivers/Z2_A1 -> Net-(C156-Pad1)
- C157 pad 1: /Stepper Drivers/Z2_B1 -> CGND
- C157 pad 2: CGND -> +24V
- C158 pad 1: +24V -> /Stepper Drivers/Y Stepper Driver/5VOUT
- C159 pad 1: +24V -> Net-(C159-Pad1)
- C159 pad 2: CGND -> Net-(C159-Pad2)
- C16 pad 1: CGND -> VCC
- C160 pad 1: Net-(C160-Pad1) -> /Stepper Drivers/Y_A2
- C161 pad 1: +24V -> /Stepper Drivers/Y_B2
- C162 pad 2: CGND -> Net-(C162-Pad2)
- C163 pad 1: Net-(C163-Pad1) -> /Stepper Drivers/Y_A1
- C164 pad 1: VCC -> /Stepper Drivers/Y_B1
- C165 pad 1: Net-(C165-Pad1) -> +24V
- C166 pad 1: CGND -> +24V
- C166 pad 2: +24V -> CGND
- C167 pad 1: /Stepper Drivers/H Stepper Driver/5VOUT -> Net-(C167-Pad1)
- C168 pad 1: Net-(C168-Pad1) -> +24V
- C168 pad 2: Net-(C168-Pad2) -> CGND
- C169 pad 1: /Stepper Drivers/H_A2 -> +24V
- C17 pad 1: VCC -> CGND
- C170 pad 1: /Stepper Drivers/H_B2 -> Net-(C170-Pad1)
- C171 pad 1: +24V -> VCC
- C171 pad 2: Net-(C171-Pad2) -> CGND
- C172 pad 1: /Stepper Drivers/H_A1 -> Net-(C172-Pad1)
- C173 pad 1: /Stepper Drivers/H_B1 -> CGND
- C173 pad 2: CGND -> +24V
- C174 pad 1: +24V -> /Stepper Drivers/X1 Stepper Driver/5VOUT
- C175 pad 1: +24V -> Net-(C175-Pad1)
- C175 pad 2: CGND -> Net-(C175-Pad2)
- C176 pad 1: Net-(C176-Pad1) -> /Stepper Drivers/X1_A2
- C177 pad 1: +24V -> /Stepper Drivers/X1_B2
- C178 pad 2: CGND -> Net-(C178-Pad2)
- C179 pad 1: Net-(C179-Pad1) -> /Stepper Drivers/X1_A1
- C180 pad 1: VCC -> /Stepper Drivers/X1_B1
- C181 pad 1: Net-(C181-Pad1) -> +24V
- C182 pad 1: CGND -> +24V
- C182 pad 2: +24V -> CGND
- C183 pad 1: /Stepper Drivers/Y Stepper Driver/5VOUT -> Net-(C183-Pad1)
- C184 pad 1: Net-(C184-Pad1) -> +24V
- C184 pad 2: Net-(C184-Pad2) -> CGND
- C185 pad 1: /Stepper Drivers/Y_A2 -> +24V
- C186 pad 1: /Stepper Drivers/Y_B2 -> Net-(C186-Pad1)
- C187 pad 1: +24V -> VCC
- C187 pad 2: Net-(C187-Pad2) -> CGND
- C188 pad 1: /Stepper Drivers/Y_A1 -> +24V
- C188 pad 2: CGND -> /Heaters/BED_HEAT
- C189 pad 1: /Stepper Drivers/Y_B1 -> +24V
- C189 pad 2: CGND -> /Heaters/E_HEAT
- C190 pad 2: CGND -> /Heaters/DOCK0_HEAT
- C191 pad 2: CGND -> /Heaters/H_HEAT
- C192 pad 1: Net-(C192-Pad1) -> +24V
- C192 pad 2: CGND -> /Heaters/DOCK1_HEAT
- C193 pad 2: CGND -> /Fans/E_FAN
- C194 pad 2: CGND -> /Fans/H_FAN
- C195 pad 1: Net-(C195-Pad1) -> +24V
- C195 pad 2: CGND -> /Fans/CASE_FAN
- C196 pad 1: VCC -> /Configuration/LCD.D15.R4--R7
- C197 pad 1: Net-(C197-Pad1) -> /Configuration/LCD.D14.R3--R6
- C198 pad 1: CGND -> /Configuration/LCD.D13.R2--R5
- C198 pad 2: +24V -> CGND
- C199 pad 1: /Stepper Drivers/X1 Stepper Driver/5VOUT -> /Configuration/LCD.D12.R1--R4
- C200 pad 1: Net-(C200-Pad1) -> /Configuration/LCD.D11.R0--R3
- C200 pad 2: Net-(C200-Pad2) -> CGND
- C201 pad 1: /Stepper Drivers/X1_A2 -> /Configuration/LCD.D10.G5--G7
- C202 pad 1: /Stepper Drivers/X1_B2 -> /Configuration/LCD.D9.G4--G6
- C203 pad 1: +24V -> /Configuration/LCD.D8.G3--G5
- C203 pad 2: Net-(C203-Pad2) -> CGND
- C204 pad 1: /Stepper Drivers/X1_A1 -> /Configuration/LCD.D7.G2--G4
- C205 pad 1: /Stepper Drivers/X1_B1 -> /Configuration/LCD.D6.G1--G3
- C206 pad 1: +24V -> /Configuration/LCD.D5.G0--G2
- C207 pad 1: +24V -> /Configuration/LCD.D4.B4--B7
- C208 pad 1: Net-(C208-Pad1) -> /Configuration/LCD.D3.B3--B6
- C209 pad 1: +24V -> /Configuration/LCD.D2.B2--B5
- C21 pad 1: CGND -> Net-(C21-Pad1)
- C210 pad 1: +24V -> /Configuration/LCD.D1.B1--B4
- C211 pad 1: Net-(C211-Pad1) -> /Configuration/LCD.D0.B0--B3
- C22 pad 1: Net-(C22-Pad1) -> Net-(C21-Pad1)
- C23 pad 1: Net-(C22-Pad1) -> VCC
- C24 pad 1: VCC -> SYS_5V
- C25 pad 1: SYS_5V -> Net-(C25-Pad1)
- C26 pad 1: Net-(C26-Pad1) -> USB_DC
- C27 pad 1: USB_DC -> VCC
- C28 pad 1: VCC -> Net-(C28-Pad1)
- C30 pad 1: Net-(C30-Pad1) -> VCC
- C31 pad 1: VCC -> VDD_PHYA
- C33 pad 1: VDD_PHYA -> /Ethernet/PHY_VDDCR
- C34 pad 1: /Ethernet/PHY_VDDCR -> VDD_PHYA
- C35 pad 1: VDD_PHYA -> /Ethernet/PHY_VDDCR
- C36 pad 1: /Ethernet/PHY_VDDCR -> /Ethernet/RD+
- C37 pad 1: /Ethernet/RD+ -> /Ethernet/RD-
- C38 pad 1: /Ethernet/RD- -> /Ethernet/TD+
- C39 pad 1: /Ethernet/TD+ -> /Ethernet/TD-
- C40 pad 1: /Ethernet/TD- -> VCC
- C42 pad 1: VCC -> Net-(C42-Pad1)
- C42 pad 2: CGND -> Net-(C42-Pad2)
- C43 pad 1: HDMI_1V8 -> Net-(C43-Pad1)
- C43 pad 2: Net-(C43-Pad2) -> Net-(C42-Pad2)
- C44 pad 1: HDMI_1V8 -> Net-(C44-Pad1)
- C44 pad 2: Net-(C43-Pad2) -> Net-(C44-Pad2)
- C45 pad 1: HDMI_1V8 -> Net-(C45-Pad1)
- C45 pad 2: Net-(C43-Pad2) -> Net-(C44-Pad2)
- C46 pad 1: /HDMI/LCD.D15.R4--R7 -> CGND
- C46 pad 2: CGND -> /BED_THERM
- C47 pad 1: HDMI_1V8 -> CGND
- C47 pad 2: Net-(C43-Pad2) -> /ADC
- C48 pad 1: /HDMI/LCD.D14.R3--R6 -> /X1_ENDSTOP
- C49 pad 1: /HDMI/LCD.D13.R2--R5 -> /Y1_ENDSTOP
- C50 pad 1: HDMI_1V8 -> /Z1_ENDSTOP
- C50 pad 2: Net-(C43-Pad2) -> CGND
- C51 pad 1: /HDMI/LCD.D12.R1--R4 -> /ENC_A
- C52 pad 1: /HDMI/LCD.D11.R0--R3 -> /ENC_B
- C53 pad 1: HDMI_1V8 -> VCC
- C53 pad 2: Net-(C43-Pad2) -> CGND
- C54 pad 1: /HDMI/LCD.D10.G5--G7 -> VCC
- C55 pad 1: /HDMI/LCD.D9.G4--G6 -> VCC
- C56 pad 1: HDMI_1V8 -> CGND
- C56 pad 2: Net-(C43-Pad2) -> VCC
- C57 pad 1: /HDMI/LCD.D8.G3--G5 -> VCC
- C58 pad 1: /HDMI/LCD.D7.G2--G4 -> VCC
- C6 pad 1: Net-(C6-Pad1) -> VCC
- C7 pad 1: VCC -> Net-(C7-Pad1)
- C75 pad 1: /Z1_ENDSTOP -> VCC
- C76 pad 1: /ENC_A -> Net-(C76-Pad1)
- C77 pad 1: /ENC_B -> CGND
- C77 pad 2: CGND -> +24V
- C78 pad 1: VCC -> /Stepper Drivers/X0 Stepper Driver/5VOUT
- C79 pad 1: VCC -> Net-(C79-Pad1)
- C79 pad 2: CGND -> Net-(C79-Pad2)
- C80 pad 1: VCC -> /Stepper Drivers/X0_A2
- C81 pad 1: CGND -> /Stepper Drivers/X0_B2
- C81 pad 2: VCC -> CGND
- C82 pad 1: VCC -> +24V
- C82 pad 2: CGND -> Net-(C82-Pad2)
- C83 pad 1: VCC -> /Stepper Drivers/X0_A1
- D17 pad 1: /HDMI/CEC -> /Endstops/Z1_IN
- D17 pad 2: Net-(D17-Pad2) -> CGND
- D18 pad 1: /Endstops/Z1_IN -> Net-(D18-Pad1)
- D19 pad 1: Net-(D19-Pad1) -> CGND
- D19 pad 2: CGND -> Net-(D19-Pad2)
- D20 pad 1: CGND -> Net-(D20-Pad1)
- D20 pad 2: Net-(D20-Pad2) -> CGND
- D22 pad 1: Net-(D22-Pad1) -> CGND
- D22 pad 2: CGND -> Net-(D22-Pad2)
- D24 pad 1: CGND -> Net-(D24-Pad1)
- D24 pad 2: Net-(D24-Pad2) -> CGND
- D26 pad 1: Net-(D26-Pad1) -> CGND
- D26 pad 2: CGND -> Net-(D26-Pad2)
- D28 pad 1: CGND -> Net-(D28-Pad1)
- D28 pad 2: Net-(D28-Pad2) -> CGND
- D29 pad 1: Net-(D29-Pad1) -> CGND
- D29 pad 2: CGND -> Net-(D29-Pad2)
- D30 pad 1: CGND -> Net-(D30-Pad1)
- D30 pad 2: Net-(D30-Pad2) -> CGND
- D31 pad 1: Net-(D31-Pad1) -> CGND
- D31 pad 2: CGND -> Net-(D31-Pad2)
- D32 pad 1: CGND -> Net-(D32-Pad1)
- D32 pad 2: Net-(D32-Pad2) -> CGND
- D33 pad 1: Net-(D33-Pad1) -> CGND
- D33 pad 2: CGND -> Net-(D33-Pad2)
- FB24 pad 1: /12MHz -> Net-(FB24-Pad1)
- FB24 pad 2: Net-(FB24-Pad2) -> /XDMA_EVENT_INTRO
- FB25 pad 1: Net-(FB25-Pad1) -> /CLKOUT2
- FB25 pad 2: /XDMA_EVENT_INTRO -> Net-(FB25-Pad2)
- FB26 pad 1: /CLKOUT2 -> Net-(C25-Pad1)
- FB26 pad 2: Net-(FB26-Pad2) -> /USB/USB.B.VBUS
- FB27 pad 1: Net-(C26-Pad1) -> VCC
- FB27 pad 2: /USB/USB.B.VBUS -> VDD_PHYA
- FB28 pad 1: VCC -> /Thermistors/BED_THERM_IN
- FB28 pad 2: VDD_PHYA -> Net-(FB28-Pad2)
- FB29 pad 1: VDD_1V8 -> /Thermistors/ADC_IN
- FB29 pad 2: HDMI_1V8 -> Net-(FB29-Pad2)
- FB30 pad 1: /Thermistors/BED_THERM_IN -> /Endstops/X1_IN
- FB31 pad 1: /Thermistors/ADC_IN -> /Endstops/Y1_IN
- FB32 pad 1: /Endstops/X1_IN -> /Endstops/Z1_IN
- FB33 pad 1: /Endstops/Y1_IN -> /Endstops/ENC_A_IN
- FB34 pad 1: /Endstops/Z1_IN -> /Endstops/ENC_B_IN
- FB35 pad 1: /Endstops/ENC_A_IN -> Net-(D18-Pad1)
- FB35 pad 2: Net-(FB35-Pad2) -> /Heaters/BED_HEAT
- FB36 pad 1: /Endstops/ENC_B_IN -> Net-(D18-Pad1)
- FB36 pad 2: Net-(FB36-Pad2) -> /Heaters/BED_HEAT
- FB37 pad 1: Net-(D19-Pad1) -> Net-(D20-Pad1)
- FB37 pad 2: /Heaters/BED_HEAT -> /Heaters/E_HEAT
- FB38 pad 1: Net-(D19-Pad1) -> Net-(D21-Pad1)
- FB38 pad 2: /Heaters/BED_HEAT -> /Heaters/DOCK0_HEAT
- FB39 pad 1: Net-(D21-Pad1) -> Net-(D24-Pad1)
- FB39 pad 2: /Heaters/E_HEAT -> /Heaters/H_HEAT
- FB40 pad 1: Net-(D22-Pad1) -> Net-(D25-Pad1)
- FB40 pad 2: /Heaters/DOCK0_HEAT -> /Heaters/DOCK1_HEAT
- FB41 pad 1: Net-(D25-Pad1) -> Net-(D28-Pad1)
- FB41 pad 2: /Heaters/H_HEAT -> /Fans/E_FAN
- FB42 pad 1: Net-(D26-Pad1) -> Net-(D30-Pad1)
- FB42 pad 2: /Heaters/DOCK1_HEAT -> /Fans/H_FAN
- FB43 pad 1: Net-(D29-Pad1) -> Net-(D32-Pad1)
- FB43 pad 2: /Fans/E_FAN -> /Fans/CASE_FAN
- P14 pad 1: /HDMI/HPD -> /JTAG/JTAG_TMS
- P14 pad 11: /HDMI/TX0- -> /TCK
- P14 pad 12: /HDMI/TXC+ -> CGND
- P14 pad 13: CGND -> /JTAG/JTAG_EMU0
- P14 pad 14: /HDMI/TXC- -> /JTAG/JTAG_EMU1
- P14 pad 15: /HDMI/CEC -> /~SYS_RESET
- P14 pad 17: /HDMI/DSCL -> /XDMA_EVENT_INTRO
- P14 pad 18: /HDMI/DSDA -> /CLKOUT2
- P14 pad 19: /HDMI/DVI_5V -> /SD.CD
- P14 pad 2: Net-(P14-Pad2) -> /JTAG/~JTAG_TRST
- P14 pad 3: /HDMI/TX2+ -> /JTAG/JTAG_TDI
- P14 pad 5: /HDMI/TX2- -> VCC
- P14 pad 6: /HDMI/TX1+ -> Net-(P14-Pad6)
- P14 pad 7: CGND -> /JTAG/JTAG_TD0
- P14 pad 8: /HDMI/TX1- -> CGND
- P14 pad 9: /HDMI/TX0+ -> /TCK
- P16 pad 4: Net-(C6-Pad1) -> Net-(C7-Pad1)
- P16 pad 5: Net-(C6-Pad1) -> Net-(C7-Pad1)
- P17 pad 1: /JTAG/JTAG_TMS -> /3V3_FILTERED
- P17 pad 2: /JTAG/~JTAG_TRST -> Net-(FB14-Pad2)
- P17 pad 3: /JTAG/JTAG_TDI -> Net-(FB15-Pad2)
- P17 pad 4: CGND -> Net-(FB16-Pad2)
- P17 pad 5: VCC -> Net-(FB17-Pad2)
- P17 pad 6: Net-(P17-Pad6) -> Net-(FB18-Pad2)
- P17 pad 7: /JTAG/JTAG_TD0 -> CGND
- P18 pad 1: /3V3_FILTERED -> /Stepper Drivers/E_A1
- P18 pad 2: Net-(FB14-Pad2) -> /Stepper Drivers/E_A2
- P18 pad 3: Net-(FB15-Pad2) -> /Stepper Drivers/E_B1
- P18 pad 4: Net-(FB16-Pad2) -> /Stepper Drivers/E_B2
- P19 pad 1: /Stepper Drivers/E_A1 -> /Stepper Drivers/H_A1
- P19 pad 2: /Stepper Drivers/E_A2 -> /Stepper Drivers/H_A2
- P19 pad 3: /Stepper Drivers/E_B1 -> /Stepper Drivers/H_B1
- P19 pad 4: /Stepper Drivers/E_B2 -> /Stepper Drivers/H_B2
- P20 pad 1: /Stepper Drivers/H_A1 -> /Stepper Drivers/X0_A1
- P20 pad 2: /Stepper Drivers/H_A2 -> /Stepper Drivers/X0_A2
- P20 pad 3: /Stepper Drivers/H_B1 -> /Stepper Drivers/X0_B1
- P20 pad 4: /Stepper Drivers/H_B2 -> /Stepper Drivers/X0_B2
- P21 pad 1: /Stepper Drivers/X0_A1 -> /Stepper Drivers/X1_B2
- P21 pad 2: /Stepper Drivers/X0_A2 -> /Stepper Drivers/X1_B1
- P21 pad 3: /Stepper Drivers/X0_B1 -> /Stepper Drivers/X1_A2
- P21 pad 4: /Stepper Drivers/X0_B2 -> /Stepper Drivers/X1_A1
- P22 pad 1: /Stepper Drivers/X1_B2 -> /Stepper Drivers/Y_A1
- P22 pad 2: /Stepper Drivers/X1_B1 -> Net-(P22-Pad2)
- P22 pad 3: /Stepper Drivers/X1_A2 -> /Stepper Drivers/Y_B1
- P22 pad 4: /Stepper Drivers/X1_A1 -> Net-(P22-Pad4)
- P23 pad 1: /Stepper Drivers/Y_A1 -> Net-(P22-Pad4)
- P23 pad 2: Net-(P23-Pad2) -> /Stepper Drivers/Y_B2
- P23 pad 3: /Stepper Drivers/Y_B1 -> Net-(P22-Pad2)
- P23 pad 4: Net-(P23-Pad4) -> /Stepper Drivers/Y_A2
- P24 pad 1: Net-(P23-Pad4) -> /Stepper Drivers/Z0_A1
- P24 pad 2: /Stepper Drivers/Y_B2 -> /Stepper Drivers/Z0_A2
- P24 pad 3: Net-(P23-Pad2) -> /Stepper Drivers/Z0_B1
- P24 pad 4: /Stepper Drivers/Y_A2 -> /Stepper Drivers/Z0_B2
- P25 pad 1: /Stepper Drivers/Z0_A1 -> /Stepper Drivers/Z1_A1
- P25 pad 2: /Stepper Drivers/Z0_A2 -> /Stepper Drivers/Z1_A2
- P25 pad 3: /Stepper Drivers/Z0_B1 -> /Stepper Drivers/Z1_B1
- P25 pad 4: /Stepper Drivers/Z0_B2 -> /Stepper Drivers/Z1_B2
- P26 pad 1: /Stepper Drivers/Z1_A1 -> /Stepper Drivers/Z2_A1
- P26 pad 2: /Stepper Drivers/Z1_A2 -> /Stepper Drivers/Z2_A2
- P26 pad 3: /Stepper Drivers/Z1_B1 -> /Stepper Drivers/Z2_B1
- P26 pad 4: /Stepper Drivers/Z1_B2 -> /Stepper Drivers/Z2_B2
- P27 pad 1: /Stepper Drivers/Z2_A1 -> /Heaters/BED_HEAT
- P27 pad 2: /Stepper Drivers/Z2_A2 -> CGND
- P28 pad 1: /Heaters/BED_HEAT -> /Heaters/E_HEAT
- P29 pad 1: /Heaters/E_HEAT -> /Heaters/H_HEAT
- P30 pad 1: /Heaters/H_HEAT -> /Heaters/DOCK0_HEAT
- P31 pad 1: /Heaters/DOCK0_HEAT -> /Heaters/DOCK1_HEAT
- P32 pad 1: /Heaters/DOCK1_HEAT -> /Fans/E_FAN
- P33 pad 1: /Fans/E_FAN -> /Fans/H_FAN
- P34 pad 1: /Fans/H_FAN -> /Fans/CASE_FAN
- P35 pad 1: /Fans/CASE_FAN -> Net-(FB19-Pad2)
- P35 pad 2: CGND -> Net-(FB20-Pad2)
- P36 pad 1: Net-(FB19-Pad2) -> Net-(F1-Pad1)
- P36 pad 2: Net-(FB20-Pad2) -> Net-(F1-Pad1)
- Q10 pad 3: Net-(D22-Pad1) -> Net-(D21-Pad1)
- Q13 pad 3: Net-(D25-Pad1) -> Net-(D24-Pad1)
- Q14 pad 3: Net-(D26-Pad1) -> Net-(D25-Pad1)
- Q16 pad 3: Net-(D29-Pad1) -> Net-(D28-Pad1)
- Q18 pad 3: Net-(D31-Pad1) -> Net-(D30-Pad1)
- Q20 pad 3: Net-(D33-Pad1) -> Net-(D32-Pad1)
- Q6 pad 3: Net-(D19-Pad1) -> Net-(D18-Pad1)
- Q9 pad 3: Net-(D21-Pad1) -> Net-(D20-Pad1)
- R100 pad 1: /HDMI/LCD.D14.R3--R6 -> /Z1_ENDSTOP
- R100 pad 2: CGND -> Net-(FB32-Pad2)
- R101 pad 1: VCC -> /Z1_ENDSTOP
- R101 pad 2: /HDMI/LCD.D13.R2--R5 -> VCC
- R102 pad 1: /HDMI/LCD.D12.R1--R4 -> /ENC_A
- R102 pad 2: CGND -> Net-(FB33-Pad2)
- R103 pad 1: /HDMI/LCD.D11.R0--R3 -> /ENC_B
- R103 pad 2: CGND -> Net-(FB34-Pad2)
- R104 pad 1: /HDMI/LCD.D15.R4--R7 -> VCC
- R104 pad 2: CGND -> /~SR_EN
- R105 pad 1: /HDMI/LCD.D10.G5--G7 -> VCC
- R105 pad 2: CGND -> /~SS_TOOLHEAD0_T
- R106 pad 1: /HDMI/LCD.D9.G4--G6 -> VCC
- R106 pad 2: CGND -> /~SS_TOOLHEAD0_NVM
- R107 pad 1: /HDMI/LCD.D8.G3--G5 -> VCC
- R107 pad 2: CGND -> /~SS_TOOLHEAD1_T
- R108 pad 1: /HDMI/LCD.D7.G2--G4 -> VCC
- R108 pad 2: CGND -> /~SS_TOOLHEAD1_NVM
- R109 pad 1: /HDMI/LCD.D6.G1--G3 -> VCC
- R109 pad 2: CGND -> /~SS_DOCK0_T
- R110 pad 2: /HDMI/LCD.D5.G0--G2 -> /~SS_DOCK0_NVM
- R111 pad 2: /HDMI/LCD.D4.B4--B7 -> /~SS_DOCK1_T
- R112 pad 2: /HDMI/LCD.D3.B3--B6 -> /~SS_DOCK1_NVM
- R113 pad 2: /HDMI/LCD.D2.B2--B5 -> /E_FAULT
- R114 pad 1: /HDMI/LCD.D1.B1--B4 -> VCC
- R114 pad 2: CGND -> /Stepper Drivers/~E_SS
- R120 pad 1: Net-(FB30-Pad2) -> VCC
- R120 pad 2: /BED_THERM -> /X2_ENDSTOP
- R121 pad 1: VDD_ADC -> VCC
- R121 pad 2: /Thermistors/ADC_IN -> /X_FAULT
- R122 pad 1: Net-(FB31-Pad2) -> VCC
- R122 pad 2: /ADC -> /Stepper Drivers/~X0_SS
- R123 pad 1: /X1_ENDSTOP -> /Stepper Drivers/X0 Stepper Driver/5VOUT
- R123 pad 2: Net-(FB32-Pad2) -> Net-(C76-Pad1)
- R124 pad 1: /X1_ENDSTOP -> /Stepper Drivers/X0 Stepper Driver/5VOUT
- R124 pad 2: VCC -> Net-(R124-Pad2)
- R125 pad 1: /Y1_ENDSTOP -> CGND
- R125 pad 2: Net-(FB33-Pad2) -> Net-(R124-Pad2)
- R126 pad 1: /Y1_ENDSTOP -> CGND
- R126 pad 2: VCC -> Net-(C87-Pad1)
- R127 pad 1: /Z1_ENDSTOP -> CGND
- R127 pad 2: Net-(FB34-Pad2) -> Net-(C90-Pad1)
- R128 pad 1: /Z1_ENDSTOP -> VCC
- R128 pad 2: VCC -> /Z2_ENDSTOP
- R129 pad 1: /ENC_A -> VCC
- R129 pad 2: Net-(FB35-Pad2) -> /Z_FAULT
- R130 pad 1: /ENC_B -> VCC
- R130 pad 2: Net-(FB36-Pad2) -> /Stepper Drivers/~Z0_SS
- R131 pad 1: VCC -> /Stepper Drivers/Z0 Stepper Driver/5VOUT
- R131 pad 2: /~SR_EN -> Net-(C92-Pad1)
- R132 pad 1: VCC -> /Stepper Drivers/Z0 Stepper Driver/5VOUT
- R132 pad 2: /~SS_TOOLHEAD0_T -> Net-(R132-Pad2)
- R133 pad 1: VCC -> CGND
- R133 pad 2: /~SS_TOOLHEAD0_NVM -> Net-(R132-Pad2)
- R134 pad 1: VCC -> CGND
- R134 pad 2: /~SS_TOOLHEAD1_T -> Net-(C103-Pad1)
- R135 pad 1: VCC -> CGND
- R135 pad 2: /~SS_TOOLHEAD1_NVM -> Net-(C106-Pad1)
- R136 pad 2: /~SS_DOCK0_T -> /Stepper Drivers/~Z1_SS
- R137 pad 1: VCC -> /Stepper Drivers/Z1 Stepper Driver/5VOUT
- R137 pad 2: /~SS_DOCK0_NVM -> Net-(C108-Pad1)
- R138 pad 1: VCC -> /Stepper Drivers/Z1 Stepper Driver/5VOUT
- R138 pad 2: /~SS_DOCK1_T -> Net-(R138-Pad2)
- R139 pad 1: VCC -> CGND
- R139 pad 2: /~SS_DOCK1_NVM -> Net-(R138-Pad2)
- R140 pad 1: VCC -> CGND
- R140 pad 2: /E_FAULT -> Net-(C119-Pad1)
- R141 pad 1: VCC -> CGND
- R141 pad 2: /Stepper Drivers/~E_SS -> Net-(C122-Pad1)
- R147 pad 1: VCC -> CGND
- R147 pad 2: /X2_ENDSTOP -> Net-(C138-Pad1)
- R148 pad 2: /X_FAULT -> /H_FAULT
- R149 pad 2: /Stepper Drivers/~X0_SS -> /Stepper Drivers/~H_SS
- R150 pad 1: /Stepper Drivers/X0 Stepper Driver/5VOUT -> /Stepper Drivers/H Stepper Driver/5VOUT
- R150 pad 2: Net-(C101-Pad1) -> Net-(C140-Pad1)
- R151 pad 1: /Stepper Drivers/X0 Stepper Driver/5VOUT -> /Stepper Drivers/H Stepper Driver/5VOUT
- R153 pad 2: Net-(C112-Pad1) -> Net-(C151-Pad1)
- R154 pad 2: Net-(C115-Pad1) -> Net-(C154-Pad1)
- R155 pad 2: /Z2_ENDSTOP -> /Y2_ENDSTOP
- R156 pad 2: /Z_FAULT -> /Y_FAULT
- R157 pad 2: /Stepper Drivers/~Z0_SS -> /Stepper Drivers/~Y_SS
- R158 pad 1: /Stepper Drivers/Z0 Stepper Driver/5VOUT -> /Stepper Drivers/Y Stepper Driver/5VOUT
- R158 pad 2: Net-(C117-Pad1) -> Net-(C156-Pad1)
- R159 pad 1: /Stepper Drivers/Z0 Stepper Driver/5VOUT -> /Stepper Drivers/Y Stepper Driver/5VOUT
- R161 pad 2: Net-(C128-Pad1) -> Net-(C167-Pad1)
- R162 pad 2: Net-(C131-Pad1) -> Net-(C170-Pad1)
- R163 pad 2: /Stepper Drivers/~Z1_SS -> /Stepper Drivers/~X1_SS
- R164 pad 1: /Stepper Drivers/Z1 Stepper Driver/5VOUT -> /Stepper Drivers/X1 Stepper Driver/5VOUT
- R164 pad 2: Net-(C133-Pad1) -> Net-(C172-Pad1)
- R165 pad 1: /Stepper Drivers/Z1 Stepper Driver/5VOUT -> /Stepper Drivers/X1 Stepper Driver/5VOUT
- R167 pad 2: Net-(C144-Pad1) -> Net-(C183-Pad1)
- R168 pad 2: Net-(C147-Pad1) -> Net-(C186-Pad1)
- R169 pad 2: /Stepper Drivers/~Z2_SS -> /CLKOUT2
- R170 pad 1: /Stepper Drivers/Z2 Stepper Driver/5VOUT -> Net-(Q5-Pad1)
- R170 pad 2: Net-(C149-Pad1) -> /PWM/BED_HEAT
- R171 pad 1: /Stepper Drivers/Z2 Stepper Driver/5VOUT -> CGND
- R171 pad 2: Net-(R171-Pad2) -> /PWM/BED_HEAT
- R172 pad 1: CGND -> +24V
- R172 pad 2: Net-(R171-Pad2) -> Net-(Q6-Pad1)
- R173 pad 1: CGND -> Net-(Q6-Pad1)
- R173 pad 2: Net-(C160-Pad1) -> Net-(Q5-Pad3)
- R174 pad 1: CGND -> Net-(D18-Pad1)
- R174 pad 2: Net-(C163-Pad1) -> Net-(D19-Pad2)
- R175 pad 1: VCC -> /Heaters/BED_HEAT
- R175 pad 2: /H_FAULT -> CGND
- R176 pad 1: VCC -> Net-(Q7-Pad1)
- R176 pad 2: /Stepper Drivers/~H_SS -> /PWM/E_HEAT
- R177 pad 1: /Stepper Drivers/H Stepper Driver/5VOUT -> Net-(Q8-Pad1)
- R177 pad 2: Net-(C165-Pad1) -> /PWM/DOCK0_HEAT
- R178 pad 1: /Stepper Drivers/H Stepper Driver/5VOUT -> CGND
- R178 pad 2: Net-(R178-Pad2) -> /PWM/E_HEAT
- R179 pad 2: Net-(R178-Pad2) -> /PWM/DOCK0_HEAT
- R180 pad 1: CGND -> +24V
- R180 pad 2: Net-(C176-Pad1) -> Net-(Q9-Pad1)
- R181 pad 1: CGND -> Net-(Q9-Pad1)
- R181 pad 2: Net-(C179-Pad1) -> Net-(Q7-Pad3)
- R182 pad 1: VCC -> +24V
- R182 pad 2: /Y2_ENDSTOP -> Net-(Q10-Pad1)
- R183 pad 1: VCC -> Net-(Q10-Pad1)
- R183 pad 2: /Y_FAULT -> Net-(Q8-Pad3)
- R184 pad 1: VCC -> Net-(D20-Pad1)
- R184 pad 2: /Stepper Drivers/~Y_SS -> Net-(D22-Pad2)
- R185 pad 1: /Stepper Drivers/Y Stepper Driver/5VOUT -> Net-(D21-Pad1)
- R185 pad 2: Net-(C181-Pad1) -> Net-(D23-Pad2)
- R186 pad 1: /Stepper Drivers/Y Stepper Driver/5VOUT -> /Heaters/E_HEAT
- R186 pad 2: Net-(R186-Pad2) -> CGND
- R187 pad 1: CGND -> /Heaters/DOCK0_HEAT
- R187 pad 2: Net-(R186-Pad2) -> CGND
- R188 pad 1: CGND -> Net-(Q11-Pad1)
- R188 pad 2: Net-(C192-Pad1) -> /PWM/H_HEAT
- R189 pad 1: CGND -> Net-(Q12-Pad1)
- R189 pad 2: Net-(C195-Pad1) -> /PWM/DOCK1_HEAT
- R190 pad 1: VCC -> CGND
- R190 pad 2: /Stepper Drivers/~X1_SS -> /PWM/H_HEAT
- R191 pad 1: /Stepper Drivers/X1 Stepper Driver/5VOUT -> CGND
- R191 pad 2: Net-(C197-Pad1) -> /PWM/DOCK1_HEAT
- R192 pad 1: /Stepper Drivers/X1 Stepper Driver/5VOUT -> +24V
- R192 pad 2: Net-(R192-Pad2) -> Net-(Q13-Pad1)
- R193 pad 1: CGND -> Net-(Q13-Pad1)
- R193 pad 2: Net-(R192-Pad2) -> Net-(Q11-Pad3)
- R194 pad 1: CGND -> +24V
- R194 pad 2: Net-(C208-Pad1) -> Net-(Q14-Pad1)
- R195 pad 1: CGND -> Net-(Q14-Pad1)
- R195 pad 2: Net-(C211-Pad1) -> Net-(Q12-Pad3)
- R196 pad 1: VCC -> Net-(D24-Pad1)
- R196 pad 2: /CLKOUT2 -> Net-(D26-Pad2)
- R197 pad 1: Net-(Q5-Pad1) -> Net-(D25-Pad1)
- R197 pad 2: /PWM/BED_HEAT -> Net-(D27-Pad2)
- R198 pad 1: CGND -> /Heaters/H_HEAT
- R198 pad 2: /PWM/BED_HEAT -> CGND
- R199 pad 1: +24V -> /Heaters/DOCK1_HEAT
- R199 pad 2: Net-(Q6-Pad1) -> CGND
- R200 pad 1: Net-(Q6-Pad1) -> Net-(Q15-Pad1)
- R200 pad 2: Net-(Q5-Pad3) -> /PWM/E_FAN
- R201 pad 1: Net-(D19-Pad1) -> CGND
- R201 pad 2: Net-(D20-Pad2) -> /PWM/E_FAN
- R202 pad 1: /Heaters/BED_HEAT -> +24V
- R202 pad 2: CGND -> Net-(Q16-Pad1)
- R203 pad 1: Net-(Q7-Pad1) -> Net-(Q16-Pad1)
- R203 pad 2: /PWM/E_HEAT -> Net-(Q15-Pad3)
- R204 pad 1: Net-(Q8-Pad1) -> Net-(D28-Pad1)
- R204 pad 2: /PWM/DOCK0_HEAT -> Net-(D29-Pad2)
- R205 pad 1: CGND -> /Fans/E_FAN
- R205 pad 2: /PWM/E_HEAT -> CGND
- R206 pad 1: CGND -> Net-(Q17-Pad1)
- R206 pad 2: /PWM/DOCK0_HEAT -> /PWM/H_FAN
- R207 pad 1: +24V -> CGND
- R207 pad 2: Net-(Q9-Pad1) -> /PWM/H_FAN
- R208 pad 1: Net-(Q9-Pad1) -> +24V
- R208 pad 2: Net-(Q7-Pad3) -> Net-(Q18-Pad1)
- R209 pad 1: +24V -> Net-(Q18-Pad1)
- R209 pad 2: Net-(Q10-Pad1) -> Net-(Q17-Pad3)
- R210 pad 1: Net-(Q10-Pad1) -> Net-(D30-Pad1)
- R210 pad 2: Net-(Q8-Pad3) -> Net-(D31-Pad2)
- R211 pad 1: Net-(D21-Pad1) -> /Fans/H_FAN
- R211 pad 2: Net-(D23-Pad2) -> CGND
- R212 pad 1: Net-(D22-Pad1) -> Net-(Q19-Pad1)
- R212 pad 2: Net-(D24-Pad2) -> /PWM/CASE_FAN
- R213 pad 1: /Heaters/E_HEAT -> CGND
- R213 pad 2: CGND -> /PWM/CASE_FAN
- R214 pad 1: /Heaters/DOCK0_HEAT -> +24V
- R214 pad 2: CGND -> Net-(Q20-Pad1)
- R215 pad 1: Net-(Q11-Pad1) -> Net-(Q20-Pad1)
- R215 pad 2: /PWM/H_HEAT -> Net-(Q19-Pad3)
- R216 pad 1: Net-(Q12-Pad1) -> Net-(D32-Pad1)
- R216 pad 2: /PWM/DOCK1_HEAT -> Net-(D33-Pad2)
- R217 pad 1: CGND -> /Fans/CASE_FAN
- R217 pad 2: /PWM/H_HEAT -> CGND
- R218 pad 1: CGND -> /Configuration/LCD.D0.B0--B3
- R218 pad 2: /PWM/DOCK1_HEAT -> CGND
- R219 pad 1: +24V -> Net-(R219-Pad1)
- R219 pad 2: Net-(Q13-Pad1) -> /Configuration/LCD.D2.B2--B5
- R220 pad 1: Net-(Q13-Pad1) -> /Configuration/LCD.D1.B1--B4
- R220 pad 2: Net-(Q11-Pad3) -> CGND
- R221 pad 1: +24V -> VCC
- R221 pad 2: Net-(Q14-Pad1) -> /Configuration/LCD.D2.B2--B5
- R222 pad 1: Net-(Q14-Pad1) -> VCC
- R222 pad 2: Net-(Q12-Pad3) -> /Configuration/LCD.D3.B3--B6
- R223 pad 1: Net-(D25-Pad1) -> VCC
- R223 pad 2: Net-(D27-Pad2) -> /Configuration/LCD.D4.B4--B7
- R224 pad 1: Net-(D26-Pad1) -> VCC
- R224 pad 2: Net-(D28-Pad2) -> /Configuration/LCD.D5.G0--G2
- R225 pad 1: /Heaters/H_HEAT -> /Configuration/LCD.D6.G1--G3
- R226 pad 1: /Heaters/DOCK1_HEAT -> /Configuration/LCD.D7.G2--G4
- R227 pad 1: Net-(Q15-Pad1) -> /Configuration/LCD.D8.G3--G5
- R227 pad 2: /PWM/E_FAN -> CGND
- R228 pad 1: CGND -> /Configuration/LCD.D9.G4--G6
- R228 pad 2: /PWM/E_FAN -> CGND
- R229 pad 1: +24V -> /Configuration/LCD.D10.G5--G7
- R229 pad 2: Net-(Q16-Pad1) -> CGND
- R230 pad 1: Net-(Q16-Pad1) -> /Configuration/LCD.D11.R0--R3
- R230 pad 2: Net-(Q15-Pad3) -> CGND
- R231 pad 1: Net-(D29-Pad1) -> /Configuration/LCD.D12.R1--R4
- R231 pad 2: Net-(D30-Pad2) -> CGND
- R232 pad 1: /Fans/E_FAN -> /Configuration/LCD.D13.R2--R5
- R233 pad 1: Net-(Q17-Pad1) -> VCC
- R233 pad 2: /PWM/H_FAN -> /Configuration/LCD.D14.R3--R6
- R234 pad 1: CGND -> /Configuration/LCD.D15.R4--R7
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Other:
- board text removed: "μHDMI"

Commit message: Read in the new netlist, HDMI removed from the layout
Parts:
- C6: value 100nF -> 22nF
- C7: value 22nF -> 100nF
- P14: value JTAG -> μSD; footprint KiMBo:JTAG -> KiMBo:SCHA5B0200
- P15: value μSD -> Ethernet; footprint KiMBo:SCHA5B0200 -> KiMBo:Ethernet-LPJ0011BBNL
- P16: value Ethernet -> JTAG; footprint KiMBo:Ethernet-LPJ0011BBNL -> KiMBo:JTAG
- R218: value 100kΩ -> 100Ω
- R219: value 100Ω -> 100kΩ
- R5: value 4.75kΩ -> 470Ω
- R6: value 470Ω -> 4.75kΩ
- moved C48 160.3 mm to (377.8, 132.8)
- moved R100 160.3 mm to (382.5, 132.8)
- moved C51 156.8 mm to (382.3, 126.9)
- moved FB31 155.9 mm to (367.6, 120.3)
- moved FB34 155.9 mm to (367.6, 127.3)
- moved C173 154.8 mm to (368.9, 160.7)
- moved C180 153.9 mm to (379.2, 160.3)
- moved R97 150.3 mm to (393.6, 124.5)
- moved C96 147.1 mm to (544.1, 12.9)
- moved R99 146.6 mm to (398.4, 118.7)
- moved C176 145.7 mm to (374.1, 160.3)
- moved C146 145.1 mm to (526.4, 42.7)
- moved R103 144.7 mm to (387.2, 132.8)
- moved C179 140.0 mm to (382.8, 154.5)
- moved C143 139.5 mm to (521.7, 42.7)
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Connections:
- C6 pad 1: VCC -> Net-(C6-Pad1)
- C7 pad 1: Net-(C7-Pad1) -> VCC
- P14 pad 1: /JTAG/JTAG_TMS -> /MMC0_DAT2
- P14 pad 10: CGND -> /SD.CD
- P14 pad 11: /TCK -> CGND
- P14 pad 13: /JTAG/JTAG_EMU0 -> CGND
- P14 pad 14: /JTAG/JTAG_EMU1 -> CGND
- P14 pad 15: /~SYS_RESET -> CGND
- P14 pad 2: /JTAG/~JTAG_TRST -> /MMC0_DAT3
- P14 pad 3: /JTAG/JTAG_TDI -> /MMC0_CMD
- P14 pad 4: CGND -> VCC
- P14 pad 5: VCC -> /MMC0_CLK
- P14 pad 6: Net-(P14-Pad6) -> CGND
- P14 pad 7: /JTAG/JTAG_TD0 -> /MMC0_DAT0
- P14 pad 8: CGND -> /MMC0_DAT1
- P14 pad 9: /TCK -> CGND
- P15 pad 1: /MMC0_DAT2 -> /Ethernet/RD+
- P15 pad 10: /SD.CD -> Net-(P15-Pad10)
- P15 pad 11: CGND -> Net-(P15-Pad11)
- P15 pad 12: CGND -> /Ethernet/YELA
- P15 pad 2: /MMC0_DAT3 -> /Ethernet/RD-
- P15 pad 3: /MMC0_CMD -> /Ethernet/TD+
- P15 pad 4: VCC -> Net-(C6-Pad1)
- P15 pad 5: /MMC0_CLK -> Net-(C6-Pad1)
- P15 pad 6: CGND -> /Ethernet/TD-
- P15 pad 7: /MMC0_DAT0 -> Net-(P15-Pad7)
- P15 pad 8: /MMC0_DAT1 -> CGND
- P15 pad 9: CGND -> /Ethernet/GRNA
- P16 pad 1: /Ethernet/RD+ -> /JTAG/JTAG_TMS
- P16 pad 10: Net-(P16-Pad10) -> CGND
- P16 pad 11: Net-(P16-Pad11) -> /TCK
- P16 pad 12: /Ethernet/YELA -> CGND
- P16 pad 13: CGND -> /JTAG/JTAG_EMU0
- P16 pad 14: CGND -> /JTAG/JTAG_EMU1
- P16 pad 2: /Ethernet/RD- -> /JTAG/~JTAG_TRST
- P16 pad 3: /Ethernet/TD+ -> /JTAG/JTAG_TDI
- P16 pad 4: Net-(C7-Pad1) -> CGND
- P16 pad 5: Net-(C7-Pad1) -> VCC
- P16 pad 6: /Ethernet/TD- -> Net-(P16-Pad6)
- P16 pad 7: Net-(P16-Pad7) -> /JTAG/JTAG_TD0
- P16 pad 9: /Ethernet/GRNA -> /TCK
- R218 pad 1: /Configuration/LCD.D0.B0--B3 -> Net-(R218-Pad1)
- R218 pad 2: CGND -> /Configuration/LCD.D2.B2--B5
- R219 pad 1: Net-(R219-Pad1) -> /Configuration/LCD.D0.B0--B3
- R219 pad 2: /Configuration/LCD.D2.B2--B5 -> CGND
- R5 pad 1: /JTAG/JTAG_EMU0 -> Net-(P15-Pad10)
- R5 pad 2: VCC -> CGND
- R6 pad 1: Net-(P16-Pad10) -> /JTAG/JTAG_EMU0
- R6 pad 2: CGND -> VCC
- R8 pad 1: Net-(P16-Pad11) -> Net-(P15-Pad11)
- R9 pad 2: Net-(C7-Pad1) -> Net-(C6-Pad1)
- SW3 pad 1: Net-(R219-Pad1) -> Net-(R218-Pad1)
- SW3 pad 3: Net-(R219-Pad1) -> Net-(R218-Pad1)
