File: KiMBo/KiMBo.kicad_pcb (KiCad board)
At the start: 6 copper layers, 187 x 127 mm, 615 parts, among them IC1 24LC32AT-I/OT, P1 TOOLHEAD0, P10 ADC, P11 Serial, P12 μUSB, P13 USB_Type_A, P14 μSD, P15 Ethernet, P16 JTAG, P17 LCD, P18 E_MOTOR, P19 H_MOTOR, P2 TOOLHEAD1, P20 X0_MOTOR, P21 X1_MOTOR, P22 Y0_MOTOR, P23 Y1_MOTOR, P24 Z0_MOTOR, P25 Z1_MOTOR, P26 Z2_MOTOR, P27 BED_HEAT, P28 E_HEAT, P29 H_HEAT, P3 DOCK0, P30 DOCK0_HEAT, P31 DOCK1_HEAT, P32 E_FAN, P33 H_FAN, P34 CASE_FAN, P35 PWM, P36 PWR_Input, P4 DOCK1, P5 X1, P6 Y1, P7 Z1, P8 ENC, P9 BED_THERM, Q1 2N7002, Q10 DMP3098L-7, Q11 2N7002, Q12 2N7002, Q13 DMP3098L-7, Q14 DMP3098L-7, Q15 2N7002, Q16 DMP3098L-7, Q17 2N7002, Q18 DMP3098L-7, Q19 2N7002, Q2 MMBT2907, Q20 DMP3098L-7, Q3 DNP-MMBT2907, Q4 IPD90P03P4-04, Q5 2N7002, Q6 IPD90P03P4-04, Q7 2N7002, Q8 2N7002, Q9 DMP3098L-7, SW1 RESET, SW2 Power, SW3 μSD_Boot, U1 OSD3358, U10 LAN8710A, U11 74HC595, U12 74HC595, U13 74HC595, U14 TMC2130, U15 TMC2130, U16 TMC2130, U17 TMC2130, U18 TMC2130, U19 TMC2130, U2 74LVC1G06, U20 TMC2130, U21 TMC2130, U22 PCA9685, U3 LM2592HVSX-5.0, U4 74LVC1G06, U5 EMMC**G-S100, U6 TPS2051B, U7 TPD4S012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

Commit message: More stepper motor driver progress
Parts:
- removed the R120 at (450.4, 98.3)
- removed the R121 at (435.0, 116.2)
- added R115: 4.7kΩ, Resistors_SMD:R_0603, F.Cu at (392.2, 50.5)
- added R116: 4.7kΩ, Resistors_SMD:R_0603, F.Cu at (387.3, 50.5)
- added R235: 100kΩ, Resistors_SMD:R_0603, F.Cu at (441.2, 114.2)
- added R236: 100kΩ, Resistors_SMD:R_0603, F.Cu at (450.0, 108.4)
- C48, C49: value 0.1μF -> 39nF
- C50, C51, C52: value 0.1μF -> 100nF
- R123, R131, R150, R158: value 2.2Ω -> 4.7kΩ
- R124, R132, R138, R144, R151, R159, R165: value 5.23kΩ -> 4.7kΩ
- R125, R133, R139, R145, R152, R160, R166: value 4.75kΩ -> 2.2Ω
- R126, R134, R140, R146, R153, R161, R167: value 220mΩ -> 5.23kΩ; footprint Resistors_SMD:R_0805 -> Resistors_SMD:R_0603
- R127, R135, R141, R147, R154, R162, R168: value 220mΩ -> 4.75kΩ; footprint Resistors_SMD:R_0805 -> Resistors_SMD:R_0603
- R128, R129, R136, R142, R148, R149, R155, R156, R163, R169: value 4.7kΩ -> 220mΩ; footprint Resistors_SMD:R_0603 -> Resistors_SMD:R_0805
- R137, R143, R164: value 2.2Ω -> 220mΩ; footprint Resistors_SMD:R_0603 -> Resistors_SMD:R_0805
- R170: value 10Ω -> 220mΩ; footprint Resistors_SMD:R_0603 -> Resistors_SMD:R_0805
- R172, R178, R179, R190, R191, R202, R208, R214: value 4.7kΩ -> 10Ω
- R176, R177, R188, R189, R200, R206, R212: value 10Ω -> 10kΩ
- R186, R187, R198, R199, R201, R207, R213: value 4.7kΩ -> 10kΩ
- R218: value 100Ω -> 10kΩ
- R219: value 100kΩ -> 10kΩ
- R220: value 100kΩ -> 100Ω
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- renumbered R115 to R117, R116 to R118, R117 to R119, R118 to R120, R119 to R121
Connections:
- P18 pad 3: /Stepper Drivers/E_B1 -> /Stepper Drivers/E_B2
- P18 pad 4: /Stepper Drivers/E_B2 -> /Stepper Drivers/E_B1
- P19 pad 3: /Stepper Drivers/H_B1 -> /Stepper Drivers/H_B2
- P19 pad 4: /Stepper Drivers/H_B2 -> /Stepper Drivers/H_B1
- P20 pad 3: /Stepper Drivers/X0_B1 -> /Stepper Drivers/X0_B2
- P20 pad 4: /Stepper Drivers/X0_B2 -> /Stepper Drivers/X0_B1
- P21 pad 1: /Stepper Drivers/X1_B2 -> /Stepper Drivers/X1_A1
- P21 pad 2: /Stepper Drivers/X1_B1 -> /Stepper Drivers/X1_A2
- P21 pad 3: /Stepper Drivers/X1_A2 -> /Stepper Drivers/X1_B2
- P21 pad 4: /Stepper Drivers/X1_A1 -> /Stepper Drivers/X1_B1
- P24 pad 3: /Stepper Drivers/Z0_B1 -> /Stepper Drivers/Z0_B2
- P24 pad 4: /Stepper Drivers/Z0_B2 -> /Stepper Drivers/Z0_B1
- P25 pad 3: /Stepper Drivers/Z1_B1 -> /Stepper Drivers/Z1_B2
- P25 pad 4: /Stepper Drivers/Z1_B2 -> /Stepper Drivers/Z1_B1
- P26 pad 3: /Stepper Drivers/Z2_B1 -> /Stepper Drivers/Z2_B2
- P26 pad 4: /Stepper Drivers/Z2_B2 -> /Stepper Drivers/Z2_B1
- R105 pad 2: /~SS_TOOLHEAD0_T -> Net-(R105-Pad2)
- R107 pad 2: /~SS_TOOLHEAD1_T -> Net-(R107-Pad2)
- R113 pad 1: VCC -> /~SS_TOOLHEAD0_T
- R113 pad 2: /E_FAULT -> Net-(R105-Pad2)
- R114 pad 1: VCC -> /~SS_TOOLHEAD1_T
- R114 pad 2: /Stepper Drivers/~E_SS -> Net-(R107-Pad2)
- R122 pad 2: /Stepper Drivers/~X0_SS -> /X2_ENDSTOP
- R123 pad 1: /Stepper Drivers/X0 Stepper Driver/5VOUT -> VCC
- R123 pad 2: Net-(C76-Pad1) -> /X_FAULT
- R124 pad 1: /Stepper Drivers/X0 Stepper Driver/5VOUT -> VCC
- R124 pad 2: Net-(R124-Pad2) -> /Stepper Drivers/~X0_SS
- R125 pad 1: CGND -> /Stepper Drivers/X0 Stepper Driver/5VOUT
- R125 pad 2: Net-(R124-Pad2) -> Net-(C76-Pad1)
- R126 pad 1: CGND -> /Stepper Drivers/X0 Stepper Driver/5VOUT
- R126 pad 2: Net-(C87-Pad1) -> Net-(R126-Pad2)
- R127 pad 2: Net-(C90-Pad1) -> Net-(R126-Pad2)
- R128 pad 1: VCC -> CGND
- R128 pad 2: /Z2_ENDSTOP -> Net-(C87-Pad1)
- R129 pad 1: VCC -> CGND
- R129 pad 2: /Z_FAULT -> Net-(C90-Pad1)
- R130 pad 2: /Stepper Drivers/~Z0_SS -> /Z2_ENDSTOP
- R131 pad 1: /Stepper Drivers/Z0 Stepper Driver/5VOUT -> VCC
- R131 pad 2: Net-(C92-Pad1) -> /Z_FAULT
- R132 pad 1: /Stepper Drivers/Z0 Stepper Driver/5VOUT -> VCC
- R132 pad 2: Net-(R132-Pad2) -> /Stepper Drivers/~Z0_SS
- R133 pad 1: CGND -> /Stepper Drivers/Z0 Stepper Driver/5VOUT
- R133 pad 2: Net-(R132-Pad2) -> Net-(C92-Pad1)
- R134 pad 1: CGND -> /Stepper Drivers/Z0 Stepper Driver/5VOUT
- R134 pad 2: Net-(C103-Pad1) -> Net-(R134-Pad2)
- R135 pad 2: Net-(C106-Pad1) -> Net-(R134-Pad2)
- R136 pad 1: VCC -> CGND
- R136 pad 2: /Stepper Drivers/~Z1_SS -> Net-(C103-Pad1)
- R137 pad 1: /Stepper Drivers/Z1 Stepper Driver/5VOUT -> CGND
- R137 pad 2: Net-(C108-Pad1) -> Net-(C106-Pad1)
- R138 pad 1: /Stepper Drivers/Z1 Stepper Driver/5VOUT -> VCC
- R138 pad 2: Net-(R138-Pad2) -> /Stepper Drivers/~Z1_SS
- R139 pad 1: CGND -> /Stepper Drivers/Z1 Stepper Driver/5VOUT
- R139 pad 2: Net-(R138-Pad2) -> Net-(C108-Pad1)
- R140 pad 1: CGND -> /Stepper Drivers/Z1 Stepper Driver/5VOUT
- R140 pad 2: Net-(C119-Pad1) -> Net-(R140-Pad2)
- R141 pad 2: Net-(C122-Pad1) -> Net-(R140-Pad2)
- R142 pad 1: VCC -> CGND
- R142 pad 2: /Stepper Drivers/~Z2_SS -> Net-(C119-Pad1)
- R143 pad 1: /Stepper Drivers/Z2 Stepper Driver/5VOUT -> CGND
- R143 pad 2: Net-(C124-Pad1) -> Net-(C122-Pad1)
- R144 pad 1: /Stepper Drivers/Z2 Stepper Driver/5VOUT -> VCC
- R144 pad 2: Net-(R144-Pad2) -> /Stepper Drivers/~Z2_SS
- R145 pad 1: CGND -> /Stepper Drivers/Z2 Stepper Driver/5VOUT
- R145 pad 2: Net-(R144-Pad2) -> Net-(C124-Pad1)
- R146 pad 1: CGND -> /Stepper Drivers/Z2 Stepper Driver/5VOUT
- R146 pad 2: Net-(C135-Pad1) -> Net-(R146-Pad2)
- R147 pad 2: Net-(C138-Pad1) -> Net-(R146-Pad2)
- R148 pad 1: VCC -> CGND
- R148 pad 2: /H_FAULT -> Net-(C135-Pad1)
- R149 pad 1: VCC -> CGND
- R149 pad 2: /Stepper Drivers/~H_SS -> Net-(C138-Pad1)
- R150 pad 1: /Stepper Drivers/H Stepper Driver/5VOUT -> VCC
- R150 pad 2: Net-(C140-Pad1) -> /H_FAULT
- R151 pad 1: /Stepper Drivers/H Stepper Driver/5VOUT -> VCC
- R151 pad 2: Net-(R151-Pad2) -> /Stepper Drivers/~H_SS
- R152 pad 1: CGND -> /Stepper Drivers/H Stepper Driver/5VOUT
- R152 pad 2: Net-(R151-Pad2) -> Net-(C140-Pad1)
- R153 pad 1: CGND -> /Stepper Drivers/H Stepper Driver/5VOUT
- R153 pad 2: Net-(C151-Pad1) -> Net-(R153-Pad2)
- R154 pad 2: Net-(C154-Pad1) -> Net-(R153-Pad2)
- R155 pad 1: VCC -> CGND
- R155 pad 2: /Y2_ENDSTOP -> Net-(C151-Pad1)
- R156 pad 1: VCC -> CGND
- R156 pad 2: /Y_FAULT -> Net-(C154-Pad1)
- R157 pad 2: /Stepper Drivers/~Y_SS -> /Y2_ENDSTOP
- R158 pad 1: /Stepper Drivers/Y Stepper Driver/5VOUT -> VCC
- R158 pad 2: Net-(C156-Pad1) -> /Y_FAULT
- R159 pad 1: /Stepper Drivers/Y Stepper Driver/5VOUT -> VCC
- R159 pad 2: Net-(R159-Pad2) -> /Stepper Drivers/~Y_SS
- R160 pad 1: CGND -> /Stepper Drivers/Y Stepper Driver/5VOUT
- R160 pad 2: Net-(R159-Pad2) -> Net-(C156-Pad1)
- R161 pad 1: CGND -> /Stepper Drivers/Y Stepper Driver/5VOUT
- R161 pad 2: Net-(C167-Pad1) -> Net-(R161-Pad2)
- R162 pad 2: Net-(C170-Pad1) -> Net-(R161-Pad2)
- R163 pad 1: VCC -> CGND
- R163 pad 2: /Stepper Drivers/~X1_SS -> Net-(C167-Pad1)
- R164 pad 1: /Stepper Drivers/X1 Stepper Driver/5VOUT -> CGND
- R164 pad 2: Net-(C172-Pad1) -> Net-(C170-Pad1)
- R165 pad 1: /Stepper Drivers/X1 Stepper Driver/5VOUT -> VCC
- R165 pad 2: Net-(R165-Pad2) -> /Stepper Drivers/~X1_SS
- R166 pad 1: CGND -> /Stepper Drivers/X1 Stepper Driver/5VOUT
- R166 pad 2: Net-(R165-Pad2) -> Net-(C172-Pad1)
- R167 pad 1: CGND -> /Stepper Drivers/X1 Stepper Driver/5VOUT
- R167 pad 2: Net-(C183-Pad1) -> Net-(R167-Pad2)
- R168 pad 2: Net-(C186-Pad1) -> Net-(R167-Pad2)
- R169 pad 1: VCC -> CGND
- R169 pad 2: /CLKOUT2 -> Net-(C183-Pad1)
- R170 pad 1: Net-(Q5-Pad1) -> CGND
- R170 pad 2: /PWM/BED_HEAT -> Net-(C186-Pad1)
- R171 pad 1: CGND -> VCC
- R171 pad 2: /PWM/BED_HEAT -> /CLKOUT2
- R172 pad 1: +24V -> Net-(Q5-Pad1)
- R172 pad 2: Net-(Q6-Pad1) -> /PWM/BED_HEAT
- R173 pad 1: Net-(Q6-Pad1) -> CGND
- R173 pad 2: Net-(Q5-Pad3) -> /PWM/BED_HEAT
- R174 pad 1: Net-(D18-Pad1) -> +24V
- R174 pad 2: Net-(D19-Pad2) -> Net-(Q6-Pad1)
- R175 pad 1: /Heaters/BED_HEAT -> Net-(Q6-Pad1)
- R175 pad 2: CGND -> Net-(Q5-Pad3)
- R176 pad 1: Net-(Q7-Pad1) -> Net-(D18-Pad1)
- R176 pad 2: /PWM/E_HEAT -> Net-(D19-Pad2)
- R177 pad 1: Net-(Q8-Pad1) -> /Heaters/BED_HEAT
- R177 pad 2: /PWM/DOCK0_HEAT -> CGND
- R178 pad 1: CGND -> Net-(Q7-Pad1)
- R179 pad 1: CGND -> Net-(Q8-Pad1)
- R180 pad 1: +24V -> CGND
- R180 pad 2: Net-(Q9-Pad1) -> /PWM/E_HEAT
- R181 pad 1: Net-(Q9-Pad1) -> CGND
- R181 pad 2: Net-(Q7-Pad3) -> /PWM/DOCK0_HEAT
- R182 pad 2: Net-(Q10-Pad1) -> Net-(Q9-Pad1)
- R183 pad 1: Net-(Q10-Pad1) -> Net-(Q9-Pad1)
- R183 pad 2: Net-(Q8-Pad3) -> Net-(Q7-Pad3)
- R184 pad 1: Net-(D20-Pad1) -> +24V
- R184 pad 2: Net-(D22-Pad2) -> Net-(Q10-Pad1)
- R185 pad 1: Net-(D21-Pad1) -> Net-(Q10-Pad1)
- R185 pad 2: Net-(D23-Pad2) -> Net-(Q8-Pad3)
- R186 pad 1: /Heaters/E_HEAT -> Net-(D20-Pad1)
- R186 pad 2: CGND -> Net-(D22-Pad2)
- R187 pad 1: /Heaters/DOCK0_HEAT -> Net-(D21-Pad1)
- R187 pad 2: CGND -> Net-(D23-Pad2)
- R188 pad 1: Net-(Q11-Pad1) -> /Heaters/E_HEAT
- R188 pad 2: /PWM/H_HEAT -> CGND
- R189 pad 1: Net-(Q12-Pad1) -> /Heaters/DOCK0_HEAT
- R189 pad 2: /PWM/DOCK1_HEAT -> CGND
- R190 pad 1: CGND -> Net-(Q11-Pad1)
- R191 pad 1: CGND -> Net-(Q12-Pad1)
- R192 pad 1: +24V -> CGND
- R192 pad 2: Net-(Q13-Pad1) -> /PWM/H_HEAT
- R193 pad 1: Net-(Q13-Pad1) -> CGND
- R193 pad 2: Net-(Q11-Pad3) -> /PWM/DOCK1_HEAT
- R194 pad 2: Net-(Q14-Pad1) -> Net-(Q13-Pad1)
- R195 pad 1: Net-(Q14-Pad1) -> Net-(Q13-Pad1)
- R195 pad 2: Net-(Q12-Pad3) -> Net-(Q11-Pad3)
- R196 pad 1: Net-(D24-Pad1) -> +24V
- R196 pad 2: Net-(D26-Pad2) -> Net-(Q14-Pad1)
- R197 pad 1: Net-(D25-Pad1) -> Net-(Q14-Pad1)
- R197 pad 2: Net-(D27-Pad2) -> Net-(Q12-Pad3)
- R198 pad 1: /Heaters/H_HEAT -> Net-(D24-Pad1)
- R198 pad 2: CGND -> Net-(D26-Pad2)
- R199 pad 1: /Heaters/DOCK1_HEAT -> Net-(D25-Pad1)
- R199 pad 2: CGND -> Net-(D27-Pad2)
- R200 pad 1: Net-(Q15-Pad1) -> /Heaters/H_HEAT
- R200 pad 2: /PWM/E_FAN -> CGND
- R201 pad 1: CGND -> /Heaters/DOCK1_HEAT
- R201 pad 2: /PWM/E_FAN -> CGND
- R202 pad 1: +24V -> Net-(Q15-Pad1)
- R202 pad 2: Net-(Q16-Pad1) -> /PWM/E_FAN
- R203 pad 1: Net-(Q16-Pad1) -> CGND
- R203 pad 2: Net-(Q15-Pad3) -> /PWM/E_FAN
- R204 pad 1: Net-(D28-Pad1) -> +24V
- R204 pad 2: Net-(D29-Pad2) -> Net-(Q16-Pad1)
- R205 pad 1: /Fans/E_FAN -> Net-(Q16-Pad1)
- R205 pad 2: CGND -> Net-(Q15-Pad3)
- R206 pad 1: Net-(Q17-Pad1) -> Net-(D28-Pad1)
- R206 pad 2: /PWM/H_FAN -> Net-(D29-Pad2)
- R207 pad 1: CGND -> /Fans/E_FAN
- R207 pad 2: /PWM/H_FAN -> CGND
- R208 pad 1: +24V -> Net-(Q17-Pad1)
- R208 pad 2: Net-(Q18-Pad1) -> /PWM/H_FAN
- R209 pad 1: Net-(Q18-Pad1) -> CGND
- R209 pad 2: Net-(Q17-Pad3) -> /PWM/H_FAN
- R210 pad 1: Net-(D30-Pad1) -> +24V
- R210 pad 2: Net-(D31-Pad2) -> Net-(Q18-Pad1)
- R211 pad 1: /Fans/H_FAN -> Net-(Q18-Pad1)
- R211 pad 2: CGND -> Net-(Q17-Pad3)
- R212 pad 1: Net-(Q19-Pad1) -> Net-(D30-Pad1)
- R212 pad 2: /PWM/CASE_FAN -> Net-(D31-Pad2)
- R213 pad 1: CGND -> /Fans/H_FAN
- R213 pad 2: /PWM/CASE_FAN -> CGND
- R214 pad 1: +24V -> Net-(Q19-Pad1)
- R214 pad 2: Net-(Q20-Pad1) -> /PWM/CASE_FAN
- R215 pad 1: Net-(Q20-Pad1) -> CGND
- R215 pad 2: Net-(Q19-Pad3) -> /PWM/CASE_FAN
- R216 pad 1: Net-(D32-Pad1) -> +24V
- R216 pad 2: Net-(D33-Pad2) -> Net-(Q20-Pad1)
- R217 pad 1: /Fans/CASE_FAN -> Net-(Q20-Pad1)
- R217 pad 2: CGND -> Net-(Q19-Pad3)
- R218 pad 1: Net-(R218-Pad1) -> Net-(D32-Pad1)
- R218 pad 2: /Configuration/LCD.D2.B2--B5 -> Net-(D33-Pad2)
- R219 pad 1: /Configuration/LCD.D0.B0--B3 -> /Fans/CASE_FAN
- R220 pad 1: /Configuration/LCD.D1.B1--B4 -> Net-(R220-Pad1)
- R220 pad 2: CGND -> /Configuration/LCD.D2.B2--B5
- R221 pad 1: VCC -> /Configuration/LCD.D0.B0--B3
- R221 pad 2: /Configuration/LCD.D2.B2--B5 -> CGND
- R222 pad 1: VCC -> /Configuration/LCD.D1.B1--B4
- R222 pad 2: /Configuration/LCD.D3.B3--B6 -> CGND
- R223 pad 2: /Configuration/LCD.D4.B4--B7 -> /Configuration/LCD.D2.B2--B5
- R224 pad 2: /Configuration/LCD.D5.G0--G2 -> /Configuration/LCD.D3.B3--B6
- R225 pad 1: /Configuration/LCD.D6.G1--G3 -> VCC
- R225 pad 2: CGND -> /Configuration/LCD.D4.B4--B7
- R226 pad 1: /Configuration/LCD.D7.G2--G4 -> VCC
- R226 pad 2: CGND -> /Configuration/LCD.D5.G0--G2
- R227 pad 1: /Configuration/LCD.D8.G3--G5 -> /Configuration/LCD.D6.G1--G3
- R228 pad 1: /Configuration/LCD.D9.G4--G6 -> /Configuration/LCD.D7.G2--G4
- R229 pad 1: /Configuration/LCD.D10.G5--G7 -> /Configuration/LCD.D8.G3--G5
- R230 pad 1: /Configuration/LCD.D11.R0--R3 -> /Configuration/LCD.D9.G4--G6
- R231 pad 1: /Configuration/LCD.D12.R1--R4 -> /Configuration/LCD.D10.G5--G7
- R232 pad 1: /Configuration/LCD.D13.R2--R5 -> /Configuration/LCD.D11.R0--R3
- R233 pad 1: VCC -> /Configuration/LCD.D12.R1--R4
- R233 pad 2: /Configuration/LCD.D14.R3--R6 -> CGND
- R234 pad 1: /Configuration/LCD.D15.R4--R7 -> /Configuration/LCD.D13.R2--R5
- SW3 pad 1: Net-(R218-Pad1) -> Net-(R220-Pad1)
- SW3 pad 3: Net-(R218-Pad1) -> Net-(R220-Pad1)
- U11 pad 15: /~SS_TOOLHEAD0_T -> Net-(R105-Pad2)
- U11 pad 2: /~SS_TOOLHEAD1_T -> Net-(R107-Pad2)
- U15 pad 23: Net-(R124-Pad2) -> Net-(R126-Pad2)
- U16 pad 23: Net-(R132-Pad2) -> Net-(R134-Pad2)
- U17 pad 23: Net-(R138-Pad2) -> Net-(R140-Pad2)
- U18 pad 23: Net-(R144-Pad2) -> Net-(R146-Pad2)
- U19 pad 23: Net-(R151-Pad2) -> Net-(R153-Pad2)
- U20 pad 23: Net-(R159-Pad2) -> Net-(R161-Pad2)
- U21 pad 23: Net-(R165-Pad2) -> Net-(R167-Pad2)
Routing:
- net +24V: track 26.5 -> 31.2 mm, vias 10 -> 11
- net Net-(R118-Pad2): track 4.90 -> 3.38 mm
- net /Stepper Drivers/E Stepper Driver/5VOUT: track 6.69 -> 5.23 mm
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- added copper zone on In4.Cu, net +24V
- added copper zone on In2.Cu, net /Stepper Drivers/E_B1
- added copper zone on In1.Cu, net CGND

Commit message: Duplicate the stepper circuit, remove extra Y connector
The Y motors will be wired in series through the motor connectors on the machine
Parts:
- removed the C59 at (194.0, 124.4)
- removed the C60 at (198.4, 135.0)
- removed the C61 at (201.9, 132.0)
- removed the C62 at (196.0, 134.8)
- removed the C63 at (200.1, 134.4)
- removed the C64 at (202.0, 128.4)
- removed the C65 at (189.0, 128.4)
- removed the C66 at (201.8, 134.4)
- removed the C67 at (199.4, 124.8)
- removed the C68 at (191.6, 124.8)
- removed the C69 at (201.9, 130.3)
- removed the C70 at (189.6, 130.5)
- removed the C71 at (188.7, 124.1)
- removed the C72 at (188.9, 136.6)
- removed the C73 at (188.2, 117.7)
- removed the C74 at (202.3, 124.1)
- removed the P18 at (199.3, 140.3)
- removed P23: Y1_MOTOR, Pin_Headers:Pin_Header_Angled_1x04
- removed the R117 at (196.0, 136.6)
- removed the R118 at (193.6, 135.3)
- removed the R119 at (191.7, 135.3)
- removed the R120 at (188.7, 126.1)
- removed the R121 at (202.3, 126.1)
- removed the U14 at (195.5, 129.5)
- added C59 (x2): 100nF, Capacitors_SMD:C_0603, F.Cu at (113.0, 142.9)
- added C59 (x2): 100nF, Capacitors_SMD:C_0603, F.Cu at (167.0, 142.9)
- added C59 (x2): 100nF, Capacitors_SMD:C_0603, F.Cu at (185.0, 142.9)
- added C59 (x2): 100nF, Capacitors_SMD:C_0603, F.Cu at (203.0, 142.9)
- added C59 (x2): 100nF, Capacitors_SMD:C_0603, F.Cu at (221.0, 142.9)
- added C59 (x2): 100nF, Capacitors_SMD:C_0603, F.Cu at (149.0, 142.9)
- added C59 (x2): 100nF, Capacitors_SMD:C_0603, F.Cu at (95.0, 142.9)
- added C59 (x2): 100nF, Capacitors_SMD:C_0603, F.Cu at (131.0, 142.9)
- added C60 (x2): 470nF, Capacitors_SMD:C_0603, F.Cu at (153.4, 153.5)
- added C60 (x2): 470nF, Capacitors_SMD:C_0603, F.Cu at (171.4, 153.5)
- added C60 (x2): 470nF, Capacitors_SMD:C_0603, F.Cu at (189.4, 153.5)
- added C60 (x2): 470nF, Capacitors_SMD:C_0603, F.Cu at (207.4, 153.5)
- added C60 (x2): 470nF, Capacitors_SMD:C_0603, F.Cu at (225.4, 153.5)
- added C60 (x2): 470nF, Capacitors_SMD:C_0603, F.Cu at (99.4, 153.5)
- added C60 (x2): 470nF, Capacitors_SMD:C_0603, F.Cu at (117.4, 153.5)
- added C60 (x2): 470nF, Capacitors_SMD:C_0603, F.Cu at (135.4, 153.5)
- added C61 (x2): 100nF, Capacitors_SMD:C_0603, F.Cu at (120.9, 150.5)
- added C61 (x2): 100nF, Capacitors_SMD:C_0603, F.Cu at (192.9, 150.5)
- added C61 (x2): 100nF, Capacitors_SMD:C_0603, F.Cu at (174.9, 150.5)
- added C61 (x2): 100nF, Capacitors_SMD:C_0603, F.Cu at (210.9, 150.5)
- added C61 (x2): 100nF, Capacitors_SMD:C_0603, F.Cu at (228.9, 150.5)
- added C61 (x2): 100nF, Capacitors_SMD:C_0603, F.Cu at (156.9, 150.5)
- added C61 (x2): 100nF, Capacitors_SMD:C_0603, F.Cu at (138.9, 150.5)
- added C61 (x2): 100nF, Capacitors_SMD:C_0603, F.Cu at (102.9, 150.5)
- added C62 (x2): 4.7μF, Capacitors_SMD:C_0603, F.Cu at (97.0, 153.3)
- added C62 (x2): 4.7μF, Capacitors_SMD:C_0603, F.Cu at (187.0, 153.3)
- added C62 (x2): 4.7μF, Capacitors_SMD:C_0603, F.Cu at (169.0, 153.3)
- added C62 (x2): 4.7μF, Capacitors_SMD:C_0603, F.Cu at (205.0, 153.3)
- added C62 (x2): 4.7μF, Capacitors_SMD:C_0603, F.Cu at (223.0, 153.3)
- added C62 (x2): 4.7μF, Capacitors_SMD:C_0603, F.Cu at (115.0, 153.3)
- added C62 (x2): 4.7μF, Capacitors_SMD:C_0603, F.Cu at (151.0, 153.3)
- added C62 (x2): 4.7μF, Capacitors_SMD:C_0603, F.Cu at (133.0, 153.3)
- added C63 (x2): 22nF, Capacitors_SMD:C_0603, F.Cu at (101.1, 152.9)
- added C63 (x2): 22nF, Capacitors_SMD:C_0603, F.Cu at (173.1, 152.9)
- added C63 (x2): 22nF, Capacitors_SMD:C_0603, F.Cu at (191.1, 152.9)
- added C63 (x2): 22nF, Capacitors_SMD:C_0603, F.Cu at (209.1, 152.9)
- added C63 (x2): 22nF, Capacitors_SMD:C_0603, F.Cu at (227.1, 152.9)
- added C63 (x2): 22nF, Capacitors_SMD:C_0603, F.Cu at (155.1, 152.9)
- added C63 (x2): 22nF, Capacitors_SMD:C_0603, F.Cu at (137.1, 152.9)
- added C63 (x2): 22nF, Capacitors_SMD:C_0603, F.Cu at (119.1, 152.9)
- added C64 (x2): 470pF, Capacitors_SMD:C_0603, F.Cu at (157.0, 146.9)
- added C64 (x2): 470pF, Capacitors_SMD:C_0603, F.Cu at (193.0, 146.9)
- added C64 (x2): 470pF, Capacitors_SMD:C_0603, F.Cu at (175.0, 146.9)
- added C64 (x2): 470pF, Capacitors_SMD:C_0603, F.Cu at (211.0, 146.9)
- added C64 (x2): 470pF, Capacitors_SMD:C_0603, F.Cu at (229.0, 146.9)
- added C64 (x2): 470pF, Capacitors_SMD:C_0603, F.Cu at (103.0, 146.9)
- added C64 (x2): 470pF, Capacitors_SMD:C_0603, F.Cu at (121.0, 146.9)
- added C64 (x2): 470pF, Capacitors_SMD:C_0603, F.Cu at (139.0, 146.9)
- added C65 (x2): 470pF, Capacitors_SMD:C_0603, F.Cu at (144.0, 146.9)
- added C65 (x2): 470pF, Capacitors_SMD:C_0603, F.Cu at (162.0, 146.9)
- added C65 (x2): 470pF, Capacitors_SMD:C_0603, F.Cu at (180.0, 146.9)
- added C65 (x2): 470pF, Capacitors_SMD:C_0603, F.Cu at (198.0, 146.9)
- added C65 (x2): 470pF, Capacitors_SMD:C_0603, F.Cu at (216.0, 146.9)
- added C65 (x2): 470pF, Capacitors_SMD:C_0603, F.Cu at (108.0, 146.9)
- added C65 (x2): 470pF, Capacitors_SMD:C_0603, F.Cu at (126.0, 146.9)
- added C65 (x2): 470pF, Capacitors_SMD:C_0603, F.Cu at (90.0, 146.9)
- added C66 (x2): 100nF, Capacitors_SMD:C_0603, F.Cu at (138.8, 152.9)
- added C66 (x2): 100nF, Capacitors_SMD:C_0603, F.Cu at (192.8, 152.9)
- added C66 (x2): 100nF, Capacitors_SMD:C_0603, F.Cu at (174.8, 152.9)
- added C66 (x2): 100nF, Capacitors_SMD:C_0603, F.Cu at (210.8, 152.9)
- added C66 (x2): 100nF, Capacitors_SMD:C_0603, F.Cu at (228.8, 152.9)
- added C66 (x2): 100nF, Capacitors_SMD:C_0603, F.Cu at (120.8, 152.9)
- added C66 (x2): 100nF, Capacitors_SMD:C_0603, F.Cu at (102.8, 152.9)
- added C66 (x2): 100nF, Capacitors_SMD:C_0603, F.Cu at (156.8, 152.9)
- added C67 (x2): 470pF, Capacitors_SMD:C_0603, F.Cu at (154.4, 143.3)
- added C67 (x2): 470pF, Capacitors_SMD:C_0603, F.Cu at (172.4, 143.3)
- added C67 (x2): 470pF, Capacitors_SMD:C_0603, F.Cu at (190.4, 143.3)
- added C67 (x2): 470pF, Capacitors_SMD:C_0603, F.Cu at (208.4, 143.3)
- added C67 (x2): 470pF, Capacitors_SMD:C_0603, F.Cu at (226.4, 143.3)
- added C67 (x2): 470pF, Capacitors_SMD:C_0603, F.Cu at (118.4, 143.3)
- added C67 (x2): 470pF, Capacitors_SMD:C_0603, F.Cu at (100.4, 143.3)
- added C67 (x2): 470pF, Capacitors_SMD:C_0603, F.Cu at (136.4, 143.3)
- added C68 (x2): 470pF, Capacitors_SMD:C_0603, F.Cu at (92.6, 143.3)
- added C68 (x2): 470pF, Capacitors_SMD:C_0603, F.Cu at (182.6, 143.3)
- added C68 (x2): 470pF, Capacitors_SMD:C_0603, F.Cu at (164.6, 143.3)
- added C68 (x2): 470pF, Capacitors_SMD:C_0603, F.Cu at (200.6, 143.3)
- added C68 (x2): 470pF, Capacitors_SMD:C_0603, F.Cu at (218.6, 143.3)
- added C68 (x2): 470pF, Capacitors_SMD:C_0603, F.Cu at (128.6, 143.3)
- added C68 (x2): 470pF, Capacitors_SMD:C_0603, F.Cu at (146.6, 143.3)
- added C68 (x2): 470pF, Capacitors_SMD:C_0603, F.Cu at (110.6, 143.3)
- added C69 (x2): 100nF, Capacitors_SMD:C_0603, F.Cu at (156.9, 148.8)
- added C69 (x2): 100nF, Capacitors_SMD:C_0603, F.Cu at (174.9, 148.8)
- added C69 (x2): 100nF, Capacitors_SMD:C_0603, F.Cu at (192.9, 148.8)
- added C69 (x2): 100nF, Capacitors_SMD:C_0603, F.Cu at (210.9, 148.8)
- added C69 (x2): 100nF, Capacitors_SMD:C_0603, F.Cu at (228.9, 148.8)
- added C69 (x2): 100nF, Capacitors_SMD:C_0603, F.Cu at (120.9, 148.8)
- added C69 (x2): 100nF, Capacitors_SMD:C_0603, F.Cu at (102.9, 148.8)
- added C69 (x2): 100nF, Capacitors_SMD:C_0603, F.Cu at (138.9, 148.8)
- added C70 (x2): 100nF, Capacitors_SMD:C_0603, F.Cu at (144.6, 149.0)
- added C70 (x2): 100nF, Capacitors_SMD:C_0603, F.Cu at (180.6, 149.0)
- added C70 (x2): 100nF, Capacitors_SMD:C_0603, F.Cu at (162.6, 149.0)
- added C70 (x2): 100nF, Capacitors_SMD:C_0603, F.Cu at (198.6, 149.0)
- added C70 (x2): 100nF, Capacitors_SMD:C_0603, F.Cu at (216.6, 149.0)
- added C70 (x2): 100nF, Capacitors_SMD:C_0603, F.Cu at (108.6, 149.0)
- added C70 (x2): 100nF, Capacitors_SMD:C_0603, F.Cu at (90.6, 149.0)
- added C70 (x2): 100nF, Capacitors_SMD:C_0603, F.Cu at (126.6, 149.0)
- added C71 (x2): 100nF, Capacitors_SMD:C_0603, F.Cu at (143.7, 142.6)
- added C71 (x2): 100nF, Capacitors_SMD:C_0603, F.Cu at (179.7, 142.6)
- added C71 (x2): 100nF, Capacitors_SMD:C_0603, F.Cu at (161.7, 142.6)
- added C71 (x2): 100nF, Capacitors_SMD:C_0603, F.Cu at (197.7, 142.6)
- added C71 (x2): 100nF, Capacitors_SMD:C_0603, F.Cu at (215.7, 142.6)
- added C71 (x2): 100nF, Capacitors_SMD:C_0603, F.Cu at (89.7, 142.6)
- added C71 (x2): 100nF, Capacitors_SMD:C_0603, F.Cu at (107.7, 142.6)
- added C71 (x2): 100nF, Capacitors_SMD:C_0603, F.Cu at (125.7, 142.6)
- added C72 (x2): 10μF, Capacitors_SMD:C_0805, F.Cu at (107.9, 155.1)
- added C72 (x2): 10μF, Capacitors_SMD:C_0805, F.Cu at (161.9, 155.1)
- added C72 (x2): 10μF, Capacitors_SMD:C_0805, F.Cu at (179.9, 155.1)
- added C72 (x2): 10μF, Capacitors_SMD:C_0805, F.Cu at (197.9, 155.1)
- added C72 (x2): 10μF, Capacitors_SMD:C_0805, F.Cu at (215.9, 155.1)
- added C72 (x2): 10μF, Capacitors_SMD:C_0805, F.Cu at (143.9, 155.1)
- added C72 (x2): 10μF, Capacitors_SMD:C_0805, F.Cu at (89.9, 155.1)
- added C72 (x2): 10μF, Capacitors_SMD:C_0805, F.Cu at (125.9, 155.1)
- added C73 (x2): 100μF, Capacitors_SMD:c_elec_8x10, F.Cu at (125.2, 136.2)
- added C73 (x2): 100μF, Capacitors_SMD:c_elec_8x10, F.Cu at (179.2, 136.2)
- added C73 (x2): 100μF, Capacitors_SMD:c_elec_8x10, F.Cu at (161.2, 136.2)
- added C73 (x2): 100μF, Capacitors_SMD:c_elec_8x10, F.Cu at (197.2, 136.2)
- added C73 (x2): 100μF, Capacitors_SMD:c_elec_8x10, F.Cu at (215.2, 136.2)
- added C73 (x2): 100μF, Capacitors_SMD:c_elec_8x10, F.Cu at (89.2, 136.2)
- added C73 (x2): 100μF, Capacitors_SMD:c_elec_8x10, F.Cu at (107.2, 136.2)
- added C73 (x2): 100μF, Capacitors_SMD:c_elec_8x10, F.Cu at (143.2, 136.2)
- added C74 (x2): 100nF, Capacitors_SMD:C_0603, F.Cu at (121.3, 142.6)
- added C74 (x2): 100nF, Capacitors_SMD:C_0603, F.Cu at (175.3, 142.6)
- added C74 (x2): 100nF, Capacitors_SMD:C_0603, F.Cu at (193.3, 142.6)
- added C74 (x2): 100nF, Capacitors_SMD:C_0603, F.Cu at (211.3, 142.6)
- added C74 (x2): 100nF, Capacitors_SMD:C_0603, F.Cu at (229.3, 142.6)
- added C74 (x2): 100nF, Capacitors_SMD:C_0603, F.Cu at (157.3, 142.6)
- added C74 (x2): 100nF, Capacitors_SMD:C_0603, F.Cu at (103.3, 142.6)
- added C74 (x2): 100nF, Capacitors_SMD:C_0603, F.Cu at (139.3, 142.6)
- added P18 (x2): E_MOTOR, Pin_Headers:Pin_Header_Angled_1x04, F.Cu at (118.3, 158.8)
- added P18 (x2): E_MOTOR, Pin_Headers:Pin_Header_Angled_1x04, F.Cu at (190.3, 158.8)
- added P18 (x2): E_MOTOR, Pin_Headers:Pin_Header_Angled_1x04, F.Cu at (172.3, 158.8)
- added P18 (x2): E_MOTOR, Pin_Headers:Pin_Header_Angled_1x04, F.Cu at (208.3, 158.8)
- added P18 (x2): E_MOTOR, Pin_Headers:Pin_Header_Angled_1x04, F.Cu at (226.3, 158.8)
- added P18 (x2): E_MOTOR, Pin_Headers:Pin_Header_Angled_1x04, F.Cu at (154.3, 158.8)
- added P18 (x2): E_MOTOR, Pin_Headers:Pin_Header_Angled_1x04, F.Cu at (100.3, 158.8)
- added P18 (x2): E_MOTOR, Pin_Headers:Pin_Header_Angled_1x04, F.Cu at (136.3, 158.8)
- added R117 (x2): 2.2Ω, Resistors_SMD:R_0603, F.Cu at (133.0, 155.1)
- added R117 (x2): 2.2Ω, Resistors_SMD:R_0603, F.Cu at (187.0, 155.1)
- added R117 (x2): 2.2Ω, Resistors_SMD:R_0603, F.Cu at (169.0, 155.1)
- added R117 (x2): 2.2Ω, Resistors_SMD:R_0603, F.Cu at (205.0, 155.1)
- added R117 (x2): 2.2Ω, Resistors_SMD:R_0603, F.Cu at (223.0, 155.1)
- added R117 (x2): 2.2Ω, Resistors_SMD:R_0603, F.Cu at (115.0, 155.1)
- added R117 (x2): 2.2Ω, Resistors_SMD:R_0603, F.Cu at (151.0, 155.1)
- added R117 (x2): 2.2Ω, Resistors_SMD:R_0603, F.Cu at (97.0, 155.1)
- added R118 (x2): 5.23kΩ, Resistors_SMD:R_0603, F.Cu at (148.6, 153.8)
- added R118 (x2): 5.23kΩ, Resistors_SMD:R_0603, F.Cu at (166.6, 153.8)
- added R118 (x2): 5.23kΩ, Resistors_SMD:R_0603, F.Cu at (184.6, 153.8)
- added R118 (x2): 5.23kΩ, Resistors_SMD:R_0603, F.Cu at (202.6, 153.8)
- added R118 (x2): 5.23kΩ, Resistors_SMD:R_0603, F.Cu at (220.6, 153.8)
- added R118 (x2): 5.23kΩ, Resistors_SMD:R_0603, F.Cu at (112.5, 153.8)
- added R118 (x2): 5.23kΩ, Resistors_SMD:R_0603, F.Cu at (94.5, 153.8)
- added R118 (x2): 5.23kΩ, Resistors_SMD:R_0603, F.Cu at (130.6, 153.8)
- added R119 (x2): 4.75kΩ, Resistors_SMD:R_0603, F.Cu at (146.7, 153.8)
- added R119 (x2): 4.75kΩ, Resistors_SMD:R_0603, F.Cu at (182.7, 153.8)
- added R119 (x2): 4.75kΩ, Resistors_SMD:R_0603, F.Cu at (164.7, 153.8)
- added R119 (x2): 4.75kΩ, Resistors_SMD:R_0603, F.Cu at (200.7, 153.8)
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Connections:
- P19 pad 1: /Stepper Drivers/H_A1 -> /Stepper Drivers/H_A2
- P19 pad 2: /Stepper Drivers/H_A2 -> /Stepper Drivers/H_A1
- P20 pad 1: /Stepper Drivers/X0_A1 -> /Stepper Drivers/X0_A2
- P20 pad 2: /Stepper Drivers/X0_A2 -> /Stepper Drivers/X0_A1
- P21 pad 1: /Stepper Drivers/X1_A1 -> /Stepper Drivers/X1_A2
- P21 pad 2: /Stepper Drivers/X1_A2 -> /Stepper Drivers/X1_A1
- P22 pad 2: Net-(P22-Pad2) -> /Stepper Drivers/Y_A2
- P22 pad 4: Net-(P22-Pad4) -> /Stepper Drivers/Y_B2
- P24 pad 1: /Stepper Drivers/Z0_A1 -> /Stepper Drivers/Z0_A2
- P24 pad 2: /Stepper Drivers/Z0_A2 -> /Stepper Drivers/Z0_A1
- P25 pad 1: /Stepper Drivers/Z1_A1 -> /Stepper Drivers/Z1_A2
- P25 pad 2: /Stepper Drivers/Z1_A2 -> /Stepper Drivers/Z1_A1
- P26 pad 1: /Stepper Drivers/Z2_A1 -> /Stepper Drivers/Z2_A2
- P26 pad 2: /Stepper Drivers/Z2_A2 -> /Stepper Drivers/Z2_A1
Routing:
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- added copper zone on In2.Cu, net /Stepper Drivers/E_A1
- added copper zone on In2.Cu, net /Stepper Drivers/E_A2
- added copper zone on In2.Cu, net /Stepper Drivers/E_B2
Other:
- board text added: "Y"
- board text removed: "Y0"
- board text removed: "Y1"

Commit message: Change associated annotations of X0, X1, Y, and Z0 stepper circuits' components
Parts:
- removed C1, C107, C109, C114, C117, C118, C119, C122, C123, C125, C130, C133, C134, C135, C138, C139, C14, C141, C146, C149, C150, C151, C154, C16, C17, C187, C19, C2, C22, C23, C25, C26, C27, C30, C31, C32, C5, C50, C51, C52, C53, C54, C55, C56, C57, C58, C7, C9: 100nF, Capacitors_SMD:C_0603
- removed C10: 470μF, KiMBo:c_elec_16x16.5
- removed C108, C124, C140: 470nF, Capacitors_SMD:C_0603
- removed C11: 220μF, KiMBo:c_elec_8x10.2
- removed C110, C126, C142, C46, C47: 4.7μF, Capacitors_SMD:C_0603
- removed C111, C127, C143, C6: 22nF, Capacitors_SMD:C_0603
- removed C112, C113, C115, C116, C128, C129, C131, C132, C144, C145, C147, C148, C33: 470pF, Capacitors_SMD:C_0603
- removed C12, C13: 22μF, Capacitors_SMD:C_0805
- removed C120, C136, C152, C34: 10μF, Capacitors_SMD:C_0805
- removed C121, C137, C153: 100μF, Capacitors_SMD:c_elec_8x10
- removed C15, C18, C20: 2.2μF, Capacitors_SMD:C_0805
- removed C188, C189, C190, C191, C192, C193, C194, C195: 4.7nF, Capacitors_SMD:C_0603
- removed C196, C197, C198, C199, C200, C201, C202, C203, C204, C205, C206, C207, C208, C209, C210, C211: 47pF, Capacitors_SMD:C_0603
- removed C21: 4.7μF, Capacitors_SMD:C_0805
- removed C24: 220μF, Capacitors_Tantalum_SMD:TantalC_SizeD_EIA-7343_Reflow
- removed C28, C29: 30pF, Capacitors_SMD:C_0603
- removed C3, C4: 10nF, Capacitors_SMD:C_0603
- removed C35: 1μF, Capacitors_SMD:C_0603
- removed C36, C37, C38, C39: DNP-15pF, Capacitors_SMD:C_0603
- removed C40, C41: 10μF, Capacitors_SMD:C_0603
- removed C42, C43, C44, C45: 18pF, Capacitors_SMD:C_0603
- removed C48, C49: 39nF, Capacitors_SMD:C_0603
- removed the C59 at (113.0, 142.9) (x2)
- removed the C59 at (167.0, 142.9) (x2)
- removed the C59 at (185.0, 142.9) (x2)
- removed the C59 at (203.0, 142.9)
- removed the C59 at (221.0, 142.9) (x2)
- removed the C59 at (149.0, 142.9) (x2)
- removed the C59 at (95.0, 142.9) (x2)
- removed the C59 at (131.0, 142.9) (x2)
- removed the C60 at (153.4, 153.5) (x2)
- removed the C60 at (171.4, 153.5) (x2)
- removed the C60 at (189.4, 153.5) (x2)
- removed the C60 at (207.4, 153.5)
- removed the C60 at (225.4, 153.5) (x2)
- removed the C60 at (99.4, 153.5) (x2)
- removed the C60 at (117.4, 153.5) (x2)
- removed the C60 at (135.4, 153.5) (x2)
- removed the C61 at (120.9, 150.5) (x2)
- removed the C61 at (192.9, 150.5) (x2)
- removed the C61 at (174.9, 150.5) (x2)
- removed the C61 at (210.9, 150.5)
- removed the C61 at (228.9, 150.5) (x2)
- removed the C61 at (156.9, 150.5) (x2)
- removed the C61 at (138.9, 150.5) (x2)
- removed the C61 at (102.9, 150.5) (x2)
- removed the C62 at (97.0, 153.3) (x2)
- removed the C62 at (187.0, 153.3) (x2)
- removed the C62 at (169.0, 153.3) (x2)
- removed the C62 at (205.0, 153.3)
- removed the C62 at (223.0, 153.3) (x2)
- removed the C62 at (115.0, 153.3) (x2)
- removed the C62 at (151.0, 153.3) (x2)
- removed the C62 at (133.0, 153.3) (x2)
- removed the C63 at (101.1, 152.9) (x2)
- removed the C63 at (173.1, 152.9) (x2)
- removed the C63 at (191.1, 152.9) (x2)
- removed the C63 at (209.1, 152.9)
- removed the C63 at (227.1, 152.9) (x2)
- removed the C63 at (155.1, 152.9) (x2)
- removed the C63 at (137.1, 152.9) (x2)
- removed the C63 at (119.1, 152.9) (x2)
- removed the C64 at (157.0, 146.9) (x2)
- removed the C64 at (193.0, 146.9) (x2)
- removed the C64 at (175.0, 146.9) (x2)
- removed the C64 at (211.0, 146.9)
- removed the C64 at (229.0, 146.9) (x2)
- removed the C64 at (103.0, 146.9) (x2)
- removed the C64 at (121.0, 146.9) (x2)
- removed the C64 at (139.0, 146.9) (x2)
- removed the C65 at (144.0, 146.9) (x2)
- removed the C65 at (162.0, 146.9) (x2)
- removed the C65 at (180.0, 146.9) (x2)
- removed the C65 at (198.0, 146.9)
- removed the C65 at (216.0, 146.9) (x2)
- removed the C65 at (108.0, 146.9) (x2)
- removed the C65 at (126.0, 146.9) (x2)
- removed the C65 at (90.0, 146.9) (x2)
- removed the C66 at (138.8, 152.9) (x2)
- removed the C66 at (192.8, 152.9) (x2)
- removed the C66 at (174.8, 152.9) (x2)
- removed the C66 at (210.8, 152.9)
- removed the C66 at (228.8, 152.9) (x2)
- removed the C66 at (120.8, 152.9) (x2)
- removed the C66 at (102.8, 152.9) (x2)
- removed the C66 at (156.8, 152.9) (x2)
- removed the C67 at (154.4, 143.3) (x2)
- removed the C67 at (172.4, 143.3) (x2)
- removed the C67 at (190.4, 143.3) (x2)
- removed the C67 at (208.4, 143.3)
- removed the C67 at (226.4, 143.3) (x2)
- removed the C67 at (118.4, 143.3) (x2)
- removed the C67 at (100.4, 143.3) (x2)
- removed the C67 at (136.4, 143.3) (x2)
- removed the C68 at (92.6, 143.3) (x2)
- removed the C68 at (182.6, 143.3) (x2)
- removed the C68 at (164.6, 143.3) (x2)
- removed the C68 at (200.6, 143.3)
- removed the C68 at (218.6, 143.3) (x2)
- removed the C68 at (128.6, 143.3) (x2)
- removed the C68 at (146.6, 143.3) (x2)
- removed the C68 at (110.6, 143.3) (x2)
- removed the C69 at (156.9, 148.8) (x2)
- removed the C69 at (174.9, 148.8) (x2)
- removed the C69 at (192.9, 148.8) (x2)
- removed the C69 at (210.9, 148.8)
- removed the C69 at (228.9, 148.8) (x2)
- removed the C69 at (120.9, 148.8) (x2)
- removed the C69 at (102.9, 148.8) (x2)
- removed the C69 at (138.9, 148.8) (x2)
- removed the C70 at (144.6, 149.0) (x2)
- removed the C70 at (180.6, 149.0) (x2)
- removed the C70 at (162.6, 149.0) (x2)
- removed the C70 at (198.6, 149.0)
- removed the C70 at (216.6, 149.0) (x2)
- removed the C70 at (108.6, 149.0) (x2)
- removed the C70 at (90.6, 149.0) (x2)
- removed the C70 at (126.6, 149.0) (x2)
- removed the C71 at (143.7, 142.6) (x2)
- removed the C71 at (179.7, 142.6) (x2)
- removed the C71 at (161.7, 142.6) (x2)
- removed the C71 at (197.7, 142.6)
- removed the C71 at (215.7, 142.6) (x2)
- removed the C71 at (89.7, 142.6) (x2)
- removed the C71 at (107.7, 142.6) (x2)
- removed the C71 at (125.7, 142.6) (x2)
- removed the C72 at (107.9, 155.1) (x2)
- removed the C72 at (161.9, 155.1) (x2)
- removed the C72 at (179.9, 155.1) (x2)
- removed the C72 at (197.9, 155.1)
- removed the C72 at (215.9, 155.1) (x2)
- removed the C72 at (143.9, 155.1) (x2)
- removed the C72 at (89.9, 155.1) (x2)
- removed the C72 at (125.9, 155.1) (x2)
- removed the C73 at (125.2, 136.2) (x2)
- removed the C73 at (179.2, 136.2) (x2)
- removed the C73 at (161.2, 136.2) (x2)
- removed the C73 at (197.2, 136.2)
- removed the C73 at (215.2, 136.2) (x2)
- removed the C73 at (89.2, 136.2) (x2)
- removed the C73 at (107.2, 136.2) (x2)
- removed the C73 at (143.2, 136.2) (x2)
- removed the C74 at (121.3, 142.6) (x2)
- removed the C74 at (175.3, 142.6) (x2)
- removed the C74 at (193.3, 142.6) (x2)
- removed the C74 at (211.3, 142.6)
- removed the C74 at (229.3, 142.6) (x2)
- removed the C74 at (157.3, 142.6) (x2)
- removed the C74 at (103.3, 142.6) (x2)
- removed the C74 at (139.3, 142.6) (x2)
- removed C8: 2.2μF, Capacitors_SMD:C_0603
- removed D1, D14, D7, D8: D5V0F1U2S9, KiMBo:SOD-923
- removed D10, D17, D2: TPD1E04U04DPYR, KiMBo:TPD_PX1SON
- removed D11, D19, D22, D23, D26, D27, D29, D3, D31, D33, D4, D5, D6: LED, LEDs:LED_0603
- removed D12: DNP-TLVH431, TO_SOT_Packages_SMD:SOT-23
- removed D13: SK54A-LTP, KiMBo:SK-DO-214AC
- removed D15: SMAZ10, KiMBo:SMA-DO-214AC
- removed D16: SMAJ26A, KiMBo:SK-DO-214AC
- removed D18: SK1545-TP, KiMBo:SK-DO-214AB
- removed D20, D21, D24, D25, D28, D30, D32: MBRA340T3, KiMBo:MBR-DO-214AC
- removed D9: TLVH431, TO_SOT_Packages_SMD:SOT-23
- removed FB1, FB19, FB2, FB21: MPZ1608S102ATA00, KiMBo:Ferrite_Bead_0603
- removed FB10, FB11, FB12, FB13, FB14, FB15, FB16, FB17, FB18, FB20, FB28, FB29, FB3, FB30, FB31, FB32, FB33, FB34, FB4, FB5, FB6, FB7, FB8, FB9: MMZ1608A252BTA00, KiMBo:Ferrite_Bead_0603
- removed FB22, FB23, FB35, FB36: BLM31SN500SN1L, Resistors_SMD:R_1206_HandSoldering
- removed FB24, FB25: BLM15AG102SN1D, Resistors_SMD:R_0402
- removed FB26, FB27: LI0805H151R-10, Resistors_SMD:R_0805
- removed FB37, FB38, FB39, FB40: FBMH4532HM132-T, KiMBo:Ferrite_Bead_1812
- removed FB41, FB42, FB43: CIM21J202NE, Resistors_SMD:R_0805
- removed IC1: 24LC32AT-I/OT, TO_SOT_Packages_SMD:SOT-23-5
- removed L1: 47μH, KiMBo:IHLP_Inductor
- removed OSC1: ASDMB, KiMBo:Crystal_SMD_ASDMB_4Pads
- removed the P18 at (118.3, 158.8) (x2)
- removed the P18 at (190.3, 158.8) (x2)
- removed the P18 at (172.3, 158.8) (x2)
- removed the P18 at (208.3, 158.8)
- removed the P18 at (226.3, 158.8) (x2)
- removed the P18 at (154.3, 158.8) (x2)
- removed the P18 at (100.3, 158.8) (x2)
- removed the P18 at (136.3, 158.8) (x2)
- removed P19: H_MOTOR, Pin_Headers:Pin_Header_Angled_1x04
- removed P25: Z1_MOTOR, Pin_Headers:Pin_Header_Angled_1x04
- removed P26: Z2_MOTOR, Pin_Headers:Pin_Header_Angled_1x04
- removed Q1, Q11, Q12, Q15, Q17, Q19, Q5, Q7, Q8: 2N7002, TO_SOT_Packages_SMD:SOT-23
- removed Q10, Q13, Q14, Q16, Q18, Q20, Q9: DMP3098L-7, TO_SOT_Packages_SMD:SOT-23
- removed Q2: MMBT2907, TO_SOT_Packages_SMD:SOT-23
- removed Q3: DNP-MMBT2907, TO_SOT_Packages_SMD:SOT-23
- removed Q4, Q6: IPD90P03P4-04, TO_SOT_Packages_SMD:TO-252-2Lead
- removed R1, R2, R3, R4: 1kΩ, Resistors_SMD:R_0603
- removed R10, R11, R141, R147, R154, R20, R26, R27, R6: 4.75kΩ, Resistors_SMD:R_0603
- removed R100, R220, R57, R58, R59, R60, R61, R62, R63, R64, R65, R66, R96, R98: 100Ω, Resistors_SMD:R_0603
- removed R101, R102, R103, R104, R105, R106, R107, R108, R109, R110, R111, R112, R113, R114, R115, R116, R12, R122, R123, R124, R13, R130, R131, R132, R138, R144, R150, R151, R157, R158, R159, R165, R171, R173, R174, R175, R180, R181, R182, R183, R184, R185, R192, R193, R194, R195, R196, R197, R203, R204, R205, R209, R210, R211, R215, R216, R217, R92, R94, R97, R99: 4.7kΩ, Resistors_SMD:R_0603
- removed the R117 at (133.0, 155.1) (x2)
- removed the R117 at (187.0, 155.1) (x2)
- removed the R117 at (169.0, 155.1) (x2)
- removed the R117 at (205.0, 155.1)
- removed the R117 at (223.0, 155.1) (x2)
- removed the R117 at (115.0, 155.1) (x2)
- removed the R117 at (151.0, 155.1) (x2)
- removed the R117 at (97.0, 155.1) (x2)
- removed the R118 at (148.6, 153.8) (x2)
- removed the R118 at (166.6, 153.8) (x2)
- removed the R118 at (184.6, 153.8) (x2)
- removed the R118 at (202.6, 153.8)
- removed the R118 at (220.6, 153.8) (x2)
- removed the R118 at (112.5, 153.8) (x2)
- removed the R118 at (94.5, 153.8) (x2)
- removed the R118 at (130.6, 153.8) (x2)
- removed the R119 at (146.7, 153.8) (x2)
- removed the R119 at (182.7, 153.8) (x2)
- removed the R119 at (164.7, 153.8) (x2)
- removed the R119 at (200.7, 153.8)
- removed the R119 at (218.7, 153.8) (x2)
- removed the R119 at (128.7, 153.8) (x2)
- removed the R119 at (110.7, 153.8) (x2)
- removed the R119 at (92.7, 153.8) (x2)
- removed the R120 at (107.7, 144.6) (x2)
- removed the R120 at (179.7, 144.6) (x2)
- removed the R120 at (161.7, 144.6) (x2)
- removed the R120 at (197.7, 144.6)
- removed the R120 at (215.7, 144.6) (x2)
- removed the R120 at (125.7, 144.6) (x2)
- removed the R120 at (89.7, 144.6) (x2)
- removed the R120 at (143.7, 144.6) (x2)
- removed the R121 at (121.3, 144.6) (x2)
- removed the R121 at (175.3, 144.6) (x2)
- removed the R121 at (193.3, 144.6) (x2)
- removed the R121 at (211.3, 144.6)
- removed the R121 at (229.3, 144.6) (x2)
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Connections:
- P22 pad 1: /Stepper Drivers/Y_A1 -> /Stepper Drivers/Y_A2
- P22 pad 2: /Stepper Drivers/Y_A2 -> /Stepper Drivers/Y_A1
- P22 pad 3: /Stepper Drivers/Y_B1 -> /Stepper Drivers/Y_B2
- P22 pad 4: /Stepper Drivers/Y_B2 -> /Stepper Drivers/Y_B1
Routing:
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- added copper zone on F.Cu, net /Stepper Drivers/X0_A1
- added copper zone on In2.Cu, net /Stepper Drivers/X0_A1
- added copper zone on F.Cu, net /Stepper Drivers/X0_A2
- added copper zone on In2.Cu, net /Stepper Drivers/X0_A2
- added copper zone on F.Cu, net /Stepper Drivers/X0_B1
- added copper zone on In2.Cu, net /Stepper Drivers/X0_B1
- added copper zone on F.Cu, net /Stepper Drivers/X0_B2
- added copper zone on In2.Cu, net /Stepper Drivers/X0_B2
- added copper zone on F.Cu, net /Stepper Drivers/X1_A1
- added copper zone on In2.Cu, net /Stepper Drivers/X1_A1
- added copper zone on F.Cu, net /Stepper Drivers/X1_A2
- added copper zone on In2.Cu, net /Stepper Drivers/X1_A2
- added copper zone on F.Cu, net /Stepper Drivers/X1_B1
- added copper zone on In2.Cu, net /Stepper Drivers/X1_B1
- added copper zone on F.Cu, net /Stepper Drivers/X1_B2
- added copper zone on In2.Cu, net /Stepper Drivers/X1_B2
- added copper zone on F.Cu, net /Stepper Drivers/Y_A1
- added copper zone on In2.Cu, net /Stepper Drivers/Y_A1
- added copper zone on F.Cu, net /Stepper Drivers/Y_A2
- added copper zone on In2.Cu, net /Stepper Drivers/Y_A2
- added copper zone on F.Cu, net /Stepper Drivers/Y_B1
- added copper zone on In2.Cu, net /Stepper Drivers/Y_B1
- added copper zone on F.Cu, net /Stepper Drivers/Y_B2
- added copper zone on In2.Cu, net /Stepper Drivers/Y_B2
- added copper zone on F.Cu, net /Stepper Drivers/Z0_A1
- added copper zone on In2.Cu, net /Stepper Drivers/Z0_A1
- added copper zone on F.Cu, net /Stepper Drivers/Z0_A2
- added copper zone on In2.Cu, net /Stepper Drivers/Z0_A2
- added copper zone on F.Cu, net /Stepper Drivers/Z0_B1
- added copper zone on In2.Cu, net /Stepper Drivers/Z0_B1
- added copper zone on F.Cu, net /Stepper Drivers/Z0_B2
- added copper zone on In2.Cu, net /Stepper Drivers/Z0_B2
