File: KiMBo/fan.sch (KiCad schematic (older format))
At the start: 36 parts, among them Q14 2N7002, Q15 DMP3098L-7, Q16 2N7002, Q17 DMP3098L-7, Q18 2N7002, Q19 DMP3098L-7

Commit message: Leave SPI0 free for a display, reassign pins so SPI1 is available
Fix some typos/errors
Parts:
- renumbered Q14 to Q15, Q15 to Q16, Q16 to Q17, Q17 to Q18, Q18 to Q19, Q19 to Q20, R219 to R221, R220 to R222, R221 to R223, R222 to R224, R223 to R225, R224 to R226, R225 to R227, R226 to R228, R227 to R229, R228 to R230, R229 to R231, R230 to R232, R231 to R233, R232 to R234, R233 to R235, R234 to R236, R235 to R237, R236 to R238
Changed lines of the file:
@@
 E_FAN
 $Comp
-L +24V #PWR0278
+L +24V #PWR0277
 U 1 1 5B5EFE55
 P 4800 4500
-F 0 "#PWR0278" H 4800 4350 50  0001 C CNN
+F 0 "#PWR0277" H 4800 4350 50  0001 C CNN
 F 1 "+24V" H 4815 4673 50  0000 C CNN
 F 2 "" H 4800 4500 50  0000 C CNN
@@
 $EndComp
 $Comp
-L GND #PWR0279
+L GND #PWR0278
 U 1 1 5B5EFE5B
 P 4200 6000
-F 0 "#PWR0279" H 4200 5750 50  0001 C CNN
+F 0 "#PWR0278" H 4200 5750 50  0001 C CNN
 F 1 "GND" H 4205 5827 50  0000 C CNN
 F 2 "" H 4200 6000 50  0000 C CNN
@@
 $EndComp
 $Comp
-L R R219
+L R R221
 U 1 1 5B5EFE68
 P 3700 5600
-F 0 "R219" V 3600 5600 50  0000 C CNN
+F 0 "R221" V 3600 5600 50  0000 C CNN
 F 1 "10Ω" V 3800 5600 50  0000 C CNN
 F 2 "" V 3630 5600 50  0001 C CNN
@@
 $EndComp
 $Comp
-L 2N7002P,215 Q14
+L 2N7002P,215 Q15
 U 1 1 5B5EFE6F
 P 4100 5600
-F 0 "Q14" H 4050 5750 40  0000 L CNN
+F 0 "Q15" H 4050 5750 40  0000 L CNN
 F 1 "2N7002" H 3850 5475 40  0000 L CNN
 F 2 "" H 3970 5702 29  0001 C CNN
@@
 $EndComp
 $Comp
-L R R223
+L R R225
 U 1 1 5B5EFE7E
 P 5150 5400
-F 0 "R223" H 5220 5446 50  0000 L CNN
+F 0 "R225" H 5220 5446 50  0000 L CNN
 F 1 "4.7kΩ" H 5220 5355 50  0000 L CNN
 F 2 "" V 5080 5400 50  0001 C CNN
@@
 $EndComp
 $Comp
-L R R221
+L R R223
 U 1 1 5B5EFE85
 P 4200 4750
-F 0 "R221" H 4270 4796 50  0000 L CNN
+F 0 "R223" H 4270 4796 50  0000 L CNN
 F 1 "4.7kΩ" H 4270 4705 50  0000 L CNN
 F 2 "" V 4130 4750 50  0001 C CNN
@@
 $EndComp
 $Comp
-L R R222
+L R R224
 U 1 1 5B5EFE8C
 P 4200 5150
-F 0 "R222" H 4270 5196 50  0000 L CNN
+F 0 "R224" H 4270 5196 50  0000 L CNN
 F 1 "4.7kΩ" H 4270 5105 50  0000 L CNN
 F 2 "" V 4130 5150 50  0001 C CNN
@@
 $EndComp
 $Comp
-L R R220
+L R R222
 U 1 1 5B5EFE93
 P 3800 5950
-F 0 "R220" V 3700 5950 50  0000 C CNN
+F 0 "R222" V 3700 5950 50  0000 C CNN
 F 1 "4.7kΩ" V 3900 5950 50  0000 C CNN
 F 2 "" V 3730 5950 50  0001 C CNN
@@
 $EndComp
 $Comp
-L R R224
+L R R226
 U 1 1 5B5EFE9A
 P 5700 5600
-F 0 "R224" H 5770 5646 50  0000 L CNN
+F 0 "R226" H 5770 5646 50  0000 L CNN
 F 1 "4.7kΩ" H 5770 5555 50  0000 L CNN
 F 2 "" V 5630 5600 50  0001 C CNN
@@
 	4200 4550 5700 4550
 $Comp
-L DMP3098L-7 Q15
+L DMP3098L-7 Q16
 U 1 1 5B5EFEC7
 P 4700 4950
-F 0 "Q15" H 4900 5100 50  0000 L CNN
+F 0 "Q16" H 4900 5100 50  0000 L CNN
 F 1 "DMP3098L-7" H 4900 5000 50  0000 L CNN
 F 2 "" H 4950 5025 50  0001 L CNN
@@
 H_FAN
 $Comp
-L +24V #PWR0280
+L +24V #PWR0279
 U 1 1 5B5F23AA
 P 8100 4500
-F 0 "#PWR0280" H 8100 4350 50  0001 C CNN
+F 0 "#PWR0279" H 8100 4350 50  0001 C CNN
 F 1 "+24V" H 8115 4673 50  0000 C CNN
 F 2 "" H 8100 4500 50  0000 C CNN
@@
 $EndComp
 $Comp
-L GND #PWR0281
+L GND #PWR0280
 U 1 1 5B5F23B0
 P 7500 6000
-F 0 "#PWR0281" H 7500 5750 50  0001 C CNN
+F 0 "#PWR0280" H 7500 5750 50  0001 C CNN
 F 1 "GND" H 7505 5827 50  0000 C CNN
 F 2 "" H 7500 6000 50  0000 C CNN
@@
 $EndComp
 $Comp
-L R R225
+L R R227
 U 1 1 5B5F23BD
 P 7000 5600
-F 0 "R225" V 6900 5600 50  0000 C CNN
+F 0 "R227" V 6900 5600 50  0000 C CNN
 F 1 "10Ω" V 7100 5600 50  0000 C CNN
 F 2 "" V 6930 5600 50  0001 C CNN
@@
 $EndComp
 $Comp
-L R R229
+L R R231
 U 1 1 5B5F23D2
 P 8450 5400
-F 0 "R229" H 8520 5446 50  0000 L CNN
+F 0 "R231" H 8520 5446 50  0000 L CNN
 F 1 "4.7kΩ" H 8520 5355 50  0000 L CNN
 F 2 "" V 8380 5400 50  0001 C CNN
@@
 $EndComp
 $Comp
-L R R227
+L R R229
 U 1 1 5B5F23D9
 P 7500 4750
-F 0 "R227" H 7570 4796 50  0000 L CNN
+F 0 "R229" H 7570 4796 50  0000 L CNN
 F 1 "4.7kΩ" H 7570 4705 50  0000 L CNN
 F 2 "" V 7430 4750 50  0001 C CNN
@@
 $EndComp
 $Comp
-L R R228
+L R R230
 U 1 1 5B5F23E0
 P 7500 5150
-F 0 "R228" H 7570 5196 50  0000 L CNN
+F 0 "R230" H 7570 5196 50  0000 L CNN
 F 1 "4.7kΩ" H 7570 5105 50  0000 L CNN
 F 2 "" V 7430 5150 50  0001 C CNN
@@
 $EndComp
 $Comp
-L R R226
+L R R228
 U 1 1 5B5F23E7
 P 7100 5950
-F 0 "R226" V 7000 5950 50  0000 C CNN
+F 0 "R228" V 7000 5950 50  0000 C CNN
 F 1 "4.7kΩ" V 7200 5950 50  0000 C CNN
 F 2 "" V 7030 5950 50  0001 C CNN
@@
 $EndComp
 $Comp
-L R R230
+L R R232
 U 1 1 5B5F23EE
 P 9000 5600
-F 0 "R230" H 9070 5646 50  0000 L CNN
+F 0 "R232" H 9070 5646 50  0000 L CNN
 F 1 "4.7kΩ" H 9070 5555 50  0000 L CNN
 F 2 "" V 8930 5600 50  0001 C CNN
@@
 	7500 4550 9000 4550
 $Comp
-L DMP3098L-7 Q17
+L DMP3098L-7 Q18
 U 1 1 5B5F241B
 P 8000 4950
-F 0 "Q17" H 8200 5100 50  0000 L CNN
+F 0 "Q18" H 8200 5100 50  0000 L CNN
 F 1 "DMP3098L-7" H 8200 5000 50  0000 L CNN
 F 2 "" H 8250 5025 50  0001 L CNN
@@
 CASE_FAN
 $Comp
-L +24V #PWR0282
+L +24V #PWR0281
 U 1 1 5B5F2995
 P 11400 4500
-F 0 "#PWR0282" H 11400 4350 50  0001 C CNN
+F 0 "#PWR0281" H 11400 4350 50  0001 C CNN
 F 1 "+24V" H 11415 4673 50  0000 C CNN
 F 2 "" H 11400 4500 50  0000 C CNN
@@
 $EndComp
 $Comp
-L GND #PWR0283
+L GND #PWR0282
 U 1 1 5B5F299B
 P 10800 6000
-F 0 "#PWR0283" H 10800 5750 50  0001 C CNN
+F 0 "#PWR0282" H 10800 5750 50  0001 C CNN
 F 1 "GND" H 10805 5827 50  0000 C CNN
 F 2 "" H 10800 6000 50  0000 C CNN
@@
 $EndComp
 $Comp
-L R R231
+L R R233
 U 1 1 5B5F29A8
 P 10300 5600
-F 0 "R231" V 10200 5600 50  0000 C CNN
+F 0 "R233" V 10200 5600 50  0000 C CNN
 F 1 "10Ω" V 10400 5600 50  0000 C CNN
 F 2 "" V 10230 5600 50  0001 C CNN
@@
 $EndComp
 $Comp
-L R R235
+L R R237
 U 1 1 5B5F29BD
 P 11750 5400
-F 0 "R235" H 11820 5446 50  0000 L CNN
+F 0 "R237" H 11820 5446 50  0000 L CNN
 F 1 "4.7kΩ" H 11820 5355 50  0000 L CNN
 F 2 "" V 11680 5400 50  0001 C CNN
@@
 $EndComp
 $Comp
-L R R233
+L R R235
 U 1 1 5B5F29C4
 P 10800 4750
-F 0 "R233" H 10870 4796 50  0000 L CNN
+F 0 "R235" H 10870 4796 50  0000 L CNN
 F 1 "4.7kΩ" H 10870 4705 50  0000 L CNN
 F 2 "" V 10730 4750 50  0001 C CNN
@@
 $EndComp
 $Comp
-L R R234
+L R R236
 U 1 1 5B5F29CB
 P 10800 5150
-F 0 "R234" H 10870 5196 50  0000 L CNN
+F 0 "R236" H 10870 5196 50  0000 L CNN
 F 1 "4.7kΩ" H 10870 5105 50  0000 L CNN
 F 2 "" V 10730 5150 50  0001 C CNN
@@
 $EndComp
 $Comp
-L R R232
+L R R234
 U 1 1 5B5F29D2
 P 10400 5950
-F 0 "R232" V 10300 5950 50  0000 C CNN
+F 0 "R234" V 10300 5950 50  0000 C CNN
 F 1 "4.7kΩ" V 10500 5950 50  0000 C CNN
 F 2 "" V 10330 5950 50  0001 C CNN
@@
 $EndComp
 $Comp
-L R R236
+L R R238
 U 1 1 5B5F29D9
 P 12300 5600
-F 0 "R236" H 12370 5646 50  0000 L CNN
+F 0 "R238" H 12370 5646 50  0000 L CNN
 F 1 "4.7kΩ" H 12370 5555 50  0000 L CNN
 F 2 "" V 12230 5600 50  0001 C CNN
@@
 	10800 4550 12300 4550
 $Comp
-L DMP3098L-7 Q19
+L DMP3098L-7 Q20
 U 1 1 5B5F2A06
 P 11300 4950
-F 0 "Q19" H 11500 5100 50  0000 L CNN
+F 0 "Q20" H 11500 5100 50  0000 L CNN
 F 1 "DMP3098L-7" H 11500 5000 50  0000 L CNN
 F 2 "" H 11550 5025 50  0001 L CNN
@@
 $EndComp
 $Comp
-L 2N7002P,215 Q16
+L 2N7002P,215 Q17
 U 1 1 5B5FA7B8
 P 7400 5600
-F 0 "Q16" H 7350 5750 40  0000 L CNN
+F 0 "Q17" H 7350 5750 40  0000 L CNN
 F 1 "2N7002" H 7150 5475 40  0000 L CNN
 F 2 "" H 7270 5702 29  0001 C CNN
@@
 $EndComp
 $Comp
-L 2N7002P,215 Q18
+L 2N7002P,215 Q19
 U 1 1 5B5FA86F
 P 10700 5600
-F 0 "Q18" H 10650 5750 40  0000 L CNN
+F 0 "Q19" H 10650 5750 40  0000 L CNN
 F 1 "2N7002" H 10450 5475 40  0000 L CNN
 F 2 "" H 10570 5702 29  0001 C CNN

Commit message: Use fixed 5V LM2592HV Buck, include SPI0 header for LCD
Parts:
- renumbered C219 to C216, C220 to C217, C221 to C218, FB38 to FB43, FB39 to FB44, FB40 to FB45, R221 to R218, R222 to R219, R223 to R220, R224 to R221, R225 to R222, R226 to R223, R227 to R224, R228 to R225, R229 to R226, R230 to R227, R231 to R228, R232 to R229, R233 to R230, R234 to R231, R235 to R232, R236 to R233, R237 to R234, R238 to R235
Changed lines of the file:
@@
 E_FAN
 $Comp
-L +24V #PWR0277
+L +24V #PWR0272
 U 1 1 5B5EFE55
 P 4800 4500
-F 0 "#PWR0277" H 4800 4350 50  0001 C CNN
+F 0 "#PWR0272" H 4800 4350 50  0001 C CNN
 F 1 "+24V" H 4815 4673 50  0000 C CNN
 F 2 "" H 4800 4500 50  0000 C CNN
@@
 $EndComp
 $Comp
-L GND #PWR0278
+L GND #PWR0273
 U 1 1 5B5EFE5B
 P 4200 6000
-F 0 "#PWR0278" H 4200 5750 50  0001 C CNN
+F 0 "#PWR0273" H 4200 5750 50  0001 C CNN
 F 1 "GND" H 4205 5827 50  0000 C CNN
 F 2 "" H 4200 6000 50  0000 C CNN
@@
 $EndComp
 $Comp
-L R R221
+L R R218
 U 1 1 5B5EFE68
 P 3700 5600
-F 0 "R221" V 3600 5600 50  0000 C CNN
+F 0 "R218" V 3600 5600 50  0000 C CNN
 F 1 "10Ω" V 3800 5600 50  0000 C CNN
 F 2 "" V 3630 5600 50  0001 C CNN
@@
 $EndComp
 $Comp
-L R R225
+L R R222
 U 1 1 5B5EFE7E
 P 5150 5400
-F 0 "R225" H 5220 5446 50  0000 L CNN
+F 0 "R222" H 5220 5446 50  0000 L CNN
 F 1 "4.7kΩ" H 5220 5355 50  0000 L CNN
 F 2 "" V 5080 5400 50  0001 C CNN
@@
 $EndComp
 $Comp
-L R R223
+L R R220
 U 1 1 5B5EFE85
 P 4200 4750
-F 0 "R223" H 4270 4796 50  0000 L CNN
+F 0 "R220" H 4270 4796 50  0000 L CNN
 F 1 "4.7kΩ" H 4270 4705 50  0000 L CNN
 F 2 "" V 4130 4750 50  0001 C CNN
@@
 $EndComp
 $Comp
-L R R224
+L R R221
 U 1 1 5B5EFE8C
 P 4200 5150
-F 0 "R224" H 4270 5196 50  0000 L CNN
+F 0 "R221" H 4270 5196 50  0000 L CNN
 F 1 "4.7kΩ" H 4270 5105 50  0000 L CNN
 F 2 "" V 4130 5150 50  0001 C CNN
@@
 $EndComp
 $Comp
-L R R222
+L R R219
 U 1 1 5B5EFE93
 P 3800 5950
-F 0 "R222" V 3700 5950 50  0000 C CNN
+F 0 "R219" V 3700 5950 50  0000 C CNN
 F 1 "4.7kΩ" V 3900 5950 50  0000 C CNN
 F 2 "" V 3730 5950 50  0001 C CNN
@@
 $EndComp
 $Comp
-L R R226
+L R R223
 U 1 1 5B5EFE9A
 P 5700 5600
-F 0 "R226" H 5770 5646 50  0000 L CNN
+F 0 "R223" H 5770 5646 50  0000 L CNN
 F 1 "4.7kΩ" H 5770 5555 50  0000 L CNN
 F 2 "" V 5630 5600 50  0001 C CNN
@@
 $EndComp
 $Comp
-L C C219
+L C C216
 U 1 1 5B5EFEA1
 P 5700 4850
-F 0 "C219" H 5815 4896 50  0000 L CNN
+F 0 "C216" H 5815 4896 50  0000 L CNN
 F 1 "4.7nF" H 5815 4805 50  0000 L CNN
 F 2 "Capacitors_SMD:C_0402" H 5738 4700 50  0001 C CNN
@@
 $EndComp
 $Comp
-L INDUCTOR_Small FB38
+L INDUCTOR_Small FB43
 U 1 1 5B5F15E2
 P 5300 5200
-F 0 "FB38" V 5485 5200 50  0000 C CNN
+F 0 "FB43" V 5485 5200 50  0000 C CNN
 F 1 "CIM21J202NE" V 5394 5200 50  0000 C CNN
 F 2 "" H 5300 5200 50  0001 C CNN
@@
 H_FAN
 $Comp
-L +24V #PWR0279
+L +24V #PWR0274
 U 1 1 5B5F23AA
 P 8100 4500
-F 0 "#PWR0279" H 8100 4350 50  0001 C CNN
+F 0 "#PWR0274" H 8100 4350 50  0001 C CNN
 F 1 "+24V" H 8115 4673 50  0000 C CNN
 F 2 "" H 8100 4500 50  0000 C CNN
@@
 $EndComp
 $Comp
-L GND #PWR0280
+L GND #PWR0275
 U 1 1 5B5F23B0
 P 7500 6000
-F 0 "#PWR0280" H 7500 5750 50  0001 C CNN
+F 0 "#PWR0275" H 7500 5750 50  0001 C CNN
 F 1 "GND" H 7505 5827 50  0000 C CNN
 F 2 "" H 7500 6000 50  0000 C CNN
@@
 $EndComp
 $Comp
-L R R227
+L R R224
 U 1 1 5B5F23BD
 P 7000 5600
-F 0 "R227" V 6900 5600 50  0000 C CNN
+F 0 "R224" V 6900 5600 50  0000 C CNN
 F 1 "10Ω" V 7100 5600 50  0000 C CNN
 F 2 "" V 6930 5600 50  0001 C CNN
@@
 $EndComp
 $Comp
-L R R231
+L R R228
 U 1 1 5B5F23D2
 P 8450 5400
-F 0 "R231" H 8520 5446 50  0000 L CNN
+F 0 "R228" H 8520 5446 50  0000 L CNN
 F 1 "4.7kΩ" H 8520 5355 50  0000 L CNN
 F 2 "" V 8380 5400 50  0001 C CNN
@@
 $EndComp
 $Comp
-L R R229
+L R R226
 U 1 1 5B5F23D9
 P 7500 4750
-F 0 "R229" H 7570 4796 50  0000 L CNN
+F 0 "R226" H 7570 4796 50  0000 L CNN
 F 1 "4.7kΩ" H 7570 4705 50  0000 L CNN
 F 2 "" V 7430 4750 50  0001 C CNN
@@
 $EndComp
 $Comp
-L R R230
+L R R227
 U 1 1 5B5F23E0
 P 7500 5150
-F 0 "R230" H 7570 5196 50  0000 L CNN
+F 0 "R227" H 7570 5196 50  0000 L CNN
 F 1 "4.7kΩ" H 7570 5105 50  0000 L CNN
 F 2 "" V 7430 5150 50  0001 C CNN
@@
 $EndComp
 $Comp
-L R R228
+L R R225
 U 1 1 5B5F23E7
 P 7100 5950
-F 0 "R228" V 7000 5950 50  0000 C CNN
+F 0 "R225" V 7000 5950 50  0000 C CNN
 F 1 "4.7kΩ" V 7200 5950 50  0000 C CNN
 F 2 "" V 7030 5950 50  0001 C CNN
@@
 $EndComp
 $Comp
-L R R232
+L R R229
 U 1 1 5B5F23EE
 P 9000 5600
-F 0 "R232" H 9070 5646 50  0000 L CNN
+F 0 "R229" H 9070 5646 50  0000 L CNN
 F 1 "4.7kΩ" H 9070 5555 50  0000 L CNN
 F 2 "" V 8930 5600 50  0001 C CNN
@@
 $EndComp
 $Comp
-L C C220
+L C C217
 U 1 1 5B5F23F5
 P 9000 4850
-F 0 "C220" H 9115 4896 50  0000 L CNN
+F 0 "C217" H 9115 4896 50  0000 L CNN
 F 1 "4.7nF" H 9115 4805 50  0000 L CNN
 F 2 "Capacitors_SMD:C_0402" H 9038 4700 50  0001 C CNN
@@
 $EndComp
 $Comp
-L INDUCTOR_Small FB39
+L INDUCTOR_Small FB44
 U 1 1 5B5F2422
 P 8600 5200
-F 0 "FB39" V 8785 5200 50  0000 C CNN
+F 0 "FB44" V 8785 5200 50  0000 C CNN
 F 1 "CIM21J202NE" V 8694 5200 50  0000 C CNN
 F 2 "" H 8600 5200 50  0001 C CNN
@@
 CASE_FAN
 $Comp
-L +24V #PWR0281
+L +24V #PWR0276
 U 1 1 5B5F2995
 P 11400 4500
-F 0 "#PWR0281" H 11400 4350 50  0001 C CNN
+F 0 "#PWR0276" H 11400 4350 50  0001 C CNN
 F 1 "+24V" H 11415 4673 50  0000 C CNN
 F 2 "" H 11400 4500 50  0000 C CNN
@@
 $EndComp
 $Comp
-L GND #PWR0282
+L GND #PWR0277
 U 1 1 5B5F299B
 P 10800 6000
-F 0 "#PWR0282" H 10800 5750 50  0001 C CNN
+F 0 "#PWR0277" H 10800 5750 50  0001 C CNN
 F 1 "GND" H 10805 5827 50  0000 C CNN
 F 2 "" H 10800 6000 50  0000 C CNN
@@
 $EndComp
 $Comp
-L R R233
+L R R230
 U 1 1 5B5F29A8
 P 10300 5600
-F 0 "R233" V 10200 5600 50  0000 C CNN
+F 0 "R230" V 10200 5600 50  0000 C CNN
 F 1 "10Ω" V 10400 5600 50  0000 C CNN
 F 2 "" V 10230 5600 50  0001 C CNN
@@
 $EndComp
 $Comp
-L R R237
+L R R234
 U 1 1 5B5F29BD
 P 11750 5400
-F 0 "R237" H 11820 5446 50  0000 L CNN
+F 0 "R234" H 11820 5446 50  0000 L CNN
 F 1 "4.7kΩ" H 11820 5355 50  0000 L CNN
 F 2 "" V 11680 5400 50  0001 C CNN
@@
 $EndComp
 $Comp
-L R R235
+L R R232
 U 1 1 5B5F29C4
 P 10800 4750
-F 0 "R235" H 10870 4796 50  0000 L CNN
+F 0 "R232" H 10870 4796 50  0000 L CNN
 F 1 "4.7kΩ" H 10870 4705 50  0000 L CNN
 F 2 "" V 10730 4750 50  0001 C CNN
@@
 $EndComp
 $Comp
-L R R236
+L R R233
 U 1 1 5B5F29CB
 P 10800 5150
-F 0 "R236" H 10870 5196 50  0000 L CNN
+F 0 "R233" H 10870 5196 50  0000 L CNN
 F 1 "4.7kΩ" H 10870 5105 50  0000 L CNN
 F 2 "" V 10730 5150 50  0001 C CNN
@@
 $EndComp
 $Comp
-L R R234
+L R R231
 U 1 1 5B5F29D2
 P 10400 5950
-F 0 "R234" V 10300 5950 50  0000 C CNN
+F 0 "R231" V 10300 5950 50  0000 C CNN
 F 1 "4.7kΩ" V 10500 5950 50  0000 C CNN
 F 2 "" V 10330 5950 50  0001 C CNN
@@
 $EndComp
 $Comp
-L R R238
+L R R235
 U 1 1 5B5F29D9
 P 12300 5600
-F 0 "R238" H 12370 5646 50  0000 L CNN
+F 0 "R235" H 12370 5646 50  0000 L CNN
 F 1 "4.7kΩ" H 12370 5555 50  0000 L CNN
 F 2 "" V 12230 5600 50  0001 C CNN
@@
 $EndComp
 $Comp
-L C C221
+L C C218
 U 1 1 5B5F29E0
 P 12300 4850
-F 0 "C221" H 12415 4896 50  0000 L CNN
+F 0 "C218" H 12415 4896 50  0000 L CNN
 F 1 "4.7nF" H 12415 4805 50  0000 L CNN
 F 2 "Capacitors_SMD:C_0402" H 12338 4700 50  0001 C CNN
@@
 $EndComp
 $Comp
-L INDUCTOR_Small FB40
+L INDUCTOR_Small FB45
 U 1 1 5B5F2A0D
 P 11900 5200
-F 0 "FB40" V 12085 5200 50  0000 C CNN
+F 0 "FB45" V 12085 5200 50  0000 C CNN
 F 1 "CIM21J202NE" V 11994 5200 50  0000 C CNN
 F 2 "" H 11900 5200 50  0001 C CNN

Commit message: Assocate more footprints
Parts:
- C216, C217, C218: footprint Capacitors_SMD:C_0402 -> Capacitors_SMD:C_0603
- D28: renamed from D27; footprint (none) -> LEDs:LED_0603
- D30: renamed from D29; footprint (none) -> LEDs:LED_0603
- D32: renamed from D31; footprint (none) -> LEDs:LED_0603
- FB43, FB44, FB45: footprint (none) -> Resistors_SMD:R_0805
- R218, R219, R220, R221, R222, R223, R224, R225, R226, R227, R228, R229, R230, R231, R232, R233, R234, R235: footprint (none) -> Resistors_SMD:R_0603
- renumbered D26 to D27, D28 to D29, D30 to D31
Changed lines of the file:
@@
 $EndComp
 $Comp
-L D_Schottky D26
+L D_Schottky D27
 U 1 1 5B5EFE61
 P 4800 5550
-F 0 "D26" V 4700 5400 50  0000 L CNN
+F 0 "D27" V 4700 5400 50  0000 L CNN
 F 1 "MBRA340T3" V 4950 5100 50  0000 L CNN
 F 2 "" H 4800 5550 50  0001 C CNN
@@
 F 0 "R218" V 3600 5600 50  0000 C CNN
 F 1 "10Ω" V 3800 5600 50  0000 C CNN
-F 2 "" V 3630 5600 50  0001 C CNN
+F 2 "Resistors_SMD:R_0603" V 3630 5600 50  0001 C CNN
 F 3 "" H 3700 5600 50  0000 C CNN
 	1    3700 5600
@@
 $EndComp
 $Comp
-L LED_Short D27
+L LED_Short D28
 U 1 1 5B5EFE77
 P 5150 5750
-F 0 "D27" V 5196 5642 50  0000 R CNN
+F 0 "D28" V 5196 5642 50  0000 R CNN
 F 1 "LED" V 5105 5642 50  0000 R CNN
-F 2 "" H 5150 5750 50  0001 C CNN
+F 2 "LEDs:LED_0603" H 5150 5750 50  0001 C CNN
 F 3 "" H 5150 5750 50  0000 C CNN
 	1    5150 5750
@@
 F 0 "R222" H 5220 5446 50  0000 L CNN
 F 1 "4.7kΩ" H 5220 5355 50  0000 L CNN
-F 2 "" V 5080 5400 50  0001 C CNN
+F 2 "Resistors_SMD:R_0603" V 5080 5400 50  0001 C CNN
 F 3 "" H 5150 5400 50  0000 C CNN
 	1    5150 5400
@@
 F 0 "R220" H 4270 4796 50  0000 L CNN
 F 1 "4.7kΩ" H 4270 4705 50  0000 L CNN
-F 2 "" V 4130 4750 50  0001 C CNN
+F 2 "Resistors_SMD:R_0603" V 4130 4750 50  0001 C CNN
 F 3 "" H 4200 4750 50  0000 C CNN
 	1    4200 4750
@@
 F 0 "R221" H 4270 5196 50  0000 L CNN
 F 1 "4.7kΩ" H 4270 5105 50  0000 L CNN
-F 2 "" V 4130 5150 50  0001 C CNN
+F 2 "Resistors_SMD:R_0603" V 4130 5150 50  0001 C CNN
 F 3 "" H 4200 5150 50  0000 C CNN
 	1    4200 5150
@@
 F 0 "R219" V 3700 5950 50  0000 C CNN
 F 1 "4.7kΩ" V 3900 5950 50  0000 C CNN
-F 2 "" V 3730 5950 50  0001 C CNN
+F 2 "Resistors_SMD:R_0603" V 3730 5950 50  0001 C CNN
 F 3 "" H 3800 5950 50  0000 C CNN
 	1    3800 5950
@@
 F 0 "R223" H 5770 5646 50  0000 L CNN
 F 1 "4.7kΩ" H 5770 5555 50  0000 L CNN
-F 2 "" V 5630 5600 50  0001 C CNN
+F 2 "Resistors_SMD:R_0603" V 5630 5600 50  0001 C CNN
 F 3 "" H 5700 5600 50  0000 C CNN
 	1    5700 5600
@@
 F 0 "C216" H 5815 4896 50  0000 L CNN
 F 1 "4.7nF" H 5815 4805 50  0000 L CNN
-F 2 "Capacitors_SMD:C_0402" H 5738 4700 50  0001 C CNN
+F 2 "Capacitors_SMD:C_0603" H 5738 4700 50  0001 C CNN
 F 3 "" H 5700 4850 50  0000 C CNN
 	1    5700 4850
@@
 F 0 "FB43" V 5485 5200 50  0000 C CNN
 F 1 "CIM21J202NE" V 5394 5200 50  0000 C CNN
-F 2 "" H 5300 5200 50  0001 C CNN
+F 2 "Resistors_SMD:R_0805" H 5300 5200 50  0001 C CNN
 F 3 "" H 5300 5200 50  0000 C CNN
 	1    5300 5200
@@
 $EndComp
 $Comp
-L D_Schottky D28
+L D_Schottky D29
 U 1 1 5B5F23B6
 P 8100 5550
-F 0 "D28" V 8000 5400 50  0000 L CNN
+F 0 "D29" V 8000 5400 50  0000 L CNN
 F 1 "MBRA340T3" V 8250 5100 50  0000 L CNN
 F 2 "" H 8100 5550 50  0001 C CNN
@@
 F 0 "R224" V 6900 5600 50  0000 C CNN
 F 1 "10Ω" V 7100 5600 50  0000 C CNN
-F 2 "" V 6930 5600 50  0001 C CNN
+F 2 "Resistors_SMD:R_0603" V 6930 5600 50  0001 C CNN
 F 3 "" H 7000 5600 50  0000 C CNN
 	1    7000 5600
@@
 $EndComp
 $Comp
-L LED_Short D29
+L LED_Short D30
 U 1 1 5B5F23CB
 P 8450 5750
-F 0 "D29" V 8496 5642 50  0000 R CNN
+F 0 "D30" V 8496 5642 50  0000 R CNN
 F 1 "LED" V 8405 5642 50  0000 R CNN
-F 2 "" H 8450 5750 50  0001 C CNN
+F 2 "LEDs:LED_0603" H 8450 5750 50  0001 C CNN
 F 3 "" H 8450 5750 50  0000 C CNN
 	1    8450 5750
@@
 F 0 "R228" H 8520 5446 50  0000 L CNN
 F 1 "4.7kΩ" H 8520 5355 50  0000 L CNN
-F 2 "" V 8380 5400 50  0001 C CNN
+F 2 "Resistors_SMD:R_0603" V 8380 5400 50  0001 C CNN
 F 3 "" H 8450 5400 50  0000 C CNN
 	1    8450 5400
@@
 F 0 "R226" H 7570 4796 50  0000 L CNN
 F 1 "4.7kΩ" H 7570 4705 50  0000 L CNN
-F 2 "" V 7430 4750 50  0001 C CNN
+F 2 "Resistors_SMD:R_0603" V 7430 4750 50  0001 C CNN
 F 3 "" H 7500 4750 50  0000 C CNN
 	1    7500 4750
@@
 F 0 "R227" H 7570 5196 50  0000 L CNN
 F 1 "4.7kΩ" H 7570 5105 50  0000 L CNN
-F 2 "" V 7430 5150 50  0001 C CNN
+F 2 "Resistors_SMD:R_0603" V 7430 5150 50  0001 C CNN
 F 3 "" H 7500 5150 50  0000 C CNN
 	1    7500 5150
@@
 F 0 "R225" V 7000 5950 50  0000 C CNN
 F 1 "4.7kΩ" V 7200 5950 50  0000 C CNN
-F 2 "" V 7030 5950 50  0001 C CNN
+F 2 "Resistors_SMD:R_0603" V 7030 5950 50  0001 C CNN
 F 3 "" H 7100 5950 50  0000 C CNN
 	1    7100 5950
@@
 F 0 "R229" H 9070 5646 50  0000 L CNN
 F 1 "4.7kΩ" H 9070 5555 50  0000 L CNN
-F 2 "" V 8930 5600 50  0001 C CNN
+F 2 "Resistors_SMD:R_0603" V 8930 5600 50  0001 C CNN
 F 3 "" H 9000 5600 50  0000 C CNN
 	1    9000 5600
@@
 F 0 "C217" H 9115 4896 50  0000 L CNN
 F 1 "4.7nF" H 9115 4805 50  0000 L CNN
-F 2 "Capacitors_SMD:C_0402" H 9038 4700 50  0001 C CNN
+F 2 "Capacitors_SMD:C_0603" H 9038 4700 50  0001 C CNN
 F 3 "" H 9000 4850 50  0000 C CNN
 	1    9000 4850
@@
 F 0 "FB44" V 8785 5200 50  0000 C CNN
 F 1 "CIM21J202NE" V 8694 5200 50  0000 C CNN
-F 2 "" H 8600 5200 50  0001 C CNN
+F 2 "Resistors_SMD:R_0805" H 8600 5200 50  0001 C CNN
 F 3 "" H 8600 5200 50  0000 C CNN
 	1    8600 5200
@@
 $EndComp
 $Comp
-L D_Schottky D30
+L D_Schottky D31
 U 1 1 5B5F29A1
 P 11400 5550
-F 0 "D30" V 11300 5400 50  0000 L CNN
+F 0 "D31" V 11300 5400 50  0000 L CNN
 F 1 "MBRA340T3" V 11550 5100 50  0000 L CNN
 F 2 "" H 11400 5550 50  0001 C CNN
@@
 F 0 "R230" V 10200 5600 50  0000 C CNN
 F 1 "10Ω" V 10400 5600 50  0000 C CNN
-F 2 "" V 10230 5600 50  0001 C CNN
+F 2 "Resistors_SMD:R_0603" V 10230 5600 50  0001 C CNN
 F 3 "" H 10300 5600 50  0000 C CNN
 	1    10300 5600
@@
 $EndComp
 $Comp
-L LED_Short D31
+L LED_Short D32
 U 1 1 5B5F29B6
 P 11750 5750
-F 0 "D31" V 11796 5642 50  0000 R CNN
+F 0 "D32" V 11796 5642 50  0000 R CNN
 F 1 "LED" V 11705 5642 50  0000 R CNN
-F 2 "" H 11750 5750 50  0001 C CNN
+F 2 "LEDs:LED_0603" H 11750 5750 50  0001 C CNN
 F 3 "" H 11750 5750 50  0000 C CNN
 	1    11750 5750
@@
 F 0 "R234" H 11820 5446 50  0000 L CNN
 F 1 "4.7kΩ" H 11820 5355 50  0000 L CNN
-F 2 "" V 11680 5400 50  0001 C CNN
+F 2 "Resistors_SMD:R_0603" V 11680 5400 50  0001 C CNN
 F 3 "" H 11750 5400 50  0000 C CNN
 	1    11750 5400
@@
 F 0 "R232" H 10870 4796 50  0000 L CNN
 F 1 "4.7kΩ" H 10870 4705 50  0000 L CNN
-F 2 "" V 10730 4750 50  0001 C CNN
+F 2 "Resistors_SMD:R_0603" V 10730 4750 50  0001 C CNN
 F 3 "" H 10800 4750 50  0000 C CNN
 	1    10800 4750
@@
 F 0 "R233" H 10870 5196 50  0000 L CNN
 F 1 "4.7kΩ" H 10870 5105 50  0000 L CNN
-F 2 "" V 10730 5150 50  0001 C CNN
+F 2 "Resistors_SMD:R_0603" V 10730 5150 50  0001 C CNN
 F 3 "" H 10800 5150 50  0000 C CNN
 	1    10800 5150
@@
 F 0 "R231" V 10300 5950 50  0000 C CNN
 F 1 "4.7kΩ" V 10500 5950 50  0000 C CNN
-F 2 "" V 10330 5950 50  0001 C CNN
+F 2 "Resistors_SMD:R_0603" V 10330 5950 50  0001 C CNN
 F 3 "" H 10400 5950 50  0000 C CNN
 	1    10400 5950
@@
 F 0 "R235" H 12370 5646 50  0000 L CNN
 F 1 "4.7kΩ" H 12370 5555 50  0000 L CNN
-F 2 "" V 12230 5600 50  0001 C CNN
+F 2 "Resistors_SMD:R_0603" V 12230 5600 50  0001 C CNN
 F 3 "" H 12300 5600 50  0000 C CNN
 	1    12300 5600
@@
 F 0 "C218" H 12415 4896 50  0000 L CNN
 F 1 "4.7nF" H 12415 4805 50  0000 L CNN
-F 2 "Capacitors_SMD:C_0402" H 12338 4700 50  0001 C CNN
+F 2 "Capacitors_SMD:C_0603" H 12338 4700 50  0001 C CNN
 F 3 "" H 12300 4850 50  0000 C CNN
 	1    12300 4850
@@
 F 0 "FB45" V 12085 5200 50  0000 C CNN
 F 1 "CIM21J202NE" V 11994 5200 50  0000 C CNN
-F 2 "" H 11900 5200 50  0001 C CNN
+F 2 "Resistors_SMD:R_0805" H 11900 5200 50  0001 C CNN
 F 3 "" H 11900 5200 50  0000 C CNN
 	1    11900 5200
