File: KiMBo/fan.sch (KiCad schematic (older format))
At the start: 36 parts, among them Q15 2N7002, Q16 DMP3098L-7, Q17 2N7002, Q18 DMP3098L-7, Q19 2N7002, Q20 DMP3098L-7

Commit message: More footprint association
Parts:
- D28: renamed from D27; footprint (none) -> KiMBo:MBR-DO-214AC
- D30: renamed from D29; footprint (none) -> KiMBo:MBR-DO-214AC
- D32: renamed from D31; footprint (none) -> KiMBo:MBR-DO-214AC
- Q15, Q16, Q17, Q18, Q19, Q20: footprint (none) -> TO_SOT_Packages_SMD:SOT-23
- renumbered D28 to D29, D30 to D31, D32 to D33
Changed lines of the file:
@@
 E_FAN
 $Comp
-L +24V #PWR0272
+L +24V #PWR0273
 U 1 1 5B5EFE55
 P 4800 4500
-F 0 "#PWR0272" H 4800 4350 50  0001 C CNN
+F 0 "#PWR0273" H 4800 4350 50  0001 C CNN
 F 1 "+24V" H 4815 4673 50  0000 C CNN
 F 2 "" H 4800 4500 50  0000 C CNN
@@
 $EndComp
 $Comp
-L GND #PWR0273
+L GND #PWR0274
 U 1 1 5B5EFE5B
 P 4200 6000
-F 0 "#PWR0273" H 4200 5750 50  0001 C CNN
+F 0 "#PWR0274" H 4200 5750 50  0001 C CNN
 F 1 "GND" H 4205 5827 50  0000 C CNN
 F 2 "" H 4200 6000 50  0000 C CNN
@@
 $EndComp
 $Comp
-L D_Schottky D27
+L D_Schottky D28
 U 1 1 5B5EFE61
 P 4800 5550
-F 0 "D27" V 4700 5400 50  0000 L CNN
+F 0 "D28" V 4700 5400 50  0000 L CNN
 F 1 "MBRA340T3" V 4950 5100 50  0000 L CNN
-F 2 "" H 4800 5550 50  0001 C CNN
+F 2 "KiMBo:MBR-DO-214AC" H 4800 5550 50  0001 C CNN
 F 3 "" H 4800 5550 50  0000 C CNN
 	1    4800 5550
@@
 F 0 "Q15" H 4050 5750 40  0000 L CNN
 F 1 "2N7002" H 3850 5475 40  0000 L CNN
-F 2 "" H 3970 5702 29  0001 C CNN
+F 2 "TO_SOT_Packages_SMD:SOT-23" H 3970 5702 29  0001 C CNN
 F 3 "" H 4100 5600 60  0000 C CNN
 	1    4100 5600
@@
 $EndComp
 $Comp
-L LED_Short D28
+L LED_Short D29
 U 1 1 5B5EFE77
 P 5150 5750
-F 0 "D28" V 5196 5642 50  0000 R CNN
+F 0 "D29" V 5196 5642 50  0000 R CNN
 F 1 "LED" V 5105 5642 50  0000 R CNN
 F 2 "LEDs:LED_0603" H 5150 5750 50  0001 C CNN
@@
 F 0 "Q16" H 4900 5100 50  0000 L CNN
 F 1 "DMP3098L-7" H 4900 5000 50  0000 L CNN
-F 2 "" H 4950 5025 50  0001 L CNN
+F 2 "TO_SOT_Packages_SMD:SOT-23" H 4950 5025 50  0001 L CNN
 F 3 "http://www.diodes.com/_files/datasheets/ds31447.pdf" H 4891 4859 50  0001 L CNN
 	1    4700 4950
@@
 H_FAN
 $Comp
-L +24V #PWR0274
+L +24V #PWR0275
 U 1 1 5B5F23AA
 P 8100 4500
-F 0 "#PWR0274" H 8100 4350 50  0001 C CNN
+F 0 "#PWR0275" H 8100 4350 50  0001 C CNN
 F 1 "+24V" H 8115 4673 50  0000 C CNN
 F 2 "" H 8100 4500 50  0000 C CNN
@@
 $EndComp
 $Comp
-L GND #PWR0275
+L GND #PWR0276
 U 1 1 5B5F23B0
 P 7500 6000
-F 0 "#PWR0275" H 7500 5750 50  0001 C CNN
+F 0 "#PWR0276" H 7500 5750 50  0001 C CNN
 F 1 "GND" H 7505 5827 50  0000 C CNN
 F 2 "" H 7500 6000 50  0000 C CNN
@@
 $EndComp
 $Comp
-L D_Schottky D29
+L D_Schottky D30
 U 1 1 5B5F23B6
 P 8100 5550
-F 0 "D29" V 8000 5400 50  0000 L CNN
+F 0 "D30" V 8000 5400 50  0000 L CNN
 F 1 "MBRA340T3" V 8250 5100 50  0000 L CNN
-F 2 "" H 8100 5550 50  0001 C CNN
+F 2 "KiMBo:MBR-DO-214AC" H 8100 5550 50  0001 C CNN
 F 3 "" H 8100 5550 50  0000 C CNN
 	1    8100 5550
@@
 $EndComp
 $Comp
-L LED_Short D30
+L LED_Short D31
 U 1 1 5B5F23CB
 P 8450 5750
-F 0 "D30" V 8496 5642 50  0000 R CNN
+F 0 "D31" V 8496 5642 50  0000 R CNN
 F 1 "LED" V 8405 5642 50  0000 R CNN
 F 2 "LEDs:LED_0603" H 8450 5750 50  0001 C CNN
@@
 F 0 "Q18" H 8200 5100 50  0000 L CNN
 F 1 "DMP3098L-7" H 8200 5000 50  0000 L CNN
-F 2 "" H 8250 5025 50  0001 L CNN
+F 2 "TO_SOT_Packages_SMD:SOT-23" H 8250 5025 50  0001 L CNN
 F 3 "http://www.diodes.com/_files/datasheets/ds31447.pdf" H 8191 4859 50  0001 L CNN
 	1    8000 4950
@@
 CASE_FAN
 $Comp
-L +24V #PWR0276
+L +24V #PWR0277
 U 1 1 5B5F2995
 P 11400 4500
-F 0 "#PWR0276" H 11400 4350 50  0001 C CNN
+F 0 "#PWR0277" H 11400 4350 50  0001 C CNN
 F 1 "+24V" H 11415 4673 50  0000 C CNN
 F 2 "" H 11400 4500 50  0000 C CNN
@@
 $EndComp
 $Comp
-L GND #PWR0277
+L GND #PWR0278
 U 1 1 5B5F299B
 P 10800 6000
-F 0 "#PWR0277" H 10800 5750 50  0001 C CNN
+F 0 "#PWR0278" H 10800 5750 50  0001 C CNN
 F 1 "GND" H 10805 5827 50  0000 C CNN
 F 2 "" H 10800 6000 50  0000 C CNN
@@
 $EndComp
 $Comp
-L D_Schottky D31
+L D_Schottky D32
 U 1 1 5B5F29A1
 P 11400 5550
-F 0 "D31" V 11300 5400 50  0000 L CNN
+F 0 "D32" V 11300 5400 50  0000 L CNN
 F 1 "MBRA340T3" V 11550 5100 50  0000 L CNN
-F 2 "" H 11400 5550 50  0001 C CNN
+F 2 "KiMBo:MBR-DO-214AC" H 11400 5550 50  0001 C CNN
 F 3 "" H 11400 5550 50  0000 C CNN
 	1    11400 5550
@@
 $EndComp
 $Comp
-L LED_Short D32
+L LED_Short D33
 U 1 1 5B5F29B6
 P 11750 5750
-F 0 "D32" V 11796 5642 50  0000 R CNN
+F 0 "D33" V 11796 5642 50  0000 R CNN
 F 1 "LED" V 11705 5642 50  0000 R CNN
 F 2 "LEDs:LED_0603" H 11750 5750 50  0001 C CNN
@@
 F 0 "Q20" H 11500 5100 50  0000 L CNN
 F 1 "DMP3098L-7" H 11500 5000 50  0000 L CNN
-F 2 "" H 11550 5025 50  0001 L CNN
+F 2 "TO_SOT_Packages_SMD:SOT-23" H 11550 5025 50  0001 L CNN
 F 3 "http://www.diodes.com/_files/datasheets/ds31447.pdf" H 11491 4859 50  0001 L CNN
 	1    11300 4950
@@
 F 0 "Q17" H 7350 5750 40  0000 L CNN
 F 1 "2N7002" H 7150 5475 40  0000 L CNN
-F 2 "" H 7270 5702 29  0001 C CNN
+F 2 "TO_SOT_Packages_SMD:SOT-23" H 7270 5702 29  0001 C CNN
 F 3 "" H 7400 5600 60  0000 C CNN
 	1    7400 5600
@@
 F 0 "Q19" H 10650 5750 40  0000 L CNN
 F 1 "2N7002" H 10450 5475 40  0000 L CNN
-F 2 "" H 10570 5702 29  0001 C CNN
+F 2 "TO_SOT_Packages_SMD:SOT-23" H 10570 5702 29  0001 C CNN
 F 3 "" H 10700 5600 60  0000 C CNN
 	1    10700 5600

Commit message: Add more footprints and more associations, one association left!
Parts:
- renumbered R218 to R227, R219 to R228, R220 to R229, R221 to R230, R222 to R231, R223 to R232, R224 to R233, R225 to R234, R226 to R235, R227 to R236, R228 to R237, R229 to R238, R230 to R239, R231 to R240, R232 to R241, R233 to R242, R234 to R243, R235 to R244
Changed lines of the file:
@@
 E_FAN
 $Comp
-L +24V #PWR0273
+L +24V #PWR0275
 U 1 1 5B5EFE55
 P 4800 4500
-F 0 "#PWR0273" H 4800 4350 50  0001 C CNN
+F 0 "#PWR0275" H 4800 4350 50  0001 C CNN
 F 1 "+24V" H 4815 4673 50  0000 C CNN
 F 2 "" H 4800 4500 50  0000 C CNN
@@
 $EndComp
 $Comp
-L GND #PWR0274
+L GND #PWR0276
 U 1 1 5B5EFE5B
 P 4200 6000
-F 0 "#PWR0274" H 4200 5750 50  0001 C CNN
+F 0 "#PWR0276" H 4200 5750 50  0001 C CNN
 F 1 "GND" H 4205 5827 50  0000 C CNN
 F 2 "" H 4200 6000 50  0000 C CNN
@@
 $EndComp
 $Comp
-L R R218
+L R R227
 U 1 1 5B5EFE68
 P 3700 5600
-F 0 "R218" V 3600 5600 50  0000 C CNN
+F 0 "R227" V 3600 5600 50  0000 C CNN
 F 1 "10Ω" V 3800 5600 50  0000 C CNN
 F 2 "Resistors_SMD:R_0603" V 3630 5600 50  0001 C CNN
@@
 $EndComp
 $Comp
-L R R222
+L R R231
 U 1 1 5B5EFE7E
 P 5150 5400
-F 0 "R222" H 5220 5446 50  0000 L CNN
+F 0 "R231" H 5220 5446 50  0000 L CNN
 F 1 "4.7kΩ" H 5220 5355 50  0000 L CNN
 F 2 "Resistors_SMD:R_0603" V 5080 5400 50  0001 C CNN
@@
 $EndComp
 $Comp
-L R R220
+L R R229
 U 1 1 5B5EFE85
 P 4200 4750
-F 0 "R220" H 4270 4796 50  0000 L CNN
+F 0 "R229" H 4270 4796 50  0000 L CNN
 F 1 "4.7kΩ" H 4270 4705 50  0000 L CNN
 F 2 "Resistors_SMD:R_0603" V 4130 4750 50  0001 C CNN
@@
 $EndComp
 $Comp
-L R R221
+L R R230
 U 1 1 5B5EFE8C
 P 4200 5150
-F 0 "R221" H 4270 5196 50  0000 L CNN
+F 0 "R230" H 4270 5196 50  0000 L CNN
 F 1 "4.7kΩ" H 4270 5105 50  0000 L CNN
 F 2 "Resistors_SMD:R_0603" V 4130 5150 50  0001 C CNN
@@
 $EndComp
 $Comp
-L R R219
+L R R228
 U 1 1 5B5EFE93
 P 3800 5950
-F 0 "R219" V 3700 5950 50  0000 C CNN
+F 0 "R228" V 3700 5950 50  0000 C CNN
 F 1 "4.7kΩ" V 3900 5950 50  0000 C CNN
 F 2 "Resistors_SMD:R_0603" V 3730 5950 50  0001 C CNN
@@
 $EndComp
 $Comp
-L R R223
+L R R232
 U 1 1 5B5EFE9A
 P 5700 5600
-F 0 "R223" H 5770 5646 50  0000 L CNN
+F 0 "R232" H 5770 5646 50  0000 L CNN
 F 1 "4.7kΩ" H 5770 5555 50  0000 L CNN
 F 2 "Resistors_SMD:R_0603" V 5630 5600 50  0001 C CNN
@@
 H_FAN
 $Comp
-L +24V #PWR0275
+L +24V #PWR0277
 U 1 1 5B5F23AA
 P 8100 4500
-F 0 "#PWR0275" H 8100 4350 50  0001 C CNN
+F 0 "#PWR0277" H 8100 4350 50  0001 C CNN
 F 1 "+24V" H 8115 4673 50  0000 C CNN
 F 2 "" H 8100 4500 50  0000 C CNN
@@
 $EndComp
 $Comp
-L GND #PWR0276
+L GND #PWR0278
 U 1 1 5B5F23B0
 P 7500 6000
-F 0 "#PWR0276" H 7500 5750 50  0001 C CNN
+F 0 "#PWR0278" H 7500 5750 50  0001 C CNN
 F 1 "GND" H 7505 5827 50  0000 C CNN
 F 2 "" H 7500 6000 50  0000 C CNN
@@
 $EndComp
 $Comp
-L R R224
+L R R233
 U 1 1 5B5F23BD
 P 7000 5600
-F 0 "R224" V 6900 5600 50  0000 C CNN
+F 0 "R233" V 6900 5600 50  0000 C CNN
 F 1 "10Ω" V 7100 5600 50  0000 C CNN
 F 2 "Resistors_SMD:R_0603" V 6930 5600 50  0001 C CNN
@@
 $EndComp
 $Comp
-L R R228
+L R R237
 U 1 1 5B5F23D2
 P 8450 5400
-F 0 "R228" H 8520 5446 50  0000 L CNN
+F 0 "R237" H 8520 5446 50  0000 L CNN
 F 1 "4.7kΩ" H 8520 5355 50  0000 L CNN
 F 2 "Resistors_SMD:R_0603" V 8380 5400 50  0001 C CNN
@@
 $EndComp
 $Comp
-L R R226
+L R R235
 U 1 1 5B5F23D9
 P 7500 4750
-F 0 "R226" H 7570 4796 50  0000 L CNN
+F 0 "R235" H 7570 4796 50  0000 L CNN
 F 1 "4.7kΩ" H 7570 4705 50  0000 L CNN
 F 2 "Resistors_SMD:R_0603" V 7430 4750 50  0001 C CNN
@@
 $EndComp
 $Comp
-L R R227
+L R R236
 U 1 1 5B5F23E0
 P 7500 5150
-F 0 "R227" H 7570 5196 50  0000 L CNN
+F 0 "R236" H 7570 5196 50  0000 L CNN
 F 1 "4.7kΩ" H 7570 5105 50  0000 L CNN
 F 2 "Resistors_SMD:R_0603" V 7430 5150 50  0001 C CNN
@@
 $EndComp
 $Comp
-L R R225
+L R R234
 U 1 1 5B5F23E7
 P 7100 5950
-F 0 "R225" V 7000 5950 50  0000 C CNN
+F 0 "R234" V 7000 5950 50  0000 C CNN
 F 1 "4.7kΩ" V 7200 5950 50  0000 C CNN
 F 2 "Resistors_SMD:R_0603" V 7030 5950 50  0001 C CNN
@@
 $EndComp
 $Comp
-L R R229
+L R R238
 U 1 1 5B5F23EE
 P 9000 5600
-F 0 "R229" H 9070 5646 50  0000 L CNN
+F 0 "R238" H 9070 5646 50  0000 L CNN
 F 1 "4.7kΩ" H 9070 5555 50  0000 L CNN
 F 2 "Resistors_SMD:R_0603" V 8930 5600 50  0001 C CNN
@@
 CASE_FAN
 $Comp
-L +24V #PWR0277
+L +24V #PWR0279
 U 1 1 5B5F2995
 P 11400 4500
-F 0 "#PWR0277" H 11400 4350 50  0001 C CNN
+F 0 "#PWR0279" H 11400 4350 50  0001 C CNN
 F 1 "+24V" H 11415 4673 50  0000 C CNN
 F 2 "" H 11400 4500 50  0000 C CNN
@@
 $EndComp
 $Comp
-L GND #PWR0278
+L GND #PWR0280
 U 1 1 5B5F299B
 P 10800 6000
-F 0 "#PWR0278" H 10800 5750 50  0001 C CNN
+F 0 "#PWR0280" H 10800 5750 50  0001 C CNN
 F 1 "GND" H 10805 5827 50  0000 C CNN
 F 2 "" H 10800 6000 50  0000 C CNN
@@
 $EndComp
 $Comp
-L R R230
+L R R239
 U 1 1 5B5F29A8
 P 10300 5600
-F 0 "R230" V 10200 5600 50  0000 C CNN
+F 0 "R239" V 10200 5600 50  0000 C CNN
 F 1 "10Ω" V 10400 5600 50  0000 C CNN
 F 2 "Resistors_SMD:R_0603" V 10230 5600 50  0001 C CNN
@@
 $EndComp
 $Comp
-L R R234
+L R R243
 U 1 1 5B5F29BD
 P 11750 5400
-F 0 "R234" H 11820 5446 50  0000 L CNN
+F 0 "R243" H 11820 5446 50  0000 L CNN
 F 1 "4.7kΩ" H 11820 5355 50  0000 L CNN
 F 2 "Resistors_SMD:R_0603" V 11680 5400 50  0001 C CNN
@@
 $EndComp
 $Comp
-L R R232
+L R R241
 U 1 1 5B5F29C4
 P 10800 4750
-F 0 "R232" H 10870 4796 50  0000 L CNN
+F 0 "R241" H 10870 4796 50  0000 L CNN
 F 1 "4.7kΩ" H 10870 4705 50  0000 L CNN
 F 2 "Resistors_SMD:R_0603" V 10730 4750 50  0001 C CNN
@@
 $EndComp
 $Comp
-L R R233
+L R R242
 U 1 1 5B5F29CB
 P 10800 5150
-F 0 "R233" H 10870 5196 50  0000 L CNN
+F 0 "R242" H 10870 5196 50  0000 L CNN
 F 1 "4.7kΩ" H 10870 5105 50  0000 L CNN
 F 2 "Resistors_SMD:R_0603" V 10730 5150 50  0001 C CNN
@@
 $EndComp
 $Comp
-L R R231
+L R R240
 U 1 1 5B5F29D2
 P 10400 5950
-F 0 "R231" V 10300 5950 50  0000 C CNN
+F 0 "R240" V 10300 5950 50  0000 C CNN
 F 1 "4.7kΩ" V 10500 5950 50  0000 C CNN
 F 2 "Resistors_SMD:R_0603" V 10330 5950 50  0001 C CNN
@@
 $EndComp
 $Comp
-L R R235
+L R R244
 U 1 1 5B5F29D9
 P 12300 5600
-F 0 "R235" H 12370 5646 50  0000 L CNN
+F 0 "R244" H 12370 5646 50  0000 L CNN
 F 1 "4.7kΩ" H 12370 5555 50  0000 L CNN
 F 2 "Resistors_SMD:R_0603" V 12230 5600 50  0001 C CNN

Commit message: Begin layout
Arrange all connectors to get a feel for the area.
Parts:
- renumbered C216 to C218, C217 to C219, C218 to C220, D28 to D29, D29 to D30, D30 to D31, D31 to D32, D32 to D33, D33 to D34
Changed lines of the file:
@@
 E_FAN
 $Comp
-L +24V #PWR0275
+L +24V #PWR0278
 U 1 1 5B5EFE55
 P 4800 4500
-F 0 "#PWR0275" H 4800 4350 50  0001 C CNN
+F 0 "#PWR0278" H 4800 4350 50  0001 C CNN
 F 1 "+24V" H 4815 4673 50  0000 C CNN
 F 2 "" H 4800 4500 50  0000 C CNN
@@
 $EndComp
 $Comp
-L GND #PWR0276
+L GND #PWR0279
 U 1 1 5B5EFE5B
 P 4200 6000
-F 0 "#PWR0276" H 4200 5750 50  0001 C CNN
+F 0 "#PWR0279" H 4200 5750 50  0001 C CNN
 F 1 "GND" H 4205 5827 50  0000 C CNN
 F 2 "" H 4200 6000 50  0000 C CNN
@@
 $EndComp
 $Comp
-L D_Schottky D28
+L D_Schottky D29
 U 1 1 5B5EFE61
 P 4800 5550
-F 0 "D28" V 4700 5400 50  0000 L CNN
+F 0 "D29" V 4700 5400 50  0000 L CNN
 F 1 "MBRA340T3" V 4950 5100 50  0000 L CNN
 F 2 "KiMBo:MBR-DO-214AC" H 4800 5550 50  0001 C CNN
@@
 $EndComp
 $Comp
-L LED_Short D29
+L LED_Short D30
 U 1 1 5B5EFE77
 P 5150 5750
-F 0 "D29" V 5196 5642 50  0000 R CNN
+F 0 "D30" V 5196 5642 50  0000 R CNN
 F 1 "LED" V 5105 5642 50  0000 R CNN
 F 2 "LEDs:LED_0603" H 5150 5750 50  0001 C CNN
@@
 $EndComp
 $Comp
-L C C216
+L C C218
 U 1 1 5B5EFEA1
 P 5700 4850
-F 0 "C216" H 5815 4896 50  0000 L CNN
+F 0 "C218" H 5815 4896 50  0000 L CNN
 F 1 "4.7nF" H 5815 4805 50  0000 L CNN
 F 2 "Capacitors_SMD:C_0603" H 5738 4700 50  0001 C CNN
@@
 H_FAN
 $Comp
-L +24V #PWR0277
+L +24V #PWR0280
 U 1 1 5B5F23AA
 P 8100 4500
-F 0 "#PWR0277" H 8100 4350 50  0001 C CNN
+F 0 "#PWR0280" H 8100 4350 50  0001 C CNN
 F 1 "+24V" H 8115 4673 50  0000 C CNN
 F 2 "" H 8100 4500 50  0000 C CNN
@@
 $EndComp
 $Comp
-L GND #PWR0278
+L GND #PWR0281
 U 1 1 5B5F23B0
 P 7500 6000
-F 0 "#PWR0278" H 7500 5750 50  0001 C CNN
+F 0 "#PWR0281" H 7500 5750 50  0001 C CNN
 F 1 "GND" H 7505 5827 50  0000 C CNN
 F 2 "" H 7500 6000 50  0000 C CNN
@@
 $EndComp
 $Comp
-L D_Schottky D30
+L D_Schottky D31
 U 1 1 5B5F23B6
 P 8100 5550
-F 0 "D30" V 8000 5400 50  0000 L CNN
+F 0 "D31" V 8000 5400 50  0000 L CNN
 F 1 "MBRA340T3" V 8250 5100 50  0000 L CNN
 F 2 "KiMBo:MBR-DO-214AC" H 8100 5550 50  0001 C CNN
@@
 $EndComp
 $Comp
-L LED_Short D31
+L LED_Short D32
 U 1 1 5B5F23CB
 P 8450 5750
-F 0 "D31" V 8496 5642 50  0000 R CNN
+F 0 "D32" V 8496 5642 50  0000 R CNN
 F 1 "LED" V 8405 5642 50  0000 R CNN
 F 2 "LEDs:LED_0603" H 8450 5750 50  0001 C CNN
@@
 $EndComp
 $Comp
-L C C217
+L C C219
 U 1 1 5B5F23F5
 P 9000 4850
-F 0 "C217" H 9115 4896 50  0000 L CNN
+F 0 "C219" H 9115 4896 50  0000 L CNN
 F 1 "4.7nF" H 9115 4805 50  0000 L CNN
 F 2 "Capacitors_SMD:C_0603" H 9038 4700 50  0001 C CNN
@@
 CASE_FAN
 $Comp
-L +24V #PWR0279
+L +24V #PWR0282
 U 1 1 5B5F2995
 P 11400 4500
-F 0 "#PWR0279" H 11400 4350 50  0001 C CNN
+F 0 "#PWR0282" H 11400 4350 50  0001 C CNN
 F 1 "+24V" H 11415 4673 50  0000 C CNN
 F 2 "" H 11400 4500 50  0000 C CNN
@@
 $EndComp
 $Comp
-L GND #PWR0280
+L GND #PWR0283
 U 1 1 5B5F299B
 P 10800 6000
-F 0 "#PWR0280" H 10800 5750 50  0001 C CNN
+F 0 "#PWR0283" H 10800 5750 50  0001 C CNN
 F 1 "GND" H 10805 5827 50  0000 C CNN
 F 2 "" H 10800 6000 50  0000 C CNN
@@
 $EndComp
 $Comp
-L D_Schottky D32
+L D_Schottky D33
 U 1 1 5B5F29A1
 P 11400 5550
-F 0 "D32" V 11300 5400 50  0000 L CNN
+F 0 "D33" V 11300 5400 50  0000 L CNN
 F 1 "MBRA340T3" V 11550 5100 50  0000 L CNN
 F 2 "KiMBo:MBR-DO-214AC" H 11400 5550 50  0001 C CNN
@@
 $EndComp
 $Comp
-L LED_Short D33
+L LED_Short D34
 U 1 1 5B5F29B6
 P 11750 5750
-F 0 "D33" V 11796 5642 50  0000 R CNN
+F 0 "D34" V 11796 5642 50  0000 R CNN
 F 1 "LED" V 11705 5642 50  0000 R CNN
 F 2 "LEDs:LED_0603" H 11750 5750 50  0001 C CNN
@@
 $EndComp
 $Comp
-L C C218
+L C C220
 U 1 1 5B5F29E0
 P 12300 4850
-F 0 "C218" H 12415 4896 50  0000 L CNN
+F 0 "C220" H 12415 4896 50  0000 L CNN
 F 1 "4.7nF" H 12415 4805 50  0000 L CNN
 F 2 "Capacitors_SMD:C_0603" H 12338 4700 50  0001 C CNN
