File: KiMBo/fan.sch (KiCad schematic (older format))
At the start: 36 parts, among them Q15 2N7002, Q16 DMP3098L-7, Q17 2N7002, Q18 DMP3098L-7, Q19 2N7002, Q20 DMP3098L-7

Commit message: Remove HDMI from the schematic
Parts:
- renumbered C218 to C193, C219 to C194, C220 to C195, D29 to D28, D30 to D29, D31 to D30, D32 to D31, D33 to D32, D34 to D33, FB43 to FB41, FB44 to FB42, FB45 to FB43, R227 to R200, R228 to R201, R229 to R202, R230 to R203, R231 to R204, R232 to R205, R233 to R206, R234 to R207, R235 to R208, R236 to R209, R237 to R210, R238 to R211, R239 to R212, R240 to R213, R241 to R214, R242 to R215, R243 to R216, R244 to R217
Changed lines of the file:
@@
 $Descr A3 16535 11693
 encoding utf-8
-Sheet 26 26
+Sheet 26 25
 Title ""
 Date ""
@@
 E_FAN
 $Comp
-L +24V #PWR0278
+L +24V #PWR0247
 U 1 1 5B5EFE55
 P 4800 4500
-F 0 "#PWR0278" H 4800 4350 50  0001 C CNN
+F 0 "#PWR0247" H 4800 4350 50  0001 C CNN
 F 1 "+24V" H 4815 4673 50  0000 C CNN
 F 2 "" H 4800 4500 50  0000 C CNN
@@
 $EndComp
 $Comp
-L GND #PWR0279
+L GND #PWR0248
 U 1 1 5B5EFE5B
 P 4200 6000
-F 0 "#PWR0279" H 4200 5750 50  0001 C CNN
+F 0 "#PWR0248" H 4200 5750 50  0001 C CNN
 F 1 "GND" H 4205 5827 50  0000 C CNN
 F 2 "" H 4200 6000 50  0000 C CNN
@@
 $EndComp
 $Comp
-L D_Schottky D29
+L D_Schottky D28
 U 1 1 5B5EFE61
 P 4800 5550
-F 0 "D29" V 4700 5400 50  0000 L CNN
+F 0 "D28" V 4700 5400 50  0000 L CNN
 F 1 "MBRA340T3" V 4950 5100 50  0000 L CNN
 F 2 "KiMBo:MBR-DO-214AC" H 4800 5550 50  0001 C CNN
@@
 $EndComp
 $Comp
-L R R227
+L R R200
 U 1 1 5B5EFE68
 P 3700 5600
-F 0 "R227" V 3600 5600 50  0000 C CNN
+F 0 "R200" V 3600 5600 50  0000 C CNN
 F 1 "10Ω" V 3800 5600 50  0000 C CNN
 F 2 "Resistors_SMD:R_0603" V 3630 5600 50  0001 C CNN
@@
 $EndComp
 $Comp
-L LED_Short D30
+L LED_Short D29
 U 1 1 5B5EFE77
 P 5150 5750
-F 0 "D30" V 5196 5642 50  0000 R CNN
+F 0 "D29" V 5196 5642 50  0000 R CNN
 F 1 "LED" V 5105 5642 50  0000 R CNN
 F 2 "LEDs:LED_0603" H 5150 5750 50  0001 C CNN
@@
 $EndComp
 $Comp
-L R R231
+L R R204
 U 1 1 5B5EFE7E
 P 5150 5400
-F 0 "R231" H 5220 5446 50  0000 L CNN
+F 0 "R204" H 5220 5446 50  0000 L CNN
 F 1 "4.7kΩ" H 5220 5355 50  0000 L CNN
 F 2 "Resistors_SMD:R_0603" V 5080 5400 50  0001 C CNN
@@
 $EndComp
 $Comp
-L R R229
+L R R202
 U 1 1 5B5EFE85
 P 4200 4750
-F 0 "R229" H 4270 4796 50  0000 L CNN
+F 0 "R202" H 4270 4796 50  0000 L CNN
 F 1 "4.7kΩ" H 4270 4705 50  0000 L CNN
 F 2 "Resistors_SMD:R_0603" V 4130 4750 50  0001 C CNN
@@
 $EndComp
 $Comp
-L R R230
+L R R203
 U 1 1 5B5EFE8C
 P 4200 5150
-F 0 "R230" H 4270 5196 50  0000 L CNN
+F 0 "R203" H 4270 5196 50  0000 L CNN
 F 1 "4.7kΩ" H 4270 5105 50  0000 L CNN
 F 2 "Resistors_SMD:R_0603" V 4130 5150 50  0001 C CNN
@@
 $EndComp
 $Comp
-L R R228
+L R R201
 U 1 1 5B5EFE93
 P 3800 5950
-F 0 "R228" V 3700 5950 50  0000 C CNN
+F 0 "R201" V 3700 5950 50  0000 C CNN
 F 1 "4.7kΩ" V 3900 5950 50  0000 C CNN
 F 2 "Resistors_SMD:R_0603" V 3730 5950 50  0001 C CNN
@@
 $EndComp
 $Comp
-L R R232
+L R R205
 U 1 1 5B5EFE9A
 P 5700 5600
-F 0 "R232" H 5770 5646 50  0000 L CNN
+F 0 "R205" H 5770 5646 50  0000 L CNN
 F 1 "4.7kΩ" H 5770 5555 50  0000 L CNN
 F 2 "Resistors_SMD:R_0603" V 5630 5600 50  0001 C CNN
@@
 $EndComp
 $Comp
-L C C218
+L C C193
 U 1 1 5B5EFEA1
 P 5700 4850
-F 0 "C218" H 5815 4896 50  0000 L CNN
+F 0 "C193" H 5815 4896 50  0000 L CNN
 F 1 "4.7nF" H 5815 4805 50  0000 L CNN
 F 2 "Capacitors_SMD:C_0603" H 5738 4700 50  0001 C CNN
@@
 $EndComp
 $Comp
-L INDUCTOR_Small FB43
+L INDUCTOR_Small FB41
 U 1 1 5B5F15E2
 P 5300 5200
-F 0 "FB43" V 5485 5200 50  0000 C CNN
+F 0 "FB41" V 5485 5200 50  0000 C CNN
 F 1 "CIM21J202NE" V 5394 5200 50  0000 C CNN
 F 2 "Resistors_SMD:R_0805" H 5300 5200 50  0001 C CNN
@@
 H_FAN
 $Comp
-L +24V #PWR0280
+L +24V #PWR0249
 U 1 1 5B5F23AA
 P 8100 4500
-F 0 "#PWR0280" H 8100 4350 50  0001 C CNN
+F 0 "#PWR0249" H 8100 4350 50  0001 C CNN
 F 1 "+24V" H 8115 4673 50  0000 C CNN
 F 2 "" H 8100 4500 50  0000 C CNN
@@
 $EndComp
 $Comp
-L GND #PWR0281
+L GND #PWR0250
 U 1 1 5B5F23B0
 P 7500 6000
-F 0 "#PWR0281" H 7500 5750 50  0001 C CNN
+F 0 "#PWR0250" H 7500 5750 50  0001 C CNN
 F 1 "GND" H 7505 5827 50  0000 C CNN
 F 2 "" H 7500 6000 50  0000 C CNN
@@
 $EndComp
 $Comp
-L D_Schottky D31
+L D_Schottky D30
 U 1 1 5B5F23B6
 P 8100 5550
-F 0 "D31" V 8000 5400 50  0000 L CNN
+F 0 "D30" V 8000 5400 50  0000 L CNN
 F 1 "MBRA340T3" V 8250 5100 50  0000 L CNN
 F 2 "KiMBo:MBR-DO-214AC" H 8100 5550 50  0001 C CNN
@@
 $EndComp
 $Comp
-L R R233
+L R R206
 U 1 1 5B5F23BD
 P 7000 5600
-F 0 "R233" V 6900 5600 50  0000 C CNN
+F 0 "R206" V 6900 5600 50  0000 C CNN
 F 1 "10Ω" V 7100 5600 50  0000 C CNN
 F 2 "Resistors_SMD:R_0603" V 6930 5600 50  0001 C CNN
@@
 $EndComp
 $Comp
-L LED_Short D32
+L LED_Short D31
 U 1 1 5B5F23CB
 P 8450 5750
-F 0 "D32" V 8496 5642 50  0000 R CNN
+F 0 "D31" V 8496 5642 50  0000 R CNN
 F 1 "LED" V 8405 5642 50  0000 R CNN
 F 2 "LEDs:LED_0603" H 8450 5750 50  0001 C CNN
@@
 $EndComp
 $Comp
-L R R237
+L R R210
 U 1 1 5B5F23D2
 P 8450 5400
-F 0 "R237" H 8520 5446 50  0000 L CNN
+F 0 "R210" H 8520 5446 50  0000 L CNN
 F 1 "4.7kΩ" H 8520 5355 50  0000 L CNN
 F 2 "Resistors_SMD:R_0603" V 8380 5400 50  0001 C CNN
@@
 $EndComp
 $Comp
-L R R235
+L R R208
 U 1 1 5B5F23D9
 P 7500 4750
-F 0 "R235" H 7570 4796 50  0000 L CNN
+F 0 "R208" H 7570 4796 50  0000 L CNN
 F 1 "4.7kΩ" H 7570 4705 50  0000 L CNN
 F 2 "Resistors_SMD:R_0603" V 7430 4750 50  0001 C CNN
@@
 $EndComp
 $Comp
-L R R236
+L R R209
 U 1 1 5B5F23E0
 P 7500 5150
-F 0 "R236" H 7570 5196 50  0000 L CNN
+F 0 "R209" H 7570 5196 50  0000 L CNN
 F 1 "4.7kΩ" H 7570 5105 50  0000 L CNN
 F 2 "Resistors_SMD:R_0603" V 7430 5150 50  0001 C CNN
@@
 $EndComp
 $Comp
-L R R234
+L R R207
 U 1 1 5B5F23E7
 P 7100 5950
-F 0 "R234" V 7000 5950 50  0000 C CNN
+F 0 "R207" V 7000 5950 50  0000 C CNN
 F 1 "4.7kΩ" V 7200 5950 50  0000 C CNN
 F 2 "Resistors_SMD:R_0603" V 7030 5950 50  0001 C CNN
@@
 $EndComp
 $Comp
-L R R238
+L R R211
 U 1 1 5B5F23EE
 P 9000 5600
-F 0 "R238" H 9070 5646 50  0000 L CNN
+F 0 "R211" H 9070 5646 50  0000 L CNN
 F 1 "4.7kΩ" H 9070 5555 50  0000 L CNN
 F 2 "Resistors_SMD:R_0603" V 8930 5600 50  0001 C CNN
@@
 $EndComp
 $Comp
-L C C219
+L C C194
 U 1 1 5B5F23F5
 P 9000 4850
-F 0 "C219" H 9115 4896 50  0000 L CNN
+F 0 "C194" H 9115 4896 50  0000 L CNN
 F 1 "4.7nF" H 9115 4805 50  0000 L CNN
 F 2 "Capacitors_SMD:C_0603" H 9038 4700 50  0001 C CNN
@@
 $EndComp
 $Comp
-L INDUCTOR_Small FB44
+L INDUCTOR_Small FB42
 U 1 1 5B5F2422
 P 8600 5200
-F 0 "FB44" V 8785 5200 50  0000 C CNN
+F 0 "FB42" V 8785 5200 50  0000 C CNN
 F 1 "CIM21J202NE" V 8694 5200 50  0000 C CNN
 F 2 "Resistors_SMD:R_0805" H 8600 5200 50  0001 C CNN
@@
 CASE_FAN
 $Comp
-L +24V #PWR0282
+L +24V #PWR0251
 U 1 1 5B5F2995
 P 11400 4500
-F 0 "#PWR0282" H 11400 4350 50  0001 C CNN
+F 0 "#PWR0251" H 11400 4350 50  0001 C CNN
 F 1 "+24V" H 11415 4673 50  0000 C CNN
 F 2 "" H 11400 4500 50  0000 C CNN
@@
 $EndComp
 $Comp
-L GND #PWR0283
+L GND #PWR0252
 U 1 1 5B5F299B
 P 10800 6000
-F 0 "#PWR0283" H 10800 5750 50  0001 C CNN
+F 0 "#PWR0252" H 10800 5750 50  0001 C CNN
 F 1 "GND" H 10805 5827 50  0000 C CNN
 F 2 "" H 10800 6000 50  0000 C CNN
@@
 $EndComp
 $Comp
-L D_Schottky D33
+L D_Schottky D32
 U 1 1 5B5F29A1
 P 11400 5550
-F 0 "D33" V 11300 5400 50  0000 L CNN
+F 0 "D32" V 11300 5400 50  0000 L CNN
 F 1 "MBRA340T3" V 11550 5100 50  0000 L CNN
 F 2 "KiMBo:MBR-DO-214AC" H 11400 5550 50  0001 C CNN
@@
 $EndComp
 $Comp
-L R R239
+L R R212
 U 1 1 5B5F29A8
 P 10300 5600
-F 0 "R239" V 10200 5600 50  0000 C CNN
+F 0 "R212" V 10200 5600 50  0000 C CNN
 F 1 "10Ω" V 10400 5600 50  0000 C CNN
 F 2 "Resistors_SMD:R_0603" V 10230 5600 50  0001 C CNN
@@
 $EndComp
 $Comp
-L LED_Short D34
+L LED_Short D33
 U 1 1 5B5F29B6
 P 11750 5750
-F 0 "D34" V 11796 5642 50  0000 R CNN
+F 0 "D33" V 11796 5642 50  0000 R CNN
 F 1 "LED" V 11705 5642 50  0000 R CNN
 F 2 "LEDs:LED_0603" H 11750 5750 50  0001 C CNN
@@
 $EndComp
 $Comp
-L R R243
+L R R216
 U 1 1 5B5F29BD
 P 11750 5400
-F 0 "R243" H 11820 5446 50  0000 L CNN
+F 0 "R216" H 11820 5446 50  0000 L CNN
 F 1 "4.7kΩ" H 11820 5355 50  0000 L CNN
 F 2 "Resistors_SMD:R_0603" V 11680 5400 50  0001 C CNN
@@
 $EndComp
 $Comp
-L R R241
+L R R214
 U 1 1 5B5F29C4
 P 10800 4750
-F 0 "R241" H 10870 4796 50  0000 L CNN
+F 0 "R214" H 10870 4796 50  0000 L CNN
 F 1 "4.7kΩ" H 10870 4705 50  0000 L CNN
 F 2 "Resistors_SMD:R_0603" V 10730 4750 50  0001 C CNN
@@
 $EndComp
 $Comp
-L R R242
+L R R215
 U 1 1 5B5F29CB
 P 10800 5150
-F 0 "R242" H 10870 5196 50  0000 L CNN
+F 0 "R215" H 10870 5196 50  0000 L CNN
 F 1 "4.7kΩ" H 10870 5105 50  0000 L CNN
 F 2 "Resistors_SMD:R_0603" V 10730 5150 50  0001 C CNN
@@
 $EndComp
 $Comp
-L R R240
+L R R213
 U 1 1 5B5F29D2
 P 10400 5950
-F 0 "R240" V 10300 5950 50  0000 C CNN
+F 0 "R213" V 10300 5950 50  0000 C CNN
 F 1 "4.7kΩ" V 10500 5950 50  0000 C CNN
 F 2 "Resistors_SMD:R_0603" V 10330 5950 50  0001 C CNN
@@
 $EndComp
 $Comp
-L R R244
+L R R217
 U 1 1 5B5F29D9
 P 12300 5600
-F 0 "R244" H 12370 5646 50  0000 L CNN
+F 0 "R217" H 12370 5646 50  0000 L CNN
 F 1 "4.7kΩ" H 12370 5555 50  0000 L CNN
 F 2 "Resistors_SMD:R_0603" V 12230 5600 50  0001 C CNN
@@
 $EndComp
 $Comp
-L C C220
+L C C195
 U 1 1 5B5F29E0
 P 12300 4850
-F 0 "C220" H 12415 4896 50  0000 L CNN
+F 0 "C195" H 12415 4896 50  0000 L CNN
 F 1 "4.7nF" H 12415 4805 50  0000 L CNN
 F 2 "Capacitors_SMD:C_0603" H 12338 4700 50  0001 C CNN
@@
 $EndComp
 $Comp
-L INDUCTOR_Small FB45
+L INDUCTOR_Small FB43
 U 1 1 5B5F2A0D
 P 11900 5200
-F 0 "FB45" V 12085 5200 50  0000 C CNN
+F 0 "FB43" V 12085 5200 50  0000 C CNN
 F 1 "CIM21J202NE" V 11994 5200 50  0000 C CNN
 F 2 "Resistors_SMD:R_0805" H 11900 5200 50  0001 C CNN

Commit message: More stepper motor driver progress
Parts:
- R206: renamed from R204; value 4.7kΩ -> 10kΩ
- R207: renamed from R205; value 4.7kΩ -> 10kΩ
- R212: renamed from R210; value 4.7kΩ -> 10kΩ
- R213: renamed from R211; value 4.7kΩ -> 10kΩ
- R218: renamed from R216; value 4.7kΩ -> 10kΩ
- R219: renamed from R217; value 4.7kΩ -> 10kΩ
- renumbered R200 to R202, R201 to R203, R202 to R204, R203 to R205, R206 to R208, R207 to R209, R208 to R210, R209 to R211, R212 to R214, R213 to R215, R214 to R216, R215 to R217
Changed lines of the file:
@@
 $Descr A3 16535 11693
 encoding utf-8
-Sheet 26 25
+Sheet 24 25
 Title ""
 Date ""
@@
 $EndComp
 $Comp
-L R R200
+L R R202
 U 1 1 5B5EFE68
 P 3700 5600
-F 0 "R200" V 3600 5600 50  0000 C CNN
+F 0 "R202" V 3600 5600 50  0000 C CNN
 F 1 "10Ω" V 3800 5600 50  0000 C CNN
 F 2 "Resistors_SMD:R_0603" V 3630 5600 50  0001 C CNN
@@
 $EndComp
 $Comp
-L R R204
+L R R206
 U 1 1 5B5EFE7E
 P 5150 5400
-F 0 "R204" H 5220 5446 50  0000 L CNN
-F 1 "4.7kΩ" H 5220 5355 50  0000 L CNN
+F 0 "R206" H 5220 5446 50  0000 L CNN
+F 1 "10kΩ" H 5220 5355 50  0000 L CNN
 F 2 "Resistors_SMD:R_0603" V 5080 5400 50  0001 C CNN
 F 3 "" H 5150 5400 50  0000 C CNN
@@
 $EndComp
 $Comp
-L R R202
+L R R204
 U 1 1 5B5EFE85
 P 4200 4750
-F 0 "R202" H 4270 4796 50  0000 L CNN
+F 0 "R204" H 4270 4796 50  0000 L CNN
 F 1 "4.7kΩ" H 4270 4705 50  0000 L CNN
 F 2 "Resistors_SMD:R_0603" V 4130 4750 50  0001 C CNN
@@
 $EndComp
 $Comp
-L R R203
+L R R205
 U 1 1 5B5EFE8C
 P 4200 5150
-F 0 "R203" H 4270 5196 50  0000 L CNN
+F 0 "R205" H 4270 5196 50  0000 L CNN
 F 1 "4.7kΩ" H 4270 5105 50  0000 L CNN
 F 2 "Resistors_SMD:R_0603" V 4130 5150 50  0001 C CNN
@@
 $EndComp
 $Comp
-L R R201
+L R R203
 U 1 1 5B5EFE93
 P 3800 5950
-F 0 "R201" V 3700 5950 50  0000 C CNN
+F 0 "R203" V 3700 5950 50  0000 C CNN
 F 1 "4.7kΩ" V 3900 5950 50  0000 C CNN
 F 2 "Resistors_SMD:R_0603" V 3730 5950 50  0001 C CNN
@@
 $EndComp
 $Comp
-L R R205
+L R R207
 U 1 1 5B5EFE9A
 P 5700 5600
-F 0 "R205" H 5770 5646 50  0000 L CNN
-F 1 "4.7kΩ" H 5770 5555 50  0000 L CNN
+F 0 "R207" H 5770 5646 50  0000 L CNN
+F 1 "10kΩ" H 5770 5555 50  0000 L CNN
 F 2 "Resistors_SMD:R_0603" V 5630 5600 50  0001 C CNN
 F 3 "" H 5700 5600 50  0000 C CNN
@@
 $EndComp
 $Comp
-L R R206
+L R R208
 U 1 1 5B5F23BD
 P 7000 5600
-F 0 "R206" V 6900 5600 50  0000 C CNN
+F 0 "R208" V 6900 5600 50  0000 C CNN
 F 1 "10Ω" V 7100 5600 50  0000 C CNN
 F 2 "Resistors_SMD:R_0603" V 6930 5600 50  0001 C CNN
@@
 $EndComp
 $Comp
-L R R210
+L R R212
 U 1 1 5B5F23D2
 P 8450 5400
-F 0 "R210" H 8520 5446 50  0000 L CNN
-F 1 "4.7kΩ" H 8520 5355 50  0000 L CNN
+F 0 "R212" H 8520 5446 50  0000 L CNN
+F 1 "10kΩ" H 8520 5355 50  0000 L CNN
 F 2 "Resistors_SMD:R_0603" V 8380 5400 50  0001 C CNN
 F 3 "" H 8450 5400 50  0000 C CNN
@@
 $EndComp
 $Comp
-L R R208
+L R R210
 U 1 1 5B5F23D9
 P 7500 4750
-F 0 "R208" H 7570 4796 50  0000 L CNN
+F 0 "R210" H 7570 4796 50  0000 L CNN
 F 1 "4.7kΩ" H 7570 4705 50  0000 L CNN
 F 2 "Resistors_SMD:R_0603" V 7430 4750 50  0001 C CNN
@@
 $EndComp
 $Comp
-L R R209
+L R R211
 U 1 1 5B5F23E0
 P 7500 5150
-F 0 "R209" H 7570 5196 50  0000 L CNN
+F 0 "R211" H 7570 5196 50  0000 L CNN
 F 1 "4.7kΩ" H 7570 5105 50  0000 L CNN
 F 2 "Resistors_SMD:R_0603" V 7430 5150 50  0001 C CNN
@@
 $EndComp
 $Comp
-L R R207
+L R R209
 U 1 1 5B5F23E7
 P 7100 5950
-F 0 "R207" V 7000 5950 50  0000 C CNN
+F 0 "R209" V 7000 5950 50  0000 C CNN
 F 1 "4.7kΩ" V 7200 5950 50  0000 C CNN
 F 2 "Resistors_SMD:R_0603" V 7030 5950 50  0001 C CNN
@@
 $EndComp
 $Comp
-L R R211
+L R R213
 U 1 1 5B5F23EE
 P 9000 5600
-F 0 "R211" H 9070 5646 50  0000 L CNN
-F 1 "4.7kΩ" H 9070 5555 50  0000 L CNN
+F 0 "R213" H 9070 5646 50  0000 L CNN
+F 1 "10kΩ" H 9070 5555 50  0000 L CNN
 F 2 "Resistors_SMD:R_0603" V 8930 5600 50  0001 C CNN
 F 3 "" H 9000 5600 50  0000 C CNN
@@
 $EndComp
 $Comp
-L R R212
+L R R214
 U 1 1 5B5F29A8
 P 10300 5600
-F 0 "R212" V 10200 5600 50  0000 C CNN
+F 0 "R214" V 10200 5600 50  0000 C CNN
 F 1 "10Ω" V 10400 5600 50  0000 C CNN
 F 2 "Resistors_SMD:R_0603" V 10230 5600 50  0001 C CNN
@@
 $EndComp
 $Comp
-L R R216
+L R R218
 U 1 1 5B5F29BD
 P 11750 5400
-F 0 "R216" H 11820 5446 50  0000 L CNN
-F 1 "4.7kΩ" H 11820 5355 50  0000 L CNN
+F 0 "R218" H 11820 5446 50  0000 L CNN
+F 1 "10kΩ" H 11820 5355 50  0000 L CNN
 F 2 "Resistors_SMD:R_0603" V 11680 5400 50  0001 C CNN
 F 3 "" H 11750 5400 50  0000 C CNN
@@
 $EndComp
 $Comp
-L R R214
+L R R216
 U 1 1 5B5F29C4
 P 10800 4750
-F 0 "R214" H 10870 4796 50  0000 L CNN
+F 0 "R216" H 10870 4796 50  0000 L CNN
 F 1 "4.7kΩ" H 10870 4705 50  0000 L CNN
 F 2 "Resistors_SMD:R_0603" V 10730 4750 50  0001 C CNN
@@
 $EndComp
 $Comp
-L R R215
+L R R217
 U 1 1 5B5F29CB
 P 10800 5150
-F 0 "R215" H 10870 5196 50  0000 L CNN
+F 0 "R217" H 10870 5196 50  0000 L CNN
 F 1 "4.7kΩ" H 10870 5105 50  0000 L CNN
 F 2 "Resistors_SMD:R_0603" V 10730 5150 50  0001 C CNN
@@
 $EndComp
 $Comp
-L R R213
+L R R215
 U 1 1 5B5F29D2
 P 10400 5950
-F 0 "R213" V 10300 5950 50  0000 C CNN
+F 0 "R215" V 10300 5950 50  0000 C CNN
 F 1 "4.7kΩ" V 10500 5950 50  0000 C CNN
 F 2 "Resistors_SMD:R_0603" V 10330 5950 50  0001 C CNN
@@
 $EndComp
 $Comp
-L R R217
+L R R219
 U 1 1 5B5F29D9
 P 12300 5600
-F 0 "R217" H 12370 5646 50  0000 L CNN
-F 1 "4.7kΩ" H 12370 5555 50  0000 L CNN
+F 0 "R219" H 12370 5646 50  0000 L CNN
+F 1 "10kΩ" H 12370 5555 50  0000 L CNN
 F 2 "Resistors_SMD:R_0603" V 12230 5600 50  0001 C CNN
 F 3 "" H 12300 5600 50  0000 C CNN
