File: KiMBo/z0_stepper.sch (KiCad schematic (older format))
At the start: 25 parts, among them U20 TMC2130

Commit message: Assocate more footprints
Parts:
- C117, C118: footprint Capacitors_SMD:C_0402 -> Capacitors_SMD:C_0603
- R146, R147, R148, R149, R150, R151: footprint (none) -> Resistors_SMD:R_0603
Changed lines of the file:
@@
 F 0 "C118" H 8865 4246 50  0000 L CNN
 F 1 "22nF" H 8865 4155 50  0000 L CNN
-F 2 "Capacitors_SMD:C_0402" H 8788 4050 50  0001 C CNN
+F 2 "Capacitors_SMD:C_0603" H 8788 4050 50  0001 C CNN
 F 3 "" H 8750 4200 50  0000 C CNN
 	1    8750 4200
@@
 F 0 "R149" V 6800 3800 50  0000 C CNN
 F 1 "2.2Ω" V 6900 3800 50  0000 C CNN
-F 2 "" V 6830 3800 50  0001 C CNN
+F 2 "Resistors_SMD:R_0603" V 6830 3800 50  0001 C CNN
 F 3 "" H 6900 3800 50  0000 C CNN
 	1    6900 3800
@@
 F 0 "R147" H 5719 4346 50  0000 L CNN
 F 1 "4.7kΩ" H 5719 4255 50  0000 L CNN
-F 2 "" V 5580 4300 50  0001 C CNN
+F 2 "Resistors_SMD:R_0603" V 5580 4300 50  0001 C CNN
 F 3 "" H 5650 4300 50  0000 C CNN
 	1    5650 4300
@@
 F 0 "C117" H 7150 4100 50  0000 L CNN
 F 1 "4.7μF" H 7150 3900 50  0000 L CNN
-F 2 "Capacitors_SMD:C_0402" H 7138 3850 50  0001 C CNN
+F 2 "Capacitors_SMD:C_0603" H 7138 3850 50  0001 C CNN
 F 3 "" H 7100 4000 50  0000 C CNN
 	1    7100 4000
@@
 F 0 "R150" H 8919 6796 50  0000 L CNN
 F 1 "5.23kΩ" H 8919 6705 50  0000 L CNN
-F 2 "" V 8780 6750 50  0001 C CNN
+F 2 "Resistors_SMD:R_0603" V 8780 6750 50  0001 C CNN
 F 3 "" H 8850 6750 50  0000 C CNN
 	1    8850 6750
@@
 F 0 "R151" V 8850 6950 50  0000 C CNN
 F 1 "4.75kΩ" V 8950 6950 50  0000 C CNN
-F 2 "" V 8980 6950 50  0001 C CNN
+F 2 "Resistors_SMD:R_0603" V 8980 6950 50  0001 C CNN
 F 3 "" H 9050 6950 50  0000 C CNN
 	1    9050 6950
@@
 F 0 "R148" H 6069 4346 50  0000 L CNN
 F 1 "4.7kΩ" H 6069 4255 50  0000 L CNN
-F 2 "" V 5930 4300 50  0001 C CNN
+F 2 "Resistors_SMD:R_0603" V 5930 4300 50  0001 C CNN
 F 3 "" H 6000 4300 50  0000 C CNN
 	1    6000 4300
@@
 F 0 "R146" H 5369 4346 50  0000 L CNN
 F 1 "4.7kΩ" H 5369 4255 50  0000 L CNN
-F 2 "" V 5230 4300 50  0001 C CNN
+F 2 "Resistors_SMD:R_0603" V 5230 4300 50  0001 C CNN
 F 3 "" H 5300 4300 50  0000 C CNN
 	1    5300 4300

Commit message: More footprint association
Parts:
- R152, R153: footprint (none) -> Resistors_SMD:R_0805
- U20: footprint (none) -> KiMBo:QFN36_5X6
Changed lines of the file:
@@
 $EndComp
 $Comp
-L GND #PWR0210
+L GND #PWR0211
 U 1 1 58C0C3E5
 P 7100 3350
-F 0 "#PWR0210" H 7100 3100 50  0001 C CNN
+F 0 "#PWR0211" H 7100 3100 50  0001 C CNN
 F 1 "GND" H 7100 3200 50  0000 C CNN
 F 2 "" H 7100 3350 50  0000 C CNN
@@
 $EndComp
 $Comp
-L GND #PWR0211
+L GND #PWR0212
 U 1 1 58C0C3F2
 P 9950 3400
-F 0 "#PWR0211" H 9950 3150 50  0001 C CNN
+F 0 "#PWR0212" H 9950 3150 50  0001 C CNN
 F 1 "GND" H 9955 3227 50  0000 C CNN
 F 2 "" H 9950 3400 50  0000 C CNN
@@
 $EndComp
 $Comp
-L +24V #PWR0212
+L +24V #PWR0213
 U 1 1 58C0C3F8
 P 8150 2900
-F 0 "#PWR0212" H 8150 2750 50  0001 C CNN
+F 0 "#PWR0213" H 8150 2750 50  0001 C CNN
 F 1 "+24V" H 8165 3073 50  0000 C CNN
 F 2 "" H 8150 2900 50  0000 C CNN
@@
 F 0 "R153" H 10300 6700 50  0000 R CNN
 F 1 "220mΩ" H 10300 6800 50  0000 R CNN
-F 2 "" V 10280 6750 50  0001 C CNN
+F 2 "Resistors_SMD:R_0805" V 10280 6750 50  0001 C CNN
 F 3 "" H 10350 6750 50  0000 C CNN
 	1    10350 6750
@@
 F 0 "R152" H 9500 6700 50  0000 R CNN
 F 1 "220mΩ" H 9500 6800 50  0000 R CNN
-F 2 "" V 9480 6750 50  0001 C CNN
+F 2 "Resistors_SMD:R_0805" V 9480 6750 50  0001 C CNN
 F 3 "" H 9550 6750 50  0000 C CNN
 	1    9550 6750
@@
 $EndComp
 $Comp
-L GND #PWR0213
+L GND #PWR0214
 U 1 1 58C0C413
 P 9250 7100
-F 0 "#PWR0213" H 9250 6850 50  0001 C CNN
+F 0 "#PWR0214" H 9250 6850 50  0001 C CNN
 F 1 "GND" H 9255 6927 50  0000 C CNN
 F 2 "" H 9250 7100 50  0000 C CNN
@@
 NoConn ~ 7300 5750
 $Comp
-L GND #PWR0214
+L GND #PWR0215
 U 1 1 58C0C436
 P 7250 6150
-F 0 "#PWR0214" H 7250 5900 50  0001 C CNN
+F 0 "#PWR0215" H 7250 5900 50  0001 C CNN
 F 1 "GND" H 7255 5977 50  0000 C CNN
 F 2 "" H 7250 6150 50  0000 C CNN
@@
 $EndComp
 $Comp
-L GND #PWR0215
+L GND #PWR0216
 U 1 1 58C0C47A
 P 8850 5250
-F 0 "#PWR0215" H 8850 5000 50  0001 C CNN
+F 0 "#PWR0216" H 8850 5000 50  0001 C CNN
 F 1 "GND" H 8850 5100 50  0000 C CNN
 F 2 "" H 8850 5250 50  0000 C CNN
@@
 $EndComp
 $Comp
-L GND #PWR0216
+L GND #PWR0217
 U 1 1 58C0C48E
 P 8850 6100
-F 0 "#PWR0216" H 8850 5850 50  0001 C CNN
+F 0 "#PWR0217" H 8850 5850 50  0001 C CNN
 F 1 "GND" H 8850 5950 50  0000 C CNN
 F 2 "" H 8850 6100 50  0000 C CNN
@@
 F 0 "U20" H 7550 6250 60  0000 C CNN
 F 1 "TMC2130" H 8300 6250 60  0000 C CNN
-F 2 "" H 8000 5050 60  0001 C CNN
+F 2 "KiMBo:QFN36_5X6" H 8000 5050 60  0001 C CNN
 F 3 "" H 8000 5050 60  0000 C CNN
 	1    8000 4750
@@
 	5300 3550 7300 3550
 $Comp
-L VDD_3V3B #PWR0217
+L VDD_3V3B #PWR0218
 U 1 1 5A313878
 P 6350 3500
-F 0 "#PWR0217" H 6350 3350 50  0001 C CNN
+F 0 "#PWR0218" H 6350 3350 50  0001 C CNN
 F 1 "VDD_3V3B" H 6365 3673 50  0000 C CNN
 F 2 "" H 6350 3500 50  0000 C CNN

Commit message: Add more footprints and more associations, one association left!
Parts:
- R160: renamed from R151; footprint Resistors_SMD:R_0603 -> Resistors_SMD:R_0805
- R162: renamed from R153; footprint Resistors_SMD:R_0805 -> Resistors_SMD:R_0603
- renumbered R146 to R155, R147 to R156, R148 to R157, R149 to R158, R150 to R159, R152 to R161
Changed lines of the file:
@@
 $EndComp
 $Comp
-L GND #PWR0211
+L GND #PWR0213
 U 1 1 58C0C3E5
 P 7100 3350
-F 0 "#PWR0211" H 7100 3100 50  0001 C CNN
+F 0 "#PWR0213" H 7100 3100 50  0001 C CNN
 F 1 "GND" H 7100 3200 50  0000 C CNN
 F 2 "" H 7100 3350 50  0000 C CNN
@@
 $EndComp
 $Comp
-L GND #PWR0212
+L GND #PWR0214
 U 1 1 58C0C3F2
 P 9950 3400
-F 0 "#PWR0212" H 9950 3150 50  0001 C CNN
+F 0 "#PWR0214" H 9950 3150 50  0001 C CNN
 F 1 "GND" H 9955 3227 50  0000 C CNN
 F 2 "" H 9950 3400 50  0000 C CNN
@@
 $EndComp
 $Comp
-L +24V #PWR0213
+L +24V #PWR0215
 U 1 1 58C0C3F8
 P 8150 2900
-F 0 "#PWR0213" H 8150 2750 50  0001 C CNN
+F 0 "#PWR0215" H 8150 2750 50  0001 C CNN
 F 1 "+24V" H 8165 3073 50  0000 C CNN
 F 2 "" H 8150 2900 50  0000 C CNN
@@
 $EndComp
 $Comp
-L R R153
+L R R162
 U 1 1 58C0C405
 P 10350 6750
-F 0 "R153" H 10300 6700 50  0000 R CNN
+F 0 "R162" H 10300 6700 50  0000 R CNN
 F 1 "220mΩ" H 10300 6800 50  0000 R CNN
-F 2 "Resistors_SMD:R_0805" V 10280 6750 50  0001 C CNN
+F 2 "Resistors_SMD:R_0603" V 10280 6750 50  0001 C CNN
 F 3 "" H 10350 6750 50  0000 C CNN
 	1    10350 6750
@@
 $EndComp
 $Comp
-L R R152
+L R R161
 U 1 1 58C0C40C
 P 9550 6750
-F 0 "R152" H 9500 6700 50  0000 R CNN
+F 0 "R161" H 9500 6700 50  0000 R CNN
 F 1 "220mΩ" H 9500 6800 50  0000 R CNN
 F 2 "Resistors_SMD:R_0805" V 9480 6750 50  0001 C CNN
@@
 $EndComp
 $Comp
-L GND #PWR0214
+L GND #PWR0216
 U 1 1 58C0C413
 P 9250 7100
-F 0 "#PWR0214" H 9250 6850 50  0001 C CNN
+F 0 "#PWR0216" H 9250 6850 50  0001 C CNN
 F 1 "GND" H 9255 6927 50  0000 C CNN
 F 2 "" H 9250 7100 50  0000 C CNN
@@
 NoConn ~ 7300 5650
 $Comp
-L R R149
+L R R158
 U 1 1 58C0C41A
 P 6900 3800
-F 0 "R149" V 6800 3800 50  0000 C CNN
+F 0 "R158" V 6800 3800 50  0000 C CNN
 F 1 "2.2Ω" V 6900 3800 50  0000 C CNN
 F 2 "Resistors_SMD:R_0603" V 6830 3800 50  0001 C CNN
@@
 NoConn ~ 7300 5750
 $Comp
-L GND #PWR0215
+L GND #PWR0217
 U 1 1 58C0C436
 P 7250 6150
-F 0 "#PWR0215" H 7250 5900 50  0001 C CNN
+F 0 "#PWR0217" H 7250 5900 50  0001 C CNN
 F 1 "GND" H 7255 5977 50  0000 C CNN
 F 2 "" H 7250 6150 50  0000 C CNN
@@
 Z0_FAULT
 $Comp
-L R R147
+L R R156
 U 1 1 58C0C444
 P 5650 4300
-F 0 "R147" H 5719 4346 50  0000 L CNN
+F 0 "R156" H 5719 4346 50  0000 L CNN
 F 1 "4.7kΩ" H 5719 4255 50  0000 L CNN
 F 2 "Resistors_SMD:R_0603" V 5580 4300 50  0001 C CNN
@@
 5VOUT
 $Comp
-L R R150
+L R R159
 U 1 1 58C0C456
 P 8850 6750
-F 0 "R150" H 8919 6796 50  0000 L CNN
+F 0 "R159" H 8919 6796 50  0000 L CNN
 F 1 "5.23kΩ" H 8919 6705 50  0000 L CNN
 F 2 "Resistors_SMD:R_0603" V 8780 6750 50  0001 C CNN
@@
 5VOUT
 $Comp
-L R R151
+L R R160
 U 1 1 58C0C45E
 P 9050 6950
-F 0 "R151" V 8850 6950 50  0000 C CNN
+F 0 "R160" V 8850 6950 50  0000 C CNN
 F 1 "4.75kΩ" V 8950 6950 50  0000 C CNN
-F 2 "Resistors_SMD:R_0603" V 8980 6950 50  0001 C CNN
+F 2 "Resistors_SMD:R_0805" V 8980 6950 50  0001 C CNN
 F 3 "" H 9050 6950 50  0000 C CNN
 	1    9050 6950
@@
 $EndComp
 $Comp
-L R R148
+L R R157
 U 1 1 58C0C465
 P 6000 4300
-F 0 "R148" H 6069 4346 50  0000 L CNN
+F 0 "R157" H 6069 4346 50  0000 L CNN
 F 1 "4.7kΩ" H 6069 4255 50  0000 L CNN
 F 2 "Resistors_SMD:R_0603" V 5930 4300 50  0001 C CNN
@@
 $EndComp
 $Comp
-L GND #PWR0216
+L GND #PWR0218
 U 1 1 58C0C47A
 P 8850 5250
-F 0 "#PWR0216" H 8850 5000 50  0001 C CNN
+F 0 "#PWR0218" H 8850 5000 50  0001 C CNN
 F 1 "GND" H 8850 5100 50  0000 C CNN
 F 2 "" H 8850 5250 50  0000 C CNN
@@
 $EndComp
 $Comp
-L GND #PWR0217
+L GND #PWR0219
 U 1 1 58C0C48E
 P 8850 6100
-F 0 "#PWR0217" H 8850 5850 50  0001 C CNN
+F 0 "#PWR0219" H 8850 5850 50  0001 C CNN
 F 1 "GND" H 8850 5950 50  0000 C CNN
 F 2 "" H 8850 6100 50  0000 C CNN
@@
 	8750 6050 8750 6000
 $Comp
-L R R146
+L R R155
 U 1 1 58C0C50F
 P 5300 4300
-F 0 "R146" H 5369 4346 50  0000 L CNN
+F 0 "R155" H 5369 4346 50  0000 L CNN
 F 1 "4.7kΩ" H 5369 4255 50  0000 L CNN
 F 2 "Resistors_SMD:R_0603" V 5230 4300 50  0001 C CNN
@@
 	5300 3550 7300 3550
 $Comp
-L VDD_3V3B #PWR0218
+L VDD_3V3B #PWR0220
 U 1 1 5A313878
 P 6350 3500
-F 0 "#PWR0218" H 6350 3350 50  0001 C CNN
+F 0 "#PWR0220" H 6350 3350 50  0001 C CNN
 F 1 "VDD_3V3B" H 6365 3673 50  0000 C CNN
 F 2 "" H 6350 3500 50  0000 C CNN

Commit message: Begin layout
Arrange all connectors to get a feel for the area.
Parts:
- renumbered C114 to C116, C115 to C117, C116 to C118, C117 to C119, C118 to C120, C119 to C121, C120 to C122, C121 to C123, C122 to C124, C123 to C125, C124 to C126, C125 to C127, C126 to C128, C127 to C129, C128 to C130, C129 to C131
Changed lines of the file:
@@
 Z0_SG
 $Comp
-L C C116
+L C C118
 U 1 1 58C0C3C9
 P 7100 3150
-F 0 "C116" H 6986 3104 50  0000 R CNN
+F 0 "C118" H 6986 3104 50  0000 R CNN
 F 1 "100nF" H 6986 3195 50  0000 R CNN
 F 2 "Capacitors_SMD:C_0603" H 7138 3000 50  0001 C CNN
@@
 $EndComp
 $Comp
-L C C121
+L C C123
 U 1 1 58C0C3D0
 P 8900 3700
-F 0 "C121" V 8850 3600 50  0000 C CNN
+F 0 "C123" V 8850 3600 50  0000 C CNN
 F 1 "100nF" V 8850 3875 50  0000 C CNN
 F 2 "Capacitors_SMD:C_0603" H 8938 3550 50  0001 C CNN
@@
 $EndComp
 $Comp
-L CP1 C128
+L CP1 C130
 U 1 1 58C0C3D7
 P 10250 3150
-F 0 "C128" H 10350 3250 50  0000 C CNN
+F 0 "C130" H 10350 3250 50  0000 C CNN
 F 1 "100μF" H 10400 3050 50  0000 C CNN
 F 2 "Capacitors_SMD:c_elec_8x10" H 10250 3150 50  0001 C CNN
@@
 $EndComp
 $Comp
-L C C124
+L C C126
 U 1 1 58C0C3DE
 P 9350 3150
-F 0 "C124" H 9250 3250 50  0000 C CNN
+F 0 "C126" H 9250 3250 50  0000 C CNN
 F 1 "100nF" H 9225 3050 50  0000 C CNN
 F 2 "Capacitors_SMD:C_0603" H 9388 3000 50  0001 C CNN
@@
 $EndComp
 $Comp
-L GND #PWR0213
+L GND #PWR0216
 U 1 1 58C0C3E5
 P 7100 3350
-F 0 "#PWR0213" H 7100 3100 50  0001 C CNN
+F 0 "#PWR0216" H 7100 3100 50  0001 C CNN
 F 1 "GND" H 7100 3200 50  0000 C CNN
 F 2 "" H 7100 3350 50  0000 C CNN
@@
 $EndComp
 $Comp
-L C C125
+L C C127
 U 1 1 58C0C3EB
 P 9650 3150
-F 0 "C125" H 9550 3250 50  0000 C CNN
+F 0 "C127" H 9550 3250 50  0000 C CNN
 F 1 "100nF" H 9525 3050 50  0000 C CNN
 F 2 "Capacitors_SMD:C_0603" H 9688 3000 50  0001 C CNN
@@
 $EndComp
 $Comp
-L GND #PWR0214
+L GND #PWR0217
 U 1 1 58C0C3F2
 P 9950 3400
-F 0 "#PWR0214" H 9950 3150 50  0001 C CNN
+F 0 "#PWR0217" H 9950 3150 50  0001 C CNN
 F 1 "GND" H 9955 3227 50  0000 C CNN
 F 2 "" H 9950 3400 50  0000 C CNN
@@
 $EndComp
 $Comp
-L +24V #PWR0215
+L +24V #PWR0218
 U 1 1 58C0C3F8
 P 8150 2900
-F 0 "#PWR0215" H 8150 2750 50  0001 C CNN
+F 0 "#PWR0218" H 8150 2750 50  0001 C CNN
 F 1 "+24V" H 8165 3073 50  0000 C CNN
 F 2 "" H 8150 2900 50  0000 C CNN
@@
 $EndComp
 $Comp
-L C C118
+L C C120
 U 1 1 58C0C3FE
 P 8750 4200
-F 0 "C118" H 8865 4246 50  0000 L CNN
+F 0 "C120" H 8865 4246 50  0000 L CNN
 F 1 "22nF" H 8865 4155 50  0000 L CNN
 F 2 "Capacitors_SMD:C_0603" H 8788 4050 50  0001 C CNN
@@
 $EndComp
 $Comp
-L GND #PWR0216
+L GND #PWR0219
 U 1 1 58C0C413
 P 9250 7100
-F 0 "#PWR0216" H 9250 6850 50  0001 C CNN
+F 0 "#PWR0219" H 9250 6850 50  0001 C CNN
 F 1 "GND" H 9255 6927 50  0000 C CNN
 F 2 "" H 9250 7100 50  0000 C CNN
@@
 $EndComp
 $Comp
-L C C115
+L C C117
 U 1 1 58C0C421
 P 6700 4000
-F 0 "C115" H 6750 4100 50  0000 L CNN
+F 0 "C117" H 6750 4100 50  0000 L CNN
 F 1 "470nF" H 6725 3900 50  0000 L CNN
 F 2 "Capacitors_SMD:C_0603" H 6738 3850 50  0001 C CNN
@@
 NoConn ~ 7300 5750
 $Comp
-L GND #PWR0217
+L GND #PWR0220
 U 1 1 58C0C436
 P 7250 6150
-F 0 "#PWR0217" H 7250 5900 50  0001 C CNN
+F 0 "#PWR0220" H 7250 5900 50  0001 C CNN
 F 1 "GND" H 7255 5977 50  0000 C CNN
 F 2 "" H 7250 6150 50  0000 C CNN
@@
 $EndComp
 $Comp
-L C C126
+L C C128
 U 1 1 58C0C43C
 P 9700 6750
-F 0 "C126" H 9750 6850 50  0000 L CNN
+F 0 "C128" H 9750 6850 50  0000 L CNN
 F 1 "100nF" H 9750 6650 50  0000 L CNN
 F 2 "Capacitors_SMD:C_0603" H 9738 6600 50  0001 C CNN
@@
 NoConn ~ 7300 4600
 $Comp
-L C C117
+L C C119
 U 1 1 58C0C44E
 P 7100 4000
-F 0 "C117" H 7150 4100 50  0000 L CNN
+F 0 "C119" H 7150 4100 50  0000 L CNN
 F 1 "4.7μF" H 7150 3900 50  0000 L CNN
 F 2 "Capacitors_SMD:C_0603" H 7138 3850 50  0001 C CNN
@@
 $EndComp
 $Comp
-L C C129
+L C C131
 U 1 1 58C0C46C
 P 10500 6750
-F 0 "C129" H 10550 6850 50  0000 L CNN
+F 0 "C131" H 10550 6850 50  0000 L CNN
 F 1 "100nF" H 10550 6650 50  0000 L CNN
 F 2 "Capacitors_SMD:C_0603" H 10538 6600 50  0001 C CNN
@@
 $EndComp
 $Comp
-L C C119
+L C C121
 U 1 1 58C0C473
 P 8750 5000
-F 0 "C119" H 8775 5100 50  0000 L CNN
+F 0 "C121" H 8775 5100 50  0000 L CNN
 F 1 "470pF" H 8750 4900 50  0000 L CNN
 F 2 "Capacitors_SMD:C_0603" H 8788 4850 50  0001 C CNN
@@
 $EndComp
 $Comp
-L GND #PWR0218
+L GND #PWR0221
 U 1 1 58C0C47A
 P 8850 5250
-F 0 "#PWR0218" H 8850 5000 50  0001 C CNN
+F 0 "#PWR0221" H 8850 5000 50  0001 C CNN
 F 1 "GND" H 8850 5100 50  0000 C CNN
 F 2 "" H 8850 5250 50  0000 C CNN
@@
 $EndComp
 $Comp
-L C C122
+L C C124
 U 1 1 58C0C480
 P 8950 5000
-F 0 "C122" H 8975 5100 50  0000 L CNN
+F 0 "C124" H 8975 5100 50  0000 L CNN
 F 1 "470pF" H 8975 4900 50  0000 L CNN
 F 2 "Capacitors_SMD:C_0603" H 8988 4850 50  0001 C CNN
@@
 $EndComp
 $Comp
-L C C120
+L C C122
 U 1 1 58C0C487
 P 8750 5850
-F 0 "C120" H 8775 5950 50  0000 L CNN
+F 0 "C122" H 8775 5950 50  0000 L CNN
 F 1 "470pF" H 8750 5750 50  0000 L CNN
 F 2 "Capacitors_SMD:C_0603" H 8788 5700 50  0001 C CNN
@@
 $EndComp
 $Comp
-L GND #PWR0219
+L GND #PWR0222
 U 1 1 58C0C48E
 P 8850 6100
-F 0 "#PWR0219" H 8850 5850 50  0001 C CNN
+F 0 "#PWR0222" H 8850 5850 50  0001 C CNN
 F 1 "GND" H 8850 5950 50  0000 C CNN
 F 2 "" H 8850 6100 50  0000 C CNN
@@
 $EndComp
 $Comp
-L C C123
+L C C125
 U 1 1 58C0C494
 P 8950 5850
-F 0 "C123" H 8975 5950 50  0000 L CNN
+F 0 "C125" H 8975 5950 50  0000 L CNN
 F 1 "470pF" H 8975 5750 50  0000 L CNN
 F 2 "Capacitors_SMD:C_0603" H 8988 5700 50  0001 C CNN
@@
 Connection ~ 5650 3550
 $Comp
-L C C127
+L C C129
 U 1 1 58C0C51A
 P 9950 3150
-F 0 "C127" H 9850 3250 50  0000 C CNN
+F 0 "C129" H 9850 3250 50  0000 C CNN
 F 1 "10μF" H 9825 3050 50  0000 C CNN
 F 2 "Capacitors_SMD:C_0805" H 9988 3000 50  0001 C CNN
@@
 	5300 3550 7300 3550
 $Comp
-L VDD_3V3B #PWR0220
+L VDD_3V3B #PWR0223
 U 1 1 5A313878
 P 6350 3500
-F 0 "#PWR0220" H 6350 3350 50  0001 C CNN
+F 0 "#PWR0223" H 6350 3350 50  0001 C CNN
 F 1 "VDD_3V3B" H 6365 3673 50  0000 C CNN
 F 2 "" H 6350 3500 50  0000 C CNN
@@
 $EndComp
 $Comp
-L C C114
+L C C116
 U 1 1 5A89B9DA
 P 6350 4000
-F 0 "C114" H 6400 4100 50  0000 L CNN
+F 0 "C116" H 6400 4100 50  0000 L CNN
 F 1 "100nF" H 6375 3900 50  0000 L CNN
 F 2 "Capacitors_SMD:C_0603" H 6388 3850 50  0001 C CNN

Commit message: Arrange connectors and E-stepper circuit
Parts:
- R160: footprint Resistors_SMD:R_0805 -> Resistors_SMD:R_0603
- R162: footprint Resistors_SMD:R_0603 -> Resistors_SMD:R_0805
Changed lines of the file:
@@
 F 0 "R162" H 10300 6700 50  0000 R CNN
 F 1 "220mΩ" H 10300 6800 50  0000 R CNN
-F 2 "Resistors_SMD:R_0603" V 10280 6750 50  0001 C CNN
+F 2 "Resistors_SMD:R_0805" V 10280 6750 50  0001 C CNN
 F 3 "" H 10350 6750 50  0000 C CNN
 	1    10350 6750
@@
 F 0 "R160" V 8850 6950 50  0000 C CNN
 F 1 "4.75kΩ" V 8950 6950 50  0000 C CNN
-F 2 "Resistors_SMD:R_0805" V 8980 6950 50  0001 C CNN
+F 2 "Resistors_SMD:R_0603" V 8980 6950 50  0001 C CNN
 F 3 "" H 9050 6950 50  0000 C CNN
 	1    9050 6950
