File: KiMBo/z0_stepper.sch (KiCad schematic (older format))
At the start: 25 parts, among them U20 TMC2130

Commit message: Remove HDMI from the schematic
Parts:
- renumbered C125 to C100, C126 to C101, C127 to C102, C128 to C103, C129 to C104, C130 to C105, C131 to C106, C116 to C91, C117 to C92, C118 to C93, C119 to C94, C120 to C95, C121 to C96, C122 to C97, C123 to C98, C124 to C99, R155 to R128, R156 to R129, R157 to R130, R158 to R131, R159 to R132, R160 to R133, R161 to R134, R162 to R135, U20 to U16
Changed lines of the file:
@@
 $Descr A3 16535 11693
 encoding utf-8
-Sheet 18 26
+Sheet 18 25
 Title ""
 Date ""
@@
 Z0_SG
 $Comp
-L C C118
+L C C93
 U 1 1 58C0C3C9
 P 7100 3150
-F 0 "C118" H 6986 3104 50  0000 R CNN
+F 0 "C93" H 6986 3104 50  0000 R CNN
 F 1 "100nF" H 6986 3195 50  0000 R CNN
 F 2 "Capacitors_SMD:C_0603" H 7138 3000 50  0001 C CNN
@@
 $EndComp
 $Comp
-L C C123
+L C C98
 U 1 1 58C0C3D0
 P 8900 3700
-F 0 "C123" V 8850 3600 50  0000 C CNN
+F 0 "C98" V 8850 3600 50  0000 C CNN
 F 1 "100nF" V 8850 3875 50  0000 C CNN
 F 2 "Capacitors_SMD:C_0603" H 8938 3550 50  0001 C CNN
@@
 $EndComp
 $Comp
-L CP1 C130
+L CP1 C105
 U 1 1 58C0C3D7
 P 10250 3150
-F 0 "C130" H 10350 3250 50  0000 C CNN
+F 0 "C105" H 10350 3250 50  0000 C CNN
 F 1 "100μF" H 10400 3050 50  0000 C CNN
 F 2 "Capacitors_SMD:c_elec_8x10" H 10250 3150 50  0001 C CNN
@@
 $EndComp
 $Comp
-L C C126
+L C C101
 U 1 1 58C0C3DE
 P 9350 3150
-F 0 "C126" H 9250 3250 50  0000 C CNN
+F 0 "C101" H 9250 3250 50  0000 C CNN
 F 1 "100nF" H 9225 3050 50  0000 C CNN
 F 2 "Capacitors_SMD:C_0603" H 9388 3000 50  0001 C CNN
@@
 $EndComp
 $Comp
-L GND #PWR0216
+L GND #PWR0185
 U 1 1 58C0C3E5
 P 7100 3350
-F 0 "#PWR0216" H 7100 3100 50  0001 C CNN
+F 0 "#PWR0185" H 7100 3100 50  0001 C CNN
 F 1 "GND" H 7100 3200 50  0000 C CNN
 F 2 "" H 7100 3350 50  0000 C CNN
@@
 $EndComp
 $Comp
-L C C127
+L C C102
 U 1 1 58C0C3EB
 P 9650 3150
-F 0 "C127" H 9550 3250 50  0000 C CNN
+F 0 "C102" H 9550 3250 50  0000 C CNN
 F 1 "100nF" H 9525 3050 50  0000 C CNN
 F 2 "Capacitors_SMD:C_0603" H 9688 3000 50  0001 C CNN
@@
 $EndComp
 $Comp
-L GND #PWR0217
+L GND #PWR0186
 U 1 1 58C0C3F2
 P 9950 3400
-F 0 "#PWR0217" H 9950 3150 50  0001 C CNN
+F 0 "#PWR0186" H 9950 3150 50  0001 C CNN
 F 1 "GND" H 9955 3227 50  0000 C CNN
 F 2 "" H 9950 3400 50  0000 C CNN
@@
 $EndComp
 $Comp
-L +24V #PWR0218
+L +24V #PWR0187
 U 1 1 58C0C3F8
 P 8150 2900
-F 0 "#PWR0218" H 8150 2750 50  0001 C CNN
+F 0 "#PWR0187" H 8150 2750 50  0001 C CNN
 F 1 "+24V" H 8165 3073 50  0000 C CNN
 F 2 "" H 8150 2900 50  0000 C CNN
@@
 $EndComp
 $Comp
-L C C120
+L C C95
 U 1 1 58C0C3FE
 P 8750 4200
-F 0 "C120" H 8865 4246 50  0000 L CNN
+F 0 "C95" H 8865 4246 50  0000 L CNN
 F 1 "22nF" H 8865 4155 50  0000 L CNN
 F 2 "Capacitors_SMD:C_0603" H 8788 4050 50  0001 C CNN
@@
 $EndComp
 $Comp
-L R R162
+L R R135
 U 1 1 58C0C405
 P 10350 6750
-F 0 "R162" H 10300 6700 50  0000 R CNN
+F 0 "R135" H 10300 6700 50  0000 R CNN
 F 1 "220mΩ" H 10300 6800 50  0000 R CNN
 F 2 "Resistors_SMD:R_0805" V 10280 6750 50  0001 C CNN
@@
 $EndComp
 $Comp
-L R R161
+L R R134
 U 1 1 58C0C40C
 P 9550 6750
-F 0 "R161" H 9500 6700 50  0000 R CNN
+F 0 "R134" H 9500 6700 50  0000 R CNN
 F 1 "220mΩ" H 9500 6800 50  0000 R CNN
 F 2 "Resistors_SMD:R_0805" V 9480 6750 50  0001 C CNN
@@
 $EndComp
 $Comp
-L GND #PWR0219
+L GND #PWR0188
 U 1 1 58C0C413
 P 9250 7100
-F 0 "#PWR0219" H 9250 6850 50  0001 C CNN
+F 0 "#PWR0188" H 9250 6850 50  0001 C CNN
 F 1 "GND" H 9255 6927 50  0000 C CNN
 F 2 "" H 9250 7100 50  0000 C CNN
@@
 NoConn ~ 7300 5650
 $Comp
-L R R158
+L R R131
 U 1 1 58C0C41A
 P 6900 3800
-F 0 "R158" V 6800 3800 50  0000 C CNN
+F 0 "R131" V 6800 3800 50  0000 C CNN
 F 1 "2.2Ω" V 6900 3800 50  0000 C CNN
 F 2 "Resistors_SMD:R_0603" V 6830 3800 50  0001 C CNN
@@
 $EndComp
 $Comp
-L C C117
+L C C92
 U 1 1 58C0C421
 P 6700 4000
-F 0 "C117" H 6750 4100 50  0000 L CNN
+F 0 "C92" H 6750 4100 50  0000 L CNN
 F 1 "470nF" H 6725 3900 50  0000 L CNN
 F 2 "Capacitors_SMD:C_0603" H 6738 3850 50  0001 C CNN
@@
 NoConn ~ 7300 5750
 $Comp
-L GND #PWR0220
+L GND #PWR0189
 U 1 1 58C0C436
 P 7250 6150
-F 0 "#PWR0220" H 7250 5900 50  0001 C CNN
+F 0 "#PWR0189" H 7250 5900 50  0001 C CNN
 F 1 "GND" H 7255 5977 50  0000 C CNN
 F 2 "" H 7250 6150 50  0000 C CNN
@@
 $EndComp
 $Comp
-L C C128
+L C C103
 U 1 1 58C0C43C
 P 9700 6750
-F 0 "C128" H 9750 6850 50  0000 L CNN
+F 0 "C103" H 9750 6850 50  0000 L CNN
 F 1 "100nF" H 9750 6650 50  0000 L CNN
 F 2 "Capacitors_SMD:C_0603" H 9738 6600 50  0001 C CNN
@@
 Z0_FAULT
 $Comp
-L R R156
+L R R129
 U 1 1 58C0C444
 P 5650 4300
-F 0 "R156" H 5719 4346 50  0000 L CNN
+F 0 "R129" H 5719 4346 50  0000 L CNN
 F 1 "4.7kΩ" H 5719 4255 50  0000 L CNN
 F 2 "Resistors_SMD:R_0603" V 5580 4300 50  0001 C CNN
@@
 NoConn ~ 7300 4600
 $Comp
-L C C119
+L C C94
 U 1 1 58C0C44E
 P 7100 4000
-F 0 "C119" H 7150 4100 50  0000 L CNN
+F 0 "C94" H 7150 4100 50  0000 L CNN
 F 1 "4.7μF" H 7150 3900 50  0000 L CNN
 F 2 "Capacitors_SMD:C_0603" H 7138 3850 50  0001 C CNN
@@
 5VOUT
 $Comp
-L R R159
+L R R132
 U 1 1 58C0C456
 P 8850 6750
-F 0 "R159" H 8919 6796 50  0000 L CNN
+F 0 "R132" H 8919 6796 50  0000 L CNN
 F 1 "5.23kΩ" H 8919 6705 50  0000 L CNN
 F 2 "Resistors_SMD:R_0603" V 8780 6750 50  0001 C CNN
@@
 5VOUT
 $Comp
-L R R160
+L R R133
 U 1 1 58C0C45E
 P 9050 6950
-F 0 "R160" V 8850 6950 50  0000 C CNN
+F 0 "R133" V 8850 6950 50  0000 C CNN
 F 1 "4.75kΩ" V 8950 6950 50  0000 C CNN
 F 2 "Resistors_SMD:R_0603" V 8980 6950 50  0001 C CNN
@@
 $EndComp
 $Comp
-L R R157
+L R R130
 U 1 1 58C0C465
 P 6000 4300
-F 0 "R157" H 6069 4346 50  0000 L CNN
+F 0 "R130" H 6069 4346 50  0000 L CNN
 F 1 "4.7kΩ" H 6069 4255 50  0000 L CNN
 F 2 "Resistors_SMD:R_0603" V 5930 4300 50  0001 C CNN
@@
 $EndComp
 $Comp
-L C C131
+L C C106
 U 1 1 58C0C46C
 P 10500 6750
-F 0 "C131" H 10550 6850 50  0000 L CNN
+F 0 "C106" H 10550 6850 50  0000 L CNN
 F 1 "100nF" H 10550 6650 50  0000 L CNN
 F 2 "Capacitors_SMD:C_0603" H 10538 6600 50  0001 C CNN
@@
 $EndComp
 $Comp
-L C C121
+L C C96
 U 1 1 58C0C473
 P 8750 5000
-F 0 "C121" H 8775 5100 50  0000 L CNN
+F 0 "C96" H 8775 5100 50  0000 L CNN
 F 1 "470pF" H 8750 4900 50  0000 L CNN
 F 2 "Capacitors_SMD:C_0603" H 8788 4850 50  0001 C CNN
@@
 $EndComp
 $Comp
-L GND #PWR0221
+L GND #PWR0190
 U 1 1 58C0C47A
 P 8850 5250
-F 0 "#PWR0221" H 8850 5000 50  0001 C CNN
+F 0 "#PWR0190" H 8850 5000 50  0001 C CNN
 F 1 "GND" H 8850 5100 50  0000 C CNN
 F 2 "" H 8850 5250 50  0000 C CNN
@@
 $EndComp
 $Comp
-L C C124
+L C C99
 U 1 1 58C0C480
 P 8950 5000
-F 0 "C124" H 8975 5100 50  0000 L CNN
+F 0 "C99" H 8975 5100 50  0000 L CNN
 F 1 "470pF" H 8975 4900 50  0000 L CNN
 F 2 "Capacitors_SMD:C_0603" H 8988 4850 50  0001 C CNN
@@
 $EndComp
 $Comp
-L C C122
+L C C97
 U 1 1 58C0C487
 P 8750 5850
-F 0 "C122" H 8775 5950 50  0000 L CNN
+F 0 "C97" H 8775 5950 50  0000 L CNN
 F 1 "470pF" H 8750 5750 50  0000 L CNN
 F 2 "Capacitors_SMD:C_0603" H 8788 5700 50  0001 C CNN
@@
 $EndComp
 $Comp
-L GND #PWR0222
+L GND #PWR0191
 U 1 1 58C0C48E
 P 8850 6100
-F 0 "#PWR0222" H 8850 5850 50  0001 C CNN
+F 0 "#PWR0191" H 8850 5850 50  0001 C CNN
 F 1 "GND" H 8850 5950 50  0000 C CNN
 F 2 "" H 8850 6100 50  0000 C CNN
@@
 $EndComp
 $Comp
-L C C125
+L C C100
 U 1 1 58C0C494
 P 8950 5850
-F 0 "C125" H 8975 5950 50  0000 L CNN
+F 0 "C100" H 8975 5950 50  0000 L CNN
 F 1 "470pF" H 8975 5750 50  0000 L CNN
 F 2 "Capacitors_SMD:C_0603" H 8988 5700 50  0001 C CNN
@@
 $EndComp
 $Comp
-L TMC2130 U20
+L TMC2130 U16
 U 1 1 58C0C49B
 P 8000 4750
-F 0 "U20" H 7550 6250 60  0000 C CNN
+F 0 "U16" H 7550 6250 60  0000 C CNN
 F 1 "TMC2130" H 8300 6250 60  0000 C CNN
 F 2 "KiMBo:QFN36_5X6" H 8000 5050 60  0001 C CNN
@@
 	8750 6050 8750 6000
 $Comp
-L R R155
+L R R128
 U 1 1 58C0C50F
 P 5300 4300
-F 0 "R155" H 5369 4346 50  0000 L CNN
+F 0 "R128" H 5369 4346 50  0000 L CNN
 F 1 "4.7kΩ" H 5369 4255 50  0000 L CNN
 F 2 "Resistors_SMD:R_0603" V 5230 4300 50  0001 C CNN
@@
 Connection ~ 5650 3550
 $Comp
-L C C129
+L C C104
 U 1 1 58C0C51A
 P 9950 3150
-F 0 "C129" H 9850 3250 50  0000 C CNN
+F 0 "C104" H 9850 3250 50  0000 C CNN
 F 1 "10μF" H 9825 3050 50  0000 C CNN
 F 2 "Capacitors_SMD:C_0805" H 9988 3000 50  0001 C CNN
@@
 	5300 3550 7300 3550
 $Comp
-L VDD_3V3B #PWR0223
+L VDD_3V3B #PWR0192
 U 1 1 5A313878
 P 6350 3500
-F 0 "#PWR0223" H 6350 3350 50  0001 C CNN
+F 0 "#PWR0192" H 6350 3350 50  0001 C CNN
 F 1 "VDD_3V3B" H 6365 3673 50  0000 C CNN
 F 2 "" H 6350 3500 50  0000 C CNN
@@
 $EndComp
 $Comp
-L C C116
+L C C91
 U 1 1 5A89B9DA
 P 6350 4000
-F 0 "C116" H 6400 4100 50  0000 L CNN
+F 0 "C91" H 6400 4100 50  0000 L CNN
 F 1 "100nF" H 6375 3900 50  0000 L CNN
 F 2 "Capacitors_SMD:C_0603" H 6388 3850 50  0001 C CNN

Commit message: More stepper motor driver progress
Parts:
- renumbered R128 to R130, R129 to R131, R130 to R132, R131 to R133, R132 to R134, R133 to R135, R134 to R136, R135 to R137
Changed lines of the file:
@@
 $Descr A3 16535 11693
 encoding utf-8
-Sheet 18 25
+Sheet 16 25
 Title ""
 Date ""
@@
 $EndComp
 $Comp
-L R R135
+L R R137
 U 1 1 58C0C405
 P 10350 6750
-F 0 "R135" H 10300 6700 50  0000 R CNN
+F 0 "R137" H 10300 6700 50  0000 R CNN
 F 1 "220mΩ" H 10300 6800 50  0000 R CNN
 F 2 "Resistors_SMD:R_0805" V 10280 6750 50  0001 C CNN
@@
 $EndComp
 $Comp
-L R R134
+L R R136
 U 1 1 58C0C40C
 P 9550 6750
-F 0 "R134" H 9500 6700 50  0000 R CNN
+F 0 "R136" H 9500 6700 50  0000 R CNN
 F 1 "220mΩ" H 9500 6800 50  0000 R CNN
 F 2 "Resistors_SMD:R_0805" V 9480 6750 50  0001 C CNN
@@
 NoConn ~ 7300 5650
 $Comp
-L R R131
+L R R133
 U 1 1 58C0C41A
 P 6900 3800
-F 0 "R131" V 6800 3800 50  0000 C CNN
+F 0 "R133" V 6800 3800 50  0000 C CNN
 F 1 "2.2Ω" V 6900 3800 50  0000 C CNN
 F 2 "Resistors_SMD:R_0603" V 6830 3800 50  0001 C CNN
@@
 Z0_FAULT
 $Comp
-L R R129
+L R R131
 U 1 1 58C0C444
 P 5650 4300
-F 0 "R129" H 5719 4346 50  0000 L CNN
+F 0 "R131" H 5719 4346 50  0000 L CNN
 F 1 "4.7kΩ" H 5719 4255 50  0000 L CNN
 F 2 "Resistors_SMD:R_0603" V 5580 4300 50  0001 C CNN
@@
 5VOUT
 $Comp
-L R R132
+L R R134
 U 1 1 58C0C456
 P 8850 6750
-F 0 "R132" H 8919 6796 50  0000 L CNN
+F 0 "R134" H 8919 6796 50  0000 L CNN
 F 1 "5.23kΩ" H 8919 6705 50  0000 L CNN
 F 2 "Resistors_SMD:R_0603" V 8780 6750 50  0001 C CNN
@@
 5VOUT
 $Comp
-L R R133
+L R R135
 U 1 1 58C0C45E
 P 9050 6950
-F 0 "R133" V 8850 6950 50  0000 C CNN
+F 0 "R135" V 8850 6950 50  0000 C CNN
 F 1 "4.75kΩ" V 8950 6950 50  0000 C CNN
 F 2 "Resistors_SMD:R_0603" V 8980 6950 50  0001 C CNN
@@
 $EndComp
 $Comp
-L R R130
+L R R132
 U 1 1 58C0C465
 P 6000 4300
-F 0 "R130" H 6069 4346 50  0000 L CNN
+F 0 "R132" H 6069 4346 50  0000 L CNN
 F 1 "4.7kΩ" H 6069 4255 50  0000 L CNN
 F 2 "Resistors_SMD:R_0603" V 5930 4300 50  0001 C CNN
@@
 	8750 6050 8750 6000
 $Comp
-L R R128
+L R R130
 U 1 1 58C0C50F
 P 5300 4300
-F 0 "R128" H 5369 4346 50  0000 L CNN
+F 0 "R130" H 5369 4346 50  0000 L CNN
 F 1 "4.7kΩ" H 5369 4255 50  0000 L CNN
 F 2 "Resistors_SMD:R_0603" V 5230 4300 50  0001 C CNN

Commit message: Daisy chain the SPI stepper motor driver interface, continue work on the E-heater layout
Parts:
- renumbered C102 to C100, C103 to C101, C104 to C102, C105 to C103, C106 to C104, C91 to C89, C92 to C90, C93 to C91, C94 to C92, C95 to C93, C96 to C94, C97 to C95, C98 to C96, C99 to C97, C100 to C98, C101 to C99, U16 to U15
Changed lines of the file:
@@
 Z0_SG
 $Comp
-L C C93
+L C C91
 U 1 1 58C0C3C9
 P 7100 3150
-F 0 "C93" H 6986 3104 50  0000 R CNN
+F 0 "C91" H 6986 3104 50  0000 R CNN
 F 1 "100nF" H 6986 3195 50  0000 R CNN
 F 2 "Capacitors_SMD:C_0603" H 7138 3000 50  0001 C CNN
@@
 $EndComp
 $Comp
-L C C98
+L C C96
 U 1 1 58C0C3D0
 P 8900 3700
-F 0 "C98" V 8850 3600 50  0000 C CNN
+F 0 "C96" V 8850 3600 50  0000 C CNN
 F 1 "100nF" V 8850 3875 50  0000 C CNN
 F 2 "Capacitors_SMD:C_0603" H 8938 3550 50  0001 C CNN
@@
 $EndComp
 $Comp
-L CP1 C105
+L CP1 C103
 U 1 1 58C0C3D7
 P 10250 3150
-F 0 "C105" H 10350 3250 50  0000 C CNN
+F 0 "C103" H 10350 3250 50  0000 C CNN
 F 1 "100μF" H 10400 3050 50  0000 C CNN
 F 2 "Capacitors_SMD:c_elec_8x10" H 10250 3150 50  0001 C CNN
@@
 $EndComp
 $Comp
-L C C101
+L C C99
 U 1 1 58C0C3DE
 P 9350 3150
-F 0 "C101" H 9250 3250 50  0000 C CNN
+F 0 "C99" H 9250 3250 50  0000 C CNN
 F 1 "100nF" H 9225 3050 50  0000 C CNN
 F 2 "Capacitors_SMD:C_0603" H 9388 3000 50  0001 C CNN
@@
 $EndComp
 $Comp
-L GND #PWR0185
+L GND #PWR165
 U 1 1 58C0C3E5
 P 7100 3350
-F 0 "#PWR0185" H 7100 3100 50  0001 C CNN
+F 0 "#PWR165" H 7100 3100 50  0001 C CNN
 F 1 "GND" H 7100 3200 50  0000 C CNN
 F 2 "" H 7100 3350 50  0000 C CNN
@@
 $EndComp
 $Comp
-L C C102
+L C C100
 U 1 1 58C0C3EB
 P 9650 3150
-F 0 "C102" H 9550 3250 50  0000 C CNN
+F 0 "C100" H 9550 3250 50  0000 C CNN
 F 1 "100nF" H 9525 3050 50  0000 C CNN
 F 2 "Capacitors_SMD:C_0603" H 9688 3000 50  0001 C CNN
@@
 $EndComp
 $Comp
-L GND #PWR0186
+L GND #PWR171
 U 1 1 58C0C3F2
 P 9950 3400
-F 0 "#PWR0186" H 9950 3150 50  0001 C CNN
+F 0 "#PWR171" H 9950 3150 50  0001 C CNN
 F 1 "GND" H 9955 3227 50  0000 C CNN
 F 2 "" H 9950 3400 50  0000 C CNN
@@
 $EndComp
 $Comp
-L +24V #PWR0187
+L +24V #PWR167
 U 1 1 58C0C3F8
 P 8150 2900
-F 0 "#PWR0187" H 8150 2750 50  0001 C CNN
+F 0 "#PWR167" H 8150 2750 50  0001 C CNN
 F 1 "+24V" H 8165 3073 50  0000 C CNN
 F 2 "" H 8150 2900 50  0000 C CNN
@@
 $EndComp
 $Comp
-L C C95
+L C C93
 U 1 1 58C0C3FE
 P 8750 4200
-F 0 "C95" H 8865 4246 50  0000 L CNN
+F 0 "C93" H 8865 4246 50  0000 L CNN
 F 1 "22nF" H 8865 4155 50  0000 L CNN
 F 2 "Capacitors_SMD:C_0603" H 8788 4050 50  0001 C CNN
@@
 $EndComp
 $Comp
-L GND #PWR0188
+L GND #PWR170
 U 1 1 58C0C413
 P 9250 7100
-F 0 "#PWR0188" H 9250 6850 50  0001 C CNN
+F 0 "#PWR170" H 9250 6850 50  0001 C CNN
 F 1 "GND" H 9255 6927 50  0000 C CNN
 F 2 "" H 9250 7100 50  0000 C CNN
@@
 $EndComp
 $Comp
-L C C92
+L C C90
 U 1 1 58C0C421
 P 6700 4000
-F 0 "C92" H 6750 4100 50  0000 L CNN
+F 0 "C90" H 6750 4100 50  0000 L CNN
 F 1 "470nF" H 6725 3900 50  0000 L CNN
 F 2 "Capacitors_SMD:C_0603" H 6738 3850 50  0001 C CNN
@@
 NoConn ~ 7300 5750
 $Comp
-L GND #PWR0189
+L GND #PWR166
 U 1 1 58C0C436
 P 7250 6150
-F 0 "#PWR0189" H 7250 5900 50  0001 C CNN
+F 0 "#PWR166" H 7250 5900 50  0001 C CNN
 F 1 "GND" H 7255 5977 50  0000 C CNN
 F 2 "" H 7250 6150 50  0000 C CNN
@@
 $EndComp
 $Comp
-L C C103
+L C C101
 U 1 1 58C0C43C
 P 9700 6750
-F 0 "C103" H 9750 6850 50  0000 L CNN
+F 0 "C101" H 9750 6850 50  0000 L CNN
 F 1 "100nF" H 9750 6650 50  0000 L CNN
 F 2 "Capacitors_SMD:C_0603" H 9738 6600 50  0001 C CNN
@@
 NoConn ~ 7300 4600
 $Comp
-L C C94
+L C C92
 U 1 1 58C0C44E
 P 7100 4000
-F 0 "C94" H 7150 4100 50  0000 L CNN
+F 0 "C92" H 7150 4100 50  0000 L CNN
 F 1 "4.7μF" H 7150 3900 50  0000 L CNN
 F 2 "Capacitors_SMD:C_0603" H 7138 3850 50  0001 C CNN
@@
 $EndComp
 $Comp
-L C C106
+L C C104
 U 1 1 58C0C46C
 P 10500 6750
-F 0 "C106" H 10550 6850 50  0000 L CNN
+F 0 "C104" H 10550 6850 50  0000 L CNN
 F 1 "100nF" H 10550 6650 50  0000 L CNN
 F 2 "Capacitors_SMD:C_0603" H 10538 6600 50  0001 C CNN
@@
 $EndComp
 $Comp
-L C C96
+L C C94
 U 1 1 58C0C473
 P 8750 5000
-F 0 "C96" H 8775 5100 50  0000 L CNN
+F 0 "C94" H 8775 5100 50  0000 L CNN
 F 1 "470pF" H 8750 4900 50  0000 L CNN
 F 2 "Capacitors_SMD:C_0603" H 8788 4850 50  0001 C CNN
@@
 $EndComp
 $Comp
-L GND #PWR0190
+L GND #PWR168
 U 1 1 58C0C47A
 P 8850 5250
-F 0 "#PWR0190" H 8850 5000 50  0001 C CNN
+F 0 "#PWR168" H 8850 5000 50  0001 C CNN
 F 1 "GND" H 8850 5100 50  0000 C CNN
 F 2 "" H 8850 5250 50  0000 C CNN
@@
 $EndComp
 $Comp
-L C C99
+L C C97
 U 1 1 58C0C480
 P 8950 5000
-F 0 "C99" H 8975 5100 50  0000 L CNN
+F 0 "C97" H 8975 5100 50  0000 L CNN
 F 1 "470pF" H 8975 4900 50  0000 L CNN
 F 2 "Capacitors_SMD:C_0603" H 8988 4850 50  0001 C CNN
@@
 $EndComp
 $Comp
-L C C97
+L C C95
 U 1 1 58C0C487
 P 8750 5850
-F 0 "C97" H 8775 5950 50  0000 L CNN
+F 0 "C95" H 8775 5950 50  0000 L CNN
 F 1 "470pF" H 8750 5750 50  0000 L CNN
 F 2 "Capacitors_SMD:C_0603" H 8788 5700 50  0001 C CNN
@@
 $EndComp
 $Comp
-L GND #PWR0191
+L GND #PWR169
 U 1 1 58C0C48E
 P 8850 6100
-F 0 "#PWR0191" H 8850 5850 50  0001 C CNN
+F 0 "#PWR169" H 8850 5850 50  0001 C CNN
 F 1 "GND" H 8850 5950 50  0000 C CNN
 F 2 "" H 8850 6100 50  0000 C CNN
@@
 $EndComp
 $Comp
-L C C100
+L C C98
 U 1 1 58C0C494
 P 8950 5850
-F 0 "C100" H 8975 5950 50  0000 L CNN
+F 0 "C98" H 8975 5950 50  0000 L CNN
 F 1 "470pF" H 8975 5750 50  0000 L CNN
 F 2 "Capacitors_SMD:C_0603" H 8988 5700 50  0001 C CNN
@@
 $EndComp
 $Comp
-L TMC2130 U16
+L TMC2130 U15
 U 1 1 58C0C49B
 P 8000 4750
-F 0 "U16" H 7550 6250 60  0000 C CNN
+F 0 "U15" H 7550 6250 60  0000 C CNN
 F 1 "TMC2130" H 8300 6250 60  0000 C CNN
 F 2 "KiMBo:QFN36_5X6" H 8000 5050 60  0001 C CNN
@@
 Connection ~ 5650 3550
 $Comp
-L C C104
+L C C102
 U 1 1 58C0C51A
 P 9950 3150
-F 0 "C104" H 9850 3250 50  0000 C CNN
+F 0 "C102" H 9850 3250 50  0000 C CNN
 F 1 "10μF" H 9825 3050 50  0000 C CNN
 F 2 "Capacitors_SMD:C_0805" H 9988 3000 50  0001 C CNN
@@
 	5300 3550 7300 3550
 $Comp
-L VDD_3V3B #PWR0192
+L VDD_3V3B #PWR164
 U 1 1 5A313878
 P 6350 3500
-F 0 "#PWR0192" H 6350 3350 50  0001 C CNN
+F 0 "#PWR164" H 6350 3350 50  0001 C CNN
 F 1 "VDD_3V3B" H 6365 3673 50  0000 C CNN
 F 2 "" H 6350 3500 50  0000 C CNN
@@
 $EndComp
 $Comp
-L C C91
+L C C89
 U 1 1 5A89B9DA
 P 6350 4000
-F 0 "C91" H 6400 4100 50  0000 L CNN
+F 0 "C89" H 6400 4100 50  0000 L CNN
 F 1 "100nF" H 6375 3900 50  0000 L CNN
 F 2 "Capacitors_SMD:C_0603" H 6388 3850 50  0001 C CNN
