File: KiMBo/eth.sch (KiCad schematic (older format))
At the start: 45 parts, among them U1 OSD3358, U11 LAN8710A, Y1 7A-25.000MAAJ-T

Commit message: Create more footprints and add more associations
Parts:
- U11: footprint (none) -> Housings_DFN_QFN:QFN-32-1EP_5x5mm_Pitch0.5mm
- Y1: footprint (none) -> KiMBo:Crystal_SMD_7A_2Pads
Changed lines of the file:
@@
 F 0 "U11" H 6450 5400 60  0000 C CNN
 F 1 "LAN8710A" H 7750 5400 60  0000 C CNN
-F 2 "" H 7450 4250 60  0001 C CNN
+F 2 "Housings_DFN_QFN:QFN-32-1EP_5x5mm_Pitch0.5mm" H 7450 4250 60  0001 C CNN
 F 3 "" H 7450 4250 60  0001 C CNN
 	1    7200 4150
@@
 F 0 "Y1" H 5200 5868 50  0000 C CNN
 F 1 "7A-25.000MAAJ-T" H 5350 5750 50  0000 C CNN
-F 2 "" H 5200 5600 50  0001 C CNN
+F 2 "KiMBo:Crystal_SMD_7A_2Pads" H 5200 5600 50  0001 C CNN
 F 3 "" H 5200 5600 50  0000 C CNN
 	1    5200 5600

Commit message: Complete footprint association
Next step is layout, adjustments may need to be made to the schematic at a later point.
Parts:
- C35, C36, C37, C38: footprint (none) -> Capacitors_SMD:C_0603
- R55, R56, R68: footprint (none) -> Resistors_SMD:R_0603
Changed lines of the file:
@@
 F 0 "R55" V 5100 5050 50  0000 C CNN
 F 1 "DNP-1MΩ" V 5300 5050 50  0000 C CNN
-F 2 "" V 5130 5050 50  0001 C CNN
+F 2 "Resistors_SMD:R_0603" V 5130 5050 50  0001 C CNN
 F 3 "" H 5200 5050 50  0000 C CNN
 	1    5200 5050
@@
 F 0 "C35" H 8350 3750 50  0000 L CNN
 F 1 "DNP-15pF" H 8350 3550 50  0000 L CNN
-F 2 "" H 8388 3500 50  0001 C CNN
+F 2 "Capacitors_SMD:C_0603" H 8388 3500 50  0001 C CNN
 F 3 "" H 8350 3650 50  0000 C CNN
 	1    8350 3650
@@
 F 0 "C36" H 8550 3750 50  0000 L CNN
 F 1 "DNP-15pF" H 8550 3475 50  0000 L CNN
-F 2 "" H 8588 3500 50  0001 C CNN
+F 2 "Capacitors_SMD:C_0603" H 8588 3500 50  0001 C CNN
 F 3 "" H 8550 3650 50  0000 C CNN
 	1    8550 3650
@@
 F 0 "C37" H 8750 3750 50  0000 L CNN
 F 1 "DNP-15pF" H 8750 3550 50  0000 L CNN
-F 2 "" H 8788 3500 50  0001 C CNN
+F 2 "Capacitors_SMD:C_0603" H 8788 3500 50  0001 C CNN
 F 3 "" H 8750 3650 50  0000 C CNN
 	1    8750 3650
@@
 F 0 "C38" H 8950 3750 50  0000 L CNN
 F 1 "DNP-15pF" H 8950 3475 50  0000 L CNN
-F 2 "" H 8988 3500 50  0001 C CNN
+F 2 "Capacitors_SMD:C_0603" H 8988 3500 50  0001 C CNN
 F 3 "" H 8950 3650 50  0000 C CNN
 	1    8950 3650
@@
 F 0 "R56" V 5043 2950 50  0000 C CNN
 F 1 "DNP-10Ω" V 5134 2950 50  0000 C CNN
-F 2 "" V 5180 2950 50  0001 C CNN
+F 2 "Resistors_SMD:R_0603" V 5180 2950 50  0001 C CNN
 F 3 "" H 5250 2950 50  0000 C CNN
 	1    5250 2950
@@
 F 0 "R68" V 5750 4800 50  0000 C CNN
 F 1 "DNP-0Ω" V 5925 4800 50  0000 C CNN
-F 2 "" V 5780 4800 50  0001 C CNN
+F 2 "Resistors_SMD:R_0603" V 5780 4800 50  0001 C CNN
 F 3 "" H 5850 4800 50  0000 C CNN
 	1    5850 4800

Commit message: Begin layout
Arrange all connectors to get a feel for the area.
Parts:
- renumbered C27 to C29, C28 to C30, C29 to C31, C30 to C32, C31 to C33, C32 to C34, C33 to C35, C34 to C36, C35 to C37, C36 to C38, C37 to C39, C38 to C40
Changed lines of the file:
@@
 $EndComp
 $Comp
-L C C27
+L C C29
 U 1 1 589D3894
 P 4950 5800
-F 0 "C27" H 5064 5846 50  0000 L CNN
+F 0 "C29" H 5064 5846 50  0000 L CNN
 F 1 "30pF" H 5064 5755 50  0000 L CNN
 F 2 "Capacitors_SMD:C_0603" H 4988 5650 50  0001 C CNN
@@
 $EndComp
 $Comp
-L C C28
+L C C30
 U 1 1 589D38D5
 P 5450 5800
-F 0 "C28" H 5565 5846 50  0000 L CNN
+F 0 "C30" H 5565 5846 50  0000 L CNN
 F 1 "30pF" H 5565 5755 50  0000 L CNN
 F 2 "Capacitors_SMD:C_0603" H 5488 5650 50  0001 C CNN
@@
 $EndComp
 $Comp
-L GND #PWR0121
+L GND #PWR0124
 U 1 1 589D3921
 P 4950 6000
-F 0 "#PWR0121" H 4950 5750 50  0001 C CNN
+F 0 "#PWR0124" H 4950 5750 50  0001 C CNN
 F 1 "GND" H 4955 5827 50  0000 C CNN
 F 2 "" H 4950 6000 50  0000 C CNN
@@
 $EndComp
 $Comp
-L GND #PWR0122
+L GND #PWR0125
 U 1 1 589D3945
 P 5450 6000
-F 0 "#PWR0122" H 5450 5750 50  0001 C CNN
+F 0 "#PWR0125" H 5450 5750 50  0001 C CNN
 F 1 "GND" H 5455 5827 50  0000 C CNN
 F 2 "" H 5450 6000 50  0000 C CNN
@@
 $EndComp
 $Comp
-L C C35
+L C C37
 U 1 1 589EEF58
 P 8350 3650
-F 0 "C35" H 8350 3750 50  0000 L CNN
+F 0 "C37" H 8350 3750 50  0000 L CNN
 F 1 "DNP-15pF" H 8350 3550 50  0000 L CNN
 F 2 "Capacitors_SMD:C_0603" H 8388 3500 50  0001 C CNN
@@
 $EndComp
 $Comp
-L C C36
+L C C38
 U 1 1 589EEFBF
 P 8550 3650
-F 0 "C36" H 8550 3750 50  0000 L CNN
+F 0 "C38" H 8550 3750 50  0000 L CNN
 F 1 "DNP-15pF" H 8550 3475 50  0000 L CNN
 F 2 "Capacitors_SMD:C_0603" H 8588 3500 50  0001 C CNN
@@
 $EndComp
 $Comp
-L C C37
+L C C39
 U 1 1 589EF023
 P 8750 3650
-F 0 "C37" H 8750 3750 50  0000 L CNN
+F 0 "C39" H 8750 3750 50  0000 L CNN
 F 1 "DNP-15pF" H 8750 3550 50  0000 L CNN
 F 2 "Capacitors_SMD:C_0603" H 8788 3500 50  0001 C CNN
@@
 $EndComp
 $Comp
-L C C38
+L C C40
 U 1 1 589EF088
 P 8950 3650
-F 0 "C38" H 8950 3750 50  0000 L CNN
+F 0 "C40" H 8950 3750 50  0000 L CNN
 F 1 "DNP-15pF" H 8950 3475 50  0000 L CNN
 F 2 "Capacitors_SMD:C_0603" H 8988 3500 50  0001 C CNN
@@
 $EndComp
 $Comp
-L GND #PWR0123
+L GND #PWR0126
 U 1 1 589EF9C7
 P 8350 3850
-F 0 "#PWR0123" H 8350 3600 50  0001 C CNN
+F 0 "#PWR0126" H 8350 3600 50  0001 C CNN
 F 1 "GND" H 8355 3677 50  0000 C CNN
 F 2 "" H 8350 3850 50  0000 C CNN
@@
 $EndComp
 $Comp
-L GND #PWR0124
+L GND #PWR0127
 U 1 1 589EFA2D
 P 8550 3850
-F 0 "#PWR0124" H 8550 3600 50  0001 C CNN
+F 0 "#PWR0127" H 8550 3600 50  0001 C CNN
 F 1 "GND" H 8555 3677 50  0000 C CNN
 F 2 "" H 8550 3850 50  0000 C CNN
@@
 $EndComp
 $Comp
-L GND #PWR0125
+L GND #PWR0128
 U 1 1 589EFA8C
 P 8750 3850
-F 0 "#PWR0125" H 8750 3600 50  0001 C CNN
+F 0 "#PWR0128" H 8750 3600 50  0001 C CNN
 F 1 "GND" H 8755 3677 50  0000 C CNN
 F 2 "" H 8750 3850 50  0000 C CNN
@@
 $EndComp
 $Comp
-L GND #PWR0126
+L GND #PWR0129
 U 1 1 589EFAEB
 P 8950 3850
-F 0 "#PWR0126" H 8950 3600 50  0001 C CNN
+F 0 "#PWR0129" H 8950 3600 50  0001 C CNN
 F 1 "GND" H 8955 3677 50  0000 C CNN
 F 2 "" H 8950 3850 50  0000 C CNN
@@
 $EndComp
 $Comp
-L GND #PWR0127
+L GND #PWR0130
 U 1 1 589F5496
 P 7200 5600
-F 0 "#PWR0127" H 7200 5350 50  0001 C CNN
+F 0 "#PWR0130" H 7200 5350 50  0001 C CNN
 F 1 "GND" H 7205 5427 50  0000 C CNN
 F 2 "" H 7200 5600 50  0000 C CNN
@@
 $EndComp
 $Comp
-L GND #PWR0128
+L GND #PWR0131
 U 1 1 589F6033
 P 8450 5600
-F 0 "#PWR0128" H 8450 5350 50  0001 C CNN
+F 0 "#PWR0131" H 8450 5350 50  0001 C CNN
 F 1 "GND" H 8455 5427 50  0000 C CNN
 F 2 "" H 8450 5600 50  0000 C CNN
@@
 $EndComp
 $Comp
-L GND #PWR0129
+L GND #PWR0132
 U 1 1 589F60CA
 P 8700 5600
-F 0 "#PWR0129" H 8700 5350 50  0001 C CNN
+F 0 "#PWR0132" H 8700 5350 50  0001 C CNN
 F 1 "GND" H 8705 5427 50  0000 C CNN
 F 2 "" H 8700 5600 50  0000 C CNN
@@
 $EndComp
 $Comp
-L C C29
+L C C31
 U 1 1 589FB905
 P 5900 2650
-F 0 "C29" H 6015 2696 50  0000 L CNN
+F 0 "C31" H 6015 2696 50  0000 L CNN
 F 1 "100nF" H 6015 2605 50  0000 L CNN
 F 2 "Capacitors_SMD:C_0603" H 5938 2500 50  0001 C CNN
@@
 $EndComp
 $Comp
-L GND #PWR0130
+L GND #PWR0133
 U 1 1 589FBD44
 P 5900 2850
-F 0 "#PWR0130" H 5900 2600 50  0001 C CNN
+F 0 "#PWR0133" H 5900 2600 50  0001 C CNN
 F 1 "GND" H 5905 2677 50  0000 C CNN
 F 2 "" H 5900 2850 50  0000 C CNN
@@
 $EndComp
 $Comp
-L C C30
+L C C32
 U 1 1 589FC806
 P 7500 1750
-F 0 "C30" H 7500 1850 50  0000 L CNN
+F 0 "C32" H 7500 1850 50  0000 L CNN
 F 1 "100nF" H 7500 1650 50  0000 L CNN
 F 2 "Capacitors_SMD:C_0603" H 7538 1600 50  0001 C CNN
@@
 $EndComp
 $Comp
-L GND #PWR0131
+L GND #PWR0134
 U 1 1 589FC878
 P 7500 1950
-F 0 "#PWR0131" H 7500 1700 50  0001 C CNN
+F 0 "#PWR0134" H 7500 1700 50  0001 C CNN
 F 1 "GND" H 7505 1777 50  0000 C CNN
 F 2 "" H 7500 1950 50  0000 C CNN
@@
 $EndComp
 $Comp
-L C C32
+L C C34
 U 1 1 589FC986
 P 7700 2450
-F 0 "C32" H 7750 2550 50  0000 L CNN
+F 0 "C34" H 7750 2550 50  0000 L CNN
 F 1 "470pF" H 7700 2350 50  0000 L CNN
 F 2 "Capacitors_SMD:C_0603" H 7738 2300 50  0001 C CNN
@@
 $EndComp
 $Comp
-L C C34
+L C C36
 U 1 1 589FCA4C
 P 7900 2450
-F 0 "C34" H 8015 2496 50  0000 L CNN
+F 0 "C36" H 8015 2496 50  0000 L CNN
 F 1 "1μF" H 8015 2405 50  0000 L CNN
 F 2 "Capacitors_SMD:C_0603" H 7938 2300 50  0001 C CNN
@@
 $EndComp
 $Comp
-L GND #PWR0132
+L GND #PWR0135
 U 1 1 589FCD92
 P 7800 2700
-F 0 "#PWR0132" H 7800 2450 50  0001 C CNN
+F 0 "#PWR0135" H 7800 2450 50  0001 C CNN
 F 1 "GND" H 7900 2600 50  0000 C CNN
 F 2 "" H 7800 2700 50  0000 C CNN
@@
 $EndComp
 $Comp
-L C C31
+L C C33
 U 1 1 589FE02F
 P 7700 1750
-F 0 "C31" H 7700 1850 50  0000 L CNN
+F 0 "C33" H 7700 1850 50  0000 L CNN
 F 1 "100nF" H 7700 1650 50  0000 L CNN
 F 2 "Capacitors_SMD:C_0603" H 7738 1600 50  0001 C CNN
@@
 $EndComp
 $Comp
-L C C33
+L C C35
 U 1 1 589FE0C1
 P 7900 1750
-F 0 "C33" H 7900 1850 50  0000 L CNN
+F 0 "C35" H 7900 1850 50  0000 L CNN
 F 1 "10μF" H 7900 1650 50  0000 L CNN
 F 2 "Capacitors_SMD:C_0805" H 7938 1600 50  0001 C CNN
@@
 $EndComp
 $Comp
-L GND #PWR0133
+L GND #PWR0136
 U 1 1 589FE46D
 P 7700 1950
-F 0 "#PWR0133" H 7700 1700 50  0001 C CNN
+F 0 "#PWR0136" H 7700 1700 50  0001 C CNN
 F 1 "GND" H 7705 1777 50  0000 C CNN
 F 2 "" H 7700 1950 50  0000 C CNN
@@
 $EndComp
 $Comp
-L GND #PWR0134
+L GND #PWR0137
 U 1 1 589FE4F9
 P 7900 1950
-F 0 "#PWR0134" H 7900 1700 50  0001 C CNN
+F 0 "#PWR0137" H 7900 1700 50  0001 C CNN
 F 1 "GND" H 7905 1777 50  0000 C CNN
 F 2 "" H 7900 1950 50  0000 C CNN
@@
 PHY_VDDCR
 $Comp
-L VDD_PHYA #PWR0135
+L VDD_PHYA #PWR0138
 U 1 1 58A03526
 P 7150 1500
-F 0 "#PWR0135" H 7150 1350 50  0001 C CNN
+F 0 "#PWR0138" H 7150 1350 50  0001 C CNN
 F 1 "VDD_PHYA" H 7165 1673 50  0000 C CNN
 F 2 "" H 7150 1500 50  0000 C CNN
@@
 $EndComp
 $Comp
-L VDD_PHYA #PWR0136
+L VDD_PHYA #PWR0139
 U 1 1 58A03EB3
 P 8650 2650
-F 0 "#PWR0136" H 8650 2500 50  0001 C CNN
+F 0 "#PWR0139" H 8650 2500 50  0001 C CNN
 F 1 "VDD_PHYA" H 8665 2823 50  0000 C CNN
 F 2 "" H 8650 2650 50  0000 C CNN
@@
 RXER/PHYAD0
 $Comp
-L GND #PWR0137
+L GND #PWR0140
 U 1 1 58A0B062
 P 8550 1700
-F 0 "#PWR0137" H 8550 1450 50  0001 C CNN
+F 0 "#PWR0140" H 8550 1450 50  0001 C CNN
 F 1 "GND" H 8555 1527 50  0000 C CNN
 F 2 "" H 8550 1700 50  0000 C CNN
@@
 MMC0_CLK
 $Comp
-L VDD_3V3B #PWR0138
+L VDD_3V3B #PWR0141
 U 1 1 5A083952
 P 5900 2400
-F 0 "#PWR0138" H 5900 2250 50  0001 C CNN
+F 0 "#PWR0141" H 5900 2250 50  0001 C CNN
 F 1 "VDD_3V3B" H 5915 2573 50  0000 C CNN
 F 2 "" H 5900 2400 50  0000 C CNN
@@
 $EndComp
 $Comp
-L VDD_3V3B #PWR0139
+L VDD_3V3B #PWR0142
 U 1 1 5A08528B
 P 10300 900
-F 0 "#PWR0139" H 10300 750 50  0001 C CNN
+F 0 "#PWR0142" H 10300 750 50  0001 C CNN
 F 1 "VDD_3V3B" H 10315 1073 50  0000 C CNN
 F 2 "" H 10300 900 50  0000 C CNN
@@
 Connection ~ 6150 2700
 $Comp
-L PWR_FLAG #FLG0140
+L PWR_FLAG #FLG0143
 U 1 1 5A0AC399
 P 6850 2400
-F 0 "#FLG0140" H 6850 2495 50  0001 C CNN
+F 0 "#FLG0143" H 6850 2495 50  0001 C CNN
 F 1 "PWR_FLAG" H 6850 2624 50  0000 C CNN
 F 2 "" H 6850 2400 50  0000 C CNN

Commit message: Remove HDMI from the schematic
Parts:
- renumbered C29 to C28, C30 to C29, C31 to C30, C32 to C31, C33 to C32, C34 to C33, C35 to C34, C36 to C35, C37 to C36, C38 to C37, C39 to C38, C40 to C39, FB28 to FB27, U11 to U10
Changed lines of the file:
@@
 $Descr A4 11693 8268
 encoding utf-8
-Sheet 8 26
+Sheet 8 25
 Title ""
 Date ""
@@
 $EndDescr
 $Comp
-L LAN8710A U11
+L LAN8710A U10
 U 1 1 589D11A4
 P 7200 4150
-F 0 "U11" H 6450 5400 60  0000 C CNN
+F 0 "U10" H 6450 5400 60  0000 C CNN
 F 1 "LAN8710A" H 7750 5400 60  0000 C CNN
 F 2 "Housings_DFN_QFN:QFN-32-1EP_5x5mm_Pitch0.5mm" H 7450 4250 60  0001 C CNN
@@
 $EndComp
 $Comp
-L C C29
+L C C28
 U 1 1 589D3894
 P 4950 5800
-F 0 "C29" H 5064 5846 50  0000 L CNN
+F 0 "C28" H 5064 5846 50  0000 L CNN
 F 1 "30pF" H 5064 5755 50  0000 L CNN
 F 2 "Capacitors_SMD:C_0603" H 4988 5650 50  0001 C CNN
@@
 $EndComp
 $Comp
-L C C30
+L C C29
 U 1 1 589D38D5
 P 5450 5800
-F 0 "C30" H 5565 5846 50  0000 L CNN
+F 0 "C29" H 5565 5846 50  0000 L CNN
 F 1 "30pF" H 5565 5755 50  0000 L CNN
 F 2 "Capacitors_SMD:C_0603" H 5488 5650 50  0001 C CNN
@@
 $EndComp
 $Comp
-L GND #PWR0124
+L GND #PWR0119
 U 1 1 589D3921
 P 4950 6000
-F 0 "#PWR0124" H 4950 5750 50  0001 C CNN
+F 0 "#PWR0119" H 4950 5750 50  0001 C CNN
 F 1 "GND" H 4955 5827 50  0000 C CNN
 F 2 "" H 4950 6000 50  0000 C CNN
@@
 $EndComp
 $Comp
-L GND #PWR0125
+L GND #PWR0120
 U 1 1 589D3945
 P 5450 6000
-F 0 "#PWR0125" H 5450 5750 50  0001 C CNN
+F 0 "#PWR0120" H 5450 5750 50  0001 C CNN
 F 1 "GND" H 5455 5827 50  0000 C CNN
 F 2 "" H 5450 6000 50  0000 C CNN
@@
 $EndComp
 $Comp
-L C C37
+L C C36
 U 1 1 589EEF58
 P 8350 3650
-F 0 "C37" H 8350 3750 50  0000 L CNN
+F 0 "C36" H 8350 3750 50  0000 L CNN
 F 1 "DNP-15pF" H 8350 3550 50  0000 L CNN
 F 2 "Capacitors_SMD:C_0603" H 8388 3500 50  0001 C CNN
@@
 $EndComp
 $Comp
-L C C38
+L C C37
 U 1 1 589EEFBF
 P 8550 3650
-F 0 "C38" H 8550 3750 50  0000 L CNN
+F 0 "C37" H 8550 3750 50  0000 L CNN
 F 1 "DNP-15pF" H 8550 3475 50  0000 L CNN
 F 2 "Capacitors_SMD:C_0603" H 8588 3500 50  0001 C CNN
@@
 $EndComp
 $Comp
-L C C39
+L C C38
 U 1 1 589EF023
 P 8750 3650
-F 0 "C39" H 8750 3750 50  0000 L CNN
+F 0 "C38" H 8750 3750 50  0000 L CNN
 F 1 "DNP-15pF" H 8750 3550 50  0000 L CNN
 F 2 "Capacitors_SMD:C_0603" H 8788 3500 50  0001 C CNN
@@
 $EndComp
 $Comp
-L C C40
+L C C39
 U 1 1 589EF088
 P 8950 3650
-F 0 "C40" H 8950 3750 50  0000 L CNN
+F 0 "C39" H 8950 3750 50  0000 L CNN
 F 1 "DNP-15pF" H 8950 3475 50  0000 L CNN
 F 2 "Capacitors_SMD:C_0603" H 8988 3500 50  0001 C CNN
@@
 $EndComp
 $Comp
-L GND #PWR0126
+L GND #PWR0121
 U 1 1 589EF9C7
 P 8350 3850
-F 0 "#PWR0126" H 8350 3600 50  0001 C CNN
+F 0 "#PWR0121" H 8350 3600 50  0001 C CNN
 F 1 "GND" H 8355 3677 50  0000 C CNN
 F 2 "" H 8350 3850 50  0000 C CNN
@@
 $EndComp
 $Comp
-L GND #PWR0127
+L GND #PWR0122
 U 1 1 589EFA2D
 P 8550 3850
-F 0 "#PWR0127" H 8550 3600 50  0001 C CNN
+F 0 "#PWR0122" H 8550 3600 50  0001 C CNN
 F 1 "GND" H 8555 3677 50  0000 C CNN
 F 2 "" H 8550 3850 50  0000 C CNN
@@
 $EndComp
 $Comp
-L GND #PWR0128
+L GND #PWR0123
 U 1 1 589EFA8C
 P 8750 3850
-F 0 "#PWR0128" H 8750 3600 50  0001 C CNN
+F 0 "#PWR0123" H 8750 3600 50  0001 C CNN
 F 1 "GND" H 8755 3677 50  0000 C CNN
 F 2 "" H 8750 3850 50  0000 C CNN
@@
 $EndComp
 $Comp
-L GND #PWR0129
+L GND #PWR0124
 U 1 1 589EFAEB
 P 8950 3850
-F 0 "#PWR0129" H 8950 3600 50  0001 C CNN
+F 0 "#PWR0124" H 8950 3600 50  0001 C CNN
 F 1 "GND" H 8955 3677 50  0000 C CNN
 F 2 "" H 8950 3850 50  0000 C CNN
@@
 $EndComp
 $Comp
-L GND #PWR0130
+L GND #PWR0125
 U 1 1 589F5496
 P 7200 5600
-F 0 "#PWR0130" H 7200 5350 50  0001 C CNN
+F 0 "#PWR0125" H 7200 5350 50  0001 C CNN
 F 1 "GND" H 7205 5427 50  0000 C CNN
 F 2 "" H 7200 5600 50  0000 C CNN
@@
 $EndComp
 $Comp
-L GND #PWR0131
+L GND #PWR0126
 U 1 1 589F6033
 P 8450 5600
-F 0 "#PWR0131" H 8450 5350 50  0001 C CNN
+F 0 "#PWR0126" H 8450 5350 50  0001 C CNN
 F 1 "GND" H 8455 5427 50  0000 C CNN
 F 2 "" H 8450 5600 50  0000 C CNN
@@
 $EndComp
 $Comp
-L GND #PWR0132
+L GND #PWR0127
 U 1 1 589F60CA
 P 8700 5600
-F 0 "#PWR0132" H 8700 5350 50  0001 C CNN
+F 0 "#PWR0127" H 8700 5350 50  0001 C CNN
 F 1 "GND" H 8705 5427 50  0000 C CNN
 F 2 "" H 8700 5600 50  0000 C CNN
@@
 $EndComp
 $Comp
-L INDUCTOR_Small FB28
+L INDUCTOR_Small FB27
 U 1 1 589FB353
 P 6550 2450
-F 0 "FB28" V 6735 2450 50  0000 C CNN
+F 0 "FB27" V 6735 2450 50  0000 C CNN
 F 1 "LI0805H151R-10" V 6650 2550 50  0000 C CNN
 F 2 "Resistors_SMD:R_0805" H 6550 2450 50  0001 C CNN
@@
 $EndComp
 $Comp
-L C C31
+L C C30
 U 1 1 589FB905
 P 5900 2650
-F 0 "C31" H 6015 2696 50  0000 L CNN
+F 0 "C30" H 6015 2696 50  0000 L CNN
 F 1 "100nF" H 6015 2605 50  0000 L CNN
 F 2 "Capacitors_SMD:C_0603" H 5938 2500 50  0001 C CNN
@@
 $EndComp
 $Comp
-L GND #PWR0133
+L GND #PWR0128
 U 1 1 589FBD44
 P 5900 2850
-F 0 "#PWR0133" H 5900 2600 50  0001 C CNN
+F 0 "#PWR0128" H 5900 2600 50  0001 C CNN
 F 1 "GND" H 5905 2677 50  0000 C CNN
 F 2 "" H 5900 2850 50  0000 C CNN
@@
 $EndComp
 $Comp
-L C C32
+L C C31
 U 1 1 589FC806
 P 7500 1750
-F 0 "C32" H 7500 1850 50  0000 L CNN
+F 0 "C31" H 7500 1850 50  0000 L CNN
 F 1 "100nF" H 7500 1650 50  0000 L CNN
 F 2 "Capacitors_SMD:C_0603" H 7538 1600 50  0001 C CNN
@@
 $EndComp
 $Comp
-L GND #PWR0134
+L GND #PWR0129
 U 1 1 589FC878
 P 7500 1950
-F 0 "#PWR0134" H 7500 1700 50  0001 C CNN
+F 0 "#PWR0129" H 7500 1700 50  0001 C CNN
 F 1 "GND" H 7505 1777 50  0000 C CNN
 F 2 "" H 7500 1950 50  0000 C CNN
@@
 $EndComp
 $Comp
-L C C34
+L C C33
 U 1 1 589FC986
 P 7700 2450
-F 0 "C34" H 7750 2550 50  0000 L CNN
+F 0 "C33" H 7750 2550 50  0000 L CNN
 F 1 "470pF" H 7700 2350 50  0000 L CNN
 F 2 "Capacitors_SMD:C_0603" H 7738 2300 50  0001 C CNN
@@
 $EndComp
 $Comp
-L C C36
+L C C35
 U 1 1 589FCA4C
 P 7900 2450
-F 0 "C36" H 8015 2496 50  0000 L CNN
+F 0 "C35" H 8015 2496 50  0000 L CNN
 F 1 "1μF" H 8015 2405 50  0000 L CNN
 F 2 "Capacitors_SMD:C_0603" H 7938 2300 50  0001 C CNN
@@
 $EndComp
 $Comp
-L GND #PWR0135
+L GND #PWR0130
 U 1 1 589FCD92
 P 7800 2700
-F 0 "#PWR0135" H 7800 2450 50  0001 C CNN
+F 0 "#PWR0130" H 7800 2450 50  0001 C CNN
 F 1 "GND" H 7900 2600 50  0000 C CNN
 F 2 "" H 7800 2700 50  0000 C CNN
@@
 $EndComp
 $Comp
-L C C33
+L C C32
 U 1 1 589FE02F
 P 7700 1750
-F 0 "C33" H 7700 1850 50  0000 L CNN
+F 0 "C32" H 7700 1850 50  0000 L CNN
 F 1 "100nF" H 7700 1650 50  0000 L CNN
 F 2 "Capacitors_SMD:C_0603" H 7738 1600 50  0001 C CNN
@@
 $EndComp
 $Comp
-L C C35
+L C C34
 U 1 1 589FE0C1
 P 7900 1750
-F 0 "C35" H 7900 1850 50  0000 L CNN
+F 0 "C34" H 7900 1850 50  0000 L CNN
 F 1 "10μF" H 7900 1650 50  0000 L CNN
 F 2 "Capacitors_SMD:C_0805" H 7938 1600 50  0001 C CNN
@@
 $EndComp
 $Comp
-L GND #PWR0136
+L GND #PWR0131
 U 1 1 589FE46D
 P 7700 1950
-F 0 "#PWR0136" H 7700 1700 50  0001 C CNN
+F 0 "#PWR0131" H 7700 1700 50  0001 C CNN
 F 1 "GND" H 7705 1777 50  0000 C CNN
 F 2 "" H 7700 1950 50  0000 C CNN
@@
 $EndComp
 $Comp
-L GND #PWR0137
+L GND #PWR0132
 U 1 1 589FE4F9
 P 7900 1950
-F 0 "#PWR0137" H 7900 1700 50  0001 C CNN
+F 0 "#PWR0132" H 7900 1700 50  0001 C CNN
 F 1 "GND" H 7905 1777 50  0000 C CNN
 F 2 "" H 7900 1950 50  0000 C CNN
@@
 PHY_VDDCR
 $Comp
-L VDD_PHYA #PWR0138
+L VDD_PHYA #PWR0133
 U 1 1 58A03526
 P 7150 1500
-F 0 "#PWR0138" H 7150 1350 50  0001 C CNN
+F 0 "#PWR0133" H 7150 1350 50  0001 C CNN
 F 1 "VDD_PHYA" H 7165 1673 50  0000 C CNN
 F 2 "" H 7150 1500 50  0000 C CNN
@@
 $EndComp
 $Comp
-L VDD_PHYA #PWR0139
+L VDD_PHYA #PWR0134
 U 1 1 58A03EB3
 P 8650 2650
-F 0 "#PWR0139" H 8650 2500 50  0001 C CNN
+F 0 "#PWR0134" H 8650 2500 50  0001 C CNN
 F 1 "VDD_PHYA" H 8665 2823 50  0000 C CNN
 F 2 "" H 8650 2650 50  0000 C CNN
@@
 RXER/PHYAD0
 $Comp
-L GND #PWR0140
+L GND #PWR0135
 U 1 1 58A0B062
 P 8550 1700
-F 0 "#PWR0140" H 8550 1450 50  0001 C CNN
+F 0 "#PWR0135" H 8550 1450 50  0001 C CNN
 F 1 "GND" H 8555 1527 50  0000 C CNN
 F 2 "" H 8550 1700 50  0000 C CNN
@@
 MMC0_CLK
 $Comp
-L VDD_3V3B #PWR0141
+L VDD_3V3B #PWR0136
 U 1 1 5A083952
 P 5900 2400
-F 0 "#PWR0141" H 5900 2250 50  0001 C CNN
+F 0 "#PWR0136" H 5900 2250 50  0001 C CNN
 F 1 "VDD_3V3B" H 5915 2573 50  0000 C CNN
 F 2 "" H 5900 2400 50  0000 C CNN
@@
 $EndComp
 $Comp
-L VDD_3V3B #PWR0142
+L VDD_3V3B #PWR0137
 U 1 1 5A08528B
 P 10300 900
-F 0 "#PWR0142" H 10300 750 50  0001 C CNN
+F 0 "#PWR0137" H 10300 750 50  0001 C CNN
 F 1 "VDD_3V3B" H 10315 1073 50  0000 C CNN
 F 2 "" H 10300 900 50  0000 C CNN
@@
 Connection ~ 6150 2700
 $Comp
-L PWR_FLAG #FLG0143
+L PWR_FLAG #FLG0138
 U 1 1 5A0AC399
 P 6850 2400
-F 0 "#FLG0143" H 6850 2495 50  0001 C CNN
+F 0 "#FLG0138" H 6850 2495 50  0001 C CNN
 F 1 "PWR_FLAG" H 6850 2624 50  0000 C CNN
 F 2 "" H 6850 2400 50  0000 C CNN

Commit message: Add F1 PTC resettable fuse at the 5V output, begin E's heater circuit layout
Parts:
- renumbered FB27 to FB31
Changed lines of the file:
@@
 $EndComp
 $Comp
-L INDUCTOR_Small FB27
+L INDUCTOR_Small FB31
 U 1 1 589FB353
 P 6550 2450
-F 0 "FB27" V 6735 2450 50  0000 C CNN
+F 0 "FB31" V 6735 2450 50  0000 C CNN
 F 1 "LI0805H151R-10" V 6650 2550 50  0000 C CNN
 F 2 "Resistors_SMD:R_0805" H 6550 2450 50  0001 C CNN

Commit message: Route 24V to the buck, add PTC fuse to 5V output
Parts:
- renumbered FB31 to FB40
Changed lines of the file:
@@
 $EndComp
 $Comp
-L INDUCTOR_Small FB31
+L INDUCTOR_Small FB40
 U 1 1 589FB353
 P 6550 2450
-F 0 "FB31" V 6735 2450 50  0000 C CNN
+F 0 "FB40" V 6735 2450 50  0000 C CNN
 F 1 "LI0805H151R-10" V 6650 2550 50  0000 C CNN
 F 2 "Resistors_SMD:R_0805" H 6550 2450 50  0001 C CNN
