File: KiMBo/e_stepper.sch (KiCad schematic (older format))
At the start: 24 parts, among them U18 TMC2130

Commit message: Arrange connectors and E-stepper circuit
Parts:
- R144: footprint Resistors_SMD:R_0805 -> Resistors_SMD:R_0603
- R146: footprint Resistors_SMD:R_0603 -> Resistors_SMD:R_0805
Changed lines of the file:
@@
 F 0 "R146" H 10500 7500 50  0000 R CNN
 F 1 "220mΩ" H 10500 7600 50  0000 R CNN
-F 2 "Resistors_SMD:R_0603" V 10480 7550 50  0001 C CNN
+F 2 "Resistors_SMD:R_0805" V 10480 7550 50  0001 C CNN
 F 3 "" H 10550 7550 50  0000 C CNN
 	1    10550 7550
@@
 F 0 "R144" V 9050 7750 50  0000 C CNN
 F 1 "4.75kΩ" V 9150 7750 50  0000 C CNN
-F 2 "Resistors_SMD:R_0805" V 9180 7750 50  0001 C CNN
+F 2 "Resistors_SMD:R_0603" V 9180 7750 50  0001 C CNN
 F 3 "" H 9250 7750 50  0000 C CNN
 	1    9250 7750

Commit message: Remove HDMI from the schematic
Parts:
- renumbered C84 to C59, C85 to C60, C86 to C61, C87 to C62, C88 to C63, C89 to C64, C90 to C65, C91 to C66, C92 to C67, C93 to C68, C94 to C69, C95 to C70, C96 to C71, C97 to C72, C98 to C73, C99 to C74, R140 to R113, R141 to R114, R142 to R115, R143 to R116, R144 to R117, R145 to R118, R146 to R119, U18 to U14
Changed lines of the file:
@@
 $Descr A3 16535 11693
 encoding utf-8
-Sheet 16 26
+Sheet 16 25
 Title ""
 Date ""
@@
 MOSI
 $Comp
-L C C86
+L C C61
 U 1 1 589B8A74
 P 7300 3950
-F 0 "C86" H 7186 3904 50  0000 R CNN
+F 0 "C61" H 7186 3904 50  0000 R CNN
 F 1 "100nF" H 7186 3995 50  0000 R CNN
 F 2 "Capacitors_SMD:C_0603" H 7338 3800 50  0001 C CNN
@@
 $EndComp
 $Comp
-L C C91
+L C C66
 U 1 1 5BA7E11F
 P 9100 4500
-F 0 "C91" V 9050 4400 50  0000 C CNN
+F 0 "C66" V 9050 4400 50  0000 C CNN
 F 1 "100nF" V 9050 4675 50  0000 C CNN
 F 2 "Capacitors_SMD:C_0603" H 9138 4350 50  0001 C CNN
@@
 $EndComp
 $Comp
-L CP1 C98
+L CP1 C73
 U 1 1 5BA7E120
 P 10450 3950
-F 0 "C98" H 10550 4050 50  0000 C CNN
+F 0 "C73" H 10550 4050 50  0000 C CNN
 F 1 "100μF" H 10600 3850 50  0000 C CNN
 F 2 "Capacitors_SMD:c_elec_8x10" H 10450 3950 50  0001 C CNN
@@
 $EndComp
 $Comp
-L C C94
+L C C69
 U 1 1 589BC941
 P 9550 3950
-F 0 "C94" H 9450 4050 50  0000 C CNN
+F 0 "C69" H 9450 4050 50  0000 C CNN
 F 1 "100nF" H 9425 3850 50  0000 C CNN
 F 2 "Capacitors_SMD:C_0603" H 9588 3800 50  0001 C CNN
@@
 $EndComp
 $Comp
-L GND #PWR0200
+L GND #PWR0169
 U 1 1 589BD203
 P 7300 4150
-F 0 "#PWR0200" H 7300 3900 50  0001 C CNN
+F 0 "#PWR0169" H 7300 3900 50  0001 C CNN
 F 1 "GND" H 7300 4000 50  0000 C CNN
 F 2 "" H 7300 4150 50  0000 C CNN
@@
 $EndComp
 $Comp
-L C C95
+L C C70
 U 1 1 589BDAA2
 P 9850 3950
-F 0 "C95" H 9750 4050 50  0000 C CNN
+F 0 "C70" H 9750 4050 50  0000 C CNN
 F 1 "100nF" H 9725 3850 50  0000 C CNN
 F 2 "Capacitors_SMD:C_0603" H 9888 3800 50  0001 C CNN
@@
 $EndComp
 $Comp
-L GND #PWR0201
+L GND #PWR0170
 U 1 1 589BE47E
 P 10150 4200
-F 0 "#PWR0201" H 10150 3950 50  0001 C CNN
+F 0 "#PWR0170" H 10150 3950 50  0001 C CNN
 F 1 "GND" H 10155 4027 50  0000 C CNN
 F 2 "" H 10150 4200 50  0000 C CNN
@@
 $EndComp
 $Comp
-L +24V #PWR0202
+L +24V #PWR0171
 U 1 1 5BA7E125
 P 8350 3700
-F 0 "#PWR0202" H 8350 3550 50  0001 C CNN
+F 0 "#PWR0171" H 8350 3550 50  0001 C CNN
 F 1 "+24V" H 8365 3873 50  0000 C CNN
 F 2 "" H 8350 3700 50  0000 C CNN
@@
 $EndComp
 $Comp
-L C C88
+L C C63
 U 1 1 589C0BAD
 P 8950 5000
-F 0 "C88" H 9065 5046 50  0000 L CNN
+F 0 "C63" H 9065 5046 50  0000 L CNN
 F 1 "22nF" H 9065 4955 50  0000 L CNN
 F 2 "Capacitors_SMD:C_0603" H 8988 4850 50  0001 C CNN
@@
 $EndComp
 $Comp
-L R R146
+L R R119
 U 1 1 589C1BED
 P 10550 7550
-F 0 "R146" H 10500 7500 50  0000 R CNN
+F 0 "R119" H 10500 7500 50  0000 R CNN
 F 1 "220mΩ" H 10500 7600 50  0000 R CNN
 F 2 "Resistors_SMD:R_0805" V 10480 7550 50  0001 C CNN
@@
 $EndComp
 $Comp
-L R R145
+L R R118
 U 1 1 589C1CA7
 P 9750 7550
-F 0 "R145" H 9700 7500 50  0000 R CNN
+F 0 "R118" H 9700 7500 50  0000 R CNN
 F 1 "220mΩ" H 9700 7600 50  0000 R CNN
 F 2 "Resistors_SMD:R_0805" V 9680 7550 50  0001 C CNN
@@
 $EndComp
 $Comp
-L GND #PWR0203
+L GND #PWR0172
 U 1 1 5BA7E129
 P 9450 7900
-F 0 "#PWR0203" H 9450 7650 50  0001 C CNN
+F 0 "#PWR0172" H 9450 7650 50  0001 C CNN
 F 1 "GND" H 9455 7727 50  0000 C CNN
 F 2 "" H 9450 7900 50  0000 C CNN
@@
 NoConn ~ 7500 6450
 $Comp
-L R R142
+L R R115
 U 1 1 5BA7E12B
 P 7100 4600
-F 0 "R142" V 7000 4600 50  0000 C CNN
+F 0 "R115" V 7000 4600 50  0000 C CNN
 F 1 "2.2Ω" V 7100 4600 50  0000 C CNN
 F 2 "Resistors_SMD:R_0603" V 7030 4600 50  0001 C CNN
@@
 $EndComp
 $Comp
-L C C85
+L C C60
 U 1 1 589C52DF
 P 6900 4800
-F 0 "C85" H 6950 4900 50  0000 L CNN
+F 0 "C60" H 6950 4900 50  0000 L CNN
 F 1 "470nF" H 6925 4700 50  0000 L CNN
 F 2 "Capacitors_SMD:C_0603" H 6938 4650 50  0001 C CNN
@@
 NoConn ~ 7500 6550
 $Comp
-L GND #PWR0204
+L GND #PWR0173
 U 1 1 589C97FF
 P 7450 6950
-F 0 "#PWR0204" H 7450 6700 50  0001 C CNN
+F 0 "#PWR0173" H 7450 6700 50  0001 C CNN
 F 1 "GND" H 7455 6777 50  0000 C CNN
 F 2 "" H 7450 6950 50  0000 C CNN
@@
 $EndComp
 $Comp
-L C C96
+L C C71
 U 1 1 5BA7E12E
 P 9900 7550
-F 0 "C96" H 9950 7650 50  0000 L CNN
+F 0 "C71" H 9950 7650 50  0000 L CNN
 F 1 "100nF" H 9950 7450 50  0000 L CNN
 F 2 "Capacitors_SMD:C_0603" H 9938 7400 50  0001 C CNN
@@
 E_FAULT
 $Comp
-L R R140
+L R R113
 U 1 1 589D21BC
 P 5850 5100
-F 0 "R140" H 5919 5146 50  0000 L CNN
+F 0 "R113" H 5919 5146 50  0000 L CNN
 F 1 "4.7kΩ" H 5919 5055 50  0000 L CNN
 F 2 "Resistors_SMD:R_0603" V 5780 5100 50  0001 C CNN
@@
 Internal\nPull-Up
 $Comp
-L C C87
+L C C62
 U 1 1 5BA7E12A
 P 7300 4800
-F 0 "C87" H 7350 4900 50  0000 L CNN
+F 0 "C62" H 7350 4900 50  0000 L CNN
 F 1 "4.7μF" H 7350 4700 50  0000 L CNN
 F 2 "Capacitors_SMD:C_0603" H 7338 4650 50  0001 C CNN
@@
 5VOUT
 $Comp
-L R R143
+L R R116
 U 1 1 589E13FD
 P 9050 7550
-F 0 "R143" H 9119 7596 50  0000 L CNN
+F 0 "R116" H 9119 7596 50  0000 L CNN
 F 1 "5.23kΩ" H 9119 7505 50  0000 L CNN
 F 2 "Resistors_SMD:R_0603" V 8980 7550 50  0001 C CNN
@@
 5VOUT
 $Comp
-L R R144
+L R R117
 U 1 1 589E24D4
 P 9250 7750
-F 0 "R144" V 9050 7750 50  0000 C CNN
+F 0 "R117" V 9050 7750 50  0000 C CNN
 F 1 "4.75kΩ" V 9150 7750 50  0000 C CNN
 F 2 "Resistors_SMD:R_0603" V 9180 7750 50  0001 C CNN
@@
 AIN_IREF=1-2.4V
 $Comp
-L R R141
+L R R114
 U 1 1 5BA7E132
 P 6200 5100
-F 0 "R141" H 6269 5146 50  0000 L CNN
+F 0 "R114" H 6269 5146 50  0000 L CNN
 F 1 "4.7kΩ" H 6269 5055 50  0000 L CNN
 F 2 "Resistors_SMD:R_0603" V 6130 5100 50  0001 C CNN
@@
 $EndComp
 $Comp
-L C C99
+L C C74
 U 1 1 5BA7E133
 P 10700 7550
-F 0 "C99" H 10750 7650 50  0000 L CNN
+F 0 "C74" H 10750 7650 50  0000 L CNN
 F 1 "100nF" H 10750 7450 50  0000 L CNN
 F 2 "Capacitors_SMD:C_0603" H 10738 7400 50  0001 C CNN
@@
 Choose  sense  resistors  in  a  way,  that  normal \nIRUN is 16 to 31 for best microstep performance.
 $Comp
-L C C89
+L C C64
 U 1 1 5BA7E134
 P 8950 5800
-F 0 "C89" H 8975 5900 50  0000 L CNN
+F 0 "C64" H 8975 5900 50  0000 L CNN
 F 1 "470pF" H 8950 5700 50  0000 L CNN
 F 2 "Capacitors_SMD:C_0603" H 8988 5650 50  0001 C CNN
@@
 $EndComp
 $Comp
-L GND #PWR0205
+L GND #PWR0174
 U 1 1 58B19D33
 P 9050 6050
-F 0 "#PWR0205" H 9050 5800 50  0001 C CNN
+F 0 "#PWR0174" H 9050 5800 50  0001 C CNN
 F 1 "GND" H 9050 5900 50  0000 C CNN
 F 2 "" H 9050 6050 50  0000 C CNN
@@
 $EndComp
 $Comp
-L C C92
+L C C67
 U 1 1 58B1B794
 P 9150 5800
-F 0 "C92" H 9175 5900 50  0000 L CNN
+F 0 "C67" H 9175 5900 50  0000 L CNN
 F 1 "470pF" H 9175 5700 50  0000 L CNN
 F 2 "Capacitors_SMD:C_0603" H 9188 5650 50  0001 C CNN
@@
 $EndComp
 $Comp
-L C C90
+L C C65
 U 1 1 58B1C6FD
 P 8950 6650
-F 0 "C90" H 8975 6750 50  0000 L CNN
+F 0 "C65" H 8975 6750 50  0000 L CNN
 F 1 "470pF" H 8950 6550 50  0000 L CNN
 F 2 "Capacitors_SMD:C_0603" H 8988 6500 50  0001 C CNN
@@
 $EndComp
 $Comp
-L GND #PWR0206
+L GND #PWR0175
 U 1 1 58B1C704
 P 9050 6900
-F 0 "#PWR0206" H 9050 6650 50  0001 C CNN
+F 0 "#PWR0175" H 9050 6650 50  0001 C CNN
 F 1 "GND" H 9050 6750 50  0000 C CNN
 F 2 "" H 9050 6900 50  0000 C CNN
@@
 $EndComp
 $Comp
-L C C93
+L C C68
 U 1 1 58B1C710
 P 9150 6650
-F 0 "C93" H 9175 6750 50  0000 L CNN
+F 0 "C68" H 9175 6750 50  0000 L CNN
 F 1 "470pF" H 9175 6550 50  0000 L CNN
 F 2 "Capacitors_SMD:C_0603" H 9188 6500 50  0001 C CNN
@@
 $EndComp
 $Comp
-L TMC2130 U18
+L TMC2130 U14
 U 1 1 5BA7E11D
 P 8200 5550
-F 0 "U18" H 7750 7050 60  0000 C CNN
+F 0 "U14" H 7750 7050 60  0000 C CNN
 F 1 "TMC2130" H 8500 7050 60  0000 C CNN
 F 2 "KiMBo:QFN36_5X6" H 8200 5850 60  0001 C CNN
@@
 $EndComp
 $Comp
-L C C97
+L C C72
 U 1 1 58B40194
 P 10150 3950
-F 0 "C97" H 10050 4050 50  0000 C CNN
+F 0 "C72" H 10050 4050 50  0000 C CNN
 F 1 "10μF" H 10025 3850 50  0000 C CNN
 F 2 "Capacitors_SMD:C_0805" H 10188 3800 50  0001 C CNN
@@
 Can extract which\nfault is occurring via SPI\nby reading DRV_STATUS reg
 $Comp
-L VDD_3V3B #PWR0207
+L VDD_3V3B #PWR0176
 U 1 1 5A2FD350
 P 6550 4300
-F 0 "#PWR0207" H 6550 4150 50  0001 C CNN
+F 0 "#PWR0176" H 6550 4150 50  0001 C CNN
 F 1 "VDD_3V3B" H 6565 4473 50  0000 C CNN
 F 2 "" H 6550 4300 50  0000 C CNN
@@
 $EndComp
 $Comp
-L C C84
+L C C59
 U 1 1 5A896678
 P 6550 4800
-F 0 "C84" H 6600 4900 50  0000 L CNN
+F 0 "C59" H 6600 4900 50  0000 L CNN
 F 1 "100nF" H 6575 4700 50  0000 L CNN
 F 2 "Capacitors_SMD:C_0603" H 6588 4650 50  0001 C CNN

Commit message: More stepper motor driver progress
Parts:
- renumbered R113 to R115, R114 to R116, R115 to R117, R116 to R118, R117 to R119, R118 to R120, R119 to R121
Changed lines of the file:
@@
 $Descr A3 16535 11693
 encoding utf-8
-Sheet 16 25
+Sheet 14 25
 Title ""
 Date ""
@@
 $EndComp
 $Comp
-L R R119
+L R R121
 U 1 1 589C1BED
 P 10550 7550
-F 0 "R119" H 10500 7500 50  0000 R CNN
+F 0 "R121" H 10500 7500 50  0000 R CNN
 F 1 "220mΩ" H 10500 7600 50  0000 R CNN
 F 2 "Resistors_SMD:R_0805" V 10480 7550 50  0001 C CNN
@@
 $EndComp
 $Comp
-L R R118
+L R R120
 U 1 1 589C1CA7
 P 9750 7550
-F 0 "R118" H 9700 7500 50  0000 R CNN
+F 0 "R120" H 9700 7500 50  0000 R CNN
 F 1 "220mΩ" H 9700 7600 50  0000 R CNN
 F 2 "Resistors_SMD:R_0805" V 9680 7550 50  0001 C CNN
@@
 NoConn ~ 7500 6450
 $Comp
-L R R115
+L R R117
 U 1 1 5BA7E12B
 P 7100 4600
-F 0 "R115" V 7000 4600 50  0000 C CNN
+F 0 "R117" V 7000 4600 50  0000 C CNN
 F 1 "2.2Ω" V 7100 4600 50  0000 C CNN
 F 2 "Resistors_SMD:R_0603" V 7030 4600 50  0001 C CNN
@@
 E_FAULT
 $Comp
-L R R113
+L R R115
 U 1 1 589D21BC
 P 5850 5100
-F 0 "R113" H 5919 5146 50  0000 L CNN
+F 0 "R115" H 5919 5146 50  0000 L CNN
 F 1 "4.7kΩ" H 5919 5055 50  0000 L CNN
 F 2 "Resistors_SMD:R_0603" V 5780 5100 50  0001 C CNN
@@
 5VOUT
 $Comp
-L R R116
+L R R118
 U 1 1 589E13FD
 P 9050 7550
-F 0 "R116" H 9119 7596 50  0000 L CNN
+F 0 "R118" H 9119 7596 50  0000 L CNN
 F 1 "5.23kΩ" H 9119 7505 50  0000 L CNN
 F 2 "Resistors_SMD:R_0603" V 8980 7550 50  0001 C CNN
@@
 5VOUT
 $Comp
-L R R117
+L R R119
 U 1 1 589E24D4
 P 9250 7750
-F 0 "R117" V 9050 7750 50  0000 C CNN
+F 0 "R119" V 9050 7750 50  0000 C CNN
 F 1 "4.75kΩ" V 9150 7750 50  0000 C CNN
 F 2 "Resistors_SMD:R_0603" V 9180 7750 50  0001 C CNN
@@
 AIN_IREF=1-2.4V
 $Comp
-L R R114
+L R R116
 U 1 1 5BA7E132
 P 6200 5100
-F 0 "R114" H 6269 5146 50  0000 L CNN
+F 0 "R116" H 6269 5146 50  0000 L CNN
 F 1 "4.7kΩ" H 6269 5055 50  0000 L CNN
 F 2 "Resistors_SMD:R_0603" V 6130 5100 50  0001 C CNN

Commit message: Daisy chain the SPI stepper motor driver interface, continue work on the E-heater layout
Parts:
- renumbered C59 to C57, C60 to C58, C61 to C59, C62 to C60, C63 to C61, C64 to C62, C65 to C63, C66 to C64, C67 to C65, C68 to C66, C69 to C67, C70 to C68, C71 to C69, C72 to C70, C73 to C71, C74 to C72, U14 to U13
Changed lines of the file:
@@
 MOSI
 $Comp
-L C C61
+L C C59
 U 1 1 589B8A74
 P 7300 3950
-F 0 "C61" H 7186 3904 50  0000 R CNN
+F 0 "C59" H 7186 3904 50  0000 R CNN
 F 1 "100nF" H 7186 3995 50  0000 R CNN
 F 2 "Capacitors_SMD:C_0603" H 7338 3800 50  0001 C CNN
@@
 $EndComp
 $Comp
-L C C66
+L C C64
 U 1 1 5BA7E11F
 P 9100 4500
-F 0 "C66" V 9050 4400 50  0000 C CNN
+F 0 "C64" V 9050 4400 50  0000 C CNN
 F 1 "100nF" V 9050 4675 50  0000 C CNN
 F 2 "Capacitors_SMD:C_0603" H 9138 4350 50  0001 C CNN
@@
 $EndComp
 $Comp
-L CP1 C73
+L CP1 C71
 U 1 1 5BA7E120
 P 10450 3950
-F 0 "C73" H 10550 4050 50  0000 C CNN
+F 0 "C71" H 10550 4050 50  0000 C CNN
 F 1 "100μF" H 10600 3850 50  0000 C CNN
 F 2 "Capacitors_SMD:c_elec_8x10" H 10450 3950 50  0001 C CNN
@@
 $EndComp
 $Comp
-L C C69
+L C C67
 U 1 1 589BC941
 P 9550 3950
-F 0 "C69" H 9450 4050 50  0000 C CNN
+F 0 "C67" H 9450 4050 50  0000 C CNN
 F 1 "100nF" H 9425 3850 50  0000 C CNN
 F 2 "Capacitors_SMD:C_0603" H 9588 3800 50  0001 C CNN
@@
 $EndComp
 $Comp
-L GND #PWR0169
+L GND #PWR149
 U 1 1 589BD203
 P 7300 4150
-F 0 "#PWR0169" H 7300 3900 50  0001 C CNN
+F 0 "#PWR149" H 7300 3900 50  0001 C CNN
 F 1 "GND" H 7300 4000 50  0000 C CNN
 F 2 "" H 7300 4150 50  0000 C CNN
@@
 $EndComp
 $Comp
-L C C70
+L C C68
 U 1 1 589BDAA2
 P 9850 3950
-F 0 "C70" H 9750 4050 50  0000 C CNN
+F 0 "C68" H 9750 4050 50  0000 C CNN
 F 1 "100nF" H 9725 3850 50  0000 C CNN
 F 2 "Capacitors_SMD:C_0603" H 9888 3800 50  0001 C CNN
@@
 $EndComp
 $Comp
-L GND #PWR0170
+L GND #PWR155
 U 1 1 589BE47E
 P 10150 4200
-F 0 "#PWR0170" H 10150 3950 50  0001 C CNN
+F 0 "#PWR155" H 10150 3950 50  0001 C CNN
 F 1 "GND" H 10155 4027 50  0000 C CNN
 F 2 "" H 10150 4200 50  0000 C CNN
@@
 $EndComp
 $Comp
-L +24V #PWR0171
+L +24V #PWR151
 U 1 1 5BA7E125
 P 8350 3700
-F 0 "#PWR0171" H 8350 3550 50  0001 C CNN
+F 0 "#PWR151" H 8350 3550 50  0001 C CNN
 F 1 "+24V" H 8365 3873 50  0000 C CNN
 F 2 "" H 8350 3700 50  0000 C CNN
@@
 $EndComp
 $Comp
-L C C63
+L C C61
 U 1 1 589C0BAD
 P 8950 5000
-F 0 "C63" H 9065 5046 50  0000 L CNN
+F 0 "C61" H 9065 5046 50  0000 L CNN
 F 1 "22nF" H 9065 4955 50  0000 L CNN
 F 2 "Capacitors_SMD:C_0603" H 8988 4850 50  0001 C CNN
@@
 $EndComp
 $Comp
-L GND #PWR0172
+L GND #PWR154
 U 1 1 5BA7E129
 P 9450 7900
-F 0 "#PWR0172" H 9450 7650 50  0001 C CNN
+F 0 "#PWR154" H 9450 7650 50  0001 C CNN
 F 1 "GND" H 9455 7727 50  0000 C CNN
 F 2 "" H 9450 7900 50  0000 C CNN
@@
 $EndComp
 $Comp
-L C C60
+L C C58
 U 1 1 589C52DF
 P 6900 4800
-F 0 "C60" H 6950 4900 50  0000 L CNN
+F 0 "C58" H 6950 4900 50  0000 L CNN
 F 1 "470nF" H 6925 4700 50  0000 L CNN
 F 2 "Capacitors_SMD:C_0603" H 6938 4650 50  0001 C CNN
@@
 NoConn ~ 7500 6550
 $Comp
-L GND #PWR0173
+L GND #PWR150
 U 1 1 589C97FF
 P 7450 6950
-F 0 "#PWR0173" H 7450 6700 50  0001 C CNN
+F 0 "#PWR150" H 7450 6700 50  0001 C CNN
 F 1 "GND" H 7455 6777 50  0000 C CNN
 F 2 "" H 7450 6950 50  0000 C CNN
@@
 $EndComp
 $Comp
-L C C71
+L C C69
 U 1 1 5BA7E12E
 P 9900 7550
-F 0 "C71" H 9950 7650 50  0000 L CNN
+F 0 "C69" H 9950 7650 50  0000 L CNN
 F 1 "100nF" H 9950 7450 50  0000 L CNN
 F 2 "Capacitors_SMD:C_0603" H 9938 7400 50  0001 C CNN
@@
 Internal\nPull-Up
 $Comp
-L C C62
+L C C60
 U 1 1 5BA7E12A
 P 7300 4800
-F 0 "C62" H 7350 4900 50  0000 L CNN
+F 0 "C60" H 7350 4900 50  0000 L CNN
 F 1 "4.7μF" H 7350 4700 50  0000 L CNN
 F 2 "Capacitors_SMD:C_0603" H 7338 4650 50  0001 C CNN
@@
 $EndComp
 $Comp
-L C C74
+L C C72
 U 1 1 5BA7E133
 P 10700 7550
-F 0 "C74" H 10750 7650 50  0000 L CNN
+F 0 "C72" H 10750 7650 50  0000 L CNN
 F 1 "100nF" H 10750 7450 50  0000 L CNN
 F 2 "Capacitors_SMD:C_0603" H 10738 7400 50  0001 C CNN
@@
 Choose  sense  resistors  in  a  way,  that  normal \nIRUN is 16 to 31 for best microstep performance.
 $Comp
-L C C64
+L C C62
 U 1 1 5BA7E134
 P 8950 5800
-F 0 "C64" H 8975 5900 50  0000 L CNN
+F 0 "C62" H 8975 5900 50  0000 L CNN
 F 1 "470pF" H 8950 5700 50  0000 L CNN
 F 2 "Capacitors_SMD:C_0603" H 8988 5650 50  0001 C CNN
@@
 $EndComp
 $Comp
-L GND #PWR0174
+L GND #PWR152
 U 1 1 58B19D33
 P 9050 6050
-F 0 "#PWR0174" H 9050 5800 50  0001 C CNN
+F 0 "#PWR152" H 9050 5800 50  0001 C CNN
 F 1 "GND" H 9050 5900 50  0000 C CNN
 F 2 "" H 9050 6050 50  0000 C CNN
@@
 $EndComp
 $Comp
-L C C67
+L C C65
 U 1 1 58B1B794
 P 9150 5800
-F 0 "C67" H 9175 5900 50  0000 L CNN
+F 0 "C65" H 9175 5900 50  0000 L CNN
 F 1 "470pF" H 9175 5700 50  0000 L CNN
 F 2 "Capacitors_SMD:C_0603" H 9188 5650 50  0001 C CNN
@@
 $EndComp
 $Comp
-L C C65
+L C C63
 U 1 1 58B1C6FD
 P 8950 6650
-F 0 "C65" H 8975 6750 50  0000 L CNN
+F 0 "C63" H 8975 6750 50  0000 L CNN
 F 1 "470pF" H 8950 6550 50  0000 L CNN
 F 2 "Capacitors_SMD:C_0603" H 8988 6500 50  0001 C CNN
@@
 $EndComp
 $Comp
-L GND #PWR0175
+L GND #PWR153
 U 1 1 58B1C704
 P 9050 6900
-F 0 "#PWR0175" H 9050 6650 50  0001 C CNN
+F 0 "#PWR153" H 9050 6650 50  0001 C CNN
 F 1 "GND" H 9050 6750 50  0000 C CNN
 F 2 "" H 9050 6900 50  0000 C CNN
@@
 $EndComp
 $Comp
-L C C68
+L C C66
 U 1 1 58B1C710
 P 9150 6650
-F 0 "C68" H 9175 6750 50  0000 L CNN
+F 0 "C66" H 9175 6750 50  0000 L CNN
 F 1 "470pF" H 9175 6550 50  0000 L CNN
 F 2 "Capacitors_SMD:C_0603" H 9188 6500 50  0001 C CNN
@@
 $EndComp
 $Comp
-L TMC2130 U14
+L TMC2130 U13
 U 1 1 5BA7E11D
 P 8200 5550
-F 0 "U14" H 7750 7050 60  0000 C CNN
+F 0 "U13" H 7750 7050 60  0000 C CNN
 F 1 "TMC2130" H 8500 7050 60  0000 C CNN
 F 2 "KiMBo:QFN36_5X6" H 8200 5850 60  0001 C CNN
@@
 $EndComp
 $Comp
-L C C72
+L C C70
 U 1 1 58B40194
 P 10150 3950
-F 0 "C72" H 10050 4050 50  0000 C CNN
+F 0 "C70" H 10050 4050 50  0000 C CNN
 F 1 "10μF" H 10025 3850 50  0000 C CNN
 F 2 "Capacitors_SMD:C_0805" H 10188 3800 50  0001 C CNN
@@
 Can extract which\nfault is occurring via SPI\nby reading DRV_STATUS reg
 $Comp
-L VDD_3V3B #PWR0176
+L VDD_3V3B #PWR148
 U 1 1 5A2FD350
 P 6550 4300
-F 0 "#PWR0176" H 6550 4150 50  0001 C CNN
+F 0 "#PWR148" H 6550 4150 50  0001 C CNN
 F 1 "VDD_3V3B" H 6565 4473 50  0000 C CNN
 F 2 "" H 6550 4300 50  0000 C CNN
@@
 $EndComp
 $Comp
-L C C59
+L C C57
 U 1 1 5A896678
 P 6550 4800
-F 0 "C59" H 6600 4900 50  0000 L CNN
+F 0 "C57" H 6600 4900 50  0000 L CNN
 F 1 "100nF" H 6575 4700 50  0000 L CNN
 F 2 "Capacitors_SMD:C_0603" H 6588 4650 50  0001 C CNN
