File: KiMBo/e_stepper.sch (KiCad schematic (older format))
At the start: 24 parts, among them U13 TMC2130

Commit message: Add ferrite beads to the 5V and 3V pins at the SPI connectors
Parts:
- renumbered C57 to C53, C58 to C54, C59 to C55, C60 to C56, C61 to C57, C62 to C58, C63 to C59, C64 to C60, C65 to C61, C66 to C62, C67 to C63, C68 to C64, C69 to C65, C70 to C66, C71 to C67, C72 to C68
Changed lines of the file:
@@
 MOSI
 $Comp
-L C C59
+L C C55
 U 1 1 589B8A74
 P 7300 3950
-F 0 "C59" H 7186 3904 50  0000 R CNN
+F 0 "C55" H 7186 3904 50  0000 R CNN
 F 1 "100nF" H 7186 3995 50  0000 R CNN
 F 2 "Capacitors_SMD:C_0603" H 7338 3800 50  0001 C CNN
@@
 $EndComp
 $Comp
-L C C64
+L C C60
 U 1 1 5BA7E11F
 P 9100 4500
-F 0 "C64" V 9050 4400 50  0000 C CNN
+F 0 "C60" V 9050 4400 50  0000 C CNN
 F 1 "100nF" V 9050 4675 50  0000 C CNN
 F 2 "Capacitors_SMD:C_0603" H 9138 4350 50  0001 C CNN
@@
 $EndComp
 $Comp
-L CP1 C71
+L CP1 C67
 U 1 1 5BA7E120
 P 10450 3950
-F 0 "C71" H 10550 4050 50  0000 C CNN
+F 0 "C67" H 10550 4050 50  0000 C CNN
 F 1 "100μF" H 10600 3850 50  0000 C CNN
 F 2 "Capacitors_SMD:c_elec_8x10" H 10450 3950 50  0001 C CNN
@@
 $EndComp
 $Comp
-L C C67
+L C C63
 U 1 1 589BC941
 P 9550 3950
-F 0 "C67" H 9450 4050 50  0000 C CNN
+F 0 "C63" H 9450 4050 50  0000 C CNN
 F 1 "100nF" H 9425 3850 50  0000 C CNN
 F 2 "Capacitors_SMD:C_0603" H 9588 3800 50  0001 C CNN
@@
 $EndComp
 $Comp
-L GND #PWR0165
+L GND #PWR0162
 U 1 1 589BD203
 P 7300 4150
-F 0 "#PWR0165" H 7300 3900 50  0001 C CNN
+F 0 "#PWR0162" H 7300 3900 50  0001 C CNN
 F 1 "GND" H 7300 4000 50  0000 C CNN
 F 2 "" H 7300 4150 50  0000 C CNN
@@
 $EndComp
 $Comp
-L C C68
+L C C64
 U 1 1 589BDAA2
 P 9850 3950
-F 0 "C68" H 9750 4050 50  0000 C CNN
+F 0 "C64" H 9750 4050 50  0000 C CNN
 F 1 "100nF" H 9725 3850 50  0000 C CNN
 F 2 "Capacitors_SMD:C_0603" H 9888 3800 50  0001 C CNN
@@
 $EndComp
 $Comp
-L GND #PWR0166
+L GND #PWR0163
 U 1 1 589BE47E
 P 10150 4200
-F 0 "#PWR0166" H 10150 3950 50  0001 C CNN
+F 0 "#PWR0163" H 10150 3950 50  0001 C CNN
 F 1 "GND" H 10155 4027 50  0000 C CNN
 F 2 "" H 10150 4200 50  0000 C CNN
@@
 $EndComp
 $Comp
-L +24V #PWR0167
+L +24V #PWR0164
 U 1 1 5BA7E125
 P 8350 3700
-F 0 "#PWR0167" H 8350 3550 50  0001 C CNN
+F 0 "#PWR0164" H 8350 3550 50  0001 C CNN
 F 1 "+24V" H 8365 3873 50  0000 C CNN
 F 2 "" H 8350 3700 50  0000 C CNN
@@
 $EndComp
 $Comp
-L C C61
+L C C57
 U 1 1 589C0BAD
 P 8950 5000
-F 0 "C61" H 9065 5046 50  0000 L CNN
+F 0 "C57" H 9065 5046 50  0000 L CNN
 F 1 "22nF" H 9065 4955 50  0000 L CNN
 F 2 "Capacitors_SMD:C_0603" H 8988 4850 50  0001 C CNN
@@
 $EndComp
 $Comp
-L GND #PWR0168
+L GND #PWR0165
 U 1 1 5BA7E129
 P 9450 7900
-F 0 "#PWR0168" H 9450 7650 50  0001 C CNN
+F 0 "#PWR0165" H 9450 7650 50  0001 C CNN
 F 1 "GND" H 9455 7727 50  0000 C CNN
 F 2 "" H 9450 7900 50  0000 C CNN
@@
 $EndComp
 $Comp
-L C C58
+L C C54
 U 1 1 589C52DF
 P 6900 4800
-F 0 "C58" H 6950 4900 50  0000 L CNN
+F 0 "C54" H 6950 4900 50  0000 L CNN
 F 1 "470nF" H 6925 4700 50  0000 L CNN
 F 2 "Capacitors_SMD:C_0603" H 6938 4650 50  0001 C CNN
@@
 NoConn ~ 7500 6550
 $Comp
-L GND #PWR0169
+L GND #PWR0166
 U 1 1 589C97FF
 P 7450 6950
-F 0 "#PWR0169" H 7450 6700 50  0001 C CNN
+F 0 "#PWR0166" H 7450 6700 50  0001 C CNN
 F 1 "GND" H 7455 6777 50  0000 C CNN
 F 2 "" H 7450 6950 50  0000 C CNN
@@
 $EndComp
 $Comp
-L C C69
+L C C65
 U 1 1 5BA7E12E
 P 9900 7550
-F 0 "C69" H 9950 7650 50  0000 L CNN
+F 0 "C65" H 9950 7650 50  0000 L CNN
 F 1 "100nF" H 9950 7450 50  0000 L CNN
 F 2 "Capacitors_SMD:C_0603" H 9938 7400 50  0001 C CNN
@@
 Internal\nPull-Up
 $Comp
-L C C60
+L C C56
 U 1 1 5BA7E12A
 P 7300 4800
-F 0 "C60" H 7350 4900 50  0000 L CNN
+F 0 "C56" H 7350 4900 50  0000 L CNN
 F 1 "4.7μF" H 7350 4700 50  0000 L CNN
 F 2 "Capacitors_SMD:C_0603" H 7338 4650 50  0001 C CNN
@@
 $EndComp
 $Comp
-L C C72
+L C C68
 U 1 1 5BA7E133
 P 10700 7550
-F 0 "C72" H 10750 7650 50  0000 L CNN
+F 0 "C68" H 10750 7650 50  0000 L CNN
 F 1 "100nF" H 10750 7450 50  0000 L CNN
 F 2 "Capacitors_SMD:C_0603" H 10738 7400 50  0001 C CNN
@@
 Choose  sense  resistors  in  a  way,  that  normal \nIRUN is 16 to 31 for best microstep performance.
 $Comp
-L C C62
+L C C58
 U 1 1 5BA7E134
 P 8950 5800
-F 0 "C62" H 8975 5900 50  0000 L CNN
+F 0 "C58" H 8975 5900 50  0000 L CNN
 F 1 "470pF" H 8950 5700 50  0000 L CNN
 F 2 "Capacitors_SMD:C_0603" H 8988 5650 50  0001 C CNN
@@
 $EndComp
 $Comp
-L GND #PWR0170
+L GND #PWR0167
 U 1 1 58B19D33
 P 9050 6050
-F 0 "#PWR0170" H 9050 5800 50  0001 C CNN
+F 0 "#PWR0167" H 9050 5800 50  0001 C CNN
 F 1 "GND" H 9050 5900 50  0000 C CNN
 F 2 "" H 9050 6050 50  0000 C CNN
@@
 $EndComp
 $Comp
-L C C65
+L C C61
 U 1 1 58B1B794
 P 9150 5800
-F 0 "C65" H 9175 5900 50  0000 L CNN
+F 0 "C61" H 9175 5900 50  0000 L CNN
 F 1 "470pF" H 9175 5700 50  0000 L CNN
 F 2 "Capacitors_SMD:C_0603" H 9188 5650 50  0001 C CNN
@@
 $EndComp
 $Comp
-L C C63
+L C C59
 U 1 1 58B1C6FD
 P 8950 6650
-F 0 "C63" H 8975 6750 50  0000 L CNN
+F 0 "C59" H 8975 6750 50  0000 L CNN
 F 1 "470pF" H 8950 6550 50  0000 L CNN
 F 2 "Capacitors_SMD:C_0603" H 8988 6500 50  0001 C CNN
@@
 $EndComp
 $Comp
-L GND #PWR0171
+L GND #PWR0168
 U 1 1 58B1C704
 P 9050 6900
-F 0 "#PWR0171" H 9050 6650 50  0001 C CNN
+F 0 "#PWR0168" H 9050 6650 50  0001 C CNN
 F 1 "GND" H 9050 6750 50  0000 C CNN
 F 2 "" H 9050 6900 50  0000 C CNN
@@
 $EndComp
 $Comp
-L C C66
+L C C62
 U 1 1 58B1C710
 P 9150 6650
-F 0 "C66" H 9175 6750 50  0000 L CNN
+F 0 "C62" H 9175 6750 50  0000 L CNN
 F 1 "470pF" H 9175 6550 50  0000 L CNN
 F 2 "Capacitors_SMD:C_0603" H 9188 6500 50  0001 C CNN
@@
 $EndComp
 $Comp
-L C C70
+L C C66
 U 1 1 58B40194
 P 10150 3950
-F 0 "C70" H 10050 4050 50  0000 C CNN
+F 0 "C66" H 10050 4050 50  0000 C CNN
 F 1 "10μF" H 10025 3850 50  0000 C CNN
 F 2 "Capacitors_SMD:C_0805" H 10188 3800 50  0001 C CNN
@@
 Can extract which\nfault is occurring via SPI\nby reading DRV_STATUS reg
 $Comp
-L VDD_3V3B #PWR0172
+L VDD_3V3B #PWR0169
 U 1 1 5A2FD350
 P 6550 4300
-F 0 "#PWR0172" H 6550 4150 50  0001 C CNN
+F 0 "#PWR0169" H 6550 4150 50  0001 C CNN
 F 1 "VDD_3V3B" H 6565 4473 50  0000 C CNN
 F 2 "" H 6550 4300 50  0000 C CNN
@@
 $EndComp
 $Comp
-L C C57
+L C C53
 U 1 1 5A896678
 P 6550 4800
-F 0 "C57" H 6600 4900 50  0000 L CNN
+F 0 "C53" H 6600 4900 50  0000 L CNN
 F 1 "100nF" H 6575 4700 50  0000 L CNN
 F 2 "Capacitors_SMD:C_0603" H 6588 4650 50  0001 C CNN

Commit message: Complete SPI, ADC, and Endstop header layout/position, add zone around the SiP
Parts:
- renumbered C53 to C55, C54 to C56, C55 to C57, C56 to C58, C57 to C59, C58 to C60, C59 to C61, C60 to C62, C61 to C63, C62 to C64, C63 to C65, C64 to C66, C65 to C67, C66 to C68, C67 to C69, C68 to C70
Changed lines of the file:
@@
 MOSI
 $Comp
-L C C55
+L C C57
 U 1 1 589B8A74
 P 7300 3950
-F 0 "C55" H 7186 3904 50  0000 R CNN
+F 0 "C57" H 7186 3904 50  0000 R CNN
 F 1 "100nF" H 7186 3995 50  0000 R CNN
 F 2 "Capacitors_SMD:C_0603" H 7338 3800 50  0001 C CNN
@@
 $EndComp
 $Comp
-L C C60
+L C C62
 U 1 1 5BA7E11F
 P 9100 4500
-F 0 "C60" V 9050 4400 50  0000 C CNN
+F 0 "C62" V 9050 4400 50  0000 C CNN
 F 1 "100nF" V 9050 4675 50  0000 C CNN
 F 2 "Capacitors_SMD:C_0603" H 9138 4350 50  0001 C CNN
@@
 $EndComp
 $Comp
-L CP1 C67
+L CP1 C69
 U 1 1 5BA7E120
 P 10450 3950
-F 0 "C67" H 10550 4050 50  0000 C CNN
+F 0 "C69" H 10550 4050 50  0000 C CNN
 F 1 "100μF" H 10600 3850 50  0000 C CNN
 F 2 "Capacitors_SMD:c_elec_8x10" H 10450 3950 50  0001 C CNN
@@
 $EndComp
 $Comp
-L C C63
+L C C65
 U 1 1 589BC941
 P 9550 3950
-F 0 "C63" H 9450 4050 50  0000 C CNN
+F 0 "C65" H 9450 4050 50  0000 C CNN
 F 1 "100nF" H 9425 3850 50  0000 C CNN
 F 2 "Capacitors_SMD:C_0603" H 9588 3800 50  0001 C CNN
@@
 $EndComp
 $Comp
-L GND #PWR0162
+L GND #PWR0164
 U 1 1 589BD203
 P 7300 4150
-F 0 "#PWR0162" H 7300 3900 50  0001 C CNN
+F 0 "#PWR0164" H 7300 3900 50  0001 C CNN
 F 1 "GND" H 7300 4000 50  0000 C CNN
 F 2 "" H 7300 4150 50  0000 C CNN
@@
 $EndComp
 $Comp
-L C C64
+L C C66
 U 1 1 589BDAA2
 P 9850 3950
-F 0 "C64" H 9750 4050 50  0000 C CNN
+F 0 "C66" H 9750 4050 50  0000 C CNN
 F 1 "100nF" H 9725 3850 50  0000 C CNN
 F 2 "Capacitors_SMD:C_0603" H 9888 3800 50  0001 C CNN
@@
 $EndComp
 $Comp
-L GND #PWR0163
+L GND #PWR0165
 U 1 1 589BE47E
 P 10150 4200
-F 0 "#PWR0163" H 10150 3950 50  0001 C CNN
+F 0 "#PWR0165" H 10150 3950 50  0001 C CNN
 F 1 "GND" H 10155 4027 50  0000 C CNN
 F 2 "" H 10150 4200 50  0000 C CNN
@@
 $EndComp
 $Comp
-L +24V #PWR0164
+L +24V #PWR0166
 U 1 1 5BA7E125
 P 8350 3700
-F 0 "#PWR0164" H 8350 3550 50  0001 C CNN
+F 0 "#PWR0166" H 8350 3550 50  0001 C CNN
 F 1 "+24V" H 8365 3873 50  0000 C CNN
 F 2 "" H 8350 3700 50  0000 C CNN
@@
 $EndComp
 $Comp
-L C C57
+L C C59
 U 1 1 589C0BAD
 P 8950 5000
-F 0 "C57" H 9065 5046 50  0000 L CNN
+F 0 "C59" H 9065 5046 50  0000 L CNN
 F 1 "22nF" H 9065 4955 50  0000 L CNN
 F 2 "Capacitors_SMD:C_0603" H 8988 4850 50  0001 C CNN
@@
 $EndComp
 $Comp
-L GND #PWR0165
+L GND #PWR0167
 U 1 1 5BA7E129
 P 9450 7900
-F 0 "#PWR0165" H 9450 7650 50  0001 C CNN
+F 0 "#PWR0167" H 9450 7650 50  0001 C CNN
 F 1 "GND" H 9455 7727 50  0000 C CNN
 F 2 "" H 9450 7900 50  0000 C CNN
@@
 $EndComp
 $Comp
-L C C54
+L C C56
 U 1 1 589C52DF
 P 6900 4800
-F 0 "C54" H 6950 4900 50  0000 L CNN
+F 0 "C56" H 6950 4900 50  0000 L CNN
 F 1 "470nF" H 6925 4700 50  0000 L CNN
 F 2 "Capacitors_SMD:C_0603" H 6938 4650 50  0001 C CNN
@@
 NoConn ~ 7500 6550
 $Comp
-L GND #PWR0166
+L GND #PWR0168
 U 1 1 589C97FF
 P 7450 6950
-F 0 "#PWR0166" H 7450 6700 50  0001 C CNN
+F 0 "#PWR0168" H 7450 6700 50  0001 C CNN
 F 1 "GND" H 7455 6777 50  0000 C CNN
 F 2 "" H 7450 6950 50  0000 C CNN
@@
 $EndComp
 $Comp
-L C C65
+L C C67
 U 1 1 5BA7E12E
 P 9900 7550
-F 0 "C65" H 9950 7650 50  0000 L CNN
+F 0 "C67" H 9950 7650 50  0000 L CNN
 F 1 "100nF" H 9950 7450 50  0000 L CNN
 F 2 "Capacitors_SMD:C_0603" H 9938 7400 50  0001 C CNN
@@
 Internal\nPull-Up
 $Comp
-L C C56
+L C C58
 U 1 1 5BA7E12A
 P 7300 4800
-F 0 "C56" H 7350 4900 50  0000 L CNN
+F 0 "C58" H 7350 4900 50  0000 L CNN
 F 1 "4.7μF" H 7350 4700 50  0000 L CNN
 F 2 "Capacitors_SMD:C_0603" H 7338 4650 50  0001 C CNN
@@
 $EndComp
 $Comp
-L C C68
+L C C70
 U 1 1 5BA7E133
 P 10700 7550
-F 0 "C68" H 10750 7650 50  0000 L CNN
+F 0 "C70" H 10750 7650 50  0000 L CNN
 F 1 "100nF" H 10750 7450 50  0000 L CNN
 F 2 "Capacitors_SMD:C_0603" H 10738 7400 50  0001 C CNN
@@
 Choose  sense  resistors  in  a  way,  that  normal \nIRUN is 16 to 31 for best microstep performance.
 $Comp
-L C C58
+L C C60
 U 1 1 5BA7E134
 P 8950 5800
-F 0 "C58" H 8975 5900 50  0000 L CNN
+F 0 "C60" H 8975 5900 50  0000 L CNN
 F 1 "470pF" H 8950 5700 50  0000 L CNN
 F 2 "Capacitors_SMD:C_0603" H 8988 5650 50  0001 C CNN
@@
 $EndComp
 $Comp
-L GND #PWR0167
+L GND #PWR0169
 U 1 1 58B19D33
 P 9050 6050
-F 0 "#PWR0167" H 9050 5800 50  0001 C CNN
+F 0 "#PWR0169" H 9050 5800 50  0001 C CNN
 F 1 "GND" H 9050 5900 50  0000 C CNN
 F 2 "" H 9050 6050 50  0000 C CNN
@@
 $EndComp
 $Comp
-L C C61
+L C C63
 U 1 1 58B1B794
 P 9150 5800
-F 0 "C61" H 9175 5900 50  0000 L CNN
+F 0 "C63" H 9175 5900 50  0000 L CNN
 F 1 "470pF" H 9175 5700 50  0000 L CNN
 F 2 "Capacitors_SMD:C_0603" H 9188 5650 50  0001 C CNN
@@
 $EndComp
 $Comp
-L C C59
+L C C61
 U 1 1 58B1C6FD
 P 8950 6650
-F 0 "C59" H 8975 6750 50  0000 L CNN
+F 0 "C61" H 8975 6750 50  0000 L CNN
 F 1 "470pF" H 8950 6550 50  0000 L CNN
 F 2 "Capacitors_SMD:C_0603" H 8988 6500 50  0001 C CNN
@@
 $EndComp
 $Comp
-L GND #PWR0168
+L GND #PWR0170
 U 1 1 58B1C704
 P 9050 6900
-F 0 "#PWR0168" H 9050 6650 50  0001 C CNN
+F 0 "#PWR0170" H 9050 6650 50  0001 C CNN
 F 1 "GND" H 9050 6750 50  0000 C CNN
 F 2 "" H 9050 6900 50  0000 C CNN
@@
 $EndComp
 $Comp
-L C C62
+L C C64
 U 1 1 58B1C710
 P 9150 6650
-F 0 "C62" H 9175 6750 50  0000 L CNN
+F 0 "C64" H 9175 6750 50  0000 L CNN
 F 1 "470pF" H 9175 6550 50  0000 L CNN
 F 2 "Capacitors_SMD:C_0603" H 9188 6500 50  0001 C CNN
@@
 $EndComp
 $Comp
-L C C66
+L C C68
 U 1 1 58B40194
 P 10150 3950
-F 0 "C66" H 10050 4050 50  0000 C CNN
+F 0 "C68" H 10050 4050 50  0000 C CNN
 F 1 "10μF" H 10025 3850 50  0000 C CNN
 F 2 "Capacitors_SMD:C_0805" H 10188 3800 50  0001 C CNN
@@
 Can extract which\nfault is occurring via SPI\nby reading DRV_STATUS reg
 $Comp
-L VDD_3V3B #PWR0169
+L VDD_3V3B #PWR0171
 U 1 1 5A2FD350
 P 6550 4300
-F 0 "#PWR0169" H 6550 4150 50  0001 C CNN
+F 0 "#PWR0171" H 6550 4150 50  0001 C CNN
 F 1 "VDD_3V3B" H 6565 4473 50  0000 C CNN
 F 2 "" H 6550 4300 50  0000 C CNN
@@
 $EndComp
 $Comp
-L C C53
+L C C55
 U 1 1 5A896678
 P 6550 4800
-F 0 "C53" H 6600 4900 50  0000 L CNN
+F 0 "C55" H 6600 4900 50  0000 L CNN
 F 1 "100nF" H 6575 4700 50  0000 L CNN
 F 2 "Capacitors_SMD:C_0603" H 6588 4650 50  0001 C CNN

Commit message: Remove the unneeded oscillator, track down which components are underneath the OSD3358 and put them on the top
Parts:
- renumbered C55 to C54, C56 to C55, C57 to C56, C58 to C57, C59 to C58, C60 to C59, C61 to C60, C62 to C61, C63 to C62, C64 to C63, C65 to C64, C66 to C65, C67 to C66, C68 to C67, C69 to C68, C70 to C69, R115 to R114, R116 to R115, R117 to R116, R118 to R117, R119 to R118, R120 to R119, R121 to R120
Changed lines of the file:
@@
 MOSI
 $Comp
-L C C57
+L C C56
 U 1 1 589B8A74
 P 7300 3950
-F 0 "C57" H 7186 3904 50  0000 R CNN
+F 0 "C56" H 7186 3904 50  0000 R CNN
 F 1 "100nF" H 7186 3995 50  0000 R CNN
 F 2 "Capacitors_SMD:C_0603" H 7338 3800 50  0001 C CNN
@@
 $EndComp
 $Comp
-L C C62
+L C C61
 U 1 1 5BA7E11F
 P 9100 4500
-F 0 "C62" V 9050 4400 50  0000 C CNN
+F 0 "C61" V 9050 4400 50  0000 C CNN
 F 1 "100nF" V 9050 4675 50  0000 C CNN
 F 2 "Capacitors_SMD:C_0603" H 9138 4350 50  0001 C CNN
@@
 $EndComp
 $Comp
-L CP1 C69
+L CP1 C68
 U 1 1 5BA7E120
 P 10450 3950
-F 0 "C69" H 10550 4050 50  0000 C CNN
+F 0 "C68" H 10550 4050 50  0000 C CNN
 F 1 "100μF" H 10600 3850 50  0000 C CNN
 F 2 "Capacitors_SMD:c_elec_8x10" H 10450 3950 50  0001 C CNN
@@
 $EndComp
 $Comp
-L C C65
+L C C64
 U 1 1 589BC941
 P 9550 3950
-F 0 "C65" H 9450 4050 50  0000 C CNN
+F 0 "C64" H 9450 4050 50  0000 C CNN
 F 1 "100nF" H 9425 3850 50  0000 C CNN
 F 2 "Capacitors_SMD:C_0603" H 9588 3800 50  0001 C CNN
@@
 $EndComp
 $Comp
-L GND #PWR0164
+L GND #PWR0162
 U 1 1 589BD203
 P 7300 4150
-F 0 "#PWR0164" H 7300 3900 50  0001 C CNN
+F 0 "#PWR0162" H 7300 3900 50  0001 C CNN
 F 1 "GND" H 7300 4000 50  0000 C CNN
 F 2 "" H 7300 4150 50  0000 C CNN
@@
 $EndComp
 $Comp
-L C C66
+L C C65
 U 1 1 589BDAA2
 P 9850 3950
-F 0 "C66" H 9750 4050 50  0000 C CNN
+F 0 "C65" H 9750 4050 50  0000 C CNN
 F 1 "100nF" H 9725 3850 50  0000 C CNN
 F 2 "Capacitors_SMD:C_0603" H 9888 3800 50  0001 C CNN
@@
 $EndComp
 $Comp
-L GND #PWR0165
+L GND #PWR0163
 U 1 1 589BE47E
 P 10150 4200
-F 0 "#PWR0165" H 10150 3950 50  0001 C CNN
+F 0 "#PWR0163" H 10150 3950 50  0001 C CNN
 F 1 "GND" H 10155 4027 50  0000 C CNN
 F 2 "" H 10150 4200 50  0000 C CNN
@@
 $EndComp
 $Comp
-L +24V #PWR0166
+L +24V #PWR0164
 U 1 1 5BA7E125
 P 8350 3700
-F 0 "#PWR0166" H 8350 3550 50  0001 C CNN
+F 0 "#PWR0164" H 8350 3550 50  0001 C CNN
 F 1 "+24V" H 8365 3873 50  0000 C CNN
 F 2 "" H 8350 3700 50  0000 C CNN
@@
 $EndComp
 $Comp
-L C C59
+L C C58
 U 1 1 589C0BAD
 P 8950 5000
-F 0 "C59" H 9065 5046 50  0000 L CNN
+F 0 "C58" H 9065 5046 50  0000 L CNN
 F 1 "22nF" H 9065 4955 50  0000 L CNN
 F 2 "Capacitors_SMD:C_0603" H 8988 4850 50  0001 C CNN
@@
 $EndComp
 $Comp
-L R R121
+L R R120
 U 1 1 589C1BED
 P 10550 7550
-F 0 "R121" H 10500 7500 50  0000 R CNN
+F 0 "R120" H 10500 7500 50  0000 R CNN
 F 1 "220mΩ" H 10500 7600 50  0000 R CNN
 F 2 "Resistors_SMD:R_0805" V 10480 7550 50  0001 C CNN
@@
 $EndComp
 $Comp
-L R R120
+L R R119
 U 1 1 589C1CA7
 P 9750 7550
-F 0 "R120" H 9700 7500 50  0000 R CNN
+F 0 "R119" H 9700 7500 50  0000 R CNN
 F 1 "220mΩ" H 9700 7600 50  0000 R CNN
 F 2 "Resistors_SMD:R_0805" V 9680 7550 50  0001 C CNN
@@
 $EndComp
 $Comp
-L GND #PWR0167
+L GND #PWR0165
 U 1 1 5BA7E129
 P 9450 7900
-F 0 "#PWR0167" H 9450 7650 50  0001 C CNN
+F 0 "#PWR0165" H 9450 7650 50  0001 C CNN
 F 1 "GND" H 9455 7727 50  0000 C CNN
 F 2 "" H 9450 7900 50  0000 C CNN
@@
 NoConn ~ 7500 6450
 $Comp
-L R R117
+L R R116
 U 1 1 5BA7E12B
 P 7100 4600
-F 0 "R117" V 7000 4600 50  0000 C CNN
+F 0 "R116" V 7000 4600 50  0000 C CNN
 F 1 "2.2Ω" V 7100 4600 50  0000 C CNN
 F 2 "Resistors_SMD:R_0603" V 7030 4600 50  0001 C CNN
@@
 $EndComp
 $Comp
-L C C56
+L C C55
 U 1 1 589C52DF
 P 6900 4800
-F 0 "C56" H 6950 4900 50  0000 L CNN
+F 0 "C55" H 6950 4900 50  0000 L CNN
 F 1 "470nF" H 6925 4700 50  0000 L CNN
 F 2 "Capacitors_SMD:C_0603" H 6938 4650 50  0001 C CNN
@@
 NoConn ~ 7500 6550
 $Comp
-L GND #PWR0168
+L GND #PWR0166
 U 1 1 589C97FF
 P 7450 6950
-F 0 "#PWR0168" H 7450 6700 50  0001 C CNN
+F 0 "#PWR0166" H 7450 6700 50  0001 C CNN
 F 1 "GND" H 7455 6777 50  0000 C CNN
 F 2 "" H 7450 6950 50  0000 C CNN
@@
 $EndComp
 $Comp
-L C C67
+L C C66
 U 1 1 5BA7E12E
 P 9900 7550
-F 0 "C67" H 9950 7650 50  0000 L CNN
+F 0 "C66" H 9950 7650 50  0000 L CNN
 F 1 "100nF" H 9950 7450 50  0000 L CNN
 F 2 "Capacitors_SMD:C_0603" H 9938 7400 50  0001 C CNN
@@
 E_FAULT
 $Comp
-L R R115
+L R R114
 U 1 1 589D21BC
 P 5850 5100
-F 0 "R115" H 5919 5146 50  0000 L CNN
+F 0 "R114" H 5919 5146 50  0000 L CNN
 F 1 "4.7kΩ" H 5919 5055 50  0000 L CNN
 F 2 "Resistors_SMD:R_0603" V 5780 5100 50  0001 C CNN
@@
 Internal\nPull-Up
 $Comp
-L C C58
+L C C57
 U 1 1 5BA7E12A
 P 7300 4800
-F 0 "C58" H 7350 4900 50  0000 L CNN
+F 0 "C57" H 7350 4900 50  0000 L CNN
 F 1 "4.7μF" H 7350 4700 50  0000 L CNN
 F 2 "Capacitors_SMD:C_0603" H 7338 4650 50  0001 C CNN
@@
 5VOUT
 $Comp
-L R R118
+L R R117
 U 1 1 589E13FD
 P 9050 7550
-F 0 "R118" H 9119 7596 50  0000 L CNN
+F 0 "R117" H 9119 7596 50  0000 L CNN
 F 1 "5.23kΩ" H 9119 7505 50  0000 L CNN
 F 2 "Resistors_SMD:R_0603" V 8980 7550 50  0001 C CNN
@@
 5VOUT
 $Comp
-L R R119
+L R R118
 U 1 1 589E24D4
 P 9250 7750
-F 0 "R119" V 9050 7750 50  0000 C CNN
+F 0 "R118" V 9050 7750 50  0000 C CNN
 F 1 "4.75kΩ" V 9150 7750 50  0000 C CNN
 F 2 "Resistors_SMD:R_0603" V 9180 7750 50  0001 C CNN
@@
 AIN_IREF=1-2.4V
 $Comp
-L R R116
+L R R115
 U 1 1 5BA7E132
 P 6200 5100
-F 0 "R116" H 6269 5146 50  0000 L CNN
+F 0 "R115" H 6269 5146 50  0000 L CNN
 F 1 "4.7kΩ" H 6269 5055 50  0000 L CNN
 F 2 "Resistors_SMD:R_0603" V 6130 5100 50  0001 C CNN
@@
 $EndComp
 $Comp
-L C C70
+L C C69
 U 1 1 5BA7E133
 P 10700 7550
-F 0 "C70" H 10750 7650 50  0000 L CNN
+F 0 "C69" H 10750 7650 50  0000 L CNN
 F 1 "100nF" H 10750 7450 50  0000 L CNN
 F 2 "Capacitors_SMD:C_0603" H 10738 7400 50  0001 C CNN
@@
 Choose  sense  resistors  in  a  way,  that  normal \nIRUN is 16 to 31 for best microstep performance.
 $Comp
-L C C60
+L C C59
 U 1 1 5BA7E134
 P 8950 5800
-F 0 "C60" H 8975 5900 50  0000 L CNN
+F 0 "C59" H 8975 5900 50  0000 L CNN
 F 1 "470pF" H 8950 5700 50  0000 L CNN
 F 2 "Capacitors_SMD:C_0603" H 8988 5650 50  0001 C CNN
@@
 $EndComp
 $Comp
-L GND #PWR0169
+L GND #PWR0167
 U 1 1 58B19D33
 P 9050 6050
-F 0 "#PWR0169" H 9050 5800 50  0001 C CNN
+F 0 "#PWR0167" H 9050 5800 50  0001 C CNN
 F 1 "GND" H 9050 5900 50  0000 C CNN
 F 2 "" H 9050 6050 50  0000 C CNN
@@
 $EndComp
 $Comp
-L C C63
+L C C62
 U 1 1 58B1B794
 P 9150 5800
-F 0 "C63" H 9175 5900 50  0000 L CNN
+F 0 "C62" H 9175 5900 50  0000 L CNN
 F 1 "470pF" H 9175 5700 50  0000 L CNN
 F 2 "Capacitors_SMD:C_0603" H 9188 5650 50  0001 C CNN
@@
 $EndComp
 $Comp
-L C C61
+L C C60
 U 1 1 58B1C6FD
 P 8950 6650
-F 0 "C61" H 8975 6750 50  0000 L CNN
+F 0 "C60" H 8975 6750 50  0000 L CNN
 F 1 "470pF" H 8950 6550 50  0000 L CNN
 F 2 "Capacitors_SMD:C_0603" H 8988 6500 50  0001 C CNN
@@
 $EndComp
 $Comp
-L GND #PWR0170
+L GND #PWR0168
 U 1 1 58B1C704
 P 9050 6900
-F 0 "#PWR0170" H 9050 6650 50  0001 C CNN
+F 0 "#PWR0168" H 9050 6650 50  0001 C CNN
 F 1 "GND" H 9050 6750 50  0000 C CNN
 F 2 "" H 9050 6900 50  0000 C CNN
@@
 $EndComp
 $Comp
-L C C64
+L C C63
 U 1 1 58B1C710
 P 9150 6650
-F 0 "C64" H 9175 6750 50  0000 L CNN
+F 0 "C63" H 9175 6750 50  0000 L CNN
 F 1 "470pF" H 9175 6550 50  0000 L CNN
 F 2 "Capacitors_SMD:C_0603" H 9188 6500 50  0001 C CNN
@@
 $EndComp
 $Comp
-L C C68
+L C C67
 U 1 1 58B40194
 P 10150 3950
-F 0 "C68" H 10050 4050 50  0000 C CNN
+F 0 "C67" H 10050 4050 50  0000 C CNN
 F 1 "10μF" H 10025 3850 50  0000 C CNN
 F 2 "Capacitors_SMD:C_0805" H 10188 3800 50  0001 C CNN
@@
 Can extract which\nfault is occurring via SPI\nby reading DRV_STATUS reg
 $Comp
-L VDD_3V3B #PWR0171
+L VDD_3V3B #PWR0169
 U 1 1 5A2FD350
 P 6550 4300
-F 0 "#PWR0171" H 6550 4150 50  0001 C CNN
+F 0 "#PWR0169" H 6550 4150 50  0001 C CNN
 F 1 "VDD_3V3B" H 6565 4473 50  0000 C CNN
 F 2 "" H 6550 4300 50  0000 C CNN
@@
 $EndComp
 $Comp
-L C C55
+L C C54
 U 1 1 5A896678
 P 6550 4800
-F 0 "C55" H 6600 4900 50  0000 L CNN
+F 0 "C54" H 6600 4900 50  0000 L CNN
 F 1 "100nF" H 6575 4700 50  0000 L CNN
 F 2 "Capacitors_SMD:C_0603" H 6588 4650 50  0001 C CNN
