File: KiMBo/therm.sch (KiCad schematic (older format))
At the start: 8 parts

Commit message: Add F1 PTC resettable fuse at the 5V output, begin E's heater circuit layout
Parts:
- renumbered FB28 to FB32, FB29 to FB33
Changed lines of the file:
@@
 $EndComp
 $Comp
-L INDUCTOR_Small FB28
+L INDUCTOR_Small FB32
 U 1 1 5B885A27
 P 6200 5250
-F 0 "FB28" V 6385 5250 50  0000 C CNN
+F 0 "FB32" V 6385 5250 50  0000 C CNN
 F 1 "MMZ1608A252BTA00" V 6294 5250 50  0000 C CNN
 F 2 "KiMBo:Ferrite_Bead_0603" H 6200 5250 50  0001 C CNN
@@
 	8750 5250 8750 5100
 $Comp
-L INDUCTOR_Small FB29
+L INDUCTOR_Small FB33
 U 1 1 5B8FFD1D
 P 9150 5250
-F 0 "FB29" V 9335 5250 50  0000 C CNN
+F 0 "FB33" V 9335 5250 50  0000 C CNN
 F 1 "MMZ1608A252BTA00" V 9244 5250 50  0000 C CNN
 F 2 "KiMBo:Ferrite_Bead_0603" H 9150 5250 50  0001 C CNN

Commit message: Route 24V to the buck, add PTC fuse to 5V output
Parts:
- renumbered FB32 to FB41, FB33 to FB42
Changed lines of the file:
@@
 $EndComp
 $Comp
-L INDUCTOR_Small FB32
+L INDUCTOR_Small FB41
 U 1 1 5B885A27
 P 6200 5250
-F 0 "FB32" V 6385 5250 50  0000 C CNN
+F 0 "FB41" V 6385 5250 50  0000 C CNN
 F 1 "MMZ1608A252BTA00" V 6294 5250 50  0000 C CNN
 F 2 "KiMBo:Ferrite_Bead_0603" H 6200 5250 50  0001 C CNN
@@
 	8750 5250 8750 5100
 $Comp
-L INDUCTOR_Small FB33
+L INDUCTOR_Small FB42
 U 1 1 5B8FFD1D
 P 9150 5250
-F 0 "FB33" V 9335 5250 50  0000 C CNN
+F 0 "FB42" V 9335 5250 50  0000 C CNN
 F 1 "MMZ1608A252BTA00" V 9244 5250 50  0000 C CNN
 F 2 "KiMBo:Ferrite_Bead_0603" H 9150 5250 50  0001 C CNN

Commit message: Add ferrite beads to the 5V and 3V pins at the SPI connectors
Parts:
- renumbered C46 to C42, C47 to C43, FB41 to FB49, FB42 to FB50
Changed lines of the file:
@@
 $EndDescr
 $Comp
-L C C46
+L C C42
 U 1 1 57931608
 P 6900 5550
-F 0 "C46" H 6785 5504 50  0000 R CNN
+F 0 "C42" H 6785 5504 50  0000 R CNN
 F 1 "4.7μF" H 6785 5595 50  0000 R CNN
 F 2 "Capacitors_SMD:C_0603" H 6938 5400 50  0001 C CNN
@@
 BED_THERM_IN
 $Comp
-L VDD_ADC #PWR0142
+L VDD_ADC #PWR0139
 U 1 1 59E74D42
 P 5800 4750
-F 0 "#PWR0142" H 5950 4700 50  0001 C CNN
+F 0 "#PWR0139" H 5950 4700 50  0001 C CNN
 F 1 "VDD_ADC" H 5820 4893 50  0000 C CNN
 F 2 "" H 5800 4750 50  0000 C CNN
@@
 $EndComp
 $Comp
-L C C47
+L C C43
 U 1 1 5AD7EE6B
 P 9850 5550
-F 0 "C47" H 9735 5504 50  0000 R CNN
+F 0 "C43" H 9735 5504 50  0000 R CNN
 F 1 "4.7μF" H 9735 5595 50  0000 R CNN
 F 2 "Capacitors_SMD:C_0603" H 9888 5400 50  0001 C CNN
@@
 ADC_IN
 $Comp
-L VDD_ADC #PWR0143
+L VDD_ADC #PWR0140
 U 1 1 5AD7EEB1
 P 8750 4750
-F 0 "#PWR0143" H 8900 4700 50  0001 C CNN
+F 0 "#PWR0140" H 8900 4700 50  0001 C CNN
 F 1 "VDD_ADC" H 8770 4893 50  0000 C CNN
 F 2 "" H 8750 4750 50  0000 C CNN
@@
 $EndComp
 $Comp
-L GND #PWR0144
+L GND #PWR0141
 U 1 1 5B331170
 P 6900 5750
-F 0 "#PWR0144" H 6900 5500 50  0001 C CNN
+F 0 "#PWR0141" H 6900 5500 50  0001 C CNN
 F 1 "GND" H 6905 5577 50  0000 C CNN
 F 2 "" H 6900 5750 50  0000 C CNN
@@
 $EndComp
 $Comp
-L GND #PWR0145
+L GND #PWR0142
 U 1 1 5B3311A0
 P 9850 5750
-F 0 "#PWR0145" H 9850 5500 50  0001 C CNN
+F 0 "#PWR0142" H 9850 5500 50  0001 C CNN
 F 1 "GND" H 9855 5577 50  0000 C CNN
 F 2 "" H 9850 5750 50  0000 C CNN
@@
 $EndComp
 $Comp
-L INDUCTOR_Small FB41
+L INDUCTOR_Small FB49
 U 1 1 5B885A27
 P 6200 5250
-F 0 "FB41" V 6385 5250 50  0000 C CNN
+F 0 "FB49" V 6385 5250 50  0000 C CNN
 F 1 "MMZ1608A252BTA00" V 6294 5250 50  0000 C CNN
 F 2 "KiMBo:Ferrite_Bead_0603" H 6200 5250 50  0001 C CNN
@@
 	8750 5250 8750 5100
 $Comp
-L INDUCTOR_Small FB42
+L INDUCTOR_Small FB50
 U 1 1 5B8FFD1D
 P 9150 5250
-F 0 "FB42" V 9335 5250 50  0000 C CNN
+F 0 "FB50" V 9335 5250 50  0000 C CNN
 F 1 "MMZ1608A252BTA00" V 9244 5250 50  0000 C CNN
 F 2 "KiMBo:Ferrite_Bead_0603" H 9150 5250 50  0001 C CNN

Commit message: Complete SPI, ADC, and Endstop header layout/position, add zone around the SiP
Parts:
- renumbered C42 to C44, C43 to C45
Connections:
- net ADC_IN: now also FB50.2; no longer FB50.1
- net BED_THERM_IN: now also FB49.2; no longer FB49.1
- net at R93.1: now also FB49.1; no longer FB49.2
- net at R95.1: now also FB50.1; no longer FB50.2
Changed lines of the file:
@@
 $EndDescr
 $Comp
-L C C42
+L C C44
 U 1 1 57931608
 P 6900 5550
-F 0 "C42" H 6785 5504 50  0000 R CNN
+F 0 "C44" H 6785 5504 50  0000 R CNN
 F 1 "4.7μF" H 6785 5595 50  0000 R CNN
 F 2 "Capacitors_SMD:C_0603" H 6938 5400 50  0001 C CNN
@@
 BED_THERM_IN
 $Comp
-L VDD_ADC #PWR0139
+L VDD_ADC #PWR0141
 U 1 1 59E74D42
 P 5800 4750
-F 0 "#PWR0139" H 5950 4700 50  0001 C CNN
+F 0 "#PWR0141" H 5950 4700 50  0001 C CNN
 F 1 "VDD_ADC" H 5820 4893 50  0000 C CNN
 F 2 "" H 5800 4750 50  0000 C CNN
@@
 $EndComp
 $Comp
-L C C43
+L C C45
 U 1 1 5AD7EE6B
 P 9850 5550
-F 0 "C43" H 9735 5504 50  0000 R CNN
+F 0 "C45" H 9735 5504 50  0000 R CNN
 F 1 "4.7μF" H 9735 5595 50  0000 R CNN
 F 2 "Capacitors_SMD:C_0603" H 9888 5400 50  0001 C CNN
@@
 ADC_IN
 $Comp
-L VDD_ADC #PWR0140
+L VDD_ADC #PWR0142
 U 1 1 5AD7EEB1
 P 8750 4750
-F 0 "#PWR0140" H 8900 4700 50  0001 C CNN
+F 0 "#PWR0142" H 8900 4700 50  0001 C CNN
 F 1 "VDD_ADC" H 8770 4893 50  0000 C CNN
 F 2 "" H 8750 4750 50  0000 C CNN
@@
 $EndComp
 $Comp
-L GND #PWR0141
+L GND #PWR0143
 U 1 1 5B331170
 P 6900 5750
-F 0 "#PWR0141" H 6900 5500 50  0001 C CNN
+F 0 "#PWR0143" H 6900 5500 50  0001 C CNN
 F 1 "GND" H 6905 5577 50  0000 C CNN
 F 2 "" H 6900 5750 50  0000 C CNN
@@
 $EndComp
 $Comp
-L GND #PWR0142
+L GND #PWR0144
 U 1 1 5B3311A0
 P 9850 5750
-F 0 "#PWR0142" H 9850 5500 50  0001 C CNN
+F 0 "#PWR0144" H 9850 5500 50  0001 C CNN
 F 1 "GND" H 9855 5577 50  0000 C CNN
 F 2 "" H 9850 5750 50  0000 C CNN
@@
 F 3 "" H 6200 5250 50  0000 C CNN
 	1    6200 5250
-	0    -1   -1   0
+	0    1    -1   0
 $EndComp
 Text Notes 8250 5200 0    60   ~ 0
@@
 F 3 "" H 9150 5250 50  0000 C CNN
 	1    9150 5250
-	0    -1   -1   0
+	0    1    -1   0
 $EndComp
 $EndSCHEMATC

Commit message: Remove the unneeded oscillator, track down which components are underneath the OSD3358 and put them on the top
Parts:
- renumbered C44 to C43, C45 to C44, R92 to R91, R93 to R92, R94 to R93, R95 to R94
Changed lines of the file:
@@
 $EndDescr
 $Comp
-L C C44
+L C C43
 U 1 1 57931608
 P 6900 5550
-F 0 "C44" H 6785 5504 50  0000 R CNN
+F 0 "C43" H 6785 5504 50  0000 R CNN
 F 1 "4.7μF" H 6785 5595 50  0000 R CNN
 F 2 "Capacitors_SMD:C_0603" H 6938 5400 50  0001 C CNN
@@
 $EndComp
 $Comp
-L R R93
+L R R92
 U 1 1 57931779
 P 6700 5250
-F 0 "R93" V 6540 5250 50  0000 C CNN
+F 0 "R92" V 6540 5250 50  0000 C CNN
 F 1 "10kΩ" V 6610 5250 50  0000 C CNN
 F 2 "Resistors_SMD:R_0603" V 6630 5250 50  0001 C CNN
@@
 $EndComp
 $Comp
-L R R92
+L R R91
 U 1 1 57931815
 P 5800 4950
-F 0 "R92" H 5650 4950 50  0000 C CNN
+F 0 "R91" H 5650 4950 50  0000 C CNN
 F 1 "4.7kΩ" H 5960 4950 50  0000 C CNN
 F 2 "Resistors_SMD:R_0603" V 5730 4950 50  0001 C CNN
@@
 BED_THERM_IN
 $Comp
-L VDD_ADC #PWR0141
+L VDD_ADC #PWR0139
 U 1 1 59E74D42
 P 5800 4750
-F 0 "#PWR0141" H 5950 4700 50  0001 C CNN
+F 0 "#PWR0139" H 5950 4700 50  0001 C CNN
 F 1 "VDD_ADC" H 5820 4893 50  0000 C CNN
 F 2 "" H 5800 4750 50  0000 C CNN
@@
 $EndComp
 $Comp
-L C C45
+L C C44
 U 1 1 5AD7EE6B
 P 9850 5550
-F 0 "C45" H 9735 5504 50  0000 R CNN
+F 0 "C44" H 9735 5504 50  0000 R CNN
 F 1 "4.7μF" H 9735 5595 50  0000 R CNN
 F 2 "Capacitors_SMD:C_0603" H 9888 5400 50  0001 C CNN
@@
 $EndComp
 $Comp
-L R R95
+L R R94
 U 1 1 5AD7EE80
 P 9650 5250
-F 0 "R95" V 9490 5250 50  0000 C CNN
+F 0 "R94" V 9490 5250 50  0000 C CNN
 F 1 "10kΩ" V 9560 5250 50  0000 C CNN
 F 2 "Resistors_SMD:R_0603" V 9580 5250 50  0001 C CNN
@@
 $EndComp
 $Comp
-L R R94
+L R R93
 U 1 1 5AD7EE87
 P 8750 4950
-F 0 "R94" H 8600 4950 50  0000 C CNN
+F 0 "R93" H 8600 4950 50  0000 C CNN
 F 1 "4.7kΩ" H 8910 4950 50  0000 C CNN
 F 2 "Resistors_SMD:R_0603" V 8680 4950 50  0001 C CNN
@@
 ADC_IN
 $Comp
-L VDD_ADC #PWR0142
+L VDD_ADC #PWR0140
 U 1 1 5AD7EEB1
 P 8750 4750
-F 0 "#PWR0142" H 8900 4700 50  0001 C CNN
+F 0 "#PWR0140" H 8900 4700 50  0001 C CNN
 F 1 "VDD_ADC" H 8770 4893 50  0000 C CNN
 F 2 "" H 8750 4750 50  0000 C CNN
@@
 $EndComp
 $Comp
-L GND #PWR0143
+L GND #PWR0141
 U 1 1 5B331170
 P 6900 5750
-F 0 "#PWR0143" H 6900 5500 50  0001 C CNN
+F 0 "#PWR0141" H 6900 5500 50  0001 C CNN
 F 1 "GND" H 6905 5577 50  0000 C CNN
 F 2 "" H 6900 5750 50  0000 C CNN
@@
 $EndComp
 $Comp
-L GND #PWR0144
+L GND #PWR0142
 U 1 1 5B3311A0
 P 9850 5750
-F 0 "#PWR0144" H 9850 5500 50  0001 C CNN
+F 0 "#PWR0142" H 9850 5500 50  0001 C CNN
 F 1 "GND" H 9855 5577 50  0000 C CNN
 F 2 "" H 9850 5750 50  0000 C CNN

Commit message: Complete parallel data bus routing from the eMMC to the CPU
Center the SiP on the PCB

Add LPFs at the I2Cs' SCL outputs
Parts:
- renumbered C43 to C44, C44 to C45, FB49 to FB50, FB50 to FB51
Changed lines of the file:
@@
 $EndDescr
 $Comp
-L C C43
+L C C44
 U 1 1 57931608
 P 6900 5550
-F 0 "C43" H 6785 5504 50  0000 R CNN
+F 0 "C44" H 6785 5504 50  0000 R CNN
 F 1 "4.7μF" H 6785 5595 50  0000 R CNN
 F 2 "Capacitors_SMD:C_0603" H 6938 5400 50  0001 C CNN
@@
 BED_THERM_IN
 $Comp
-L VDD_ADC #PWR0139
+L VDD_ADC #PWR0140
 U 1 1 59E74D42
 P 5800 4750
-F 0 "#PWR0139" H 5950 4700 50  0001 C CNN
+F 0 "#PWR0140" H 5950 4700 50  0001 C CNN
 F 1 "VDD_ADC" H 5820 4893 50  0000 C CNN
 F 2 "" H 5800 4750 50  0000 C CNN
@@
 $EndComp
 $Comp
-L C C44
+L C C45
 U 1 1 5AD7EE6B
 P 9850 5550
-F 0 "C44" H 9735 5504 50  0000 R CNN
+F 0 "C45" H 9735 5504 50  0000 R CNN
 F 1 "4.7μF" H 9735 5595 50  0000 R CNN
 F 2 "Capacitors_SMD:C_0603" H 9888 5400 50  0001 C CNN
@@
 ADC_IN
 $Comp
-L VDD_ADC #PWR0140
+L VDD_ADC #PWR0141
 U 1 1 5AD7EEB1
 P 8750 4750
-F 0 "#PWR0140" H 8900 4700 50  0001 C CNN
+F 0 "#PWR0141" H 8900 4700 50  0001 C CNN
 F 1 "VDD_ADC" H 8770 4893 50  0000 C CNN
 F 2 "" H 8750 4750 50  0000 C CNN
@@
 $EndComp
 $Comp
-L GND #PWR0141
+L GND #PWR0142
 U 1 1 5B331170
 P 6900 5750
-F 0 "#PWR0141" H 6900 5500 50  0001 C CNN
+F 0 "#PWR0142" H 6900 5500 50  0001 C CNN
 F 1 "GND" H 6905 5577 50  0000 C CNN
 F 2 "" H 6900 5750 50  0000 C CNN
@@
 $EndComp
 $Comp
-L GND #PWR0142
+L GND #PWR0143
 U 1 1 5B3311A0
 P 9850 5750
-F 0 "#PWR0142" H 9850 5500 50  0001 C CNN
+F 0 "#PWR0143" H 9850 5500 50  0001 C CNN
 F 1 "GND" H 9855 5577 50  0000 C CNN
 F 2 "" H 9850 5750 50  0000 C CNN
@@
 $EndComp
 $Comp
-L INDUCTOR_Small FB49
+L INDUCTOR_Small FB50
 U 1 1 5B885A27
 P 6200 5250
-F 0 "FB49" V 6385 5250 50  0000 C CNN
+F 0 "FB50" V 6385 5250 50  0000 C CNN
 F 1 "MMZ1608A252BTA00" V 6294 5250 50  0000 C CNN
 F 2 "KiMBo:Ferrite_Bead_0603" H 6200 5250 50  0001 C CNN
@@
 	8750 5250 8750 5100
 $Comp
-L INDUCTOR_Small FB50
+L INDUCTOR_Small FB51
 U 1 1 5B8FFD1D
 P 9150 5250
-F 0 "FB50" V 9335 5250 50  0000 C CNN
+F 0 "FB51" V 9335 5250 50  0000 C CNN
 F 1 "MMZ1608A252BTA00" V 9244 5250 50  0000 C CNN
 F 2 "KiMBo:Ferrite_Bead_0603" H 9150 5250 50  0001 C CNN

Commit message: Routing open-drain output inverters, SOT-5 I2C EEPROM, begin adding bypass caps around the eMMC
Parts:
- renumbered C44 to C45, C45 to C46, FB50 to FB51, FB51 to FB52
Changed lines of the file:
@@
 $EndDescr
 $Comp
-L C C44
+L C C45
 U 1 1 57931608
 P 6900 5550
-F 0 "C44" H 6785 5504 50  0000 R CNN
+F 0 "C45" H 6785 5504 50  0000 R CNN
 F 1 "4.7μF" H 6785 5595 50  0000 R CNN
 F 2 "Capacitors_SMD:C_0603" H 6938 5400 50  0001 C CNN
@@
 BED_THERM_IN
 $Comp
-L VDD_ADC #PWR0140
+L VDD_ADC #PWR0141
 U 1 1 59E74D42
 P 5800 4750
-F 0 "#PWR0140" H 5950 4700 50  0001 C CNN
+F 0 "#PWR0141" H 5950 4700 50  0001 C CNN
 F 1 "VDD_ADC" H 5820 4893 50  0000 C CNN
 F 2 "" H 5800 4750 50  0000 C CNN
@@
 $EndComp
 $Comp
-L C C45
+L C C46
 U 1 1 5AD7EE6B
 P 9850 5550
-F 0 "C45" H 9735 5504 50  0000 R CNN
+F 0 "C46" H 9735 5504 50  0000 R CNN
 F 1 "4.7μF" H 9735 5595 50  0000 R CNN
 F 2 "Capacitors_SMD:C_0603" H 9888 5400 50  0001 C CNN
@@
 ADC_IN
 $Comp
-L VDD_ADC #PWR0141
+L VDD_ADC #PWR0142
 U 1 1 5AD7EEB1
 P 8750 4750
-F 0 "#PWR0141" H 8900 4700 50  0001 C CNN
+F 0 "#PWR0142" H 8900 4700 50  0001 C CNN
 F 1 "VDD_ADC" H 8770 4893 50  0000 C CNN
 F 2 "" H 8750 4750 50  0000 C CNN
@@
 $EndComp
 $Comp
-L GND #PWR0142
+L GND #PWR0143
 U 1 1 5B331170
 P 6900 5750
-F 0 "#PWR0142" H 6900 5500 50  0001 C CNN
+F 0 "#PWR0143" H 6900 5500 50  0001 C CNN
 F 1 "GND" H 6905 5577 50  0000 C CNN
 F 2 "" H 6900 5750 50  0000 C CNN
@@
 $EndComp
 $Comp
-L GND #PWR0143
+L GND #PWR0144
 U 1 1 5B3311A0
 P 9850 5750
-F 0 "#PWR0143" H 9850 5500 50  0001 C CNN
+F 0 "#PWR0144" H 9850 5500 50  0001 C CNN
 F 1 "GND" H 9855 5577 50  0000 C CNN
 F 2 "" H 9850 5750 50  0000 C CNN
@@
 $EndComp
 $Comp
-L INDUCTOR_Small FB50
+L INDUCTOR_Small FB51
 U 1 1 5B885A27
 P 6200 5250
-F 0 "FB50" V 6385 5250 50  0000 C CNN
+F 0 "FB51" V 6385 5250 50  0000 C CNN
 F 1 "MMZ1608A252BTA00" V 6294 5250 50  0000 C CNN
 F 2 "KiMBo:Ferrite_Bead_0603" H 6200 5250 50  0001 C CNN
@@
 	8750 5250 8750 5100
 $Comp
-L INDUCTOR_Small FB51
+L INDUCTOR_Small FB52
 U 1 1 5B8FFD1D
 P 9150 5250
-F 0 "FB51" V 9335 5250 50  0000 C CNN
+F 0 "FB52" V 9335 5250 50  0000 C CNN
 F 1 "MMZ1608A252BTA00" V 9244 5250 50  0000 C CNN
 F 2 "KiMBo:Ferrite_Bead_0603" H 9150 5250 50  0001 C CNN
